File: Hardware/FC0/FC0.kicad_pcb (KiCad board)
At the start: 4 copper layers, 66 x 57 mm, 84 parts, among them J1 Micro_SD_Card, J10 UART conn6, J11 I2C conn4, J12 I2C conn4, J13 SWD_CONN4, J14 USB_B_Micro, J2 Power Conn6, J3 ADC6.6 conn4, J4 ADC3.3 conn4, J5 PWM_SIG, J6 PWM_POWER, J7 UART conn6, J8 UART conn4, J9 UART conn4, SW1 NRST, SW2 SW_SPDT, U1 PCA9685PW, U2 MPU-9250, U3 MS5611-01BA, U4 STM32F405RGTx, U5 AMS1117-3.3, U6 USBLC6-2SC6, Y1 X322516MLB4SI

Commit message: updated FC0
added information about silkscreen errors
fixed silkscreen errors
Other:
- board text added: "перепутана шелкография у первой партии плат на схеме ошибка устранена C12-C13 С9--С17 С10-с18"
- board text added: "слой, назначение, заливка 1 SIGNAL (GND) 2 (GND) 3 (POWER) 4 SIGNAL (GND)"
- board text removed: "1 SIGNAL (GND) 2 (GND) 3 (POWER) 4 SIGNAL (GND)"
- board text removed: "ОСИ ДЛЯ ГИРОСКОПА"
- board text removed: "проверить распиновку датчиков"
Changed lines of the file:
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@@
     (property "Sheetname" "MCU")
     (attr smd)
-    (fp_text reference "C17" (at 2.8833 -1.517 90) (layer "F.SilkS")
+    (fp_text reference "C17" (at 2.8833 0.007 90) (layer "F.SilkS")
       (effects (font (size 0.8 0.8) (thickness 0.13)))
     )
@@
     (property "Sheetname" "MCU")
     (attr smd)
-    (fp_text reference "C13" (at 3.595 -1.43) (layer "F.SilkS")
+    (fp_text reference "C13" (at 3.595 -0.012) (layer "F.SilkS")
       (effects (font (size 0.8 0.8) (thickness 0.13)))
     )
@@
     (property "Sheetname" "MCU")
     (attr smd)
-    (fp_text reference "C18" (at 2.991 -1.512) (layer "F.SilkS")
+    (fp_text reference "C18" (at 2.991 0.139) (layer "F.SilkS")
       (effects (font (size 0.8 0.8) (thickness 0.13)))
     )
@@
     (property "Sheetname" "MCU")
     (attr smd)
-    (fp_text reference "C9" (at -2.6293 -1.5564 90) (layer "F.SilkS")
+    (fp_text reference "C9" (at -2.6293 -0.0324 90) (layer "F.SilkS")
       (effects (font (size 0.8 0.8) (thickness 0.13)))
     )
@@
     (property "Sheetname" "MCU")
     (attr smd)
-    (fp_text reference "C10" (at -2.991 -1.536) (layer "F.SilkS")
+    (fp_text reference "C10" (at -2.991 -0.139) (layer "F.SilkS")
       (effects (font (size 0.8 0.8) (thickness 0.13)))
     )
@@
     (property "Sheetname" "MCU")
     (attr smd)
-    (fp_text reference "C12" (at 3.595 1.512) (layer "F.SilkS")
+    (fp_text reference "C12" (at 3.595 -0.012) (layer "F.SilkS")
       (effects (font (size 0.8 0.8) (thickness 0.13)))
     )
@@
     (effects (font (size 0.8 0.8) (thickness 0.13)))
   )
-  (gr_text "проверить распиновку датчиков" (at 149.098 160.782) (layer "Dwgs.User")
-    (effects (font (size 1.5 1.5) (thickness 0.3)))
+  (gr_text "слой, назначение, заливка\n1 SIGNAL (GND)\n2 (GND)\n3 (POWER)\n4 SIGNAL (GND)" (at 184.658 96) (layer "User.1")
+    (effects (font (size 1.5 1.5) (thickness 0.3)) (justify left))
   )
-  (gr_text "1 SIGNAL (GND)\n2 (GND)\n3 (POWER)\n4 SIGNAL (GND)" (at 83.566 99.822) (layer "User.1")
-    (effects (font (size 1 1) (thickness 0.15)))
-  )
-  (gr_text "ОСИ ДЛЯ ГИРОСКОПА" (at 185.674 101.854) (layer "User.1")
-    (effects (font (size 1.5 1.5) (thickness 0.3)))
+  (gr_text "перепутана шелкография у первой партии плат\nна схеме ошибка устранена\nC12-C13 \nС9--С17\nС10-с18" (at 185 113) (layer "User.2")
+    (effects (font (size 1.5 1.5) (thickness 0.3)) (justify left))
   )
   (dimension (type aligned) (layer "User.1")
