File: Hardware/ciam/impeller/impeller/impeller.kicad_pcb (KiCad board)
At the start: 4 copper layers, 113.7 x 86.6 mm, 255 parts, among them J1 PLS-3, J10 Micro-Fit_2x5P, J11 Micro-Fit_2x5P, J12 Micro-Fit_2x5P, J13 Micro-Fit_2x12P, J14 PLS-5, J16 Micro-Fit_2x2P, J2 Conn_02x05_SWD, J3 USB_B_Micro, J4 Micro_SD_Card_Con, J5 PicoBlade_1x2P, J6 Micro-Fit_2x2P, J7 Micro-Fit_2x2P, J8 Micro-Fit_2x5P, J9 Micro-Fit_2x5P, Q1 BSS138, Q10 BSS138, Q11 BSS138, Q12 BSS138, Q2 BSS138, Q3 BSS138, Q4 BSS138, Q5 BSS138, Q6 BSS138, Q7 BSS138, Q8 BSS138, Q9 BSS138, SW1 KLS7-TS6601-11-180, SW2 DS1040-06RN, SW3 DS1040-06RN, U1 STM32F405VGT6, U10 G3VM61D1, U11 G3VM61D1, U12 G3VM61D1, U13 G3VM61D1, U14 G3VM61D1, U15 G3VM61D1, U16 G3VM61D1, U17 G3VM61D1, U18 TLP291, U19 TLP291, U2 LDL1117S33R, U20 TLP291, U21 TLP291, U22 TLP291, U23 TLP291, U24 TLP291, U25 TLP291, U26 TLP291, U27 TLP291, U28 B0505MT-1WR4, U29 B0505MT-1WR4, U3 TEL 5-1211, U30 TLP291, U31 TLP291, U32 TLP291, U33 TLP291, U34 TLP291, U35 B0505MT-1WR4, U36 HCPL-0630, U37 HCPL-0630, U38 HCPL-0630, U39 HCPL-0630, U4 ISO1050DUB, U40 HCPL-0630, U41 B0505MT-1WR4, U42 USBLC6-2SC6, U43 HCPL-0630, U44 LDL1117S33R, U45 B0505MT-1WR4, U5 ISO1050DUB, U6 B0505MT-1WR4, U7 B0505MT-1WR4, U8 G3VM61D1, U9 G3VM61D1, Y1 KSE-7K32768KDY2400A3, Y2 KSE-7U08000MAB143ZA3

Commit message: Updated CIAM project
Parts:
- added J17: Micro-Fit_2x2P, Connector_Molex:Molex_Micro-Fit_3.0_43045-0400_2x02_P3.00mm_Horizontal, F.Cu at (124.6, 106.5)
- added R105: 1k, Resistor_SMD:R_0603_1608Metric, F.Cu at (127.4, 104.2)
- added R106: 2k, Resistor_SMD:R_0603_1608Metric, F.Cu at (127.4, 102.8)
- added R107: 1k, Resistor_SMD:R_0603_1608Metric, F.Cu at (118.9, 104.3)
- added R108: 2k, Resistor_SMD:R_0603_1608Metric, F.Cu at (118.9, 102.8)
- SW2, SW3: footprint Button_Switch_THT:SW_DIP_SPSTx08_Slide_9.78x22.5mm_W7.62mm_P2.54mm -> Button_Switch_THT:SW_DIP_SPSTx06_Slide_9.78x17.42mm_W7.62mm_P2.54mm
- moved C29 232.4 mm to (123.9, 44.4), turned to 90 degrees
- moved C30 231.0 mm to (122.0, 44.4), turned to 90 degrees
- moved C32 212.5 mm to (108.0, 40.6), turned to 90 degrees
- moved R14 197.6 mm to (129.9, 29.8), turned to 90 degrees
- moved C40 197.1 mm to (101.6, 42.2)
- moved R11 196.4 mm to (123.8, 32.3), turned to 90 degrees
- moved C39 196.3 mm to (101.6, 44.1)
- moved C42 195.9 mm to (101.6, 56.1)
- moved C41 195.3 mm to (101.6, 58.1)
- moved R13 195.0 mm to (127.9, 30.6), turned to 90 degrees
- moved U5 195.0 mm to (115.0, 44.4), turned to 180 degrees
- moved C34 195.0 mm to (90.0, 45.1), turned to 90 degrees
- moved U7 194.0 mm to (101.6, 50.2), turned to 90 degrees
- moved R10 193.8 mm to (121.7, 33.1), turned to 90 degrees
- moved C27 193.4 mm to (85.3, 44.4), turned to 90 degrees
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Connections:
- C31 pad 2: GND1 -> GND2
- C33 pad 2: GND1 -> GND2
- C35 pad 2: GND1 -> GND2
- C36 pad 2: GND1 -> GND2
- D1 pad 1: Net-(J6-Pin_1) -> /CAN/CAN2-
- D1 pad 2: Net-(J6-Pin_2) -> /CAN/CAN2+
- D1 pad 3: GND1 -> GND2
- D2 pad 1: Net-(J7-Pin_1) -> /CAN/CAN1-
- D2 pad 2: Net-(J7-Pin_2) -> /CAN/CAN1+
- J6 pad 1: Net-(J6-Pin_1) -> /CAN/CAN2-
- J6 pad 2: Net-(J6-Pin_2) -> /CAN/CAN2+
- J6 pad 4: GND1 -> GND2
- J7 pad 1: Net-(J7-Pin_1) -> /CAN/CAN1-
- J7 pad 2: Net-(J7-Pin_2) -> /CAN/CAN1+
- L1 pad 1: Net-(J6-Pin_1) -> /CAN/CAN2_-
- L1 pad 2: Net-(U4-CANL) -> /CAN/CAN2-
- L1 pad 3: Net-(U4-CANH) -> /CAN/CAN2+
- L1 pad 4: Net-(J6-Pin_2) -> /CAN/CAN2_+
- L2 pad 1: Net-(J7-Pin_1) -> /CAN/CAN1_-
- L2 pad 2: Net-(U5-CANL) -> /CAN/CAN1-
- L2 pad 3: Net-(U5-CANH) -> /CAN/CAN1+
- L2 pad 4: Net-(J7-Pin_2) -> /CAN/CAN1_+
- R3 pad 1: Net-(J6-Pin_1) -> /CAN/CAN2-
- R4 pad 1: Net-(J7-Pin_1) -> /CAN/CAN1-
- R5 pad 1: Net-(J6-Pin_2) -> /CAN/CAN2+
- R6 pad 1: Net-(J7-Pin_2) -> /CAN/CAN1+
- U1 pad 35: unconnected-(U1-PB0-Pad35) -> ThrustLever1
- U1 pad 36: unconnected-(U1-PB1-Pad36) -> ThrustLever2
- U1 pad 63: unconnected-(U1-PC6-Pad63) -> CAN1_A0
- U1 pad 64: unconnected-(U1-PC7-Pad64) -> CAN1_A1
- U1 pad 67: unconnected-(U1-PA8-Pad67) -> CAN1_A2
- U1 pad 68: unconnected-(U1-PA9-Pad68) -> CAN1_A3
- U1 pad 69: unconnected-(U1-PA10-Pad69) -> CAN1_A4
- U1 pad 77: unconnected-(U1-PA15-Pad77) -> CAN1_A5
- U1 pad 85: unconnected-(U1-PD4-Pad85) -> CAN2_A0
- U1 pad 86: unconnected-(U1-PD5-Pad86) -> CAN2_A1
- U1 pad 87: unconnected-(U1-PD6-Pad87) -> CAN2_A2
- U1 pad 88: unconnected-(U1-PD7-Pad88) -> CAN2_A3
- U1 pad 90: unconnected-(U1-PB4-Pad90) -> CAN2_A4
- U1 pad 93: unconnected-(U1-PB7-Pad93) -> CAN2_A5
- U4 pad 2: CAN1_RX -> CAN2_RX
- U4 pad 3: CAN1_TX -> CAN2_TX
- U4 pad 5: GND1 -> GND2
- U4 pad 6: Net-(U4-CANL) -> /CAN/CAN2_-
- U4 pad 7: Net-(U4-CANH) -> /CAN/CAN2_+
- U5 pad 2: CAN2_RX -> CAN1_RX
- U5 pad 3: CAN2_TX -> CAN1_TX
- U5 pad 6: Net-(U5-CANL) -> /CAN/CAN1_-
- U5 pad 7: Net-(U5-CANH) -> /CAN/CAN1_+
- U6 pad 6: GND1 -> GND2
- U6 pad 7: GND1 -> GND2
Routing:
- net CAN2_A4: track 0.00 -> 113.5 mm
- net CAN2_A3: track 0.00 -> 113.1 mm
- net CAN2_A2: track 0.00 -> 111.2 mm
- net CAN2_A1: track 0.00 -> 109.5 mm
- net CAN2_A0: track 0.00 -> 108.0 mm
- net CAN2_A5: track 0.00 -> 100.2 mm
- net CAN1_A0: track 0.00 -> 82.5 mm, vias 0 -> 2
- net CAN1_A5: track 0.00 -> 81.7 mm, vias 0 -> 2
- net CAN1_A1: track 0.00 -> 80.2 mm, vias 0 -> 2
- net CAN2_TX: track 0.00 -> 78.9 mm, vias 0 -> 2
- net CAN1_A4: track 0.00 -> 78.7 mm, vias 0 -> 2
- net CAN1_A2: track 0.00 -> 78.5 mm, vias 0 -> 2
- net CAN1_A3: track 0.00 -> 78.4 mm, vias 0 -> 2
- net CAN2_RX: track 0.00 -> 77.5 mm, vias 0 -> 2
- net CAN1_TX: track 1.68 -> 44.6 mm, vias 1 -> 4
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Other:
- board size 113.7 x 86.6 mm -> 147.4 x 88.4 mm
