File: Hardware/ciam/impeller/impeller/can.kicad_sch (KiCad schematic)
At the start: 20 parts, among them J1 Conn_01x04, SW1 SW_DIP_x06, U3 ISO1050DUB, U4 B0505MT-1WR4

Commit message: updated ciam project
Parts:
- added C10, C8: 1u, symbol Device:C_Small
- added C14: 4u7, symbol Device:C_Small
- added C16: 10u, symbol Device:C_Small
- added C17: 4n7, symbol Device:C_Small
- added C9: 100n, symbol Device:C_Small
- added D1: PESD1CAN, symbol Power_Protection:PRTR5V0U2X
- added J1: Micro-Fit_1x4P, symbol Connector_Generic:Conn_01x04
- added L1: B82789C0513H002, symbol Device:L_Coupled_1243
- added R1, R2: 60, symbol Device:R_Small
- added R3, R4, R5, R6, R7, R8: 10k, symbol Device:R_Small
- added SW1: SW_DIP_x06, symbol Switch:SW_DIP_x06
- added U3: ISO1050DUB, Package_SO:SOP-8_6.62x9.15mm_P2.54mm, symbol Interface_CAN_LIN:ISO1050DUB
- added U4: B0505MT-1WR4, symbol Interface_CAN_LIN:ISO1050DUB
- J1: value Conn_01x04 -> Micro-Fit_1x4P
Connections:
- net GND: now also C14.2, C8.2, C9.2, SW1.10, SW1.11, SW1.12, SW1.7, SW1.8, SW1.9, U3.4 (GND1), U4.1 (gnd), U4.2 (gnd)
- net GND1: now also J1.4 (Pin_4), C10.2, C16.2, C17.2, D1.3, J1.4 (Pin_4), U3.5 (GND2), U4.6 (0V), U4.7 (0V); no longer J1.1 (Pin_1)
- net VDD_3V3: now also C8.1, C9.1, R3.1, R4.1, R5.1, R6.1, R7.1, R8.1, U3.1 (VCC1)
- net VDD_5V0: now also C14.1, U4.13 (Vin), U4.14 (Vin)
- net at C10.1, C16.1, U3.8 (VCC2)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: now also J1.3 (Pin_3); no longer J1.2 (Pin_2)
- net at D1.2, L1.4, R2.1: now also J1.2 (Pin_2); no longer J1.3 (Pin_3)
- net at D1.1, L1.1, R1.1: now also J1.1 (Pin_1); no longer J1.4 (Pin_4)
- new net: D1.1, J1.1 (Pin_1), L1.1, R1.1
- new net: L1.2, U3.6 (CANL)
- new net: L1.3, U3.7 (CANH)
- new net: D1.2, J1.2 (Pin_2), L1.4, R2.1
- new net: C17.1, R1.2, R2.2
- new net: C10.1, C16.1, J1.3 (Pin_3), U3.8 (VCC2), U4.8 (+Vo)
- new net CAN2_A0: R3.2, SW1.1
- new net CAN2_A1: R4.2, SW1.2
- new net CAN2_A2: R5.2, SW1.3
- new net CAN2_A3: R8.2, SW1.4
- new net CAN2_A4: R7.2, SW1.5
- new net CAN2_A5: R6.2, SW1.6
- new net CAN2_RX: U3.2 (RXD)
- new net CAN2_TX: U3.3 (TXD)
Other:
- note added: "1 CAN L 2 CAN H 3 +5V 4 GND"
- note added: "CAN 1"
- note added: "CAN 1 address"
- note added: "CAN 2"
- note added: "CAN 2 address"
- note removed: "ДОБАВИТЬ 2 CAN ШИНУ!!!!!11!!111!!!!11"
- moved on the sheet: C10, C14, C16, C17, C8, C9, D1, J1, L1, R1, R2, R3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

Commit message: updated impeller project
Parts:
- removed C16: 10u, symbol Device:C_Small
- removed R2: 60, symbol Device:R_Small
- added C16: 10u, symbol Device:C_Small
- added C16 (x4): 0.1u, symbol Device:C_Small
- added R2 (x2): 240, symbol Device:R_Small
- added R2: 60, symbol Device:R_Small
- added R2 (x2): 0, symbol Device:R_Small
- C14: value 4u7 -> 10u
- SW1: value SW_DIP_x06 -> DS1040-06RN
Connections:
- net GND: now also C16.2, C16.2
- net GND1: now also C16.2, C16.2, C16.2, R2.1, R2.1
- net VDD_5V0: now also C16.1, C16.1
- net at D1.2, J1.2 (Pin_2), L1.4: now also R2.1
- net at C10.1, C16.1, U3.8 (VCC2)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: now also C16.1, R2.1, R2.2; no longer J1.3 (Pin_3)
- net at C17.1, R1.2: now also R2.2
- net at C10.1, U3.8 (VCC2), U4.8 (+Vo): now also C16.1, C16.1, R2.1, R2.2; no longer J1.3 (Pin_3)
- new net: J1.3 (Pin_3), R2.2 (x2)
Other:
- note added: "1 CAN L 2 CAN H 3 V_EXT 4 GND_EXT"
- note removed: "1 CAN L 2 CAN H 3 +5V 4 GND"
- note removed: "CAN 2"
- moved on the sheet: C14, C16, C8, R3, R4, R5, R6, R7, R8, SW1, U4

Commit message: multiple fixes
Parts:
- removed R2 (x2): 240, symbol Device:R_Small
- C10, C8: footprint (none) -> Capacitor_SMD:C_0805_2012Metric; Ссылка (none) -> https://www.chipdip.ru/product/grm21br71e105k; Цена (none) -> 13
- C14, C16: footprint (none) -> Capacitor_SMD:C_0805_2012Metric; Ссылка (none) -> https://www.chipdip.ru/product/grm21br61e106ka73l; Цена (none) -> 13
- C16: value 0.1u -> 100n; footprint (none) -> Capacitor_SMD:C_0805_2012Metric; Ссылка (none) -> https://www.chipdip.ru/product/grm21br71h104k; Цена (none) -> 13
- C17: footprint (none) -> Capacitor_SMD:C_0805_2012Metric; Ссылка (none) -> https://www.chipdip.ru/product/grm216r71h472k; Цена (none) -> 8
- C9: footprint (none) -> Capacitor_SMD:C_0805_2012Metric; Ссылка (none) -> https://www.chipdip.ru/product/grm21br71h104k; Цена (none) -> 13
- D1: Ссылка (none) -> https://www.chipdip.ru/product/pesd1can.215; Цена (none) -> 87
- J1: value Micro-Fit_1x4P -> Micro-Fit_2x2P; Ссылка (none) -> https://www.chipdip.ru/product/sct3001wv-2x02p; Цена (none) -> 26
- L1: Ссылка (none) -> https://www.chipdip.ru/product0/8002015174; Цена (none) -> 510
- R1, R2: footprint (none) -> Resistor_SMD:R_0603_1608Metric
- R2: footprint (none) -> Resistor_SMD:R_0805_2012Metric; Ссылка (none) -> https://www.chipdip.ru/product/0.125w-0805-peremychka-0-om; Цена (none) -> 5
- R3, R4, R5, R6, R7, R8: footprint (none) -> Resistor_SMD:R_0805_2012Metric; Ссылка (none) -> https://www.chipdip.ru/product/0.125w-0805-10-kom-5; Цена (none) -> 5
- SW1: Ссылка (none) -> https://www.chipdip.ru/product/ds1040-06rn; Цена (none) -> 38
- U3: Ссылка (none) -> https://energoflot.ru/item/ISO1050DUB; Цена (none) -> 225
- U4: Ссылка (none) -> https://www.chipdip.ru/product0/8003333290; Цена (none) -> 120

Commit message: updated bom
Parts:
- C10, C8: Человекопонятное название (none) -> Конденсатор 1мкФ
- C14, C16: Человекопонятное название (none) -> Конденсатор 10мкФ
- C16, C9: Человекопонятное название (none) -> Конденсатор 100нФ
- C17: Человекопонятное название (none) -> Конденсатор 4.7нФ
- D1: Человекопонятное название (none) -> Защитный диод от ESD для CAN шины
- J1: Человекопонятное название (none) -> Разъем Micro-Fit 2x2 М
- L1: Человекопонятное название (none) -> Подавитель синфазных помех
- R1, R2: Человекопонятное название (none) -> Резистор 60 Ом
- R2: Человекопонятное название (none) -> Резистор 0 ОМ (перемычка)
- R3, R4, R5, R6, R7, R8: Человекопонятное название (none) -> Резистор 10k Ом
- SW1: Человекопонятное название (none) -> DIP переключатель 6pin красный
- U3: Человекопонятное название (none) -> Изолированный приемопередатчик интерфейса CAN
- U4: Человекопонятное название (none) -> DC/DC преобразователь

Commit message: Updated CIAM project
Parts:
- D1: footprint (none) -> Package_TO_SOT_SMD:SOT-23
- J1: footprint (none) -> Connector_Molex:Molex_Micro-Fit_3.0_43045-0400_2x02_P3.00mm_Horizontal; Ссылка https://www.chipdip.ru/product/sct3001wv-2x02p -> https://www.chipdip.ru/product/sct3001wr-2x02p
- L1: footprint (none) -> user_lib:B82789C0513H002
- SW1: footprint (none) -> Button_Switch_THT:SW_DIP_SPSTx08_Slide_9.78x22.5mm_W7.62mm_P2.54mm
- U4: footprint (none) -> user_lib:B0505MT-1WR4
Changed lines of the file:
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@@
       (effects (font (size 1.27 1.27)))
     )
-    (property "Footprint" "" (at 194.945 36.195 0)
+    (property "Footprint" "user_lib:B82789C0513H002" (at 194.945 36.195 0)
       (effects (font (size 1.27 1.27)) hide)
     )
@@
       (effects (font (size 1.27 1.27)))
     )
-    (property "Footprint" "" (at 231.775 88.9 0)
+    (property "Footprint" "user_lib:B0505MT-1WR4" (at 231.775 88.9 0)
       (effects (font (size 1.27 1.27) italic) hide)
     )
@@
       (effects (font (size 1.27 1.27)))
     )
-    (property "Footprint" "" (at 100.33 88.9 0)
+    (property "Footprint" "user_lib:B0505MT-1WR4" (at 100.33 88.9 0)
       (effects (font (size 1.27 1.27) italic) hide)
     )
@@
       (effects (font (size 1.27 1.27)))
     )
-    (property "Footprint" "" (at 238.76 140.97 0)
+    (property "Footprint" "Button_Switch_THT:SW_DIP_SPSTx08_Slide_9.78x22.5mm_W7.62mm_P2.54mm" (at 238.76 140.97 0)
       (effects (font (size 1.27 1.27)) hide)
     )
@@
       (effects (font (size 1.27 1.27)))
     )
-    (property "Footprint" "" (at 36.195 89.535 0)
+    (property "Footprint" "Package_TO_SOT_SMD:SOT-23" (at 36.195 89.535 0)
       (effects (font (size 1.27 1.27)) hide)
     )
@@
       (effects (font (size 1.27 1.27)))
     )
-    (property "Footprint" "" (at 33.02 69.215 0)
-      (effects (font (size 1.27 1.27)) hide)
-    )
-    (property "Datasheet" "~" (at 33.02 69.215 0)
-      (effects (font (size 1.27 1.27)) hide)
-    )
-    (property "Ссылка" "https://www.chipdip.ru/product/sct3001wv-2x02p" (at 33.02 69.215 0)
+    (property "Footprint" "Connector_Molex:Molex_Micro-Fit_3.0_43045-0400_2x02_P3.00mm_Horizontal" (at 33.02 69.215 0)
+      (effects (font (size 1.27 1.27)) hide)
+    )
+    (property "Datasheet" "" (at 33.02 69.215 0)
+      (effects (font (size 1.27 1.27)) hide)
+    )
+    (property "Ссылка" "https://www.chipdip.ru/product/sct3001wr-2x02p" (at 33.02 69.215 0)
       (effects (font (size 1.27 1.27)) hide)
     )
@@
       (effects (font (size 1.27 1.27)))
     )
-    (property "Footprint" "" (at 106.68 140.97 0)
+    (property "Footprint" "Button_Switch_THT:SW_DIP_SPSTx08_Slide_9.78x22.5mm_W7.62mm_P2.54mm" (at 106.68 140.97 0)
       (effects (font (size 1.27 1.27)) hide)
     )
@@
       (effects (font (size 1.27 1.27)))
     )
-    (property "Footprint" "" (at 63.5 36.195 0)
+    (property "Footprint" "user_lib:B82789C0513H002" (at 63.5 36.195 0)
       (effects (font (size 1.27 1.27)) hide)
     )
@@
       (effects (font (size 1.27 1.27)))
     )
-    (property "Footprint" "" (at 164.465 69.215 0)
-      (effects (font (size 1.27 1.27)) hide)
-    )
-    (property "Datasheet" "~" (at 164.465 69.215 0)
-      (effects (font (size 1.27 1.27)) hide)
-    )
-    (property "Ссылка" "https://www.chipdip.ru/product/sct3001wv-2x02p" (at 164.465 69.215 0)
+    (property "Footprint" "Connector_Molex:Molex_Micro-Fit_3.0_43045-0400_2x02_P3.00mm_Horizontal" (at 164.465 69.215 0)
+      (effects (font (size 1.27 1.27)) hide)
+    )
+    (property "Datasheet" "" (at 164.465 69.215 0)
+      (effects (font (size 1.27 1.27)) hide)
+    )
+    (property "Ссылка" "https://www.chipdip.ru/product/sct3001wr-2x02p" (at 164.465 69.215 0)
       (effects (font (size 1.27 1.27)) hide)
     )
@@
       (effects (font (size 1.27 1.27)))
     )
-    (property "Footprint" "" (at 167.64 89.535 0)
-      (effects (font (size 1.27 1.27)) hide)
-    )
+    (property "Footprint" "Package_TO_SOT_SMD:SOT-23" (at 167.64 89.535 0)
+      (effects (font (size 1.27 1.27)) hide)
+    )

Commit message: Updated CIAM project
Parts:
- SW1: footprint Button_Switch_THT:SW_DIP_SPSTx08_Slide_9.78x22.5mm_W7.62mm_P2.54mm -> Button_Switch_THT:SW_DIP_SPSTx06_Slide_9.78x17.42mm_W7.62mm_P2.54mm
Connections:
- net CAN1_RX: now also U3.2 (RXD); no longer U3.2 (RXD)
- net CAN1_TX: now also U3.3 (TXD); no longer U3.3 (TXD)
- net CAN2_RX: now also U3.2 (RXD); no longer U3.2 (RXD)
- net CAN2_TX: now also U3.3 (TXD); no longer U3.3 (TXD)
- net GND1: no longer C10.2, C16.2, C16.2, C17.2, D1.3, J1.4 (Pin_4), U3.5 (GND2), U4.6 (0V), U4.7 (0V)
- net CAN1-: now reaches D1.1, J1.1 (Pin_1), R1.1
- net CAN1-: now also L1.2; no longer L1.1
- net CAN1_-: now reaches U3.6 (CANL)
- net CAN1_-: now also L1.1; no longer L1.2
- net CAN1+: now reaches L1.3
- net CAN1+: now also D1.2, J1.2 (Pin_2), R2.1; no longer U3.7 (CANH)
- net CAN2+: now reaches D1.2, J1.2 (Pin_2), R2.1
- net CAN2+: now also L1.3; no longer L1.4
- net CAN2-: now reaches D1.1, J1.1 (Pin_1), R1.1
- net CAN2-: now also L1.2; no longer L1.1
- net CAN2_-: now reaches U3.6 (CANL)
- net CAN2_-: now also L1.1; no longer L1.2
- net CAN2_+: now reaches U3.7 (CANH)
- net CAN2_+: now also L1.4; no longer L1.3
- new net CAN1_+: L1.4, U3.7 (CANH)
- new net GND2: C10.2, C16.2, C16.2, C17.2, D1.3, J1.4 (Pin_4), U3.5 (GND2), U4.6 (0V), U4.7 (0V)
Other:
- note added: "CAN 2"
