File: Hardware/ciam/impeller/impeller/connectors.kicad_sch (KiCad schematic)
At the start: 15 parts, among them J12 Micro-Fit_2x2P, J29 USB_A, J4 MicroFit_2x2, J4 Pinheader_2x5, U19 TLP521-2, U2 B0503S-1WR3, U4 USBLC6-2SC6

Commit message: updated impeller project
Parts:
- removed C48: 10u, symbol Device:C
- removed C49: 4u7, symbol Device:C
- removed J4: Pinheader_2x5, Connector_PinHeader_1.27mm:PinHeader_2x05_P1.27mm_Vertical, symbol Connector_Generic:Conn_02x05_Odd_Even
- removed J4: MicroFit_2x2, symbol Connector_Generic:Conn_02x02_Odd_Even
- removed R54 (x2): 470, symbol Device:R_Small
- removed R56 (x2): 10k, symbol Device:R_Small
- removed U19: TLP521-2, symbol Isolator:TLP291
- removed U2: B0503S-1WR3, symbol Converter_DCDC:TMR-1211
- added C14: 4u7, symbol Device:C_Small
- added C16: 10u, symbol Device:C_Small
- added C59: 100n, symbol Device:C_Small
- added C62: 100n, symbol Device:C
- added C63: 4u7, symbol Device:C
- added J17: Conn_01x05, symbol Connector_Generic:Conn_01x05
- added Q1, Q2: BSS138, Package_TO_SOT_SMD:SOT-23, symbol Transistor_FET:BSS138
- added R100, R101, R102, R99: 10k, symbol Device:R_Small
- added R51 (x2): 220, symbol Device:R_Small
- added U4: B0505MT-1WR4, symbol Interface_CAN_LIN:ISO1050DUB
- added U46: HCPL-0630, Package_SO:SOIC-8_3.9x4.9mm_P1.27mm, symbol Isolator:HCPL-0630
- added U47: LDL1117S33R, Package_TO_SOT_SMD:SOT-223-3_TabPin2, symbol Regulator_Linear:LD1117S33TR_SOT223
Connections:
- net GND: now also J12.2 (Pin_2), J12.4 (Pin_4), C14.2, J17.2 (Pin_2), U4.1 (gnd), U4.2 (gnd)
- net NRST: now also J17.5 (Pin_5)
- net SWD_SWCLK: now also J17.3 (Pin_3)
- net SWD_SWDIO: now also J17.1 (Pin_1)
- net USART3_RX: now also R51.1
- net USART3_TX: now also R51.1
- net VDD_3V3: now also J17.4 (Pin_4), U46.2 (C1), U46.3 (C2)
- net VDD_5V0: now also C14.1, C16.1, C59.1, C62.1, R101.1, R99.1, U4.13 (Vin), U4.14 (Vin), U4.8 (+Vo), U46.8 (VCC), U47.3 (VI)
- net at J12.3 (Pin_3): now also Q2.2 (S), R102.2; no longer J12.1 (Pin_1)
- new net: C16.2, C59.2, C62.2, C63.2, U4.6 (0V), U4.7 (0V), U46.5 (GND), U47.1 (GND)
- new net: R51.2, U46.4 (A2)
- new net: R51.2, U46.1 (A1)
- new net: Q2.3 (D), R101.2, U46.6 (VO2)
- new net: Q1.3 (D), R99.2, U46.7 (VO1)
- new net: C63.1, Q1.1 (G), Q2.1 (G), R100.1, R102.1, U47.2 (VO)
- new net: J12.1 (Pin_1), Q1.2 (S), R100.2
- no-connect marks 2 -> 0
Other:
- note removed: "UART3 RPi<->Stm32"
- moved on the sheet: J12

Commit message: multiple fixes
Parts:
- C14, C63: footprint (none) -> Capacitor_SMD:C_0805_2012Metric; Ссылка (none) -> https://www.chipdip.ru/product/grm21br61e475ka12l; Цена (none) -> 13
- C16: footprint (none) -> Capacitor_SMD:C_0805_2012Metric; Ссылка (none) -> https://www.chipdip.ru/product/grm21br61e106ka73l; Цена (none) -> 13
- C20: Ссылка (none) -> https://www.chipdip.ru/product/grm188r71h104k; Цена (none) -> 19
- C59, C62: footprint (none) -> Capacitor_SMD:C_0805_2012Metric; Ссылка (none) -> https://www.chipdip.ru/product/grm21br71h104k; Цена (none) -> 13
- D3: renamed from D13; Ссылка (none) -> https://www.chipdip.ru/product/ss24-umw; Цена (none) -> 5
- J12: Ссылка (none) -> https://www.chipdip.ru/product/sct3001wv-2x02p; Цена (none) -> 26
- J14: renamed from J17; value Conn_01x05 -> PLS-5; Ссылка (none) -> https://www.chipdip.ru/product/pls-5; Цена (none) -> 8
- J29: value USB_A -> USBA-1J; Ссылка (none) -> https://www.chipdip.ru/product/usba-1j; Цена (none) -> 22
- Q1, Q2: Ссылка (none) -> https://www.chipdip.ru/product/bss138-umw; Цена (none) -> 3
- R100, R101, R102, R99: footprint (none) -> Resistor_SMD:R_0805_2012Metric; Ссылка (none) -> https://www.chipdip.ru/product/0.125w-0805-10-kom-5; Цена (none) -> 5
- R51: footprint (none) -> Resistor_SMD:R_0603_1608Metric; Ссылка (none) -> https://www.chipdip.ru/product/0.1w-0603-220-om-1; Цена (none) -> 5
- U4: Ссылка (none) -> https://www.chipdip.ru/product0/8003333290; Цена (none) -> 120
- U4: Ссылка (none) -> https://www.chipdip.ru/product/usblc6-2sc6; Цена (none) -> 25
- U47: Ссылка (none) -> https://www.chipdip.ru/product/ldl1117s33r-stm; Цена (none) -> 33
Other:
- moved on the sheet: J12

Commit message: updated bom
Parts:
- C14, C63: Человекопонятное название (none) -> Конденсатор 4.7мкФ
- C16: Человекопонятное название (none) -> Конденсатор 10мкФ
- C20, C59, C62: Человекопонятное название (none) -> Конденсатор 100нФ
- D3: Человекопонятное название (none) -> Диод Шоттки
- J12: Человекопонятное название (none) -> Разъем Micro-Fit 2x2 М
- J14: Человекопонятное название (none) -> Вилка штыревая 1x5
- J29: Человекопонятное название (none) -> Разъем USB A
- Q1, Q2: Человекопонятное название (none) -> Транзистор полевой n типа
- R100, R101, R102, R99: Человекопонятное название (none) -> Резистор 10k Ом
- R51: Человекопонятное название (none) -> Резистор 220 Ом
- U4: Человекопонятное название (none) -> DC/DC преобразователь
- U4: Человекопонятное название (none) -> Защита интерфейса USB от электростатических разрядов
- U46: Человекопонятное название (none) -> Оптопара двухканальная с логическими уровнями на выходе
- U47: Человекопонятное название (none) -> LDO-стабилизатор напряжения
Changed lines of the file:
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@@
+      (effects (font (size 1.27 1.27)) hide)
+    )
+    (property "Человекопонятное название" "Конденсатор 100нФ" (at 100.33 148.59 0)
       (effects (font (size 1.27 1.27)) hide)
     )
@@
     )
     (property "Цена" "5" (at 66.04 118.745 0)
+      (effects (font (size 1.27 1.27)) hide)
+    )
+    (property "Человекопонятное название" "Резистор 220 Ом" (at 66.04 118.745 0)
       (effects (font (size 1.27 1.27)) hide)
     )
@@
     )
     (property "Цена" "" (at 77.47 111.125 0)
+      (effects (font (size 1.27 1.27)) hide)
+    )
+    (property "Человекопонятное название" "Оптопара двухканальная с логическими уровнями на выходе" (at 77.47 111.125 0)
       (effects (font (size 1.27 1.27)) hide)
     )
@@
       (effects (font (size 1.27 1.27)) hide)
     )
+    (property "Человекопонятное название" "Конденсатор 10мкФ" (at 72.39 147.32 0)
+      (effects (font (size 1.27 1.27)) hide)
+    )
     (pin "1")
     (pin "2")
@@
       (effects (font (size 1.27 1.27)) hide)
     )
+    (property "Человекопонятное название" "Конденсатор 4.7мкФ" (at 135.255 148.59 0)
+      (effects (font (size 1.27 1.27)) hide)
+    )
     (pin "1")
     (pin "2")
@@
       (effects (font (size 1.27 1.27)) hide)
     )
+    (property "Человекопонятное название" "LDO-стабилизатор напряжения" (at 116.205 143.51 0)
+      (effects (font (size 1.27 1.27)) hide)
+    )
     (pin "1")
     (pin "2")
@@
       (effects (font (size 1.27 1.27)) hide)
     )
+    (property "Человекопонятное название" "Резистор 10k Ом" (at 127.635 113.665 0)
+      (effects (font (size 1.27 1.27)) hide)
+    )
     (pin "1")
     (pin "2")
@@
       (effects (font (size 1.27 1.27)) hide)
     )
+    (property "Человекопонятное название" "Разъем Micro-Fit 2x2 М" (at 151.13 106.045 0)
+      (effects (font (size 1.27 1.27)) hide)
+    )
     (pin "1")
     (pin "2")
@@
     )
     (property "Цена" "5" (at 127.635 100.965 0)
+      (effects (font (size 1.27 1.27)) hide)
+    )
+    (property "Человекопонятное название" "Резистор 10k Ом" (at 127.635 100.965 0)
       (effects (font (size 1.27 1.27)) hide)
     )
@@
       (effects (font (size 1.27 1.27)) hide)
     )
+    (property "Человекопонятное название" "Разъем USB A" (at 43.18 52.07 0)
+      (effects (font (size 1.27 1.27)) hide)
+    )
     (pin "1")
     (pin "2")
@@
       (effects (font (size 1.27 1.27)) hide)
     )
+    (property "Человекопонятное название" "Резистор 220 Ом" (at 66.04 103.505 0)
+      (effects (font (size 1.27 1.27)) hide)
+    )
     (pin "1")
     (pin "2")
@@
       (effects (font (size 1.27 1.27)) hide)
     )
+    (property "Человекопонятное название" "Транзистор полевой n типа" (at 121.285 116.205 0)
+      (effects (font (size 1.27 1.27)) hide)
+    )
     (pin "1")
     (pin "2")
@@
     )
     (property "Цена" "120" (at 51.435 146.05 0)
+      (effects (font (size 1.27 1.27)) hide)
+    )
+    (property "Человекопонятное название" "DC/DC преобразователь" (at 51.435 146.05 0)
       (effects (font (size 1.27 1.27)) hide)
     )
@@
       (effects (font (size 1.27 1.27)) hide)
     )
+    (property "Человекопонятное название" "Конденсатор 100нФ" (at 33.655 52.705 0)
+      (effects (font (size 1.27 1.27)) hide)
+    )
     (pin "1")
     (pin "2")
@@
       (effects (font (size 1.27 1.27)) hide)
     )
+    (property "Человекопонятное название" "Вилка штыревая 1x5" (at 155.575 45.085 0)
+      (effects (font (size 1.27 1.27)) hide)
+    )
     (pin "1")
     (pin "2")
@@
       (effects (font (size 1.27 1.27)) hide)
     )
+    (property "Человекопонятное название" "Конденсатор 4.7мкФ" (at 35.56 147.32 0)
+      (effects (font (size 1.27 1.27)) hide)
+    )
     (pin "1")
     (pin "2")
@@
       (effects (font (size 1.27 1.27)) hide)
     )
+    (property "Человекопонятное название" "Транзистор полевой n типа" (at 121.285 103.505 0)
+      (effects (font (size 1.27 1.27)) hide)
+    )
     (pin "1")
     (pin "2")
@@
     )
     (property "Цена" "25" (at 92.075 53.34 0)
+      (effects (font (size 1.27 1.27)) hide)
+    )
+    (property "Человекопонятное название" "Защита интерфейса USB от электростатических разрядов" (at 92.075 53.34 0)
       (effects (font (size 1.27 1.27)) hide)
     )
@@
       (effects (font (size 1.27 1.27)) hide)
     )
+    (property "Человекопонятное название" "Диод Шоттки" (at 57.785 46.99 0)
+      (effects (font (size 1.27 1.27)) hide)
+    )
     (pin "1")
     (pin "2")
@@
       (effects (font (size 1.27 1.27)) hide)
     )
+    (property "Человекопонятное название" "Резистор 10k Ом" (at 114.935 113.665 0)
+      (effects (font (size 1.27 1.27)) hide)
+    )
     (pin "1")
     (pin "2")
@@
     )
     (property "Цена" "5" (at 114.935 100.965 0)
+      (effects (font (size 1.27 1.27)) hide)
+    )
+    (property "Человекопонятное название" "Резистор 10k Ом" (at 114.935 100.965 0)
       (effects (font (size 1.27 1.27)) hide)
     )
@@
       (effects (font (size 1.27 1.27)) hide)
     )
+    (property "Человекопонятное название" "Конденсатор 100нФ" (at 85.725 100.965 0)
+      (effects (font (size 1.27 1.27)) hide)
+    )

Commit message: Updated CIAM project
Parts:
- removed D3: ss24, symbol Device:D_Schottky
- removed J29: USBA-1J, symbol Connector:USB_A
- added C23: 100n, Capacitor_SMD:C_0603_1608Metric, symbol Device:C_Small
- added J16: Conn_02x05_SWD, Connector_PinHeader_1.27mm:PinHeader_2x05_P1.27mm_Vertical, symbol Connector_Generic:Conn_02x05_Odd_Even
- added J3: USB_B_Micro, user_lib:U-F-M5DD-W-2-SUS, symbol Connector:USB_B_Micro
- added J4: Micro_SD_Card_Con, sd:TF01A, symbol Connector:Micro_SD_Card_Det1
- added R17, R18, R19, R20, R21, R22: 100k, Resistor_SMD:R_0603_1608Metric, symbol Device:R_Small
- J12: footprint (none) -> Connector_Molex:Molex_Micro-Fit_3.0_43045-0400_2x02_P3.00mm_Horizontal; Ссылка https://www.chipdip.ru/product/sct3001wv-2x02p -> https://www.chipdip.ru/product/sct3001wr-2x02p
- J14: footprint (none) -> Connector_PinHeader_2.54mm:PinHeader_1x05_P2.54mm_Vertical
- U4: footprint (none) -> user_lib:B0505MT-1WR4
Connections:
- net GND: now also C23.1, J16.3 (Pin_3), J16.5 (Pin_5), J16.9 (Pin_9), J3.5 (GND), J3.6 (Shield), J4.10 (SHIELD), J4.6 (VSS); no longer J12.2 (Pin_2), J12.4 (Pin_4)
- net NRST: now also J16.10 (Pin_10)
- net SWD_SWCLK: now also J16.4 (Pin_4)
- net SWD_SWDIO: now also J16.2 (Pin_2)
- net VDD_3V3: now also C23.2, J16.1 (Pin_1), J4.4 (VDD), R17.1, R18.1, R19.1, R20.1, R21.1, R22.1
- net VDD_5V0: no longer C16.1, C20.1, C59.1, C62.1, R101.1, R99.1, U4.8 (+Vo), U46.8 (VCC), U47.3 (VI)
- net usb_conn_d+: now also J3.3 (D+)
- net usb_conn_d-: now also J3.2 (D-)
- net GND_ISO_UART3: now reaches C16.2, C59.2, C62.2, C63.2, U4.6 (0V), U4.7 (0V), U46.5 (GND), U47.1 (GND)
- net GND_ISO_UART3: now also J12.2 (Pin_2), J12.4 (Pin_4)
- new net SDIO_CLK: J4.5 (CLK)
- new net SDIO_CMD: J4.3 (CMD), R20.2
- new net SDIO_DAT0: J4.7 (DAT0), R19.2
- new net SDIO_DAT1: J4.8 (DAT1), R18.2
- new net SDIO_DAT2: J4.1 (DAT2), R22.2
- new net SDIO_DAT3: J4.2 (DAT3/CD), R21.2
- new net SD_CD: J4.9 (DET), R17.2
- new net SWD_SWO: J16.6 (Pin_6)
- new net VDD_5V0_ISO_UART3: C16.1, C59.1, C62.1, R101.1, R99.1, U4.8 (+Vo), U46.8 (VCC), U47.3 (VI)
- new net VDD_5V_VBUS: C20.1, J3.1 (VBUS)
- no-connect marks 0 -> 3
Other:
- note added: "Micro SD"
- note added: "SWD"
- note removed: "РУД"
- moved on the sheet: C14, C16, C59, C62, C63, J12, J14, Q1, Q2, R100, R101, R102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

Commit message: added thrust lever
Parts:
- added J12: Micro-Fit_2x2P, Connector_Molex:Molex_Micro-Fit_3.0_43045-0400_2x02_P3.00mm_Horizontal, symbol Connector_Generic:Conn_02x02_Odd_Even
- added R51 (x2): 220, Resistor_SMD:R_0603_1608Metric, symbol Device:R_Small
- added R52 (x2): 360, Resistor_SMD:R_0603_1608Metric, symbol Device:R_Small
- R17, R18, R19, R20, R21, R22: Ссылка (none) -> https://www.chipdip.ru/product/0.1w-0603-100-kom-1; Цена (none) -> 5; Человекопонятное название (none) -> Резистор 100k Ом
Connections:
- net GND: now also R52.1, R52.1
- net VDD_5V0: now also J12.1 (Pin_1), J12.3 (Pin_3)
- new net: J12.2 (Pin_2), R51.1
- new net: J12.4 (Pin_4), R51.1
- new net ThrustLever1: R51.2, R52.2
- new net ThrustLever2: R51.2, R52.2
Other:
- note added: "Thrust lever"
- moved on the sheet: J14, J16

Commit message: updated thrust level voltage divider
Parts:
- R51: value 220 -> 1k; Ссылка https://www.chipdip.ru/product/0.1w-0603-220-om-1 -> https://www.chipdip.ru/product/0.1w-0603-1-kom-1
- R52: value 360 -> 2k; Ссылка https://www.chipdip.ru/product/0.1w-0603-360-om-1 -> https://www.chipdip.ru/product/0.1w-0603-2-kom-1
Changed lines of the file:
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@@
       (effects (font (size 1.27 1.27)))
     )
-    (property "Value" "360" (at 219.075 142.875 90)
+    (property "Value" "2k" (at 219.075 142.875 90)
       (effects (font (size 1.27 1.27)))
     )
@@
       (effects (font (size 1.27 1.27)) hide)
     )
-    (property "Ссылка" "https://www.chipdip.ru/product/0.1w-0603-360-om-1" (at 219.075 144.78 0)
+    (property "Ссылка" "https://www.chipdip.ru/product/0.1w-0603-2-kom-1" (at 219.075 144.78 0)
       (effects (font (size 1.27 1.27)) hide)
     )
@@
     )
   )
+  (symbol (lib_id "Device:R_Small") (at 219.075 153.035 270) (unit 1)
+    (in_bom yes) (on_board yes) (dnp no)
+    (property "Reference" "R52" (at 219.075 154.94 90)
+      (effects (font (size 1.27 1.27)))
+    )
+    (property "Value" "2k" (at 219.075 151.13 90)
+      (effects (font (size 1.27 1.27)))
+    )
+    (property "Footprint" "Resistor_SMD:R_0603_1608Metric" (at 219.075 153.035 0)
+      (effects (font (size 1.27 1.27)) hide)
+    )
+    (property "Datasheet" "~" (at 219.075 153.035 0)
+      (effects (font (size 1.27 1.27)) hide)
+    )
+    (property "Ссылка" "https://www.chipdip.ru/product/0.1w-0603-2-kom-1" (at 219.075 153.035 0)
+      (effects (font (size 1.27 1.27)) hide)
+    )
+    (property "Цена" "5" (at 219.075 153.035 0)
+      (effects (font (size 1.27 1.27)) hide)
+    )
+    (property "Человекопонятное название" "Резистор 360 Ом" (at 219.075 153.035 0)
+      (effects (font (size 1.27 1.27)) hide)
+    )
+    (pin "1")
+    (pin "2")
+    (instances
+      (project "impeller"
+        (path "/dc9d3fdd-86e3-4a65-b009-b0cbd29a6eee/7a5f1b8e-a29e-483a-94c0-c542bb8c7cf0"
+          (reference "R52") (unit 1)
+        )
+        (path "/dc9d3fdd-86e3-4a65-b009-b0cbd29a6eee/5a3c1b9c-681a-4723-b2b5-156fdda94574"
+          (reference "R106") (unit 1)
+        )
+      )
+    )
+  )
   (symbol (lib_id "Device:R_Small") (at 127.635 125.73 0) (mirror y) (unit 1)
     (in_bom yes) (on_board yes) (dnp no)
@@
     )
   )
-  (symbol (lib_id "Device:R_Small") (at 219.075 153.035 270) (unit 1)
-    (in_bom yes) (on_board yes) (dnp no)
-    (property "Reference" "R52" (at 219.075 154.94 90)
-      (effects (font (size 1.27 1.27)))
-    )
-    (property "Value" "360" (at 219.075 151.13 90)
-      (effects (font (size 1.27 1.27)))
-    )
-    (property "Footprint" "Resistor_SMD:R_0603_1608Metric" (at 219.075 153.035 0)
-      (effects (font (size 1.27 1.27)) hide)
-    )
-    (property "Datasheet" "~" (at 219.075 153.035 0)
-      (effects (font (size 1.27 1.27)) hide)
-    )
-    (property "Ссылка" "https://www.chipdip.ru/product/0.1w-0603-360-om-1" (at 219.075 153.035 0)
-      (effects (font (size 1.27 1.27)) hide)
-    )
-    (property "Цена" "5" (at 219.075 153.035 0)
-      (effects (font (size 1.27 1.27)) hide)
-    )
-    (property "Человекопонятное название" "Резистор 360 Ом" (at 219.075 153.035 0)
-      (effects (font (size 1.27 1.27)) hide)
-    )
-    (pin "1")
-    (pin "2")
-    (instances
-      (project "impeller"
-        (path "/dc9d3fdd-86e3-4a65-b009-b0cbd29a6eee/7a5f1b8e-a29e-483a-94c0-c542bb8c7cf0"
-          (reference "R52") (unit 1)
-        )
-        (path "/dc9d3fdd-86e3-4a65-b009-b0cbd29a6eee/5a3c1b9c-681a-4723-b2b5-156fdda94574"
-          (reference "R106") (unit 1)
-        )
-      )
-    )
-  )
   (symbol (lib_id "Device:R_Small") (at 66.04 115.57 90) (unit 1)
     (in_bom yes) (on_board yes) (dnp no)
@@
       (effects (font (size 1.27 1.27)))
     )
-    (property "Value" "220" (at 208.915 142.875 90)
+    (property "Value" "1k" (at 208.915 142.875 90)
       (effects (font (size 1.27 1.27)))
     )
@@
       (effects (font (size 1.27 1.27)) hide)
     )
-    (property "Ссылка" "https://www.chipdip.ru/product/0.1w-0603-220-om-1" (at 208.915 144.78 0)
+    (property "Ссылка" "https://www.chipdip.ru/product/0.1w-0603-1-kom-1" (at 208.915 144.78 0)
       (effects (font (size 1.27 1.27)) hide)
     )
@@
     )
   )
-  (symbol (lib_id "Device:R_Small") (at 208.915 153.035 90) (unit 1)
-    (in_bom yes) (on_board yes) (dnp no)
-    (property "Reference" "R51" (at 208.915 154.94 90)
-      (effects (font (size 1.27 1.27)))
-    )
-    (property "Value" "220" (at 208.915 151.13 90)
-      (effects (font (size 1.27 1.27)))
-    )
-    (property "Footprint" "Resistor_SMD:R_0603_1608Metric" (at 208.915 153.035 0)
-      (effects (font (size 1.27 1.27)) hide)
-    )
-    (property "Datasheet" "~" (at 208.915 153.035 0)
-      (effects (font (size 1.27 1.27)) hide)
-    )
-    (property "Ссылка" "https://www.chipdip.ru/product/0.1w-0603-220-om-1" (at 208.915 153.035 0)
-      (effects (font (size 1.27 1.27)) hide)
-    )
-    (property "Цена" "5" (at 208.915 153.035 0)
-      (effects (font (size 1.27 1.27)) hide)
-    )
-    (property "Человекопонятное название" "Резистор 220 Ом" (at 208.915 153.035 0)
-      (effects (font (size 1.27 1.27)) hide)
-    )
-    (pin "1")
-    (pin "2")
-    (instances
-      (project "impeller"
-        (path "/dc9d3fdd-86e3-4a65-b009-b0cbd29a6eee/7a5f1b8e-a29e-483a-94c0-c542bb8c7cf0"
-          (reference "R51") (unit 1)
-        )
-        (path "/dc9d3fdd-86e3-4a65-b009-b0cbd29a6eee/0a393be1-a79e-48b5-bd67-1675300f121e"
-          (reference "R97") (unit 1)
-        )
-        (path "/dc9d3fdd-86e3-4a65-b009-b0cbd29a6eee/5a3c1b9c-681a-4723-b2b5-156fdda94574"
-          (reference "R105") (unit 1)
-        )
-      )
-    )
-  )
   (symbol (lib_id "Connector_Generic:Conn_01x05") (at 209.55 107.95 0) (unit 1)
     (in_bom yes) (on_board yes) (dnp no)
@@
         )
       )
+    )
+  )
+  (symbol (lib_id "Device:R_Small") (at 208.915 153.035 90) (unit 1)
+    (in_bom yes) (on_board yes) (dnp no)
+    (property "Reference" "R51" (at 208.915 154.94 90)
+      (effects (font (size 1.27 1.27)))
+    )
+    (property "Value" "1k" (at 208.915 151.13 90)
+      (effects (font (size 1.27 1.27)))
+    )
+    (property "Footprint" "Resistor_SMD:R_0603_1608Metric" (at 208.915 153.035 0)
+      (effects (font (size 1.27 1.27)) hide)
+    )
+    (property "Datasheet" "~" (at 208.915 153.035 0)
+      (effects (font (size 1.27 1.27)) hide)
+    )
+    (property "Ссылка" "https://www.chipdip.ru/product/0.1w-0603-1-kom-1" (at 208.915 153.035 0)
+      (effects (font (size 1.27 1.27)) hide)
+    )
+    (property "Цена" "5" (at 208.915 153.035 0)
+      (effects (font (size 1.27 1.27)) hide)
+    )
+    (property "Человекопонятное название" "Резистор 220 Ом" (at 208.915 153.035 0)
+      (effects (font (size 1.27 1.27)) hide)
+    )
+    (pin "1")
+    (pin "2")
+    (instances
+      (project "impeller"
+        (path "/dc9d3fdd-86e3-4a65-b009-b0cbd29a6eee/7a5f1b8e-a29e-483a-94c0-c542bb8c7cf0"
+          (reference "R51") (unit 1)
+        )
+        (path "/dc9d3fdd-86e3-4a65-b009-b0cbd29a6eee/0a393be1-a79e-48b5-bd67-1675300f121e"
+          (reference "R97") (unit 1)
+        )
+        (path "/dc9d3fdd-86e3-4a65-b009-b0cbd29a6eee/5a3c1b9c-681a-4723-b2b5-156fdda94574"
+          (reference "R105") (unit 1)
+        )
+      )

Commit message: Updated CIAM project
Parts:
- R51: Человекопонятное название Резистор 220 Ом -> Резистор 1К ОМ
- R52: Человекопонятное название Резистор 360 Ом -> Резистор 2К ОМ
Changed lines of the file:
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@@
       (effects (font (size 1.27 1.27)) hide)
     )
-    (property "Человекопонятное название" "Резистор 360 Ом" (at 219.075 144.78 0)
+    (property "Человекопонятное название" "Резистор 2К ОМ" (at 219.075 144.78 0)
       (effects (font (size 1.27 1.27)) hide)
     )
@@
       (effects (font (size 1.27 1.27)) hide)
     )
-    (property "Человекопонятное название" "Резистор 360 Ом" (at 219.075 153.035 0)
+    (property "Человекопонятное название" "Резистор 2К ОМ" (at 219.075 153.035 0)
       (effects (font (size 1.27 1.27)) hide)
     )
@@
       (effects (font (size 1.27 1.27)) hide)
     )
-    (property "Человекопонятное название" "Резистор 220 Ом" (at 208.915 144.78 0)
+    (property "Человекопонятное название" "Резистор 1К ОМ" (at 208.915 144.78 0)
       (effects (font (size 1.27 1.27)) hide)
     )
@@
       (effects (font (size 1.27 1.27)) hide)
     )
-    (property "Человекопонятное название" "Резистор 220 Ом" (at 208.915 153.035 0)
-      (effects (font (size 1.27 1.27)) hide)
-    )
+    (property "Человекопонятное название" "Резистор 1К ОМ" (at 208.915 153.035 0)
+      (effects (font (size 1.27 1.27)) hide)
+    )
