File: Hardware/ciam/impeller/impeller/connectors.kicad_sch (KiCad schematic)
At the start: 35 parts, among them J12 Micro-Fit_2x2P, J14 PLS-5, J16 Conn_02x05_SWD, J3 USB_B_Micro, J4 Micro_SD_Card_Con, Q1 BSS138, Q2 BSS138, U4 B0505MT-1WR4, U4 USBLC6-2SC6, U46 HCPL-0630, U47 LDL1117S33R

Commit message: added rpi shield project
Parts:
- C23: Ссылка (none) -> https://www.chipdip.ru/product/grm188r71h104k
Changed lines of the file:
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@@
+      (effects (font (size 1.27 1.27)) hide)
+    )
+    (property "Ссылка" "https://www.chipdip.ru/product/grm188r71h104k" (at 220.98 67.31 0)
       (effects (font (size 1.27 1.27)) hide)
     )

Commit message: fixed uart
Parts:
- removed C59: 100n, Capacitor_SMD:C_0805_2012Metric, symbol Device:C_Small
- removed C62: 100n, Capacitor_SMD:C_0805_2012Metric, symbol Device:C
- removed C63: 4u7, Capacitor_SMD:C_0805_2012Metric, symbol Device:C
- removed Q1, Q2: BSS138, Package_TO_SOT_SMD:SOT-23, symbol Transistor_FET:BSS138
- removed R100, R101, R102, R99: 10k, Resistor_SMD:R_0805_2012Metric, symbol Device:R_Small
- removed R51 (x2): 220, Resistor_SMD:R_0603_1608Metric, symbol Device:R_Small
- removed U46: HCPL-0630, Package_SO:SOIC-8_3.9x4.9mm_P1.27mm, symbol Isolator:HCPL-0630
- removed U47: LDL1117S33R, Package_TO_SOT_SMD:SOT-223-3_TabPin2, symbol Regulator_Linear:LD1117S33TR_SOT223
- added C9 (x2): 100n, Capacitor_SMD:C_0805_2012Metric, symbol Device:C_Small
- added Q5: BSS138, Package_TO_SOT_SMD:SOT-23, symbol Transistor_FET:BSS138
- added R37: 360, Resistor_SMD:R_0603_1608Metric, symbol Device:R_Small
- added R51: 220, Resistor_SMD:R_0603_1608Metric, symbol Device:R_Small
- added R77, R87: 10k, Resistor_SMD:R_0805_2012Metric, symbol Device:R_Small
- added U46 (x2): HCPL-0600, Package_SO:SO-8_3.9x4.9mm_P1.27mm, symbol Isolator:HCPL-0630
Connections:
- net GND: now also C9.2, U46.5 (GND)
- net USART3_RX: now also Q5.2 (S), R87.2
- net USART3_TX: now also U46.3 (Cathode)
- net VDD_3V3: now also Q5.1 (G), R51.1, R87.1
- net VDD_5V0: now also C9.1, R77.1, U46.7 (VE), U46.8 (VCC)
- net at J12.3 (Pin_3): now also J12.1 (Pin_1), U46.3 (Cathode), U46.6 (VOut)
- net GND_ISO_UART3 renamed GND_UART_ISO
- net GND_UART_ISO: now also C9.2, U46.5 (GND)
- net VDD_5V0_ISO_UART3 renamed 5V0_UART_ISO
- net 5V0_UART_ISO: now also C9.1, R37.2, U46.7 (VE), U46.8 (VCC)
- new net: R37.1, U46.2 (Anode)
- new net: Q5.3 (D), R77.2, U46.6 (VOut)
- new net: R51.2, U46.2 (Anode)
Other:
- note added: "0"
- moved on the sheet: C14, C16, J12, R51, R52, U4

Commit message: Updated CIAM project
Connections:
- net GND_UART_ISO: now also J12.1 (Pin_2); no longer J12.2 (Pin_2)
- net at J12.3 (Pin_3), U46.3 (Cathode): no longer J12.1 (Pin_1), U46.6 (VOut)
- new net: J12.2 (Pin_1), U46.6 (VOut)
Other:
- note removed: "0"
Changed lines of the file:
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@@
   (junction (at 81.915 170.815) (diameter 0) (color 0 0 0 0)
   )
-  (junction (at 123.19 125.73) (diameter 0) (color 0 0 0 0)
-  )
   (junction (at 107.315 170.815) (diameter 0) (color 0 0 0 0)
   )
@@
   )
   (junction (at 85.725 132.08) (diameter 0) (color 0 0 0 0)
-  )
-  (junction (at 123.19 123.19) (diameter 0) (color 0 0 0 0)
   )
   (junction (at 182.245 32.385) (diameter 0) (color 0 0 0 0)
@@
     (stroke (width 0) (type default))
   )
-  (wire (pts (xy 102.87 123.19) (xy 123.19 123.19))
-    (stroke (width 0) (type default))
-  )
   (wire (pts (xy 170.18 43.18) (xy 205.105 43.18))
     (stroke (width 0) (type default))
@@
     (stroke (width 0) (type default))
   )
-  (wire (pts (xy 123.19 123.19) (xy 125.73 123.19))
+  (wire (pts (xy 102.87 123.19) (xy 125.73 123.19))
     (stroke (width 0) (type default))
   )
@@
   )
   (polyline (pts (xy 172.085 83.82) (xy 172.085 189.23))
-    (stroke (width 0) (type default))
-  )
-  (wire (pts (xy 123.19 123.19) (xy 123.19 125.73))
     (stroke (width 0) (type default))
   )
@@
   (text "SWD" (at 259.715 129.54 0)
     (effects (font (size 1.27 1.27)) (justify left bottom))
-  )
-  (text "0" (at 36.195 120.65 0)
-    (effects (font (size 2.54 2.54) (thickness 0.508) bold) (justify left bottom))
   )
   (text "Serial wire debug (SWD)" (at 192.405 128.905 0)
@@
     )
   )
-  (symbol (lib_id "Connector_Generic:Conn_02x02_Odd_Even") (at 130.81 123.19 0) (unit 1)
+  (symbol (lib_name "Conn_02x02_Odd_Even_1") (lib_id "Connector_Generic:Conn_02x02_Odd_Even") (at 130.81 123.19 0) (unit 1)
     (in_bom yes) (on_board yes) (dnp no)
     (property "Reference" "J12" (at 132.08 117.475 0)
@@
     )
     (pin "1")
+    (pin "3")
     (pin "2")
-    (pin "3")
     (pin "4")
     (instances
