File: Hardware/ciam/impeller/impeller/impeller.kicad_sch (KiCad schematic)
At the start: 30 parts, among them J1 PLS-3, SW1 KLS7-TS6601-11-180, U1 STM32F405VGT6, Y1 KSE-7K32768KDY2400A3, Y1 KSE-7U08000MAB143ZA3

Commit message: Updated CIAM project
Connections:
- net CAN1_A0: now also U1.63 (PC6)
- net CAN1_A1: now also U1.64 (PC7)
- net CAN1_A2: now also U1.67 (PA8)
- net CAN1_A3: now also U1.68 (PA9)
- net CAN1_A4: now also U1.69 (PA10)
- net CAN1_A5: now also U1.77 (PA15)
- net CAN2_A0: now also U1.85 (PD4)
- net CAN2_A1: now also U1.86 (PD5)
- net CAN2_A2: now also U1.87 (PD6)
- net CAN2_A3: now also U1.88 (PD7)
- net CAN2_A4: now also U1.90 (PB4)
- net CAN2_A5: now also U1.93 (PB7)
- net ThrustLever1: now reaches U1.35 (PB0)
- net ThrustLever2: now reaches U1.36 (PB1)
Changed lines of the file:
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@@
     )
   )
-  (global_label "CAN1_A1" (shape input) (at 116.84 168.275 180) (fields_autoplaced)
-    (effects (font (size 1.27 1.27)) (justify right))
-    (property "Intersheetrefs" "${INTERSHEET_REFS}" (at 105.7699 168.275 0)
-      (effects (font (size 1.27 1.27)) (justify right) hide)
-    )
-  )
-  (global_label "CAN2_A5" (shape input) (at 116.84 163.195 180) (fields_autoplaced)
-    (effects (font (size 1.27 1.27)) (justify right))
-    (property "Intersheetrefs" "${INTERSHEET_REFS}" (at 105.7699 163.195 0)
-      (effects (font (size 1.27 1.27)) (justify right) hide)
+  (global_label "CAN1_A1" (shape input) (at 81.915 151.13 0) (fields_autoplaced)
+    (effects (font (size 1.27 1.27)) (justify left))
+    (property "Intersheetrefs" "${INTERSHEET_REFS}" (at 93.0645 151.13 0)
+      (effects (font (size 1.27 1.27)) (justify left) hide)
+    )
+  )
+  (global_label "CAN2_A5" (shape input) (at 81.915 107.95 0) (fields_autoplaced)
+    (effects (font (size 1.27 1.27)) (justify left))
+    (property "Intersheetrefs" "${INTERSHEET_REFS}" (at 93.0645 107.95 0)
+      (effects (font (size 1.27 1.27)) (justify left) hide)
     )
   )
@@
     )
   )
-  (global_label "CAN1_A0" (shape input) (at 116.84 165.735 180) (fields_autoplaced)
-    (effects (font (size 1.27 1.27)) (justify right))
-    (property "Intersheetrefs" "${INTERSHEET_REFS}" (at 105.7699 165.735 0)
-      (effects (font (size 1.27 1.27)) (justify right) hide)
+  (global_label "CAN1_A0" (shape input) (at 81.915 148.59 0) (fields_autoplaced)
+    (effects (font (size 1.27 1.27)) (justify left))
+    (property "Intersheetrefs" "${INTERSHEET_REFS}" (at 93.0645 148.59 0)
+      (effects (font (size 1.27 1.27)) (justify left) hide)
     )
   )
@@
     )
   )
-  (global_label "CAN2_A3" (shape input) (at 116.84 158.115 180) (fields_autoplaced)
-    (effects (font (size 1.27 1.27)) (justify right))
-    (property "Intersheetrefs" "${INTERSHEET_REFS}" (at 105.7699 158.115 0)
+  (global_label "CAN2_A3" (shape input) (at 36.195 130.81 180) (fields_autoplaced)
+    (effects (font (size 1.27 1.27)) (justify right))
+    (property "Intersheetrefs" "${INTERSHEET_REFS}" (at 25.1249 130.81 0)
       (effects (font (size 1.27 1.27)) (justify right) hide)
     )
@@
     )
   )
-  (global_label "CAN2_A1" (shape input) (at 116.84 153.035 180) (fields_autoplaced)
-    (effects (font (size 1.27 1.27)) (justify right))
-    (property "Intersheetrefs" "${INTERSHEET_REFS}" (at 105.7699 153.035 0)
+  (global_label "CAN2_A1" (shape input) (at 36.195 125.73 180) (fields_autoplaced)
+    (effects (font (size 1.27 1.27)) (justify right))
+    (property "Intersheetrefs" "${INTERSHEET_REFS}" (at 25.1249 125.73 0)
       (effects (font (size 1.27 1.27)) (justify right) hide)
     )
@@
     )
   )
-  (global_label "CAN2_A0" (shape input) (at 116.84 150.495 180) (fields_autoplaced)
-    (effects (font (size 1.27 1.27)) (justify right))
-    (property "Intersheetrefs" "${INTERSHEET_REFS}" (at 105.7699 150.495 0)
-      (effects (font (size 1.27 1.27)) (justify right) hide)
-    )
-  )
-  (global_label "CAN1_A5" (shape input) (at 116.84 178.435 180) (fields_autoplaced)
-    (effects (font (size 1.27 1.27)) (justify right))
-    (property "Intersheetrefs" "${INTERSHEET_REFS}" (at 105.7699 178.435 0)
-      (effects (font (size 1.27 1.27)) (justify right) hide)
+  (global_label "CAN2_A0" (shape input) (at 36.195 123.19 180) (fields_autoplaced)
+    (effects (font (size 1.27 1.27)) (justify right))
+    (property "Intersheetrefs" "${INTERSHEET_REFS}" (at 25.1249 123.19 0)
+      (effects (font (size 1.27 1.27)) (justify right) hide)
+    )
+  )
+  (global_label "CAN1_A5" (shape input) (at 81.915 85.09 0) (fields_autoplaced)
+    (effects (font (size 1.27 1.27)) (justify left))
+    (property "Intersheetrefs" "${INTERSHEET_REFS}" (at 93.0645 85.09 0)
+      (effects (font (size 1.27 1.27)) (justify left) hide)
     )
   )
@@
     )
   )
-  (global_label "CAN2_A2" (shape input) (at 116.84 155.575 180) (fields_autoplaced)
-    (effects (font (size 1.27 1.27)) (justify right))
-    (property "Intersheetrefs" "${INTERSHEET_REFS}" (at 105.7699 155.575 0)
+  (global_label "CAN2_A2" (shape input) (at 36.195 128.27 180) (fields_autoplaced)
+    (effects (font (size 1.27 1.27)) (justify right))
+    (property "Intersheetrefs" "${INTERSHEET_REFS}" (at 25.1249 128.27 0)
       (effects (font (size 1.27 1.27)) (justify right) hide)
     )
@@
     )
   )
-  (global_label "CAN2_A4" (shape input) (at 116.84 160.655 180) (fields_autoplaced)
-    (effects (font (size 1.27 1.27)) (justify right))
-    (property "Intersheetrefs" "${INTERSHEET_REFS}" (at 105.7699 160.655 0)
-      (effects (font (size 1.27 1.27)) (justify right) hide)
+  (global_label "CAN2_A4" (shape input) (at 81.915 100.33 0) (fields_autoplaced)
+    (effects (font (size 1.27 1.27)) (justify left))
+    (property "Intersheetrefs" "${INTERSHEET_REFS}" (at 93.0645 100.33 0)
+      (effects (font (size 1.27 1.27)) (justify left) hide)
     )
   )
@@
     )
   )
+  (global_label "ThrustLever2" (shape input) (at 81.915 92.71 0) (fields_autoplaced)
+    (effects (font (size 1.27 1.27)) (justify left))
+    (property "Intersheetrefs" "${INTERSHEET_REFS}" (at 96.795 92.71 0)
+      (effects (font (size 1.27 1.27)) (justify left) hide)
+    )
+  )
   (global_label "IND7_3V3" (shape input) (at 119.38 158.115 0) (fields_autoplaced)
     (effects (font (size 1.27 1.27)) (justify left))
@@
     )
   )
-  (global_label "CAN1_A3" (shape input) (at 116.84 173.355 180) (fields_autoplaced)
-    (effects (font (size 1.27 1.27)) (justify right))
-    (property "Intersheetrefs" "${INTERSHEET_REFS}" (at 105.7699 173.355 0)
-      (effects (font (size 1.27 1.27)) (justify right) hide)
+  (global_label "CAN1_A3" (shape input) (at 81.915 69.85 0) (fields_autoplaced)
+    (effects (font (size 1.27 1.27)) (justify left))
+    (property "Intersheetrefs" "${INTERSHEET_REFS}" (at 93.0645 69.85 0)
+      (effects (font (size 1.27 1.27)) (justify left) hide)
     )
   )
@@
     )
   )
-  (global_label "CAN1_A4" (shape input) (at 116.84 175.895 180) (fields_autoplaced)
-    (effects (font (size 1.27 1.27)) (justify right))
-    (property "Intersheetrefs" "${INTERSHEET_REFS}" (at 105.7699 175.895 0)
-      (effects (font (size 1.27 1.27)) (justify right) hide)
+  (global_label "ThrustLever1" (shape input) (at 81.915 90.17 0) (fields_autoplaced)
+    (effects (font (size 1.27 1.27)) (justify left))
+    (property "Intersheetrefs" "${INTERSHEET_REFS}" (at 96.795 90.17 0)
+      (effects (font (size 1.27 1.27)) (justify left) hide)
+    )
+  )
+  (global_label "CAN1_A4" (shape input) (at 81.915 72.39 0) (fields_autoplaced)
+    (effects (font (size 1.27 1.27)) (justify left))
+    (property "Intersheetrefs" "${INTERSHEET_REFS}" (at 93.0645 72.39 0)
+      (effects (font (size 1.27 1.27)) (justify left) hide)
     )
   )
@@
     )
   )
-  (global_label "CAN1_A2" (shape input) (at 116.84 170.815 180) (fields_autoplaced)
-    (effects (font (size 1.27 1.27)) (justify right))
-    (property "Intersheetrefs" "${INTERSHEET_REFS}" (at 105.7699 170.815 0)
-      (effects (font (size 1.27 1.27)) (justify right) hide)
-    )
-  )
+  (global_label "CAN1_A2" (shape input) (at 81.915 67.31 0) (fields_autoplaced)
+    (effects (font (size 1.27 1.27)) (justify left))
+    (property "Intersheetrefs" "${INTERSHEET_REFS}" (at 93.0645 67.31 0)
+      (effects (font (size 1.27 1.27)) (justify left) hide)
+    )
+  )

Commit message: Updated CIAM project
Parts:
- added H1 (x2): MH_M3_Corner, user_lib:MountingHole_3.2mm_M3_Pad_Via_5mm, symbol Mechanical:MountingHole
- renumbered C16 to C10, C14 to C16, C1 to C3, C13 to C9
Connections:
- net Encoder1_A: now also U1.45 (PE14)
- net Encoder1_B: now also U1.44 (PE13)
- net Encoder2_A: now also U1.42 (PE11)
- net Encoder2_B: now also U1.41 (PE10)
- net Encoder3_A: now also U1.39 (PE8)
- net Encoder3_B: now also U1.40 (PE9)
- net Encoder4_A: now also U1.48 (PB11)
- net Encoder4_B: now also U1.51 (PB12)
- net Encoder5_A: now also U1.47 (PB10)
- net Encoder5_B: now also U1.46 (PE15)
- net IND10_3V3: now also U1.53 (PB14)
- net IND1_3V3: now also U1.54 (PB15)
- net IND2_3V3: now also U1.58 (PD11)
- net IND3_3V3: now also U1.59 (PD12)
- net IND4_3V3: now also U1.57 (PD10)
- net IND5_3V3: now also U1.62 (PD15)
- net IND6_3V3: now also U1.23 (PA0)
- net IND7_3V3: now also U1.61 (PD14)
- net IND8_3V3: now also U1.60 (PD13)
- net IND9_3V3: now also U1.52 (PB13)
- net PushSwitch_Stop_board: now also U1.25 (PA2)
- net PushSwitch_Stop_cocpit: now also U1.24 (PA1)
- net PushSwitch_Sync: now also U1.29 (PA4)
- net ToggleSwitch_AircraftPWR: now also U1.26 (PA3)
- net ToggleSwitch_AirfieldPWR: now also U1.34 (PC5)
- net ToggleSwitch_Bat1: now also U1.96 (PB9)
- net ToggleSwitch_Bat2: now also U1.98 (PE1)
- net ToggleSwitch_Bat3: now also U1.2 (PE3)
- net ToggleSwitch_Bat4: now also U1.95 (PB8)
- net ToggleSwitch_Bat_GND: now also U1.97 (PE0)
- net ToggleSwitch_Imp1: now also U1.7 (PC13)
- net ToggleSwitch_Imp2: now also U1.1 (PE2)
- net ToggleSwitch_Imp3: now also U1.5 (PE6)
- net ToggleSwitch_Imp4: now also U1.4 (PE5)
- net ToggleSwitch_Imp5: now also U1.3 (PE4)
