File: Hardware/ciam/impeller/impeller/impeller.kicad_sch (KiCad schematic)
At the start: 32 parts, among them J1 PLS-3, SW1 KLS7-TS6601-11-180, U1 STM32F405VGT6, Y1 KSE-7K32768KDY2400A3, Y1 KSE-7U08000MAB143ZA3

Commit message: updated piezo module
Parts:
- renumbered C10 to C11, C11 to C12, C12 to C13, C13 to C14, C14 to C15, C15 to C18, C16 to C19, C3 to C4, C6 to C5, C7 to C6, C8 to C7, C9 to C8, Y1 to Y2
