File: Hardware/ciam/impeller/impeller/power.kicad_sch (KiCad schematic)
At the start: 10 parts, among them J2 Picoblade_1x2, U1 LDL1117S33, U2 TMR-1211

Commit message: updated ciam project
Parts:
- removed J2: Picoblade_1x2, symbol Connector_Generic:Conn_01x02
- added J12: Micro-Fit_2x2P, symbol Connector_Generic:Conn_02x02_Odd_Even
- U2: value TMR-1211 -> TEL 3-2411; footprint Converter_DCDC:Converter_DCDC_TRACO_TMR-xxxx_THT -> (none)
Connections:
- net GND: now also U2.10 (-VOUT), U2.15 (-VOUT); no longer U2.7 (-VOUT)
- net VDD_5V0: now also U2.11 (+VOUT), U2.14 (+VOUT); no longer U2.6 (+VOUT)
- net at C1.2: now also U2.12 (-VIN), U2.13 (-VIN), J12.1 (Pin_1), J12.3 (Pin_3); no longer U2.1 (-VIN)
- net at C1.1: now also U2.1 (+VIN), U2.24 (+VIN), J12.2 (Pin_2), J12.4 (Pin_4); no longer U2.2 (+VIN)
- no-connect marks 1 -> 0
Other:
- moved on the sheet: C1, C2, C3, C4, C5, C6, C7, U1

Commit message: updated impeller project
Parts:
- removed C3: 1u, symbol Device:C
- removed C4, C5: 100n, symbol Device:C
- removed C6: 4u7, symbol Device:C
- removed C7: 47u, symbol Device:C_Polarized
- removed J12: Micro-Fit_2x2P, symbol Connector_Generic:Conn_02x02_Odd_Even
- removed U1: LDL1117S33, Package_TO_SOT_SMD:SOT-223-3_TabPin2, symbol Regulator_Linear:LD1117S33TR_SOT223
- removed U2: TEL 3-2411, symbol Converter_DCDC:TMR-1211
- added C2: 47u, symbol Device:C_Polarized
- added C20, C23: 4u7, symbol Device:C
- added C21, C24: 100n, symbol Device:C
- added J2: PicoBlade_1x2P, symbol Connector_Generic:Conn_01x02
- added U3: LDL1117S33R, Package_TO_SOT_SMD:SOT-223-3_TabPin2, symbol Regulator_Linear:LD1117S33TR_SOT223
- added U4: TMR-1211, Converter_DCDC:Converter_DCDC_TRACO_TMR-xxxx_THT, symbol Converter_DCDC:TMR-1211
Connections:
- net GND: now also C2.2, C20.2, C21.2, C23.2, C24.2, U3.1 (GND), U4.7 (-VOUT)
- net VDD_3V3: now also C2.1, C23.1, C24.1, U3.2 (VO)
- net VDD_5V0: now also C20.1, C21.1, U3.3 (VI), U4.6 (+VOUT)
- net at C1.2: now also J2.1 (Pin_1), U4.1 (-VIN)
- net at C1.1: now also J2.2 (Pin_2), U4.2 (+VIN)
- no-connect marks 0 -> 1
Other:
- moved on the sheet: C1, C2

Commit message: multiple fixes
Parts:
- added D4, D5: FYLS-1206SRC, symbol Device:LED
- added R97: 150, Resistor_SMD:R_0603_1608Metric, symbol Device:R
- added R98: 65, Resistor_SMD:R_0603_1608Metric, symbol Device:R
- C1: footprint (none) -> Capacitor_SMD:C_0805_2012Metric; Ссылка (none) -> https://www.chipdip.ru/product/grm21br61e475ka12l; Цена (none) -> 13
- C2: footprint (none) -> Capacitor_SMD:CP_Elec_6.3x5.4; Ссылка (none) -> https://www.chipdip.ru/product0/9000565730; Цена (none) -> 16
- C22: renamed from C20; footprint (none) -> Capacitor_SMD:C_0805_2012Metric; Ссылка (none) -> https://www.chipdip.ru/product/grm21br61e475ka12l; Цена (none) -> 13
- C23: renamed from C21; footprint (none) -> Capacitor_SMD:C_0805_2012Metric; Ссылка (none) -> https://www.chipdip.ru/product/grm21br71h104k; Цена (none) -> 13
- C25: renamed from C23; footprint (none) -> Capacitor_SMD:C_0805_2012Metric; Ссылка (none) -> https://www.chipdip.ru/product/grm21br61e475ka12l; Цена (none) -> 13
- C26: renamed from C24; footprint (none) -> Capacitor_SMD:C_0805_2012Metric; Ссылка (none) -> https://www.chipdip.ru/product/grm21br71h104k; Цена (none) -> 13
- J5: renamed from J2; Ссылка (none) -> https://www.chipdip.ru/product/sct1251wv-2p; Цена (none) -> 8
- U2: renamed from U3; Ссылка (none) -> https://www.chipdip.ru/product/ldl1117s33r-stm; Цена (none) -> 33
- U3: renamed from U4; Ссылка (none) -> https://www.chipdip.ru/product0/8002030343; Цена (none) -> 5230
Connections:
- net GND: now also R97.2, R98.2
- net VDD_3V3: now also D5.2 (A)
- net VDD_5V0: now also D4.2 (A)
- new net: D5.1 (K), R98.1
- new net: D4.1 (K), R97.1

Commit message: updated bom
Parts:
- C1, C22, C25: Человекопонятное название (none) -> Конденсатор 4.7мкФ
- C2: Человекопонятное название (none) -> Конденсатор 47мкФ
- C23, C26: Человекопонятное название (none) -> Конденсатор 100нФ
- D4, D5: Человекопонятное название (none) -> Светодиод красный
- J5: Человекопонятное название (none) -> Разъем Picoblade 1x2
- R97: Человекопонятное название (none) -> Резистор 150 Ом
- R98: Человекопонятное название (none) -> Резистор 65 Ом
- U2: Человекопонятное название (none) -> LDO-стабилизатор напряжения
- U3: Человекопонятное название (none) -> DC-DC преобразователь
Changed lines of the file:
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@@
+      (effects (font (size 1.27 1.27)) hide)
+    )
+    (property "Человекопонятное название" "Резистор 65 Ом" (at 100.965 115.57 0)
       (effects (font (size 1.27 1.27)) hide)
     )
@@
     )
     (property "Цена" "13" (at 126.365 66.675 0)
+      (effects (font (size 1.27 1.27)) hide)
+    )
+    (property "Человекопонятное название" "Конденсатор 100нФ" (at 126.365 66.675 0)
       (effects (font (size 1.27 1.27)) hide)
     )
@@
     )
     (property "Цена" "5230" (at 80.01 66.675 0)
+      (effects (font (size 1.27 1.27)) hide)
+    )
+    (property "Человекопонятное название" "DC-DC преобразователь" (at 80.01 66.675 0)
       (effects (font (size 1.27 1.27)) hide)
     )
@@
       (effects (font (size 1.27 1.27)) hide)
     )
+    (property "Человекопонятное название" "Светодиод красный" (at 100.965 105.41 0)
+      (effects (font (size 1.27 1.27)) hide)
+    )
     (pin "1")
     (pin "2")
@@
       (effects (font (size 1.27 1.27)) hide)
     )
+    (property "Человекопонятное название" "LDO-стабилизатор напряжения" (at 142.24 61.595 0)
+      (effects (font (size 1.27 1.27)) hide)
+    )
     (pin "1")
     (pin "2")
@@
     )
     (property "Цена" "16" (at 104.14 66.675 0)
+      (effects (font (size 1.27 1.27)) hide)
+    )
+    (property "Человекопонятное название" "Конденсатор 47мкФ" (at 104.14 66.675 0)
       (effects (font (size 1.27 1.27)) hide)
     )
@@
       (effects (font (size 1.27 1.27)) hide)
     )
+    (property "Человекопонятное название" "Конденсатор 4.7мкФ" (at 165.1 66.675 0)
+      (effects (font (size 1.27 1.27)) hide)
+    )
     (pin "1")
     (pin "2")
@@
     )
     (property "Цена" "13" (at 176.53 66.675 0)
+      (effects (font (size 1.27 1.27)) hide)
+    )
+    (property "Человекопонятное название" "Конденсатор 100нФ" (at 176.53 66.675 0)
       (effects (font (size 1.27 1.27)) hide)
     )
@@
       (effects (font (size 1.27 1.27)) hide)
     )
+    (property "Человекопонятное название" "Светодиод красный" (at 78.74 105.41 0)
+      (effects (font (size 1.27 1.27)) hide)
+    )
     (pin "1")
     (pin "2")
@@
       (effects (font (size 1.27 1.27)) hide)
     )
+    (property "Человекопонятное название" "Разъем Picoblade 1x2" (at 34.29 64.135 0)
+      (effects (font (size 1.27 1.27)) hide)
+    )
     (pin "1")
     (pin "2")
@@
     )
     (property "Цена" "16" (at 154.305 66.675 0)
+      (effects (font (size 1.27 1.27)) hide)
+    )
+    (property "Человекопонятное название" "Конденсатор 47мкФ" (at 154.305 66.675 0)
       (effects (font (size 1.27 1.27)) hide)
     )
@@
       (effects (font (size 1.27 1.27)) hide)
     )
+    (property "Человекопонятное название" "Резистор 150 Ом" (at 78.74 115.57 0)
+      (effects (font (size 1.27 1.27)) hide)
+    )
     (pin "1")
     (pin "2")
@@
       (effects (font (size 1.27 1.27)) hide)
     )
+    (property "Человекопонятное название" "Конденсатор 4.7мкФ" (at 114.935 66.675 0)
+      (effects (font (size 1.27 1.27)) hide)
+    )
     (pin "1")
     (pin "2")
@@
       (effects (font (size 1.27 1.27)) hide)
     )
+    (property "Человекопонятное название" "Конденсатор 4.7мкФ" (at 52.705 66.675 0)
+      (effects (font (size 1.27 1.27)) hide)
+    )

Commit message: updated bom
Parts:
- U3: value TMR-1211 -> TMR 3-1211; Ссылка https://www.chipdip.ru/product0/8002030343 -> https://www.chipdip.ru/product/tmr-3-1211; Цена 5230 -> 2130
Changed lines of the file:
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@@
       (effects (font (size 1.27 1.27)))
     )
-    (property "Value" "TMR-1211" (at 80.01 57.785 0)
+    (property "Value" "TMR 3-1211" (at 80.01 57.785 0)
       (effects (font (size 1.27 1.27)))
     )
@@
       (effects (font (size 1.27 1.27)) hide)
     )
-    (property "Ссылка" "https://www.chipdip.ru/product0/8002030343" (at 80.01 66.675 0)
+    (property "Ссылка" "https://www.chipdip.ru/product/tmr-3-1211" (at 80.01 66.675 0)
       (effects (font (size 1.27 1.27)) hide)
     )
-    (property "Цена" "5230" (at 80.01 66.675 0)
+    (property "Цена" "2130" (at 80.01 66.675 0)
       (effects (font (size 1.27 1.27)) hide)
     )

Commit message: changed 12-5V dc-dc converter
Parts:
- U3: value TMR 3-1211 -> TEL 5-1211; Ссылка https://www.chipdip.ru/product/tmr-3-1211 -> https://www.chipdip.ru/product/tel-5-1211; Цена 2130 -> 2 500
Connections:
- net GND: now also U3.16 (-VOUT); no longer U3.7 (-VOUT)
- net VDD_5V0: now also U3.14 (+VOUT); no longer U3.6 (+VOUT)
- net at C1.2, J5.1 (Pin_1): now also U3.2 (-VIN), U3.3 (-VIN); no longer U3.1 (-VIN)
- net at C1.1, J5.2 (Pin_2): now also U3.22 (+VIN), U3.23 (+VIN); no longer U3.2 (+VIN)
- no-connect marks 1 -> 0
Changed lines of the file:
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@@
   (junction (at 104.14 61.595) (diameter 0) (color 0 0 0 0)
   )
+  (junction (at 64.77 61.595) (diameter 0) (color 0 0 0 0)
+  )
   (junction (at 100.965 122.555) (diameter 0) (color 0 0 0 0)
   )
@@
   (junction (at 114.935 61.595) (diameter 0) (color 0 0 0 0)
   )
-  (no_connect (at 67.31 66.675))
+  (junction (at 64.77 71.755) (diameter 0) (color 0 0 0 0)
+  )
   (wire (pts (xy 126.365 61.595) (xy 126.365 62.865))
     (stroke (width 0) (type default))
   )
+  (wire (pts (xy 67.31 64.135) (xy 64.77 64.135))
+    (stroke (width 0) (type default))
+  )
   (wire (pts (xy 39.37 61.595) (xy 52.705 61.595))
     (stroke (width 0) (type default))
@@
     (stroke (width 0) (type default))
   )
+  (wire (pts (xy 64.77 71.755) (xy 67.31 71.755))
+    (stroke (width 0) (type default))
+  )
   (wire (pts (xy 104.14 61.595) (xy 114.935 61.595))
     (stroke (width 0) (type default))
@@
     (stroke (width 0) (type default))
   )
+  (wire (pts (xy 64.77 69.215) (xy 64.77 71.755))
+    (stroke (width 0) (type default))
+  )
+  (wire (pts (xy 64.77 64.135) (xy 64.77 61.595))
+    (stroke (width 0) (type default))
+  )
   (wire (pts (xy 149.86 61.595) (xy 154.305 61.595))
     (stroke (width 0) (type default))
@@
     (stroke (width 0) (type default))
   )
-  (wire (pts (xy 52.705 61.595) (xy 67.31 61.595))
+  (wire (pts (xy 52.705 61.595) (xy 64.77 61.595))
     (stroke (width 0) (type default))
   )
@@
     (stroke (width 0) (type default))
   )
-  (wire (pts (xy 52.705 71.755) (xy 67.31 71.755))
+  (wire (pts (xy 52.705 71.755) (xy 64.77 71.755))
     (stroke (width 0) (type default))
   )
@@
     (stroke (width 0) (type default))
   )
+  (wire (pts (xy 67.31 69.215) (xy 64.77 69.215))
+    (stroke (width 0) (type default))
+  )
   (wire (pts (xy 78.74 122.555) (xy 100.965 122.555))
     (stroke (width 0) (type default))
@@
   )
   (wire (pts (xy 98.425 61.595) (xy 104.14 61.595))
+    (stroke (width 0) (type default))
+  )
+  (wire (pts (xy 64.77 61.595) (xy 67.31 61.595))
     (stroke (width 0) (type default))
   )
@@
   (symbol (lib_name "TMR-1211_1") (lib_id "Converter_DCDC:TMR-1211") (at 80.01 66.675 0) (unit 1)
     (in_bom yes) (on_board yes) (dnp no) (fields_autoplaced)
-    (property "Reference" "U3" (at 80.01 55.245 0)
+    (property "Reference" "U3" (at 80.01 54.61 0)
       (effects (font (size 1.27 1.27)))
     )
-    (property "Value" "TMR 3-1211" (at 80.01 57.785 0)
+    (property "Value" "TEL 5-1211" (at 80.01 57.15 0)
       (effects (font (size 1.27 1.27)))
     )
-    (property "Footprint" "Converter_DCDC:Converter_DCDC_TRACO_TMR-xxxx_THT" (at 80.01 75.565 0)
-      (effects (font (size 1.27 1.27)) hide)
-    )
-    (property "Datasheet" "https://www.tracopower.com/products/tmr2.pdf" (at 80.01 79.375 0)
-      (effects (font (size 1.27 1.27)) hide)
-    )
-    (property "Ссылка" "https://www.chipdip.ru/product/tmr-3-1211" (at 80.01 66.675 0)
-      (effects (font (size 1.27 1.27)) hide)
-    )
-    (property "Цена" "2130" (at 80.01 66.675 0)
-      (effects (font (size 1.27 1.27)) hide)
-    )
-    (property "Человекопонятное название" "DC-DC преобразователь" (at 80.01 66.675 0)
-      (effects (font (size 1.27 1.27)) hide)
-    )
-    (pin "1")
+    (property "Footprint" "Converter_DCDC:Converter_DCDC_TRACO_TMR-xxxx_THT" (at 80.645 86.36 0)
+      (effects (font (size 1.27 1.27)) hide)
+    )
+    (property "Datasheet" "" (at 80.645 90.17 0)
+      (effects (font (size 1.27 1.27)) hide)
+    )
+    (property "Ссылка" "https://www.chipdip.ru/product/tel-5-1211" (at 78.74 83.185 0)
+      (effects (font (size 1.27 1.27)) hide)
+    )
+    (property "Цена" "2 500" (at 80.01 78.74 0)
+      (effects (font (size 1.27 1.27)) hide)
+    )
+    (property "Человекопонятное название" "DC-DC преобразователь" (at 78.74 80.645 0)
+      (effects (font (size 1.27 1.27)) hide)
+    )
+    (pin "14")
+    (pin "16")
     (pin "2")
+    (pin "22")
+    (pin "23")
     (pin "3")
-    (pin "5")
-    (pin "6")
-    (pin "7")
-    (pin "8")
     (instances
       (project "impeller"

Commit message: Updated CIAM project
Parts:
- added C62: 100n, Capacitor_SMD:C_0805_2012Metric, symbol Device:C
- added D3: ss24, user_lib:SS24, symbol Device:D_Schottky
- D4, D5: footprint (none) -> Resistor_SMD:R_1206_3216Metric_Pad1.30x1.75mm_HandSolder
- J5: footprint (none) -> Connector_Molex:Molex_PicoBlade_53047-0210_1x02_P1.25mm_Vertical
- U3: footprint Converter_DCDC:Converter_DCDC_TRACO_TMR-xxxx_THT -> user_lib:TEL 5-1211
Connections:
- net VDD_5V0: now also D3.1 (K)
- net at C1.2, J5.1 (Pin_1), U3.2 (-VIN)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: now also C62.2
- net at C1.1, J5.2 (Pin_2), U3.22 (+VIN)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: now also C62.1
- new net VDD_5V_VBUS: D3.2 (A)
Other:
- moved on the sheet: C1

Commit message: Updated CIAM project
Parts:
- renumbered C62 to C21, C22 to C23, C23 to C24, C25 to C26, C26 to C27, D4 to D1, D5 to D3, J5 to J2, R97 to R3, R98 to R4, U2 to U3
