File: Hardware/ciam/impeller/impeller/power.kicad_sch (KiCad schematic)
At the start: 16 parts, among them J2 PicoBlade_1x2P, U3 LDL1117S33R, U3 TEL 5-1211

Commit message: updated piezo module
Parts:
- renumbered C1 to C20, C2 to C22, C2 to C25, D3 to D2
