File: Hardware/ciam/impeller/impeller/encoders.kicad_sch (KiCad schematic)
At the start: 33 parts, among them J11 Micro-Fit_2x2P, J12 Micro-Fit_2x2P, J13 Micro-Fit_2x2P, J14 Micro-Fit_2x2P, J9 Micro-Fit_2x2P, U19 TLP521-2, U4 B0505MT-1WR4

Commit message: updated impeller project
Parts:
- removed R54 (x10): 470, symbol Device:R_Small
- removed R56 (x10): 10k, symbol Device:R_Small
- removed U19 (x5): TLP521-2, symbol Isolator:TLP291
- added C49, C50, C51, C52, C53: 100n, symbol Device:C_Small
- added Q11, Q12, Q13, Q14, Q15, Q16, Q17, Q18, Q19, Q20: BSS138, Package_TO_SOT_SMD:SOT-23, symbol Transistor_FET:BSS138
- added R51 (x10): 330, symbol Device:R_Small
- added R63, R64, R66, R67, R69, R70, R72, R73, R75, R76, R78, R79, R81, R82, R84, R85, R87, R88, R90, R91: 10k, symbol Device:R_Small
- added U28, U29, U30, U31, U32: HCPL-0630, Package_SO:SOIC-8_3.9x4.9mm_P1.27mm, symbol Isolator:HCPL-0630
- renumbered J9 to J15
Connections:
- net Encoder1_A: now also Q11.2 (S), R64.2
- net Encoder1_B: now also Q12.2 (S), R67.2
- net Encoder2_A: now also Q13.2 (S), R70.2
- net Encoder2_B: now also Q14.2 (S), R73.2
- net Encoder3_A: now also Q15.2 (S), R76.2
- net Encoder3_B: now also Q16.2 (S), R79.2
- net Encoder4_A: now also Q17.2 (S), R82.2
- net Encoder4_B: now also Q18.2 (S), R85.2
- net Encoder5_A: now also Q19.2 (S), R88.2
- net Encoder5_B: now also Q20.2 (S), R91.2
- net GND: now also C49.1, C50.1, C51.1, C52.1, C53.1, U28.5 (GND), U29.5 (GND), U30.5 (GND), U31.5 (GND), U32.5 (GND)
- net VDD_3V3: now also Q11.1 (G), Q12.1 (G), Q13.1 (G), Q14.1 (G), Q15.1 (G), Q16.1 (G), Q17.1 (G), Q18.1 (G), Q19.1 (G), Q20.1 (G), R64.1, R67.1, R70.1, R73.1, R76.1, R79.1, R82.1, R85.1, R88.1, R91.1
- net VDD_5V0: now also C49.2, C50.2, C51.2, C52.2, C53.2, R63.1, R66.1, R69.1, R72.1, R75.1, R78.1, R81.1, R84.1, R87.1, R90.1, U28.8 (VCC), U29.8 (VCC), U30.8 (VCC), U31.8 (VCC), U32.8 (VCC)
- net at C16.1, U4.8 (+Vo): now also R51.1, R51.1, R51.1, R51.1, R51.1, R51.1, R51.1, R51.1, R51.1, R51.1
- net at J11.2 (Pin_2): now also U28.2 (C1)
- net at J11.4 (Pin_4): now also U28.3 (C2)
- net at J15.2 (Pin_2): now also U32.2 (C1)
- net at J15.4 (Pin_4): now also U32.3 (C2)
- net at J12.2 (Pin_2): now also U29.2 (C1)
- net at J12.4 (Pin_4): now also U29.3 (C2)
- net at J13.2 (Pin_2): now also U30.2 (C1)
- net at J13.4 (Pin_4): now also U30.3 (C2)
- net at J14.2 (Pin_2): now also U31.2 (C1)
- net at J14.4 (Pin_4): now also U31.3 (C2)
- new net: R51.2, U32.1 (A1)
- new net: R51.2, U28.1 (A1)
- new net: Q11.3 (D), R63.2, U28.7 (VO1)
- new net: R51.2, U28.4 (A2)
- new net: Q12.3 (D), R66.2, U28.6 (VO2)
- new net: Q20.3 (D), R90.2, U32.6 (VO2)
- new net: R51.2, U30.1 (A1)
- new net: Q19.3 (D), R87.2, U32.7 (VO1)
- new net: Q15.3 (D), R75.2, U30.7 (VO1)
- new net: Q14.3 (D), R72.2, U29.6 (VO2)
- new net: R51.2, U31.1 (A1)
- new net: R51.2, U32.4 (A2)
- new net: Q16.3 (D), R78.2, U30.6 (VO2)
- new net: Q18.3 (D), R84.2, U31.6 (VO2)
- new net: R51.2, U31.4 (A2)
- new net: Q17.3 (D), R81.2, U31.7 (VO1)
- new net: R51.2, U29.1 (A1)
- new net: R51.2, U29.4 (A2)
- new net: Q13.3 (D), R69.2, U29.7 (VO1)
- new net: R51.2, U30.4 (A2)
Other:
- moved on the sheet: C14, C16, J15, U4

Commit message: multiple fixes
Parts:
- removed J11, J12, J13, J14, J15: Micro-Fit_2x2P, symbol Connector_Generic:Conn_02x02_Odd_Even
- added J13: Micro-Fit_2x12P, symbol Connector_Generic:Conn_02x12_Odd_Even
- C14: footprint (none) -> Capacitor_SMD:C_0805_2012Metric; Ссылка (none) -> https://www.chipdip.ru/product/grm21br61e475ka12l; Цена (none) -> 13
- C16: footprint (none) -> Capacitor_SMD:C_0805_2012Metric; Ссылка (none) -> https://www.chipdip.ru/product/grm21br61e106ka73l; Цена (none) -> 13
- C49, C50, C51, C52, C53: footprint (none) -> Capacitor_SMD:C_0805_2012Metric; Ссылка (none) -> https://www.chipdip.ru/product/grm21br71h104k; Цена (none) -> 13
- Q1: renamed from Q11; Ссылка (none) -> https://www.chipdip.ru/product/bss138-umw; Цена (none) -> 3
- Q10: renamed from Q20; Ссылка (none) -> https://www.chipdip.ru/product/bss138-umw; Цена (none) -> 3
- Q2: renamed from Q12; Ссылка (none) -> https://www.chipdip.ru/product/bss138-umw; Цена (none) -> 3
- Q3: renamed from Q13; Ссылка (none) -> https://www.chipdip.ru/product/bss138-umw; Цена (none) -> 3
- Q4: renamed from Q14; Ссылка (none) -> https://www.chipdip.ru/product/bss138-umw; Цена (none) -> 3
- Q5: renamed from Q15; Ссылка (none) -> https://www.chipdip.ru/product/bss138-umw; Цена (none) -> 3
- Q6: renamed from Q16; Ссылка (none) -> https://www.chipdip.ru/product/bss138-umw; Цена (none) -> 3
- Q7: renamed from Q17; Ссылка (none) -> https://www.chipdip.ru/product/bss138-umw; Цена (none) -> 3
- Q8: renamed from Q18; Ссылка (none) -> https://www.chipdip.ru/product/bss138-umw; Цена (none) -> 3
- Q9: renamed from Q19; Ссылка (none) -> https://www.chipdip.ru/product/bss138-umw; Цена (none) -> 3
- R51: footprint (none) -> Resistor_SMD:R_0603_1608Metric; Ссылка (none) -> https://www.chipdip.ru/product/0.1w-0603-330-om-1; Цена (none) -> 5
- R61: renamed from R63; footprint (none) -> Resistor_SMD:R_0805_2012Metric; Ссылка (none) -> https://www.chipdip.ru/product/0.125w-0805-10-kom-5; Цена (none) -> 5
- R62: renamed from R64; footprint (none) -> Resistor_SMD:R_0805_2012Metric; Ссылка (none) -> https://www.chipdip.ru/product/0.125w-0805-10-kom-5; Цена (none) -> 5
- R64: renamed from R66; footprint (none) -> Resistor_SMD:R_0805_2012Metric; Ссылка (none) -> https://www.chipdip.ru/product/0.125w-0805-10-kom-5; Цена (none) -> 5
- R65: renamed from R67; footprint (none) -> Resistor_SMD:R_0805_2012Metric; Ссылка (none) -> https://www.chipdip.ru/product/0.125w-0805-10-kom-5; Цена (none) -> 5
- R67: renamed from R69; footprint (none) -> Resistor_SMD:R_0805_2012Metric; Ссылка (none) -> https://www.chipdip.ru/product/0.125w-0805-10-kom-5; Цена (none) -> 5
- R68: renamed from R70; footprint (none) -> Resistor_SMD:R_0805_2012Metric; Ссылка (none) -> https://www.chipdip.ru/product/0.125w-0805-10-kom-5; Цена (none) -> 5
- R70: renamed from R72; footprint (none) -> Resistor_SMD:R_0805_2012Metric; Ссылка (none) -> https://www.chipdip.ru/product/0.125w-0805-10-kom-5; Цена (none) -> 5
- R71: renamed from R73; footprint (none) -> Resistor_SMD:R_0805_2012Metric; Ссылка (none) -> https://www.chipdip.ru/product/0.125w-0805-10-kom-5; Цена (none) -> 5
- R73: renamed from R75; footprint (none) -> Resistor_SMD:R_0805_2012Metric; Ссылка (none) -> https://www.chipdip.ru/product/0.125w-0805-10-kom-5; Цена (none) -> 5
- R74: renamed from R76; footprint (none) -> Resistor_SMD:R_0805_2012Metric; Ссылка (none) -> https://www.chipdip.ru/product/0.125w-0805-10-kom-5; Цена (none) -> 5
- R76: renamed from R78; footprint (none) -> Resistor_SMD:R_0805_2012Metric; Ссылка (none) -> https://www.chipdip.ru/product/0.125w-0805-10-kom-5; Цена (none) -> 5
- R77: renamed from R79; footprint (none) -> Resistor_SMD:R_0805_2012Metric; Ссылка (none) -> https://www.chipdip.ru/product/0.125w-0805-10-kom-5; Цена (none) -> 5
- R79: renamed from R81; footprint (none) -> Resistor_SMD:R_0805_2012Metric; Ссылка (none) -> https://www.chipdip.ru/product/0.125w-0805-10-kom-5; Цена (none) -> 5
- R80: renamed from R82; footprint (none) -> Resistor_SMD:R_0805_2012Metric; Ссылка (none) -> https://www.chipdip.ru/product/0.125w-0805-10-kom-5; Цена (none) -> 5
- R82: renamed from R84; footprint (none) -> Resistor_SMD:R_0805_2012Metric; Ссылка (none) -> https://www.chipdip.ru/product/0.125w-0805-10-kom-5; Цена (none) -> 5
- R83: renamed from R85; footprint (none) -> Resistor_SMD:R_0805_2012Metric; Ссылка (none) -> https://www.chipdip.ru/product/0.125w-0805-10-kom-5; Цена (none) -> 5
- R85: renamed from R87; footprint (none) -> Resistor_SMD:R_0805_2012Metric; Ссылка (none) -> https://www.chipdip.ru/product/0.125w-0805-10-kom-5; Цена (none) -> 5
- R86: renamed from R88; footprint (none) -> Resistor_SMD:R_0805_2012Metric; Ссылка (none) -> https://www.chipdip.ru/product/0.125w-0805-10-kom-5; Цена (none) -> 5
- R88: renamed from R90; footprint (none) -> Resistor_SMD:R_0805_2012Metric; Ссылка (none) -> https://www.chipdip.ru/product/0.125w-0805-10-kom-5; Цена (none) -> 5
- R89: renamed from R91; footprint (none) -> Resistor_SMD:R_0805_2012Metric; Ссылка (none) -> https://www.chipdip.ru/product/0.125w-0805-10-kom-5; Цена (none) -> 5
- U4: Ссылка (none) -> https://www.chipdip.ru/product0/8003333290; Цена (none) -> 120
- renumbered U28 to U36, U29 to U37, U30 to U38, U31 to U39, U32 to U40
Connections:
- net GND: now also J13.1 (Pin_1), J13.11 (Pin_11), J13.13 (Pin_13), J13.15 (Pin_15), J13.17 (Pin_17), J13.19 (Pin_19), J13.21 (Pin_21), J13.22 (Pin_22), J13.23 (Pin_23), J13.24 (Pin_24), J13.3 (Pin_3), J13.5 (Pin_5), J13.7 (Pin_7), J13.9 (Pin_9)
- net at U36.2 (C1): now also J13.2 (Pin_2)
- net at U36.3 (C2): now also J13.4 (Pin_4)
- net at U40.2 (C1): now also J13.18 (Pin_18)
- net at U40.3 (C2): now also J13.20 (Pin_20)
- net at U37.2 (C1): now also J13.6 (Pin_6)
- net at U37.3 (C2): now also J13.8 (Pin_8)
- net at U39.2 (C1): now also J13.14 (Pin_14)
- net at U39.3 (C2): now also J13.16 (Pin_16)
- net at U38.2 (C1): now also J13.10 (Pin_10)
- net at U38.3 (C2): now also J13.12 (Pin_12)
Other:
- moved on the sheet: C14, C16, C49, C50, C51, C52, C53, Q1, Q10, Q2, Q3, Q4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

Commit message: fixed bug in encoders sheet
Connections:
- net GND: no longer J13.1 (Pin_1), J13.11 (Pin_11), J13.13 (Pin_13), J13.15 (Pin_15), J13.17 (Pin_17), J13.19 (Pin_19), J13.21 (Pin_21), J13.22 (Pin_22), J13.23 (Pin_23), J13.24 (Pin_24), J13.3 (Pin_3), J13.5 (Pin_5), J13.7 (Pin_7), J13.9 (Pin_9)
- net at C16.2, U4.6 (0V), U4.7 (0V): now also J13.1 (Pin_1), J13.11 (Pin_11), J13.13 (Pin_13), J13.15 (Pin_15), J13.17 (Pin_17), J13.19 (Pin_19), J13.21 (Pin_21), J13.22 (Pin_22), J13.23 (Pin_23), J13.24 (Pin_24), J13.3 (Pin_3), J13.5 (Pin_5), J13.7 (Pin_7), J13.9 (Pin_9)
Changed lines of the file:
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@@
-    (stroke (width 0) (type default))
-  )
-  (wire (pts (xy 50.8 190.5) (xy 118.745 190.5))
     (stroke (width 0) (type default))
   )
@@
     (stroke (width 0) (type default))
   )
+  (wire (pts (xy 31.115 190.5) (xy 118.745 190.5))
+    (stroke (width 0) (type default))
+  )
   (wire (pts (xy 104.775 111.76) (xy 114.935 111.76))
     (stroke (width 0) (type default))
@@
     (stroke (width 0) (type default))
   )
-  (wire (pts (xy 31.115 115.57) (xy 31.115 119.38))
+  (wire (pts (xy 31.115 115.57) (xy 31.115 190.5))
     (stroke (width 0) (type default))
   )
@@
         )
       )
-    )
-  )
-  (symbol (lib_id "power:GND") (at 31.115 119.38 0) (unit 1)
-    (in_bom yes) (on_board yes) (dnp no) (fields_autoplaced)
-    (property "Reference" "#PWR032" (at 31.115 125.73 0)
-      (effects (font (size 1.27 1.27)) hide)
-    )
-    (property "Value" "GND" (at 31.115 123.825 0)
-      (effects (font (size 1.27 1.27)))
-    )
-    (property "Footprint" "" (at 31.115 119.38 0)
-      (effects (font (size 1.27 1.27)) hide)
-    )
-    (property "Datasheet" "" (at 31.115 119.38 0)
-      (effects (font (size 1.27 1.27)) hide)
-    )
-    (pin "1")
-    (instances
-      (project "impeller"
-        (path "/dc9d3fdd-86e3-4a65-b009-b0cbd29a6eee/0a393be1-a79e-48b5-bd67-1675300f121e"
-          (reference "#PWR032") (unit 1)
-        )
-      )

Commit message: updated bom
Parts:
- C14: Человекопонятное название (none) -> Конденсатор 4.7мкФ
- C16: Человекопонятное название (none) -> Конденсатор 10мкФ
- C49, C50, C51, C52, C53: Человекопонятное название (none) -> Конденсатор 100нФ
- J13: Человекопонятное название (none) -> Разъем Micro-Fit 2x12 М
- Q1, Q10, Q2, Q3, Q4, Q5, Q6, Q7, Q8, Q9: Человекопонятное название (none) -> Транзистор полевой n типа
- R51: Человекопонятное название (none) -> Резистор 330 Ом
- R61, R62, R64, R65, R67, R68, R70, R71, R73, R74, R76, R77, R79, R80, R82, R83, R85, R86, R88, R89: Человекопонятное название (none) -> Резистор 10k Ом
- U36, U37, U38, U39, U40: Человекопонятное название (none) -> Оптопара двухканальная с логическими уровнями на выходе
- U4: Человекопонятное название (none) -> DC/DC преобразователь

Commit message: Updated CIAM project
Parts:
- J13: footprint (none) -> Connector_Molex:Molex_Micro-Fit_3.0_43045-2400_2x12_P3.00mm_Horizontal; Ссылка https://www.chipdip.ru/product/sct3001wv-2x12p -> https://www.chipdip.ru/product/sct3001wr-2x12p
- U4: footprint (none) -> user_lib:B0505MT-1WR4
Changed lines of the file:
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@@
       (effects (font (size 1.27 1.27)))
     )
-    (property "Footprint" "" (at 139.7 194.31 0)
+    (property "Footprint" "user_lib:B0505MT-1WR4" (at 139.7 194.31 0)
       (effects (font (size 1.27 1.27) italic) hide)
     )
@@
       (effects (font (size 1.27 1.27)))
     )
-    (property "Footprint" "" (at 38.735 96.52 0)
-      (effects (font (size 1.27 1.27)) hide)
-    )
-    (property "Datasheet" "~" (at 38.735 96.52 0)
-      (effects (font (size 1.27 1.27)) hide)
-    )
-    (property "Ссылка" "https://www.chipdip.ru/product/sct3001wv-2x12p" (at 38.735 96.52 0)
-      (effects (font (size 1.27 1.27)) hide)
-    )
+    (property "Footprint" "Connector_Molex:Molex_Micro-Fit_3.0_43045-2400_2x12_P3.00mm_Horizontal" (at 38.735 96.52 0)
+      (effects (font (size 1.27 1.27)) hide)
+    )
+    (property "Datasheet" "" (at 38.735 96.52 0)
+      (effects (font (size 1.27 1.27)) hide)
+    )
+    (property "Ссылка" "https://www.chipdip.ru/product/sct3001wr-2x12p" (at 38.735 96.52 0)
+      (effects (font (size 1.27 1.27)) hide)
+    )

Commit message: Updated CIAM project
Parts:
- renumbered C49 to C50, C50 to C51, C51 to C52, C52 to C53, C53 to C54, J13 to J10, R61 to R73, R64 to R74, R67 to R75, R70 to R76, R73 to R77, R76 to R78, R82 to R80, R85 to R81, R88 to R82, R62 to R83, R65 to R84, R68 to R85, R71 to R86, R74 to R87, R77 to R88, R80 to R89, R83 to R90, R86 to R91, R89 to R92
Connections:
- net at C16.2, J10.1 (Pin_1), J10.11 (Pin_21)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: now also J10.10 (Pin_19), J10.12 (Pin_23), J10.14 (Pin_4), J10.2 (Pin_3), J10.4 (Pin_7), J10.6 (Pin_11), J10.8 (Pin_15); no longer J10.15 (Pin_15), J10.17 (Pin_17), J10.19 (Pin_19), J10.21 (Pin_21), J10.22 (Pin_22), J10.23 (Pin_23), J10.24 (Pin_24)
- net at U36.2 (C1): now also J10.24 (Pin_24); no longer J10.2 (Pin_2)
- net at U36.3 (C2): now also J10.23 (Pin_22); no longer J10.4 (Pin_4)
- net at U39.2 (C1): now also J10.18 (Pin_12); no longer J10.14 (Pin_14)
- net at U39.3 (C2): now also J10.17 (Pin_10); no longer J10.16 (Pin_16)
- net at U37.2 (C1): now also J10.22 (Pin_20); no longer J10.6 (Pin_6)
- net at U37.3 (C2): now also J10.21 (Pin_18); no longer J10.8 (Pin_8)
- net at U38.2 (C1): now also J10.20 (Pin_16); no longer J10.10 (Pin_10)
- net at U38.3 (C2): now also J10.19 (Pin_14); no longer J10.12 (Pin_12)
- net at U40.2 (C1): now also J10.16 (Pin_8); no longer J10.18 (Pin_18)
- net at U40.3 (C2): now also J10.15 (Pin_6); no longer J10.20 (Pin_20)

Commit message: updated piezo module
Parts:
- renumbered C16 to C55, C14 to C56, R51 to R63, R51 to R64, R51 to R65, R51 to R66, R51 to R67, R51 to R68, R51 to R69, R51 to R70, R51 to R71, R51 to R72, U4 to U41
