File: Hardware/ciam/impeller/impeller/indicators.kicad_sch (KiCad schematic)
At the start: 42 parts, among them J4 Micro-Fit_2x5P, J7 Micro-Fit_2x5P, K1 SRD-05VDC-SL-C, Q5 BSS138

Commit message: updated impeller project
Parts:
- removed D1 (x10): 1N4148W, Diode_SMD:D_SOD-123, symbol Diode:1N4148W
- removed J4, J7: Micro-Fit_2x5P, symbol Connector_Generic:Conn_02x05_Odd_Even
- removed K1 (x10): SRD-05VDC-SL-C, Relay_THT:Relay_SPDT_SANYOU_SRD_Series_Form_C, symbol Relay:SANYOU_SRD_Form_C
- removed Q5 (x10): BSS138, Package_TO_SOT_SMD:SOT-23, symbol Transistor_FET:BSS138
- removed R6 (x10): 100k, Resistor_SMD:R_0603_1608Metric, symbol Device:R_Small
- added J5, J6: Micro-Fit_2x5P, symbol Connector_Generic:Conn_02x05_Odd_Even
- added R23, R24, R25, R26, R27, R28, R29, R30, R31, R32: 220, symbol Device:R_Small
- added U2 (x10): G3VM61D1, symbol Relay_SolidState:S216S01
Connections:
- net GNDPWR: now also J5.10 (Pin_10), J5.2 (Pin_2), J5.4 (Pin_4), J5.6 (Pin_6), J5.8 (Pin_8), J6.10 (Pin_10), J6.2 (Pin_2), J6.4 (Pin_4), J6.6 (Pin_6), J6.8 (Pin_8), U2.3, U2.3, U2.3, U2.3, U2.3, U2.3, U2.3, U2.3, U2.3, U2.3
- net IND10_3V3: now also R32.2
- net IND10_V24: now also J6.9 (Pin_9), U2.4
- net IND1_3V3: now also R23.2
- net IND1_V24: now also J5.1 (Pin_1), U2.4
- net IND2_3V3: now also R24.2
- net IND2_V24: now also J5.3 (Pin_3), U2.4
- net IND3_3V3: now also R25.2
- net IND3_V24: now also J5.5 (Pin_5), U2.4
- net IND4_3V3: now also R26.2
- net IND4_V24: now also J5.7 (Pin_7), U2.4
- net IND5_3V3: now also R27.2
- net IND5_V24: now also J5.9 (Pin_9), U2.4
- net IND6_3V3: now also R28.2
- net IND6_V24: now also J6.1 (Pin_1), U2.4
- net IND7_3V3: now also R29.2
- net IND7_V24: now also J6.3 (Pin_3), U2.4
- net IND8_3V3: now also R30.2
- net IND8_V24: now also J6.5 (Pin_5), U2.4
- net IND9_3V3: now also R31.2
- net IND9_V24: now also J6.7 (Pin_7), U2.4
- new net: R28.1, U2.2
- new net: R24.1, U2.2
- new net: R25.1, U2.2
- new net: R31.1, U2.2
- new net: R32.1, U2.2
- new net: R29.1, U2.2
- new net: R30.1, U2.2
- new net: R27.1, U2.2
- new net: R26.1, U2.2
- new net: R23.1, U2.2
- new net VDD_3V3: U2.1, U2.1, U2.1, U2.1, U2.1, U2.1, U2.1, U2.1, U2.1, U2.1
- no-connect marks 10 -> 0
Other:
- note added: "GNDPWR от бортового питания 24В"

Commit message: multiple fixes
Parts:
- J8: renamed from J5; Ссылка (none) -> https://www.chipdip.ru/product/sct3001fh-2x5p; Цена (none) -> 34
- J9: renamed from J6; Ссылка (none) -> https://www.chipdip.ru/product/sct3001fh-2x5p; Цена (none) -> 34
- R21: renamed from R23; footprint (none) -> Resistor_SMD:R_0603_1608Metric; Ссылка (none) -> https://www.chipdip.ru/product/0.1w-0603-220-om-1; Цена (none) -> 5
- R22: renamed from R24; footprint (none) -> Resistor_SMD:R_0603_1608Metric; Ссылка (none) -> https://www.chipdip.ru/product/0.1w-0603-220-om-1; Цена (none) -> 5
- R23: renamed from R25; footprint (none) -> Resistor_SMD:R_0603_1608Metric; Ссылка (none) -> https://www.chipdip.ru/product/0.1w-0603-220-om-1; Цена (none) -> 5
- R24: renamed from R26; footprint (none) -> Resistor_SMD:R_0603_1608Metric; Ссылка (none) -> https://www.chipdip.ru/product/0.1w-0603-220-om-1; Цена (none) -> 5
- R25: renamed from R27; footprint (none) -> Resistor_SMD:R_0603_1608Metric; Ссылка (none) -> https://www.chipdip.ru/product/0.1w-0603-220-om-1; Цена (none) -> 5
- R26: renamed from R28; footprint (none) -> Resistor_SMD:R_0603_1608Metric; Ссылка (none) -> https://www.chipdip.ru/product/0.1w-0603-220-om-1; Цена (none) -> 5
- R27: renamed from R29; footprint (none) -> Resistor_SMD:R_0603_1608Metric; Ссылка (none) -> https://www.chipdip.ru/product/0.1w-0603-220-om-1; Цена (none) -> 5
- R28: renamed from R30; footprint (none) -> Resistor_SMD:R_0603_1608Metric; Ссылка (none) -> https://www.chipdip.ru/product/0.1w-0603-220-om-1; Цена (none) -> 5
- R29: renamed from R31; footprint (none) -> Resistor_SMD:R_0603_1608Metric; Ссылка (none) -> https://www.chipdip.ru/product/0.1w-0603-220-om-1; Цена (none) -> 5
- R30: renamed from R32; footprint (none) -> Resistor_SMD:R_0603_1608Metric; Ссылка (none) -> https://www.chipdip.ru/product/0.1w-0603-220-om-1; Цена (none) -> 5
- U2: Ссылка (none) -> https://www.chipdip.ru/product0/8006782491; Цена (none) -> 710

Commit message: updated bom
Parts:
- J8, J9: Человекопонятное название (none) -> Разъем Micro-Fit 2x5 М
- R21, R22, R23, R24, R25, R26, R27, R28, R29, R30: Человекопонятное название (none) -> Резистор 220 Ом
- U2: Человекопонятное название (none) -> Оптореле
Changed lines of the file:
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@@
+      (effects (font (size 1.27 1.27)) hide)
+    )
+    (property "Человекопонятное название" "Разъем Micro-Fit 2x5 М" (at 212.725 107.315 0)
       (effects (font (size 1.27 1.27)) hide)
     )
@@
       (effects (font (size 1.27 1.27)) hide)
     )
+    (property "Человекопонятное название" "Оптореле" (at 102.235 110.49 0)
+      (effects (font (size 1.27 1.27)) hide)
+    )
     (pin "1")
     (pin "2")
@@
       (effects (font (size 1.27 1.27)) hide)
     )
+    (property "Человекопонятное название" "Оптореле" (at 102.235 59.69 0)
+      (effects (font (size 1.27 1.27)) hide)
+    )
     (pin "1")
     (pin "2")
@@
       (effects (font (size 1.27 1.27)) hide)
     )
+    (property "Человекопонятное название" "Резистор 220 Ом" (at 90.17 74.93 0)
+      (effects (font (size 1.27 1.27)) hide)
+    )
     (pin "1")
     (pin "2")
@@
       (effects (font (size 1.27 1.27)) hide)
     )
+    (property "Человекопонятное название" "Оптореле" (at 102.235 148.59 0)
+      (effects (font (size 1.27 1.27)) hide)
+    )
     (pin "1")
     (pin "2")
@@
       (effects (font (size 1.27 1.27)) hide)
     )
+    (property "Человекопонятное название" "Резистор 220 Ом" (at 90.17 163.83 0)
+      (effects (font (size 1.27 1.27)) hide)
+    )
     (pin "1")
     (pin "2")
@@
     )
     (property "Цена" "710" (at 102.235 123.19 0)
+      (effects (font (size 1.27 1.27)) hide)
+    )
+    (property "Человекопонятное название" "Оптореле" (at 102.235 123.19 0)
       (effects (font (size 1.27 1.27)) hide)
     )
@@
     )
     (property "Цена" "34" (at 175.895 107.315 0)
+      (effects (font (size 1.27 1.27)) hide)
+    )
+    (property "Человекопонятное название" "Разъем Micro-Fit 2x5 М" (at 175.895 107.315 0)
       (effects (font (size 1.27 1.27)) hide)
     )
@@
       (effects (font (size 1.27 1.27)) hide)
     )
+    (property "Человекопонятное название" "Резистор 220 Ом" (at 90.17 125.73 0)
+      (effects (font (size 1.27 1.27)) hide)
+    )
     (pin "1")
     (pin "2")
@@
     )
     (property "Цена" "5" (at 90.17 113.03 0)
+      (effects (font (size 1.27 1.27)) hide)
+    )
+    (property "Человекопонятное название" "Резистор 220 Ом" (at 90.17 113.03 0)
       (effects (font (size 1.27 1.27)) hide)
     )
@@
       (effects (font (size 1.27 1.27)) hide)
     )
+    (property "Человекопонятное название" "Резистор 220 Ом" (at 90.17 138.43 0)
+      (effects (font (size 1.27 1.27)) hide)
+    )
     (pin "1")
     (pin "2")
@@
       (effects (font (size 1.27 1.27)) hide)
     )
+    (property "Человекопонятное название" "Оптореле" (at 102.235 97.79 0)
+      (effects (font (size 1.27 1.27)) hide)
+    )
     (pin "1")
     (pin "2")
@@
       (effects (font (size 1.27 1.27)) hide)
     )
+    (property "Человекопонятное название" "Оптореле" (at 102.235 85.09 0)
+      (effects (font (size 1.27 1.27)) hide)
+    )
     (pin "1")
     (pin "2")
@@
     )
     (property "Цена" "710" (at 102.235 46.99 0)
+      (effects (font (size 1.27 1.27)) hide)
+    )
+    (property "Человекопонятное название" "Оптореле" (at 102.235 46.99 0)
       (effects (font (size 1.27 1.27)) hide)
     )
@@
       (effects (font (size 1.27 1.27)) hide)
     )
+    (property "Человекопонятное название" "Резистор 220 Ом" (at 90.17 49.53 0)
+      (effects (font (size 1.27 1.27)) hide)
+    )
     (pin "1")
     (pin "2")
@@
       (effects (font (size 1.27 1.27)) hide)
     )
+    (property "Человекопонятное название" "Оптореле" (at 102.235 72.39 0)
+      (effects (font (size 1.27 1.27)) hide)
+    )
     (pin "1")
     (pin "2")
@@
       (effects (font (size 1.27 1.27)) hide)
     )
+    (property "Человекопонятное название" "Оптореле" (at 102.235 161.29 0)
+      (effects (font (size 1.27 1.27)) hide)
+    )
     (pin "1")
     (pin "2")
@@
       (effects (font (size 1.27 1.27)) hide)
     )
+    (property "Человекопонятное название" "Резистор 220 Ом" (at 90.17 100.33 0)
+      (effects (font (size 1.27 1.27)) hide)
+    )
     (pin "1")
     (pin "2")
@@
       (effects (font (size 1.27 1.27)) hide)
     )
+    (property "Человекопонятное название" "Резистор 220 Ом" (at 90.17 151.13 0)
+      (effects (font (size 1.27 1.27)) hide)
+    )
     (pin "1")
     (pin "2")
@@
       (effects (font (size 1.27 1.27)) hide)
     )
+    (property "Человекопонятное название" "Оптореле" (at 102.235 135.89 0)
+      (effects (font (size 1.27 1.27)) hide)
+    )
     (pin "1")
     (pin "2")
@@
       (effects (font (size 1.27 1.27)) hide)
     )
+    (property "Человекопонятное название" "Резистор 220 Ом" (at 90.17 87.63 0)
+      (effects (font (size 1.27 1.27)) hide)
+    )
     (pin "1")
     (pin "2")
@@
       (effects (font (size 1.27 1.27)) hide)
     )
+    (property "Человекопонятное название" "Резистор 220 Ом" (at 90.17 62.23 0)
+      (effects (font (size 1.27 1.27)) hide)
+    )

Commit message: Updated CIAM project
Parts:
- J8, J9: footprint (none) -> Connector_Molex:Molex_Micro-Fit_3.0_43045-1000_2x05_P3.00mm_Horizontal; Ссылка https://www.chipdip.ru/product/sct3001fh-2x5p -> https://www.chipdip.ru/product/sct3001wr-2x05p
- U2: footprint (none) -> user_lib:G3VM61D1
Changed lines of the file:
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@@
       (effects (font (size 1.27 1.27)))
     )
-    (property "Footprint" "" (at 212.725 107.315 0)
-      (effects (font (size 1.27 1.27)) hide)
-    )
-    (property "Datasheet" "~" (at 212.725 107.315 0)
-      (effects (font (size 1.27 1.27)) hide)
-    )
-    (property "Ссылка" "https://www.chipdip.ru/product/sct3001fh-2x5p" (at 212.725 107.315 0)
+    (property "Footprint" "Connector_Molex:Molex_Micro-Fit_3.0_43045-1000_2x05_P3.00mm_Horizontal" (at 212.725 107.315 0)
+      (effects (font (size 1.27 1.27)) hide)
+    )
+    (property "Datasheet" "" (at 212.725 107.315 0)
+      (effects (font (size 1.27 1.27)) hide)
+    )
+    (property "Ссылка" "https://www.chipdip.ru/product/sct3001wr-2x05p" (at 212.725 107.315 0)
       (effects (font (size 1.27 1.27)) hide)
     )
@@
       (effects (font (size 1.27 1.27)))
     )
-    (property "Footprint" "" (at 97.155 115.57 0)
+    (property "Footprint" "user_lib:G3VM61D1" (at 97.155 115.57 0)
       (effects (font (size 1.27 1.27) italic) (justify left) hide)
     )
@@
       (effects (font (size 1.27 1.27)))
     )
-    (property "Footprint" "" (at 97.155 64.77 0)
+    (property "Footprint" "user_lib:G3VM61D1" (at 97.155 64.77 0)
       (effects (font (size 1.27 1.27) italic) (justify left) hide)
     )
@@
       (effects (font (size 1.27 1.27)))
     )
-    (property "Footprint" "" (at 97.155 153.67 0)
+    (property "Footprint" "user_lib:G3VM61D1" (at 97.155 153.67 0)
       (effects (font (size 1.27 1.27) italic) (justify left) hide)
     )
@@
       (effects (font (size 1.27 1.27)))
     )
-    (property "Footprint" "" (at 97.155 128.27 0)
+    (property "Footprint" "user_lib:G3VM61D1" (at 97.155 128.27 0)
       (effects (font (size 1.27 1.27) italic) (justify left) hide)
     )
@@
       (effects (font (size 1.27 1.27)))
     )
-    (property "Footprint" "" (at 175.895 107.315 0)
-      (effects (font (size 1.27 1.27)) hide)
-    )
-    (property "Datasheet" "~" (at 175.895 107.315 0)
-      (effects (font (size 1.27 1.27)) hide)
-    )
-    (property "Ссылка" "https://www.chipdip.ru/product/sct3001fh-2x5p" (at 175.895 107.315 0)
+    (property "Footprint" "Connector_Molex:Molex_Micro-Fit_3.0_43045-1000_2x05_P3.00mm_Horizontal" (at 175.895 107.315 0)
+      (effects (font (size 1.27 1.27)) hide)
+    )
+    (property "Datasheet" "" (at 175.895 107.315 0)
+      (effects (font (size 1.27 1.27)) hide)
+    )
+    (property "Ссылка" "https://www.chipdip.ru/product/sct3001wr-2x05p" (at 175.895 107.315 0)
       (effects (font (size 1.27 1.27)) hide)
     )
@@
       (effects (font (size 1.27 1.27)))
     )
-    (property "Footprint" "" (at 97.155 102.87 0)
+    (property "Footprint" "user_lib:G3VM61D1" (at 97.155 102.87 0)
       (effects (font (size 1.27 1.27) italic) (justify left) hide)
     )
@@
       (effects (font (size 1.27 1.27)))
     )
-    (property "Footprint" "" (at 97.155 90.17 0)
+    (property "Footprint" "user_lib:G3VM61D1" (at 97.155 90.17 0)
       (effects (font (size 1.27 1.27) italic) (justify left) hide)
     )
@@
       (effects (font (size 1.27 1.27)))
     )
-    (property "Footprint" "" (at 97.155 52.07 0)
+    (property "Footprint" "user_lib:G3VM61D1" (at 97.155 52.07 0)
       (effects (font (size 1.27 1.27) italic) (justify left) hide)
     )
@@
       (effects (font (size 1.27 1.27)))
     )
-    (property "Footprint" "" (at 97.155 77.47 0)
+    (property "Footprint" "user_lib:G3VM61D1" (at 97.155 77.47 0)
       (effects (font (size 1.27 1.27) italic) (justify left) hide)
     )
@@
       (effects (font (size 1.27 1.27)))
     )
-    (property "Footprint" "" (at 97.155 166.37 0)
+    (property "Footprint" "user_lib:G3VM61D1" (at 97.155 166.37 0)
       (effects (font (size 1.27 1.27) italic) (justify left) hide)
     )
@@
       (effects (font (size 1.27 1.27)))
     )
-    (property "Footprint" "" (at 97.155 140.97 0)
-      (effects (font (size 1.27 1.27) italic) (justify left) hide)
-    )
+    (property "Footprint" "user_lib:G3VM61D1" (at 97.155 140.97 0)
+      (effects (font (size 1.27 1.27) italic) (justify left) hide)
+    )

Commit message: Updated CIAM project
Parts:
- renumbered J8 to J5, J9 to J6, R21 to R23, R22 to R24, R23 to R25, R24 to R26, R25 to R27, R26 to R28, R27 to R29, R28 to R30, R29 to R31, R30 to R32
Connections:
- net GNDPWR: now also J5.7 (Pin_4), J5.9 (Pin_8); no longer J5.2 (Pin_2), J5.4 (Pin_4), J6.10 (Pin_10), J6.2 (Pin_2), J6.4 (Pin_4), J6.6 (Pin_6), J6.8 (Pin_8), U2.3, U2.3, U2.3, U2.3, U2.3
- net IND10_V24: now also J6.5 (Pin_9); no longer J6.9 (Pin_9)
- net IND2_V24: now also J5.2 (Pin_3); no longer J5.3 (Pin_3)
- net IND3_V24: now also J5.3 (Pin_5); no longer J5.5 (Pin_5)
- net IND4_V24: now also J5.4 (Pin_7); no longer J5.7 (Pin_7)
- net IND5_V24: now also J5.5 (Pin_9); no longer J5.9 (Pin_9)
- net IND6_V24: now also U2.4; no longer U2.4
- net IND7_V24: now also J6.2 (Pin_3), U2.4; no longer J6.3 (Pin_3), U2.4
- net IND8_V24: now also J6.3 (Pin_5), U2.4; no longer J6.5 (Pin_5), U2.4
- net IND9_V24: now also J6.4 (Pin_7), U2.4; no longer J6.7 (Pin_7), U2.4
- net at U2.2: now also R29.1; no longer R28.1
- net at U2.2: now also R30.1; no longer R31.1
- net at U2.2: now also R31.1; no longer R29.1
- net at U2.2: now also R28.1; no longer R30.1
- new net GND3: J6.10 (Pin_10), J6.6 (Pin_2), J6.7 (Pin_4), J6.8 (Pin_6), J6.9 (Pin_8), U2.3, U2.3, U2.3, U2.3, U2.3
Other:
- moved on the sheet: U2

Commit message: updated piezo module
Parts:
- renumbered U2 to U10, U2 to U11, U2 to U12, U2 to U13, U2 to U14, U2 to U15, U2 to U16, U2 to U17, U2 to U8, U2 to U9
