File: Hardware/ciam/impeller/rpi_power_shield/power_sheld.kicad_pcb (KiCad board)
At the start: 2 copper layers, 5 parts

Commit message: Updated CIAM project
Parts:
- removed REF**: PinHeader_2x20_P2.54mm_Vertical, Connector_PinHeader_2.54mm:PinHeader_2x20_P2.54mm_Vertical
- removed REF** (x4): MountingHole_3.2mm_M3_Pad_Via, MountingHole:MountingHole_3.2mm_M3_Pad_Via
- added C1: 10u, Capacitor_THT:CP_Radial_D10.0mm_P5.00mm, F.Cu at (58.2, 99.3)
- added C10: 100n, Capacitor_SMD:C_1206_3216Metric, F.Cu at (69.3, 126.8)
- added C11: 100n, Capacitor_SMD:C_1206_3216Metric, F.Cu at (69.3, 130.1)
- added C12: 10u, Capacitor_THT:CP_Radial_D10.0mm_P5.00mm, F.Cu at (58.2, 134.0)
- added C13: 1u, Capacitor_SMD:C_1206_3216Metric, F.Cu at (69.3, 133.4)
- added C14: 100n, Capacitor_SMD:C_1206_3216Metric, F.Cu at (69.3, 136.8)
- added C15: 100u, Capacitor_THT:CP_Radial_D6.3mm_P2.50mm, F.Cu at (96.4, 141.4)
- added C16: 100n, Capacitor_SMD:C_0805_2012Metric, F.Cu at (104.4, 124.3)
- added C17: 4u7, Capacitor_SMD:C_0805_2012Metric, F.Cu at (104.4, 127.3)
- added C18: 10u, Capacitor_SMD:C_0805_2012Metric, F.Cu at (104.4, 130.3)
- added C19: 100n, Capacitor_SMD:C_0805_2012Metric, F.Cu at (104.4, 133.3)
- added C2: 10u, Capacitor_THT:CP_Radial_D10.0mm_P5.00mm, F.Cu at (58.2, 110.9)
- added C20: 4u7, Capacitor_SMD:C_0805_2012Metric, F.Cu at (104.4, 136.3)
- added C3: 330p, Capacitor_SMD:C_1206_3216Metric, F.Cu at (69.3, 110.0)
- added C4: 330p, Capacitor_SMD:C_1206_3216Metric, F.Cu at (69.3, 113.3)
- added C5: 220u, Capacitor_THT:CP_Radial_D10.0mm_P5.00mm, F.Cu at (58.2, 122.5)
- added C6: 330p, Capacitor_SMD:C_1206_3216Metric, F.Cu at (69.3, 116.7)
- added C7: 330p, Capacitor_SMD:C_1206_3216Metric, F.Cu at (69.3, 120.0)
- added C8: 100n, Capacitor_SMD:C_1206_3216Metric, F.Cu at (69.3, 123.4)
- added C9: 22u, Capacitor_Tantalum_SMD:CP_EIA-7343-31_Kemet-D, F.Cu at (93.5, 90.5)
- added D1: SS54C, Diode_SMD:D_SMC, F.Cu at (94.0, 76.0)
- added D2: SS54C, Diode_SMD:D_SMC, F.Cu at (94.0, 83.8)
- added D3: FYLS-1206SRC, Resistor_SMD:R_1206_3216Metric_Pad1.30x1.75mm_HandSolder, F.Cu at (57.7, 141.4)
- added D4: FYLS-1206SRC, Resistor_SMD:R_1206_3216Metric_Pad1.30x1.75mm_HandSolder, F.Cu at (57.7, 144.7)
- added H1: MountingHole, MountingHole:MountingHole_2.7mm_M2.5_Pad_Via, F.Cu at (173.6, 121.1)
- added H2: MountingHole, MountingHole:MountingHole_2.7mm_M2.5_Pad_Via, F.Cu at (115.6, 121.1)
- added H3: MountingHole, MountingHole:MountingHole_2.7mm_M2.5_Pad_Via, F.Cu at (173.6, 72.1)
- added H4: MountingHole, MountingHole:MountingHole_2.7mm_M2.5_Pad_Via, F.Cu at (115.6, 72.1)
- added J1: Micro-fit_1x2P, Connector_Molex:Molex_Micro-Fit_3.0_43045-0200_2x01_P3.00mm_Horizontal, F.Cu at (88.3, 132.7)
- added J2: RPi, Connector_PinSocket_2.54mm:PinSocket_2x20_P2.54mm_Vertical, F.Cu at (120.5, 71.4)
- added J3: Micro-fit_1x2P, Connector_Molex:Molex_Micro-Fit_3.0_43045-0200_2x01_P3.00mm_Horizontal, F.Cu at (97.5, 132.7)
- added J4: Micro-Fit_2x2P, Connector_Molex:Molex_Micro-Fit_3.0_43045-0400_2x02_P3.00mm_Horizontal, F.Cu at (102.4, 103.1)
- added K1: NRP-12-C-05D-H, user_lib:NRP-12-C-05D-H, F.Cu at (94.6, 101.2)
- added L1: B82721-K2222-U30, user_lib:B82721-K2222-U30, F.Cu at (81.9, 115.5)
- added Q1: BSS138, Package_TO_SOT_SMD:SOT-23, F.Cu at (104.9, 110.5)
- added Q2: BSS138, Package_TO_SOT_SMD:SOT-23, F.Cu at (104.9, 115.0)
- added Q3: BSS138, Package_TO_SOT_SMD:SOT-23, F.Cu at (104.9, 119.5)
- added R1: R_reg, Resistor_SMD:R_0603_1608Metric, F.Cu at (101.5, 73.4)
- added R10: 10k, Resistor_SMD:R_0805_2012Metric, F.Cu at (105.7, 82.5)
- added R11: 220, Resistor_SMD:R_0603_1608Metric, F.Cu at (101.5, 88.4)
- added R12: 10k, Resistor_SMD:R_0805_2012Metric, F.Cu at (105.7, 85.4)
- added R13: 10k, Resistor_SMD:R_0805_2012Metric, F.Cu at (105.7, 88.3)
- added R14: 220, Resistor_SMD:R_0603_1608Metric, F.Cu at (101.5, 91.0)
- added R2: R_reg, Resistor_SMD:R_0603_1608Metric, F.Cu at (101.5, 75.9)
- added R3: 10k, Resistor_SMD:R_0805_2012Metric, F.Cu at (105.7, 73.6)
- added R4: 10k, Resistor_SMD:R_0805_2012Metric, F.Cu at (105.7, 76.5)
- added R5: 1k5, Resistor_SMD:R_0603_1608Metric, F.Cu at (101.5, 78.4)
- added R6: 2k, Resistor_SMD:R_0603_1608Metric, F.Cu at (101.5, 80.9)
- added R7: 360, Resistor_SMD:R_0603_1608Metric, F.Cu at (101.5, 83.4)
- added R8: 360, Resistor_SMD:R_0603_1608Metric, F.Cu at (101.5, 85.9)
- added R9: 10k, Resistor_SMD:R_0805_2012Metric, F.Cu at (105.7, 79.5)
- added U1: VDV8-1E05, user_lib:VDV8-1E05, F.Cu at (68.0, 82.8)
- added U2: L4940V5, Package_TO_SOT_THT:TO-220-3_Horizontal_TabDown, F.Cu at (75.4, 143.0)
- added U3: HCPL-0630, Package_SO:SOIC-8_3.9x4.9mm_P1.27mm, F.Cu at (106.4, 141.1)
- added U4: LDL1117S33R, Package_TO_SOT_SMD:SOT-223-3_TabPin2, F.Cu at (88.6, 141.6)
- added U5: B0505MT-1WR4, user_lib:B0505MT-1WR4, F.Cu at (97.0, 114.3)
Other:
- board outline added: 65 x 56 mm
- board text removed: "2x18650"
- board text removed: "VDV8"

Commit message: Updated CIAM project
Parts:
- C3, C4, C7, C8, R1, R2: moved to B.Cu
- moved C1 114.8 mm to (171.8, 82.7), turned to 90 degrees
- moved C2 111.1 mm to (169.3, 109.1)
- moved C3 98.4 mm to (163.6, 81.6), turned to 90 degrees
- moved C5 95.1 mm to (153.3, 119.3)
- moved C12 93.0 mm to (135.4, 82.1)
- moved C4 92.0 mm to (155.6, 81.5)
- moved L1 90.9 mm to (170.4, 94.7), turned to 90 degrees
- moved C6 87.6 mm to (156.9, 112.9), turned to 180 degrees
- moved C7 87.4 mm to (156.2, 110.1), turned to 135 degrees
- moved U1 86.3 mm to (153.6, 94.5), turned to 90 degrees
- moved C13 81.5 mm to (131.4, 80.6), turned to 90 degrees
- moved J1 78.8 mm to (165.2, 115.2), turned to 180 degrees
- moved C11 77.6 mm to (129.1, 80.6), turned to 90 degrees
- moved U2 74.8 mm to (139.7, 104.8), turned to 180 degrees
- moved C8 70.9 mm to (138.4, 107.5), turned to 180 degrees
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Connections:
- net Net-(J1-Pin_1) renamed /GND_9-70_IN
- net Net-(J1-Pin_2) renamed /VDD_9-70_IN
- net Net-(J3-Pin_2) renamed /BATT_7.4_IN
- U1 pad 24: (no net) -> Net-(U1-SHIELD)
Routing:
- net Net-(U1-SHIELD): track 0.00 -> 69.3 mm
- net Net-(C1-Pad2): track 0.00 -> 46.8 mm
- net GND: track 0.00 -> 43.6 mm
- net Net-(C1-Pad1): track 0.00 -> 22.7 mm
- net /GND_9-70_IN: track 0.00 -> 22.6 mm
- net 5V0_SENS: track 0.00 -> 19.0 mm
- net /VDD_9-70_IN: track 0.00 -> 15.8 mm
- net /BATT_7.4_IN: track 0.00 -> 14.0 mm
- net Net-(U1-REG): track 0.00 -> 5.42 mm

Commit message: Updated CIAM project
Parts:
- C3: moved to F.Cu
- J2: moved to B.Cu
- moved R11 141.2 mm to (-39.8, 86.9)
- moved R14 141.2 mm to (-39.8, 89.4)
- moved U4 141.2 mm to (-52.6, 140.1)
- moved U5 141.2 mm to (-44.2, 112.8)
- moved C16 141.2 mm to (-36.9, 122.7)
- moved C17 141.2 mm to (-36.9, 125.7)
- moved C18 141.2 mm to (-36.9, 128.7)
- moved C19 141.2 mm to (-36.9, 131.7)
- moved C20 141.2 mm to (-36.9, 134.8)
- moved Q2 141.2 mm to (-36.3, 113.4)
- moved Q3 141.2 mm to (-36.3, 117.9)
- moved R10 141.2 mm to (-35.6, 80.9)
- moved R12 141.2 mm to (-35.6, 83.8)
- moved R13 141.2 mm to (-35.6, 86.8)
- moved R9 141.2 mm to (-35.6, 77.9)
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Routing:
- net VDD_5V0: track 0.00 -> 96.9 mm, vias 0 -> 1
- net 5V0_SENS: track 19.0 -> 82.1 mm
- net GND: track 43.6 -> 88.4 mm, vias 0 -> 3
- net UART_TX: track 0.00 -> 37.3 mm
- net UART_RX: track 0.00 -> 37.3 mm
- net RELAY_SIG: track 0.00 -> 27.3 mm
- net Net-(U2-OUT): track 0.00 -> 24.9 mm
- net Net-(J2-Pin_37): track 0.00 -> 20.5 mm
- net Net-(J2-Pin_33): track 0.00 -> 13.8 mm
- net Net-(D2-A): track 0.00 -> 7.32 mm
- net Net-(D3-K): track 0.00 -> 1.99 mm
- net Net-(D4-K): track 0.00 -> 1.99 mm
- net Net-(C1-Pad2): track 46.8 -> 45.3 mm
- net Net-(U1-SHIELD): track 69.3 -> 70.6 mm

Commit message: Updated CIAM project
Parts:
- removed C20: 4u7, Capacitor_SMD:C_0805_2012Metric
- removed Q3: BSS138, Package_TO_SOT_SMD:SOT-23
- removed R13: 10k, Resistor_SMD:R_0805_2012Metric
- removed R14: 220, Resistor_SMD:R_0603_1608Metric
- added TP1: TestPoint, TestPoint:TestPoint_THTPad_1.5x1.5mm_Drill0.7mm, F.Cu at (130.7, 107.4)
- added TP2: TestPoint, TestPoint:TestPoint_THTPad_1.5x1.5mm_Drill0.7mm, F.Cu at (125.1, 107.4)
- C14, Q2, R10, R5, R6, R9: moved to B.Cu
- C16: value 100n -> 4u7; moved to B.Cu
- C17: value 4u7 -> 100n
- C18: value 10u -> 100n
- C19: value 100n -> 10u; moved to B.Cu
- D3, D4: footprint Resistor_SMD:R_1206_3216Metric_Pad1.30x1.75mm_HandSolder -> Diode_SMD:D_1206_3216Metric
- R12: value 10k -> 360; footprint Resistor_SMD:R_0805_2012Metric -> Resistor_SMD:R_0603_1608Metric
- U3: value HCPL-0630 -> B0505MT-1WR4; footprint Package_SO:SOIC-8_3.9x4.9mm_P1.27mm -> user_lib:B0505MT-1WR4; moved to B.Cu
- U4: value LDL1117S33R -> HCPL-0600; footprint Package_TO_SOT_SMD:SOT-223-3_TabPin2 -> Package_SO:SO-8_3.9x4.9mm_P1.27mm
- U5: value B0505MT-1WR4 -> HCPL-0600; footprint user_lib:B0505MT-1WR4 -> Package_SO:SO-8_3.9x4.9mm_P1.27mm
- moved U4 170.7 mm to (115.5, 110.0), turned to -90 degrees
- moved R10 165.3 mm to (128.4, 102.3), turned to -90 degrees
- moved U5 165.1 mm to (120.9, 110.0), turned to 90 degrees
- moved R9 162.7 mm to (125.7, 99.4)
- moved Q2 162.4 mm to (125.7, 102.3), turned to -90 degrees
- moved C17 159.7 mm to (121.5, 105.3)
- moved C14 159.1 mm to (119.5, 77.5), turned to 135 degrees
- moved R11 157.8 mm to (116.9, 105.5), turned to 180 degrees
- moved R12 157.8 mm to (119.3, 114.4), turned to 180 degrees
- moved C19 155.9 mm to (118.3, 116.3)
- moved C16 155.8 mm to (117.9, 104.5)
- moved U3 155.5 mm to (117.9, 110.4), turned to -90 degrees
- moved C18 152.4 mm to (114.8, 114.7), turned to 180 degrees
- moved R5 71.0 mm to (148.8, 76.7)
- moved R6 68.7 mm to (151.0, 77.5), turned to -90 degrees
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Connections:
- C16 pad 1: /5V_ISO -> VDD_5V0
- C16 pad 2: /GND_UART_ISO -> GND
- J4 pad 1: Net-(J4-Pin_1) -> /GND_UART_ISO
- J4 pad 2: /GND_UART_ISO -> Net-(J4-Pin_1)
- Q2 pad 1: /3V3_ISO -> VDD_3V3
- Q2 pad 2: Net-(J4-Pin_1) -> UART_RX
- R10 pad 1: /3V3_ISO -> VDD_5V0
- R10 pad 2: Net-(J4-Pin_1) -> Net-(Q2-D)
- R11 pad 1: UART_TX -> VDD_3V3
- R11 pad 2: Net-(U3-A1) -> Net-(U4-Anode)
- R12 pad 1: /5V_ISO -> Net-(U5-Anode)
- R12 pad 2: Net-(Q3-D) -> /5V_ISO
- R9 pad 1: /5V_ISO -> VDD_3V3
- R9 pad 2: Net-(Q2-D) -> UART_RX
- U3 pad 1: Net-(U3-A1) -> GND
- U3 pad 2: VDD_3V3 -> GND
- U3 pad 6: Net-(Q3-D) -> /GND_UART_ISO
- U3 pad 7: Net-(Q2-D) -> /GND_UART_ISO
- U4 pad 1: /GND_UART_ISO -> (no net)
- U4 pad 2: /3V3_ISO -> Net-(U4-Anode)
- U4 pad 3: /5V_ISO -> UART_TX
- U5 pad 1: GND -> (no net)
- U5 pad 2: GND -> Net-(U5-Anode)
- U5 pad 6: /GND_UART_ISO -> Net-(Q2-D)
- U5 pad 7: /GND_UART_ISO -> VDD_5V0
- U5 pad 8: /5V_ISO -> VDD_5V0
Routing:
- net VDD_5V0: track 96.9 -> 169.5 mm, vias 1 -> 3
- net /GND_UART_ISO: track 0.00 -> 45.4 mm, vias 0 -> 1
- net VDD_3V3: track 0.00 -> 42.4 mm, vias 0 -> 1
- net GND: track 88.4 -> 123.5 mm, vias 3 -> 12
- net UART_TX: track 37.3 -> 53.9 mm, vias 0 -> 1
- net 5V0_SENS: track 82.1 -> 97.3 mm
- net Net-(J4-Pin_1): track 0.00 -> 14.6 mm
- net /5V_ISO: track 0.00 -> 13.2 mm, vias 0 -> 1
- net /BATT_7.4_IN: track 14.0 -> 25.6 mm
- net Net-(Q2-D): track 0.00 -> 10.5 mm, vias 0 -> 1
- net Net-(J4-Pin_3): track 0.00 -> 8.78 mm
- net Net-(D2-A): track 7.32 -> 12.6 mm
- net UART_RX: track 37.3 -> 42.5 mm
- net Net-(C1-Pad2): track 45.3 -> 47.9 mm
- net Net-(C1-Pad1): track 22.7 -> 25.2 mm
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- added copper zone on B.Cu, net GND
Other:
- board text added: "+"
- board text added: "-"
- board text added: "BATT"
- board text added: "BATT CHECK"
- board text added: "DC 24V"
- board text added: "GND"
- board text added: "PWR"
- board text added: "UART RX"
- board text added: "UART TX"
- board text added: "VDD 7V4"
- board text added: "VDD 9-70"
- board text added: "БАТ"
- board text added: "ПУ"

Commit message: Updated CIAM project
Parts:
- moved R3 15.5 mm to (142.2, 79.2)
Routing:
- net VDD_5V0: track 169.5 -> 180.8 mm
- net RELAY_SIG: track 27.3 -> 31.8 mm
- net Net-(U2-OUT): track 24.9 -> 24.4 mm
Other:
- board text added: "hdmi в ложементе сделать охлаждение для сарая(для стабилизатора напряжения опционально) зарядка для аккумулятора встроенная -> не нужен внешний разъём, проверки напряжения, дополнительное место и тп"
