File: Hardware/Penguin Junior/Connectors.kicad_sch (KiCad schematic)
At the start: 28 parts, among them J1 USB_B_Micro, J10 Conn_01x06_UART, J10 Conn_01x06_servo, J10 Conn_01x06_servo_5V, J10 Conn_01x06_servo_GND, J11 Conn_01x06_UART, J14 Conn_01x04_UART, J16 Conn_02x05_SWD, J2 Conn_01x03_Video, J2 Micro_SD_Card_Det1, J5 Conn_01x03_Video, J9 Conn_01x04_I2C, U2 USBLC6-2SC6

Commit message: Updated project
Parts:
- removed J10: Conn_01x06_servo_GND, Connector_PinHeader_2.54mm:PinHeader_1x06_P2.54mm_Vertical, symbol Connector_Generic:Conn_01x06
- removed J10: Conn_01x06_servo, Connector_PinHeader_2.54mm:PinHeader_1x06_P2.54mm_Vertical, symbol Connector_Generic:Conn_01x06
- removed J10: Conn_01x06_servo_5V, Connector_PinHeader_2.54mm:PinHeader_1x06_P2.54mm_Vertical, symbol Connector_Generic:Conn_01x06
- removed U2: USBLC6-2SC6, Package_TO_SOT_SMD:SOT-23-6, symbol Power_Protection:USBLC6-2SC6
- added J10, J11, J12: Conn_01x10, Connector_PinHeader_2.54mm:PinHeader_1x10_P2.54mm_Vertical, symbol Connector_Generic:Conn_01x10
- added J16: Conn_02x05_SWD, Connector_PinHeader_1.27mm:PinHeader_2x05_P1.27mm_Vertical, symbol Connector_Generic:Conn_02x05_Odd_Even
- added JP1: SolderJumper_2_Open, Jumper:SolderJumper-2_P1.3mm_Open_Pad1.0x1.5mm, symbol Jumper:SolderJumper_2_Open
- added R14 (x4): 22, Resistor_SMD:R_0402_1005Metric, symbol Device:R_Small
- added R2: 10K, Resistor_SMD:R_0402_1005Metric, symbol Device:R
- C15, C16: footprint Capacitor_SMD:C_0603_1608Metric -> Capacitor_SMD:C_0402_1005Metric
- R14, R3, R4, R5, R6, R7, R8: footprint Resistor_SMD:R_0603_1608Metric -> Resistor_SMD:R_0402_1005Metric
Connections:
- net GND: now also J11.1 (Pin_1), J11.10 (Pin_10), J11.2 (Pin_2), J11.3 (Pin_3), J11.4 (Pin_4), J11.5 (Pin_5), J11.6 (Pin_6), J11.7 (Pin_7), J11.8 (Pin_8), J11.9 (Pin_9), J16.1 (Pin_1)
- net TM2_CH1: now also R14.1; no longer R14.1
- net TM3_CH1: now also R14.1; no longer R14.1
- net TM3_CH2: now also R14.1; no longer R14.1
- net TM3_CH3: now also R14.1; no longer R14.1
- net TM4_CH3: now also R14.1; no longer R14.1
- net TM4_CH4: now also R14.1; no longer R14.1
- net USB_OTG_FS_D+: now also J1.3 (D+)
- net USB_OTG_FS_D-: now also J1.2 (D-)
- net VDD_3V3: now also J16.3 (Pin_3), JP1.1 (A); no longer J16.1 (Pin_1)
- net VDD_5V: now also J16.5 (Pin_5)
- net VDD_5V_SERVO: now also J12.1 (Pin_1), J12.10 (Pin_10), J12.2 (Pin_2), J12.3 (Pin_3), J12.4 (Pin_4), J12.5 (Pin_5), J12.6 (Pin_6), J12.7 (Pin_7), J12.8 (Pin_8), J12.9 (Pin_9), J16.7 (Pin_7)
- net at R14.2: now also J10.6 (Pin_6)
- net at R14.2: now also J10.3 (Pin_3)
- net at R14.2: now also J10.2 (Pin_2)
- net at R14.2: now also J10.4 (Pin_4)
- net at R14.2: now also J10.1 (Pin_1)
- net at R14.2: now also J10.5 (Pin_5)
- net SYS_JTMS-SWCLK renamed SYS_JTCK-SWCLK
- net SYS_JTMS-SWO renamed SYS_JTDO-SWO
- new net: J10.9 (Pin_9), R14.2
- new net: J16.2 (Pin_2), R2.2
- new net: J10.8 (Pin_8), R14.2
- new net: J16.1 (Pin_1), JP1.2 (B)
- new net: J10.10 (Pin_10), R14.2
- new net: J10.7 (Pin_7), R14.2
- new net 3V3_JP: J16.4 (Pin_4)
- new net 5V0_JP: J16.6 (Pin_6)
- new net 5V0_SERVO_JP: J16.8 (Pin_8)
- new net BOOT0: R2.1
- new net TM12_CH1: R14.1
- new net TM12_CH2: R14.1
- new net TM13_CH1: R14.1
- new net TM3_CH4: R14.1
Other:
- moved on the sheet: C16

Commit message: Updated Penguin project
Parts:
- J10, J11: footprint Connector_Molex:Molex_PicoBlade_53047-0610_1x06_P1.25mm_Vertical -> user_lib:Molex_PicoBlade_53047-0610_1x06_P1.25mm_Vertical
- J14, J9: footprint Connector_Molex:Molex_PicoBlade_53047-0410_1x04_P1.25mm_Vertical -> user_lib:Molex_PicoBlade_53047-0410_1x04_P1.25mm_Vertical
- J2, J5: footprint Connector_Molex:Molex_PicoBlade_53047-0310_1x03_P1.25mm_Vertical -> user_lib:Molex_PicoBlade_53047-0310_1x03_P1.25mm_Vertical
- R2: footprint Resistor_SMD:R_0402_1005Metric -> Resistor_SMD:R_0603_1608Metric
Connections:
- net 3V3_JP: now also J16.2 (Pin_2); no longer J16.4 (Pin_4)
- net 5V0_JP: now also J16.10 (Pin_10); no longer J16.6 (Pin_6)
- net 5V0_SERVO_JP: now also J16.4 (Pin_4), J16.6 (Pin_6); no longer J16.8 (Pin_8)
- net GND: now also J16.8 (Pin_8); no longer J16.1 (Pin_1)
- net TM12_CH1: now also R14.1; no longer R14.1
- net TM12_CH2: now also R14.1; no longer R14.1
- net TM2_CH1: now also R14.1; no longer R14.1
- net TM3_CH1: now also R14.1; no longer R14.1
- net TM3_CH2: now also R14.1; no longer R14.1
- net TM3_CH3: now also R14.1; no longer R14.1
- net TM3_CH4: now also R14.1; no longer R14.1
- net TM4_CH3: now also R14.1; no longer R14.1
- net TM4_CH4: now also R14.1; no longer R14.1
- net VDD_3V3: now also J16.1 (Pin_1); no longer J16.3 (Pin_3)
- net VDD_5V: now also J16.9 (Pin_9); no longer J16.5 (Pin_5)
- net VDD_5V_SERVO: now also J16.3 (Pin_3), J16.5 (Pin_5); no longer J16.7 (Pin_7)
- net at R2.2: now also J16.7 (Pin_7); no longer J16.2 (Pin_2)
Other:
- moved on the sheet: J16, R2

Commit message: Updated Penguin project
Parts:
- R2: footprint Resistor_SMD:R_0603_1608Metric -> Resistor_SMD:R_0402_1005Metric
Connections:
- net TM12_CH2: now also R14.1; no longer R14.1
- net TM3_CH1: now also R14.1; no longer R14.1
- net TM3_CH2: now also R14.1; no longer R14.1
- net TM4_CH3: now also R14.1; no longer R14.1
- net TM4_CH4: now also R14.1; no longer R14.1

Commit message: Updated Penguin project
Parts:
- added R14 (x2): 33, Resistor_SMD:R_0402_1005Metric, symbol Device:R_Small
Connections:
- net GND: now also R14.1, R14.2
- net at R14.2: now also J10.2 (Pin_2); no longer J10.6 (Pin_6)
- net at R14.2: now also J10.4 (Pin_4); no longer J10.3 (Pin_3)
- net at R14.2: now also J10.3 (Pin_3); no longer J10.2 (Pin_2)
- net at R14.2: now also J10.6 (Pin_6); no longer J10.4 (Pin_4)
- net at J10.5 (Pin_5): now also R14.2; no longer R14.2
- net at J10.7 (Pin_7): now also R14.2; no longer R14.2
- net TM12_CH2 renamed TM12_CH2/ADC1_EXTI15
- net TM12_CH2/ADC1_EXTI15: now also R14.2
- net TM2_CH1 renamed TM2_CH1/ADC2_EXTI15
- net TM2_CH1/ADC2_EXTI15: now also R14.1
Other:
- moved on the sheet: J10, J11, J12, R14

Commit message: Updated Penguin project
Parts:
- JP1: footprint Jumper:SolderJumper-2_P1.3mm_Open_Pad1.0x1.5mm -> Jumper:SolderJumper-2_P1.3mm_Open_RoundedPad1.0x1.5mm
- renumbered J11 to J10, J12 to J11, J10 to J9
Other:
- note added: "R_4"
- note added: "R_5"
- moved on the sheet: C16, J1, J16, J5, JP1, R2

Commit message: Updated Penguin project
Parts:
- R14: value 22 -> 220
- R14: value 33 -> 330
Changed lines of the file:
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@@
       (effects (font (size 1.27 1.27)))
     )
-    (property "Value" "22" (at 182.245 169.545 90)
+    (property "Value" "220" (at 182.245 169.545 90)
       (effects (font (size 1.27 1.27)))
     )
@@
       (effects (font (size 1.27 1.27)))
     )
-    (property "Value" "22" (at 182.245 151.765 90)
+    (property "Value" "220" (at 182.245 151.765 90)
       (effects (font (size 1.27 1.27)))
     )
@@
       (effects (font (size 1.27 1.27)))
     )
-    (property "Value" "22" (at 182.245 156.845 90)
+    (property "Value" "220" (at 182.245 156.845 90)
       (effects (font (size 1.27 1.27)))
     )
@@
       (effects (font (size 1.27 1.27)))
     )
-    (property "Value" "33" (at 151.765 158.115 0)
+    (property "Value" "330" (at 151.765 158.115 0)
       (effects (font (size 1.27 1.27)))
     )
@@
       (effects (font (size 1.27 1.27)))
     )
-    (property "Value" "33" (at 145.415 158.115 0)
+    (property "Value" "330" (at 145.415 158.115 0)
       (effects (font (size 1.27 1.27)))
     )
@@
       (effects (font (size 1.27 1.27)))
     )
-    (property "Value" "22" (at 182.245 154.305 90)
+    (property "Value" "220" (at 182.245 154.305 90)
       (effects (font (size 1.27 1.27)))
     )
@@
       (effects (font (size 1.27 1.27)))
     )
-    (property "Value" "22" (at 182.245 167.005 90)
+    (property "Value" "220" (at 182.245 167.005 90)
       (effects (font (size 1.27 1.27)))
     )
@@
       (effects (font (size 1.27 1.27)))
     )
-    (property "Value" "22" (at 182.245 161.925 90)
+    (property "Value" "220" (at 182.245 161.925 90)
       (effects (font (size 1.27 1.27)))
     )
@@
       (effects (font (size 1.27 1.27)))
     )
-    (property "Value" "22" (at 182.245 172.085 90)
+    (property "Value" "220" (at 182.245 172.085 90)
       (effects (font (size 1.27 1.27)))
     )
@@
       (effects (font (size 1.27 1.27)))
     )
-    (property "Value" "22" (at 182.245 149.225 90)
+    (property "Value" "220" (at 182.245 149.225 90)
       (effects (font (size 1.27 1.27)))
     )
@@
       (effects (font (size 1.27 1.27)))
     )
-    (property "Value" "22" (at 182.245 159.385 90)
+    (property "Value" "220" (at 182.245 159.385 90)
       (effects (font (size 1.27 1.27)))
     )
@@
       (effects (font (size 1.27 1.27)))
     )
-    (property "Value" "22" (at 182.245 164.465 90)
-      (effects (font (size 1.27 1.27)))
-    )
+    (property "Value" "220" (at 182.245 164.465 90)
+      (effects (font (size 1.27 1.27)))
+    )

Commit message: Penguin Junior 1.1 release
Parts:
- removed C14: 10u, Capacitor_SMD:C_0603_1608Metric, symbol Device:C_Small
Other:
- note removed: "R_4"
- note removed: "R_5"
- moved on the sheet: C15
Changed lines of the file:
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@@
   (junction (at 241.3 30.48) (diameter 0) (color 0 0 0 0)
-  )
-  (junction (at 241.3 38.1) (diameter 0) (color 0 0 0 0)
   )
   (no_connect (at 43.815 187.325))
@@
     (stroke (width 0) (type default))
   )
-  (wire (pts (xy 250.19 30.48) (xy 250.19 31.75))
-    (stroke (width 0) (type default))
-  )
   (wire (pts (xy 273.685 75.565) (xy 273.685 79.375))
     (stroke (width 0) (type default))
   )
-  (wire (pts (xy 241.3 38.1) (xy 241.3 36.83))
-    (stroke (width 0) (type default))
-  )
   (wire (pts (xy 69.85 40.64) (xy 69.85 52.07))
     (stroke (width 0) (type default))
@@
     (stroke (width 0) (type default))
   )
-  (wire (pts (xy 241.3 38.1) (xy 241.3 40.64))
+  (wire (pts (xy 241.3 36.83) (xy 241.3 40.64))
     (stroke (width 0) (type default))
   )
@@
     (stroke (width 0) (type default))
   )
-  (wire (pts (xy 250.19 38.1) (xy 241.3 38.1))
-    (stroke (width 0) (type default))
-  )
   (wire (pts (xy 229.87 160.655) (xy 229.87 163.195))
     (stroke (width 0) (type default))
@@
     (stroke (width 0) (type default))
   )
-  (wire (pts (xy 241.3 30.48) (xy 250.19 30.48))
-    (stroke (width 0) (type default))
-  )
   (wire (pts (xy 207.01 155.575) (xy 208.28 155.575))
     (stroke (width 0) (type default))
@@
     (stroke (width 0) (type default))
   )
-  (wire (pts (xy 250.19 36.83) (xy 250.19 38.1))
-    (stroke (width 0) (type default))
-  )
   (wire (pts (xy 227.965 79.375) (xy 227.965 65.405))
     (stroke (width 0) (type default))
@@
     (stroke (width 0) (type default))
   )
-  (text "R_5" (at 148.59 156.21 90)
-    (effects (font (size 0.7 0.7)) (justify right bottom))
-  )
-  (text "R_4" (at 154.94 156.21 90)
-    (effects (font (size 0.7 0.7)) (justify right bottom))
-  )
   (global_label "VDD_3V3" (shape input) (at 81.28 34.29 90) (fields_autoplaced)
     (effects (font (size 1.27 1.27)) (justify left))
@@
     (property "Intersheetrefs" "${INTERSHEET_REFS}" (at 33.655 126.6455 90)
       (effects (font (size 1.27 1.27)) (justify left) hide)
-    )
-  )
-  (symbol (lib_id "Device:C_Small") (at 241.3 34.29 180) (unit 1)
-    (in_bom yes) (on_board yes) (dnp no)
-    (property "Reference" "C14" (at 238.76 34.29 90)
-      (effects (font (size 1.27 1.27)))
-    )
-    (property "Value" "10u" (at 243.84 34.29 90)
-      (effects (font (size 1.27 1.27)))
-    )
-    (property "Footprint" "Capacitor_SMD:C_0603_1608Metric" (at 241.3 34.29 0)
-      (effects (font (size 1.27 1.27)) hide)
-    )
-    (property "Datasheet" "~" (at 241.3 34.29 0)
-      (effects (font (size 1.27 1.27)) hide)
-    )
-    (pin "1")
-    (pin "2")
-    (instances
-      (project "Penguin Junior"
-        (path "/dfff5ef9-3e3a-4442-aa32-5f49584e77ca"
-          (reference "C14") (unit 1)
-        )
-        (path "/dfff5ef9-3e3a-4442-aa32-5f49584e77ca/cdfcf036-4a9f-4e8f-b9af-f5f7029d25f4"
-          (reference "C23") (unit 1)
-        )
-      )
     )
   )
@@
     )
   )
-  (symbol (lib_id "Device:C_Small") (at 250.19 34.29 180) (unit 1)
-    (in_bom yes) (on_board yes) (dnp no)
-    (property "Reference" "C15" (at 247.65 34.29 90)
-      (effects (font (size 1.27 1.27)))
-    )
-    (property "Value" "100n" (at 252.73 34.29 90)
-      (effects (font (size 1.27 1.27)))
-    )
-    (property "Footprint" "Capacitor_SMD:C_0402_1005Metric" (at 250.19 34.29 0)
-      (effects (font (size 1.27 1.27)) hide)
-    )
-    (property "Datasheet" "~" (at 250.19 34.29 0)
-      (effects (font (size 1.27 1.27)) hide)
-    )
+  (symbol (lib_id "Device:C_Small") (at 241.3 34.29 180) (unit 1)
+    (in_bom yes) (on_board yes) (dnp no)
+    (property "Reference" "C15" (at 238.76 34.29 90)
+      (effects (font (size 1.27 1.27)))
+    )
+    (property "Value" "100n" (at 243.84 34.29 90)
+      (effects (font (size 1.27 1.27)))
+    )
+    (property "Footprint" "Capacitor_SMD:C_0402_1005Metric" (at 241.3 34.29 0)
+      (effects (font (size 1.27 1.27)) hide)
+    )
+    (property "Datasheet" "~" (at 241.3 34.29 0)
+      (effects (font (size 1.27 1.27)) hide)
+    )

Commit message: Updated KiCad version
Parts:
- renumbered C15 to C24, C16 to C25, J2 to J3, J1 to J5, R2 to R10, R3 to R11, R4 to R12, R5 to R13, R6 to R14, R7 to R15, R8 to R16
