File: Hardware/Penguin Junior/Connectors.kicad_sch (KiCad schematic)
At the start: 35 parts, among them J10 Conn_01x06_UART, J10 Conn_01x10, J11 Conn_01x06_UART, J11 Conn_01x10, J14 Conn_01x04_UART, J16 Conn_02x05_SWD, J2 Conn_01x03_Video, J3 Micro_SD_Card_Det1, J5 Conn_01x03_Video, J5 USB_B_Micro, J9 Conn_01x04_I2C, J9 Conn_01x10

Commit message: Penguin Junior 1.2 prototype
Parts:
- removed J16: Conn_02x05_SWD, Connector_PinHeader_1.27mm:PinHeader_2x05_P1.27mm_Vertical, symbol Connector_Generic:Conn_02x05_Odd_Even
- added JP4, JP5, JP6: SolderJumper_2_Open, Jumper:SolderJumper-2_P1.3mm_Open_RoundedPad1.0x1.5mm, symbol Jumper:SolderJumper_2_Open
- added R39: 10K, Resistor_SMD:R_0402_1005Metric, symbol Device:R
Connections:
- net VDD_3V3 is gone; now on net 3V3_JP: C24.2, J3.4 (VDD), JP1.1 (A), R11.1, R12.1, R13.1, R14.1, R15.1, R16.2
- net 3V3_JP: now also JP6.2 (B)
- net 5V0_JP: now also J10.1 (Pin_1), J11.1 (Pin_1), J14.1 (Pin_1), J9.1 (Pin_1), JP4.2 (B)
- net 5V0_SERVO_JP: now also JP5.1 (A)
- net BOOT0: now also R39.1; no longer R10.1
- net GND: now also R10.2
- net VDD_5V_SERVO: now also JP5.2 (B)
- removed net VDD_5V: J10.1 (Pin_1), J11.1 (Pin_1), J14.1 (Pin_1), J2.1 (Pin_1), J5.1 (Pin_1), J9.1 (Pin_1)
- new net: J2.1 (Pin_1), J5.1 (Pin_1), JP4.1 (A)
- new net: JP6.1 (A), R10.1, R39.2
Other:
- moved on the sheet: C24, J2, J5, R10

Commit message: Update Penguin concept
Parts:
- added JP2: SolderJumper_2_Open, Jumper:SolderJumper-2_P1.3mm_Open_RoundedPad1.0x1.5mm, symbol Jumper:SolderJumper_2_Open
- J3: footprint sd:TF01A -> sd:TF01A-NEW
Connections:
- net 5V0_SERVO_JP: now also JP2.1 (A)
- net VDD_5V_SERVO: now also JP2.2 (B)
Other:
- moved on the sheet: JP5
Changed lines of the file:
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@@
 	)
 	(junction
+		(at 57.15 44.45)
+		(diameter 0)
+		(color 0 0 0 0)
+	)
+	(junction
 		(at 229.87 168.275)
 		(diameter 0)
@@
 	)
 	(junction
+		(at 41.275 44.45)
+		(diameter 0)
+		(color 0 0 0 0)
+	)
+	(junction
 		(at 147.955 153.035)
 		(diameter 0)
@@
 	(wire
 		(pts
+			(xy 57.15 44.45) (xy 64.77 44.45)
+		)
+		(stroke
+			(width 0)
+			(type default)
+		)
+	)
+	(wire
+		(pts
 			(xy 87.63 44.45) (xy 87.63 46.99)
 		)
@@
 	(wire
 		(pts
+			(xy 57.15 48.26) (xy 57.15 44.45)
+		)
+		(stroke
+			(width 0)
+			(type default)
+		)
+	)
+	(wire
+		(pts
 			(xy 73.66 144.145) (xy 78.74 144.145)
 		)
@@
 	(wire
 		(pts
+			(xy 52.705 48.26) (xy 57.15 48.26)
+		)
+		(stroke
+			(width 0)
+			(type default)
+		)
+	)
+	(wire
+		(pts
 			(xy 180.34 155.575) (xy 185.42 155.575)
 		)
@@
 	(wire
 		(pts
+			(xy 41.275 44.45) (xy 37.465 44.45)
+		)
+		(stroke
+			(width 0)
+			(type default)
+		)
+	)
+	(wire
+		(pts
 			(xy 59.055 75.565) (xy 59.055 73.66)
 		)
@@
 	(wire
 		(pts
+			(xy 41.275 44.45) (xy 45.085 44.45)
+		)
+		(stroke
+			(width 0)
+			(type default)
+		)
+	)
+	(wire
+		(pts
 			(xy 227.965 79.375) (xy 227.965 65.405)
 		)
@@
 	(wire
 		(pts
+			(xy 41.275 48.26) (xy 41.275 44.45)
+		)
+		(stroke
+			(width 0)
+			(type default)
+		)
+	)
+	(wire
+		(pts
 			(xy 229.87 168.275) (xy 231.14 168.275)
 		)
@@
 	(wire
 		(pts
-			(xy 45.085 44.45) (xy 64.77 44.45)
+			(xy 52.705 44.45) (xy 57.15 44.45)
 		)
 		(stroke
@@
 	(wire
 		(pts
+			(xy 45.085 48.26) (xy 41.275 48.26)
+		)
+		(stroke
+			(width 0)
+			(type default)
+		)
+	)
+	(wire
+		(pts
 			(xy 43.18 81.28) (xy 43.18 93.98)
 		)
@@
 	(symbol
 		(lib_id "Jumper:SolderJumper_2_Open")
+		(at 48.895 48.26 0)
+		(mirror x)
+		(unit 1)
+		(exclude_from_sim no)
+		(in_bom yes)
+		(on_board yes)
+		(dnp no)
+		(property "Reference" "JP2"
+			(at 48.895 54.61 0)
+			(effects
+				(font
+					(size 1.27 1.27)
+				)
+			)
+		)
+		(property "Value" "SolderJumper_2_Open"
+			(at 48.895 52.07 0)
+			(effects
+				(font
+					(size 1.27 1.27)
+				)
+			)
+		)
+		(property "Footprint" "Jumper:SolderJumper-2_P1.3mm_Open_RoundedPad1.0x1.5mm"
+			(at 48.895 48.26 0)
+			(effects
+				(font
+					(size 1.27 1.27)
+				)
+				(hide yes)
+			)
+		)
+		(property "Datasheet" "~"
+			(at 48.895 48.26 0)
+			(effects
+				(font
+					(size 1.27 1.27)
+				)
+				(hide yes)
+			)
+		)
+		(property "Description" ""
+			(at 48.895 48.26 0)
+			(effects
+				(font
+					(size 1.27 1.27)
+				)
+				(hide yes)
+			)
+		)
+		(pin "1"
+		)
+		(pin "2"
+		)
+		(instances
+			(project "Penguin Junior"
+				(path "/dfff5ef9-3e3a-4442-aa32-5f49584e77ca/cdfcf036-4a9f-4e8f-b9af-f5f7029d25f4"
+					(reference "JP2")
+					(unit 1)
+				)
+			)
+		)
+	)
+	(symbol
+		(lib_id "Jumper:SolderJumper_2_Open")
 		(at 111.76 90.805 270)
 		(mirror x)
@@
 	(symbol
 		(lib_id "Jumper:SolderJumper_2_Open")
-		(at 41.275 44.45 0)
+		(at 48.895 44.45 0)
 		(unit 1)
 		(exclude_from_sim no)
@@
 		(fields_autoplaced yes)
 		(property "Reference" "JP5"
-			(at 41.275 38.1 0)
+			(at 48.895 38.1 0)
 			(effects
 				(font
@@
 		)
 		(property "Value" "SolderJumper_2_Open"
-			(at 41.275 40.64 0)
+			(at 48.895 40.64 0)
 			(effects
 				(font
@@
 		)
 		(property "Footprint" "Jumper:SolderJumper-2_P1.3mm_Open_RoundedPad1.0x1.5mm"
-			(at 41.275 44.45 0)
+			(at 48.895 44.45 0)
 			(effects
 				(font
@@
 		)
 		(property "Datasheet" "~"
-			(at 41.275 44.45 0)
+			(at 48.895 44.45 0)
 			(effects
 				(font
@@
 		)
 		(property "Description" ""
-			(at 41.275 44.45 0)
+			(at 48.895 44.45 0)
 			(effects
 				(font
@@
 			)
 		)
-		(property "Footprint" "sd:TF01A"
+		(property "Footprint" "sd:TF01A-NEW"
 			(at 304.165 45.085 0)
 			(effects

Commit message: Update 1.2 project
Parts:
- removed J5: USB_B_Micro, user_lib:U-F-M5DD-W-2-SUS, symbol Connector:USB_B_Micro
- added J5: USB_C, user_lib:HCTL HC-TYPE-C-16P-01M, symbol Connector:USB_C_Receptacle_USB2.0_16P
Connections:
- net GND: now also J5.A1 (GND), J5.A12 (GND), J5.B1 (GND), J5.B12 (GND), J5.S1 (SHIELD)
- net USB_OTG_FS_D+: now also J5.A6 (D+), J5.B6 (D+)
- net USB_OTG_FS_D-: now also J5.A7 (D-), J5.B7 (D-)
- net VDD_5V_USB: now also J5.A4 (VBUS), J5.A9 (VBUS), J5.B4 (VBUS), J5.B9 (VBUS)
- no-connect marks 5 -> 8
Other:
- moved on the sheet: C25

Commit message: Penguin Junior 1.2 production
Parts:
- renumbered J11 to J10, J3 to J2, J5 to J4, J9 to J8, J10 to J9, JP6 to JP1, JP5 to JP2, JP2 to JP3, JP4 to JP5, JP1 to JP6, R11 to R15, R12 to R16, R13 to R17, R14 to R18, R15 to R19, R16 to R20, R10 to R21, R39 to R22
Connections:
- net I2C1_SCL: now also J11.4 (Pin_4)
- net I2C1_SDA: now also J11.5 (Pin_5)
- no-connect marks 8 -> 6
