File: Hardware/Penguin Junior/Power.kicad_sch (KiCad schematic)
At the start: 36 parts, among them U6 ST1S14PHR, U7 INA219AxD, U8 LDL1117_3V3

Commit message: Updated project
Parts:
- removed D4: SS54, Diode_SMD:D_SMA, symbol Device:D_Schottky
- removed JP1, JP2: INA219_ADDR, Jumper:SolderJumper-3_P1.3mm_Open_Pad1.0x1.5mm, symbol Jumper:SolderJumper_3_Bridged12
- removed JP3, JP4, JP5: Jumper_2_Bridged, Connector_PinHeader_1.27mm:PinHeader_1x02_P1.27mm_Vertical, symbol Jumper:Jumper_2_Bridged
- added J1: Conn_01x01, user_lib:ContactPlatform_7.0x7.0, symbol Connector_Generic:Conn_01x01
- added JP3 (x2): SolderJumper_3_Open, Jumper:SolderJumper-3_P1.3mm_Open_Pad1.0x1.5mm, symbol Jumper:SolderJumper_3_Open
- C26, C27, C28, C32: footprint Capacitor_SMD:C_0603_1608Metric -> Capacitor_SMD:C_0402_1005Metric
- C29: footprint Capacitor_SMD:C_2220_5650Metric -> Capacitor_SMD:C_1210_3225Metric
- C30: footprint Capacitor_SMD:C_1206_3216Metric -> Capacitor_SMD:C_0603_1608Metric
- C33, C34: footprint Capacitor_SMD:C_0805_2012Metric -> Capacitor_SMD:C_0402_1005Metric
- R27: renamed from R24; value 0m5 -> 0m2; footprint Resistor_SMD:R_2512_6332Metric -> user_lib:R2725
- R28: renamed from R25; footprint Resistor_SMD:R_0603_1608Metric -> Resistor_SMD:R_0402_1005Metric
- R29: renamed from R26; footprint Resistor_SMD:R_0603_1608Metric -> Resistor_SMD:R_0402_1005Metric
- R30: renamed from R27; footprint Resistor_SMD:R_0805_2012Metric -> Resistor_SMD:R_0402_1005Metric
- R31: renamed from R28; footprint Resistor_SMD:R_0805_2012Metric -> Resistor_SMD:R_0603_1608Metric
- R32: renamed from R29; footprint Resistor_SMD:R_0805_2012Metric -> Resistor_SMD:R_0603_1608Metric
- R5: footprint Resistor_SMD:R_0603_1608Metric -> Resistor_SMD:R_0402_1005Metric
- renumbered D5 to D4, D6 to D5, D7 to D6
Connections:
- net GND: now also J1.1 (Pin_1), JP3.1 (A), JP3.1 (A)
- net VDD_3V3: now also JP3.3 (B), JP3.3 (B)
- net VDD_BUCK_6-26_IN: no longer C29.2, C30.2, U6.5 (EN2), U6.7 (VIN)
- net VDD_BUCK_6-26_OUT: now also C29.2, C30.2, U6.5 (EN2), U6.7 (VIN)
- net 5V0_JP: now reaches F1.1, F2.2
- net at U7.1 (A1): now also JP3.2 (C)
- net at U7.2 (A0): now also JP3.2 (C)
- net 3V3_JP: now reaches C34.1, U8.2 (VO)
- net VDD_BUCK_5V renamed 5V0_SERVO_JP
Other:
- note removed: "изменить резистор на: https://www.lcsc.com/product-detail/Current-Sense-Resistors-Shunt-Resistors_RALEC-LR2725-24R0002F1_C304390.html"
- moved on the sheet: D4, D5, F1, F2

Commit message: Updated Penguin project
Parts:
- added R36: 75, Resistor_SMD:R_0603_1608Metric, symbol Device:R_Small
- C30: footprint Capacitor_SMD:C_0603_1608Metric -> Capacitor_SMD:C_0805_2012Metric
Connections:
- net 5V0_JP: now also D4.1 (K), D5.1 (K); no longer F2.2
- net 5V0_SERVO_JP: now also F2.1; no longer C22.1, C32.2, L1.2, R30.2, R31.2
- net GND: now also R36.1; no longer R32.1
- new net: R32.1, R36.2
- new net VDD_BUCK_5V: C22.1, C32.2, F2.2, L1.2, R30.2, R31.2
Other:
- note added: "или 0"
- moved on the sheet: D4, D5, F1, F2

Commit message: Updated Penguin project
Changed lines of the file:
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@@
     (effects (font (size 1.27 1.27)) (justify left top))
   )
-  (text_box "r_2=r_1/((v_out/1.22)-1)"
-    (at 157.48 79.375 0) (size 27.94 3.175)
+  (text_box "r_2=r_1/((v/1.22)-1)"
+    (at 157.48 79.375 0) (size 22.86 3.175)
     (stroke (width 0) (type default))
     (fill (type none))

Commit message: Updated Penguin project
Connections:
- net GND: now also R5.1; no longer D1.1 (K)
- net VDD_5V: now also D1.2 (A); no longer R5.1
- net at R5.2: now also D1.1 (K); no longer D1.2 (A)
Other:
- moved on the sheet: D1, R5
Changed lines of the file:
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@@
     )
   )
-  (symbol (lib_id "Device:R") (at 103.505 111.76 90) (unit 1)
-    (in_bom yes) (on_board yes) (dnp no)
-    (property "Reference" "R5" (at 103.505 109.22 90)
-      (effects (font (size 1.27 1.27)))
-    )
-    (property "Value" "220" (at 103.505 114.3 90)
-      (effects (font (size 1.27 1.27)))
-    )
-    (property "Footprint" "Resistor_SMD:R_0402_1005Metric" (at 103.505 113.538 90)
-      (effects (font (size 1.27 1.27)) hide)
-    )
-    (property "Datasheet" "~" (at 103.505 111.76 0)
+  (symbol (lib_id "Device:R") (at 112.395 111.76 270) (mirror x) (unit 1)
+    (in_bom yes) (on_board yes) (dnp no)
+    (property "Reference" "R5" (at 112.395 109.22 90)
+      (effects (font (size 1.27 1.27)))
+    )
+    (property "Value" "220" (at 112.395 114.3 90)
+      (effects (font (size 1.27 1.27)))
+    )
+    (property "Footprint" "Resistor_SMD:R_0402_1005Metric" (at 112.395 113.538 90)
+      (effects (font (size 1.27 1.27)) hide)
+    )
+    (property "Datasheet" "~" (at 112.395 111.76 0)
       (effects (font (size 1.27 1.27)) hide)
     )
@@
     )
   )
-  (symbol (lib_id "Device:LED") (at 112.395 111.76 0) (mirror y) (unit 1)
-    (in_bom yes) (on_board yes) (dnp no)
-    (property "Reference" "D1" (at 112.395 109.22 0)
-      (effects (font (size 1.27 1.27)))
-    )
-    (property "Value" "LED_5V" (at 112.395 115.57 0)
-      (effects (font (size 1.27 1.27)))
-    )
-    (property "Footprint" "LED_SMD:LED_0603_1608Metric" (at 112.395 111.76 0)
-      (effects (font (size 1.27 1.27)) hide)
-    )
-    (property "Datasheet" "~" (at 112.395 111.76 0)
-      (effects (font (size 1.27 1.27)) hide)
-    )
+  (symbol (lib_id "Device:LED") (at 103.505 111.76 0) (mirror y) (unit 1)
+    (in_bom yes) (on_board yes) (dnp no)
+    (property "Reference" "D1" (at 103.505 109.22 0)
+      (effects (font (size 1.27 1.27)))
+    )
+    (property "Value" "LED_5V" (at 103.505 115.57 0)
+      (effects (font (size 1.27 1.27)))
+    )
+    (property "Footprint" "LED_SMD:LED_0603_1608Metric" (at 103.505 111.76 0)
+      (effects (font (size 1.27 1.27)) hide)
+    )
+    (property "Datasheet" "~" (at 103.505 111.76 0)
+      (effects (font (size 1.27 1.27)) hide)
+    )

Commit message: Updated Penguin project
Parts:
- JP3: footprint Jumper:SolderJumper-3_P1.3mm_Open_Pad1.0x1.5mm -> Jumper:SolderJumper-3_P1.3mm_Open_RoundedPad1.0x1.5mm_NumberLabels
- renumbered D5 to D4, D6 to D5, D4 to D6, F2 to F1, F1 to F2, R31 to R1, R32 to R2, R27 to R29, R36 to R3, R28 to R30, R29 to R31, R30 to R32, U6 to U5, U7 to U6, U8 to U7
Other:
- note added: "R_3"

Commit message: Updated Penguin project
Parts:
- R30, R31: value 22 -> 220
Changed lines of the file:
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@@
       (effects (font (size 1.27 1.27)) (justify left))
     )
-    (property "Value" "22" (at 27.94 46.355 0)
+    (property "Value" "220" (at 27.94 46.355 0)
       (effects (font (size 1.27 1.27)) (justify left))
     )
@@
       (effects (font (size 1.27 1.27)) (justify left))
     )
-    (property "Value" "22" (at 13.97 46.355 0)
-      (effects (font (size 1.27 1.27)) (justify left))
-    )
+    (property "Value" "220" (at 13.97 46.355 0)
+      (effects (font (size 1.27 1.27)) (justify left))
+    )

Commit message: Penguin Junior 1.1 release
Other:
- note removed: "R_1"
- note removed: "R_2"
- note removed: "R_3"
- moved on the sheet: C33, C34, D1, R5, U7

Commit message: Updated KiCad version
Parts:
- renumbered C22 to C31, J1 to J14, JP3 to JP2
