File: Hardware/Penguin Junior/OSD.kicad_sch (KiCad schematic)
At the start: 13 parts, among them Q1 BSS138, U4 MAX7456, Y1 27MHz

Commit message: Updated project
Parts:
- C17, C18, C19, C22: footprint Capacitor_SMD:C_0603_1608Metric -> Capacitor_SMD:C_0402_1005Metric
- C20, C21: footprint Capacitor_SMD:C_0603_1608Metric -> Capacitor_SMD:C_1206_3216Metric
- R6: renamed from R8; footprint Resistor_SMD:R_0603_1608Metric -> Resistor_SMD:R_0402_1005Metric
- R7: renamed from R9; footprint Resistor_SMD:R_0603_1608Metric -> Resistor_SMD:R_0402_1005Metric
- R8: renamed from R10; footprint Resistor_SMD:R_0603_1608Metric -> Resistor_SMD:R_0402_1005Metric
- R9: renamed from R11; footprint Resistor_SMD:R_0603_1608Metric -> Resistor_SMD:R_0402_1005Metric
Connections:
- net SDOUT: no longer names the net of Q1.3 (D), R8.2, U4.11 (SDOUT)
Other:
- moved on the sheet: R9
Changed lines of the file:
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@@
+    (stroke (width 0) (type default))
+  )
+  (wire (pts (xy 191.135 113.03) (xy 191.135 111.76))
     (stroke (width 0) (type default))
   )
@@
     (stroke (width 0) (type default))
   )
-  (wire (pts (xy 191.135 119.38) (xy 191.135 120.65))
+  (wire (pts (xy 191.135 120.65) (xy 191.135 121.92))
     (stroke (width 0) (type default))
   )
@@
     (stroke (width 0) (type default))
   )
-  (wire (pts (xy 104.775 106.68) (xy 99.06 106.68))
+  (wire (pts (xy 99.06 106.68) (xy 141.605 106.68))
     (stroke (width 0) (type default))
   )
@@
   (wire (pts (xy 155.575 72.39) (xy 155.575 76.2))
     (stroke (width 0) (type default))
-  )
-  (wire (pts (xy 139.7 106.68) (xy 141.605 106.68))
-    (stroke (width 0) (type default))
-  )
-  (label "SDOUT" (at 139.7 106.68 270) (fields_autoplaced)
-    (effects (font (size 1.27 1.27)) (justify right bottom))
-  )
-  (label "SDOUT" (at 104.775 106.68 0) (fields_autoplaced)
-    (effects (font (size 1.27 1.27)) (justify left bottom))
   )
   (global_label "VDD_5V" (shape input) (at 99.06 91.44 90) (fields_autoplaced)
@@
       (effects (font (size 1.27 1.27)))
     )
-    (property "Footprint" "Capacitor_SMD:C_0603_1608Metric" (at 189.865 103.1748 0)
+    (property "Footprint" "Capacitor_SMD:C_1206_3216Metric" (at 189.865 103.1748 0)
       (effects (font (size 1.27 1.27)) hide)
     )
@@
     )
   )
-  (symbol (lib_id "Device:R") (at 191.135 115.57 180) (unit 1)
-    (in_bom yes) (on_board yes) (dnp no) (fields_autoplaced)
-    (property "Reference" "R11" (at 193.04 114.3 0)
+  (symbol (lib_id "Device:R") (at 191.135 116.84 180) (unit 1)
+    (in_bom yes) (on_board yes) (dnp no) (fields_autoplaced)
+    (property "Reference" "R9" (at 193.04 115.57 0)
       (effects (font (size 1.27 1.27)) (justify right))
     )
-    (property "Value" "75" (at 193.04 116.84 0)
+    (property "Value" "75" (at 193.04 118.11 0)
       (effects (font (size 1.27 1.27)) (justify right))
     )
-    (property "Footprint" "Resistor_SMD:R_0603_1608Metric" (at 192.913 115.57 90)
-      (effects (font (size 1.27 1.27)) hide)
-    )
-    (property "Datasheet" "~" (at 191.135 115.57 0)
-      (effects (font (size 1.27 1.27)) hide)
-    )
-    (pin "1")
-    (pin "2")
-    (instances
-      (project "Penguin Junior"
-        (path "/dfff5ef9-3e3a-4442-aa32-5f49584e77ca/48ae4edb-0e13-4619-bf0c-b661f0a0817d"
-          (reference "R11") (unit 1)
+    (property "Footprint" "Resistor_SMD:R_0402_1005Metric" (at 192.913 116.84 90)
+      (effects (font (size 1.27 1.27)) hide)
+    )
+    (property "Datasheet" "~" (at 191.135 116.84 0)
+      (effects (font (size 1.27 1.27)) hide)
+    )
+    (pin "1")
+    (pin "2")
+    (instances
+      (project "Penguin Junior"
+        (path "/dfff5ef9-3e3a-4442-aa32-5f49584e77ca/48ae4edb-0e13-4619-bf0c-b661f0a0817d"
+          (reference "R9") (unit 1)
         )
       )
@@
       (effects (font (size 1.27 1.27)) (justify left))
     )
-    (property "Footprint" "Capacitor_SMD:C_0603_1608Metric" (at 227.0252 83.185 0)
+    (property "Footprint" "Capacitor_SMD:C_0402_1005Metric" (at 227.0252 83.185 0)
       (effects (font (size 1.27 1.27)) hide)
     )
@@
       (effects (font (size 1.27 1.27)) (justify left))
     )
-    (property "Footprint" "Capacitor_SMD:C_0603_1608Metric" (at 238.4552 83.185 0)
+    (property "Footprint" "Capacitor_SMD:C_0402_1005Metric" (at 238.4552 83.185 0)
       (effects (font (size 1.27 1.27)) hide)
     )
@@
   (symbol (lib_id "Device:R") (at 205.105 97.79 90) (unit 1)
     (in_bom yes) (on_board yes) (dnp no) (fields_autoplaced)
-    (property "Reference" "R8" (at 205.105 92.075 90)
+    (property "Reference" "R6" (at 205.105 92.075 90)
       (effects (font (size 1.27 1.27)))
     )
@@
       (effects (font (size 1.27 1.27)))
     )
-    (property "Footprint" "Resistor_SMD:R_0603_1608Metric" (at 205.105 99.568 90)
+    (property "Footprint" "Resistor_SMD:R_0402_1005Metric" (at 205.105 99.568 90)
       (effects (font (size 1.27 1.27)) hide)
     )
@@
       (project "Penguin Junior"
         (path "/dfff5ef9-3e3a-4442-aa32-5f49584e77ca/48ae4edb-0e13-4619-bf0c-b661f0a0817d"
-          (reference "R8") (unit 1)
+          (reference "R6") (unit 1)
         )
       )
@@
       (effects (font (size 1.27 1.27)))
     )
-    (property "Footprint" "Capacitor_SMD:C_0603_1608Metric" (at 180.34 110.7948 0)
+    (property "Footprint" "Capacitor_SMD:C_0402_1005Metric" (at 180.34 110.7948 0)
       (effects (font (size 1.27 1.27)) hide)
     )
@@
   (symbol (lib_id "Device:R") (at 80.645 99.695 0) (unit 1)
     (in_bom yes) (on_board yes) (dnp no) (fields_autoplaced)
-    (property "Reference" "R9" (at 82.55 98.425 0)
+    (property "Reference" "R7" (at 82.55 98.425 0)
       (effects (font (size 1.27 1.27)) (justify left))
     )
@@
       (effects (font (size 1.27 1.27)) (justify left))
     )
-    (property "Footprint" "Resistor_SMD:R_0603_1608Metric" (at 78.867 99.695 90)
+    (property "Footprint" "Resistor_SMD:R_0402_1005Metric" (at 78.867 99.695 90)
       (effects (font (size 1.27 1.27)) hide)
     )
@@
       (project "Penguin Junior"
         (path "/dfff5ef9-3e3a-4442-aa32-5f49584e77ca/48ae4edb-0e13-4619-bf0c-b661f0a0817d"
-          (reference "R9") (unit 1)
-        )
-      )
-    )
-  )
-  (symbol (lib_id "power:GND") (at 191.135 120.65 0) (unit 1)
-    (in_bom yes) (on_board yes) (dnp no) (fields_autoplaced)
-    (property "Reference" "#PWR014" (at 191.135 127 0)
-      (effects (font (size 1.27 1.27)) hide)
-    )
-    (property "Value" "GND" (at 191.135 125.095 0)
-      (effects (font (size 1.27 1.27)))
-    )
-    (property "Footprint" "" (at 191.135 120.65 0)
-      (effects (font (size 1.27 1.27)) hide)
-    )
-    (property "Datasheet" "" (at 191.135 120.65 0)
+          (reference "R7") (unit 1)
+        )
+      )
+    )
+  )
+  (symbol (lib_id "power:GND") (at 191.135 121.92 0) (unit 1)
+    (in_bom yes) (on_board yes) (dnp no) (fields_autoplaced)
+    (property "Reference" "#PWR014" (at 191.135 128.27 0)
+      (effects (font (size 1.27 1.27)) hide)
+    )
+    (property "Value" "GND" (at 191.135 126.365 0)
+      (effects (font (size 1.27 1.27)))
+    )
+    (property "Footprint" "" (at 191.135 121.92 0)
+      (effects (font (size 1.27 1.27)) hide)
+    )
+    (property "Datasheet" "" (at 191.135 121.92 0)
       (effects (font (size 1.27 1.27)) hide)
     )
@@
       (effects (font (size 1.27 1.27)) (justify left))
     )
-    (property "Footprint" "Capacitor_SMD:C_0603_1608Metric" (at 249.8852 83.185 0)
+    (property "Footprint" "Capacitor_SMD:C_0402_1005Metric" (at 249.8852 83.185 0)
       (effects (font (size 1.27 1.27)) hide)
     )
@@
       (effects (font (size 1.27 1.27)))
     )
-    (property "Footprint" "Capacitor_SMD:C_0603_1608Metric" (at 189.865 96.8248 0)
+    (property "Footprint" "Capacitor_SMD:C_1206_3216Metric" (at 189.865 96.8248 0)
       (effects (font (size 1.27 1.27)) hide)
     )
@@
   (symbol (lib_id "Device:R") (at 99.06 99.695 0) (unit 1)
     (in_bom yes) (on_board yes) (dnp no) (fields_autoplaced)
-    (property "Reference" "R10" (at 100.965 98.425 0)
+    (property "Reference" "R8" (at 100.965 98.425 0)
       (effects (font (size 1.27 1.27)) (justify left))
     )
@@
       (effects (font (size 1.27 1.27)) (justify left))
     )
-    (property "Footprint" "Resistor_SMD:R_0603_1608Metric" (at 97.282 99.695 90)
+    (property "Footprint" "Resistor_SMD:R_0402_1005Metric" (at 97.282 99.695 90)
       (effects (font (size 1.27 1.27)) hide)
     )
@@
       (project "Penguin Junior"
         (path "/dfff5ef9-3e3a-4442-aa32-5f49584e77ca/48ae4edb-0e13-4619-bf0c-b661f0a0817d"
-          (reference "R10") (unit 1)
-        )
-      )
+          (reference "R8") (unit 1)
+        )
+      )

Commit message: Updated Penguin project
Other:
- moved on the sheet: R9
Changed lines of the file:
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@@
     (stroke (width 0) (type default))
   )
-  (wire (pts (xy 170.815 97.79) (xy 182.245 97.79))
+  (wire (pts (xy 175.895 97.79) (xy 182.245 97.79))
     (stroke (width 0) (type default))
   )
@@
     (stroke (width 0) (type default))
   )
-  (wire (pts (xy 169.545 101.6) (xy 170.815 101.6))
+  (wire (pts (xy 169.545 101.6) (xy 175.895 101.6))
     (stroke (width 0) (type default))
   )
@@
     (stroke (width 0) (type default))
   )
-  (wire (pts (xy 170.815 101.6) (xy 170.815 97.79))
+  (wire (pts (xy 175.895 101.6) (xy 175.895 97.79))
     (stroke (width 0) (type default))
   )
@@
     )
   )
-  (symbol (lib_id "Device:R") (at 191.135 116.84 180) (unit 1)
-    (in_bom yes) (on_board yes) (dnp no) (fields_autoplaced)
-    (property "Reference" "R9" (at 193.04 115.57 0)
+  (symbol (lib_id "Device:R") (at 191.135 116.84 0) (mirror x) (unit 1)
+    (in_bom yes) (on_board yes) (dnp no)
+    (property "Reference" "R9" (at 189.23 115.57 0)
       (effects (font (size 1.27 1.27)) (justify right))
     )
-    (property "Value" "75" (at 193.04 118.11 0)
+    (property "Value" "75" (at 189.23 118.11 0)
       (effects (font (size 1.27 1.27)) (justify right))
     )
-    (property "Footprint" "Resistor_SMD:R_0402_1005Metric" (at 192.913 116.84 90)
-      (effects (font (size 1.27 1.27)) hide)
-    )
+    (property "Footprint" "Resistor_SMD:R_0402_1005Metric" (at 189.357 116.84 90)
+      (effects (font (size 1.27 1.27)) hide)
+    )

Commit message: Updated Penguin project
Other:
- note added: "проверить токи"
Changed lines of the file:
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@@
     (stroke (width 0) (type default))
+  )
+  (text "проверить токи" (at 97.155 110.49 0)
+    (effects (font (size 1.27 1.27)) (justify left bottom))
   )
   (global_label "VDD_5V" (shape input) (at 99.06 91.44 90) (fields_autoplaced)

Commit message: Updated Penguin project
Other:
- moved on the sheet: C20, C21
Changed lines of the file:
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@@
     (stroke (width 0) (type default))
   )
-  (wire (pts (xy 189.865 104.14) (xy 195.58 104.14))
+  (wire (pts (xy 189.23 104.14) (xy 195.58 104.14))
     (stroke (width 0) (type default))
   )
@@
     (stroke (width 0) (type default))
   )
-  (wire (pts (xy 175.895 97.79) (xy 182.245 97.79))
-    (stroke (width 0) (type default))
-  )
-  (wire (pts (xy 169.545 104.14) (xy 182.245 104.14))
+  (wire (pts (xy 175.895 97.79) (xy 181.61 97.79))
+    (stroke (width 0) (type default))
+  )
+  (wire (pts (xy 169.545 104.14) (xy 181.61 104.14))
     (stroke (width 0) (type default))
   )
@@
     (stroke (width 0) (type default))
   )
-  (wire (pts (xy 189.865 97.79) (xy 195.58 97.79))
+  (wire (pts (xy 189.23 97.79) (xy 195.58 97.79))
     (stroke (width 0) (type default))
   )
@@
     )
   )
-  (symbol (lib_id "Device:C_Polarized") (at 186.055 104.14 90) (unit 1)
+  (symbol (lib_id "Device:C_Polarized") (at 185.42 104.14 90) (unit 1)
     (in_bom yes) (on_board yes) (dnp no)
-    (property "Reference" "C21" (at 189.865 101.6 90)
-      (effects (font (size 1.27 1.27)))
-    )
-    (property "Value" "47" (at 189.23 107.315 90)
-      (effects (font (size 1.27 1.27)))
-    )
-    (property "Footprint" "Capacitor_SMD:C_1206_3216Metric" (at 189.865 103.1748 0)
-      (effects (font (size 1.27 1.27)) hide)
-    )
-    (property "Datasheet" "~" (at 186.055 104.14 0)
+    (property "Reference" "C21" (at 189.23 101.6 90)
+      (effects (font (size 1.27 1.27)))
+    )
+    (property "Value" "47" (at 188.595 107.315 90)
+      (effects (font (size 1.27 1.27)))
+    )
+    (property "Footprint" "Capacitor_SMD:C_1206_3216Metric" (at 189.23 103.1748 0)
+      (effects (font (size 1.27 1.27)) hide)
+    )
+    (property "Datasheet" "~" (at 185.42 104.14 0)
       (effects (font (size 1.27 1.27)) hide)
     )
@@
     )
   )
-  (symbol (lib_id "Device:C_Polarized") (at 186.055 97.79 90) (unit 1)
-    (in_bom yes) (on_board yes) (dnp no) (fields_autoplaced)
-    (property "Reference" "C20" (at 185.166 90.805 90)
-      (effects (font (size 1.27 1.27)))
-    )
-    (property "Value" "47" (at 185.166 93.345 90)
-      (effects (font (size 1.27 1.27)))
-    )
-    (property "Footprint" "Capacitor_SMD:C_1206_3216Metric" (at 189.865 96.8248 0)
-      (effects (font (size 1.27 1.27)) hide)
-    )
-    (property "Datasheet" "~" (at 186.055 97.79 0)
-      (effects (font (size 1.27 1.27)) hide)
-    )
+  (symbol (lib_id "Device:C_Polarized") (at 185.42 97.79 90) (unit 1)
+    (in_bom yes) (on_board yes) (dnp no) (fields_autoplaced)
+    (property "Reference" "C20" (at 184.531 90.805 90)
+      (effects (font (size 1.27 1.27)))
+    )
+    (property "Value" "47" (at 184.531 93.345 90)
+      (effects (font (size 1.27 1.27)))
+    )
+    (property "Footprint" "Capacitor_SMD:C_1206_3216Metric" (at 189.23 96.8248 0)
+      (effects (font (size 1.27 1.27)) hide)
+    )
+    (property "Datasheet" "~" (at 185.42 97.79 0)
+      (effects (font (size 1.27 1.27)) hide)
+    )

Commit message: Updated Penguin project
Parts:
- C20, C21: footprint Capacitor_SMD:C_1206_3216Metric -> Capacitor_Tantalum_SMD:CP_EIA-3216-12_Kemet-S
Changed lines of the file:
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@@
       (effects (font (size 1.27 1.27)))
     )
-    (property "Footprint" "Capacitor_SMD:C_1206_3216Metric" (at 189.23 103.1748 0)
+    (property "Footprint" "Capacitor_Tantalum_SMD:CP_EIA-3216-12_Kemet-S" (at 189.23 103.1748 0)
       (effects (font (size 1.27 1.27)) hide)
     )
@@
   (symbol (lib_id "power:GND") (at 226.06 87.63 0) (unit 1)
     (in_bom yes) (on_board yes) (dnp no)
-    (property "Reference" "#PWR012" (at 226.06 93.98 0)
+    (property "Reference" "#PWR011" (at 226.06 93.98 0)
       (effects (font (size 1.27 1.27)) hide)
     )
@@
       (project "Penguin Junior"
         (path "/dfff5ef9-3e3a-4442-aa32-5f49584e77ca/48ae4edb-0e13-4619-bf0c-b661f0a0817d"
-          (reference "#PWR012") (unit 1)
+          (reference "#PWR011") (unit 1)
         )
       )
@@
   (symbol (lib_id "power:GND") (at 191.135 121.92 0) (unit 1)
     (in_bom yes) (on_board yes) (dnp no) (fields_autoplaced)
-    (property "Reference" "#PWR014" (at 191.135 128.27 0)
+    (property "Reference" "#PWR013" (at 191.135 128.27 0)
       (effects (font (size 1.27 1.27)) hide)
     )
@@
       (project "Penguin Junior"
         (path "/dfff5ef9-3e3a-4442-aa32-5f49584e77ca/48ae4edb-0e13-4619-bf0c-b661f0a0817d"
-          (reference "#PWR014") (unit 1)
+          (reference "#PWR013") (unit 1)
         )
       )
@@
       (effects (font (size 1.27 1.27)))
     )
-    (property "Footprint" "Capacitor_SMD:C_1206_3216Metric" (at 189.23 96.8248 0)
+    (property "Footprint" "Capacitor_Tantalum_SMD:CP_EIA-3216-12_Kemet-S" (at 189.23 96.8248 0)
       (effects (font (size 1.27 1.27)) hide)
     )
@@
   (symbol (lib_id "power:GND") (at 153.035 125.73 0) (unit 1)
     (in_bom yes) (on_board yes) (dnp no) (fields_autoplaced)
-    (property "Reference" "#PWR015" (at 153.035 132.08 0)
+    (property "Reference" "#PWR014" (at 153.035 132.08 0)
       (effects (font (size 1.27 1.27)) hide)
     )
@@
       (project "Penguin Junior"
         (path "/dfff5ef9-3e3a-4442-aa32-5f49584e77ca/48ae4edb-0e13-4619-bf0c-b661f0a0817d"
-          (reference "#PWR015") (unit 1)
+          (reference "#PWR014") (unit 1)
         )
       )
@@
   (symbol (lib_id "power:GND") (at 118.745 94.615 0) (unit 1)
     (in_bom yes) (on_board yes) (dnp no) (fields_autoplaced)
-    (property "Reference" "#PWR013" (at 118.745 100.965 0)
+    (property "Reference" "#PWR012" (at 118.745 100.965 0)
       (effects (font (size 1.27 1.27)) hide)
     )
@@
       (project "Penguin Junior"
         (path "/dfff5ef9-3e3a-4442-aa32-5f49584e77ca/48ae4edb-0e13-4619-bf0c-b661f0a0817d"
-          (reference "#PWR013") (unit 1)
-        )
-      )
+          (reference "#PWR012") (unit 1)
+        )
+      )

Commit message: Penguin Junior 1.1 release
Other:
- moved on the sheet: C17, C18, C19, C20, C21, C22, Q1, R6, R7, R8, R9, U4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

Commit message: Updated KiCad version
Parts:
- renumbered Y1 to Y2

Commit message: Penguin Junior 1.2 production
Parts:
- renumbered C17 to C18, C18 to C19, C19 to C20, C20 to C21, C21 to C22, C22 to C23, R6 to R11, R7 to R12, R8 to R13, R9 to R14
Changed lines of the file:
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@@
 		(on_board yes)
 		(dnp no)
-		(property "Reference" "C21"
+		(property "Reference" "C22"
 			(at 163.83 99.06 90)
 			(effects
@@
 			(project "Penguin Junior"
 				(path "/dfff5ef9-3e3a-4442-aa32-5f49584e77ca/48ae4edb-0e13-4619-bf0c-b661f0a0817d"
-					(reference "C21")
+					(reference "C22")
 					(unit 1)
 				)
@@
 		(on_board yes)
 		(dnp no)
-		(property "Reference" "#PWR011"
+		(property "Reference" "#PWR014"
 			(at 215.9 86.995 0)
 			(effects
@@
 			(project "Penguin Junior"
 				(path "/dfff5ef9-3e3a-4442-aa32-5f49584e77ca/48ae4edb-0e13-4619-bf0c-b661f0a0817d"
-					(reference "#PWR011")
+					(reference "#PWR014")
 					(unit 1)
 				)
@@
 		(on_board yes)
 		(dnp no)
-		(property "Reference" "R9"
+		(property "Reference" "R14"
 			(at 163.83 113.03 0)
 			(effects
@@
 			(project "Penguin Junior"
 				(path "/dfff5ef9-3e3a-4442-aa32-5f49584e77ca/48ae4edb-0e13-4619-bf0c-b661f0a0817d"
-					(reference "R9")
+					(reference "R14")
 					(unit 1)
 				)
@@
 		(dnp no)
 		(fields_autoplaced yes)
-		(property "Reference" "C17"
+		(property "Reference" "C18"
 			(at 219.71 71.12 0)
 			(effects
@@
 			(project "Penguin Junior"
 				(path "/dfff5ef9-3e3a-4442-aa32-5f49584e77ca/48ae4edb-0e13-4619-bf0c-b661f0a0817d"
-					(reference "C17")
+					(reference "C18")
 					(unit 1)
 				)
@@
 		(dnp no)
 		(fields_autoplaced yes)
-		(property "Reference" "C18"
+		(property "Reference" "C19"
 			(at 231.14 71.12 0)
 			(effects
@@
 			(project "Penguin Junior"
 				(path "/dfff5ef9-3e3a-4442-aa32-5f49584e77ca/48ae4edb-0e13-4619-bf0c-b661f0a0817d"
-					(reference "C18")
+					(reference "C19")
 					(unit 1)
 				)
@@
 		(dnp no)
 		(fields_autoplaced yes)
-		(property "Reference" "R6"
+		(property "Reference" "R11"
 			(at 179.705 89.535 90)
 			(effects
@@
 			(project "Penguin Junior"
 				(path "/dfff5ef9-3e3a-4442-aa32-5f49584e77ca/48ae4edb-0e13-4619-bf0c-b661f0a0817d"
-					(reference "R6")
+					(reference "R11")
 					(unit 1)
 				)
@@
 		(on_board yes)
 		(dnp no)
-		(property "Reference" "C22"
+		(property "Reference" "C23"
 			(at 151.13 113.665 90)
 			(effects
@@
 			(project "Penguin Junior"
 				(path "/dfff5ef9-3e3a-4442-aa32-5f49584e77ca/48ae4edb-0e13-4619-bf0c-b661f0a0817d"
-					(reference "C22")
+					(reference "C23")
 					(unit 1)
 				)
@@
 		(dnp no)
 		(fields_autoplaced yes)
-		(property "Reference" "R7"
+		(property "Reference" "R12"
 			(at 57.15 95.885 0)
 			(effects
@@
 			(project "Penguin Junior"
 				(path "/dfff5ef9-3e3a-4442-aa32-5f49584e77ca/48ae4edb-0e13-4619-bf0c-b661f0a0817d"
-					(reference "R7")
+					(reference "R12")
 					(unit 1)
 				)
@@
 		(dnp no)
 		(fields_autoplaced yes)
-		(property "Reference" "#PWR013"
+		(property "Reference" "#PWR016"
 			(at 165.735 125.73 0)
 			(effects
@@
 			(project "Penguin Junior"
 				(path "/dfff5ef9-3e3a-4442-aa32-5f49584e77ca/48ae4edb-0e13-4619-bf0c-b661f0a0817d"
-					(reference "#PWR013")
+					(reference "#PWR016")
 					(unit 1)
 				)
@@
 		(dnp no)
 		(fields_autoplaced yes)
-		(property "Reference" "C19"
+		(property "Reference" "C20"
 			(at 242.57 71.12 0)
 			(effects
@@
 			(project "Penguin Junior"
 				(path "/dfff5ef9-3e3a-4442-aa32-5f49584e77ca/48ae4edb-0e13-4619-bf0c-b661f0a0817d"
-					(reference "C19")
+					(reference "C20")
 					(unit 1)
 				)
@@
 		(dnp no)
 		(fields_autoplaced yes)
-		(property "Reference" "C20"
+		(property "Reference" "C21"
 			(at 159.131 88.265 90)
 			(effects
@@
 			(project "Penguin Junior"
 				(path "/dfff5ef9-3e3a-4442-aa32-5f49584e77ca/48ae4edb-0e13-4619-bf0c-b661f0a0817d"
-					(reference "C20")
+					(reference "C21")
 					(unit 1)
 				)
@@
 		(dnp no)
 		(fields_autoplaced yes)
-		(property "Reference" "R8"
+		(property "Reference" "R13"
 			(at 75.565 95.885 0)
 			(effects
@@
 			(project "Penguin Junior"
 				(path "/dfff5ef9-3e3a-4442-aa32-5f49584e77ca/48ae4edb-0e13-4619-bf0c-b661f0a0817d"
-					(reference "R8")
+					(reference "R13")
 					(unit 1)
 				)
@@
 		(dnp no)
 		(fields_autoplaced yes)
-		(property "Reference" "#PWR014"
+		(property "Reference" "#PWR017"
 			(at 127.635 129.54 0)
 			(effects
@@
 			(project "Penguin Junior"
 				(path "/dfff5ef9-3e3a-4442-aa32-5f49584e77ca/48ae4edb-0e13-4619-bf0c-b661f0a0817d"
-					(reference "#PWR014")
+					(reference "#PWR017")
 					(unit 1)
 				)
@@
 		(dnp no)
 		(fields_autoplaced yes)
-		(property "Reference" "#PWR012"
+		(property "Reference" "#PWR015"
 			(at 93.345 98.425 0)
 			(effects
@@
 			(project "Penguin Junior"
 				(path "/dfff5ef9-3e3a-4442-aa32-5f49584e77ca/48ae4edb-0e13-4619-bf0c-b661f0a0817d"
-					(reference "#PWR012")
-					(unit 1)
-				)
+					(reference "#PWR015")
+					(unit 1)
+				)
