File: Hardware/Penguin Junior/Sensors.kicad_sch (KiCad schematic)
At the start: 5 parts, among them U2 MS5611-01BA, U3 BMI088

Commit message: Updated project
Parts:
- C14, C15, C16: footprint Capacitor_SMD:C_0603_1608Metric -> Capacitor_SMD:C_0402_1005Metric
- U2: footprint Package_LGA:LGA-8_3x5mm_P1.25mm -> user_lib:LGA-8_3x5mm_P1.25mm_handsolder
Changed lines of the file:
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@@
       (effects (font (size 1.27 1.27)))
     )
-    (property "Footprint" "Capacitor_SMD:C_0603_1608Metric" (at 208.28 89.8398 0)
+    (property "Footprint" "Capacitor_SMD:C_0402_1005Metric" (at 208.28 89.8398 0)
       (effects (font (size 1.27 1.27)) hide)
     )
@@
       (effects (font (size 1.27 1.27)))
     )
-    (property "Footprint" "Capacitor_SMD:C_0603_1608Metric" (at 218.44 89.8398 0)
+    (property "Footprint" "Capacitor_SMD:C_0402_1005Metric" (at 218.44 89.8398 0)
       (effects (font (size 1.27 1.27)) hide)
     )
@@
       (effects (font (size 1.27 1.27)) (justify left))
     )
-    (property "Footprint" "Capacitor_SMD:C_0603_1608Metric" (at 205.4352 43.815 0)
+    (property "Footprint" "Capacitor_SMD:C_0402_1005Metric" (at 205.4352 43.815 0)
       (effects (font (size 1.27 1.27)) hide)
     )
@@
       (effects (font (size 1.27 1.27)) (justify left))
     )
-    (property "Footprint" "Package_LGA:LGA-8_3x5mm_P1.25mm" (at 189.865 40.005 0)
+    (property "Footprint" "user_lib:LGA-8_3x5mm_P1.25mm_handsolder" (at 189.865 40.005 0)
       (effects (font (size 1.27 1.27)) hide)
     )

Commit message: Penguin Junior 1.1 release
Parts:
- removed U2: MS5611-01BA, user_lib:LGA-8_3x5mm_P1.25mm_handsolder, symbol Sensor_Pressure:MS5611-01BA
- added C35: 100n, Capacitor_SMD:C_0402_1005Metric, symbol Device:C
- added U2: BMP388, user_lib:LGA-10_2x2x0.75mm, symbol user_lib:BMP388
Connections:
- net GND: now also C14.1, C35.2, U2.3 (VSS), U2.8 (VSS), U2.9 (VSS); no longer C14.2
- net SPI1_CLK: now also U2.2 (SCK)
- net SPI1_MISO: now also U3.10 (SDO2), U3.15 (SDO1), U2.5 (SDO); no longer U3.9 (SDA/SDI)
- net SPI1_MOSI: now also U3.9 (SDA/SDI), U2.4 (SDI); no longer U3.10 (SDO2), U3.15 (SDO1)
- net SPI1_MS5611_CS: now also U2.6 (CSB)
- net VDD_3V3: now also C14.2, C35.1, U2.1 (VDDIO), U2.10 (VDD); no longer C14.1
- no-connect marks 0 -> 1
Other:
- moved on the sheet: C15, C16, U3

Commit message: Penguin Junior 1.2 production
Parts:
- renumbered C15 to C14, C16 to C15, C14 to C16, C35 to C17, U3 to U2, U2 to U3
Changed lines of the file:
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@@
 		(on_board yes)
 		(dnp no)
-		(property "Reference" "U3"
+		(property "Reference" "U2"
 			(at 96.1741 81.915 0)
 			(effects
@@
 			(project "Penguin Junior"
 				(path "/dfff5ef9-3e3a-4442-aa32-5f49584e77ca/a70a2c87-1506-4cd3-8dac-29ef9684c58b"
-					(reference "U3")
+					(reference "U2")
 					(unit 1)
 				)
@@
 		(dnp no)
 		(fields_autoplaced yes)
-		(property "Reference" "C14"
+		(property "Reference" "C16"
 			(at 191.008 81.661 90)
 			(effects
@@
 			(project "Penguin Junior"
 				(path "/dfff5ef9-3e3a-4442-aa32-5f49584e77ca/a70a2c87-1506-4cd3-8dac-29ef9684c58b"
-					(reference "C14")
+					(reference "C16")
 					(unit 1)
 				)
@@
 		(dnp no)
 		(fields_autoplaced yes)
-		(property "Reference" "C35"
+		(property "Reference" "C17"
 			(at 211.836 81.661 90)
 			(effects
@@
 			(project "Penguin Junior"
 				(path "/dfff5ef9-3e3a-4442-aa32-5f49584e77ca/a70a2c87-1506-4cd3-8dac-29ef9684c58b"
-					(reference "C35")
+					(reference "C17")
 					(unit 1)
 				)
@@
 		(on_board yes)
 		(dnp no)
-		(property "Reference" "#PWR036"
+		(property "Reference" "#PWR010"
 			(at 219.71 97.282 0)
 			(effects
@@
 			(project "Penguin Junior"
 				(path "/dfff5ef9-3e3a-4442-aa32-5f49584e77ca/a70a2c87-1506-4cd3-8dac-29ef9684c58b"
-					(reference "#PWR036")
+					(reference "#PWR010")
 					(unit 1)
 				)
@@
 		(on_board yes)
 		(dnp no)
-		(property "Reference" "U2"
+		(property "Reference" "U3"
 			(at 206.248 92.202 0)
 			(effects
@@
 			(project "Penguin Junior"
 				(path "/dfff5ef9-3e3a-4442-aa32-5f49584e77ca/a70a2c87-1506-4cd3-8dac-29ef9684c58b"
-					(reference "U2")
+					(reference "U3")
 					(unit 1)
 				)
@@
 		(dnp no)
 		(fields_autoplaced yes)
-		(property "Reference" "C15"
+		(property "Reference" "C14"
 			(at 87.63 71.755 90)
 			(effects
@@
 			(project "Penguin Junior"
 				(path "/dfff5ef9-3e3a-4442-aa32-5f49584e77ca/a70a2c87-1506-4cd3-8dac-29ef9684c58b"
-					(reference "C15")
+					(reference "C14")
 					(unit 1)
 				)
@@
 		(on_board yes)
 		(dnp no)
-		(property "Reference" "#PWR037"
+		(property "Reference" "#PWR09"
 			(at 185.928 96.774 0)
 			(effects
@@
 			(project "Penguin Junior"
 				(path "/dfff5ef9-3e3a-4442-aa32-5f49584e77ca/a70a2c87-1506-4cd3-8dac-29ef9684c58b"
-					(reference "#PWR037")
+					(reference "#PWR09")
 					(unit 1)
 				)
@@
 		(dnp no)
 		(fields_autoplaced yes)
-		(property "Reference" "#PWR010"
+		(property "Reference" "#PWR013"
 			(at 91.44 129.54 0)
 			(effects
@@
 			(project "Penguin Junior"
 				(path "/dfff5ef9-3e3a-4442-aa32-5f49584e77ca/a70a2c87-1506-4cd3-8dac-29ef9684c58b"
-					(reference "#PWR010")
+					(reference "#PWR013")
 					(unit 1)
 				)
@@
 		(dnp no)
 		(fields_autoplaced yes)
-		(property "Reference" "#PWR09"
+		(property "Reference" "#PWR011"
 			(at 109.22 116.84 0)
 			(effects
@@
 			(project "Penguin Junior"
 				(path "/dfff5ef9-3e3a-4442-aa32-5f49584e77ca/a70a2c87-1506-4cd3-8dac-29ef9684c58b"
-					(reference "#PWR09")
+					(reference "#PWR011")
 					(unit 1)
 				)
@@
 		(dnp no)
 		(fields_autoplaced yes)
-		(property "Reference" "C16"
+		(property "Reference" "C15"
 			(at 97.79 71.755 90)
 			(effects
@@
 			(project "Penguin Junior"
 				(path "/dfff5ef9-3e3a-4442-aa32-5f49584e77ca/a70a2c87-1506-4cd3-8dac-29ef9684c58b"
-					(reference "C16")
+					(reference "C15")
 					(unit 1)
 				)
@@
 		(on_board yes)
 		(dnp no)
-		(property "Reference" "#PWR06"
+		(property "Reference" "#PWR012"
 			(at 199.39 124.968 0)
 			(effects
@@
 			(project "Penguin Junior"
 				(path "/dfff5ef9-3e3a-4442-aa32-5f49584e77ca/a70a2c87-1506-4cd3-8dac-29ef9684c58b"
-					(reference "#PWR06")
-					(unit 1)
-				)
+					(reference "#PWR012")
+					(unit 1)
+				)
