File: Hardware/CAN sensor net/Master board/Master board.kicad_pcb (KiCad board)
At the start: 2 copper layers, 72 parts, among them J1 Micro_SD_Card_Con, J2 USB_B_Micro, J3 Conn_02x05_SWD, J4 XT60, J5 532610671, J6 532610671, J7 DC-005, SW1 SW_Push, SW2 SW_SPDT, U1 STM32F405RGTx, U2 USBLC6-2SC6, U3 ST1S14PHR, U4 LDL1117_3V3, U5 SN65HVD230, U6 SN65HVD230, Y1 16MHz

Commit message: changed xt60 to xt30
Parts:
- J4: footprint Connector_AMASS:AMASS_XT60PW-M_1x02_P7.20mm_Horizontal -> Connector_AMASS:AMASS_XT30PW-M_1x02_P2.50mm_Horizontal
- moved J4 7.86 mm to (106.3, 44.5)
Changed lines of the file:
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@@
 		)
 	)
-	(footprint "Connector_AMASS:AMASS_XT60PW-M_1x02_P7.20mm_Horizontal"
+	(footprint "Connector_AMASS:AMASS_XT30PW-M_1x02_P2.50mm_Horizontal"
 		(layer "F.Cu")
-		(at 100.59 49.88)
-		(descr "Connector XT60 Horizontal PCB Female, https://www.tme.eu/en/Document/9b8d0c5eb7094295f3d3112c214d3ade/XT60PW%20SPEC.pdf")
-		(tags "RC Connector XT60")
+		(at 106.3 44.475)
+		(descr "Connector XT30 Horizontal PCB Male, https://www.tme.eu/en/Document/ce4077e36b79046da520ca73227e15de/XT30PW%20SPEC.pdf")
+		(tags "RC Connector XT30")
 		(property "Reference" "J4"
-			(at 3.6 -17.5 0)
+			(at -2.5 -14.5 0)
 			(layer "F.SilkS")
 			(effects
@@
 		)
 		(property "Value" "XT60"
-			(at 3.6 4 0)
+			(at -2.5 3.5 0)
 			(layer "F.Fab")
 			(effects
@@
 			)
 		)
-		(property "Footprint" "Connector_AMASS:AMASS_XT60PW-M_1x02_P7.20mm_Horizontal"
+		(property "Footprint" "Connector_AMASS:AMASS_XT30PW-M_1x02_P2.50mm_Horizontal"
 			(at 0 0 0)
 			(unlocked yes)
@@
 		(attr through_hole)
 		(fp_line
-			(start -4.26 -16.46)
-			(end -4.26 -2.15)
-			(stroke
-				(width 0.12)
-				(type solid)
-			)
-			(layer "F.SilkS")
-		)
-		(fp_line
-			(start -4.26 -16.46)
-			(end 11.46 -16.46)
-			(stroke
-				(width 0.12)
-				(type solid)
-			)
-			(layer "F.SilkS")
-		)
-		(fp_line
-			(start 2.31 1.96)
-			(end 6.05 1.96)
-			(stroke
-				(width 0.12)
-				(type solid)
-			)
-			(layer "F.SilkS")
-		)
-		(fp_line
-			(start 11.46 -16.46)
-			(end 11.46 -2.15)
+			(start -8.15 -11.11)
+			(end -7.56 -11.11)
+			(stroke
+				(width 0.12)
+				(type solid)
+			)
+			(layer "F.SilkS")
+		)
+		(fp_line
+			(start -8.15 -8.89)
+			(end -7.56 -8.89)
+			(stroke
+				(width 0.12)
+				(type solid)
+			)
+			(layer "F.SilkS")
+		)
+		(fp_line
+			(start -7.56 -13.21)
+			(end -7.56 -11.11)
+			(stroke
+				(width 0.12)
+				(type solid)
+			)
+			(layer "F.SilkS")
+		)
+		(fp_line
+			(start -7.56 -13.21)
+			(end 2.56 -13.21)
+			(stroke
+				(width 0.12)
+				(type solid)
+			)
+			(layer "F.SilkS")
+		)
+		(fp_line
+			(start -7.56 -8.89)
+			(end -7.56 -3.99)
+			(stroke
+				(width 0.12)
+				(type solid)
+			)
+			(layer "F.SilkS")
+		)
+		(fp_line
+			(start -7.56 -3.99)
+			(end 2.56 -3.99)
+			(stroke
+				(width 0.12)
+				(type solid)
+			)
+			(layer "F.SilkS")
+		)
+		(fp_line
+			(start 2.56 -13.21)
+			(end 2.56 -11.11)
+			(stroke
+				(width 0.12)
+				(type solid)
+			)
+			(layer "F.SilkS")
+		)
+		(fp_line
+			(start 2.56 -11.11)
+			(end 3.15 -11.11)
+			(stroke
+				(width 0.12)
+				(type solid)
+			)
+			(layer "F.SilkS")
+		)
+		(fp_line
+			(start 2.56 -8.89)
+			(end 2.56 -3.99)
+			(stroke
+				(width 0.12)
+				(type solid)
+			)
+			(layer "F.SilkS")
+		)
+		(fp_line
+			(start 2.56 -8.89)
+			(end 3.15 -8.89)
 			(stroke
 				(width 0.12)
@@
 		)
 		(fp_arc
-			(start -2.266806 1.372958)
-			(mid -3.727162 -0.126139)
-			(end -4.26 -2.15)
+			(start -8.15 -8.89)
+			(mid -9.26 -10)
+			(end -8.15 -11.11)
 			(stroke
 				(width 0.12)
@@
 		)
 		(fp_arc
-			(start 11.46 -2.15)
-			(mid 10.653852 0.294722)
-			(end 8.551648 1.780413)
-			(stroke
-				(width 0.12)
-				(type solid)
-			)
-			(layer "F.SilkS")
-		)
-		(fp_line
-			(start -4.65 -16.85)
-			(end -4.65 2.55)
+			(start 3.15 -11.11)
+			(mid 4.26 -10)
+			(end 3.15 -8.89)
+			(stroke
+				(width 0.12)
+				(type solid)
+			)
+			(layer "F.SilkS")
+		)
+		(fp_line
+			(start -9.65 -13.6)
+			(end -9.65 2.25)
 			(stroke
 				(width 0.05)
@@
 		)
 		(fp_line
-			(start -4.65 -16.85)
-			(end 11.85 -16.85)
+			(start -9.65 -13.6)
+			(end 4.65 -13.6)
 			(stroke
 				(width 0.05)
@@
 		)
 		(fp_line
-			(start 11.85 -16.85)
-			(end 11.85 2.55)
+			(start -9.65 2.25)
+			(end 4.65 2.25)
 			(stroke
 				(width 0.05)
@@
 		)
 		(fp_line
-			(start 11.85 2.55)
-			(end -4.65 2.55)
+			(start 4.65 -13.6)
+			(end 4.65 2.25)
 			(stroke
 				(width 0.05)
@@
 		)
 		(fp_line
-			(start -4.15 -16.35)
-			(end -4.15 -2.15)
-			(stroke
-				(width 0.1)
-				(type solid)
-			)
-			(layer "F.Fab")
-		)
-		(fp_line
-			(start -4.15 -16.35)
-			(end 11.35 -16.35)
-			(stroke
-				(width 0.1)
-				(type solid)
-			)
-			(layer "F.Fab")
-		)
-		(fp_line
-			(start -0.15 1.85)
-			(end 7.35 1.85)
-			(stroke
-				(width 0.1)
-				(type solid)
-			)
-			(layer "F.Fab")
-		)
-		(fp_line
-			(start 11.35 -16.35)
-			(end 11.35 -2.15)
+			(start -8.15 -11)
+			(end -7.45 -11)
+			(stroke
+				(width 0.1)
+				(type solid)
+			)
+			(layer "F.Fab")
+		)
+		(fp_line
+			(start -8.15 -9)
+			(end -7.45 -9)
+			(stroke
+				(width 0.1)
+				(type solid)
+			)
+			(layer "F.Fab")
+		)
+		(fp_line
+			(start -7.45 -13.1)
+			(end -7.45 -11)
+			(stroke
+				(width 0.1)
+				(type solid)
+			)
+			(layer "F.Fab")
+		)
+		(fp_line
+			(start -7.45 -13.1)
+			(end 2.45 -13.1)
+			(stroke
+				(width 0.1)
+				(type solid)
+			)
+			(layer "F.Fab")
+		)
+		(fp_line
+			(start -7.45 -9)
+			(end -7.45 -4.1)
+			(stroke
+				(width 0.1)
+				(type solid)
+			)
+			(layer "F.Fab")
+		)
+		(fp_line
+			(start -7.45 -4.1)
+			(end 2.45 -4.1)
+			(stroke
+				(width 0.1)
+				(type solid)
+			)
+			(layer "F.Fab")
+		)
+		(fp_line
+			(start 2.45 -13.1)
+			(end 2.45 -11)
+			(stroke
+				(width 0.1)
+				(type solid)
+			)
+			(layer "F.Fab")
+		)
+		(fp_line
+			(start 2.45 -11)
+			(end 3.15 -11)
+			(stroke
+				(width 0.1)
+				(type solid)
+			)
+			(layer "F.Fab")
+		)
+		(fp_line
+			(start 2.45 -9)
+			(end 2.45 -4.1)
+			(stroke
+				(width 0.1)
+				(type solid)
+			)
+			(layer "F.Fab")
+		)
+		(fp_line
+			(start 2.45 -9)
+			(end 3.15 -9)
 			(stroke
 				(width 0.1)
@@
 		)
 		(fp_arc
-			(start -0.15 1.85)
-			(mid -2.978427 0.678427)
-			(end -4.15 -2.15)
+			(start -8.15 -9)
+			(mid -9.15 -10)
+			(end -8.15 -11)
 			(stroke
 				(width 0.1)
@@
 		)
 		(fp_arc
-			(start 11.35 -2.15)
-			(mid 10.178427 0.678427)
-			(end 7.35 1.85)
+			(start 3.15 -11)
+			(mid 4.15 -10)
+			(end 3.15 -9)
 			(stroke
 				(width 0.1)
@@
 		)
 		(fp_text user "+"
-			(at 9.5 2.5 0)
+			(at -8 0 0)
 			(layer "F.SilkS")
 			(effects
@@
 		)
 		(fp_text user "-"
-			(at -2.8 2.5 0)
+			(at 3 0 0)
 			(layer "F.SilkS")
 			(effects
@@
 		)
 		(fp_text user "${REFERENCE}"
-			(at 3.6 -3.6 0)
+			(at -2.5 -3 0)
 			(layer "F.Fab")
 			(effects
@@
 			)
 		)
-		(pad "" thru_hole rect
-			(at -3.15 -6)
-			(size 0.9 2)
-			(drill oval 0.6 1.7)
+		(pad "" thru_hole circle
+			(at -8 -10)
+			(size 1.4 1.4)
+			(drill 1)
 			(layers "*.Cu" "*.Mask")
 			(remove_unused_layers no)
 		)
-		(pad "" thru_hole rect
-			(at 10.35 -6)
-			(size 0.9 2)
-			(drill oval 0.6 1.7)
+		(pad "" thru_hole circle
+			(at 3 -10)
+			(size 1.4 1.4)
+			(drill 1)
 			(layers "*.Cu" "*.Mask")
 			(remove_unused_layers no)
 		)
-		(pad "1" thru_hole roundrect
+		(pad "1" thru_hole rect
 			(at 0 0)
-			(size 4.1 4.1)
-			(drill 2.7)
+			(size 3.5 3.5)
+			(drill 1.9)
 			(layers "*.Cu" "*.Mask")
 			(remove_unused_layers no)
-			(roundrect_rratio 0.25)
 			(net 1 "GND")
 			(pinfunction "Pin_1")
@@
 		)
 		(pad "2" thru_hole circle
-			(at 7.2 0)
-			(size 4.1 4.1)
-			(drill 2.7)
+			(at -5 0)
+			(size 3.5 3.5)
+			(drill 1.9)
 			(layers "*.Cu" "*.Mask")
 			(remove_unused_layers no)
@@
 			(pintype "passive")
 		)
-		(model "${KICAD8_3DMODEL_DIR}/Connector_AMASS.3dshapes/AMASS_XT60PW-M_1x02_P7.20mm_Horizontal.wrl"
+		(model "${KICAD8_3DMODEL_DIR}/Connector_AMASS.3dshapes/AMASS_XT30PW-M_1x02_P2.50mm_Horizontal.wrl"
 			(offset
 				(xyz 0 0 0)
@@
 			)
 		)
-		(model "${KIPRJMOD}/packages3D/XT60PW-M--3DModel-STEP-269445.STEP"
+		(model "${KIPRJMOD}/packages3D/XT30PW-M--3DModel-STEP-1.STEP"
 			(offset
-				(xyz 3.5 6 0)
+				(xyz -2.5 10 0)
 			)
 			(scale

Commit message: Master board сoncept
Parts:
- removed J7: DC-005, Connector_BarrelJack:BarrelJack_Horizontal
- removed JP2: Jumper_2_Bridged, Connector_PinHeader_2.54mm:PinHeader_1x02_P2.54mm_Vertical
- added D7: LED, LED_SMD:LED_1206_3216Metric, F.Cu at (213.1, 90.0)
- added R20: 220, Resistor_SMD:R_0603_1608Metric, F.Cu at (164.5, 89.3)
- C1, C10, C11, C12, C13, C16, C2, C21, C22, C23, C24, C3, C4, C5, C6, C7, C8, C9: footprint Capacitor_SMD:C_0402_1005Metric -> Capacitor_SMD:C_0603_1608Metric
- C17, D2, J1, JP1, U3, U4: moved to B.Cu
- C18: footprint Capacitor_SMD:C_0805_2012Metric -> Capacitor_SMD:C_0603_1608Metric
- R12: footprint Resistor_SMD:R_0402_1005Metric -> Resistor_SMD:R_0603_1608Metric
- moved J2 130.6 mm to (195.8, 110.2), turned to 180 degrees
- moved J1 121.4 mm to (186.6, 88.9), turned to -90 degrees
- moved J3 118.0 mm to (186.3, 104.1), turned to 90 degrees
- moved U2 117.1 mm to (196.0, 103.7), turned to -90 degrees
- moved J4 116.4 mm to (203.8, 108.1), turned to -90 degrees
- moved U4 113.6 mm to (206.7, 97.1), turned to -90 degrees
- moved U3 110.8 mm to (213.3, 105.5), turned to -90 degrees
- moved J6 110.0 mm to (173.3, 105.8), turned to -90 degrees
- moved JP1 108.6 mm to (186.6, 106.9), turned to 180 degrees
- moved J5 107.5 mm to (173.2, 91.4), turned to -90 degrees
- moved C19 105.7 mm to (213.1, 96.4), turned to 90 degrees
- moved D2 102.0 mm to (213.4, 89.1), turned to -90 degrees
- moved L1 100.3 mm to (206.9, 88.5)
- moved C17 99.0 mm to (207.6, 105.6), turned to 90 degrees
- moved U1 96.7 mm to (196.2, 94.9)
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Connections:
- C22 pad 1: Net-(JP2-A) -> VDD_3V3
- U4 pad 2: Net-(JP2-A) -> VDD_3V3
Routing:
- net Net-(D1-RK): vias 0 -> 1
- net Net-(D1-GK): vias 0 -> 1
- net Net-(D1-BK): vias 0 -> 1
Other:
- board outline added: 47.2 x 28.9 mm

Commit message: minor fixes
Parts:
- added C25: 100n, Capacitor_SMD:C_0603_1608Metric, F.Cu at (93.6, 65.1)
- added U7: W25Q32FVSSIG, Package_SO:SOIC-8_5.23x5.23mm_P1.27mm, F.Cu at (96.8, 60.5)
- R12: value 47K -> 47k
- R13: value 10K -> 10k
- R14, R15: value 1K -> 1k

Commit message: Bugfix
Parts:
- C17, D2, U3, U4: moved to F.Cu
- U1, U5, U6: moved to B.Cu
- moved C14 166.8 mm to (228.0, 132.3)
- moved R4 166.8 mm to (228.0, 137.4)
- moved R5 166.8 mm to (228.0, 139.9)
- moved R6 166.8 mm to (228.0, 142.4)
- moved R7 166.8 mm to (232.0, 132.3)
- moved R8 166.8 mm to (232.0, 134.8)
- moved R9 166.8 mm to (232.0, 137.4)
- moved R1 101.0 mm to (188.1, 130.7)
- moved R19 101.0 mm to (192.1, 133.2)
- moved R2 101.0 mm to (188.1, 133.2)
- moved R21 101.0 mm to (192.1, 135.7)
- moved R22 101.0 mm to (192.1, 138.3)
- moved R23 101.0 mm to (192.1, 140.8)
- moved R3 101.0 mm to (188.1, 135.7)
- moved R18 100.5 mm to (204.5, 112.0)
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Routing:
- net Net-(D5-K): vias 0 -> 1
- net Net-(D1-RK): vias 1 -> 0
- net Net-(D1-GK): vias 1 -> 0
- net Net-(D1-BK): vias 1 -> 0
Other:
- board text added: "led"
- board text added: "разъём программатора юарт??"

Commit message: Added UART port
Parts:
- added J7: 530470310, Connector_Molex:Molex_PicoBlade_53047-0310_1x03_P1.25mm_Vertical, F.Cu at (69.2, 134.0)
- added JP2: SolderJumper_2_Open, Jumper:SolderJumper-2_P1.3mm_Open_RoundedPad1.0x1.5mm, F.Cu at (68.9, 123.6)
- added JP3: SolderJumper_2_Open, Jumper:SolderJumper-2_P1.3mm_Open_RoundedPad1.0x1.5mm, F.Cu at (68.9, 127.2)
- added R24: 10k, Resistor_SMD:R_0603_1608Metric, F.Cu at (127.2, 94.5)
- C20: footprint Capacitor_SMD:C_0402_1005Metric -> Capacitor_SMD:C_0603_1608Metric
- R10, R11, R4, R5, R6, R7, R8, R9: value 100k -> 10k
- U2: moved to B.Cu
- moved J1 181.6 mm to (29.6, 115.5), turned to 0 degrees
- moved C24 136.3 mm to (252.5, 96.2)
- moved C23 136.1 mm to (252.7, 89.2)
- moved J6 119.2 mm to (58.7, 138.8)
- moved J5 119.2 mm to (58.7, 124.3)
- moved R5 116.0 mm to (121.2, 94.5)
- moved R6 116.0 mm to (121.2, 97.0)
- moved R7 115.6 mm to (121.2, 99.5)
- moved R8 115.6 mm to (121.2, 102.1)
- moved R9 115.6 mm to (121.2, 104.6)
- moved C14 105.7 mm to (127.7, 98.8)
- moved R4 105.7 mm to (127.7, 103.8)
- moved R16 64.1 mm to (73.0, 123.1)
- moved R17 64.1 mm to (73.0, 125.6)
- moved U5 30.1 mm to (210.6, 88.9)
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Connections:
- net LED1 renamed LED3
- net LED2 renamed LED4
- R10 pad 1: VDD_5V_USB -> VBUS_DETECT
- R10 pad 2: VBUS_DETECT -> GND
- R11 pad 1: VBUS_DETECT -> VDD_5V_USB
- R11 pad 2: GND -> VBUS_DETECT
- R16 pad 2: CAN0_L -> Net-(JP2-B)
- R17 pad 2: CAN1_L -> Net-(JP3-B)
- SW2 pad 2: BOOT0 -> Net-(SW2-B)
- U2 pad 5: VDD_5V_VBUS -> VDD_5V_USB
Routing:
- net USB_D+: track 0.00 -> 2.23 mm
- net USB_D-: track 0.00 -> 2.23 mm
- net Net-(D5-K): vias 1 -> 0
Other:
- board size 47.2 x 28.9 mm -> 161.7 x 61.8 mm
- copper layers 2 -> 4

Commit message: PCB prototype
Parts:
- added F1: RUEF300, user_lib:RUEF300, F.Cu at (76.9, 135.0)
- added H1: MountingHole, MountingHole:MountingHole_2.2mm_M2_Pad_Via, F.Cu at (97.1, 143.4)
- added H2: MountingHole, MountingHole:MountingHole_2.2mm_M2_Pad_Via, F.Cu at (64.8, 119.6)
- added H3: MountingHole, MountingHole:MountingHole_2.2mm_M2_Pad_Via, F.Cu at (64.9, 143.5)
- D3, D4, U4: moved to B.Cu
- JP1: moved to F.Cu
- moved U5 154.2 mm to (59.9, 121.7), turned to 90 degrees
- moved C19 139.1 mm to (77.5, 127.1), turned to 180 degrees
- moved U1 136.3 mm to (67.5, 131.7), turned to 90 degrees
- moved U3 132.0 mm to (72.7, 135.8)
- moved D2 129.1 mm to (92.8, 135.1), turned to 90 degrees
- moved D7 129.0 mm to (80.3, 134.8), turned to 90 degrees
- moved L1 127.3 mm to (91.6, 142.5)
- moved U2 125.9 mm to (71.9, 120.7), turned to 90 degrees
- moved SW1 124.7 mm to (84.7, 143.5), turned to -90 degrees
- moved J2 124.5 mm to (71.7, 119.7), turned to 0 degrees
- moved U7 122.7 mm to (65.4, 131.5)
- moved U6 122.4 mm to (59.0, 141.1), turned to -90 degrees
- moved J3 122.2 mm to (76.7, 142.5)
- moved D5 122.0 mm to (63.7, 124.3), turned to 90 degrees
- moved C17 119.4 mm to (84.4, 134.2)
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Connections:
- C19 pad 1: VDD_7V0 -> Net-(C19-Pad1)
- C20 pad 2: VDD_7V0 -> Net-(C19-Pad1)
- L1 pad 2: VDD_7V0 -> Net-(C19-Pad1)
- R12 pad 2: VDD_7V0 -> Net-(C19-Pad1)
- R13 pad 2: VDD_7V0 -> Net-(C19-Pad1)
Routing:
- net USB_D+: track 2.23 -> 0.00 mm
- net USB_D-: track 2.23 -> 0.00 mm
- net CAN0_L: vias 0 -> 1
- net CAN0_H: vias 0 -> 1
Other:
- board size 161.7 x 61.8 mm -> 44 x 28.9 mm

Commit message: New best debug connector model
Parts:
- added H2: MountingHole, MountingHole:MountingHole_2.2mm_M2_Pad_Via, F.Cu at (194.0, 75.3)
- added H4: MountingHole, MountingHole:MountingHole_2.2mm_M2_Pad_Via, F.Cu at (103.1, 140.2)
- added J5: 532610671, Connector_Molex:Molex_PicoBlade_53261-0671_1x06-1MP_P1.25mm_Horizontal, F.Cu at (148.7, 76.4)
- added J6: 532610671, Connector_Molex:Molex_PicoBlade_53261-0671_1x06-1MP_P1.25mm_Horizontal, F.Cu at (148.7, 90.9)
- moved J1 30.9 mm to (62.6, 129.6), turned to 0 degrees
- moved U7 30.1 mm to (94.5, 123.9)
- moved H1 24.6 mm to (103.1, 119.6)
- moved H3 23.9 mm to (64.8, 119.6)
- moved J4 15.6 mm to (93.4, 140.3)
- moved U1 14.8 mm to (82.1, 129.2)
- moved J3 8.04 mm to (84.7, 141.9)
- moved U6 0.45 mm to (58.6, 140.8)
Other:
- board size 44 x 28.9 mm -> 186.8 x 93.7 mm

Commit message: Concept no trace
Parts:
- removed the H1 at (103.1, 119.6)
- removed the H2 at (194.0, 75.3)
- removed H4: MountingHole, MountingHole:MountingHole_2.2mm_M2_Pad_Via
- added H1: MountingHole, MountingHole:MountingHole_2.2mm_M2_Pad_Via, F.Cu at (70.3, 121.0)
- added H1: MountingHole, MountingHole:MountingHole_2.2mm_M2_Pad_Via, F.Cu at (79.7, 141.8)
- added H1: MountingHole, MountingHole:MountingHole_2.2mm_M2_Pad_Via, F.Cu at (155.2, 89.2)
- added J7: 530470310, Connector_Molex:Molex_PicoBlade_53261-0371_1x03-1MP_P1.25mm_Horizontal, F.Cu at (64.1, 138.7)
- added REF**: Molex_PicoBlade_53261-0271_1x02-1MP_P1.25mm_Horizontal, Connector_Molex:Molex_PicoBlade_53261-0271_1x02-1MP_P1.25mm_Horizontal, F.Cu at (86.0, 138.4)
- J7: footprint Connector_Molex:Molex_PicoBlade_53047-0310_1x03_P1.25mm_Vertical -> Connector_Molex:Molex_PicoBlade_53261-0371_1x03-1MP_P1.25mm_Horizontal
- JP2, JP3, R16, R17, R24: moved to B.Cu
- SW2: footprint user_lib:MSS-12D16 -> Button_Switch_SMD:SW_SPDT_PCM12; moved to B.Cu
- U5, U6: moved to F.Cu
- moved D7 105.0 mm to (161.0, 67.7), turned to 180 degrees
- moved H3 103.8 mm to (155.2, 68.6)
- moved J5 98.0 mm to (64.1, 126.1)
- moved D4 92.6 mm to (157.6, 63.5), turned to 90 degrees
- moved U3 90.4 mm to (140.7, 76.3), turned to 0 degrees
- moved D8 89.5 mm to (150.4, 85.9)
- moved D1 88.2 mm to (150.3, 92.0)
- moved L1 88.0 mm to (142.0, 70.4), turned to 90 degrees
- moved C17 86.2 mm to (147.8, 75.8)
- moved C18 86.1 mm to (145.5, 76.3), turned to 90 degrees
- moved D3 85.6 mm to (155.3, 63.5), turned to 90 degrees
- moved D2 84.9 mm to (147.2, 69.9)
- moved J4 84.7 mm to (151.7, 78.9)
- moved C19 81.7 mm to (136.4, 70.4), turned to 90 degrees
- moved J7 80.5 mm to (162.2, 88.9)
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Connections:
- J5 pad 1: VDD_7V0 -> (no net)
- J5 pad 2: VDD_7V0 -> (no net)
- J5 pad 3: CAN0_H -> (no net)
- J5 pad 4: CAN0_L -> (no net)
- J5 pad 5: GND -> (no net)
- J5 pad 6: GND -> (no net)
- J5 pad 3: CAN0_H -> CAN0_-
- J5 pad 4: CAN0_L -> CAN0_+
- J6 pad 3: CAN1_H -> CAN1_-
- J6 pad 4: CAN1_L -> CAN1_+
- J6 pad 1: VDD_7V0 -> (no net)
- J6 pad 2: VDD_7V0 -> (no net)
- J6 pad 3: CAN1_H -> (no net)
- J6 pad 4: CAN1_L -> (no net)
- J6 pad 5: GND -> (no net)
- J6 pad 6: GND -> (no net)
- JP2 pad 1: CAN0_L -> Net-(JP2-A)
- JP2 pad 2: Net-(JP2-B) -> CAN0_+
- JP3 pad 1: CAN1_L -> CAN1_-
- R16 pad 1: CAN0_H -> CAN0_-
- R16 pad 2: Net-(JP2-B) -> Net-(JP2-A)
- R17 pad 1: CAN1_H -> CAN1_+
- U2 pad 1: USB_D+ -> /Connectors/usb_conn_d-
- U2 pad 3: USB_D- -> /Connectors/usb_conn_d+
- U2 pad 4: /Connectors/usb_conn_d- -> USB_D+
- U2 pad 6: /Connectors/usb_conn_d+ -> USB_D-
- U5 pad 6: CAN0_L -> CAN0_-
- U5 pad 7: CAN0_H -> CAN0_+
- U6 pad 6: CAN1_L -> CAN1_-
- U6 pad 7: CAN1_H -> CAN1_+
Routing:
- net VDD_7V0: track 0.00 -> 47.1 mm, vias 0 -> 4
- net Net-(C19-Pad1): track 0.00 -> 13.5 mm
- net CAN0_-: track 0.00 -> 11.0 mm, vias 0 -> 1
- net CAN1_+: track 0.00 -> 10.9 mm, vias 0 -> 1
- net /Connectors/usb_conn_d-: track 0.00 -> 10.1 mm, vias 0 -> 1
- net /Connectors/usb_conn_d+: track 0.00 -> 9.90 mm, vias 0 -> 1
- net CAN0_+: track 0.00 -> 7.91 mm, vias 0 -> 1
- net CAN1_-: track 0.00 -> 7.79 mm, vias 0 -> 1
- net USB_D+: track 0.00 -> 3.06 mm
- net USB_D-: track 0.00 -> 3.02 mm
- net Net-(JP2-A): track 0.00 -> 1.91 mm
- net Net-(JP3-B): track 0.00 -> 1.91 mm
- net GND: vias 0 -> 4
- net CAN0_L: vias 1 -> 0
- net CAN0_H: vias 1 -> 0
Other:
- board size 186.8 x 93.7 mm -> 193.9 x 117.5 mm
- board text added: "юарт??"
- board text removed: "разъём программатора юарт??"
