File: Hardware/CAN sensor net/Master board/Master board.kicad_pcb (KiCad board)
At the start: 4 copper layers, 193.9 x 117.5 mm, 88 parts, among them J1 Micro_SD_Card_Con, J2 USB_B_Micro, J3 Conn_02x05_SWD, J4 XT60, J5 532610671, J6 532610671, J7 530470310, SW1 SW_Push, SW2 SW_SPDT, U1 STM32F405RGTx, U2 USBLC6-2SC6, U3 ST1S14PHR, U4 LDL1117_3V3, U5 SN65HVD230, U6 SN65HVD230, U7 W25Q32FVSSIG, Y1 16MHz

Commit message: Minor changes
Parts:
- removed the H1 at (70.3, 121.0)
- removed the H1 at (79.7, 141.8)
- removed the J5 at (64.1, 126.1)
- removed the J6 at (85.9, 126.0)
- removed the J7 at (64.1, 138.7)
- removed REF**: Molex_PicoBlade_53261-0271_1x02-1MP_P1.25mm_Horizontal, Connector_Molex:Molex_PicoBlade_53261-0271_1x02-1MP_P1.25mm_Horizontal
- SW2: moved to F.Cu
- moved C25 77.2 mm to (134.3, 104.9), turned to 90 degrees
- moved SW2 28.2 mm to (148.4, 91.4)
- moved JP1 17.2 mm to (87.8, 66.1)
- moved D8 10.4 mm to (140.0, 85.7)
- moved U7 10.2 mm to (130.2, 86.0)
- moved D1 7.59 mm to (145.9, 85.8)
- moved R24 2.55 mm to (122.5, 89.7)
- moved R13 0.15 mm to (134.5, 78.0)
- moved U4 0.10 mm to (130.2, 86.2), turned to -90 degrees
Routing:
- net DEBUG_SWDIO: track 0.00 -> 20.5 mm
- net DEBUG_SWO: track 0.00 -> 16.8 mm
- net DEBUG_SWCLK: track 0.00 -> 13.2 mm
Other:
- board text added: "кто прочитал тот лох"

Commit message: Pre-production
Parts:
- C1, C10, C11, C12, C13, C2, C25, C3, C4, C5, C6, C7, C8, R4, R5, R6, R7, R8, R9, U7, Y1: moved to B.Cu
- D3, D4, R24: moved to F.Cu
- J4: value XT60 -> XT30
- moved C23 133.8 mm to (120.4, 69.6), turned to -90 degrees
- moved C24 130.9 mm to (121.9, 87.6), turned to 90 degrees
- moved R18 97.6 mm to (172.7, 107.2)
- moved C15 80.6 mm to (138.0, 87.6)
- moved C11 74.3 mm to (142.5, 68.8), turned to -90 degrees
- moved R10 74.3 mm to (141.1, 107.7)
- moved C10 73.7 mm to (139.1, 67.5)
- moved R11 73.5 mm to (141.0, 109.4)
- moved R9 72.7 mm to (129.6, 79.9), turned to 90 degrees
- moved R8 71.5 mm to (128.1, 79.9), turned to 90 degrees
- moved C6 70.6 mm to (148.0, 72.1)
- moved R7 70.4 mm to (126.7, 79.9), turned to 90 degrees
- moved R5 69.6 mm to (120.7, 92.1)
- moved Y1 68.0 mm to (139.6, 70.0), turned to 0 degrees
- moved R6 67.3 mm to (119.9, 90.6)
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Connections:
- net CAN0_+ renamed CAN0_H+
- net CAN0_- renamed CAN0_L-
- net CAN1_+ renamed CAN1_H+
- net CAN1_- renamed CAN1_L-
- J7 pad 1: unconnected-(J7-Pin_1-Pad1) -> GND
- J7 pad 2: unconnected-(J7-Pin_2-Pad2) -> UART1_TX
- J7 pad 3: unconnected-(J7-Pin_3-Pad3) -> UART1_RX
- SW2 pad 1: VDD_3V3 -> GND
- SW2 pad 3: GND -> VDD_3V3
- U1 pad 21: unconnected-(U1-PA5-Pad21) -> SPI_CLK
- U1 pad 22: unconnected-(U1-PA6-Pad22) -> SPI_MISO
- U1 pad 23: unconnected-(U1-PA7-Pad23) -> SPI_MOSI
- U1 pad 42: unconnected-(U1-PA9-Pad42) -> UART1_TX
- U1 pad 43: unconnected-(U1-PA10-Pad43) -> UART1_RX
- U1 pad 57: unconnected-(U1-PB5-Pad57) -> CAN1_RX
- U1 pad 58: unconnected-(U1-PB6-Pad58) -> CAN1_TX
- U1 pad 61: unconnected-(U1-PB8-Pad61) -> CAN0_RX
- U1 pad 62: unconnected-(U1-PB9-Pad62) -> CAN0_TX
Routing:
- net SDIO_D0: track 0.00 -> 44.4 mm
- net NRST: track 0.00 -> 41.9 mm
- net SDIO_D1: track 0.00 -> 39.0 mm
- net GND: track 0.00 -> 38.6 mm, vias 4 -> 32
- net VDD_3V3: track 0.00 -> 37.0 mm, vias 0 -> 13
- net CAN1_TX: track 0.00 -> 29.0 mm, vias 0 -> 1
- net CAN1_RX: track 0.00 -> 24.0 mm, vias 0 -> 1
- net UART1_RX: track 0.00 -> 23.8 mm, vias 0 -> 1
- net UART1_TX: track 0.00 -> 23.3 mm, vias 0 -> 1
- net CAN0_RX: track 0.00 -> 22.6 mm, vias 0 -> 1
- net SDIO_CMD: track 0.00 -> 19.1 mm
- net SDIO_D3: track 0.00 -> 18.9 mm
- net BOOT0: track 0.00 -> 18.5 mm, vias 0 -> 1
- net CAN0_TX: track 0.00 -> 17.2 mm, vias 0 -> 1
- net SDIO_CK: track 0.00 -> 14.8 mm, vias 0 -> 2
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- added copper zone on In1.Cu, net GND
- added copper zone on In2.Cu, net GND
- added copper zone on F.Cu, net Net-(C19-Pad1)
- added copper zone on F.Cu, net Net-(D2-K)
- added copper zone on F.Cu, net Net-(D3-K)
- added copper zone on F.Cu, net Net-(J4-Pin_2)
- added copper zone on F.Cu, net Net-(U3-FB)
- added copper zone on B.Cu, net VDD_3V3
Other:
- board size 193.9 x 117.5 mm -> 136.5 x 28.9 mm
- board text added: "SD"
- board text added: "usb 5v0"
- board text added: "подписи светодиодов, коннекторов и пинов UART распиновка boot0 распиновка и подключение flash"
- board text removed: "кто прочитал тот лох"
- board text removed: "юарт??"

Commit message: Minor fixes
Parts:
- moved D1 13.3 mm to (142.4, 85.4)
- moved D8 12.9 mm to (147.5, 85.6)
- moved R24 2.02 mm to (151.2, 87.6)
Routing:
- net BOOT0: track 18.5 -> 6.94 mm
Other:
- board text added: "0"
- board text added: "1"
- board text added: "A"
- board text added: "B"
- board text added: "CAN0"
- board text added: "CAN1"
- board text added: "PWR"
- board text added: "RESET"
- board text added: "UART"
Changed lines of the file:
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@@
 	(footprint "LED_SMD:LED_Cree-PLCC4_3.2x2.8mm_CCW"
 		(layer "F.Cu")
-		(at 140.063 98.46 180)
+		(at 142.433 85.411 180)
 		(descr "3.2mm x 2.8mm PLCC4 RGB LED, https://assets.cree-led.com/a/ds/h/HB-CLV1A-FKB.pdf")
 		(tags "LED Cree PLCC-4 3528 CLV1A-FKB")
@@
 	(footprint "Resistor_SMD:R_0603_1608Metric"
 		(layer "F.Cu")
-		(at 149.232 87.339 -90)
+		(at 151.239 87.604 -90)
 		(descr "Resistor SMD 0603 (1608 Metric), square (rectangular) end terminal, IPC_7351 nominal, (Body size source: IPC-SM-782 page 72, https://www.pcb-3d.com/wordpress/wp-content/uploads/ipc-sm-782a_amendment_1_and_2.pdf), generated with kicad-footprint-generator")
 		(tags "resistor")
@@
 			(at 0 -4.4 90)
 			(layer "F.SilkS")
+			(hide yes)
 			(effects
 				(font
@@
 	(footprint "LED_SMD:LED_Cree-PLCC4_3.2x2.8mm_CCW"
 		(layer "F.Cu")
-		(at 147.033 98.496)
+		(at 147.523 85.584)
 		(descr "3.2mm x 2.8mm PLCC4 RGB LED, https://assets.cree-led.com/a/ds/h/HB-CLV1A-FKB.pdf")
 		(tags "LED Cree PLCC-4 3528 CLV1A-FKB")
@@
 		)
 	)
+	(gr_rect
+		(start 140.101 82.111)
+		(end 144.683 87.339)
+		(stroke
+			(width 0.1)
+			(type default)
+		)
+		(fill none)
+		(layer "F.SilkS")
+	)
+	(gr_rect
+		(start 145.203 82.434)
+		(end 149.831 87.524)
+		(stroke
+			(width 0.1)
+			(type default)
+		)
+		(fill none)
+		(layer "F.SilkS")
+	)
 	(gr_line
 		(start 165.399 67.807)
@@
 		(layer "User.2")
 	)
+	(gr_text "0"
+		(at 145.847 94.805 0)
+		(layer "F.SilkS")
+		(effects
+			(font
+				(size 1 1)
+				(thickness 0.1)
+			)
+			(justify left bottom)
+		)
+	)
+	(gr_text "UART"
+		(at 157.238 93.367 0)
+		(layer "F.SilkS")
+		(effects
+			(font
+				(size 1 1)
+				(thickness 0.1)
+			)
+			(justify left bottom)
+		)
+	)
+	(gr_text "CAN0"
+		(at 115.184 80.234 0)
+		(layer "F.SilkS")
+		(effects
+			(font
+				(size 1 1)
+				(thickness 0.1)
+			)
+			(justify left bottom)
+		)
+	)
+	(gr_text "RESET"
+		(at 114.373 95.134 0)
+		(layer "F.SilkS")
+		(effects
+			(font
+				(size 1 1)
+				(thickness 0.1)
+			)
+			(justify left bottom)
+		)
+	)
+	(gr_text "CAN1"
+		(at 115.165 82.607 0)
+		(layer "F.SilkS")
+		(effects
+			(font
+				(size 1 1)
+				(thickness 0.1)
+			)
+			(justify left bottom)
+		)
+	)
+	(gr_text "B"
+		(at 146.761 83.715 0)
+		(layer "F.SilkS")
+		(effects
+			(font
+				(size 1 1)
+				(thickness 0.1)
+			)
+			(justify left bottom)
+		)
+	)
+	(gr_text "1"
+		(at 149.984 94.771 0)
+		(layer "F.SilkS")
+		(effects
+			(font
+				(size 1 1)
+				(thickness 0.1)
+			)
+			(justify left bottom)
+		)
+	)
+	(gr_text "A"
+		(at 141.81 83.553 0)
+		(layer "F.SilkS")
+		(effects
+			(font
+				(size 1 1)
+				(thickness 0.1)
+			)
+			(justify left bottom)
+		)
+	)
+	(gr_text "PWR"
+		(at 157.304 70.89 0)
+		(layer "F.SilkS")
+		(effects
+			(font
+				(size 1 1)
+				(thickness 0.1)
+			)
+			(justify left bottom)
+		)
+	)
 	(gr_text "SD"
 		(at 122.445 114.492 0)
@@
 		(net 45)
 	)
-	(segment
-		(start 143.758 81.04)
-		(end 139.983 81.04)
-		(width 0.5)
-		(layer "F.Cu")
-		(net 51)
-	)
-	(segment
-		(start 149.232 86.514)
-		(end 143.758 81.04)
-		(width 0.5)
-		(layer "F.Cu")
-		(net 51)
-	)
 	(via

Commit message: Piezo concept (full)
Parts:
- D1, D8: footprint LED_SMD:LED_Cree-PLCC4_3.2x2.8mm_CCW -> LED_SMD:LED_RGB_Wuerth-PLCC4_3.2x2.8mm_150141M173100
- moved D8 0.20 mm to (147.7, 85.5)
Changed lines of the file:
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@@
 			)
 		)
+		(property ki_fp_filters "*Fuse*")
+		(sheetname "Power")
+		(sheetfile "power.kicad_sch")
 		(attr through_hole)
 		(fp_line
@@
 		)
 	)
-	(footprint "LED_SMD:LED_Cree-PLCC4_3.2x2.8mm_CCW"
+	(footprint "LED_SMD:LED_RGB_Wuerth-PLCC4_3.2x2.8mm_150141M173100"
 		(layer "F.Cu")
 		(at 142.433 85.411 180)
-		(descr "3.2mm x 2.8mm PLCC4 RGB LED, https://assets.cree-led.com/a/ds/h/HB-CLV1A-FKB.pdf")
-		(tags "LED Cree PLCC-4 3528 CLV1A-FKB")
+		(descr "3.2mm x 2.8mm PLCC4 LED, https://www.we-online.de/katalog/datasheet/150141M173100.pdf")
+		(tags "LED RGB Wurth PLCC-4 3528")
 		(property "Reference" "D1"
-			(at 0 -2.65 180)
+			(at 0 -2.4 180)
 			(layer "F.SilkS")
 			(hide yes)
@@
 		)
 		(property "Value" "LED_RGBA"
-			(at 0 2.65 180)
+			(at 0 2.5 180)
 			(layer "F.Fab")
 			(effects
@@
 			)
 		)
-		(property "Footprint" "LED_SMD:LED_Cree-PLCC4_3.2x2.8mm_CCW"
+		(property "Footprint" "LED_SMD:LED_RGB_Wuerth-PLCC4_3.2x2.8mm_150141M173100"
 			(at 0 0 180)
 			(unlocked yes)
@@
 		(attr smd)
 		(fp_line
-			(start -1.95 1.5)
-			(end 1.95 1.5)
+			(start -2.3 1.51)
+			(end 2.3 1.51)
 			(stroke
 				(width 0.12)
@@
 		)
 		(fp_line
-			(start -1.95 -0.7)
-			(end -1.95 -1.5)
+			(start -2.5 -0.7)
+			(end -2.5 -1.51)
 			(stroke
 				(width 0.12)
@@
 		)
 		(fp_line
-			(start -1.95 -1.5)
-			(end 1.95 -1.5)
+			(start -2.5 -1.51)
+			(end 2.3 -1.51)
 			(stroke
 				(width 0.12)
@@
 		)
 		(fp_line
-			(start 2.2 1.75)
-			(end 2.2 -1.75)
+			(start 2.55 1.65)
+			(end 2.55 -1.65)
 			(stroke
 				(width 0.05)
@@
 		)
 		(fp_line
-			(start 2.2 -1.75)
-			(end -2.2 -1.75)
+			(start 2.55 -1.65)
+			(end -2.55 -1.65)
 			(stroke
 				(width 0.05)
@@
 		)
 		(fp_line
-			(start -2.2 1.75)
-			(end 2.2 1.75)
+			(start -2.55 1.65)
+			(end 2.55 1.65)
 			(stroke
 				(width 0.05)
@@
 		)
 		(fp_line
-			(start -2.2 -1.75)
-			(end -2.2 1.75)
+			(start -2.55 -1.65)
+			(end -2.55 1.65)
 			(stroke
 				(width 0.05)
@@
 		)
 		(pad "1" smd rect
-			(at -1.25 -0.7 180)
-			(size 1 0.8)
+			(at 1.55 -0.7 180)
+			(size 1.5 0.9)
 			(layers "F.Cu" "F.Paste" "F.Mask")
 			(net 16 "Net-(D1-RK)")
@@
 		)
 		(pad "2" smd rect
-			(at -1.25 0.7 180)
-			(size 1 0.8)
+			(at 1.55 0.7 180)
+			(size 1.5 0.9)
 			(layers "F.Cu" "F.Paste" "F.Mask")
 			(net 17 "Net-(D1-GK)")
@@
 		)
 		(pad "3" smd rect
-			(at 1.25 0.7 180)
-			(size 1 0.8)
+			(at -1.55 -0.7 180)
+			(size 1.5 0.9)
 			(layers "F.Cu" "F.Paste" "F.Mask")
 			(net 18 "Net-(D1-BK)")
@@
 		)
 		(pad "4" smd rect
-			(at 1.25 -0.7 180)
-			(size 1 0.8)
+			(at -1.55 0.7 180)
+			(size 1.5 0.9)
 			(layers "F.Cu" "F.Paste" "F.Mask")
 			(net 2 "VDD_3V3")
@@
 			(pintype "passive")
 		)
-		(model "${KICAD8_3DMODEL_DIR}/LED_SMD.3dshapes/LED_Cree-PLCC4_3.2x2.8mm_CCW.wrl"
+		(model "${KICAD8_3DMODEL_DIR}/LED_SMD.3dshapes/LED_RGB_Wuerth-PLCC4_3.2x2.8mm_150141M173100.wrl"
 			(offset
 				(xyz 0 0 0)
@@
 			)
 		)
-		(model "${KIPRJMOD}/packages3D/LED_3528_RGB.STEP"
-			(offset
-				(xyz 0 0 0)
-			)
-			(scale
-				(xyz 1 1 1)
-			)
-			(rotate
-				(xyz -90 0 0)
-			)
-		)
 	)
 	(footprint "Package_SO:SOIC-8_3.9x4.9mm_P1.27mm"
@@
 		)
 	)
-	(footprint "LED_SMD:LED_Cree-PLCC4_3.2x2.8mm_CCW"
+	(footprint "LED_SMD:LED_RGB_Wuerth-PLCC4_3.2x2.8mm_150141M173100"
 		(layer "F.Cu")
-		(at 147.523 85.584)
-		(descr "3.2mm x 2.8mm PLCC4 RGB LED, https://assets.cree-led.com/a/ds/h/HB-CLV1A-FKB.pdf")
-		(tags "LED Cree PLCC-4 3528 CLV1A-FKB")
+		(at 147.711 85.532)
+		(descr "3.2mm x 2.8mm PLCC4 LED, https://www.we-online.de/katalog/datasheet/150141M173100.pdf")
+		(tags "LED RGB Wurth PLCC-4 3528")
 		(property "Reference" "D8"
-			(at 0 -2.65 0)
+			(at 0 -2.4 0)
 			(layer "F.SilkS")
 			(hide yes)
@@
 		)
 		(property "Value" "LED_RGBA"
-			(at 0 2.65 0)
+			(at 0 2.5 0)
 			(layer "F.Fab")
 			(effects
@@
 			)
 		)
-		(property "Footprint" "LED_SMD:LED_Cree-PLCC4_3.2x2.8mm_CCW"
+		(property "Footprint" "LED_SMD:LED_RGB_Wuerth-PLCC4_3.2x2.8mm_150141M173100"
 			(at 0 0 0)
 			(unlocked yes)
@@
 		(attr smd)
 		(fp_line
-			(start -1.95 -1.5)
-			(end 1.95 -1.5)
+			(start -2.5 -1.51)
+			(end 2.3 -1.51)
 			(stroke
 				(width 0.12)
@@
 		)
 		(fp_line
-			(start -1.95 -0.7)
-			(end -1.95 -1.5)
+			(start -2.5 -0.7)
+			(end -2.5 -1.51)
 			(stroke
 				(width 0.12)
@@
 		)
 		(fp_line
-			(start -1.95 1.5)
-			(end 1.95 1.5)
+			(start -2.3 1.51)
+			(end 2.3 1.51)
 			(stroke
 				(width 0.12)
@@
 		)
 		(fp_line
-			(start -2.2 -1.75)
-			(end -2.2 1.75)
+			(start -2.55 -1.65)
+			(end -2.55 1.65)
 			(stroke
 				(width 0.05)
@@
 		)
 		(fp_line
-			(start -2.2 1.75)
-			(end 2.2 1.75)
+			(start -2.55 1.65)
+			(end 2.55 1.65)
 			(stroke
 				(width 0.05)
@@
 		)
 		(fp_line
-			(start 2.2 -1.75)
-			(end -2.2 -1.75)
+			(start 2.55 -1.65)
+			(end -2.55 -1.65)
 			(stroke
 				(width 0.05)
@@
 		)
 		(fp_line
-			(start 2.2 1.75)
-			(end 2.2 -1.75)
+			(start 2.55 1.65)
+			(end 2.55 -1.65)
 			(stroke
 				(width 0.05)
@@
 		)
 		(fp_text user "${REFERENCE}"
-			(at -0.08 1.32 0)
+			(at 0 0 0)
 			(layer "F.Fab")
 			(effects
@@
 		)
 		(pad "1" smd rect
-			(at -1.25 -0.7)
-			(size 1 0.8)
+			(at 1.55 -0.7)
+			(size 1.5 0.9)
 			(layers "F.Cu" "F.Paste" "F.Mask")
 			(net 23 "Net-(D8-RK)")
@@
 		)
 		(pad "2" smd rect
-			(at -1.25 0.7)
-			(size 1 0.8)
+			(at 1.55 0.7)
+			(size 1.5 0.9)
 			(layers "F.Cu" "F.Paste" "F.Mask")
 			(net 21 "Net-(D8-GK)")
@@
 		)
 		(pad "3" smd rect
-			(at 1.25 0.7)
-			(size 1 0.8)
+			(at -1.55 -0.7)
+			(size 1.5 0.9)
 			(layers "F.Cu" "F.Paste" "F.Mask")
 			(net 22 "Net-(D8-BK)")
@@
 		)
 		(pad "4" smd rect
-			(at 1.25 -0.7)
-			(size 1 0.8)
+			(at -1.55 0.7)
+			(size 1.5 0.9)
 			(layers "F.Cu" "F.Paste" "F.Mask")
 			(net 2 "VDD_3V3")
@@
 			(pintype "passive")
 		)
-		(model "${KICAD8_3DMODEL_DIR}/LED_SMD.3dshapes/LED_Cree-PLCC4_3.2x2.8mm_CCW.wrl"
+		(model "${KICAD8_3DMODEL_DIR}/LED_SMD.3dshapes/LED_RGB_Wuerth-PLCC4_3.2x2.8mm_150141M173100.wrl"
 			(offset
 				(xyz 0 0 0)
@@
 			)
 		)
-		(model "${KIPRJMOD}/packages3D/LED_3528_RGB.STEP"
-			(offset
-				(xyz 0 0 0)
-			)
-			(scale
-				(xyz 1 1 1)
-			)
-			(rotate
-				(xyz -90 0 0)
-			)
-		)

Commit message: Update
Parts:
- added G***: LOGO, Logos:platypus_16_9.3, F.Cu at (120.6, 80.8)
- C14, R20: moved to B.Cu
- R4: moved to F.Cu
- moved R20 44.1 mm to (158.9, 71.8), turned to -90 degrees
- moved R19 41.0 mm to (141.4, 83.5), turned to 90 degrees
- moved R4 35.5 mm to (138.4, 83.0), turned to 45 degrees
- moved C9 11.7 mm to (116.9, 96.1), turned to 180 degrees
- moved D5 8.46 mm to (124.9, 73.4), turned to 180 degrees
- moved D6 8.39 mm to (124.9, 88.0)
- moved C23 4.43 mm to (121.8, 73.8), turned to 90 degrees
- moved C14 4.36 mm to (126.7, 79.9), turned to -90 degrees
- moved R7 4.19 mm to (127.9, 75.9), turned to -90 degrees
- moved D1 3.41 mm to (145.8, 86.0), turned to -90 degrees
- moved D8 2.17 mm to (149.8, 86.1), turned to 90 degrees
- moved R24 1.92 mm to (149.3, 87.6)
- moved C15 1.86 mm to (136.3, 86.8), turned to 90 degrees
- moved C25 1.25 mm to (156.7, 72.9)
- moved D7 0.45 mm to (161.3, 68.1), turned to 0 degrees
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Connections:
- U1 pad 11: unconnected-(U1-PC3-Pad11) -> SD_CD
- U1 pad 41: unconnected-(U1-PA8-Pad41) -> LED4
Routing:
- net SD_CD: track 0.00 -> 28.1 mm, vias 0 -> 2
- net Net-(D6-K): track 0.00 -> 21.1 mm
- net FLASH_CS: track 0.00 -> 20.4 mm
- net BOOT0: track 6.94 -> 21.3 mm
- net SPI_MISO: track 8.13 -> 17.9 mm
- net NRST: track 41.9 -> 37.7 mm
- net Net-(D7-K): track 0.00 -> 3.26 mm, vias 0 -> 1
- net VDD_3V3: track 37.0 -> 40.2 mm, vias 13 -> 15
- net SDIO_CK: track 14.8 -> 17.2 mm
- net SPI_CLK: track 7.85 -> 9.79 mm
- net Net-(SW2-B): track 0.00 -> 1.92 mm
- net SDIO_CMD: track 19.1 -> 17.3 mm
- net SPI_MOSI: track 8.29 -> 10.0 mm
- net LED4: track 0.00 -> 1.51 mm, vias 0 -> 1
- net GND: track 38.6 -> 39.9 mm, vias 32 -> 33
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
Commit message: Piezo fixes
Parts:
- JP1, R1, R2, R21, R22, R23, R3: moved to B.Cu
- moved R18 61.5 mm to (122.6, 71.5), turned to 180 degrees
- moved R23 39.8 mm to (149.3, 85.0), turned to -90 degrees
- moved R22 36.9 mm to (150.8, 85.0), turned to -90 degrees
- moved R3 35.0 mm to (146.2, 85.4), turned to -90 degrees
- moved R21 33.6 mm to (149.3, 88.1), turned to -90 degrees
- moved R2 32.1 mm to (147.6, 85.4), turned to -90 degrees
- moved R1 29.3 mm to (146.2, 88.3), turned to -90 degrees
- moved R11 26.7 mm to (141.3, 82.7)
- moved R10 26.5 mm to (141.3, 81.2), turned to 180 degrees
- moved R24 10.0 mm to (139.9, 84.1), turned to 0 degrees
- moved JP1 8.95 mm to (116.8, 92.0), turned to -90 degrees
- moved C9 5.43 mm to (120.5, 92.0), turned to -90 degrees
- moved C15 2.71 mm to (138.9, 87.6), turned to 0 degrees
- moved R19 2.47 mm to (139.9, 85.6), turned to 0 degrees
- moved R4 1.06 mm to (137.4, 82.6), turned to 0 degrees
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Connections:
- D5 pad 1: Net-(D5-K) -> LED3
- D5 pad 2: VDD_3V3 -> Net-(D5-A)
- J5 pad MP: (no net) -> GND
- J6 pad MP: (no net) -> GND
- J7 pad MP: (no net) -> GND
- R18 pad 1: Net-(D5-K) -> Net-(D5-A)
- R18 pad 2: LED3 -> VDD_3V3
- U1 pad 20: unconnected-(U1-PA4-Pad20) -> FLASH_CS
- U1 pad 30: unconnected-(U1-PB11-Pad30) -> VBUS_DETECT
- U1 pad 33: unconnected-(U1-PB12-Pad33) -> LED2_RGB_GREEN
- U1 pad 34: unconnected-(U1-PB13-Pad34) -> LED1_RGB_GREEN
- U1 pad 35: unconnected-(U1-PB14-Pad35) -> LED1_RGB_RED
- U1 pad 36: unconnected-(U1-PB15-Pad36) -> LED2_RGB_RED
- U1 pad 37: unconnected-(U1-PC6-Pad37) -> LED1_RGB_BLUE
- U1 pad 38: unconnected-(U1-PC7-Pad38) -> LED2_RGB_BLUE
- U1 pad 56: unconnected-(U1-PB4-Pad56) -> LED3
Routing:
- net LED3: track 0.00 -> 23.9 mm, vias 0 -> 1
- net BOOT0: track 21.3 -> 9.99 mm
- net LED2_RGB_BLUE: track 0.00 -> 11.1 mm
- net LED2_RGB_RED: track 0.00 -> 10.2 mm
- net VDD_3V3: track 40.2 -> 50.1 mm, vias 15 -> 17
- net Net-(SW2-B): track 1.92 -> 11.8 mm
- net Net-(J3-Pin_1): track 0.00 -> 9.37 mm, vias 0 -> 1
- net LED2_RGB_GREEN: track 0.00 -> 7.08 mm
- net LED1_RGB_BLUE: track 0.00 -> 6.60 mm
- net VBUS_DETECT: track 0.00 -> 6.30 mm, vias 0 -> 1
- net VDD_5V_USB: track 9.68 -> 15.2 mm
- net LED1_RGB_GREEN: track 0.00 -> 4.48 mm
- net LED1_RGB_RED: track 0.00 -> 3.64 mm
- net Net-(D6-K): track 21.1 -> 18.4 mm
- net NRST: track 37.7 -> 40.2 mm
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Other:
- board size 136.5 x 28.9 mm -> 58.5 x 28.9 mm

Commit message: Master board pre-production
Parts:
- added G***: LOGO, Logos:name_11_2.0, F.Cu at (126.4, 68.5)
- moved R10 2.32 mm to (143.5, 80.5), turned to 90 degrees
- moved R11 1.44 mm to (141.3, 81.2)
- turned U2 to -90 degrees
Connections:
- U2 pad 1: /Connectors/usb_conn_d- -> USB_D+
- U2 pad 3: /Connectors/usb_conn_d+ -> USB_D-
- U2 pad 4: USB_D+ -> /Connectors/usb_conn_d-
- U2 pad 6: USB_D- -> /Connectors/usb_conn_d+
Routing:
- net VDD_7V0: track 38.4 -> 2.69 mm
- net GND: track 41.4 -> 47.1 mm, vias 62 -> 63
- net VDD_3V3: track 50.1 -> 47.2 mm
- net VDD_5V_USB: track 15.2 -> 16.8 mm
- net VBUS_DETECT: track 6.30 -> 4.95 mm
- net Net-(D6-K): track 18.4 -> 18.9 mm
- net DEBUG_SWO: track 19.9 -> 20.4 mm
- added copper zone on B.Cu, net GND
- added copper zone on F.Cu, net GND
- added copper zone on In1.Cu, net VDD_3V3
- added copper zone on In1.Cu, net VDD_7V0
Other:
- board text added: "04/24"
- board text added: "120R"
- board text added: "GND"
- board text added: "RX"
- board text added: "TX"

Commit message: Master and Piezo ready to production
Parts:
- turned G*** to 0 degrees
Other:
- board text added: "7V0"
- board text added: "CANH"
- board text added: "CANL"
- board text added: "SWD_3V3"
- board text added: "ПОВОРОТ: -3"
- board text removed: "SD"
- board text removed: "led"
- board text removed: "usb 5v0"
- board text removed: "подписи светодиодов, коннекторов и пинов UART распиновка boot0 распиновка и подключение flash"
