File: Hardware/CAN sensor net/Master board/Master board.kicad_sch (KiCad schematic)
At the start: 35 parts, among them SW1 SW_Push, SW2 SW_SPDT, U1 STM32F405RGTx, U5 SN65HVD230, U6 SN65HVD230, Y1 16MHz

Commit message: Master board сoncept
Parts:
- added D7: LED, LED_SMD:LED_1206_3216Metric, symbol Device:LED
- added R20: 220, Resistor_SMD:R_0603_1608Metric, symbol Device:R
- C1, C10, C11, C12, C13, C2, C23, C24, C3, C4, C5, C6, C7, C8, C9: footprint Capacitor_SMD:C_0402_1005Metric -> Capacitor_SMD:C_0603_1608Metric
Connections:
- net GND: now also R20.2
- net VDD_3V3: now also D7.2 (A)
- new net: D7.1 (K), R20.1

Commit message: added spi flash memory
Parts:
- added C25: 100n, Capacitor_SMD:C_0603_1608Metric, symbol Device:C_Small
- added U7: W25Q32FVSSIG, Package_SO:SOIC-8_5.23x5.23mm_P1.27mm, symbol Memory_Flash:W25Q32JVSS
Connections:
- net GND: now also C25.1, U7.4 (GND)
- net VDD_3V3: now also C25.2, U7.7 (IO3), U7.8 (VCC)
- new net FLASH_CS: U7.1 (~{CS})
- new net SPI_CLK: U7.6 (CLK)
- new net SPI_MISO: U7.2 (DO(IO1))
- new net SPI_MOSI: U7.5 (DI(IO0))
- no-connect marks 2 -> 3
Other:
- note added: "Flash memory"
- moved on the sheet: C1, C10, C11, C12, C13, C2, C23, C24, C3, C4, C5, C6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

Commit message: Bugfix
Parts:
- added R24: 10k, Resistor_SMD:R_0603_1608Metric, symbol Device:R_Small
Connections:
- net BOOT0: now also R24.1; no longer SW2.2 (B)
- net LED1 renamed LED3
- net LED2 renamed LED4
- new net: R24.2, SW2.2 (B)

Commit message: added solder jumpers for 120R CAN
Parts:
- added JP2, JP3: SolderJumper_2_Open, symbol Jumper:SolderJumper_2_Open
Connections:
- net CAN0_L: now also JP2.1 (A); no longer R16.2
- net CAN1_L: now also JP3.1 (A); no longer R17.2
- new net: JP3.2 (B), R17.2
- new net: JP2.2 (B), R16.2

Commit message: Added UART port
Parts:
- JP2, JP3: footprint (none) -> Jumper:SolderJumper-2_P1.3mm_Open_RoundedPad1.0x1.5mm
Changed lines of the file:
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@@
 			)
 		)
-		(property "Footprint" ""
+		(property "Footprint" "Jumper:SolderJumper-2_P1.3mm_Open_RoundedPad1.0x1.5mm"
 			(at 264.16 139.065 0)
 			(effects
@@
 			)
 		)
-		(property "Footprint" ""
+		(property "Footprint" "Jumper:SolderJumper-2_P1.3mm_Open_RoundedPad1.0x1.5mm"
 			(at 200.025 139.065 0)
 			(effects

Commit message: PCB prototype
Parts:
- added H1, H2, H3: MountingHole, MountingHole:MountingHole_2.2mm_M2_Pad_Via, symbol Mechanical:MountingHole
Changed lines of the file:
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@@
 		)
 	)
+	(polyline
+		(pts
+			(xy 108.585 13.97) (xy 108.585 44.45)
+		)
+		(stroke
+			(width 0)
+			(type default)
+		)
+	)
 	(wire
 		(pts
@@
 		)
 	)
-	(polyline
-		(pts
-			(xy 108.585 45.085) (xy 108.585 14.605)
-		)
-		(stroke
-			(width 0)
-			(type default)
-		)
-	)
 	(wire
 		(pts
@@
 	)
 	(symbol
+		(lib_id "Mechanical:MountingHole")
+		(at 147.32 177.165 0)
+		(unit 1)
+		(exclude_from_sim no)
+		(in_bom yes)
+		(on_board yes)
+		(dnp no)
+		(fields_autoplaced yes)
+		(property "Reference" "H3"
+			(at 149.86 175.8949 0)
+			(effects
+				(font
+					(size 1.27 1.27)
+				)
+				(justify left)
+			)
+		)
+		(property "Value" "MountingHole"
+			(at 149.86 178.4349 0)
+			(effects
+				(font
+					(size 1.27 1.27)
+				)
+				(justify left)
+			)
+		)
+		(property "Footprint" "MountingHole:MountingHole_2.2mm_M2_Pad_Via"
+			(at 147.32 177.165 0)
+			(effects
+				(font
+					(size 1.27 1.27)
+				)
+				(hide yes)
+			)
+		)
+		(property "Datasheet" "~"
+			(at 147.32 177.165 0)
+			(effects
+				(font
+					(size 1.27 1.27)
+				)
+				(hide yes)
+			)
+		)
+		(property "Description" "Mounting Hole without connection"
+			(at 147.32 177.165 0)
+			(effects
+				(font
+					(size 1.27 1.27)
+				)
+				(hide yes)
+			)
+		)
+		(instances
+			(project "Master board"
+				(path "/11ca9491-ebda-4c18-be98-3e552caaabb4"
+					(reference "H3")
+					(unit 1)
+				)
+			)
+		)
+	)
+	(symbol
 		(lib_id "Device:R")
 		(at 205.74 73.66 90)
@@
 	)
 	(symbol
+		(lib_id "Mechanical:MountingHole")
+		(at 147.32 172.085 0)
+		(unit 1)
+		(exclude_from_sim no)
+		(in_bom yes)
+		(on_board yes)
+		(dnp no)
+		(fields_autoplaced yes)
+		(property "Reference" "H2"
+			(at 149.86 170.8149 0)
+			(effects
+				(font
+					(size 1.27 1.27)
+				)
+				(justify left)
+			)
+		)
+		(property "Value" "MountingHole"
+			(at 149.86 173.3549 0)
+			(effects
+				(font
+					(size 1.27 1.27)
+				)
+				(justify left)
+			)
+		)
+		(property "Footprint" "MountingHole:MountingHole_2.2mm_M2_Pad_Via"
+			(at 147.32 172.085 0)
+			(effects
+				(font
+					(size 1.27 1.27)
+				)
+				(hide yes)
+			)
+		)
+		(property "Datasheet" "~"
+			(at 147.32 172.085 0)
+			(effects
+				(font
+					(size 1.27 1.27)
+				)
+				(hide yes)
+			)
+		)
+		(property "Description" "Mounting Hole without connection"
+			(at 147.32 172.085 0)
+			(effects
+				(font
+					(size 1.27 1.27)
+				)
+				(hide yes)
+			)
+		)
+		(instances
+			(project "Master board"
+				(path "/11ca9491-ebda-4c18-be98-3e552caaabb4"
+					(reference "H2")
+					(unit 1)
+				)
+			)
+		)
+	)
+	(symbol
 		(lib_name "GND_1")
 		(lib_id "power:GND")
@@
 					(unit 1)
 				)
+			)
+		)
+	)
+	(symbol
+		(lib_id "Mechanical:MountingHole")
+		(at 147.32 167.005 0)
+		(unit 1)
+		(exclude_from_sim no)
+		(in_bom yes)
+		(on_board yes)
+		(dnp no)
+		(fields_autoplaced yes)
+		(property "Reference" "H1"
+			(at 149.86 165.7349 0)
+			(effects
+				(font
+					(size 1.27 1.27)
+				)
+				(justify left)
+			)
+		)
+		(property "Value" "MountingHole"
+			(at 149.86 168.2749 0)
+			(effects
+				(font
+					(size 1.27 1.27)
+				)
+				(justify left)
+			)
+		)
+		(property "Footprint" "MountingHole:MountingHole_2.2mm_M2_Pad_Via"
+			(at 147.32 167.005 0)
+			(effects
+				(font
+					(size 1.27 1.27)
+				)
+				(hide yes)
+			)
+		)
+		(property "Datasheet" "~"
+			(at 147.32 167.005 0)
+			(effects
+				(font
+					(size 1.27 1.27)
+				)
+				(hide yes)
+			)
+		)
+		(property "Description" "Mounting Hole without connection"
+			(at 147.32 167.005 0)
+			(effects
+				(font
+					(size 1.27 1.27)
+				)
+				(hide yes)
+			)
+		)
+		(instances
+			(project "Master board"
+				(path "/11ca9491-ebda-4c18-be98-3e552caaabb4"
+					(reference "H1")
+					(unit 1)
+				)

Commit message: Concept no trace
Parts:
- SW2: footprint user_lib:MSS-12D16 -> Button_Switch_SMD:SW_SPDT_PCM12
Connections:
- net at R16.2: now also JP2.1 (A); no longer JP2.2 (B)
- net CAN0_H renamed CAN0_+
- net CAN0_+: now also JP2.2 (B); no longer R16.1
- net CAN0_L renamed CAN0_-
- net CAN0_-: now also R16.1; no longer JP2.1 (A)
- net CAN1_H renamed CAN1_+
- net CAN1_L renamed CAN1_-
Other:
- moved on the sheet: JP2, R16
Changed lines of the file:
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@@
 		)
 	)
-	(global_label "CAN1_TX"
+	(global_label "CAN0_+"
 		(shape input)
-		(at 235.585 132.715 180)
+		(at 203.835 128.905 0)
 		(fields_autoplaced yes)
 		(effects
@@
 				(size 1.27 1.27)
 			)
-			(justify right)
+			(justify left)
 		)
 		(property "Intersheetrefs" "${INTERSHEET_REFS}"
-			(at 224.5565 132.715 0)
+			(at 214.2588 128.905 0)
 			(effects
 				(font
 					(size 1.27 1.27)
 				)
-				(justify right)
+				(justify left)
 				(hide yes)
 			)
 		)
 	)
-	(global_label "VBUS_DETECT"
+	(global_label "CAN1_TX"
 		(shape input)
-		(at 110.49 154.94 0)
+		(at 235.585 132.715 180)
 		(fields_autoplaced yes)
 		(effects
@@
 				(size 1.27 1.27)
 			)
-			(justify left)
+			(justify right)
 		)
 		(property "Intersheetrefs" "${INTERSHEET_REFS}"
-			(at 126.1146 154.94 0)
+			(at 224.5565 132.715 0)
 			(effects
 				(font
 					(size 1.27 1.27)
 				)
-				(justify left)
+				(justify right)
 				(hide yes)
 			)
 		)
 	)
-	(global_label "LED2_RGB_GREEN"
+	(global_label "VBUS_DETECT"
 		(shape input)
-		(at 214.63 97.155 0)
+		(at 110.49 154.94 0)
 		(fields_autoplaced yes)
 		(effects
@@
 		)
 		(property "Intersheetrefs" "${INTERSHEET_REFS}"
-			(at 234.1855 97.155 0)
+			(at 126.1146 154.94 0)
 			(effects
 				(font
@@
 		)
 	)
-	(global_label "CAN0_H"
+	(global_label "LED2_RGB_GREEN"
 		(shape input)
-		(at 203.835 128.905 0)
+		(at 214.63 97.155 0)
 		(fields_autoplaced yes)
 		(effects
@@
 		)
 		(property "Intersheetrefs" "${INTERSHEET_REFS}"
-			(at 214.0169 128.905 0)
+			(at 234.1855 97.155 0)
 			(effects
 				(font
@@
 		)
 	)
-	(global_label "CAN1_H"
+	(global_label "CAN1_+"
 		(shape input)
 		(at 267.97 128.905 0)
@@
 		)
 		(property "Intersheetrefs" "${INTERSHEET_REFS}"
-			(at 278.1519 128.905 0)
+			(at 278.3938 128.905 0)
 			(effects
 				(font
@@
 		)
 	)
+	(global_label "CAN0_-"
+		(shape input)
+		(at 203.835 144.145 0)
+		(fields_autoplaced yes)
+		(effects
+			(font
+				(size 1.27 1.27)
+			)
+			(justify left)
+		)
+		(property "Intersheetrefs" "${INTERSHEET_REFS}"
+			(at 214.2588 144.145 0)
+			(effects
+				(font
+					(size 1.27 1.27)
+				)
+				(justify left)
+				(hide yes)
+			)
+		)
+	)
 	(global_label "FLASH_CS"
 		(shape input)
@@
 		)
 	)
-	(global_label "CAN1_L"
+	(global_label "CAN1_-"
 		(shape input)
 		(at 267.97 144.145 0)
@@
 		)
 		(property "Intersheetrefs" "${INTERSHEET_REFS}"
-			(at 277.8495 144.145 0)
+			(at 278.3938 144.145 0)
 			(effects
 				(font
@@
 		)
 	)
-	(global_label "CAN0_L"
-		(shape input)
-		(at 203.835 144.145 0)
-		(fields_autoplaced yes)
-		(effects
-			(font
-				(size 1.27 1.27)
-			)
-			(justify left)
-		)
-		(property "Intersheetrefs" "${INTERSHEET_REFS}"
-			(at 213.7145 144.145 0)
-			(effects
-				(font
-					(size 1.27 1.27)
-				)
-				(justify left)
-				(hide yes)
-			)
-		)
-	)
 	(global_label "VDD_3V3"
 		(shape input)
@@
 	(symbol
 		(lib_id "Jumper:SolderJumper_2_Open")
-		(at 200.025 139.065 90)
+		(at 200.025 133.985 90)
 		(unit 1)
 		(exclude_from_sim no)
@@
 		(dnp no)
 		(property "Reference" "JP2"
-			(at 201.295 139.065 90)
+			(at 201.295 133.985 90)
 			(effects
 				(font
@@
 		)
 		(property "Value" "SolderJumper_2_Open"
-			(at 202.565 140.3349 90)
+			(at 202.565 135.2549 90)
 			(effects
 				(font
@@
 		)
 		(property "Footprint" "Jumper:SolderJumper-2_P1.3mm_Open_RoundedPad1.0x1.5mm"
-			(at 200.025 139.065 0)
+			(at 200.025 133.985 0)
 			(effects
 				(font
@@
 		)
 		(property "Datasheet" "~"
-			(at 200.025 139.065 0)
+			(at 200.025 133.985 0)
 			(effects
 				(font
@@
 		)
 		(property "Description" "Solder Jumper, 2-pole, open"
-			(at 200.025 139.065 0)
+			(at 200.025 133.985 0)
 			(effects
 				(font
@@
 			)
 		)
-		(property "Footprint" "user_lib:MSS-12D16"
+		(property "Footprint" "Button_Switch_SMD:SW_SPDT_PCM12"
 			(at 90.805 31.75 0)
 			(effects
@@
 	(symbol
 		(lib_id "Device:R_Small")
-		(at 200.025 132.715 0)
+		(at 200.025 140.335 180)
 		(unit 1)
 		(exclude_from_sim no)
@@
 		(dnp no)
 		(property "Reference" "R16"
-			(at 201.295 131.445 0)
+			(at 205.105 141.605 0)
 			(effects
 				(font
@@
 		)
 		(property "Value" "120"
-			(at 201.295 133.985 0)
+			(at 205.105 139.065 0)
 			(effects
 				(font
@@
 		)
 		(property "Footprint" "Resistor_SMD:R_0603_1608Metric"
-			(at 200.025 132.715 0)
+			(at 200.025 140.335 0)
 			(effects
 				(font
@@
 		)
 		(property "Datasheet" "~"
-			(at 200.025 132.715 0)
+			(at 200.025 140.335 0)
 			(effects
 				(font
@@
 		)
 		(property "Description" "Resistor, small symbol"
-			(at 200.025 132.715 0)
+			(at 200.025 140.335 0)
 			(effects
 				(font

Commit message: added band pass filter to piezo board
Changed lines of the file:
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@@
+		)
+	)
+	(global_label "UART1_TX"
+		(shape input)
+		(at 110.49 110.49 0)
+		(fields_autoplaced yes)
+		(effects
+			(font
+				(size 1.27 1.27)
+			)
+			(justify left)
+		)
+		(property "Intersheetrefs" "${INTERSHEET_REFS}"
+			(at 122.4861 110.49 0)
+			(effects
+				(font
+					(size 1.27 1.27)
+				)
+				(justify left)
+				(hide yes)
+			)
 		)
 	)
@@
 				(hide yes)
 			)
+		)
+	)
+	(global_label "UART1_RX"
+		(shape input)
+		(at 110.49 113.03 0)
+		(fields_autoplaced yes)
+		(effects
+			(font
+				(size 1.27 1.27)
+			)
+			(justify left)
+		)
+		(property "Intersheetrefs" "${INTERSHEET_REFS}"
+			(at 122.7885 113.03 0)
+			(effects
+				(font
+					(size 1.27 1.27)
+				)
+				(justify left)
+				(hide yes)
+			)
