File: Hardware/CAN sensor net/Master board/power.kicad_sch (KiCad schematic)
At the start: 20 parts, among them J4 XT60, J7 DC-005, U3 ST1S14PHR, U4 LDL1117_3V3

Commit message: changed xt60 to xt30
Parts:
- J4: footprint Connector_AMASS:AMASS_XT60PW-M_1x02_P7.20mm_Horizontal -> Connector_AMASS:AMASS_XT30PW-M_1x02_P2.50mm_Horizontal
Changed lines of the file:
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@@
 			)
 		)
-		(property "Footprint" "Connector_AMASS:AMASS_XT60PW-M_1x02_P7.20mm_Horizontal"
+		(property "Footprint" "Connector_AMASS:AMASS_XT30PW-M_1x02_P2.50mm_Horizontal"
 			(at 27.305 60.96 0)
 			(effects

Commit message: Master board сoncept
Parts:
- removed J7: DC-005, Connector_BarrelJack:BarrelJack_Horizontal, symbol Connector:Conn_Coaxial_Power
- removed JP2: Jumper_2_Bridged, Connector_PinHeader_2.54mm:PinHeader_1x02_P2.54mm_Vertical, symbol Jumper:Jumper_2_Bridged
- C16, C21, C22: footprint Capacitor_SMD:C_0402_1005Metric -> Capacitor_SMD:C_0603_1608Metric
- C18: footprint Capacitor_SMD:C_0805_2012Metric -> Capacitor_SMD:C_0603_1608Metric
- R12: footprint Resistor_SMD:R_0402_1005Metric -> Resistor_SMD:R_0603_1608Metric
Connections:
- net VDD_3V3: now also C22.1, U4.2 (VO)
Changed lines of the file:
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@@
-	)
-	(junction
-		(at 34.29 88.9)
-		(diameter 0)
-		(color 0 0 0 0)
 	)
 	(junction
@@
 	)
 	(junction
-		(at 34.29 58.42)
-		(diameter 0)
-		(color 0 0 0 0)
-	)
-	(junction
 		(at 40.64 88.9)
 		(diameter 0)
@@
 	(wire
 		(pts
-			(xy 34.29 88.9) (xy 40.64 88.9)
-		)
-		(stroke
-			(width 0)
-			(type default)
-		)
-	)
-	(wire
-		(pts
 			(xy 98.425 73.66) (xy 98.425 76.2)
 		)
@@
 	(wire
 		(pts
-			(xy 209.55 68.58) (xy 216.535 68.58)
-		)
-		(stroke
-			(width 0)
-			(type default)
-		)
-	)
-	(wire
-		(pts
 			(xy 90.17 58.42) (xy 98.425 58.42)
 		)
@@
 	(wire
 		(pts
+			(xy 209.55 62.23) (xy 209.55 68.58)
+		)
+		(stroke
+			(width 0)
+			(type default)
+		)
+	)
+	(wire
+		(pts
 			(xy 170.18 68.58) (xy 181.61 68.58)
 		)
@@
 	(wire
 		(pts
-			(xy 226.695 68.58) (xy 231.775 68.58)
-		)
-		(stroke
-			(width 0)
-			(type default)
-		)
-	)
-	(wire
-		(pts
-			(xy 32.385 58.42) (xy 34.29 58.42)
-		)
-		(stroke
-			(width 0)
-			(type default)
-		)
-	)
-	(wire
-		(pts
 			(xy 170.18 64.77) (xy 170.18 68.58)
 		)
@@
 	(wire
 		(pts
-			(xy 34.29 58.42) (xy 34.29 69.215)
-		)
-		(stroke
-			(width 0)
-			(type default)
-		)
-	)
-	(wire
-		(pts
 			(xy 123.19 63.5) (xy 123.19 67.945)
 		)
@@
 	(wire
 		(pts
-			(xy 34.29 58.42) (xy 53.975 58.42)
+			(xy 32.385 58.42) (xy 53.975 58.42)
 		)
 		(stroke
@@
 	(wire
 		(pts
-			(xy 34.29 93.345) (xy 34.29 88.9)
+			(xy 40.64 92.71) (xy 40.64 88.9)
 		)
 		(stroke
@@
 	(wire
 		(pts
-			(xy 231.775 65.405) (xy 231.775 68.58)
-		)
-		(stroke
-			(width 0)
-			(type default)
-		)
-	)
-	(wire
-		(pts
 			(xy 98.425 68.58) (xy 98.425 73.66)
 		)
@@
 		(pts
 			(xy 181.61 78.74) (xy 181.61 82.55)
-		)
-		(stroke
-			(width 0)
-			(type default)
-		)
-	)
-	(wire
-		(pts
-			(xy 34.29 76.835) (xy 34.29 88.9)
 		)
 		(stroke
@@
 	(global_label "VDD_3V3"
 		(shape input)
-		(at 231.775 65.405 90)
+		(at 209.55 62.23 90)
 		(fields_autoplaced yes)
 		(effects
@@
 		)
 		(property "Intersheetrefs" "${INTERSHEET_REFS}"
-			(at 231.6956 54.8881 90)
+			(at 209.4706 51.7131 90)
 			(effects
 				(font
@@
 			)
 		)
-		(property "Footprint" "Capacitor_SMD:C_0402_1005Metric"
+		(property "Footprint" "Capacitor_SMD:C_0603_1608Metric"
 			(at 180.6448 77.47 0)
 			(effects
@@
 			)
 		)
-		(property "Footprint" "Capacitor_SMD:C_0805_2012Metric"
+		(property "Footprint" "Capacitor_SMD:C_0603_1608Metric"
 			(at 62.865 66.04 0)
 			(effects
@@
 	(symbol
 		(lib_id "power:GND")
-		(at 34.29 93.345 0)
+		(at 40.64 92.71 0)
 		(unit 1)
 		(exclude_from_sim no)
@@
 		(dnp no)
 		(property "Reference" "#PWR012"
-			(at 34.29 99.695 0)
+			(at 40.64 99.06 0)
 			(effects
 				(font
@@
 		)
 		(property "Value" "GND"
-			(at 34.29 97.155 0)
+			(at 40.64 96.52 0)
 			(effects
 				(font
@@
 		)
 		(property "Footprint" ""
-			(at 34.29 93.345 0)
+			(at 40.64 92.71 0)
 			(effects
 				(font
@@
 		)
 		(property "Datasheet" ""
-			(at 34.29 93.345 0)
+			(at 40.64 92.71 0)
 			(effects
 				(font
@@
 		)
 		(property "Description" ""
-			(at 34.29 93.345 0)
+			(at 40.64 92.71 0)
 			(effects
 				(font
@@
 			)
 		)
-		(property "Footprint" "Capacitor_SMD:C_0402_1005Metric"
+		(property "Footprint" "Capacitor_SMD:C_0603_1608Metric"
 			(at 98.425 60.96 0)
 			(effects
@@
 			)
 		)
-		(property "Footprint" "Capacitor_SMD:C_0402_1005Metric"
+		(property "Footprint" "Capacitor_SMD:C_0603_1608Metric"
 			(at 210.5152 77.47 0)
 			(effects
@@
 	)
 	(symbol
-		(lib_id "Jumper:Jumper_2_Bridged")
-		(at 221.615 68.58 0)
-		(unit 1)
-		(exclude_from_sim no)
-		(in_bom yes)
-		(on_board yes)
-		(dnp no)
-		(property "Reference" "JP2"
-			(at 221.615 66.675 0)
-			(effects
-				(font
-					(size 1.27 1.27)
-				)
-			)
-		)
-		(property "Value" "Jumper_2_Bridged"
-			(at 221.615 65.405 0)
-			(effects
-				(font
-					(size 1.27 1.27)
-				)
-				(hide yes)
-			)
-		)
-		(property "Footprint" "Connector_PinHeader_2.54mm:PinHeader_1x02_P2.54mm_Vertical"
-			(at 221.615 68.58 0)
-			(effects
-				(font
-					(size 1.27 1.27)
-				)
-				(hide yes)
-			)
-		)
-		(property "Datasheet" "~"
-			(at 221.615 68.58 0)
-			(effects
-				(font
-					(size 1.27 1.27)
-				)
-				(hide yes)
-			)
-		)
-		(property "Description" "Jumper, 2-pole, closed/bridged"
-			(at 221.615 68.58 0)
-			(effects
-				(font
-					(size 1.27 1.27)
-				)
-				(hide yes)
-			)
-		)
-		(pin "1"
-		)
-		(pin "2"
-		)
-		(instances
-			(project "Master board"
-				(path "/11ca9491-ebda-4c18-be98-3e552caaabb4/16e6c27b-6e16-4080-b5a9-f4080643e90c"
-					(reference "JP2")
-					(unit 1)
-				)
-			)
-		)
-	)
-	(symbol
 		(lib_id "Device:R_Small")
 		(at 104.14 66.04 90)
@@
 			)
 		)
-		(property "Footprint" "Resistor_SMD:R_0402_1005Metric"
+		(property "Footprint" "Resistor_SMD:R_0603_1608Metric"
 			(at 104.14 66.04 0)
 			(effects
@@
 					(unit 1)
 				)
-			)
-		)
-	)
-	(symbol
-		(lib_id "Connector:Conn_Coaxial_Power")
-		(at 34.29 71.755 0)
-		(unit 1)
-		(exclude_from_sim no)
-		(in_bom yes)
-		(on_board yes)
-		(dnp no)
-		(property "Reference" "J7"
-			(at 28.575 72.39 0)
-			(effects
-				(font
-					(size 1.27 1.27)
-				)
-				(justify left)
-			)
-		)
-		(property "Value" "DC-005"
-			(at 24.13 74.93 0)
-			(effects
-				(font
-					(size 1.27 1.27)
-				)
-				(justify left)
-			)
-		)
-		(property "Footprint" "Connector_BarrelJack:BarrelJack_Horizontal"
-			(at 34.29 73.025 0)
-			(effects
-				(font
-					(size 1.27 1.27)
-				)
-				(hide yes)
-			)
-		)
-		(property "Datasheet" "~"
-			(at 34.29 73.025 0)
-			(effects
-				(font
-					(size 1.27 1.27)
-				)
-				(hide yes)
-			)
-		)
-		(property "Description" "coaxial connector (BNC, SMA, SMB, SMC, Cinch/RCA, LEMO, ...)"
-			(at 34.29 71.755 0)
-			(effects
-				(font
-					(size 1.27 1.27)
-				)
-				(hide yes)
-			)
-		)
-		(pin "1"
-		)
-		(pin "2"
-		)
-		(instances
-			(project "Master board"
-				(path "/11ca9491-ebda-4c18-be98-3e552caaabb4/16e6c27b-6e16-4080-b5a9-f4080643e90c"
-					(reference "J7")
-					(unit 1)
-				)

Commit message: minor fixes
Parts:
- R12: value 47K -> 47k
- R13: value 10K -> 10k
- R14, R15: value 1K -> 1k
Changed lines of the file:
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@@
 			)
 		)
-		(property "Value" "10K"
+		(property "Value" "10k"
 			(at 100.33 67.31 90)
 			(effects
@@
 			)
 		)
-		(property "Value" "47K"
+		(property "Value" "47k"
 			(at 100.33 64.77 90)
 			(effects
@@
 			)
 		)
-		(property "Value" "1K"
+		(property "Value" "1k"
 			(at 101.6 80.645 0)
 			(effects
@@
 			)
 		)
-		(property "Value" "1K"
+		(property "Value" "1k"
 			(at 101.6 86.995 0)
 			(effects

Commit message: Bugfix
Other:
- moved on the sheet: C16, C17, C18

Commit message: Added UART port
Parts:
- C20: footprint Capacitor_SMD:C_0402_1005Metric -> Capacitor_SMD:C_0603_1608Metric
Changed lines of the file:
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@@
 			)
 		)
-		(property "Footprint" "Capacitor_SMD:C_0402_1005Metric"
+		(property "Footprint" "Capacitor_SMD:C_0603_1608Metric"
 			(at 104.14 73.66 0)
 			(effects

Commit message: PCB prototype
Parts:
- added F1: RUEF300, user_lib:RUEF300, symbol Device:Fuse
Connections:
- net VDD_7V0: now also F1.1; no longer C19.1, C20.2, L1.2, R12.2, R13.2
- new net: C19.1, C20.2, F1.2, L1.2, R12.2, R13.2

Commit message: Pre-production
Parts:
- J4: value XT60 -> XT30
Changed lines of the file:
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@@
 		(fields_autoplaced yes)
 		(property "Reference" "J4"
-			(at 27.305 52.705 0)
+			(at 27.305 52.07 0)
 			(effects
 				(font
@@
 			)
 		)
-		(property "Value" "XT60"
-			(at 27.305 55.245 0)
+		(property "Value" "XT30"
+			(at 27.305 54.61 0)
 			(effects
 				(font
