File: Hardware/CAN sensor net/Piezo module/power.kicad_sch (KiCad schematic)
At the start: 10 parts, among them U5 L79L05_SOT89, U6 L78L05_SOT89, U7 LD3985M33R_SOT23

Commit message: updated piezo board schematics
Parts:
- C13: renamed from C17; footprint (none) -> Capacitor_SMD:C_0603_1608Metric
- C14: renamed from C16; footprint (none) -> Capacitor_SMD:C_0603_1608Metric
- C15: renamed from C19; footprint (none) -> Capacitor_SMD:C_0603_1608Metric
- C16: renamed from C18; footprint (none) -> Capacitor_SMD:C_0603_1608Metric
- C17: renamed from C15; footprint (none) -> Capacitor_SMD:C_0603_1608Metric
- C18: renamed from C14; footprint (none) -> Capacitor_SMD:C_0603_1608Metric
- C19: renamed from C20; footprint (none) -> Capacitor_SMD:C_0603_1608Metric
- renumbered U6 to U4, U7 to U5, U5 to U6
Changed lines of the file:
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@@
 		(dnp no)
 		(fields_autoplaced yes)
-		(property "Reference" "U7"
+		(property "Reference" "U5"
 			(at 167.64 33.02 0)
 			(effects
@@
 			(project "Piezo module"
 				(path "/0a58466e-2312-402a-82c7-7de62fe91dff/7eeb67e6-b678-4ad5-b1f2-da2d9412fd6e"
-					(reference "U7")
+					(reference "U5")
 					(unit 1)
 				)
@@
 		(on_board yes)
 		(dnp no)
-		(property "Reference" "C20"
+		(property "Reference" "C19"
 			(at 174.625 46.355 0)
 			(effects
@@
 			)
 		)
-		(property "Footprint" ""
+		(property "Footprint" "Capacitor_SMD:C_0603_1608Metric"
 			(at 179.705 48.26 0)
 			(effects
@@
 			(project "Piezo module"
 				(path "/0a58466e-2312-402a-82c7-7de62fe91dff/7eeb67e6-b678-4ad5-b1f2-da2d9412fd6e"
-					(reference "C20")
+					(reference "C19")
 					(unit 1)
 				)
@@
 		(on_board yes)
 		(dnp no)
-		(property "Reference" "C18"
+		(property "Reference" "C16"
 			(at 185.42 42.545 0)
 			(effects
@@
 			)
 		)
-		(property "Footprint" ""
+		(property "Footprint" "Capacitor_SMD:C_0603_1608Metric"
 			(at 190.5 44.45 0)
 			(effects
@@
 			(project "Piezo module"
 				(path "/0a58466e-2312-402a-82c7-7de62fe91dff/7eeb67e6-b678-4ad5-b1f2-da2d9412fd6e"
-					(reference "C18")
+					(reference "C16")
 					(unit 1)
 				)
@@
 		(on_board yes)
 		(dnp no)
-		(property "Reference" "C19"
+		(property "Reference" "C15"
 			(at 146.685 42.545 0)
 			(effects
@@
 			)
 		)
-		(property "Footprint" ""
+		(property "Footprint" "Capacitor_SMD:C_0603_1608Metric"
 			(at 144.78 44.45 0)
 			(effects
@@
 			(project "Piezo module"
 				(path "/0a58466e-2312-402a-82c7-7de62fe91dff/7eeb67e6-b678-4ad5-b1f2-da2d9412fd6e"
-					(reference "C19")
+					(reference "C15")
 					(unit 1)
 				)
@@
 		(on_board yes)
 		(dnp no)
-		(property "Reference" "#PWR016"
+		(property "Reference" "#PWR011"
 			(at 123.825 41.91 0)
 			(effects
@@
 			(project "Piezo module"
 				(path "/0a58466e-2312-402a-82c7-7de62fe91dff/7eeb67e6-b678-4ad5-b1f2-da2d9412fd6e"
-					(reference "#PWR016")
+					(reference "#PWR011")
 					(unit 1)
 				)
@@
 		(on_board yes)
 		(dnp no)
-		(property "Reference" "#PWR015"
+		(property "Reference" "#PWR012"
 			(at 34.925 59.69 0)
 			(effects
@@
 			(project "Piezo module"
 				(path "/0a58466e-2312-402a-82c7-7de62fe91dff/7eeb67e6-b678-4ad5-b1f2-da2d9412fd6e"
-					(reference "#PWR015")
+					(reference "#PWR012")
 					(unit 1)
 				)
@@
 		(on_board yes)
 		(dnp no)
-		(property "Reference" "C17"
+		(property "Reference" "C13"
 			(at 91.44 37.465 0)
 			(effects
@@
 			)
 		)
-		(property "Footprint" ""
+		(property "Footprint" "Capacitor_SMD:C_0603_1608Metric"
 			(at 89.535 39.37 0)
 			(effects
@@
 			(project "Piezo module"
 				(path "/0a58466e-2312-402a-82c7-7de62fe91dff/7eeb67e6-b678-4ad5-b1f2-da2d9412fd6e"
-					(reference "C17")
+					(reference "C13")
 					(unit 1)
 				)
@@
 		(on_board yes)
 		(dnp no)
-		(property "Reference" "C14"
+		(property "Reference" "C18"
 			(at 55.88 43.18 0)
 			(effects
@@
 			)
 		)
-		(property "Footprint" ""
+		(property "Footprint" "Capacitor_SMD:C_0603_1608Metric"
 			(at 62.865 45.085 0)
 			(effects
@@
 			(project "Piezo module"
 				(path "/0a58466e-2312-402a-82c7-7de62fe91dff/7eeb67e6-b678-4ad5-b1f2-da2d9412fd6e"
-					(reference "C14")
+					(reference "C18")
 					(unit 1)
 				)
@@
 		(on_board yes)
 		(dnp no)
-		(property "Reference" "C15"
+		(property "Reference" "C17"
 			(at 36.83 43.18 0)
 			(effects
@@
 			)
 		)
-		(property "Footprint" ""
+		(property "Footprint" "Capacitor_SMD:C_0603_1608Metric"
 			(at 34.925 45.085 0)
 			(effects
@@
 			(project "Piezo module"
 				(path "/0a58466e-2312-402a-82c7-7de62fe91dff/7eeb67e6-b678-4ad5-b1f2-da2d9412fd6e"
-					(reference "C15")
+					(reference "C17")
 					(unit 1)
 				)
@@
 		(dnp no)
 		(fields_autoplaced yes)
-		(property "Reference" "U6"
+		(property "Reference" "U4"
 			(at 48.895 31.75 0)
 			(effects
@@
 			(project "Piezo module"
 				(path "/0a58466e-2312-402a-82c7-7de62fe91dff/7eeb67e6-b678-4ad5-b1f2-da2d9412fd6e"
-					(reference "U6")
+					(reference "U4")
 					(unit 1)
 				)
@@
 		(on_board yes)
 		(dnp no)
-		(property "Reference" "C16"
+		(property "Reference" "C14"
 			(at 110.49 37.465 0)
 			(effects
@@
 			)
 		)
-		(property "Footprint" ""
+		(property "Footprint" "Capacitor_SMD:C_0603_1608Metric"
 			(at 117.475 39.37 0)
 			(effects
@@
 			(project "Piezo module"
 				(path "/0a58466e-2312-402a-82c7-7de62fe91dff/7eeb67e6-b678-4ad5-b1f2-da2d9412fd6e"
-					(reference "C16")
+					(reference "C14")
 					(unit 1)
 				)
@@
 		(dnp no)
 		(fields_autoplaced yes)
-		(property "Reference" "U5"
+		(property "Reference" "U6"
 			(at 103.505 50.8 0)
 			(effects
@@
 			(project "Piezo module"
 				(path "/0a58466e-2312-402a-82c7-7de62fe91dff/7eeb67e6-b678-4ad5-b1f2-da2d9412fd6e"
-					(reference "U5")
-					(unit 1)
-				)
+					(reference "U6")
+					(unit 1)
+				)

Commit message: Bugfix
Parts:
- added D4, D5: PMEG2020EH, Diode_SMD:D_SOD-123F, symbol Device:D_Schottky
Connections:
- net GND: now also C15.2, C16.2, C19.2, U5.2 (GND)
- net VDD_7V0: now also D4.2 (A); no longer C15.1, U5.1 (VIN), U5.3 (INH)
- new net: C15.1, D4.1 (K), D5.1 (K), U5.1 (VIN), U5.3 (INH)
- new net VDD_5V_USB: D5.2 (A)
Other:
- moved on the sheet: C15, C16, C19, U5

Commit message: Minor fixes
Other:
- moved on the sheet: C15, C16, C19, D4, D5, U5
