File: Hardware/CAN sensor net/Piezo module/Piezo module.kicad_sch (KiCad schematic)
At the start: 40 parts, among them SW1 SW_Push, SW2 SW_SPDT, U1 SN65HVD230, U2 STM32F103C8Tx, U3 W25Q32FVSSIG, Y1 16MHz

Commit message: Piezo concept (full)
Parts:
- added H1, H2: MountingHole, MountingHole:MountingHole_2.2mm_M2_Pad_Via, symbol Mechanical:MountingHole
- added TP5, TP6, TP7: TestPoint, TestPoint:TestPoint_Pad_D1.0mm, symbol Connector:TestPoint
- D2: footprint LED_SMD:LED_Cree-PLCC4_3.2x2.8mm_CCW -> LED_SMD:LED_RGB_Wuerth-PLCC4_3.2x2.8mm_150141M173100
Connections:
- net ADC_CS: now also U2.14 (PA4)
- net ADC_DRDY: now also U2.18 (PB0)
- net ADDR_0: now also U2.22 (PB11)
- net ADDR_1: now also U2.25 (PB12)
- net ADDR_2: now also U2.26 (PB13)
- net ADDR_3: now also U2.27 (PB14)
- net ADDR_4: now also U2.4 (PC15)
- net CAN_RX: now also U2.45 (PB8)
- net CAN_TX: now also U2.46 (PB9)
- net FLASH_CS: now also U2.2 (PC13)
- net LED: now also U2.40 (PB4)
- net LED_RGB_BLUE: now also U2.11 (PA1)
- net LED_RGB_GREEN: now also U2.38 (PA15)
- net LED_RGB_RED: now also U2.10 (PA0)
- net SPI_CLK: now also U2.15 (PA5)
- net SPI_MISO: now also U2.16 (PA6)
- net SPI_MOSI: now also U2.17 (PA7)
- net UART1_RX: now also U2.43 (PB7)
- net UART1_TX: now also U2.42 (PB6)
- net VBUS_DETECT: now also U2.20 (PB2)
- net SYS_JTMS-SWDIO: now reaches U2.34 (PA13)
- net SYS_JTMS-SWDIO: now also TP7.1
- net SYS_JTCK-SWCLK: now reaches U2.37 (PA14)
- net SYS_JTCK-SWCLK: now also TP6.1
- net SYS_JTDO-SWO: now reaches U2.39 (PB3)
- net SYS_JTDO-SWO: now also TP5.1
- net CAN_H renamed CAN_+
- net CAN_+: now also JP3.1 (A); no longer R13.1
- net CAN_L renamed CAN_-
- net CAN_-: now also R13.1; no longer JP3.1 (A)
Other:
- moved on the sheet: JP3, R13

Commit message: Finished piezo board
Parts:
- TP5, TP6, TP7: footprint TestPoint:TestPoint_Pad_D1.0mm -> TestPoint:TestPoint_THTPad_D1.0mm_Drill0.5mm
Changed lines of the file:
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@@
 	)
 	(junction
+		(at 200.025 109.22)
+		(diameter 0)
+		(color 0 0 0 0)
+	)
+	(junction
 		(at 274.955 118.11)
 		(diameter 0)
@@
 	)
 	(junction
-		(at 200.025 109.22)
-		(diameter 0)
-		(color 0 0 0 0)
-	)
-	(junction
 		(at 168.275 127)
 		(diameter 0)
@@
 	(wire
 		(pts
+			(xy 200.025 110.49) (xy 200.025 109.22)
+		)
+		(stroke
+			(width 0)
+			(type default)
+		)
+	)
+	(wire
+		(pts
 			(xy 245.11 72.39) (xy 245.11 80.01)
 		)
@@
 		)
 	)
-	(polyline
+	(wire
 		(pts
-			(xy 173.99 138.43) (xy 127 138.43)
+			(xy 200.025 109.22) (xy 203.835 109.22)
 		)
 		(stroke
@@
 		)
 	)
-	(wire
+	(polyline
 		(pts
-			(xy 259.715 42.545) (xy 259.715 43.815)
+			(xy 173.99 138.43) (xy 127 138.43)
 		)
 		(stroke
@@
 	(wire
 		(pts
-			(xy 200.025 118.11) (xy 200.025 118.745)
+			(xy 259.715 42.545) (xy 259.715 43.815)
 		)
 		(stroke
@@
 	(wire
 		(pts
+			(xy 200.025 118.11) (xy 200.025 118.745)
+		)
+		(stroke
+			(width 0)
+			(type default)
+		)
+	)
+	(wire
+		(pts
 			(xy 174.625 35.56) (xy 167.005 35.56)
 		)
@@
 	(wire
 		(pts
-			(xy 200.025 109.22) (xy 203.835 109.22)
-		)
-		(stroke
-			(width 0)
-			(type default)
-		)
-	)
-	(wire
-		(pts
 			(xy 140.97 35.56) (xy 140.97 38.1)
 		)
@@
 	(wire
 		(pts
-			(xy 200.025 110.49) (xy 200.025 109.22)
-		)
-		(stroke
-			(width 0)
-			(type default)
-		)
-	)
-	(wire
-		(pts
 			(xy 253.365 106.045) (xy 253.365 107.315)
 		)
@@
 			)
 		)
-		(property "Footprint" "TestPoint:TestPoint_Pad_D1.0mm"
+		(property "Footprint" "TestPoint:TestPoint_THTPad_D1.0mm_Drill0.5mm"
 			(at 96.52 179.705 0)
 			(effects
@@
 			)
 		)
-		(property "Footprint" "TestPoint:TestPoint_Pad_D1.0mm"
+		(property "Footprint" "TestPoint:TestPoint_THTPad_D1.0mm_Drill0.5mm"
 			(at 96.52 182.245 0)
 			(effects
@@
 			)
 		)
-		(property "Footprint" "TestPoint:TestPoint_Pad_D1.0mm"
+		(property "Footprint" "TestPoint:TestPoint_THTPad_D1.0mm_Drill0.5mm"
 			(at 96.52 184.785 0)
 			(effects
