File: Hardware/CAN sensor net/Piezo module/Piezo module.kicad_sch (KiCad schematic)
At the start: 45 parts, among them SW1 SW_Push, SW2 SW_SPDT, U1 SN65HVD230, U2 STM32F103C8Tx, U3 W25Q32FVSSIG, Y1 16MHz

Commit message: Piezo production
Connections:
- net ADDR_0: now also JP6.2 (B), R8.1, U2.4 (PC15); no longer JP1.2 (B), R12.1, U2.22 (PB11)
- net ADDR_1: now also JP5.2 (B), R9.1, U2.27 (PB14); no longer JP2.2 (B), R11.1, U2.25 (PB12)
- net ADDR_3: now also JP2.2 (B), R11.1, U2.25 (PB12); no longer JP5.2 (B), R9.1, U2.27 (PB14)
- net ADDR_4: now also JP1.2 (B), R12.1, U2.22 (PB11); no longer JP6.2 (B), R8.1, U2.4 (PC15)
- net GND: now also SW2.MP

Commit message: Master and Piezo fixes
Parts:
- D2: footprint LED_SMD:LED_RGB_Wuerth-PLCC4_3.2x2.8mm_150141M173100 -> user_lib:LED_RGB_promelec
Connections:
- net LED_RGB_BLUE: now also R5.2; no longer R2.2
- net LED_RGB_RED: now also R2.2; no longer R5.2
- net VDD_3V3: now also D2.2 (A); no longer D2.4 (A)
- net at D2.1 (RK): now also R2.1; no longer R5.1
- net at R4.1: now also D2.4 (GK); no longer D2.2 (GK)
- net at D2.3 (BK): now also R5.1; no longer R2.1
Other:
- moved on the sheet: D2
