File: Hardware/CAN sensor net/Piezo module/piezo.kicad_sch (KiCad schematic)
At the start: 13 parts, among them J4 532610271, U8 TL072, U9 ADS1120-PW

Commit message: Bugfix
Parts:
- J4: footprint (none) -> Connector_Molex:Molex_PicoBlade_53261-0271_1x02-1MP_P1.25mm_Horizontal
Other:
- moved on the sheet: U8C
Changed lines of the file:
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@@
-	(wire
-		(pts
-			(xy 50.165 46.355) (xy 50.165 49.53)
-		)
-		(stroke
-			(width 0)
-			(type default)
-		)
-	)
 	(wire
 		(pts
@@
 		(pts
 			(xy 50.8 78.74) (xy 52.705 78.74)
-		)
-		(stroke
-			(width 0)
-			(type default)
-		)
-	)
-	(wire
-		(pts
-			(xy 34.925 52.07) (xy 34.925 49.53)
 		)
 		(stroke
@@
 	(text "BZX84C3V3"
 		(exclude_from_sim no)
-		(at 159.385 67.31 90)
+		(at 170.815 71.12 0)
 		(effects
 			(font
@@
 	(global_label "VDD_5V0"
 		(shape input)
-		(at 50.165 46.355 90)
+		(at 259.715 65.405 90)
 		(fields_autoplaced yes)
 		(effects
@@
 		)
 		(property "Intersheetrefs" "${INTERSHEET_REFS}"
-			(at 50.165 35.266 90)
+			(at 259.715 54.316 90)
 			(effects
 				(font
@@
 		)
 	)
+	(global_label "VDD_-5V0"
+		(shape input)
+		(at 259.715 80.645 270)
+		(fields_autoplaced yes)
+		(effects
+			(font
+				(size 1.27 1.27)
+			)
+			(justify right)
+		)
+		(property "Intersheetrefs" "${INTERSHEET_REFS}"
+			(at 259.715 93.3064 90)
+			(effects
+				(font
+					(size 1.27 1.27)
+				)
+				(justify right)
+				(hide yes)
+			)
+		)
+	)
 	(global_label "SPI_MISO"
 		(shape input)
@@
 				)
 				(justify left)
-				(hide yes)
-			)
-		)
-	)
-	(global_label "VDD_-5V0"
-		(shape input)
-		(at 34.925 52.07 270)
-		(fields_autoplaced yes)
-		(effects
-			(font
-				(size 1.27 1.27)
-			)
-			(justify right)
-		)
-		(property "Intersheetrefs" "${INTERSHEET_REFS}"
-			(at 34.925 64.7314 90)
-			(effects
-				(font
-					(size 1.27 1.27)
-				)
-				(justify right)
 				(hide yes)
 			)
@@
 			)
 		)
-		(property "Footprint" ""
+		(property "Footprint" "Connector_Molex:Molex_PicoBlade_53261-0271_1x02-1MP_P1.25mm_Horizontal"
 			(at 45.72 76.2 0)
 			(effects
@@
 	(symbol
 		(lib_id "Amplifier_Operational:TL072")
-		(at 42.545 52.07 270)
+		(at 262.255 73.025 0)
 		(unit 3)
 		(exclude_from_sim no)
@@
 		(dnp no)
 		(property "Reference" "U8"
-			(at 39.6875 51.7524 90)
+			(at 261.9374 75.8825 0)
 			(effects
 				(font
@@
 		)
 		(property "Value" "TL072"
-			(at 39.6875 54.2924 90)
+			(at 261.62 71.755 0)
 			(effects
 				(font
@@
 		)
 		(property "Footprint" ""
-			(at 42.545 52.07 0)
+			(at 262.255 73.025 0)
 			(effects
 				(font
@@
 		)
 		(property "Datasheet" "http://www.ti.com/lit/ds/symlink/tl071.pdf"
-			(at 42.545 52.07 0)
+			(at 262.255 73.025 0)
 			(effects
 				(font
@@
 		)
 		(property "Description" "Dual Low-Noise JFET-Input Operational Amplifiers, DIP-8/SOIC-8"
-			(at 42.545 52.07 0)
-			(effects
-				(font
+			(at 262.255 73.025 0)
+			(effects
+				(font

Commit message: updated piezo module
Other:
- note added: "Мб лучше зафильтровать питание аналоговое"
Changed lines of the file:
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@@
+		)
+	)
+	(text "Мб лучше зафильтровать питание аналоговое"
+		(exclude_from_sim no)
+		(at 233.68 52.07 0)
+		(effects
+			(font
+				(size 1.27 1.27)
+			)
 		)
 	)

Commit message: added band pass filter to piezo board
Parts:
- added C24: 10n, Capacitor_SMD:C_0603_1608Metric, symbol Device:C_Small
- added C25: 1u, Capacitor_SMD:C_0603_1608Metric, symbol Device:C_Small
- added C26: 100n, Capacitor_SMD:C_0603_1608Metric, symbol Device:C_Small
- added C27: 1u, symbol Device:C_Small
- added L2: 27n, symbol Device:L_Small
- added R23, R24: 1k, symbol Device:R_Small
- C22: value 100n -> 100u; footprint Capacitor_SMD:C_0603_1608Metric -> (none)
Connections:
- net GND: now also C24.1, C25.1, C26.1, C27.1, R24.1; no longer C22.1
- net VDD_3V3: now also C24.2, C25.2, C26.2, L2.2; no longer C22.2, U9.12 (AVDD)
- net at RV1.1: now also C22.2, C27.2, R24.2; no longer J4.1 (Pin_1)
- new net: C22.1, R23.2
- new net: J4.1 (Pin_1), R23.1
- new net: L2.1, U9.12 (AVDD)
Other:
- note added: "C1"
- note added: "C2"
- note added: "R1"
- note added: "R2"
- note added: "VDDA"
- note added: "f_low = 0.5*pi*R1*C1 f_high = 0.5*pi*R2*C2"
- note removed: "Мб лучше зафильтровать питание аналоговое"
- moved on the sheet: C21, D2, D6, J4, R10, R11, R12, R13, R9, RV1, U8A, U8B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

Commit message: updated piezo board schematics
Parts:
- removed C22: 100u, symbol Device:C_Small
- removed C27: 1u, symbol Device:C_Small
- removed L2: 27n, symbol Device:L_Small
- removed R23, R24: 1k, symbol Device:R_Small
- added C25: 10u, Capacitor_SMD:C_0603_1608Metric, symbol Device:C_Small
- added C26: 1u, Capacitor_SMD:C_0603_1608Metric, symbol Device:C_Small
- added L1: 27n, Inductor_SMD:L_0603_1608Metric, symbol Device:L_Small
- added R19: 470, Resistor_SMD:R_0603_1608Metric, symbol Device:R_Small
- added R22: 10k, Resistor_SMD:R_0603_1608Metric, symbol Device:R_Small
- added TP1, TP2, TP3: Signal, TestPoint:TestPoint_Bridge_Pitch2.54mm_Drill1.0mm, symbol Connector:TestPoint
- added TP4: GND, TestPoint:TestPoint_Bridge_Pitch5.08mm_Drill1.3mm, symbol Connector:TestPoint
- R16: renamed from R12; footprint (none) -> Resistor_SMD:R_0603_1608Metric
- R17: renamed from R13; footprint (none) -> Resistor_SMD:R_0603_1608Metric
- R18: renamed from R11; footprint (none) -> Resistor_SMD:R_0603_1608Metric
- R20: renamed from R9; footprint (none) -> Resistor_SMD:R_0603_1608Metric
- R21: renamed from R10; footprint (none) -> Resistor_SMD:R_0603_1608Metric
- RV1: footprint (none) -> Potentiometer_SMD:Potentiometer_Bourns_3224W_Vertical
- U8: footprint (none) -> Package_SO:SO-8_3.9x4.9mm_P1.27mm
- renumbered C24 to C21, C25 to C22, C26 to C23, C21 to C24, D6 to D4, D2 to D5, J4 to J5
Connections:
- net GND: now also C26.1, R22.1, TP4.1
- net VDD_3V3: now also L1.2; no longer C21.2, C22.2, C23.2
- net at RV1.1: now also C26.2, R19.2, TP3.1
- net at J5.1 (Pin_1): now also C25.1, TP2.1
- net at D4.1 (A), D5.3 (K), R18.2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: now also TP1.1
- net at U9.12 (AVDD): now also C21.2, C22.2, C23.2, L1.1
- new net: C25.2, R19.1, R22.2
Other:
- note added: "<-INT"
- note removed: "C1"
- note removed: "C2"
- note removed: "R1"
- note removed: "R2"
- note removed: "f_low = 0.5*pi*R1*C1 f_high = 0.5*pi*R2*C2"

Commit message: Bugfix
Parts:
- TP4: footprint TestPoint:TestPoint_Bridge_Pitch5.08mm_Drill1.3mm -> TestPoint:TestPoint_Bridge_Pitch6.35mm_Drill1.3mm
- renumbered D4 to D6, D5 to D7
Changed lines of the file:
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@@
 		(dnp no)
 		(fields_autoplaced yes)
-		(property "Reference" "D4"
+		(property "Reference" "D6"
 			(at 185.42 78.7399 90)
 			(effects
@@
 			(project "Piezo module"
 				(path "/0a58466e-2312-402a-82c7-7de62fe91dff/74f4a990-612a-4918-b03d-ff48b2807170"
-					(reference "D4")
+					(reference "D6")
 					(unit 1)
 				)
@@
 		(dnp no)
 		(fields_autoplaced yes)
-		(property "Reference" "D5"
+		(property "Reference" "D7"
 			(at 185.42 91.4399 90)
 			(effects
@@
 			(project "Piezo module"
 				(path "/0a58466e-2312-402a-82c7-7de62fe91dff/74f4a990-612a-4918-b03d-ff48b2807170"
-					(reference "D5")
+					(reference "D7")
 					(unit 1)
 				)
@@
 			)
 		)
-		(property "Footprint" "TestPoint:TestPoint_Bridge_Pitch5.08mm_Drill1.3mm"
+		(property "Footprint" "TestPoint:TestPoint_Bridge_Pitch6.35mm_Drill1.3mm"
 			(at 45.72 111.125 0)
 			(effects

Commit message: Minor fixes
Connections:
- net GND: now also U8.5 (+); no longer U8.3 (+)
- net at R16.1, R17.1: now also U8.3 (+); no longer U8.5 (+)
- net at R20.2, R21.1: now also U8.2 (-); no longer U8.6 (-)
- net at R18.1, R21.2: now also U8.1; no longer U8.7
- net at R20.1, RV1.3: now also U8.7; no longer U8.1
- net at RV1.2: now also U8.6 (-); no longer U8.2 (-)
Other:
- moved on the sheet: U8A, U8B

Commit message: Finished piezo board
Connections:
- net GND: now also J5.1 (Pin_1); no longer J5.2 (Pin_2)
- net at C25.1, TP2.1: now also J5.2 (Pin_2); no longer J5.1 (Pin_1)
Other:
- moved on the sheet: J5
Changed lines of the file:
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@@
 	(symbol
 		(lib_id "Connector_Generic:Conn_01x02")
-		(at 34.925 88.9 0)
-		(mirror y)
+		(at 34.925 91.44 180)
 		(unit 1)
 		(exclude_from_sim no)
@@
 		(dnp no)
 		(property "Reference" "J5"
-			(at 31.75 88.8999 0)
+			(at 31.75 91.4401 0)
 			(effects
 				(font
@@
 		)
 		(property "Value" "532610271"
-			(at 31.75 91.4399 0)
+			(at 31.75 88.9001 0)
 			(effects
 				(font
@@
 		)
 		(property "Footprint" "Connector_Molex:Molex_PicoBlade_53261-0271_1x02-1MP_P1.25mm_Horizontal"
-			(at 34.925 88.9 0)
+			(at 34.925 91.44 0)
 			(effects
 				(font
@@
 		)
 		(property "Datasheet" "~"
-			(at 34.925 88.9 0)
+			(at 34.925 91.44 0)
 			(effects
 				(font
@@
 		)
 		(property "Description" "Generic connector, single row, 01x02, script generated (kicad-library-utils/schlib/autogen/connector/)"
-			(at 34.925 88.9 0)
+			(at 34.925 91.44 0)
 			(effects
 				(font
