File: Hardware/CAN sensor net/Piezo module/Piezo module.kicad_pcb (KiCad board)
At the start: 2 copper layers, 40 parts, among them J1 532610671, J2 532610671, J4 532610271, U1 STM32F103C8Tx, U2 SN65HVD230, U3 W25Q32FVSSIG, U4 USBLC6-2SC6, U5 L79L05_SOT89, U6 L78L05_SOT89, U7 LD3985M33R_SOT23, U9 ADS1120-PW, Y1 16MHz

Commit message: updated piezo board schematics
Parts:
- added C13: 330n, Capacitor_SMD:C_0603_1608Metric, F.Cu at (70.0, 78.1)
- added C14: 100n, Capacitor_SMD:C_0603_1608Metric, F.Cu at (70.0, 80.7)
- added C15: 1u, Capacitor_SMD:C_0603_1608Metric, F.Cu at (70.0, 83.2)
- added C16: 1u, Capacitor_SMD:C_0603_1608Metric, F.Cu at (70.0, 85.7)
- added C17: 330n, Capacitor_SMD:C_0603_1608Metric, F.Cu at (70.0, 88.2)
- added C18: 100n, Capacitor_SMD:C_0603_1608Metric, F.Cu at (70.0, 90.7)
- added C19: 10n, Capacitor_SMD:C_0603_1608Metric, F.Cu at (70.0, 93.2)
- added C21: 10n, Capacitor_SMD:C_0603_1608Metric, F.Cu at (95.7, 78.4)
- added C23: 100n, Capacitor_SMD:C_0603_1608Metric, F.Cu at (95.7, 83.4)
- added C25: 10u, Capacitor_SMD:C_0603_1608Metric, F.Cu at (76.0, 78.1)
- added C26: 1u, Capacitor_SMD:C_0603_1608Metric, F.Cu at (76.0, 80.7)
- added J3: USB_B_Micro, user_lib:U-F-M5DD-W-2-SUS, F.Cu at (98.5, 105.1)
- added J4: 530470310, Connector_Molex:Molex_PicoBlade_53261-0371_1x03-1MP_P1.25mm_Horizontal, F.Cu at (99.6, 98.4)
- added JP1: SolderJumper_2_Open, Jumper:SolderJumper-2_P1.3mm_Open_RoundedPad1.0x1.5mm, F.Cu at (80.4, 78.9)
- added JP2: SolderJumper_2_Open, Jumper:SolderJumper-2_P1.3mm_Open_RoundedPad1.0x1.5mm, F.Cu at (80.4, 82.5)
- added JP3: SolderJumper_2_Open, Jumper:SolderJumper-2_P1.3mm_Open_RoundedPad1.0x1.5mm, F.Cu at (80.4, 86.0)
- added JP4: SolderJumper_2_Open, Jumper:SolderJumper-2_P1.3mm_Open_RoundedPad1.0x1.5mm, F.Cu at (80.4, 89.5)
- added JP5: SolderJumper_2_Open, Jumper:SolderJumper-2_P1.3mm_Open_RoundedPad1.0x1.5mm, F.Cu at (80.4, 93.1)
- added JP6: SolderJumper_2_Open, Jumper:SolderJumper-2_P1.3mm_Open_RoundedPad1.0x1.5mm, F.Cu at (80.4, 96.7)
- added L1: 27n, Inductor_SMD:L_0603_1608Metric, F.Cu at (92.2, 78.4)
- added R1: 10k, Resistor_SMD:R_0603_1608Metric, F.Cu at (84.6, 78.4)
- added R10: 10k, Resistor_SMD:R_0603_1608Metric, F.Cu at (84.6, 88.4)
- added R11: 10k, Resistor_SMD:R_0603_1608Metric, F.Cu at (84.6, 90.9)
- added R12: 10k, Resistor_SMD:R_0603_1608Metric, F.Cu at (84.6, 93.4)
- added R16: 1k, Resistor_SMD:R_0603_1608Metric, F.Cu at (95.7, 88.4)
- added R17: 330, Resistor_SMD:R_0603_1608Metric, F.Cu at (95.7, 90.9)
- added R18: 100k, Resistor_SMD:R_0603_1608Metric, F.Cu at (99.7, 78.4)
- added R19: 470, Resistor_SMD:R_0603_1608Metric, F.Cu at (99.7, 80.9)
- added R20: 1k, Resistor_SMD:R_0603_1608Metric, F.Cu at (99.7, 83.4)
- added R21: 1k, Resistor_SMD:R_0603_1608Metric, F.Cu at (99.7, 85.9)
- added R22: 10k, Resistor_SMD:R_0603_1608Metric, F.Cu at (99.7, 88.4)
- added R7: 4k7, Resistor_SMD:R_0603_1608Metric, F.Cu at (84.6, 80.9)
- added R8: 10k, Resistor_SMD:R_0603_1608Metric, F.Cu at (84.6, 83.4)
- added R9: 10k, Resistor_SMD:R_0603_1608Metric, F.Cu at (84.6, 85.9)
- added RV1: 3224W-1-103E, Potentiometer_SMD:Potentiometer_Bourns_3224W_Vertical, F.Cu at (104.9, 86.7)
- added SW1: SW_Push, user_lib:button_small, F.Cu at (88.8, 91.3)
- added SW2: SW_SPDT, Button_Switch_SMD:SW_SPDT_PCM12, F.Cu at (86.8, 71.6)
- added TP1: Signal, TestPoint:TestPoint_Bridge_Pitch2.54mm_Drill1.0mm, F.Cu at (74.7, 100.8)
- added TP2: Signal, TestPoint:TestPoint_Bridge_Pitch2.54mm_Drill1.0mm, F.Cu at (86.3, 100.8)
- added TP3: Signal, TestPoint:TestPoint_Bridge_Pitch2.54mm_Drill1.0mm, F.Cu at (80.5, 100.8)
- added TP4: GND, TestPoint:TestPoint_Bridge_Pitch5.08mm_Drill1.3mm, F.Cu at (66.1, 100.8)
- added U8: TL072, Package_SO:SO-8_3.9x4.9mm_P1.27mm, F.Cu at (105.9, 80.5)
- C22: value 100n -> 1u
- moved C22 51.0 mm to (95.7, 80.9)
- renumbered C9 to C1, C13 to C10, C5 to C11, C10 to C12, C1 to C2, C11 to C20, C21 to C24, C2 to C3, C3 to C4, C4 to C5, C12 to C9, D3 to D1, D1 to D2, D4 to D3, D6 to D4, D2 to D5, J4 to J5, R1 to R13, R5 to R14, R8 to R15, R6 to R3, R3 to R4, R4 to R5, R7 to R6, U2 to U1, U1 to U2, U6 to U4, U7 to U5, U5 to U6, U4 to U7
Connections:
- C22 pad 2: VDD_3V3 -> Net-(U9-AVDD)
- J1 pad 3: CAN_H -> CAN_L-
- J1 pad 4: CAN_L -> CAN_H+
- J2 pad 3: CAN_H -> CAN_L-
- J2 pad 4: CAN_L -> CAN_H+
- R13 pad 2: CAN_L -> Net-(JP3-B)
- U7 pad 5: VDD_5V_VBUS -> VDD_5V_USB
- U9 pad 12: VDD_3V3 -> Net-(U9-AVDD)
Other:
- board text added: "Проверь распиновку у преобразователей"

Commit message: Bugfix
Parts:
- TP4: footprint TestPoint:TestPoint_Bridge_Pitch5.08mm_Drill1.3mm -> TestPoint:TestPoint_Bridge_Pitch6.35mm_Drill1.3mm
- moved SW2 77.0 mm to (86.6, 148.6), turned to 90 degrees
- moved U1 71.7 mm to (80.0, 147.7)
- moved D1 71.5 mm to (66.1, 144.8)
- moved D3 71.3 mm to (66.2, 148.0)
- moved RV1 71.1 mm to (71.1, 149.3)
- moved U3 69.7 mm to (83.0, 140.1)
- moved D2 68.7 mm to (73.6, 143.3)
- moved U8 57.8 mm to (81.8, 133.0)
- moved J5 54.1 mm to (111.4, 147.5), turned to 90 degrees
- moved SW1 50.6 mm to (63.9, 135.4)
- moved J4 48.6 mm to (104.0, 146.8), turned to -90 degrees
- moved J3 41.4 mm to (71.0, 136.0)
- moved J1 34.1 mm to (104.0, 134.3), turned to -90 degrees
- moved U9 27.4 mm to (127.1, 88.8)
- moved TP4 27.3 mm to (64.8, 128.0)
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Connections:
- J4 pad 1: UART1_RX -> GND
- J4 pad 3: GND -> UART1_RX
- SW2 pad 1: VDD_3V3 -> GND
- SW2 pad 3: GND -> VDD_3V3
Other:
- board outline added: 99.8 x 90.1 mm
- board text removed: "Проверь распиновку у преобразователей"

Commit message: Minor fixes
Parts:
- added D4: PMEG2020EH, Diode_SMD:D_SOD-123F, F.Cu at (87.3, 111.5)
- added D5: PMEG2020EH, Diode_SMD:D_SOD-123F, F.Cu at (87.3, 114.8)
- moved C24 66.7 mm to (70.3, 96.2), turned to 180 degrees
- moved D7 61.3 mm to (75.5, 91.6)
- moved D6 61.1 mm to (75.9, 95.5)
- moved R15 56.4 mm to (75.8, 88.9)
- moved C20 56.4 mm to (75.8, 83.9)
- moved R14 56.4 mm to (75.8, 86.4)
- moved U4 53.8 mm to (91.1, 96.2)
- moved U6 53.1 mm to (90.8, 90.3)
- moved U5 50.3 mm to (103.5, 98.1)
- moved Y1 37.4 mm to (97.7, 95.6)
- moved U7 34.4 mm to (91.2, 83.8)
- moved J4 24.7 mm to (118.0, 126.4)
- moved J5 24.7 mm to (125.4, 127.1)
- moved J1 24.7 mm to (118.0, 113.9)
- moved J2 24.7 mm to (125.4, 113.9)
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- renumbered D4 to D6, D5 to D7
Connections:
- C15 pad 1: VDD_7V0 -> Net-(D4-K)
- C15 pad 2: Net-(U5-GND) -> GND
- C16 pad 2: Net-(U5-GND) -> GND
- C19 pad 2: Net-(U5-GND) -> GND
- R16 pad 1: Net-(U8B-+) -> Net-(U8A-+)
- R17 pad 1: Net-(U8B-+) -> Net-(U8A-+)
- R20 pad 2: Net-(U8B--) -> Net-(U8A--)
- R21 pad 1: Net-(U8B--) -> Net-(U8A--)
- RV1 pad 2: Net-(U8A--) -> Net-(U8B--)
- U5 pad 1: VDD_7V0 -> Net-(D4-K)
- U5 pad 2: Net-(U5-GND) -> GND
- U5 pad 3: VDD_7V0 -> Net-(D4-K)
- U8 pad 1: Net-(R20-Pad1) -> Net-(R18-Pad1)
- U8 pad 3: GND -> Net-(U8A-+)
- U8 pad 5: Net-(U8B-+) -> GND
- U8 pad 7: Net-(R18-Pad1) -> Net-(R20-Pad1)
Routing:
- net Net-(R20-Pad1): track 0.00 -> 6.30 mm
- net Net-(R18-Pad1): track 0.00 -> 1.85 mm
- net Net-(U8A--): track 0.00 -> 1.82 mm
Other:
- board size 99.8 x 90.1 mm -> 69.7 x 58.2 mm
- board text added: "CAN"
- board text added: "PWR"

Commit message: Piezo concept (full)
Parts:
- added D8: PMEG2020EH, Diode_SMD:D_SOD-123F, B.Cu at (139.1, 101.3)
- added H1: MountingHole, MountingHole:MountingHole_2.2mm_M2_Pad_Via, F.Cu at (161.7, 90.8)
- added H2: MountingHole, MountingHole:MountingHole_2.2mm_M2_Pad_Via, F.Cu at (141.9, 111.1)
- added TP5: TestPoint, TestPoint:TestPoint_Pad_D1.0mm, B.Cu at (133.5, 92.0)
- added TP6: TestPoint, TestPoint:TestPoint_Pad_D1.0mm, B.Cu at (133.5, 96.0)
- added TP7: TestPoint, TestPoint:TestPoint_Pad_D1.0mm, B.Cu at (133.5, 99.2)
- C10, C15, C16, C17, C18, C19, C2, C21, C22, C23, C24, C3, C4, C5, C6, C7, C8, C9, D4, D5, D7, JP1, JP2, JP3, JP4, JP5, JP6, L1, R1, R10, R11, R12, R13, R15, R20, R21, R3, R6, R7, SW2, U2, U4, U5, U7, U9, Y1: moved to B.Cu
- D2: footprint LED_SMD:LED_Cree-PLCC4_3.2x2.8mm_CCW -> LED_SMD:LED_RGB_Wuerth-PLCC4_3.2x2.8mm_150141M173100
- moved C17 96.5 mm to (165.1, 104.7)
- moved RV1 95.7 mm to (161.5, 105.1), turned to 180 degrees
- moved C24 93.1 mm to (163.4, 98.5), turned to -90 degrees
- moved C18 93.1 mm to (162.6, 100.9), turned to 180 degrees
- moved JP1 92.7 mm to (168.0, 109.2), turned to 180 degrees
- moved C25 92.7 mm to (163.4, 109.0), turned to 90 degrees
- moved SW1 92.4 mm to (151.1, 91.8)
- moved C14 89.5 mm to (158.0, 97.1), turned to 90 degrees
- moved JP2 88.4 mm to (164.7, 109.2), turned to 180 degrees
- moved JP3 88.2 mm to (168.3, 92.4), turned to 180 degrees
- moved C26 87.7 mm to (159.0, 109.0), turned to 90 degrees
- moved D2 85.9 mm to (155.3, 105.0), turned to 180 degrees
- moved C13 85.3 mm to (154.0, 93.3), turned to -90 degrees
- moved TP1 84.8 mm to (155.2, 89.9)
- moved R11 84.4 mm to (166.3, 112.0), turned to -90 degrees
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Connections:
- J1 pad 3: CAN_L- -> CAN_-
- J1 pad 4: CAN_H+ -> CAN_+
- J1 pad MP: (no net) -> unconnected-(J1-PadMP)_0
- J2 pad 3: CAN_L- -> CAN_-
- J2 pad 4: CAN_H+ -> CAN_+
- J2 pad MP: (no net) -> unconnected-(J2-PadMP)
- J4 pad 2: UART1_TX -> Net-(D8-K)
- J4 pad MP: (no net) -> unconnected-(J4-PadMP)_0
- J5 pad MP: (no net) -> unconnected-(J5-PadMP)_0
- JP3 pad 1: CAN_L -> CAN_+
- R13 pad 1: CAN_H -> CAN_-
- U1 pad 6: CAN_L -> CAN_-
- U1 pad 7: CAN_H -> CAN_+
- U2 pad 10: unconnected-(U2-PA0-Pad10) -> LED_RGB_RED
- U2 pad 11: unconnected-(U2-PA1-Pad11) -> LED_RGB_BLUE
- U2 pad 14: unconnected-(U2-PA4-Pad14) -> ADC_CS
- U2 pad 15: unconnected-(U2-PA5-Pad15) -> SPI_CLK
- U2 pad 16: unconnected-(U2-PA6-Pad16) -> SPI_MISO
- U2 pad 17: unconnected-(U2-PA7-Pad17) -> SPI_MOSI
- U2 pad 18: unconnected-(U2-PB0-Pad18) -> ADC_DRDY
- U2 pad 2: unconnected-(U2-PC13-Pad2) -> FLASH_CS
- U2 pad 20: unconnected-(U2-PB2-Pad20) -> VBUS_DETECT
- U2 pad 22: unconnected-(U2-PB11-Pad22) -> ADDR_0
- U2 pad 25: unconnected-(U2-PB12-Pad25) -> ADDR_1
- U2 pad 26: unconnected-(U2-PB13-Pad26) -> ADDR_2
- U2 pad 27: unconnected-(U2-PB14-Pad27) -> ADDR_3
- U2 pad 34: unconnected-(U2-PA13-Pad34) -> SYS_JTMS-SWDIO
- U2 pad 37: unconnected-(U2-PA14-Pad37) -> SYS_JTCK-SWCLK
- U2 pad 38: unconnected-(U2-PA15-Pad38) -> LED_RGB_GREEN
- U2 pad 39: unconnected-(U2-PB3-Pad39) -> SYS_JTDO-SWO
- U2 pad 4: unconnected-(U2-PC15-Pad4) -> ADDR_4
- U2 pad 40: unconnected-(U2-PB4-Pad40) -> LED
- U2 pad 42: unconnected-(U2-PB6-Pad42) -> UART1_TX
- U2 pad 43: unconnected-(U2-PB7-Pad43) -> UART1_RX
- U2 pad 45: unconnected-(U2-PB8-Pad45) -> CAN_RX
- U2 pad 46: unconnected-(U2-PB9-Pad46) -> CAN_TX
Routing:
- net GND: track 0.00 -> 84.0 mm, vias 0 -> 26
- net CAN_+: track 0.00 -> 48.5 mm, vias 0 -> 1
- net VDD_3V3: track 0.00 -> 48.4 mm, vias 0 -> 13
- net VDD_7V0: track 0.00 -> 46.4 mm, vias 0 -> 5
- net CAN_-: track 0.00 -> 44.8 mm, vias 0 -> 1
- net Net-(U8A--): track 1.82 -> 37.3 mm, vias 0 -> 1
- net VDD_5V_USB: track 0.00 -> 32.9 mm, vias 0 -> 2
- net SYS_JTMS-SWDIO: track 0.00 -> 26.4 mm
- net Net-(D6-A): track 0.00 -> 25.3 mm, vias 0 -> 1
- net SYS_JTDO-SWO: track 0.00 -> 22.4 mm
- net ADDR_0: track 0.00 -> 21.3 mm
- net SPI_MISO: track 0.00 -> 20.3 mm, vias 0 -> 1
- net SYS_JTCK-SWCLK: track 0.00 -> 19.1 mm, vias 0 -> 3
- net ADDR_4: track 0.00 -> 18.6 mm, vias 0 -> 2
- net Net-(C26-Pad2): track 0.00 -> 17.9 mm
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- added copper zone on B.Cu, net GND
- added copper zone on F.Cu, net GND
- added copper zone on In2.Cu, net GND
- added copper zone on In1.Cu, net VDD_3V3
Other:
- board size 69.7 x 58.2 mm -> 38.3 x 25.1 mm
- copper layers 2 -> 4
- board text added: "+"
- board text added: "-"
- board text added: "0"
- board text added: "1"
- board text added: "2"
- board text added: "3"
- board text added: "4"
- board text added: "7V0"
- board text added: "ADC"
- board text added: "CAN_H"
- board text added: "CAN_L"
- board text added: "CLK"
- board text added: "FC1"
- board text added: "FILTER"
- board text added: "GND"
- board text added: "IN"
- board text added: "IO"
- board text added: "PIEZO"
- board text added: "RESET"
- board text added: "RX"
- board text added: "SWO"
- board text added: "TX"
- board text added: "X"
- board text added: "Y"
- board text added: "Z"
- board text added: "концепт: перетрассировать полностью проверить существующие подписи (+ подписи коннекторов и терминатора?) проверить заливки добавить MP у остальных плат"

Commit message: Update
Routing:
- net ADDR_4: track 18.6 -> 17.9 mm
- net SPI_CLK: track 11.8 -> 11.2 mm
- net VDD_7V0: track 46.4 -> 47.0 mm
- net CAN_TX: track 4.04 -> 3.46 mm
Other:
- board text added: "120R"
- board text added: "CAN_OUT"

Commit message: Finished piezo board
Parts:
- R20: moved to F.Cu
- TP5, TP6, TP7: footprint TestPoint:TestPoint_Pad_D1.0mm -> TestPoint:TestPoint_THTPad_D1.0mm_Drill0.5mm
- moved R20 8.82 mm to (158.0, 102.2), turned to 90 degrees
- moved R11 8.70 mm to (166.5, 103.3), turned to 180 degrees
- moved R21 1.59 mm to (158.4, 93.1), turned to 0 degrees
- moved R10 1.58 mm to (166.2, 111.2), turned to 0 degrees
- moved C17 1.06 mm to (164.3, 105.5), turned to -90 degrees
- moved R12 1.01 mm to (165.8, 105.5), turned to 90 degrees
- moved C1 0.88 mm to (149.8, 97.2), turned to 0 degrees
- moved R17 0.81 mm to (158.0, 99.2), turned to 90 degrees
- moved C14 0.79 mm to (158.0, 96.3)
- moved R16 0.74 mm to (155.6, 101.8)
- moved D2 0.67 mm to (154.7, 105.0)
- moved C20 0.66 mm to (147.7, 105.9), turned to 180 degrees
- moved R4 0.66 mm to (150.6, 105.9)
- moved R8 0.46 mm to (154.2, 108.1)
- moved TP6 0.40 mm to (133.9, 96.0)
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Connections:
- C25 pad 1: Net-(J5-Pin_1) -> Net-(J5-Pin_2)
- J5 pad 1: Net-(J5-Pin_1) -> GND
- J5 pad 2: GND -> Net-(J5-Pin_2)
- TP2 pad 1: Net-(J5-Pin_1) -> Net-(J5-Pin_2)
Routing:
- net GND: track 84.1 -> 37.7 mm, vias 26 -> 25
- net VDD_7V0: track 47.0 -> 15.8 mm
- net Net-(U8A--): track 37.3 -> 13.7 mm
- net Net-(J5-Pin_2): track 0.00 -> 20.1 mm
- net Net-(J5-Pin_1): track 14.9 -> 0.00 mm
- net ADDR_1: track 16.6 -> 29.1 mm
- net VDD_3V3: track 48.4 -> 60.7 mm, vias 13 -> 12
- net CAN_-: track 44.8 -> 55.2 mm
- net VDD_5V_USB: track 32.9 -> 25.3 mm
- net RCC_OSC_OUT: track 6.57 -> 0.00 mm
- net Net-(D6-A): track 25.3 -> 30.5 mm
- net VDD_-5V0: track 3.36 -> 0.00 mm
- net Net-(R18-Pad1): track 9.54 -> 12.8 mm, vias 1 -> 2
- net Net-(R20-Pad1): track 9.96 -> 12.2 mm, vias 1 -> 0
- net CAN_+: track 48.5 -> 50.6 mm
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- added copper zone on B.Cu, net ADDR_0
- added copper zone on B.Cu, net RCC_OSC_OUT
- added copper zone on F.Cu, net VDD_-5V0
- added copper zone on B.Cu, net VDD_3V3
- added copper zone on F.Cu, net VDD_3V3
- added copper zone on F.Cu, net VDD_5V_USB
- added copper zone on F.Cu, net VDD_7V0
- added copper zone on In1.Cu, net VDD_7V0
Other:
- board text added: "добавить MP у остальных плат 4 -> 0 или 0 -> 4 piezo + can out"
- board text removed: "CAN_OUT"
- board text removed: "PIEZO"
- board text removed: "концепт: перетрассировать полностью проверить существующие подписи (+ подписи коннекторов и терминатора?) проверить заливки добавить MP у остальных плат"

Commit message: Piezo production
Parts:
- added G***: LOGO, Logos:name_10_1.8, F.Cu at (144.5, 92.3)
Connections:
- J1 pad MP: unconnected-(J1-PadMP)_0 -> GND
- J2 pad MP: unconnected-(J2-PadMP) -> GND
- J4 pad MP: unconnected-(J4-PadMP)_0 -> GND
- J5 pad MP: unconnected-(J5-PadMP)_0 -> GND
- JP1 pad 2: ADDR_0 -> ADDR_4
- JP2 pad 2: ADDR_1 -> ADDR_3
- JP5 pad 2: ADDR_3 -> ADDR_1
- JP6 pad 2: ADDR_4 -> ADDR_0
- R11 pad 1: ADDR_1 -> ADDR_3
- R12 pad 1: ADDR_0 -> ADDR_4
- R8 pad 1: ADDR_4 -> ADDR_0
- R9 pad 1: ADDR_3 -> ADDR_1
- SW2 pad MP: unconnected-(SW2-PadMP)_0 -> GND
- U2 pad 22: ADDR_0 -> ADDR_4
- U2 pad 25: ADDR_1 -> ADDR_3
- U2 pad 27: ADDR_3 -> ADDR_1
- U2 pad 4: ADDR_4 -> ADDR_0
Routing:
- net ADDR_3: track 10.9 -> 29.1 mm, vias 1 -> 0
- net ADDR_1: track 29.1 -> 10.9 mm, vias 0 -> 1
- net GND: track 37.7 -> 28.1 mm, vias 25 -> 65
- net ADDR_4: track 19.2 -> 21.5 mm, vias 2 -> 0
- net ADDR_0: track 21.5 -> 19.2 mm, vias 0 -> 2
- net Net-(U9-AVDD): track 6.39 -> 8.66 mm
- net Net-(U8A--): track 13.7 -> 14.8 mm
- net unconnected-(SW2-PadMP)_0: vias 1 -> 0
- net unconnected-(SW2-PadMP): vias 1 -> 0
- net unconnected-(J5-PadMP)_0: vias 5 -> 0
- net unconnected-(J5-PadMP): vias 4 -> 0
- net unconnected-(J4-PadMP)_0: vias 5 -> 0
- net unconnected-(J4-PadMP): vias 5 -> 0
- net unconnected-(J2-PadMP)_0: vias 5 -> 0
- net unconnected-(J2-PadMP): vias 5 -> 0
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- added copper zone on B.Cu, net ADDR_4
- removed copper zone on B.Cu, net ADDR_0
Other:
- board text added: "04/24"
- board text added: "добавить MP у остальных плат"
- board text removed: "добавить MP у остальных плат 4 -> 0 или 0 -> 4 piezo + can out"

Commit message: Piezo fixes
Changed lines of the file:
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@@
 			)
 		)
-		(property ki_fp_filters "LED* LED_SMD:* LED_THT:*")
-		(sheetname "Корневой лист")
-		(sheetfile "Piezo module.kicad_sch")
 		(attr smd)
 		(fp_line
-			(start -2.285 -1.135)
-			(end -2.285 1.135)
+			(start -0.57 -0.8)
+			(end -0.57 0.8)
 			(stroke
-				(width 0.12)
-				(type solid)
-			)
-			(layer "F.SilkS")
-		)
-		(fp_line
-			(start -2.285 1.135)
-			(end 1.6 1.135)
-			(stroke
-				(width 0.12)
-				(type solid)
+				(width 0.15)
+				(type default)
 			)
 			(layer "F.SilkS")
@@
 			)
 		)
-		(property ki_fp_filters "LED* LED_SMD:* LED_THT:*")
-		(sheetname "Корневой лист")
-		(sheetfile "Piezo module.kicad_sch")
 		(attr smd)
 		(fp_line
-			(start -2.285 1.135)
-			(end 1.6 1.135)
-			(stroke
-				(width 0.12)
-				(type solid)
-			)
-			(layer "F.SilkS")
-		)
-		(fp_line
-			(start -2.285 -1.135)
-			(end -2.285 1.135)
-			(stroke
-				(width 0.12)
-				(type solid)
-			)
-			(layer "F.SilkS")
-		)
-		(fp_line
-			(start 1.6 -1.135)
-			(end -2.285 -1.135)
+			(start -0.57 -0.8)
+			(end -0.57 0.8)
 			(stroke
-				(width 0.12)
-				(type solid)
+				(width 0.15)
+				(type default)
 			)
 			(layer "F.SilkS")
@@
 			)
 		)
-		(property ki_fp_filters "LED* LED_SMD:* LED_THT:*")
-		(sheetname "Корневой лист")
-		(sheetfile "Piezo module.kicad_sch")
 		(attr smd)
 		(fp_line
-			(start -2.3 1.51)
-			(end 2.3 1.51)
+			(start 0.503 0)
+			(end 0.503 1.09)
 			(stroke
 				(width 0.12)
-				(type solid)
+				(type default)
 			)
 			(layer "F.SilkS")
 		)
 		(fp_line
-			(start -2.5 -0.7)
-			(end -2.5 -1.51)
+			(start 0.503 0)
+			(end -1.54 0)
 			(stroke
 				(width 0.12)
-				(type solid)
+				(type default)
 			)
 			(layer "F.SilkS")
 		)
 		(fp_line
-			(start -2.5 -1.51)
-			(end 2.3 -1.51)
+			(start 0.206 0.7)
+			(end -0.574 0.7)
 			(stroke
 				(width 0.12)
-				(type solid)
+				(type default)
+			)
+			(layer "F.SilkS")
+		)
+		(fp_line
+			(start -0.184 0.31)
+			(end -0.184 1.09)
+			(stroke
+				(width 0.12)
+				(type default)
 			)
 			(layer "F.SilkS")
@@
 	)
 	(gr_line
-		(start 139.456 102.88)
+		(start 141.726 98.995)
+		(end 141.726 102.88)
+		(stroke
+			(width 0.12)
+			(type default)
+		)
+		(layer "F.SilkS")
+	)
+	(gr_line
+		(start 141.726 102.88)
 		(end 133.0545 102.88)
 		(stroke
