File: Hardware/CAN sensor net/Piezo module/Piezo module.kicad_pcb (KiCad board)
At the start: 4 copper layers, 38.3 x 25.1 mm, 91 parts, among them J1 532610671, J2 532610671, J3 USB_B_Micro, J4 530470310, J5 532610271, SW1 SW_Push, SW2 SW_SPDT, U1 SN65HVD230, U2 STM32F103C8Tx, U3 W25Q32FVSSIG, U4 L78L05_SOT89, U5 LD3985M33R_SOT23, U6 L79L05_SOT89, U7 USBLC6-2SC6, U8 TL072, U9 ADS1120-PW, Y1 16MHz

Commit message: Master and Piezo fixes
Parts:
- D2: footprint LED_SMD:LED_RGB_Wuerth-PLCC4_3.2x2.8mm_150141M173100 -> user_lib:LED_RGB_promelec
- moved R2 1.46 mm to (152.7, 101.8)
- moved R5 1.46 mm to (154.1, 101.8)
Connections:
- D2 pad 2: Net-(D2-GK) -> VDD_3V3
- D2 pad 4: VDD_3V3 -> Net-(D2-GK)
- R2 pad 1: Net-(D2-BK) -> Net-(D2-RK)
- R2 pad 2: LED_RGB_BLUE -> LED_RGB_RED
- R5 pad 1: Net-(D2-RK) -> Net-(D2-BK)
- R5 pad 2: LED_RGB_RED -> LED_RGB_BLUE
Other:
- board text removed: "FC1"
- board text removed: "X"
- board text removed: "Y"
- board text removed: "Z"
- board text removed: "добавить MP у остальных плат"
Changed lines of the file:
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@@
 			)
 		)
+		(property ki_fp_filters "LED* LED_SMD:* LED_THT:*")
+		(sheetname "Корневой лист")
+		(sheetfile "Piezo module.kicad_sch")
 		(attr smd)
 		(fp_line
@@
 			)
 		)
+		(property ki_fp_filters "LED* LED_SMD:* LED_THT:*")
+		(sheetname "Корневой лист")
+		(sheetfile "Piezo module.kicad_sch")
 		(attr smd)
 		(fp_line
@@
 	(footprint "Resistor_SMD:R_0603_1608Metric"
 		(layer "F.Cu")
-		(at 154.149 101.832 90)
+		(at 152.687 101.832 90)
 		(descr "Resistor SMD 0603 (1608 Metric), square (rectangular) end terminal, IPC_7351 nominal, (Body size source: IPC-SM-782 page 72, https://www.pcb-3d.com/wordpress/wp-content/uploads/ipc-sm-782a_amendment_1_and_2.pdf), generated with kicad-footprint-generator")
 		(tags "resistor")
@@
 			(layers "F.Cu" "F.Paste" "F.Mask")
 			(roundrect_rratio 0.25)
-			(net 8 "Net-(D2-BK)")
+			(net 9 "Net-(D2-RK)")
 			(pintype "passive")
 		)
@@
 			(layers "F.Cu" "F.Paste" "F.Mask")
 			(roundrect_rratio 0.25)
-			(net 16 "LED_RGB_BLUE")
+			(net 18 "LED_RGB_RED")
 			(pintype "passive")
 		)
@@
 			)
 		)
+		(property ki_fp_filters "Connector*:*_1x??_*")
+		(sheetname "Connectors")
+		(sheetfile "connectors.kicad_sch")
 		(attr smd)
 		(fp_line
@@
 		)
 	)
-	(footprint "LED_SMD:LED_RGB_Wuerth-PLCC4_3.2x2.8mm_150141M173100"
+	(footprint "user_lib:LED_RGB_promelec"
 		(layer "F.Cu")
 		(at 154.667 104.963 180)
@@
 			)
 		)
-		(property "Footprint" "LED_SMD:LED_RGB_Wuerth-PLCC4_3.2x2.8mm_150141M173100"
+		(property "Footprint" "user_lib:LED_RGB_promelec"
 			(at 0 0 180)
 			(unlocked yes)
@@
 			)
 		)
+		(property ki_fp_filters "LED* LED_SMD:* LED_THT:*")
+		(sheetname "Корневой лист")
+		(sheetfile "Piezo module.kicad_sch")
 		(attr smd)
 		(fp_line
@@
 		)
 		(fp_line
-			(start 1.6 -1.4)
-			(end -1.6 -1.4)
+			(start 1.6 0.4)
+			(end 0.6 1.4)
 			(stroke
 				(width 0.1)
@@
 		)
 		(fp_line
-			(start -0.6 -1.4)
-			(end -1.6 -0.4)
+			(start 1.6 -1.4)
+			(end -1.6 -1.4)
 			(stroke
 				(width 0.1)
@@
 		)
 		(pad "2" smd rect
-			(at 1.55 -0.7 180)
+			(at -1.55 0.7 180)
 			(size 1.5 0.9)
 			(layers "F.Cu" "F.Paste" "F.Mask")
-			(net 10 "Net-(D2-GK)")
-			(pinfunction "GK")
+			(net 1 "VDD_3V3")
+			(pinfunction "A")
 			(pintype "passive")
 		)
@@
 		)
 		(pad "4" smd rect
-			(at -1.55 0.7 180)
+			(at 1.55 -0.7 180)
 			(size 1.5 0.9)
 			(layers "F.Cu" "F.Paste" "F.Mask")
-			(net 1 "VDD_3V3")
-			(pinfunction "A")
+			(net 10 "Net-(D2-GK)")
+			(pinfunction "GK")
 			(pintype "passive")
 		)
@@
 			)
 			(rotate
-				(xyz 0 0 0)
+				(xyz 0 0 180)
 			)
 		)
@@
 	(footprint "Resistor_SMD:R_0603_1608Metric"
 		(layer "F.Cu")
-		(at 152.687 101.832 90)
+		(at 154.149 101.832 90)
 		(descr "Resistor SMD 0603 (1608 Metric), square (rectangular) end terminal, IPC_7351 nominal, (Body size source: IPC-SM-782 page 72, https://www.pcb-3d.com/wordpress/wp-content/uploads/ipc-sm-782a_amendment_1_and_2.pdf), generated with kicad-footprint-generator")
 		(tags "resistor")
@@
 			(layers "F.Cu" "F.Paste" "F.Mask")
 			(roundrect_rratio 0.25)
-			(net 9 "Net-(D2-RK)")
+			(net 8 "Net-(D2-BK)")
 			(pintype "passive")
 		)
@@
 			(layers "F.Cu" "F.Paste" "F.Mask")
 			(roundrect_rratio 0.25)
-			(net 18 "LED_RGB_RED")
+			(net 16 "LED_RGB_BLUE")
 			(pintype "passive")
 		)
@@
 		(layer "Edge.Cuts")
 	)
-	(gr_circle
-		(center 180.799 99.608)
-		(end 181.748992 99.608)
-		(stroke
-			(width 0.2)
-			(type solid)
-		)
-		(fill solid)
-		(layer "User.2")
-	)
-	(gr_line
-		(start 188.993 99.627)
-		(end 187.346 100.689)
-		(stroke
-			(width 0.2)
-			(type default)
-		)
-		(layer "User.2")
-	)
-	(gr_line
-		(start 188.993 99.627)
-		(end 183.208003 99.608)
-		(stroke
-			(width 0.2)
-			(type default)
-		)
-		(layer "User.2")
-	)
-	(gr_line
-		(start 187.322 98.361)
-		(end 188.993 99.627)
-		(stroke
-			(width 0.2)
-			(type default)
-		)
-		(layer "User.2")
-	)
-	(gr_line
-		(start 179.691 93.237)
-		(end 180.795 91.824)
-		(stroke
-			(width 0.2)
-			(type default)
-		)
-		(layer "User.2")
-	)
-	(gr_circle
-		(center 180.799 99.608)
-		(end 183.208003 99.608)
-		(stroke
-			(width 0.2)
-			(type default)
-		)
-		(fill none)
-		(layer "User.2")
-	)
-	(gr_line
-		(start 180.795 91.824)
-		(end 181.803 93.309)
-		(stroke
-			(width 0.2)
-			(type default)
-		)
-		(layer "User.2")
-	)
-	(gr_line
-		(start 180.799 97.198997)
-		(end 180.794966 91.824001)
-		(stroke
-			(width 0.2)
-			(type default)
-		)
-		(layer "User.2")
-	)
 	(gr_text "7V0"
 		(at 137.2 94.238 0)
@@
 	)
 	(gr_text "120R"
-		(at 165.66 93.35 270)
+		(at 170.52 94.781 0)
 		(layer "B.SilkS")
 		(effects
@@
 			)
 			(justify left bottom)
-		)
-	)
-	(gr_text "X"
-		(at 187.945 103.047 0)
-		(layer "User.2")
-		(effects
-			(font
-				(size 1.5 1.5)
-				(thickness 0.3)
-				(bold yes)
-			)
-			(justify left bottom)
-		)
-	)
-	(gr_text "Z"
-		(at 177.007 103.554 0)
-		(layer "User.2")
-		(effects
-			(font
-				(size 1.5 1.5)
-				(thickness 0.3)
-				(bold yes)
-			)
-			(justify left bottom)
-		)
-	)
-	(gr_text "FC1"
-		(at 184.016 97.126 0)
-		(layer "User.2")
-		(effects
-			(font
-				(size 1.5 1.5)
-				(thickness 0.3)
-				(bold yes)
-			)
-			(justify left bottom)
-		)
-	)
-	(gr_text "добавить MP у остальных плат"
-		(at 137.547 87.023 0)
-		(layer "User.2")
-		(effects
-			(font
-				(size 1 1)
-				(thickness 0.15)
-			)
-			(justify left bottom)
-		)
-	)
-	(gr_text "Y"
-		(at 182.695 93.666 0)
-		(layer "User.2")
-		(effects
-			(font
-				(size 1.5 1.5)
-				(thickness 0.3)
-				(bold yes)
-			)
-			(justify left bottom)
