File: Hardware/CAN sensor net/IMU module/connectors.kicad_sch (KiCad schematic)
At the start: 9 parts, among them J1 532610671, J2 532610671, J3 USB_B_Micro, J4 530470310, U5 USBLC6-2SC6

Commit message: IMU update
Connections:
- net GND: now also J1.MP, J2.MP, J4.MP
Changed lines of the file:
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@@
 	(wire
 		(pts
-			(xy 172.085 54.61) (xy 172.085 51.435)
+			(xy 172.085 55.245) (xy 172.085 51.435)
 		)
 		(stroke
@@
 	(wire
 		(pts
-			(xy 194.31 80.01) (xy 194.31 82.55)
+			(xy 194.31 80.01) (xy 194.31 83.82)
 		)
 		(stroke
@@
 	(wire
 		(pts
-			(xy 203.835 54.61) (xy 203.835 51.435)
+			(xy 203.835 55.245) (xy 203.835 51.435)
 		)
 		(stroke
@@
 	(symbol
 		(lib_id "power:GND")
-		(at 203.835 54.61 0)
+		(at 203.835 55.245 0)
 		(unit 1)
 		(exclude_from_sim no)
@@
 		(dnp no)
 		(property "Reference" "#PWR013"
-			(at 203.835 60.96 0)
+			(at 203.835 61.595 0)
 			(effects
 				(font
@@
 		)
 		(property "Value" "GND"
-			(at 203.835 58.42 0)
+			(at 203.835 59.055 0)
 			(effects
 				(font
@@
 		)
 		(property "Footprint" ""
-			(at 203.835 54.61 0)
+			(at 203.835 55.245 0)
 			(effects
 				(font
@@
 		)
 		(property "Datasheet" ""
-			(at 203.835 54.61 0)
+			(at 203.835 55.245 0)
 			(effects
 				(font
@@
 		)
 		(property "Description" ""
-			(at 203.835 54.61 0)
+			(at 203.835 55.245 0)
 			(effects
 				(font
@@
 	)
 	(symbol
+		(lib_id "power:GND")
+		(at 215.9 55.245 0)
+		(unit 1)
+		(exclude_from_sim no)
+		(in_bom yes)
+		(on_board yes)
+		(dnp no)
+		(property "Reference" "#PWR028"
+			(at 215.9 61.595 0)
+			(effects
+				(font
+					(size 1.27 1.27)
+				)
+				(hide yes)
+			)
+		)
+		(property "Value" "GND"
+			(at 215.9 59.055 0)
+			(effects
+				(font
+					(size 1.27 1.27)
+				)
+			)
+		)
+		(property "Footprint" ""
+			(at 215.9 55.245 0)
+			(effects
+				(font
+					(size 1.27 1.27)
+				)
+				(hide yes)
+			)
+		)
+		(property "Datasheet" ""
+			(at 215.9 55.245 0)
+			(effects
+				(font
+					(size 1.27 1.27)
+				)
+				(hide yes)
+			)
+		)
+		(property "Description" ""
+			(at 215.9 55.245 0)
+			(effects
+				(font
+					(size 1.27 1.27)
+				)
+				(hide yes)
+			)
+		)
+		(pin "1"
+		)
+		(instances
+			(project "IMU module"
+				(path "/62238c1b-6f7a-4963-9d99-86e391606da3/78b5b684-d926-4716-ab30-8bfd5bbd500c"
+					(reference "#PWR028")
+					(unit 1)
+				)
+			)
+		)
+	)
+	(symbol
+		(lib_id "power:GND")
+		(at 184.15 55.245 0)
+		(unit 1)
+		(exclude_from_sim no)
+		(in_bom yes)
+		(on_board yes)
+		(dnp no)
+		(property "Reference" "#PWR027"
+			(at 184.15 61.595 0)
+			(effects
+				(font
+					(size 1.27 1.27)
+				)
+				(hide yes)
+			)
+		)
+		(property "Value" "GND"
+			(at 184.15 59.055 0)
+			(effects
+				(font
+					(size 1.27 1.27)
+				)
+			)
+		)
+		(property "Footprint" ""
+			(at 184.15 55.245 0)
+			(effects
+				(font
+					(size 1.27 1.27)
+				)
+				(hide yes)
+			)
+		)
+		(property "Datasheet" ""
+			(at 184.15 55.245 0)
+			(effects
+				(font
+					(size 1.27 1.27)
+				)
+				(hide yes)
+			)
+		)
+		(property "Description" ""
+			(at 184.15 55.245 0)
+			(effects
+				(font
+					(size 1.27 1.27)
+				)
+				(hide yes)
+			)
+		)
+		(pin "1"
+		)
+		(instances
+			(project "IMU module"
+				(path "/62238c1b-6f7a-4963-9d99-86e391606da3/78b5b684-d926-4716-ab30-8bfd5bbd500c"
+					(reference "#PWR027")
+					(unit 1)
+				)
+			)
+		)
+	)
+	(symbol
+		(lib_id "power:GND")
+		(at 201.295 83.82 0)
+		(unit 1)
+		(exclude_from_sim no)
+		(in_bom yes)
+		(on_board yes)
+		(dnp no)
+		(property "Reference" "#PWR029"
+			(at 201.295 90.17 0)
+			(effects
+				(font
+					(size 1.27 1.27)
+				)
+				(hide yes)
+			)
+		)
+		(property "Value" "GND"
+			(at 201.295 87.63 0)
+			(effects
+				(font
+					(size 1.27 1.27)
+				)
+			)
+		)
+		(property "Footprint" ""
+			(at 201.295 83.82 0)
+			(effects
+				(font
+					(size 1.27 1.27)
+				)
+				(hide yes)
+			)
+		)
+		(property "Datasheet" ""
+			(at 201.295 83.82 0)
+			(effects
+				(font
+					(size 1.27 1.27)
+				)
+				(hide yes)
+			)
+		)
+		(property "Description" ""
+			(at 201.295 83.82 0)
+			(effects
+				(font
+					(size 1.27 1.27)
+				)
+				(hide yes)
+			)
+		)
+		(pin "1"
+		)
+		(instances
+			(project "IMU module"
+				(path "/62238c1b-6f7a-4963-9d99-86e391606da3/78b5b684-d926-4716-ab30-8bfd5bbd500c"
+					(reference "#PWR029")
+					(unit 1)
+				)
+			)
+		)
+	)
+	(symbol
 		(lib_id "Connector:USB_B_Micro")
 		(at 43.18 52.07 0)
@@
 	)
 	(symbol
+		(lib_name "Conn_01x06_1")
 		(lib_id "Connector_Generic:Conn_01x06")
 		(at 215.9 43.815 0)
@@
 		)
 		(pin "1"
+		)
+		(pin "MP"
 		)
 		(instances
@@
 	(symbol
 		(lib_id "power:GND")
-		(at 172.085 54.61 0)
+		(at 172.085 55.245 0)
 		(unit 1)
 		(exclude_from_sim no)
@@
 		(dnp no)
 		(property "Reference" "#PWR012"
-			(at 172.085 60.96 0)
+			(at 172.085 61.595 0)
 			(effects
 				(font
@@
 		)
 		(property "Value" "GND"
-			(at 172.085 58.42 0)
+			(at 172.085 59.055 0)
 			(effects
 				(font
@@
 		)
 		(property "Footprint" ""
-			(at 172.085 54.61 0)
+			(at 172.085 55.245 0)
 			(effects
 				(font
@@
 		)
 		(property "Datasheet" ""
-			(at 172.085 54.61 0)
+			(at 172.085 55.245 0)
 			(effects
 				(font
@@
 		)
 		(property "Description" ""
-			(at 172.085 54.61 0)
+			(at 172.085 55.245 0)
 			(effects
 				(font
@@
 		(pin "1"
 		)
+		(pin "MP"
+		)
 		(instances
 			(project "IMU module"
@@
 		(lib_name "GND_1")
 		(lib_id "power:GND")
-		(at 194.31 82.55 0)
+		(at 194.31 83.82 0)
 		(unit 1)
 		(exclude_from_sim no)
@@
 		(dnp no)
 		(property "Reference" "#PWR017"
-			(at 194.31 88.9 0)
+			(at 194.31 90.17 0)
 			(effects
 				(font
@@
 		)
 		(property "Value" "GND"
-			(at 194.31 86.36 0)
+			(at 194.31 87.63 0)
 			(effects
 				(font
@@
 		)
 		(property "Footprint" ""
-			(at 194.31 82.55 0)
+			(at 194.31 83.82 0)
 			(effects
 				(font
@@
 		)
 		(property "Datasheet" ""
-			(at 194.31 82.55 0)
+			(at 194.31 83.82 0)
 			(effects
 				(font
@@
 		)
 		(property "Description" "Power symbol creates a global label with name \"GND\" , ground"
-			(at 194.31 82.55 0)
+			(at 194.31 83.82 0)
 			(effects
 				(font
@@
 		(pin "1"
 		)
+		(pin "MP"
+		)
 		(instances
