File: Hardware/CAN sensor net/IMU module/IMU module.kicad_pcb (KiCad board)
At the start: 2 copper layers, 78 parts, among them J1 532610671, J2 532610671, J3 USB_B_Micro, J4 530470310, SW1 SW_Push, SW2 SW_SPDT, U1 SN65HVD230, U2 STM32F103C8Tx, U3 W25Q32FVSSIG, U4 LD3985M33R_SOT23, U5 USBLC6-2SC6, U6 BMI088, U7 ICM-42688-P, U8 MPU-9250, Y1 16MHz

Commit message: IMU update
Parts:
- moved C3 109.6 mm to (197.3, 107.5)
- moved C6 107.0 mm to (197.3, 109.0)
- moved C4 106.3 mm to (199.2, 97.8), turned to 180 degrees
- moved C2 98.7 mm to (188.7, 97.8)
- moved C8 97.3 mm to (186.6, 103.4), turned to -90 degrees
- moved C5 96.7 mm to (190.6, 95.8), turned to 180 degrees
- moved C7 95.2 mm to (188.1, 103.4), turned to -90 degrees
- moved U2 83.3 mm to (193.9, 101.7)
- moved SW2 80.1 mm to (183.2, 66.9), turned to 180 degrees
- moved U1 80.1 mm to (182.5, 81.3), turned to 180 degrees
- moved Y1 76.8 mm to (187.3, 74.7), turned to -90 degrees
- moved U3 74.6 mm to (193.3, 85.3), turned to 180 degrees
- moved J2 72.5 mm to (210.7, 80.7), turned to 90 degrees
- moved SW1 71.7 mm to (196.3, 57.3)
- moved U6 63.5 mm to (203.1, 78.0), turned to 90 degrees
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Connections:
- J1 pad MP: (no net) -> GND
- J2 pad MP: (no net) -> GND
- J4 pad MP: (no net) -> GND
Routing:
- net unconnected-(U2-PB6-Pad42): track 0.00 -> 21.1 mm
- net CAN_TX: track 0.00 -> 21.1 mm
- net unconnected-(U2-PB7-Pad43): track 0.00 -> 18.6 mm
- net CAN_RX: track 0.00 -> 18.2 mm
- net VDD_3V3: track 0.00 -> 15.0 mm
- net GND: track 0.00 -> 11.3 mm
- net USB_D+: track 0.00 -> 8.59 mm
- net USB_D-: track 0.00 -> 7.02 mm
- net /Connectors/usb_conn_d-: track 0.00 -> 4.49 mm
- net /Connectors/usb_conn_d+: track 0.00 -> 4.49 mm
- net RCC_OSC_IN: track 0.00 -> 4.13 mm
- net CAN-: track 0.00 -> 2.55 mm
- net CAN+: track 0.00 -> 2.54 mm
- net RCC_OSC_OUT: track 0.00 -> 2.17 mm
Other:
- board outline added: 50.1 x 25.5 mm

Commit message: Added Li-Io balanserer
Other:
- board text added: "ОСИ"
Changed lines of the file:
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@@
 		(tags "solder jumper open")
 		(property "Reference" "JP6"
-			(at 0 -1.8 270)
+			(at 0 -1.8 -90)
 			(layer "F.SilkS")
 			(hide yes)
@@
 		)
 		(property "Value" "SolderJumper_2_Open"
-			(at 0 1.9 270)
+			(at 0 1.9 -90)
 			(layer "F.Fab")
 			(effects
@@
 		(tags "capacitor")
 		(property "Reference" "C3"
-			(at 0 -1.43 360)
+			(at 0 -1.43 0)
 			(layer "F.SilkS")
 			(hide yes)
@@
 		)
 		(property "Value" "100n"
-			(at 0 1.43 360)
+			(at 0 1.43 0)
 			(layer "F.Fab")
 			(effects
@@
 		)
 		(fp_text user "${REFERENCE}"
-			(at 0 0 360)
+			(at 0 0 0)
 			(layer "F.Fab")
 			(effects
@@
 		(tags "solder jumper open")
 		(property "Reference" "JP3"
-			(at 0 -1.8 270)
+			(at 0 -1.8 -90)
 			(layer "F.SilkS")
 			(hide yes)
@@
 		)
 		(property "Value" "SolderJumper_2_Open"
-			(at 0 1.9 270)
+			(at 0 1.9 -90)
 			(layer "F.Fab")
 			(effects
@@
 		(tags "solder jumper open")
 		(property "Reference" "JP5"
-			(at 0 -1.8 270)
+			(at 0 -1.8 -90)
 			(layer "F.SilkS")
 			(hide yes)
@@
 		)
 		(property "Value" "SolderJumper_2_Open"
-			(at 0 1.9 270)
+			(at 0 1.9 -90)
 			(layer "F.Fab")
 			(effects
@@
 		(tags "solder jumper open")
 		(property "Reference" "JP1"
-			(at 0 -1.8 270)
+			(at 0 -1.8 -90)
 			(layer "F.SilkS")
 			(hide yes)
@@
 		)
 		(property "Value" "SolderJumper_2_Open"
-			(at 0 1.9 270)
+			(at 0 1.9 -90)
 			(layer "F.Fab")
 			(effects
@@
 		(tags "SOT TO_SOT_SMD")
 		(property "Reference" "U5"
-			(at 0 -2.4 360)
+			(at 0 -2.4 0)
 			(layer "F.SilkS")
 			(hide yes)
@@
 		)
 		(property "Value" "USBLC6-2SC6"
-			(at 0 2.4 360)
+			(at 0 2.4 0)
 			(layer "F.Fab")
 			(effects
@@
 		)
 		(fp_text user "${REFERENCE}"
-			(at 0 0 360)
+			(at 0 0 0)
 			(layer "F.Fab")
 			(effects
@@
 		(tags "solder jumper open")
 		(property "Reference" "JP4"
-			(at 0 -1.8 270)
+			(at 0 -1.8 -90)
 			(layer "F.SilkS")
 			(hide yes)
@@
 		)
 		(property "Value" "SolderJumper_2_Open"
-			(at 0 1.9 270)
+			(at 0 1.9 -90)
 			(layer "F.Fab")
 			(effects
@@
 		(tags "solder jumper open")
 		(property "Reference" "JP2"
-			(at 0 -1.8 270)
+			(at 0 -1.8 -90)
 			(layer "F.SilkS")
 			(hide yes)
@@
 		)
 		(property "Value" "SolderJumper_2_Open"
-			(at 0 1.9 270)
+			(at 0 1.9 -90)
 			(layer "F.Fab")
 			(effects
@@
 		(tags "LQFP QFP")
 		(property "Reference" "U2"
-			(at 0 -5.85 360)
+			(at 0 -5.85 0)
 			(layer "F.SilkS")
 			(hide yes)
@@
 		)
 		(property "Value" "STM32F103C8Tx"
-			(at 0 5.85 360)
+			(at 0 5.85 0)
 			(layer "F.Fab")
 			(effects
@@
 		)
 		(fp_text user "${REFERENCE}"
-			(at 0 0 360)
+			(at 0 0 0)
 			(layer "F.Fab")
 			(effects
@@
 		(layer "Edge.Cuts")
 	)
+	(gr_text "ОСИ"
+		(at 219.568 87.321 0)
+		(layer "F.Cu")
+		(effects
+			(font
+				(size 20 20)
+				(thickness 2.5)
+			)
+			(justify left bottom)
+		)
+	)
 	(segment
