File: Hardware/CAN sensor net/IMU module/imu.kicad_sch (KiCad schematic)
At the start: 11 parts, among them U6 BMI088, U7 ICM-42688-P, U8 MPU-9250

Commit message: Update IMU
Connections:
- net GND: no longer U6.2 (NC), U7.10 (RESV), U7.11 (RESV), U7.2 (RESV), U7.3 (RESV)
Changed lines of the file:
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@@
-	)
-	(junction
-		(at 168.275 70.485)
-		(diameter 0)
-		(color 0 0 0 0)
 	)
 	(junction
@@
 	)
 	(junction
-		(at 262.89 66.675)
-		(diameter 0)
-		(color 0 0 0 0)
-	)
-	(junction
-		(at 262.89 71.755)
-		(diameter 0)
-		(color 0 0 0 0)
-	)
-	(junction
 		(at 232.41 34.925)
 		(diameter 0)
@@
 	)
 	(junction
-		(at 262.89 64.135)
-		(diameter 0)
-		(color 0 0 0 0)
-	)
-	(junction
 		(at 224.79 34.925)
-		(diameter 0)
-		(color 0 0 0 0)
-	)
-	(junction
-		(at 262.89 61.595)
 		(diameter 0)
 		(color 0 0 0 0)
@@
 	(wire
 		(pts
-			(xy 258.445 59.055) (xy 262.89 59.055)
-		)
-		(stroke
-			(width 0)
-			(type default)
-		)
-	)
-	(wire
-		(pts
 			(xy 86.995 91.44) (xy 79.375 91.44)
 		)
@@
 	(wire
 		(pts
-			(xy 168.275 67.945) (xy 168.275 70.485)
+			(xy 168.275 67.945) (xy 168.275 86.36)
 		)
 		(stroke
@@
 	(wire
 		(pts
-			(xy 258.445 66.675) (xy 262.89 66.675)
-		)
-		(stroke
-			(width 0)
-			(type default)
-		)
-	)
-	(wire
-		(pts
-			(xy 258.445 64.135) (xy 262.89 64.135)
-		)
-		(stroke
-			(width 0)
-			(type default)
-		)
-	)
-	(wire
-		(pts
 			(xy 235.585 34.925) (xy 238.125 34.925)
 		)
@@
 		)
 	)
-	(wire
-		(pts
-			(xy 168.275 86.36) (xy 168.275 70.485)
-		)
-		(stroke
-			(width 0)
-			(type default)
-		)
-	)
 	(polyline
 		(pts
@@
 	(wire
 		(pts
-			(xy 262.89 64.135) (xy 262.89 66.675)
-		)
-		(stroke
-			(width 0)
-			(type default)
-		)
-	)
-	(wire
-		(pts
 			(xy 150.495 86.36) (xy 168.275 86.36)
 		)
@@
 	(wire
 		(pts
-			(xy 262.89 61.595) (xy 262.89 64.135)
-		)
-		(stroke
-			(width 0)
-			(type default)
-		)
-	)
-	(wire
-		(pts
 			(xy 164.465 67.945) (xy 168.275 67.945)
 		)
@@
 	(wire
 		(pts
-			(xy 258.445 61.595) (xy 262.89 61.595)
-		)
-		(stroke
-			(width 0)
-			(type default)
-		)
-	)
-	(wire
-		(pts
 			(xy 40.005 71.12) (xy 40.005 91.44)
 		)
@@
 	(wire
 		(pts
-			(xy 262.89 59.055) (xy 262.89 61.595)
-		)
-		(stroke
-			(width 0)
-			(type default)
-		)
-	)
-	(wire
-		(pts
 			(xy 168.275 38.735) (xy 168.275 40.64)
 		)
@@
 	(wire
 		(pts
-			(xy 168.275 70.485) (xy 164.465 70.485)
-		)
-		(stroke
-			(width 0)
-			(type default)
-		)
-	)
-	(wire
-		(pts
 			(xy 147.955 86.36) (xy 150.495 86.36)
 		)
@@
 		)
 		(stroke
-			(width 0)
-			(type default)
-		)
-	)
-	(wire
-		(pts
-			(xy 262.89 66.675) (xy 262.89 71.755)
-		)
-		(stroke

Commit message: IMU production
Parts:
- removed C20, C21, C24: 100n, Capacitor_SMD:C_0603_1608Metric, symbol Device:C_Small
- removed U8: MPU-9250, Sensor_Motion:InvenSense_QFN-24_3x3mm_P0.4mm, symbol Sensor_Motion:MPU-9250
Connections:
- no-connect marks 2 -> 0
Other:
- note removed: "Gyro Accel Mag MPU9250"
- moved on the sheet: C17, C18, C19, C22, C23, U6, U7
