File: Hardware/ciam/impeller18/switches.kicad_sch (KiCad schematic)
At the start: 179 parts, among them J2 Conn_02x09_Odd_Even, J3 Conn_02x09_Odd_Even, J4 Conn_02x08_Odd_Even, J5 Conn_02x04_Odd_Even, Q1 BSS138, Q10 BSS138, Q11 BSS138, Q12 BSS138, Q13 BSS138, Q14 BSS138, Q15 BSS138, Q16 BSS138, Q17 BSS138, Q18 BSS138, Q19 BSS138, Q2 BSS138, Q20 BSS138, Q21 BSS138, Q22 BSS138, Q23 BSS138, Q24 BSS138, Q25 BSS138, Q26 BSS138, Q27 BSS138, Q28 BSS138, Q29 BSS138, Q3 BSS138, Q30 BSS138, Q4 BSS138, Q5 BSS138, Q6 BSS138, Q7 BSS138, Q8 BSS138, Q9 BSS138, U10 TLP291-4, U11 TLP291, U12 TLP291-4, U13 TLP291-4, U14 TLP291-4, U15 TLP291, U16 TLP291, U17 TLP291-4, U18 B0505MT-1WR4, U19 B0505MT-1WR4, U20 B0505MT-1WR4, U8 TLP291-4, U9 TLP291-4

Commit message: updated impeller18 schamatic
Parts:
- removed U11: TLP291, Package_SO:SOIC-4_4.55x2.6mm_P1.27mm, symbol Isolator:TLP291
- removed U14: TLP291-4, Package_SO:SOIC-16_4.55x10.3mm_P1.27mm, symbol Isolator:TLP291-4
- added U11: TLP291-4, symbol Isolator:TLP291-4
- J2, J3: value Conn_02x09_Odd_Even -> 430451800
- J4: value Conn_02x08_Odd_Even -> 430451600
- J5: value Conn_02x04_Odd_Even -> 430450800
- Q1, Q10, Q11, Q12, Q13, Q14, Q15, Q16, Q17, Q18, Q19, Q2, Q20, Q21, Q22, Q23, Q24, Q25, Q26, Q27, Q28, Q29, Q3, Q30, Q4, Q5, Q6, Q7, Q8, Q9: footprint Package_TO_SOT_SMD:SOT-23 -> (none)
- U10, U12, U13, U17, U8, U9: footprint Package_SO:SOIC-16_4.55x10.3mm_P1.27mm -> (none)
- U15, U16: footprint Package_SO:SOIC-4_4.55x2.6mm_P1.27mm -> (none)
Connections:
- net SWITCH_5.1_EXT is gone; now on net SWITCH_4.1_EXT: J5.1 (Pin_1), R116.2
- net SWITCH_5.2_EXT is gone; now on net SWITCH_4.2_EXT: J5.3 (Pin_3), R120.2
- net SWITCH_5.3_EXT is gone; now on net SWITCH_4.3_EXT: J5.5 (Pin_5), R124.2
- net GND: now also U11.11, U11.13, U11.15, U11.9
- net GND_IN: now also U11.2, U11.4, U11.6, U11.8
- net SWITCH_1.1_EXT: no longer J2.1 (Pin_1)
- net SWITCH_1.2_EXT: no longer J2.3 (Pin_3)
- net SWITCH_1.3_EXT: no longer J2.5 (Pin_5)
- net SWITCH_1.4_EXT: no longer J2.7 (Pin_7)
- net SWITCH_1.5_EXT: no longer J2.9 (Pin_9)
- net SWITCH_1.6_EXT: no longer J2.11 (Pin_11)
- net SWITCH_1.7_EXT: no longer J2.13 (Pin_13)
- net SWITCH_1.8_EXT: no longer J2.15 (Pin_15)
- net SWITCH_1.9_EXT: no longer J2.17 (Pin_17)
- net SWITCH_2.1_EXT: now also J2.1 (Pin_1)
- net SWITCH_2.2_EXT: now also J2.3 (Pin_3)
- net SWITCH_2.3_EXT: now also J2.5 (Pin_5)
- net SWITCH_2.4_EXT: now also J2.7 (Pin_7)
- net SWITCH_2.5_EXT: now also J2.9 (Pin_9)
- net SWITCH_2.6_EXT: now also J2.11 (Pin_11)
- net SWITCH_2.7_EXT: now also J2.13 (Pin_13)
- net SWITCH_2.8_EXT: now also J2.15 (Pin_15)
- net SWITCH_2.9_EXT: now also J2.17 (Pin_17)
- net SWITCH_4.1_EXT: no longer J4.11 (Pin_11), R78.2
- net SWITCH_4.2_EXT: no longer J4.13 (Pin_13), R90.2
- net SWITCH_4.3_EXT: no longer J4.15 (Pin_15), R102.2
- net at R86.2: now also U11.3
- net at R63.2: now also U11.1
- net at R98.2: now also U11.5
- net at R110.2: now also U11.7
- net SWITCH_1.1_INPUT renamed SWITCH_1.1_3V3
- net SWITCH_1.2_INPUT renamed SWITCH_1.2_3V3
- net SWITCH_1.3_INPUT renamed SWITCH_1.3_3V3
- net SWITCH_1.4_INPUT renamed SWITCH_1.4_3V3
- net SWITCH_1.5_INPUT renamed SWITCH_1.5_3V3
- net SWITCH_1.6_INPUT renamed SWITCH_1.6_3V3
- net SWITCH_1.7_INPUT renamed SWITCH_1.7_3V3
- net SWITCH_1.8_INPUT renamed SWITCH_1.8_3V3
- net SWITCH_1.9_INPUT renamed SWITCH_1.9_3V3
- net SWITCH_2.1_INPUT renamed SWITCH_2.1_3V3
- net SWITCH_2.2_INPUT renamed SWITCH_2.2_3V3
- net SWITCH_2.3_INPUT renamed SWITCH_2.3_3V3
- net SWITCH_2.4_INPUT renamed SWITCH_2.4_3V3
- net SWITCH_2.5_INPUT renamed SWITCH_2.5_3V3
- net SWITCH_2.6_INPUT renamed SWITCH_2.6_3V3
- net SWITCH_2.7_INPUT renamed SWITCH_2.7_3V3
- net SWITCH_2.8_INPUT renamed SWITCH_2.8_3V3
- net SWITCH_2.9_INPUT renamed SWITCH_2.9_3V3
- net SWITCH_3.1_INPUT renamed SWITCH_3.1_3V3
- net SWITCH_3.2_INPUT renamed SWITCH_3.2_3V3
- net SWITCH_3.3_INPUT renamed SWITCH_3.3_3V3
- net SWITCH_3.4_INPUT renamed SWITCH_3.4_3V3
- net SWITCH_3.5_INPUT renamed SWITCH_3.5_3V3
- net SWITCH_3.5_3V3: now also U11.16
- net SWITCH_4.1_INPUT renamed SWITCH_3.6_3V3
- net SWITCH_3.6_3V3: now also U11.14
- net SWITCH_4.2_INPUT renamed SWITCH_3.7_3V3
- net SWITCH_3.7_3V3: now also U11.12
- net SWITCH_4.3_INPUT renamed SWITCH_3.8_3V3
- net SWITCH_3.8_3V3: now also U11.10
- net SWITCH_5.1_INPUT renamed SWITCH_4.1_3V3
- net SWITCH_5.2_INPUT renamed SWITCH_4.2_3V3
- net SWITCH_5.3_INPUT renamed SWITCH_4.3_3V3
- net SWITCH_5.4_EXT renamed SWITCH_4.4_EXT
- net SWITCH_5.4_INPUT renamed SWITCH_4.4_3V3
- new net SWITCH_3.6_EXT: J4.11 (Pin_11), R78.2
- new net SWITCH_3.7_EXT: J4.13 (Pin_13), R90.2
- new net SWITCH_3.8_EXT: J4.15 (Pin_15), R102.2
- no-connect marks 4 -> 0
Other:
- moved on the sheet: C29, C30, C31, C32, C33, C34, C35, C36, C37, C38, C39, C40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
