File: Hardware/ciam/impeller18/encoders.kicad_sch (KiCad schematic)
At the start: 0 parts

Commit message: updated schematics
Parts:
- added C64, C67, C72, C73: 100n, symbol Device:C_Small
- added C65, C66: 10u, symbol Device:C_Small
- added C68: 1u, symbol Device:C
- added C69, C71: 100n, symbol Device:C
- added C70: 4u7, symbol Device:C
- added J5: 430451600, symbol Connector_Generic:Conn_02x08_Odd_Even
- added R187, R189, R195, R200, R202, R207, R209, R211: 1M, symbol Device:R_Small
- added R188, R193, R197, R201, R206, R208, R210, R212: 110k, symbol Device:R_Small
- added R190, R192, R196, R198, R203, R205: 1k, symbol Device:R_Small
- added R191, R194, R199, R204: 150, symbol Device:R_Small
- added U43: LDL1117S33R, symbol Regulator_Linear:LD1117S33TR_SOT223
- added U44: B0505MT-1WR4, symbol Interface_CAN_LIN:ISO1050DUB
- added U45, U49: HCPL-0600, Package_SO:SOIC-8_3.9x4.9mm_P1.27mm, symbol Isolator:HCPL-0600
- added U46: MCP3008, symbol Analog_ADC:MCP3008
- added U47: HCPL-0630, Package_SO:SOIC-8_3.9x4.9mm_P1.27mm, symbol Isolator:HCPL-0630
- added U48, U50: ~, symbol user_lib:IP4220
- added U51: MCP3002, symbol Analog_ADC:MCP3002
Connections:
- new net: R192.2, U45.7 (EN)
- new net: R203.2, U49.7 (EN)
- new net: R191.1, U45.2 (A)
- new net: R199.1, U47.4 (A2)
- new net: R204.1, U49.2 (A)
- new net: U46.12 (Dout), U49.3 (C)
- new net: R198.2, U46.10 (~{CS}/SHDN), U47.6 (VO2)
- new net: R190.1, U45.6 (VO), U46.13 (CLK)
- new net: R194.2, U47.1 (A1)
- new net: R196.1, U46.11 (Din), U47.7 (VO1)
- new net 3V3: R191.2, R194.1, R199.2, R203.1, R205.2, U49.8 (VCC)
- new net 3V3_ADC: C70.1, C71.1, C72.1, C73.1, R190.2, R192.1, R196.2, R198.1, R204.2, U43.2 (VO), U45.8 (VCC), U46.15 (Vref), U46.16 (Vdd), U47.8 (VCC), U48.5 (VDD), U50.5 (VDD)
- new net 5V0: C66.1, C67.1, U44.13 (Vin), U44.14 (Vin)
- new net 5V0_ADC: C64.1, C65.1, C68.1, C69.1, U43.3 (VI), U44.8 (+Vo)
- new net ADC_30V_IN_1: J5.1 (Pin_1), R187.1, U48.1 (IO1)
- new net ADC_30V_IN_2: J5.5 (Pin_5), R189.1, U48.4 (IO3)
- new net ADC_30V_IN_3: J5.3 (Pin_3), R195.1, U48.3 (IO2)
- new net ADC_30V_IN_4: J5.7 (Pin_7), R200.1, U48.6 (IO4)
- new net ADC_30V_IN_5: J5.9 (Pin_9), R202.1, U50.1 (IO1)
- new net ADC_30V_IN_6: J5.11 (Pin_11), R207.1, U50.3 (IO2)
- new net ADC_30V_IN_7: J5.13 (Pin_13), R209.1, U50.4 (IO3)
- new net ADC_30V_IN_8: J5.15 (Pin_15), R211.1, U50.6 (IO4)
- new net ADC_3V3_IN_1: R187.2, R188.2, U46.1 (CH0)
- new net ADC_3V3_IN_2: R189.2, R193.2, U46.2 (CH1)
- new net ADC_3V3_IN_3: R195.2, R197.2, U46.3 (CH2)
- new net ADC_3V3_IN_4: R200.2, R201.2, U46.4 (CH3)
- new net ADC_3V3_IN_5: R202.2, R206.2, U46.5 (CH4)
- new net ADC_3V3_IN_6: R207.2, R208.2, U46.6 (CH5)
- new net ADC_3V3_IN_7: R209.2, R210.2, U46.7 (CH6)
- new net ADC_3V3_IN_8: R211.2, R212.2, U46.8 (CH7)
- new net GND: C66.2, C67.2, U44.1 (gnd), U44.2 (gnd), U49.5 (GND)
- new net GND_ADC: C64.2, C65.2, C68.2, C69.2, C70.2, C71.2, C72.2, C73.2, J5.10 (Pin_10), J5.12 (Pin_12), J5.14 (Pin_14), J5.16 (Pin_16), J5.2 (Pin_2), J5.4 (Pin_4), J5.6 (Pin_6), J5.8 (Pin_8), R188.1, R193.1, R197.1, R201.1, R206.1, R208.1, R210.1, R212.1, U43.1 (GND), U44.6 (0V), U44.7 (0V), U45.5 (GND), U46.14 (AGND), U46.9 (DGND), U47.5 (GND), U48.2 (GND), U50.2 (GND)
- new net SPI1_STM32_ADC8_CS: U47.3 (C2)
- new net SPI1_STM32_CLK: U45.3 (C)
- new net SPI1_STM32_MISO: R205.1, U49.6 (VO)
- new net SPI1_STM32_MOSI: U47.2 (C1)
