File: Hardware/ciam/impeller18/indicators.kicad_sch (KiCad schematic)
At the start: 19 parts, among them J6 Conn_02x09_Odd_Even, U21 G3VM61VY2, U22 G3VM61VY2, U23 G3VM61VY2, U24 G3VM61VY2, U25 G3VM61VY2, U26 G3VM61VY2, U27 G3VM61VY2, U28 G3VM61VY2, U29 G3VM61VY2

Commit message: updated impeller18 schamatic
Parts:
- J7: renamed from J6; value Conn_02x09_Odd_Even -> 430451800
- renumbered R132 to R136, R133 to R137, R134 to R138, R135 to R139, R136 to R140, R137 to R141, R138 to R142, R139 to R143, R140 to R144, U21 to U24, U22 to U25, U23 to U26, U24 to U27, U25 to U28, U26 to U29, U27 to U30, U28 to U31, U29 to U32
Other:
- moved on the sheet: J7

Commit message: updated schematics
Parts:
- renumbered J7 to J10, R136 to R139, R137 to R140, R138 to R141, R139 to R142, R140 to R143, R141 to R144, R142 to R145, R143 to R146, R144 to R147, U24 to U27, U25 to U28, U26 to U29, U27 to U30, U28 to U31, U29 to U32, U30 to U33, U31 to U34, U32 to U35
Changed lines of the file:
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@@
 		(on_board yes)
 		(dnp no)
-		(property "Reference" "R139"
+		(property "Reference" "R142"
 			(at 51.435 76.835 90)
 			(effects
@@
 			(project "impeller18"
 				(path "/4ccab03b-4b1c-4c61-9fa8-19853ef32b4d/e2502236-aeb0-4ddd-871d-5a73d5946ae5"
-					(reference "R139")
+					(reference "R142")
 					(unit 1)
 				)
@@
 		(on_board yes)
 		(dnp no)
-		(property "Reference" "U28"
+		(property "Reference" "U31"
 			(at 63.5 88.9 0)
 			(effects
@@
 			(project "impeller18"
 				(path "/4ccab03b-4b1c-4c61-9fa8-19853ef32b4d/e2502236-aeb0-4ddd-871d-5a73d5946ae5"
-					(reference "U28")
+					(reference "U31")
 					(unit 1)
 				)
@@
 		(on_board yes)
 		(dnp no)
-		(property "Reference" "U27"
+		(property "Reference" "U30"
 			(at 63.5 76.2 0)
 			(effects
@@
 			(project "impeller18"
 				(path "/4ccab03b-4b1c-4c61-9fa8-19853ef32b4d/e2502236-aeb0-4ddd-871d-5a73d5946ae5"
-					(reference "U27")
+					(reference "U30")
 					(unit 1)
 				)
@@
 		(on_board yes)
 		(dnp no)
-		(property "Reference" "#PWR097"
+		(property "Reference" "#PWR0120"
 			(at 73.66 163.195 0)
 			(effects
@@
 			(project "impeller18"
 				(path "/4ccab03b-4b1c-4c61-9fa8-19853ef32b4d/e2502236-aeb0-4ddd-871d-5a73d5946ae5"
-					(reference "#PWR097")
+					(reference "#PWR0120")
 					(unit 1)
 				)
@@
 		(dnp no)
 		(fields_autoplaced yes)
-		(property "Reference" "#PWR098"
+		(property "Reference" "#PWR0121"
 			(at 81.28 184.15 0)
 			(effects
@@
 			(project "impeller18"
 				(path "/4ccab03b-4b1c-4c61-9fa8-19853ef32b4d/e2502236-aeb0-4ddd-871d-5a73d5946ae5"
-					(reference "#PWR098")
+					(reference "#PWR0121")
 					(unit 1)
 				)
@@
 		(on_board yes)
 		(dnp no)
-		(property "Reference" "U24"
+		(property "Reference" "U27"
 			(at 63.5 38.1 0)
 			(effects
@@
 			(project "impeller18"
 				(path "/4ccab03b-4b1c-4c61-9fa8-19853ef32b4d/e2502236-aeb0-4ddd-871d-5a73d5946ae5"
-					(reference "U24")
+					(reference "U27")
 					(unit 1)
 				)
@@
 		(on_board yes)
 		(dnp no)
-		(property "Reference" "R137"
+		(property "Reference" "R140"
 			(at 51.435 51.435 90)
 			(effects
@@
 			(project "impeller18"
 				(path "/4ccab03b-4b1c-4c61-9fa8-19853ef32b4d/e2502236-aeb0-4ddd-871d-5a73d5946ae5"
-					(reference "R137")
+					(reference "R140")
 					(unit 1)
 				)
@@
 		(on_board yes)
 		(dnp no)
-		(property "Reference" "U25"
+		(property "Reference" "U28"
 			(at 63.5 50.8 0)
 			(effects
@@
 			(project "impeller18"
 				(path "/4ccab03b-4b1c-4c61-9fa8-19853ef32b4d/e2502236-aeb0-4ddd-871d-5a73d5946ae5"
-					(reference "U25")
+					(reference "U28")
 					(unit 1)
 				)
@@
 		(on_board yes)
 		(dnp no)
-		(property "Reference" "U32"
+		(property "Reference" "U35"
 			(at 63.5 139.7 0)
 			(effects
@@
 			(project "impeller18"
 				(path "/4ccab03b-4b1c-4c61-9fa8-19853ef32b4d/e2502236-aeb0-4ddd-871d-5a73d5946ae5"
-					(reference "U32")
+					(reference "U35")
 					(unit 1)
 				)
@@
 		(on_board yes)
 		(dnp no)
-		(property "Reference" "U31"
+		(property "Reference" "U34"
 			(at 63.5 127 0)
 			(effects
@@
 			(project "impeller18"
 				(path "/4ccab03b-4b1c-4c61-9fa8-19853ef32b4d/e2502236-aeb0-4ddd-871d-5a73d5946ae5"
-					(reference "U31")
+					(reference "U34")
 					(unit 1)
 				)
@@
 		(on_board yes)
 		(dnp no)
-		(property "Reference" "R142"
+		(property "Reference" "R145"
 			(at 51.435 114.935 90)
 			(effects
@@
 			(project "impeller18"
 				(path "/4ccab03b-4b1c-4c61-9fa8-19853ef32b4d/e2502236-aeb0-4ddd-871d-5a73d5946ae5"
-					(reference "R142")
+					(reference "R145")
 					(unit 1)
 				)
@@
 		(on_board yes)
 		(dnp no)
-		(property "Reference" "R141"
+		(property "Reference" "R144"
 			(at 51.435 102.235 90)
 			(effects
@@
 			(project "impeller18"
 				(path "/4ccab03b-4b1c-4c61-9fa8-19853ef32b4d/e2502236-aeb0-4ddd-871d-5a73d5946ae5"
-					(reference "R141")
+					(reference "R144")
 					(unit 1)
 				)
@@
 		(on_board yes)
 		(dnp no)
-		(property "Reference" "U29"
+		(property "Reference" "U32"
 			(at 63.5 101.6 0)
 			(effects
@@
 			(project "impeller18"
 				(path "/4ccab03b-4b1c-4c61-9fa8-19853ef32b4d/e2502236-aeb0-4ddd-871d-5a73d5946ae5"
-					(reference "U29")
+					(reference "U32")
 					(unit 1)
 				)
@@
 		(dnp no)
 		(fields_autoplaced yes)
-		(property "Reference" "J7"
+		(property "Reference" "J10"
 			(at 67.31 177.8 0)
 			(effects
@@
 			(project "impeller18"
 				(path "/4ccab03b-4b1c-4c61-9fa8-19853ef32b4d/e2502236-aeb0-4ddd-871d-5a73d5946ae5"
-					(reference "J7")
+					(reference "J10")
 					(unit 1)
 				)
@@
 		(on_board yes)
 		(dnp no)
-		(property "Reference" "U26"
+		(property "Reference" "U29"
 			(at 63.5 63.5 0)
 			(effects
@@
 			(project "impeller18"
 				(path "/4ccab03b-4b1c-4c61-9fa8-19853ef32b4d/e2502236-aeb0-4ddd-871d-5a73d5946ae5"
-					(reference "U26")
+					(reference "U29")
 					(unit 1)
 				)
@@
 		(on_board yes)
 		(dnp no)
-		(property "Reference" "U30"
+		(property "Reference" "U33"
 			(at 63.5 114.3 0)
 			(effects
@@
 			(project "impeller18"
 				(path "/4ccab03b-4b1c-4c61-9fa8-19853ef32b4d/e2502236-aeb0-4ddd-871d-5a73d5946ae5"
-					(reference "U30")
+					(reference "U33")
 					(unit 1)
 				)
@@
 		(on_board yes)
 		(dnp no)
-		(property "Reference" "R143"
+		(property "Reference" "R146"
 			(at 51.435 127.635 90)
 			(effects
@@
 			(project "impeller18"
 				(path "/4ccab03b-4b1c-4c61-9fa8-19853ef32b4d/e2502236-aeb0-4ddd-871d-5a73d5946ae5"
-					(reference "R143")
+					(reference "R146")
 					(unit 1)
 				)
@@
 		(on_board yes)
 		(dnp no)
-		(property "Reference" "R140"
+		(property "Reference" "R143"
 			(at 51.435 89.535 90)
 			(effects
@@
 			(project "impeller18"
 				(path "/4ccab03b-4b1c-4c61-9fa8-19853ef32b4d/e2502236-aeb0-4ddd-871d-5a73d5946ae5"
-					(reference "R140")
+					(reference "R143")
 					(unit 1)
 				)
@@
 		(on_board yes)
 		(dnp no)
-		(property "Reference" "R138"
+		(property "Reference" "R141"
 			(at 51.435 64.135 90)
 			(effects
@@
 			(project "impeller18"
 				(path "/4ccab03b-4b1c-4c61-9fa8-19853ef32b4d/e2502236-aeb0-4ddd-871d-5a73d5946ae5"
-					(reference "R138")
+					(reference "R141")
 					(unit 1)
 				)
@@
 		(dnp no)
 		(fields_autoplaced yes)
-		(property "Reference" "#PWR096"
+		(property "Reference" "#PWR0119"
 			(at 35.56 40.64 0)
 			(effects
@@
 			(project "impeller18"
 				(path "/4ccab03b-4b1c-4c61-9fa8-19853ef32b4d/e2502236-aeb0-4ddd-871d-5a73d5946ae5"
-					(reference "#PWR096")
+					(reference "#PWR0119")
 					(unit 1)
 				)
@@
 		(on_board yes)
 		(dnp no)
-		(property "Reference" "R144"
+		(property "Reference" "R147"
 			(at 51.435 140.335 90)
 			(effects
@@
 			(project "impeller18"
 				(path "/4ccab03b-4b1c-4c61-9fa8-19853ef32b4d/e2502236-aeb0-4ddd-871d-5a73d5946ae5"
-					(reference "R144")
+					(reference "R147")
 					(unit 1)
 				)
@@
 		(on_board yes)
 		(dnp no)
-		(property "Reference" "R136"
+		(property "Reference" "R139"
 			(at 51.435 38.735 90)
 			(effects
@@
 			(project "impeller18"
 				(path "/4ccab03b-4b1c-4c61-9fa8-19853ef32b4d/e2502236-aeb0-4ddd-871d-5a73d5946ae5"
-					(reference "R136")
-					(unit 1)
-				)
+					(reference "R139")
+					(unit 1)
+				)

Commit message: updated impeller18 schematics
Parts:
- added J15: 430451800, symbol Connector_Generic:Conn_02x09_Odd_Even
- added R219, R220, R221, R222, R223, R224, R225, R226, R227: 220, symbol Device:R_Small
- added U55, U56, U57, U58, U59, U60, U61, U62, U63: G3VM61VY2, symbol Relay_SolidState:ASSR-1218
Connections:
- net 12V0: now also J15.10 (Pin_10), J15.12 (Pin_12), J15.14 (Pin_14), J15.16 (Pin_16), J15.18 (Pin_18), J15.2 (Pin_2), J15.4 (Pin_4), J15.6 (Pin_6), J15.8 (Pin_8)
- net 3V3: now also R219.1, R220.1, R221.1, R222.1, R223.1, R224.1, R225.1, R226.1, R227.1
- net GND_12V: now also U55.4, U56.4, U57.4, U58.4, U59.4, U60.4, U61.4, U62.4, U63.4
- new net: R225.2, U61.1
- new net: R220.2, U56.1
- new net: R227.2, U63.1
- new net: R223.2, U59.1
- new net: R222.2, U58.1
- new net: R226.2, U62.1
- new net: R224.2, U60.1
- new net: R219.2, U55.1
- new net: R221.2, U57.1
- new net LED10_GREEN_EXT: J15.1 (Pin_1), U55.3
- new net LED10_G_INPUT: U55.2
- new net LED11_GREEN_EXT: J15.3 (Pin_3), U56.3
- new net LED11_G_INPUT: U56.2
- new net LED12_GREEN_EXT: J15.5 (Pin_5), U57.3
- new net LED12_G_INPUT: U57.2
- new net LED13_GREEN_EXT: J15.7 (Pin_7), U58.3
- new net LED13_G_INPUT: U58.2
- new net LED14_GREEN_EXT: J15.9 (Pin_9), U59.3
- new net LED14_G_INPUT: U59.2
- new net LED15_GREEN_EXT: J15.11 (Pin_11), U60.3
- new net LED15_G_INPUT: U60.2
- new net LED16_GREEN_EXT: J15.13 (Pin_13), U61.3
- new net LED16_G_INPUT: U61.2
- new net LED17_GREEN_EXT: J15.15 (Pin_15), U62.3
- new net LED17_G_INPUT: U62.2
- new net LED18_GREEN_EXT: J15.17 (Pin_17), U63.3
- new net LED18_G_INPUT: U63.2

Commit message: updated schematics
Parts:
- added J11: 430450600, symbol Connector_Generic:Conn_02x03_Odd_Even
- added R138, R141, R144: 220, symbol Device:R_Small
- added U29, U32, U35: G3VM61VY2, symbol Relay_SolidState:ASSR-1218
- renumbered J10 to J12, J15 to J13, R139 to R136, R219 to R137, R140 to R139, R220 to R140, R141 to R142, R221 to R143, R142 to R145, R222 to R146, R143 to R147, R223 to R148, R144 to R149, R224 to R150, R145 to R151, R225 to R152, R146 to R153, R226 to R154, R147 to R155, R227 to R156, U55 to U28, U28 to U30, U56 to U31, U29 to U33, U57 to U34, U30 to U36, U58 to U37, U31 to U38, U59 to U39, U32 to U40, U60 to U41, U33 to U42, U61 to U43, U34 to U44, U62 to U45, U35 to U46, U63 to U47
Connections:
- net 12V0: now also J11.2 (Pin_2), J11.4 (Pin_4), J11.6 (Pin_6)
- net 3V3: now also R138.1, R141.1, R144.1
- net GND_12V: now also U29.4, U32.4, U35.4
- net LED10_GREEN_EXT renamed LED10_EXT_12V
- net LED10_G_INPUT renamed LED10_EXT
- net LED11_GREEN_EXT renamed LED11_EXT_12V
- net LED11_G_INPUT renamed LED11_EXT
- net LED12_GREEN_EXT renamed LED12_EXT_12V
- net LED12_G_INPUT renamed LED12_EXT
- net LED13_GREEN_EXT renamed LED13_EXT_12V
- net LED13_G_INPUT renamed LED13_EXT
- net LED14_GREEN_EXT renamed LED14_EXT_12V
- net LED14_G_INPUT renamed LED14_EXT
- net LED15_GREEN_EXT renamed LED15_EXT_12V
- net LED15_G_INPUT renamed LED15_EXT
- net LED16_GREEN_EXT renamed LED16_EXT_12V
- net LED16_G_INPUT renamed LED16_EXT
- net LED17_GREEN_EXT renamed LED17_EXT_12V
- net LED17_G_INPUT renamed LED17_EXT
- net LED18_GREEN_EXT renamed LED18_EXT_12V
- net LED18_G_INPUT renamed LED18_EXT
- net LED1_GREEN_EXT renamed LED1_EXT_12V
- net LED1_G_INPUT renamed LED1_EXT
- net LED2_GREEN_EXT renamed LED2_EXT_12V
- net LED2_G_INPUT renamed LED2_EXT
- net LED3_GREEN_EXT renamed LED3_EXT_12V
- net LED3_G_INPUT renamed LED3_EXT
- net LED4_GREEN_EXT renamed LED4_EXT_12V
- net LED4_G_INPUT renamed LED4_EXT
- net LED5_GREEN_EXT renamed LED5_EXT_12V
- net LED5_G_INPUT renamed LED5_EXT
- net LED6_GREEN_EXT renamed LED6_EXT_12V
- net LED6_G_INPUT renamed LED6_EXT
- net LED7_GREEN_EXT renamed LED7_EXT_12V
- net LED7_G_INPUT renamed LED7_EXT
- net LED8_GREEN_EXT renamed LED8_EXT_12V
- net LED8_G_INPUT renamed LED8_EXT
- net LED9_GREEN_EXT renamed LED9_EXT_12V
- net LED9_G_INPUT renamed LED9_EXT
- new net: R144.2, U35.1
- new net: R138.2, U29.1
- new net: R141.2, U32.1
- new net LED19_EXT: U29.2
- new net LED19_EXT_12V: J11.1 (Pin_1), U29.3
- new net LED20_EXT: U32.2
- new net LED20_EXT_12V: J11.3 (Pin_3), U32.3
- new net LED21_EXT: U35.2
- new net LED21_EXT_12V: J11.5 (Pin_5), U35.3

Commit message: updated schematics
Parts:
- added C107: 470u, symbol Device:C_Polarized_Small
- added C108: 100u, symbol Device:C_Polarized_Small
- added U68: SCWN06A-12, symbol user_lib:SCWN06A-12
Connections:
- net 12V0: now also U68.22 (+VIN), U68.23 (+VIN); no longer J11.2 (Pin_2), J11.4 (Pin_4), J11.6 (Pin_6), J12.10 (Pin_10), J12.12 (Pin_12), J12.14 (Pin_14), J12.16 (Pin_16), J12.18 (Pin_18), J12.2 (Pin_2), J12.4 (Pin_4), J12.6 (Pin_6), J12.8 (Pin_8), J13.10 (Pin_10), J13.12 (Pin_12), J13.14 (Pin_14), J13.16 (Pin_16), J13.18 (Pin_18), J13.2 (Pin_2), J13.4 (Pin_4), J13.6 (Pin_6), J13.8 (Pin_8)
- net GND_12V: now also U68.2 (-VIN), U68.3 (-VIN); no longer U27.4, U28.4, U29.4, U30.4, U31.4, U32.4, U33.4, U34.4, U35.4, U36.4, U37.4, U38.4, U39.4, U40.4, U41.4, U42.4, U43.4, U44.4, U45.4, U46.4, U47.4
- new net 12V0_LED: C107.1, C108.1, J11.2 (Pin_2), J11.4 (Pin_4), J11.6 (Pin_6), J12.10 (Pin_10), J12.12 (Pin_12), J12.14 (Pin_14), J12.16 (Pin_16), J12.18 (Pin_18), J12.2 (Pin_2), J12.4 (Pin_4), J12.6 (Pin_6), J12.8 (Pin_8), J13.10 (Pin_10), J13.12 (Pin_12), J13.14 (Pin_14), J13.16 (Pin_16), J13.18 (Pin_18), J13.2 (Pin_2), J13.4 (Pin_4), J13.6 (Pin_6), J13.8 (Pin_8), U68.14 (+VOUT)
- new net GND_LED: C107.2, C108.2, U27.4, U28.4, U29.4, U30.4, U31.4, U32.4, U33.4, U34.4, U35.4, U36.4, U37.4, U38.4, U39.4, U40.4, U41.4, U42.4, U43.4, U44.4, U45.4, U46.4, U47.4, U68.16 (-VOUT)

Commit message: updated schematics
Parts:
- added D17: FYLS-0603BUGC, symbol Device:LED
- added R181: 470, symbol Device:R_Small
- J12: renamed from J11; footprint (none) -> Connector_Molex:Molex_Micro-Fit_3.0_43045-0600_2x03_P3.00mm_Horizontal
- J13: renamed from J12; footprint (none) -> Connector_Molex:Molex_Micro-Fit_3.0_43045-1800_2x09_P3.00mm_Horizontal
- J14: renamed from J13; footprint (none) -> Connector_Molex:Molex_Micro-Fit_3.0_43045-1800_2x09_P3.00mm_Horizontal
- renumbered C107 to C88, C108 to C89, R136 to R160, R137 to R161, R138 to R162, R139 to R163, R140 to R164, R141 to R165, R142 to R166, R143 to R167, R144 to R168, R145 to R169, R146 to R170, R147 to R171, R148 to R172, R149 to R173, R150 to R174, R151 to R175, R152 to R176, R153 to R177, R154 to R178, R155 to R179, R156 to R180, U27 to U33, U28 to U34, U29 to U35, U30 to U36, U31 to U37, U32 to U38, U33 to U39, U34 to U40, U35 to U41, U36 to U42, U37 to U43, U38 to U44, U39 to U45, U40 to U46, U41 to U47, U42 to U48, U43 to U49, U44 to U50, U45 to U51, U46 to U52, U47 to U53, U68 to U54
Connections:
- net 12V0_LED: now also R181.1
- net GND_LED: now also D17.1 (K)
- new net: D17.2 (A), R181.2

Commit message: updated schematics
Parts:
- C88: Мин. кол-во (none) -> 15; Ссылка (none) -> https://www.promelec.ru/product/365892/; Цена (none) -> 34; Человекопонятное название (none) -> Конденсатор алюминиевый электролитический 470мкФ 25В
- C89: Мин. кол-во (none) -> 16; Ссылка (none) -> https://www.promelec.ru/product/367658/; Цена (none) -> 33; Человекопонятное название (none) -> Конденсатор алюминиевый электролитический 100мкФ 50В
- D17: footprint (none) -> LED_SMD:LED_0603_1608Metric; Мин. кол-во (none) -> 3; Ссылка (none) -> https://www.promelec.ru/product/324327/; Цена (none) -> 5; Человекопонятное название (none) -> Светодиод smd 1,6х0,8мм/зеленый/568нм/65мкд/прозрачный/130°
- J15: renamed from J12; footprint Connector_Molex:Molex_Micro-Fit_3.0_43045-0600_2x03_P3.00mm_Horizontal -> (none); Мин. кол-во (none) -> 8; Ссылка (none) -> https://www.promelec.ru/product/355066/; Цена (none) -> 68; Человекопонятное название (none) -> Разъем типа провод-плата, 3 мм, 6 контакт(-ов)
- J16: renamed from J13; footprint Connector_Molex:Molex_Micro-Fit_3.0_43045-1800_2x09_P3.00mm_Horizontal -> (none); Мин. кол-во (none) -> 3; Ссылка (none) -> https://www.promelec.ru/product/474708/; Цена (none) -> 175; Человекопонятное название (none) -> Соединитель провод-плата HDR 18 контакт(ов) 3мм угловой сер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
- J17: renamed from J14; footprint Connector_Molex:Molex_Micro-Fit_3.0_43045-1800_2x09_P3.00mm_Horizontal -> (none); Мин. кол-во (none) -> 3; Ссылка (none) -> https://www.promelec.ru/product/474708/; Цена (none) -> 175; Человекопонятное название (none) -> Соединитель провод-плата HDR 18 контакт(ов) 3мм угловой сер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
- R168: renamed from R160; Мин. кол-во (none) -> 100; Ссылка (none) -> https://www.promelec.ru/product/46446/; Цена (none) -> 1; Человекопонятное название (none) -> Толстопленочный ЧИП-резистор 0603 220Ом
- R169: renamed from R161; Мин. кол-во (none) -> 100; Ссылка (none) -> https://www.promelec.ru/product/46446/; Цена (none) -> 1; Человекопонятное название (none) -> Толстопленочный ЧИП-резистор 0603 220Ом
- R170: renamed from R162; Мин. кол-во (none) -> 100; Ссылка (none) -> https://www.promelec.ru/product/46446/; Цена (none) -> 1; Человекопонятное название (none) -> Толстопленочный ЧИП-резистор 0603 220Ом
- R171: renamed from R163; Мин. кол-во (none) -> 100; Ссылка (none) -> https://www.promelec.ru/product/46446/; Цена (none) -> 1; Человекопонятное название (none) -> Толстопленочный ЧИП-резистор 0603 220Ом
- R172: renamed from R164; Мин. кол-во (none) -> 100; Ссылка (none) -> https://www.promelec.ru/product/46446/; Цена (none) -> 1; Человекопонятное название (none) -> Толстопленочный ЧИП-резистор 0603 220Ом
- R173: renamed from R165; Мин. кол-во (none) -> 100; Ссылка (none) -> https://www.promelec.ru/product/46446/; Цена (none) -> 1; Человекопонятное название (none) -> Толстопленочный ЧИП-резистор 0603 220Ом
- R174: renamed from R166; Мин. кол-во (none) -> 100; Ссылка (none) -> https://www.promelec.ru/product/46446/; Цена (none) -> 1; Человекопонятное название (none) -> Толстопленочный ЧИП-резистор 0603 220Ом
- R175: renamed from R167; Мин. кол-во (none) -> 100; Ссылка (none) -> https://www.promelec.ru/product/46446/; Цена (none) -> 1; Человекопонятное название (none) -> Толстопленочный ЧИП-резистор 0603 220Ом
- R176: renamed from R168; Мин. кол-во (none) -> 100; Ссылка (none) -> https://www.promelec.ru/product/46446/; Цена (none) -> 1; Человекопонятное название (none) -> Толстопленочный ЧИП-резистор 0603 220Ом
- R177: renamed from R169; Мин. кол-во (none) -> 100; Ссылка (none) -> https://www.promelec.ru/product/46446/; Цена (none) -> 1; Человекопонятное название (none) -> Толстопленочный ЧИП-резистор 0603 220Ом
- R178: renamed from R170; Мин. кол-во (none) -> 100; Ссылка (none) -> https://www.promelec.ru/product/46446/; Цена (none) -> 1; Человекопонятное название (none) -> Толстопленочный ЧИП-резистор 0603 220Ом
- R179: renamed from R171; Мин. кол-во (none) -> 100; Ссылка (none) -> https://www.promelec.ru/product/46446/; Цена (none) -> 1; Человекопонятное название (none) -> Толстопленочный ЧИП-резистор 0603 220Ом
- R180: renamed from R172; Мин. кол-во (none) -> 100; Ссылка (none) -> https://www.promelec.ru/product/46446/; Цена (none) -> 1; Человекопонятное название (none) -> Толстопленочный ЧИП-резистор 0603 220Ом
- R181: renamed from R173; Мин. кол-во (none) -> 100; Ссылка (none) -> https://www.promelec.ru/product/46446/; Цена (none) -> 1; Человекопонятное название (none) -> Толстопленочный ЧИП-резистор 0603 220Ом
- R182: renamed from R174; Мин. кол-во (none) -> 100; Ссылка (none) -> https://www.promelec.ru/product/46446/; Цена (none) -> 1; Человекопонятное название (none) -> Толстопленочный ЧИП-резистор 0603 220Ом
- R183: renamed from R175; Мин. кол-во (none) -> 100; Ссылка (none) -> https://www.promelec.ru/product/46446/; Цена (none) -> 1; Человекопонятное название (none) -> Толстопленочный ЧИП-резистор 0603 220Ом
- R184: renamed from R176; Мин. кол-во (none) -> 100; Ссылка (none) -> https://www.promelec.ru/product/46446/; Цена (none) -> 1; Человекопонятное название (none) -> Толстопленочный ЧИП-резистор 0603 220Ом
- R185: renamed from R177; Мин. кол-во (none) -> 100; Ссылка (none) -> https://www.promelec.ru/product/46446/; Цена (none) -> 1; Человекопонятное название (none) -> Толстопленочный ЧИП-резистор 0603 220Ом
- R186: renamed from R178; Мин. кол-во (none) -> 100; Ссылка (none) -> https://www.promelec.ru/product/46446/; Цена (none) -> 1; Человекопонятное название (none) -> Толстопленочный ЧИП-резистор 0603 220Ом
- R187: renamed from R179; Мин. кол-во (none) -> 100; Ссылка (none) -> https://www.promelec.ru/product/46446/; Цена (none) -> 1; Человекопонятное название (none) -> Толстопленочный ЧИП-резистор 0603 220Ом
- R188: renamed from R180; Мин. кол-во (none) -> 100; Ссылка (none) -> https://www.promelec.ru/product/46446/; Цена (none) -> 1; Человекопонятное название (none) -> Толстопленочный ЧИП-резистор 0603 220Ом
- R189: renamed from R181; Мин. кол-во (none) -> 100; Ссылка (none) -> https://www.promelec.ru/product/109567/; Цена (none) -> 1; Человекопонятное название (none) -> Толстопленочный ЧИП-резистор 0603 470Ом
- U35: renamed from U33; Мин. кол-во (none) -> 5; Ссылка (none) -> https://www.promelec.ru/product/423382/; Цена (none) -> 112; Человекопонятное название (none) -> Реле твердотельное
- U36: renamed from U34; Мин. кол-во (none) -> 5; Ссылка (none) -> https://www.promelec.ru/product/423382/; Цена (none) -> 112; Человекопонятное название (none) -> Реле твердотельное
- U37: renamed from U35; Мин. кол-во (none) -> 5; Ссылка (none) -> https://www.promelec.ru/product/423382/; Цена (none) -> 112; Человекопонятное название (none) -> Реле твердотельное
- U38: renamed from U36; Мин. кол-во (none) -> 5; Ссылка (none) -> https://www.promelec.ru/product/423382/; Цена (none) -> 112; Человекопонятное название (none) -> Реле твердотельное
- U39: renamed from U37; Мин. кол-во (none) -> 5; Ссылка (none) -> https://www.promelec.ru/product/423382/; Цена (none) -> 112; Человекопонятное название (none) -> Реле твердотельное
- U40: renamed from U38; Мин. кол-во (none) -> 5; Ссылка (none) -> https://www.promelec.ru/product/423382/; Цена (none) -> 112; Человекопонятное название (none) -> Реле твердотельное
- U41: renamed from U39; Мин. кол-во (none) -> 5; Ссылка (none) -> https://www.promelec.ru/product/423382/; Цена (none) -> 112; Человекопонятное название (none) -> Реле твердотельное
- U42: renamed from U40; Мин. кол-во (none) -> 5; Ссылка (none) -> https://www.promelec.ru/product/423382/; Цена (none) -> 112; Человекопонятное название (none) -> Реле твердотельное
- U43: renamed from U41; Мин. кол-во (none) -> 5; Ссылка (none) -> https://www.promelec.ru/product/423382/; Цена (none) -> 112; Человекопонятное название (none) -> Реле твердотельное
- U44: renamed from U42; Мин. кол-во (none) -> 5; Ссылка (none) -> https://www.promelec.ru/product/423382/; Цена (none) -> 112; Человекопонятное название (none) -> Реле твердотельное
- U45: renamed from U43; Мин. кол-во (none) -> 5; Ссылка (none) -> https://www.promelec.ru/product/423382/; Цена (none) -> 112; Человекопонятное название (none) -> Реле твердотельное
- U46: renamed from U44; Мин. кол-во (none) -> 5; Ссылка (none) -> https://www.promelec.ru/product/423382/; Цена (none) -> 112; Человекопонятное название (none) -> Реле твердотельное
- U47: renamed from U45; Мин. кол-во (none) -> 5; Ссылка (none) -> https://www.promelec.ru/product/423382/; Цена (none) -> 112; Человекопонятное название (none) -> Реле твердотельное
- U48: renamed from U46; Мин. кол-во (none) -> 5; Ссылка (none) -> https://www.promelec.ru/product/423382/; Цена (none) -> 112; Человекопонятное название (none) -> Реле твердотельное
- U49: renamed from U47; Мин. кол-во (none) -> 5; Ссылка (none) -> https://www.promelec.ru/product/423382/; Цена (none) -> 112; Человекопонятное название (none) -> Реле твердотельное
- U50: renamed from U48; Мин. кол-во (none) -> 5; Ссылка (none) -> https://www.promelec.ru/product/423382/; Цена (none) -> 112; Человекопонятное название (none) -> Реле твердотельное
- U51: renamed from U49; Мин. кол-во (none) -> 5; Ссылка (none) -> https://www.promelec.ru/product/423382/; Цена (none) -> 112; Человекопонятное название (none) -> Реле твердотельное
- U52: renamed from U50; Мин. кол-во (none) -> 5; Ссылка (none) -> https://www.promelec.ru/product/423382/; Цена (none) -> 112; Человекопонятное название (none) -> Реле твердотельное
- U53: renamed from U51; Мин. кол-во (none) -> 5; Ссылка (none) -> https://www.promelec.ru/product/423382/; Цена (none) -> 112; Человекопонятное название (none) -> Реле твердотельное
- U54: renamed from U52; Мин. кол-во (none) -> 5; Ссылка (none) -> https://www.promelec.ru/product/423382/; Цена (none) -> 112; Человекопонятное название (none) -> Реле твердотельное
- U55: renamed from U53; Мин. кол-во (none) -> 5; Ссылка (none) -> https://www.promelec.ru/product/423382/; Цена (none) -> 112; Человекопонятное название (none) -> Реле твердотельное
- U56: renamed from U54; Мин. кол-во (none) -> 1; Ссылка (none) -> https://www.chipdip.ru/product/scwn06a-12; Цена (none) -> 1020; Человекопонятное название (none) -> DC/DC преобразователь, 6Вт, вход 9-18В, выход 12В/500мА

Commit message: updatec schematics
Parts:
- added TP25, TP26: TestPoint, symbol Connector:TestPoint
Connections:
- net 12V0_LED: now also TP25.1
- net GND_LED: now also TP26.1
