File: Hardware/ciam/impeller18/indicators.kicad_sch (KiCad schematic)
At the start: 52 parts, among them J15 430450600, J16 430451800, J17 430451800, U35 G3VM61VY2, U36 G3VM61VY2, U37 G3VM61VY2, U38 G3VM61VY2, U39 G3VM61VY2, U40 G3VM61VY2, U41 G3VM61VY2, U42 G3VM61VY2, U43 G3VM61VY2, U44 G3VM61VY2, U45 G3VM61VY2, U46 G3VM61VY2, U47 G3VM61VY2, U48 G3VM61VY2, U49 G3VM61VY2, U50 G3VM61VY2, U51 G3VM61VY2, U52 G3VM61VY2, U53 G3VM61VY2, U54 G3VM61VY2, U55 G3VM61VY2, U56 SCWN06A-12

Commit message: added footprints
Parts:
- C88: footprint (none) -> Capacitor_THT:CP_Radial_D12.5mm_P5.00mm
- C89: footprint (none) -> Capacitor_THT:CP_Radial_D8.0mm_P3.50mm
- J15: footprint (none) -> Connector_Molex:Molex_Micro-Fit_3.0_43045-0600_2x03_P3.00mm_Horizontal
- J16, J17: footprint (none) -> Connector_Molex:Molex_Micro-Fit_3.0_43045-1800_2x09_P3.00mm_Horizontal
- R168, R169, R170, R171, R172, R173, R174, R175, R176, R177, R178, R179, R180, R181, R182, R183, R184, R185, R186, R187, R188, R189: footprint (none) -> Resistor_SMD:R_0603_1608Metric
- TP25, TP26: footprint (none) -> TestPoint:TestPoint_THTPad_D1.5mm_Drill0.7mm
Changed lines of the file:
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@@
 			)
 		)
-		(property "Footprint" ""
+		(property "Footprint" "Resistor_SMD:R_0603_1608Metric"
 			(at 51.435 80.645 0)
 			(effects
@@
 			)
 		)
-		(property "Footprint" ""
+		(property "Footprint" "Resistor_SMD:R_0603_1608Metric"
 			(at 186.055 67.945 0)
 			(effects
@@
 			)
 		)
-		(property "Footprint" ""
+		(property "Footprint" "Resistor_SMD:R_0603_1608Metric"
 			(at 117.475 55.245 0)
 			(effects
@@
 			)
 		)
-		(property "Footprint" ""
+		(property "Footprint" "Resistor_SMD:R_0603_1608Metric"
 			(at 117.475 144.145 0)
 			(effects
@@
 			)
 		)
-		(property "Footprint" ""
+		(property "Footprint" "TestPoint:TestPoint_THTPad_D1.5mm_Drill0.7mm"
 			(at 90.17 250.825 0)
 			(effects
@@
 			)
 		)
-		(property "Footprint" ""
+		(property "Footprint" "Resistor_SMD:R_0603_1608Metric"
 			(at 117.475 93.345 0)
 			(effects
@@
 			)
 		)
-		(property "Footprint" ""
+		(property "Footprint" "Resistor_SMD:R_0603_1608Metric"
 			(at 186.055 42.545 0)
 			(effects
@@
 			)
 		)
-		(property "Footprint" ""
+		(property "Footprint" "Resistor_SMD:R_0603_1608Metric"
 			(at 117.475 80.645 0)
 			(effects
@@
 			)
 		)
-		(property "Footprint" ""
+		(property "Footprint" "Connector_Molex:Molex_Micro-Fit_3.0_43045-1800_2x09_P3.00mm_Horizontal"
 			(at 132.08 193.675 0)
 			(effects
@@
 			)
 		)
-		(property "Footprint" ""
+		(property "Footprint" "Capacitor_THT:CP_Radial_D8.0mm_P3.50mm"
 			(at 118.11 235.585 0)
 			(effects
@@
 			)
 		)
-		(property "Footprint" ""
+		(property "Footprint" "Resistor_SMD:R_0603_1608Metric"
 			(at 51.435 55.245 0)
 			(effects
@@
 			)
 		)
-		(property "Footprint" ""
+		(property "Footprint" "Resistor_SMD:R_0603_1608Metric"
 			(at 186.055 55.245 0)
 			(effects
@@
 			)
 		)
-		(property "Footprint" ""
+		(property "Footprint" "Resistor_SMD:R_0603_1608Metric"
 			(at 117.475 42.545 0)
 			(effects
@@
 			)
 		)
-		(property "Footprint" ""
+		(property "Footprint" "Resistor_SMD:R_0603_1608Metric"
 			(at 117.475 131.445 0)
 			(effects
@@
 			)
 		)
-		(property "Footprint" ""
+		(property "Footprint" "Resistor_SMD:R_0603_1608Metric"
 			(at 51.435 118.745 0)
 			(effects
@@
 			)
 		)
-		(property "Footprint" ""
+		(property "Footprint" "Resistor_SMD:R_0603_1608Metric"
 			(at 117.475 118.745 0)
 			(effects
@@
 			)
 		)
-		(property "Footprint" ""
+		(property "Footprint" "Resistor_SMD:R_0603_1608Metric"
 			(at 51.435 106.045 0)
 			(effects
@@
 			)
 		)
-		(property "Footprint" ""
+		(property "Footprint" "Connector_Molex:Molex_Micro-Fit_3.0_43045-1800_2x09_P3.00mm_Horizontal"
 			(at 66.04 193.675 0)
 			(effects
@@
 			)
 		)
-		(property "Footprint" ""
+		(property "Footprint" "Resistor_SMD:R_0603_1608Metric"
 			(at 117.475 67.945 0)
 			(effects
@@
 			)
 		)
-		(property "Footprint" ""
+		(property "Footprint" "Resistor_SMD:R_0603_1608Metric"
 			(at 145.415 230.505 0)
 			(effects
@@
 			)
 		)
-		(property "Footprint" ""
+		(property "Footprint" "Capacitor_THT:CP_Radial_D12.5mm_P5.00mm"
 			(at 107.95 235.585 0)
 			(effects
@@
 			)
 		)
-		(property "Footprint" ""
+		(property "Footprint" "Resistor_SMD:R_0603_1608Metric"
 			(at 51.435 131.445 0)
 			(effects
@@
 			)
 		)
-		(property "Footprint" ""
+		(property "Footprint" "Resistor_SMD:R_0603_1608Metric"
 			(at 51.435 93.345 0)
 			(effects
@@
 			)
 		)
-		(property "Footprint" ""
+		(property "Footprint" "Resistor_SMD:R_0603_1608Metric"
 			(at 51.435 67.945 0)
 			(effects
@@
 			)
 		)
-		(property "Footprint" ""
+		(property "Footprint" "TestPoint:TestPoint_THTPad_D1.5mm_Drill0.7mm"
 			(at 90.17 255.27 0)
 			(effects
@@
 			)
 		)
-		(property "Footprint" ""
+		(property "Footprint" "Resistor_SMD:R_0603_1608Metric"
 			(at 51.435 144.145 0)
 			(effects
@@
 			)
 		)
-		(property "Footprint" ""
+		(property "Footprint" "Resistor_SMD:R_0603_1608Metric"
 			(at 51.435 42.545 0)
 			(effects
@@
 			)
 		)
-		(property "Footprint" ""
+		(property "Footprint" "Connector_Molex:Molex_Micro-Fit_3.0_43045-0600_2x03_P3.00mm_Horizontal"
 			(at 199.39 191.77 0)
 			(effects
@@
 			)
 		)
-		(property "Footprint" ""
+		(property "Footprint" "Resistor_SMD:R_0603_1608Metric"
 			(at 117.475 106.045 0)
 			(effects

Commit message: Minor changes
Other:
- moved on the sheet: TP25, TP26
Changed lines of the file:
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@@
 	(wire
 		(pts
-			(xy 90.17 260.35) (xy 94.615 260.35)
+			(xy 179.07 241.935) (xy 179.07 246.38)
 		)
 		(stroke
@@
 	(wire
 		(pts
-			(xy 90.17 255.905) (xy 94.615 255.905)
+			(xy 179.07 227.33) (xy 179.07 222.885)
 		)
 		(stroke
@@
 	(symbol
 		(lib_id "Connector:TestPoint")
-		(at 90.17 255.905 90)
+		(at 179.07 227.33 180)
 		(unit 1)
 		(exclude_from_sim no)
@@
 		(dnp no)
 		(property "Reference" "TP25"
-			(at 82.55 256.54 90)
+			(at 185.42 229.235 0)
 			(effects
 				(font
@@
 		)
 		(property "Value" "TestPoint"
-			(at 85.09 254.635 90)
+			(at 189.23 231.775 0)
 			(effects
 				(font
@@
 		)
 		(property "Footprint" "TestPoint:TestPoint_THTPad_D1.5mm_Drill0.7mm"
-			(at 90.17 250.825 0)
+			(at 173.99 227.33 0)
 			(effects
 				(font
@@
 		)
 		(property "Datasheet" "~"
-			(at 90.17 250.825 0)
+			(at 173.99 227.33 0)
 			(effects
 				(font
@@
 		)
 		(property "Description" "test point"
-			(at 90.17 255.905 0)
+			(at 179.07 227.33 0)
 			(effects
 				(font
@@
 	(symbol
 		(lib_id "power:+12V")
-		(at 94.615 255.905 270)
+		(at 179.07 222.885 0)
 		(unit 1)
 		(exclude_from_sim no)
@@
 		(on_board yes)
 		(dnp no)
-		(fields_autoplaced yes)
 		(property "Reference" "#PWR0280"
-			(at 90.805 255.905 0)
+			(at 179.07 226.695 0)
 			(effects
 				(font
@@
 		)
 		(property "Value" "12V0_LED"
-			(at 97.79 255.9049 90)
+			(at 174.625 218.44 0)
 			(effects
 				(font
@@
 		)
 		(property "Footprint" ""
-			(at 94.615 255.905 0)
+			(at 179.07 222.885 0)
 			(effects
 				(font
@@
 		)
 		(property "Datasheet" ""
-			(at 94.615 255.905 0)
+			(at 179.07 222.885 0)
 			(effects
 				(font
@@
 		)
 		(property "Description" "Power symbol creates a global label with name \"+12V\""
-			(at 94.615 255.905 0)
+			(at 179.07 222.885 0)
 			(effects
 				(font
@@
 	(symbol
 		(lib_id "power:GND")
-		(at 94.615 260.35 90)
+		(at 179.07 246.38 0)
 		(unit 1)
 		(exclude_from_sim no)
@@
 		(dnp no)
 		(property "Reference" "#PWR0279"
-			(at 100.965 260.35 0)
+			(at 179.07 252.73 0)
 			(effects
 				(font
@@
 		)
 		(property "Value" "GND_LED"
-			(at 102.235 260.35 90)
+			(at 179.07 250.825 0)
 			(effects
 				(font
@@
 		)
 		(property "Footprint" ""
-			(at 94.615 260.35 0)
+			(at 179.07 246.38 0)
 			(effects
 				(font
@@
 		)
 		(property "Datasheet" ""
-			(at 94.615 260.35 0)
+			(at 179.07 246.38 0)
 			(effects
 				(font
@@
 		)
 		(property "Description" "Power symbol creates a global label with name \"GND\" , ground"
-			(at 94.615 260.35 0)
+			(at 179.07 246.38 0)
 			(effects
 				(font
@@
 	(symbol
 		(lib_id "Connector:TestPoint")
-		(at 90.17 260.35 90)
+		(at 179.07 241.935 0)
 		(unit 1)
 		(exclude_from_sim no)
@@
 		(dnp no)
 		(property "Reference" "TP26"
-			(at 82.55 260.985 90)
+			(at 180.34 237.49 0)
 			(effects
 				(font
@@
 		)
 		(property "Value" "TestPoint"
-			(at 85.09 259.08 90)
+			(at 180.34 240.03 0)
 			(effects
 				(font
@@
 		)
 		(property "Footprint" "TestPoint:TestPoint_THTPad_D1.5mm_Drill0.7mm"
-			(at 90.17 255.27 0)
+			(at 184.15 241.935 0)
 			(effects
 				(font
@@
 		)
 		(property "Datasheet" "~"
-			(at 90.17 255.27 0)
+			(at 184.15 241.935 0)
 			(effects
 				(font
@@
 		)
 		(property "Description" "test point"
-			(at 90.17 260.35 0)
+			(at 179.07 241.935 0)
 			(effects
 				(font

Commit message: Updated packeges
Parts:
- J15: footprint Connector_Molex:Molex_Micro-Fit_3.0_43045-0600_2x03_P3.00mm_Horizontal -> user_lib:430450600
- J16, J17: footprint Connector_Molex:Molex_Micro-Fit_3.0_43045-1800_2x09_P3.00mm_Horizontal -> user_lib:430451800
Other:
- note added: "32.4 м"
Changed lines of the file:
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@@
 		)
 	)
+	(text "32.4 м"
+		(exclude_from_sim no)
+		(at 231.775 146.685 0)
+		(effects
+			(font
+				(size 12.7 12.7)
+				(thickness 2.54)
+				(bold yes)
+			)
+		)
+	)
 	(label "LED7_EXT_12V"
 		(at 91.44 123.825 180)
@@
 			)
 		)
-		(property "Footprint" "Connector_Molex:Molex_Micro-Fit_3.0_43045-1800_2x09_P3.00mm_Horizontal"
+		(property "Footprint" "user_lib:430451800"
 			(at 132.08 193.675 0)
 			(effects
@@
 			)
 		)
-		(property "Footprint" "Connector_Molex:Molex_Micro-Fit_3.0_43045-1800_2x09_P3.00mm_Horizontal"
+		(property "Footprint" "user_lib:430451800"
 			(at 66.04 193.675 0)
 			(effects
@@
 			)
 		)
-		(property "Footprint" "Connector_Molex:Molex_Micro-Fit_3.0_43045-0600_2x03_P3.00mm_Horizontal"
+		(property "Footprint" "user_lib:430450600"
 			(at 199.39 191.77 0)
 			(effects

Commit message: Updated packeges
Parts:
- U35, U36, U37, U38, U39, U40, U41, U42, U43, U44, U45, U46, U47, U48, U49, U50, U51, U52, U53, U54, U55: footprint (none) -> user_lib:G3VM-61VY2TR
- U56: footprint (none) -> user_lib:SCWN06A-12
Changed lines of the file:
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@@
 			)
 		)
-		(property "Footprint" ""
+		(property "Footprint" "user_lib:G3VM-61VY2TR"
 			(at 58.42 100.965 0)
 			(effects
@@
 			)
 		)
-		(property "Footprint" ""
+		(property "Footprint" "user_lib:G3VM-61VY2TR"
 			(at 58.42 88.265 0)
 			(effects
@@
 			)
 		)
-		(property "Footprint" ""
+		(property "Footprint" "user_lib:G3VM-61VY2TR"
 			(at 124.46 126.365 0)
 			(effects
@@
 			)
 		)
-		(property "Footprint" ""
+		(property "Footprint" "user_lib:SCWN06A-12"
 			(at 91.567 246.507 0)
 			(effects
@@
 			)
 		)
-		(property "Footprint" ""
+		(property "Footprint" "user_lib:G3VM-61VY2TR"
 			(at 58.42 50.165 0)
 			(effects
@@
 			)
 		)
-		(property "Footprint" ""
+		(property "Footprint" "user_lib:G3VM-61VY2TR"
 			(at 124.46 139.065 0)
 			(effects
@@
 			)
 		)
-		(property "Footprint" ""
+		(property "Footprint" "user_lib:G3VM-61VY2TR"
 			(at 124.46 113.665 0)
 			(effects
@@
 			)
 		)
-		(property "Footprint" ""
+		(property "Footprint" "user_lib:G3VM-61VY2TR"
 			(at 58.42 62.865 0)
 			(effects
@@
 			)
 		)
-		(property "Footprint" ""
+		(property "Footprint" "user_lib:G3VM-61VY2TR"
 			(at 58.42 151.765 0)
 			(effects
@@
 			)
 		)
-		(property "Footprint" ""
+		(property "Footprint" "user_lib:G3VM-61VY2TR"
 			(at 58.42 139.065 0)
 			(effects
@@
 			)
 		)
-		(property "Footprint" ""
+		(property "Footprint" "user_lib:G3VM-61VY2TR"
 			(at 58.42 113.665 0)
 			(effects
@@
 			)
 		)
-		(property "Footprint" ""
+		(property "Footprint" "user_lib:G3VM-61VY2TR"
 			(at 58.42 75.565 0)
 			(effects
@@
 			)
 		)
-		(property "Footprint" ""
+		(property "Footprint" "user_lib:G3VM-61VY2TR"
 			(at 193.04 50.165 0)
 			(effects
@@
 			)
 		)
-		(property "Footprint" ""
+		(property "Footprint" "user_lib:G3VM-61VY2TR"
 			(at 124.46 151.765 0)
 			(effects
@@
 			)
 		)
-		(property "Footprint" ""
+		(property "Footprint" "user_lib:G3VM-61VY2TR"
 			(at 193.04 75.565 0)
 			(effects
@@
 			)
 		)
-		(property "Footprint" ""
+		(property "Footprint" "user_lib:G3VM-61VY2TR"
 			(at 124.46 75.565 0)
 			(effects
@@
 			)
 		)
-		(property "Footprint" ""
+		(property "Footprint" "user_lib:G3VM-61VY2TR"
 			(at 124.46 50.165 0)
 			(effects
@@
 			)
 		)
-		(property "Footprint" ""
+		(property "Footprint" "user_lib:G3VM-61VY2TR"
 			(at 58.42 126.365 0)
 			(effects
@@
 			)
 		)
-		(property "Footprint" ""
+		(property "Footprint" "user_lib:G3VM-61VY2TR"
 			(at 124.46 100.965 0)
 			(effects
@@
 			)
 		)
-		(property "Footprint" ""
+		(property "Footprint" "user_lib:G3VM-61VY2TR"
 			(at 193.04 62.865 0)
 			(effects
@@
 			)
 		)
-		(property "Footprint" ""
+		(property "Footprint" "user_lib:G3VM-61VY2TR"
 			(at 124.46 62.865 0)
 			(effects
@@
 			)
 		)
-		(property "Footprint" ""
+		(property "Footprint" "user_lib:G3VM-61VY2TR"
 			(at 124.46 88.265 0)
 			(effects
