File: Hardware/ciam/impeller18/impeller18.kicad_sch (KiCad schematic)
At the start: 0 parts

Commit message: updated impeller18 schamatic
Other:
- sheet Switches renamed Switches_1
- added sheet Digital inputs 5V (digital_inputs.kicad_sch)
- added sheet Switches_2 (switches_2.kicad_sch)
- sheet Switches_1: file switches.kicad_sch -> switches_1.kicad_sch
Changed lines of the file:
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@@
 	(sheet
 		(at 93.98 15.875)
-		(size 23.495 16.51)
-		(fields_autoplaced yes)
-		(stroke
-			(width 0.1524)
-			(type solid)
-		)
-		(fill
-			(color 0 0 0 0.0000)
-		)
-		(property "Sheetname" "Switches"
+		(size 27.94 16.51)
+		(fields_autoplaced yes)
+		(stroke
+			(width 0.1524)
+			(type solid)
+		)
+		(fill
+			(color 0 0 0 0.0000)
+		)
+		(property "Sheetname" "Switches_1"
 			(at 93.98 15.1634 0)
 			(effects
@@
 			)
 		)
-		(property "Sheetfile" "switches.kicad_sch"
+		(property "Sheetfile" "switches_1.kicad_sch"
 			(at 93.98 32.9696 0)
 			(effects
@@
 			(project "impeller18"
 				(path "/4ccab03b-4b1c-4c61-9fa8-19853ef32b4d"
-					(page "6")
+					(page "9")
 				)
 			)
@@
 				)
 			)
+		)
+	)
+	(sheet
+		(at 124.46 15.875)
+		(size 23.495 16.51)
+		(fields_autoplaced yes)
+		(stroke
+			(width 0.1524)
+			(type solid)
+		)
+		(fill
+			(color 0 0 0 0.0000)
+		)
+		(property "Sheetname" "Digital inputs 5V"
+			(at 124.46 15.1634 0)
+			(effects
+				(font
+					(size 1.27 1.27)
+				)
+				(justify left bottom)
+			)
+		)
+		(property "Sheetfile" "digital_inputs.kicad_sch"
+			(at 124.46 32.9696 0)
+			(effects
+				(font
+					(size 1.27 1.27)
+				)
+				(justify left top)
+			)
+		)
+		(instances
+			(project "impeller18"
+				(path "/4ccab03b-4b1c-4c61-9fa8-19853ef32b4d"
+					(page "10")
+				)
+			)
+		)
+	)
+	(sheet
+		(at 93.98 38.1)
+		(size 27.94 16.51)
+		(fields_autoplaced yes)
+		(stroke
+			(width 0.1524)
+			(type solid)
+		)
+		(fill
+			(color 0 0 0 0.0000)
+		)
+		(property "Sheetname" "Switches_2"
+			(at 93.98 37.3884 0)
+			(effects
+				(font
+					(size 1.27 1.27)
+				)
+				(justify left bottom)
+			)
+		)
+		(property "Sheetfile" "switches_2.kicad_sch"
+			(at 93.98 55.1946 0)
+			(effects
+				(font
+					(size 1.27 1.27)
+				)
+				(justify left top)
+			)
+		)
+		(instances
+			(project "impeller18"
+				(path "/4ccab03b-4b1c-4c61-9fa8-19853ef32b4d"
+					(page "6")
+				)
+			)

Commit message: updated schematics
Parts:
- added C1, C2: 2u2, Capacitor_SMD:C_0603_1608Metric, symbol Device:C
- added C10, C11, C12, C13, C14, C15, C16, C18, C20, C4, C5, C6, C7, C8, C9: 100n, symbol Device:C_Small
- added C17, C19: 1u, symbol Device:C_Small
- added C21, C23: 15p, Capacitor_SMD:C_0603_1608Metric, symbol Device:C_Small
- added C22: 100n, Capacitor_SMD:C_0603_1608Metric, symbol Device:C
- added C24, C25: 8p, Capacitor_SMD:C_0603_1608Metric, symbol Device:C_Small
- added C3: 4u7, symbol Device:C_Small
- added R1: 10k, Resistor_SMD:R_0603_1608Metric, symbol Device:R
- added SW1: SW_RESET, user_lib:tactile switch 6x6mm smd, symbol Switch:SW_Push
- added SW2: SW_BOOT0, user_lib:MSS-12D16, symbol Switch:SW_SPDT
- added U1: STM32F427ZGTx, Package_QFP:LQFP-144_20x20mm_P0.5mm, symbol MCU_ST_STM32F4:STM32F427ZGTx
- added Y1: KSE-7K32768KDY2400A3, user_lib:KSE-7K32768KDY2400A3, symbol Device:Crystal
- added Y2: X322516MLB4SI, Crystal:Crystal_SMD_3225-4Pin_3.2x2.5mm, symbol Device:Crystal_GND24
Connections:
- new net: R1.2, SW2.2 (B)
- new net 3V3: C10.1, C11.1, C12.1, C13.1, C14.1, C15.1, C17.1, C18.1, C19.1, C20.1, C3.1, C4.1, C5.1, C6.1, C7.1, C8.1, C9.1, SW2.1 (A), U1.108 (VDD), U1.121 (VDD), U1.131 (VDD), U1.144 (VDD), U1.17 (VDD), U1.30 (VDD), U1.33 (VDDA), U1.39 (VDD), U1.52 (VDD), U1.62 (VDD), U1.72 (VDD), U1.84 (VDD), U1.95 (VDD)
- new net 3V3_VBAT: C16.1, U1.6 (VBAT)
- new net BOOT0: R1.1, U1.138 (BOOT0)
- new net DEBUG_SWD_CLK: U1.109 (PA14)
- new net DEBUG_SWD_IO: U1.105 (PA13)
- new net DEBUG_SWD_SWO: U1.133 (PB3)
- new net GND: C1.2, C10.2, C11.2, C12.2, C13.2, C14.2, C15.2, C16.2, C17.2, C18.2, C19.2, C2.2, C20.2, C21.1, C22.2, C23.1, C24.2, C25.2, C3.2, C4.2, C5.2, C6.2, C7.2, C8.2, C9.2, SW1.2, SW2.3 (C), U1.107 (VSS), U1.120 (VSS), U1.130 (VSS), U1.16 (VSS), U1.31 (VSSA), U1.38 (VSS), U1.51 (VSS), U1.61 (VSS), U1.83 (VSS), U1.94 (VSS), Y2.2, Y2.4
- new net HSE_IN: C24.1, U1.23 (PH0), Y2.1
- new net HSE_OUT: C25.1, U1.24 (PH1), Y2.3
- new net LSE_IN: C21.2, U1.8 (PC14), Y1.2
- new net LSE_OUT: C23.2, U1.9 (PC15), Y1.1
- new net NRST: C22.1, SW1.1, U1.25 (NRST)
- new net SDIO_CLK: U1.113 (PC12)
- new net SDIO_CMD: U1.116 (PD2)
- new net SDIO_DAT0: U1.98 (PC8)
- new net SDIO_DAT1: U1.99 (PC9)
- new net SDIO_DAT2: U1.111 (PC10)
- new net SDIO_DAT3: U1.112 (PC11)
- new net VCAP_1: C1.1, U1.71 (VCAP_1)
- new net VCAP_2: C2.1, U1.106 (VCAP_2)
Other:
- sheet ADC renamed ADC_EXT
- sheet Encoders renamed ADC_RUD
- added sheet STM32 Peripherals (stm32_peripherals.kicad_sch)
- sheet ADC_RUD: file encoders.kicad_sch -> adc_rud.kicad_sch
- note added: "BOOT0"
- note added: "HSE"
- note added: "KSE-7K32768KDY2400A3 32.768 KHz 12.5pF"
- note added: "LSE"
- note added: "POWER SUPPLY"
- note added: "RESET"
- note added: "VBAT"
- note added: "VCAP"
- note added: "VDD"
- note added: "VDDA"
- note added: "VREF"
- note added: "X322516MLB4SI 16MHz 9pF"

Commit message: updated impeller18 schematics
Parts:
- removed C25: 8p, Capacitor_SMD:C_0603_1608Metric, symbol Device:C_Small
- added BT1: KLS5-CR2032-01, user_lib:KLS5-CR2032-01, symbol Device:Battery_Cell
- added C107: 8p, Capacitor_SMD:C_0603_1608Metric, symbol Device:C_Small
- added SW3: SW_SPDT, symbol Switch:SW_SPDT
- SW2: value SW_BOOT0 -> SW_SPDT; footprint user_lib:MSS-12D16 -> (none)
Connections:
- net 3V3: now also U1.143 (PDR_ON), U1.32 (VREF+), SW3.1 (A)
- net 3V3_VBAT: now also SW2.2 (B)
- net GND: now also C24.1, Y2.1, Y2.3, BT1.2 (-), C107.1, SW3.3 (C); no longer C24.2, SW2.3 (C), Y2.2, Y2.4
- net HSE_IN: now also C24.2, Y2.2; no longer C24.1, Y2.1
- net HSE_OUT: now also Y2.4, C107.2; no longer Y2.3
- net at R1.2: now also SW3.2 (B); no longer SW2.2 (B)
- net USB_VBUS: now reaches U1.101 (PA9)
- net USB_D-: now reaches U1.103 (PA11)
- net USB_D+: now reaches U1.104 (PA12)
- new net: BT1.1 (+), SW2.3 (C)
Other:
- added sheet Fan (fan.kicad_sch)
- note added: "KSE-7K32768KDY2400A3 32.768 KHz 12.5 pF"
- note added: "X322516MLB4SI 16 MHz 9 pF"
- note removed: "KSE-7K32768KDY2400A3 32.768 KHz 12.5pF"
- note removed: "X322516MLB4SI 16MHz 9pF"

Commit message: updated schematics
Parts:
- added J1: BH1,27-10-G, symbol Connector_Generic:Conn_02x05_Odd_Even
- added J2: PLS-6, symbol Connector_Generic:Conn_01x06
- added JP1: SolderJumper2, symbol Jumper:SolderJumper_2_Open
- SW2: renamed from SW3; value SW_SPDT -> MSS-12D16
- SW3: renamed from SW2; value SW_SPDT -> MSS-12D16
- renumbered C24 to C21, C21 to C22, C22 to C23, C23 to C24, C107 to C25, Y2 to Y1, Y1 to Y2
Connections:
- net 3V3: now also J2.4 (Pin_4), JP1.1 (A)
- net DEBUG_SWD_CLK: now also J1.4 (Pin_4), J2.3 (Pin_3)
- net DEBUG_SWD_IO: now also J1.2 (Pin_2), J2.1 (Pin_1)
- net DEBUG_SWD_SWO: now also J1.6 (Pin_6), J2.6 (Pin_6)
- net GND: now also J1.3 (Pin_3), J1.5 (Pin_5), J1.9 (Pin_9), J2.2 (Pin_2)
- net NRST: now also J1.10 (Pin_10), J2.5 (Pin_5)
- new net: J1.1 (Pin_1), JP1.2 (B)
- no-connect marks 0 -> 2
Other:
- sheet ADC_EXT renamed ADC8
- note added: "SWD debug connnectors"

Commit message: updated schematics
Parts:
- added J23: Conn_01x03, symbol Connector_Generic:Conn_01x03
- BT1: Ссылка https://www.chipdip.ru/product/bh-642 -> (none); Цена 16 -> (none); Человекопонятное название Разъем для плоской батарейки 3В -> (none)
- C22, C24: Ссылка https://www.chipdip.ru/product/grm1885c2a150j -> (none); Цена 6 -> (none); Человекопонятное название Конденсатор 15пФ -> (none)
- Y2: Ссылка https://www.chipdip.ru/product0/8022143960 -> (none); Человекопонятное название Кристаллический резонатор 32КГц -> (none)
Connections:
- net GND: now also J23.3 (Pin_3)
- new net UART1_STM32_RX: J23.1 (Pin_1)
- new net UART1_STM32_TX: J23.2 (Pin_2)
Other:
- note added: "UART1"
- note added: "Вместо X вписать номер (UART1 занят)"
- moved on the sheet: J2

Commit message: updated schematics
Parts:
- BT1: footprint user_lib:KLS5-CR2032-01 -> (none); Мин. кол-во (none) -> 1; Ссылка (none) -> https://www.chipdip.ru/product/bh-642; Цена (none) -> 18; Человекопонятное название (none) -> Батарейный отсек на 1xCR2032
- C1, C2: Мин. кол-во (none) -> 10; Ссылка (none) -> https://www.chipdip.ru/product/grm188r61a225k; Цена (none) -> 13; Человекопонятное название (none) -> Конденсатор керамический smd 2.2мкФ
- C10, C11, C12, C13, C14, C15, C16, C18, C20, C4, C5, C6, C7, C8, C9: Мин. кол-во (none) -> 300; Ссылка (none) -> https://www.promelec.ru/product/323633/; Цена (none) -> 2; Человекопонятное название (none) -> Керамический ЧИП-конденсатор 0603 X7R 0.1мкФ
- C17, C19: Мин. кол-во (none) -> 200; Ссылка (none) -> https://www.promelec.ru/product/334556/; Цена (none) -> 1; Человекопонятное название (none) -> Керамический ЧИП-конденсатор 0603 X7R 1мкФ
- C21, C25: footprint Capacitor_SMD:C_0603_1608Metric -> (none); Мин. кол-во (none) -> 500; Ссылка (none) -> https://www.promelec.ru/product/428876/; Цена (none) -> 1; Человекопонятное название (none) -> Керамический ЧИП-конденсатор 0603 NP0 8пФ
- C22, C24: footprint Capacitor_SMD:C_0603_1608Metric -> (none); Мин. кол-во (none) -> 10; Ссылка (none) -> https://www.chipdip.ru/product/grm1885c1h150j; Цена (none) -> 7; Человекопонятное название (none) -> Конденсатор керамический smd 15пФ
- C23: footprint Capacitor_SMD:C_0603_1608Metric -> (none); Мин. кол-во (none) -> 300; Ссылка (none) -> https://www.promelec.ru/product/323633/; Цена (none) -> 2; Человекопонятное название (none) -> Керамический ЧИП-конденсатор 0603 X7R 0.1мкФ
- C3: Мин. кол-во (none) -> 200; Ссылка (none) -> https://www.promelec.ru/product/315964/; Цена (none) -> 4; Человекопонятное название (none) -> Керамический ЧИП-конденсатор 0603 X5R 4.7мкФ
- J2: renamed from J1; Мин. кол-во (none) -> 1; Ссылка (none) -> https://energoflot.ru/item/C3503-10SGB000R+BH1%2C27-10-G; Цена (none) -> 97; Человекопонятное название (none) -> Разъем штыревой 1x05 1.27x1.27
- J3: renamed from J23; value Conn_01x03 -> 530470310; Мин. кол-во (none) -> 1; Ссылка (none) -> https://energoflot.ru/item/530470310; Цена (none) -> 20; Человекопонятное название (none) -> Разъем PicoBlade штекер на плату прямой 1,25мм 3pin
- R1: footprint Resistor_SMD:R_0603_1608Metric -> (none); Мин. кол-во (none) -> 1000; Ссылка (none) -> https://www.promelec.ru/product/344748/; Цена (none) -> 1; Человекопонятное название (none) -> Толстопленочный ЧИП-резистор 0603 10кОм
- SW1: value SW_RESET -> B3F1060; footprint user_lib:tactile switch 6x6mm smd -> (none); Мин. кол-во (none) -> 1; Ссылка (none) -> https://www.promelec.ru/product/430220/; Цена (none) -> 15; Человекопонятное название (none) -> Кнопка тактильная 6х6 h=7мм
- U1: footprint Package_QFP:LQFP-144_20x20mm_P0.5mm -> (none); Мин. кол-во (none) -> 1; Ссылка (none) -> https://www.promelec.ru/product/241424/; Цена (none) -> 726; Человекопонятное название (none) -> Микроконтроллер STM 32
- Y1: footprint Crystal:Crystal_SMD_3225-4Pin_3.2x2.5mm -> (none); Мин. кол-во (none) -> 1; Ссылка (none) -> https://energoflot.ru/item/X322516MLB4SI; Цена (none) -> 5; Человекопонятное название (none) -> Резонатор кварцевый smd
- Y2: footprint user_lib:KSE-7K32768KDY2400A3 -> (none); Мин. кол-во (none) -> 1; Ссылка (none) -> https://www.chipdip.ru/product0/8022143960; Цена 34 -> 36; Человекопонятное название (none) -> SMD-резонатор
- renumbered J2 to J1

Commit message: updatec schematics
Parts:
- added J26: PLS-3, symbol Connector_Generic:Conn_01x03
- added TP1, TP2: TestPoint, symbol Connector:TestPoint
- J3: value 530470310 -> PLS-3; Мин. кол-во 1 -> (none); Ссылка https://energoflot.ru/item/530470310 -> (none); Цена 20 -> (none); Человекопонятное название Разъем PicoBlade штекер на плату прямой 1,25мм 3pin -> (none)
Connections:
- net GND: now also J26.3 (Pin_3)
- net HSE_IN: now also TP1.1
- net LSE_IN: now also TP2.1
- net UARTX_STM32_RX: now also J26.2 (Pin_2)
- net UARTX_STM32_TX: now also J26.1 (Pin_1)
Other:
- note added: "UART"
- note added: "Вместо X вписать номер (UART1 занят) 1. тут 2. на этом листе где коннекторы 3. в rpi"
- note removed: "UART1"
- note removed: "Вместо X вписать номер (UART1 занят)"
