File: Hardware/ciam/impeller18/adc.kicad_sch (KiCad schematic)
At the start: 49 parts, among them J18 430451600, Q36 BSS138, U57 B0505MT-1WR4, U58 HCPL-0600, U59 MCP3008, U60 HCPL-0630, U61 IP4220, U62 HCPL-0600, U63 IP4220

Commit message: Minor changes
Other:
- moved on the sheet: TP27, TP28
Changed lines of the file:
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@@
 	(wire
 		(pts
-			(xy 200.66 76.835) (xy 205.105 76.835)
+			(xy 278.13 64.135) (xy 278.13 68.58)
 		)
 		(stroke
@@
 	(wire
 		(pts
-			(xy 200.66 72.39) (xy 205.105 72.39)
+			(xy 278.13 49.53) (xy 278.13 45.085)
 		)
 		(stroke
@@
 	(symbol
 		(lib_id "Connector:TestPoint")
-		(at 200.66 76.835 90)
+		(at 278.13 64.135 0)
 		(unit 1)
 		(exclude_from_sim no)
@@
 		(dnp no)
 		(property "Reference" "TP28"
-			(at 193.04 77.47 90)
+			(at 279.4 59.69 0)
 			(effects
 				(font
@@
 		)
 		(property "Value" "TestPoint"
-			(at 195.58 75.565 90)
+			(at 279.4 62.23 0)
 			(effects
 				(font
@@
 		)
 		(property "Footprint" "TestPoint:TestPoint_THTPad_D1.5mm_Drill0.7mm"
-			(at 200.66 71.755 0)
+			(at 283.21 64.135 0)
 			(effects
 				(font
@@
 		)
 		(property "Datasheet" "~"
-			(at 200.66 71.755 0)
+			(at 283.21 64.135 0)
 			(effects
 				(font
@@
 		)
 		(property "Description" "test point"
-			(at 200.66 76.835 0)
+			(at 278.13 64.135 0)
 			(effects
 				(font
@@
 	(symbol
 		(lib_id "power:+5V")
-		(at 205.105 72.39 270)
+		(at 278.13 45.085 0)
 		(unit 1)
 		(exclude_from_sim no)
@@
 		(fields_autoplaced yes)
 		(property "Reference" "#PWR0282"
-			(at 201.295 72.39 0)
+			(at 278.13 48.895 0)
 			(effects
 				(font
@@
 		)
 		(property "Value" "5V0_ADC"
-			(at 208.28 72.3899 90)
+			(at 278.1299 41.91 90)
 			(effects
 				(font
@@
 		)
 		(property "Footprint" ""
-			(at 205.105 72.39 0)
+			(at 278.13 45.085 0)
 			(effects
 				(font
@@
 		)
 		(property "Datasheet" ""
-			(at 205.105 72.39 0)
+			(at 278.13 45.085 0)
 			(effects
 				(font
@@
 		)
 		(property "Description" "Power symbol creates a global label with name \"+5V\""
-			(at 205.105 72.39 0)
+			(at 278.13 45.085 0)
 			(effects
 				(font
@@
 	(symbol
 		(lib_id "power:GND")
-		(at 205.105 76.835 90)
+		(at 278.13 68.58 0)
 		(unit 1)
 		(exclude_from_sim no)
@@
 		(dnp no)
 		(property "Reference" "#PWR0281"
-			(at 211.455 76.835 0)
+			(at 278.13 74.93 0)
 			(effects
 				(font
@@
 		)
 		(property "Value" "GND_ADC"
-			(at 212.725 76.835 90)
+			(at 278.13 76.2 90)
 			(effects
 				(font
@@
 		)
 		(property "Footprint" ""
-			(at 205.105 76.835 0)
+			(at 278.13 68.58 0)
 			(effects
 				(font
@@
 		)
 		(property "Datasheet" ""
-			(at 205.105 76.835 0)
+			(at 278.13 68.58 0)
 			(effects
 				(font
@@
 		)
 		(property "Description" ""
-			(at 205.105 76.835 0)
+			(at 278.13 68.58 0)
 			(effects
 				(font
@@
 	(symbol
 		(lib_id "Connector:TestPoint")
-		(at 200.66 72.39 90)
+		(at 278.13 49.53 180)
 		(unit 1)
 		(exclude_from_sim no)
@@
 		(dnp no)
 		(property "Reference" "TP27"
-			(at 193.04 73.025 90)
+			(at 284.48 51.435 0)
 			(effects
 				(font
@@
 		)
 		(property "Value" "TestPoint"
-			(at 195.58 71.12 90)
+			(at 288.29 53.975 0)
 			(effects
 				(font
@@
 		)
 		(property "Footprint" "TestPoint:TestPoint_THTPad_D1.5mm_Drill0.7mm"
-			(at 200.66 67.31 0)
+			(at 273.05 49.53 0)
 			(effects
 				(font
@@
 		)
 		(property "Datasheet" "~"
-			(at 200.66 67.31 0)
+			(at 273.05 49.53 0)
 			(effects
 				(font
@@
 		)
 		(property "Description" "test point"
-			(at 200.66 72.39 0)
+			(at 278.13 49.53 0)
 			(effects
 				(font

Commit message: Updated packeges
Parts:
- J18: footprint Connector_Molex:Molex_Micro-Fit_3.0_43045-1600_2x08_P3.00mm_Horizontal -> user_lib:430451600
Changed lines of the file:
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@@
 			)
 		)
-		(property "Footprint" "Connector_Molex:Molex_Micro-Fit_3.0_43045-1600_2x08_P3.00mm_Horizontal"
+		(property "Footprint" "user_lib:430451600"
 			(at 59.055 157.48 0)
 			(effects

Commit message: Updated 3D models
Parts:
- renumbered C90 to C105, C91 to C106, C92 to C107, C93 to C108, C94 to C109, C95 to C110, J18 to J26, Q36 to Q58, R190 to R250, R191 to R251, R192 to R252, R193 to R253, R194 to R254, R195 to R255, R196 to R256, R197 to R257, R198 to R258, R199 to R259, R200 to R260, R201 to R261, R202 to R262, R203 to R263, R204 to R264, R205 to R265, R206 to R266, R207 to R267, R208 to R268, R209 to R269, R210 to R270, R211 to R271, R212 to R272, R213 to R273, R214 to R274, R215 to R275, R216 to R276, R217 to R277, R218 to R278, R219 to R279, R220 to R280, TP27 to TP38, TP28 to TP39, U57 to U56, U58 to U57, U59 to U58, U60 to U59, U61 to U60, U62 to U61, U63 to U62

Commit message: updated bom
Parts:
- renumbered C105 to C108, C106 to C109, C107 to C110, C108 to C111, C109 to C112, C110 to C113
Changed lines of the file:
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@@
 		(on_board yes)
 		(dnp no)
-		(property "Reference" "C106"
+		(property "Reference" "C109"
 			(at 184.785 58.42 0)
 			(effects
@@
 			(project "impeller18"
 				(path "/4ccab03b-4b1c-4c61-9fa8-19853ef32b4d/bb535897-f2f1-40b8-a983-287c6650a9b5"
-					(reference "C106")
+					(reference "C109")
 					(unit 1)
 				)
@@
 		(on_board yes)
 		(dnp no)
-		(property "Reference" "C107"
+		(property "Reference" "C110"
 			(at 221.615 58.42 0)
 			(effects
@@
 			(project "impeller18"
 				(path "/4ccab03b-4b1c-4c61-9fa8-19853ef32b4d/bb535897-f2f1-40b8-a983-287c6650a9b5"
-					(reference "C107")
+					(reference "C110")
 					(unit 1)
 				)
@@
 		(on_board yes)
 		(dnp no)
-		(property "Reference" "C105"
+		(property "Reference" "C108"
 			(at 175.26 58.42 0)
 			(effects
@@
 			(project "impeller18"
 				(path "/4ccab03b-4b1c-4c61-9fa8-19853ef32b4d/bb535897-f2f1-40b8-a983-287c6650a9b5"
-					(reference "C105")
+					(reference "C108")
 					(unit 1)
 				)
@@
 		(on_board yes)
 		(dnp no)
-		(property "Reference" "C110"
+		(property "Reference" "C113"
 			(at 217.17 104.775 90)
 			(effects
@@
 			(project "impeller18"
 				(path "/4ccab03b-4b1c-4c61-9fa8-19853ef32b4d/bb535897-f2f1-40b8-a983-287c6650a9b5"
-					(reference "C110")
+					(reference "C113")
 					(unit 1)
 				)
@@
 		(on_board yes)
 		(dnp no)
-		(property "Reference" "C109"
+		(property "Reference" "C112"
 			(at 196.85 104.775 90)
 			(effects
@@
 			(project "impeller18"
 				(path "/4ccab03b-4b1c-4c61-9fa8-19853ef32b4d/bb535897-f2f1-40b8-a983-287c6650a9b5"
-					(reference "C109")
+					(reference "C112")
 					(unit 1)
 				)
@@
 		(on_board yes)
 		(dnp no)
-		(property "Reference" "C108"
+		(property "Reference" "C111"
 			(at 231.14 58.42 0)
 			(effects
@@
 			(project "impeller18"
 				(path "/4ccab03b-4b1c-4c61-9fa8-19853ef32b4d/bb535897-f2f1-40b8-a983-287c6650a9b5"
-					(reference "C108")
+					(reference "C111")
 					(unit 1)
 				)

Commit message: Update PCB concept
Connections:
- net ADC_30V_IN_1: now also J26.9 (Pin_9); no longer J26.1 (Pin_1)
- net ADC_30V_IN_2: now also J26.10 (Pin_10); no longer J26.5 (Pin_5)
- net ADC_30V_IN_3: now also J26.11 (Pin_11); no longer J26.3 (Pin_3)
- net ADC_30V_IN_4: now also J26.12 (Pin_12); no longer J26.7 (Pin_7)
- net ADC_30V_IN_5: now also J26.13 (Pin_13); no longer J26.9 (Pin_9)
- net ADC_30V_IN_6: now also J26.14 (Pin_14); no longer J26.11 (Pin_11)
- net ADC_30V_IN_7: now also J26.15 (Pin_15); no longer J26.13 (Pin_13)
- net ADC_30V_IN_8: now also J26.16 (Pin_16); no longer J26.15 (Pin_15)
- net GND_ADC: now also J26.1 (Pin_1), J26.3 (Pin_3), J26.5 (Pin_5), J26.7 (Pin_7); no longer J26.10 (Pin_10), J26.12 (Pin_12), J26.14 (Pin_14), J26.16 (Pin_16)
Other:
- moved on the sheet: J26

Commit message: Daily PCB update
Parts:
- renumbered R250 to R254, R251 to R255, R252 to R256, R253 to R257, R254 to R258, R255 to R259, R256 to R260, R257 to R261, R258 to R262, R259 to R263, R260 to R264, R261 to R265, R262 to R266, R263 to R267, R264 to R268, R265 to R269, R266 to R270, R267 to R271, R268 to R272, R269 to R273, R270 to R274, R271 to R275, R272 to R276, R273 to R277, R274 to R278, R275 to R279, R276 to R280, R277 to R281, R278 to R282, R279 to R283, R280 to R284, TP38 to TP39, TP39 to TP40

Commit message: Update PCB concept
Parts:
- removed R260, R262, R267: 10k, Resistor_SMD:R_0603_1608Metric, symbol Device:R_Small
- removed R275, R281, R283: 1M, Resistor_SMD:R_0603_1608Metric, symbol Device:R_Small
- removed R279, R282, R284: 200k, Resistor_SMD:R_0603_1608Metric, symbol Device:R_Small
- added R257, R258: 1k, Resistor_SMD:R_0603_1608Metric, symbol Device:R_Small
- added R265: 1M, Resistor_SMD:R_0603_1608Metric, symbol Device:R_Small
- added R271, R276, R277, R278: 200k, Resistor_SMD:R_0603_1608Metric, symbol Device:R_Small
- R255: value 1M -> 1k; Ссылка https://www.promelec.ru/product/22010/ -> https://www.promelec.ru/product/22771/; Человекопонятное название Толстопленочный ЧИП-резистор 0603 1МОм -> Толстопленочный ЧИП-резистор 0603 1кОм
- R256: value 200k -> 1k; Ссылка https://www.promelec.ru/product/57740/ -> https://www.promelec.ru/product/22771/; Человекопонятное название Толстопленочный ЧИП-резистор 0603 200кОм -> Толстопленочный ЧИП-резистор 0603 1кОм
- R264, R270: value 200k -> 1M; Ссылка https://www.promelec.ru/product/57740/ -> https://www.promelec.ru/product/22010/; Человекопонятное название Толстопленочный ЧИП-резистор 0603 200кОм -> Толстопленочный ЧИП-резистор 0603 1МОм
- R266, R269: value 10k -> 1M; Мин. кол-во 1000 -> 100; Ссылка https://www.promelec.ru/product/344748/ -> https://www.promelec.ru/product/22010/; Человекопонятное название Толстопленочный ЧИП-резистор 0603 10кОм -> Толстопленочный ЧИП-резистор 0603 1МОм
- R272: value 10k -> 200k; Мин. кол-во 1000 -> 100; Ссылка https://www.promelec.ru/product/344748/ -> https://www.promelec.ru/product/57740/; Человекопонятное название Толстопленочный ЧИП-резистор 0603 10кОм -> Толстопленочный ЧИП-резистор 0603 200кОм
- R273: value 1M -> 200k; Ссылка https://www.promelec.ru/product/22010/ -> https://www.promelec.ru/product/57740/; Человекопонятное название Толстопленочный ЧИП-резистор 0603 1МОм -> Толстопленочный ЧИП-резистор 0603 200кОм
- TP33: renamed from TP39; footprint TestPoint:TestPoint_THTPad_D1.5mm_Drill0.7mm -> TestPoint:TestPoint_THTPad_D2.0mm_Drill1.0mm
- TP34: renamed from TP40; footprint TestPoint:TestPoint_THTPad_D1.5mm_Drill0.7mm -> TestPoint:TestPoint_THTPad_D2.0mm_Drill1.0mm
- renumbered J26 to J29, R258 to R259, R261 to R260, R265 to R261, R271 to R262, R257 to R267, R259 to R275, R276 to R279, R277 to R280, R278 to R281, R280 to R282
Connections:
- net ADC_30V_1 is gone; now on net SPI_ADC8_CLK: R255.1
- net ADC_30V_5 is gone; now on net ADC_5V_3: R273.1
- net ADC_30V_IN_2 is gone; now on an unnamed net: J29.10 (Pin_10)
- net ADC_30V_IN_4 is gone; now on an unnamed net: J29.12 (Pin_12)
- net ADC_30V_IN_7 is gone; now on an unnamed net: J29.15 (Pin_15)
- net 3V3: now also U57.2 (A), U59.1 (A1), U59.4 (A2); no longer R260.2, R261.2, R262.2, R266.1, R272.1
- net 5V0_ADC: now also C113.2, R255.2, R256.2, U61.2 (A), R257.2, R258.2; no longer C113.1, R269.2, R282.1
- net ADC_5V_1: now also R266.2, R274.1, U60.3 (IO2); no longer R255.2, R256.2, U60.1 (IO1)
- net ADC_5V_2: now also R275.1, U60.1 (IO1); no longer R275.2, U60.3 (IO2)
- net ADC_5V_3: now also U60.6 (IO4), R265.2; no longer R263.2, R264.2, U60.4 (IO3)
- net ADC_5V_4: now also U60.4 (IO3), R276.1; no longer R270.2, U60.6 (IO4)
- net ADC_5V_5: now also R264.2, R272.1, U62.3 (IO2); no longer R273.2, R274.2, U62.1 (IO1)
- net ADC_5V_6: now also R269.2, U62.1 (IO1), R277.1; no longer U62.3 (IO2)
- net ADC_5V_7: now also R263.2, U62.6 (IO4), R271.1; no longer U62.4 (IO3)
- net ADC_5V_8: now also R270.2, U62.4 (IO3), R278.1; no longer U62.6 (IO4)
- net GND_ADC: now also C113.1, R272.2, R273.2, R274.2, R275.2, R271.2, R276.2, R277.2, R278.2; no longer C113.2, R256.1, R264.1, R270.1, R274.1, R275.1
- net SPI1_STM32_ADC8_CS: now also R262.1; no longer R272.2, U59.3 (C2)
- net SPI1_STM32_CLK: now also R260.2; no longer U57.3 (C)
- net SPI1_STM32_MOSI: now also R261.2; no longer R266.2, U59.2 (C1)
- net SPI_ADC8_CS: now also R258.1; no longer R269.1
- net SPI_ADC8_MISO: now also R256.1, R282.2; no longer U61.3 (C)
- net SPI_ADC8_MOSI: now also R257.1
- net at R260.1: now also U57.3 (C); no longer U57.2 (A)
- net at R261.1: now also U59.2 (C1); no longer U59.1 (A1)
- net ADC_30V_2: no longer names the net of R267.1
- net ADC_30V_3: no longer names the net of R263.1
- net ADC_30V_4: no longer names the net of R268.1
- net ADC_30V_IN_1: no longer names the net of J29.9 (Pin_9)
- net ADC_30V_IN_1: now also R266.1
- net ADC_30V_IN_3: no longer names the net of J29.11 (Pin_11)
- net ADC_30V_IN_3: now also R265.1
- net ADC_30V_IN_5: no longer names the net of J29.13 (Pin_13)
- net ADC_30V_IN_5: now also R264.1
- net ADC_30V_IN_6: no longer names the net of J29.14 (Pin_14)
- net ADC_30V_IN_6: now also R269.1
- net ADC_30V_IN_8: no longer names the net of J29.16 (Pin_16)
- net ADC_30V_IN_8: now also R270.1
- new net: R282.1, U61.3 (C)
- new net: R262.2, U59.3 (C2)
Other:
- note added: "перeкинуть резистор????"
- moved on the sheet: C112, C113, J29, Q58, R259, R260, R261, R262, R267, R275, R279, R280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

Commit message: Zone borders
Parts:
- D18: footprint LED_SMD:LED_0603_1608Metric -> user_lib:LED_0603_1608Metric
Changed lines of the file:
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@@
 			)
 		)
-		(property "Footprint" "LED_SMD:LED_0603_1608Metric"
+		(property "Footprint" "user_lib:LED_0603_1608Metric"
 			(at 252.095 63.5 0)
 			(effects
