File: Hardware/ciam/impeller18/switches_1.kicad_sch (KiCad schematic)
At the start: 108 parts, among them J3 430451800, J4 430451800, Q1 BSS138, Q10 BSS138, Q11 BSS138, Q12 BSS138, Q13 BSS138, Q14 BSS138, Q15 BSS138, Q16 BSS138, Q17 BSS138, Q18 BSS138, Q2 BSS138, Q3 BSS138, Q4 BSS138, Q5 BSS138, Q6 BSS138, Q7 BSS138, Q8 BSS138, Q9 BSS138, U12 TLP291-4, U13 TLP291-4, U14 TLP291-4, U15 TLP291-4, U16 TLP291, U17 TLP291, U18 B0505MT-1WR4, U19 B0505MT-1WR4

Commit message: updated schematics
Parts:
- renumbered C42 to C71, C43 to C72, C44 to C73, C45 to C74, C46 to C75, C47 to C76, C48 to C77, C49 to C78, J3 to J5, J4 to J6, R16 to R23, R17 to R24, R18 to R25, R19 to R26, R20 to R27, R21 to R28, R22 to R29, R23 to R30, R24 to R31, R25 to R32, R26 to R33, R27 to R34, R28 to R35, R29 to R36, R30 to R37, R31 to R38, R32 to R39, R33 to R40, R34 to R41, R35 to R42, R36 to R43, R37 to R44, R38 to R45, R39 to R46, R40 to R47, R41 to R48, R42 to R49, R43 to R50, R44 to R51, R45 to R52, R46 to R53, R47 to R54, R48 to R55, R49 to R56, R50 to R57, R51 to R58, R52 to R59, R53 to R60, R54 to R61, R55 to R62, R56 to R63, R57 to R64, R58 to R65, R59 to R66, R60 to R67, R61 to R68, R62 to R69, R63 to R70, R64 to R71, R65 to R72, R66 to R73, R67 to R74, R68 to R75, R69 to R76, R70 to R77, R71 to R78, R72 to R79, R73 to R80, R74 to R81, R75 to R82, R76 to R83, R77 to R84, R78 to R85, R79 to R86, R80 to R87, R81 to R88, R82 to R89, R83 to R90, R84 to R91, R85 to R92, R86 to R93, R87 to R94, U12 to U13, U13 to U14, U14 to U15, U15 to U16, U16 to U17, U17 to U18, U18 to U19, U19 to U20
Connections:
- net SWITCH_1.1_EXT: now also J5.1 (Pin_1)
- net SWITCH_1.2_EXT: now also J5.3 (Pin_3)
- net SWITCH_1.3_EXT: now also J5.5 (Pin_5)
- net SWITCH_1.4_EXT: now also J5.7 (Pin_7)
- net SWITCH_1.5_EXT: now also J5.9 (Pin_9)
- net SWITCH_1.6_EXT: now also J5.11 (Pin_11)
- net SWITCH_1.7_EXT: now also J5.13 (Pin_13)
- net SWITCH_1.8_EXT: now also J5.15 (Pin_15)
- net SWITCH_1.9_EXT: now also J5.17 (Pin_17)
- net SWITCH_2.1_EXT: no longer J5.1 (Pin_1)
- net SWITCH_2.2_EXT: no longer J5.3 (Pin_3)
- net SWITCH_2.3_EXT: no longer J5.5 (Pin_5)
- net SWITCH_2.4_EXT: no longer J5.7 (Pin_7)
- net SWITCH_2.5_EXT: no longer J5.9 (Pin_9)
- net SWITCH_2.6_EXT: no longer J5.11 (Pin_11)
- net SWITCH_2.7_EXT: no longer J5.13 (Pin_13)
- net SWITCH_2.8_EXT: no longer J5.15 (Pin_15)
- net SWITCH_2.9_EXT: no longer J5.17 (Pin_17)

Commit message: updated schematics
Parts:
- removed C71: 100n, symbol Device:C_Small
- removed C72, C73: 10u, symbol Device:C_Small
- removed U19: B0505MT-1WR4, symbol Interface_CAN_LIN:ISO1050DUB
- added C75, C76: 10u, symbol Device:C_Small
- added C77: 100n, symbol Device:C_Small
- added D8, D9: FYLS-0603BUGC, symbol Device:LED
- added R89, R90: 150, symbol Device:R_Small
- added U20: B0505MT-1WR4, symbol Interface_CAN_LIN:ISO1050DUB
- renumbered C75 to C70, C76 to C71, C77 to C72, C78 to C73, J5 to J6, J6 to J7, R23 to R17, R24 to R18, R25 to R19, R26 to R20, R27 to R21, R28 to R22, R29 to R23, R30 to R24, R31 to R25, R32 to R26, R33 to R27, R34 to R28, R35 to R29, R36 to R30, R37 to R31, R38 to R32, R39 to R33, R40 to R34, R41 to R35, R42 to R36, R43 to R37, R44 to R38, R45 to R39, R46 to R40, R47 to R41, R48 to R42, R49 to R43, R50 to R44, R51 to R45, R52 to R46, R53 to R47, R54 to R48, R55 to R49, R56 to R50, R57 to R51, R58 to R52, R59 to R53, R60 to R54, R61 to R55, R62 to R56, R63 to R57, R64 to R58, R65 to R59, R66 to R60, R67 to R61, R68 to R62, R69 to R63, R70 to R64, R71 to R65, R72 to R66, R73 to R67, R74 to R68, R75 to R69, R76 to R70, R77 to R71, R78 to R72, R79 to R73, R80 to R74, R81 to R75, R82 to R76, R83 to R77, R84 to R78, R85 to R79, R86 to R80, R87 to R81, R88 to R82, R89 to R83, R90 to R84, R91 to R85, R92 to R86, R93 to R87, R94 to R88, U20 to U19
Connections:
- net 5V0: now also C76.1, C77.1, U20.13 (Vin), U20.14 (Vin); no longer C74.1
- net 5V0_SWITCHES_1: now also R89.1
- net 5V0_SWITCHES_2: now also C74.1, C75.1, R90.1, U20.8 (+Vo)
- net GND: now also C76.2, C77.2, U20.1 (gnd), U20.2 (gnd); no longer C74.2
- net GND_IN: now also C74.2, C75.2, D8.1 (K), D9.1 (K), U20.6 (0V), U20.7 (0V)
- new net: D9.2 (A), R90.2
- new net: D8.2 (A), R89.2
Other:
- moved on the sheet: C70, C71, C72, C73, U19

Commit message: Added Li-Io balanserer
Parts:
- added J20: 430451800, symbol Connector_Generic:Conn_02x09_Odd_Even
Connections:
- net SWITCH_1.1_EXT: now also J20.1 (Pin_1)
- net SWITCH_1.2_EXT: now also J20.3 (Pin_3)
- net SWITCH_1.3_EXT: now also J20.5 (Pin_5)
- net SWITCH_1.4_EXT: now also J20.7 (Pin_7)
- net SWITCH_1.5_EXT: now also J20.9 (Pin_9)
- net SWITCH_1.6_EXT: now also J20.11 (Pin_11)
- net SWITCH_1.7_EXT: now also J20.13 (Pin_13)
- net SWITCH_1.8_EXT: now also J20.15 (Pin_15)
- net SWITCH_1.9_EXT: now also J20.17 (Pin_17)
- net SWITCH_2.1_EXT: now also J20.2 (Pin_2)
- net SWITCH_2.2_EXT: now also J20.4 (Pin_4)
- net SWITCH_2.3_EXT: now also J20.6 (Pin_6)
- net SWITCH_2.4_EXT: now also J20.8 (Pin_8)
- net SWITCH_2.5_EXT: now also J20.10 (Pin_10)
- net SWITCH_2.6_EXT: now also J20.12 (Pin_12)
- net SWITCH_2.7_EXT: now also J20.14 (Pin_14)
- net SWITCH_2.8_EXT: now also J20.16 (Pin_16)
- net SWITCH_2.9_EXT: now also J20.18 (Pin_18)

Commit message: updated schematics
Parts:
- removed R89, R90: 150, symbol Device:R_Small
- added R113, R114: 360, symbol Device:R_Small
- C76: renamed from C70; Ссылка https://www.chipdip.ru/product/grm21br71h104k -> (none); Цена 13 -> (none); Человекопонятное название Конденсатор 100нФ -> (none)
- C77: renamed from C71; Ссылка https://www.chipdip.ru/product/grm21br61e106ka73l -> (none); Цена 13 -> (none); Человекопонятное название Конденсатор 10мкФ -> (none)
- C78: renamed from C72; Ссылка https://www.chipdip.ru/product/grm21br61e106ka73l -> (none); Цена 13 -> (none); Человекопонятное название Конденсатор 10мкФ -> (none)
- C79: renamed from C73; Ссылка https://www.chipdip.ru/product/grm21br71h104k -> (none); Цена 13 -> (none); Человекопонятное название Конденсатор 100нФ -> (none)
- C80: renamed from C74; Ссылка https://www.chipdip.ru/product/grm21br71h104k -> (none); Цена 13 -> (none); Человекопонятное название Конденсатор 100нФ -> (none)
- C81: renamed from C75; Ссылка https://www.chipdip.ru/product/grm21br61e106ka73l -> (none); Цена 13 -> (none); Человекопонятное название Конденсатор 10мкФ -> (none)
- C82: renamed from C76; Ссылка https://www.chipdip.ru/product/grm21br61e106ka73l -> (none); Цена 13 -> (none); Человекопонятное название Конденсатор 10мкФ -> (none)
- C83: renamed from C77; Ссылка https://www.chipdip.ru/product/grm21br71h104k -> (none); Цена 13 -> (none); Человекопонятное название Конденсатор 100нФ -> (none)
- J6: footprint (none) -> Connector_Molex:Molex_Micro-Fit_3.0_43045-1800_2x09_P3.00mm_Horizontal
- J7: renamed from J20; footprint (none) -> Connector_Molex:Molex_Micro-Fit_3.0_43045-1800_2x09_P3.00mm_Horizontal
- J8: renamed from J7; footprint (none) -> Connector_Molex:Molex_Micro-Fit_3.0_43045-1800_2x09_P3.00mm_Horizontal
- U23: renamed from U17; Ссылка https://www.chipdip.ru/product/tlp291-gb-tp-se-t -> (none); Цена 62 -> (none); Человекопонятное название Оптопара с транзисторным выходом -> (none)
- U24: renamed from U18; Ссылка https://www.chipdip.ru/product/tlp291-gb-tp-se-t -> (none); Цена 62 -> (none); Человекопонятное название Оптопара с транзисторным выходом -> (none)
- U25: renamed from U19; Ссылка https://www.chipdip.ru/product0/8003333290 -> (none); Цена 120 -> (none); Человекопонятное название DC/DC преобразователь -> (none)
- U26: renamed from U20; Ссылка https://www.chipdip.ru/product0/8003333290 -> (none); Цена 120 -> (none); Человекопонятное название DC/DC преобразователь -> (none)
- renumbered D8 to D14, D9 to D15, Q6 to Q10, Q7 to Q11, Q8 to Q12, Q9 to Q13, Q10 to Q14, Q11 to Q15, Q12 to Q16, Q13 to Q17, Q14 to Q18, Q15 to Q19, Q16 to Q20, Q17 to Q21, Q18 to Q22, Q1 to Q5, Q2 to Q6, Q3 to Q7, Q4 to Q8, Q5 to Q9, R76 to R100, R77 to R101, R78 to R102, R79 to R103, R80 to R104, R81 to R105, R82 to R106, R83 to R107, R84 to R108, R85 to R109, R86 to R110, R87 to R111, R88 to R112, R17 to R41, R18 to R42, R19 to R43, R20 to R44, R21 to R45, R22 to R46, R23 to R47, R24 to R48, R25 to R49, R26 to R50, R27 to R51, R28 to R52, R29 to R53, R30 to R54, R31 to R55, R32 to R56, R33 to R57, R34 to R58, R35 to R59, R36 to R60, R37 to R61, R38 to R62, R39 to R63, R40 to R64, R41 to R65, R42 to R66, R43 to R67, R44 to R68, R45 to R69, R46 to R70, R47 to R71, R48 to R72, R49 to R73, R50 to R74, R51 to R75, R52 to R76, R53 to R77, R54 to R78, R55 to R79, R56 to R80, R57 to R81, R58 to R82, R59 to R83, R60 to R84, R61 to R85, R62 to R86, R63 to R87, R64 to R88, R65 to R89, R66 to R90, R67 to R91, R68 to R92, R69 to R93, R70 to R94, R71 to R95, R72 to R96, R73 to R97, R74 to R98, R75 to R99, U13 to U19, U14 to U20, U15 to U21, U16 to U22
Connections:
- net 5V0_SWITCHES_1: now also R113.2
- net 5V0_SWITCHES_2: now also R114.2
- net at D15.2 (A): now also R114.1
- net at D14.2 (A): now also R113.1

Commit message: updated schematics
Parts:
- C76, C79, C80, C83: Мин. кол-во (none) -> 300; Ссылка (none) -> https://www.promelec.ru/product/323633/; Цена (none) -> 2; Человекопонятное название (none) -> Керамический ЧИП-конденсатор 0603 X7R 0.1мкФ
- C77, C78, C81, C82: Мин. кол-во (none) -> 200; Ссылка (none) -> https://www.promelec.ru/product/430347/; Цена (none) -> 4; Человекопонятное название (none) -> Керамический ЧИП-конденсатор 0603 X5R 10мкФ
- D14, D15: footprint (none) -> LED_SMD:LED_0603_1608Metric; Мин. кол-во (none) -> 3; Ссылка (none) -> https://www.promelec.ru/product/324327/; Цена (none) -> 5; Человекопонятное название (none) -> Светодиод smd 1,6х0,8мм/зеленый/568нм/65мкд/прозрачный/130°
- J10: renamed from J8; footprint Connector_Molex:Molex_Micro-Fit_3.0_43045-1800_2x09_P3.00mm_Horizontal -> (none); Мин. кол-во (none) -> 3; Ссылка (none) -> https://www.promelec.ru/product/474708/; Цена (none) -> 175; Человекопонятное название (none) -> Соединитель провод-плата HDR 18 контакт(ов) 3мм угловой сер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
- J8: renamed from J6; footprint Connector_Molex:Molex_Micro-Fit_3.0_43045-1800_2x09_P3.00mm_Horizontal -> (none); Мин. кол-во (none) -> 3; Ссылка (none) -> https://www.promelec.ru/product/474708/; Цена (none) -> 175; Человекопонятное название (none) -> Соединитель провод-плата HDR 18 контакт(ов) 3мм угловой сер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
- J9: renamed from J7; footprint Connector_Molex:Molex_Micro-Fit_3.0_43045-1800_2x09_P3.00mm_Horizontal -> (none); Мин. кол-во (none) -> 3; Ссылка (none) -> https://www.promelec.ru/product/474708/; Цена (none) -> 175; Человекопонятное название (none) -> Соединитель провод-плата HDR 18 контакт(ов) 3мм угловой сер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
- Q10, Q11, Q12, Q13, Q14, Q15, Q16, Q17, Q18, Q19, Q20, Q21, Q22, Q5, Q6, Q7, Q8, Q9: Мин. кол-во (none) -> 38; Ссылка (none) -> https://www.promelec.ru/product/303635/; Цена (none) -> 14; Человекопонятное название (none) -> Транзистор полевой N-канальный
- R100, R107, R108, R43, R44, R51, R52, R59, R60, R67, R68, R75, R76, R83, R84, R91, R92, R99: Мин. кол-во (none) -> 100; Ссылка (none) -> https://www.promelec.ru/product/23650/; Цена (none) -> 1; Человекопонятное название (none) -> Толстопленочный ЧИП-резистор 0603 360кОм
- R101, R103, R109, R111, R113, R114, R45, R47, R53, R55, R61, R63, R69, R71, R77, R79, R85, R87, R93, R95: Мин. кол-во (none) -> 100; Ссылка (none) -> https://www.promelec.ru/product/46471/; Цена (none) -> 1; Человекопонятное название (none) -> Толстопленочный ЧИП-резистор 0603 360Ом
- R102, R104, R110, R112, R46, R48, R54, R56, R62, R64, R70, R72, R78, R80, R86, R88, R94, R96: Мин. кол-во (none) -> 1000; Ссылка (none) -> https://www.promelec.ru/product/344748/; Цена (none) -> 1; Человекопонятное название (none) -> Толстопленочный ЧИП-резистор 0603 10кОм
- R105, R106, R41, R42, R49, R50, R57, R58, R65, R66, R73, R74, R81, R82, R89, R90, R97, R98: Мин. кол-во (none) -> 100; Ссылка (none) -> https://www.promelec.ru/product/22010/; Цена (none) -> 1; Человекопонятное название (none) -> Толстопленочный ЧИП-резистор 0603 1МОм
- U19, U20, U21, U22: Мин. кол-во (none) -> 1; Ссылка (none) -> https://www.chipdip.ru/product/tlp291-4-gb-tp-e-t; Цена (none) -> 340; Человекопонятное название (none) -> Оптопара с транзисторным выходом 4-х канальная
- U23, U24: Мин. кол-во (none) -> 1; Ссылка (none) -> https://www.chipdip.ru/product/tlp291-gb-tp-se-t; Цена (none) -> 62; Человекопонятное название (none) -> Оптопара с транзисторным выходом
- U25, U26: Мин. кол-во (none) -> 1; Ссылка (none) -> https://www.chipdip.ru/product/b0505mt-1wr4; Цена (none) -> 230; Человекопонятное название (none) -> DC/DC преобразователь, 1Вт, вход 4.5-5.5В, выход 5В/200мА

Commit message: updatec schematics
Parts:
- added TP17, TP18, TP23, TP24: TestPoint, symbol Connector:TestPoint
Connections:
- net 5V0_SWITCHES_1: now also TP17.1
- net 5V0_SWITCHES_2: now also TP23.1
- net GND_IN: now also TP18.1, TP24.1

Commit message: added footprints
Parts:
- C76, C77, C78, C79, C80, C81, C82, C83: footprint (none) -> Capacitor_SMD:C_0603_1608Metric
- J10, J8, J9: footprint (none) -> Connector_Molex:Molex_Micro-Fit_3.0_43045-1800_2x09_P3.00mm_Horizontal
- Q10, Q11, Q12, Q13, Q14, Q15, Q16, Q17, Q18, Q19, Q20, Q21, Q22, Q5, Q6, Q7, Q8, Q9: footprint (none) -> Package_TO_SOT_SMD:SOT-23
- R100, R101, R102, R103, R104, R105, R106, R107, R108, R109, R110, R111, R112, R113, R114, R41, R42, R43, R44, R45, R46, R47, R48, R49, R50, R51, R52, R53, R54, R55, R56, R57, R58, R59, R60, R61, R62, R63, R64, R65, R66, R67, R68, R69, R70, R71, R72, R73, R74, R75, R76, R77, R78, R79, R80, R81, R82, R83, R84, R85, R86, R87, R88, R89, R90, R91, R92, R93, R94, R95, R96, R97, R98, R99: footprint (none) -> Resistor_SMD:R_0603_1608Metric
- TP17, TP18, TP23, TP24: footprint (none) -> TestPoint:TestPoint_THTPad_D1.5mm_Drill0.7mm
- U19, U20, U21, U22: footprint (none) -> Package_SO:SOIC-16_4.55x10.3mm_P1.27mm
- U23, U24: footprint (none) -> Package_SO:SOIC-4_4.55x2.6mm_P1.27mm
- U25, U26: footprint (none) -> user_lib:B0505MT-1WR4

Commit message: Minor changes
Other:
- moved on the sheet: C76, C77, C78, C79, D14, J8, J9, R113, TP17, TP18, TP23, TP24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
