File: Hardware/ciam/impeller18/rpi.kicad_sch (KiCad schematic)
At the start: 12 parts, among them J7 Raspberry Pi 4

Commit message: added footprints
Parts:
- C73, C74, C75: footprint (none) -> Capacitor_SMD:C_0603_1608Metric
- D12, D13: footprint (none) -> user_lib:LED_RGB_promelec
- R35, R36, R37, R38, R39, R40: footprint (none) -> Resistor_SMD:R_0603_1608Metric
Changed lines of the file:
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@@
 			)
 		)
-		(property "Footprint" ""
+		(property "Footprint" "user_lib:LED_RGB_promelec"
 			(at 273.685 127.635 0)
 			(effects
@@
 			)
 		)
-		(property "Footprint" ""
+		(property "Footprint" "Resistor_SMD:R_0603_1608Metric"
 			(at 285.115 128.143 90)
 			(effects
@@
 			)
 		)
-		(property "Footprint" ""
+		(property "Footprint" "Capacitor_SMD:C_0603_1608Metric"
 			(at 177.8 70.485 0)
 			(effects
@@
 			)
 		)
-		(property "Footprint" ""
+		(property "Footprint" "Capacitor_SMD:C_0603_1608Metric"
 			(at 177.8 64.77 0)
 			(effects
@@
 			)
 		)
-		(property "Footprint" ""
+		(property "Footprint" "user_lib:LED_RGB_promelec"
 			(at 273.685 100.33 0)
 			(effects
@@
 			)
 		)
-		(property "Footprint" ""
+		(property "Footprint" "Resistor_SMD:R_0603_1608Metric"
 			(at 285.115 133.223 90)
 			(effects
@@
 			)
 		)
-		(property "Footprint" ""
+		(property "Footprint" "Resistor_SMD:R_0603_1608Metric"
 			(at 285.115 100.838 90)
 			(effects
@@
 			)
 		)
-		(property "Footprint" ""
+		(property "Footprint" "Resistor_SMD:R_0603_1608Metric"
 			(at 285.115 105.918 90)
 			(effects
@@
 			)
 		)
-		(property "Footprint" ""
+		(property "Footprint" "Capacitor_SMD:C_0603_1608Metric"
 			(at 177.8 76.2 0)
 			(effects
@@
 			)
 		)
-		(property "Footprint" ""
+		(property "Footprint" "Resistor_SMD:R_0603_1608Metric"
 			(at 285.115 95.758 90)
 			(effects
@@
 			)
 		)
-		(property "Footprint" ""
+		(property "Footprint" "Resistor_SMD:R_0603_1608Metric"
 			(at 285.115 123.063 90)
 			(effects

Commit message: Minor changes
Parts:
- added J27: PLS-6, Connector_PinHeader_2.54mm:PinHeader_1x06_P2.54mm_Vertical, symbol Connector_Generic:Conn_01x06
Connections:
- net GND: now also J27.6 (Pin_6)
- net SPI1_RPi_CAN0_CS: now also J27.4 (Pin_4)
- net SPI1_RPi_CAN1_CS: now also J27.5 (Pin_5)
- net SPI1_RPi_MISO: now also J27.3 (Pin_3)
- net SPI1_RPi_SCK: now also J27.1 (Pin_1)
- net SPI0_RPi_MOSI renamed SPI1_RPi_MOSI
- net SPI1_RPi_MOSI: now also J27.2 (Pin_2)
Other:
- note added: "ПРОВЕРИТЬ СВЕТОДИОДЫ"
- note added: "когда подключим светодиоды?"

Commit message: bugfixes
Parts:
- added F2: MF-LSMF300/24X-2, Fuse:Fuse_2920_7451Metric, symbol Device:Polyfuse_Small
Connections:
- net 5V0: now also F2.2; no longer C73.2, C74.2, C75.2, J7.2 (5V), J7.4 (5V)
- new net: C73.2, C74.2, C75.2, F2.1, J7.2 (5V), J7.4 (5V)
Changed lines of the file:
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@@
+	(wire
+		(pts
+			(xy 185.42 55.245) (xy 185.42 56.515)
+		)
+		(stroke
+			(width 0)
+			(type default)
+		)
+	)
 	(wire
 		(pts
@@
 	(symbol
 		(lib_id "power:+5V")
-		(at 185.42 61.595 0)
+		(at 185.42 55.245 0)
 		(unit 1)
 		(exclude_from_sim no)
@@
 		(dnp no)
 		(property "Reference" "#PWR0103"
-			(at 185.42 65.405 0)
+			(at 185.42 59.055 0)
 			(effects
 				(font
@@
 		)
 		(property "Value" "5V0"
-			(at 185.42 57.785 0)
+			(at 185.42 51.435 0)
 			(effects
 				(font
@@
 		)
 		(property "Footprint" ""
-			(at 185.42 61.595 0)
+			(at 185.42 55.245 0)
 			(effects
 				(font
@@
 		)
 		(property "Datasheet" ""
-			(at 185.42 61.595 0)
+			(at 185.42 55.245 0)
 			(effects
 				(font
@@
 		)
 		(property "Description" "Power symbol creates a global label with name \"+5V\""
-			(at 185.42 61.595 0)
+			(at 185.42 55.245 0)
 			(effects
 				(font
@@
 					(unit 1)
 				)
+			)
+		)
+	)
+	(symbol
+		(lib_id "Device:Polyfuse_Small")
+		(at 185.42 59.055 180)
+		(unit 1)
+		(exclude_from_sim no)
+		(in_bom yes)
+		(on_board yes)
+		(dnp no)
+		(property "Reference" "F2"
+			(at 188.595 57.785 0)
+			(effects
+				(font
+					(size 1.27 1.27)
+				)
+			)
+		)
+		(property "Value" "MF-LSMF300/24X-2"
+			(at 197.485 60.96 0)
+			(effects
+				(font
+					(size 1.27 1.27)
+				)
+			)
+		)
+		(property "Footprint" "Fuse:Fuse_2920_7451Metric"
+			(at 184.15 53.975 0)
+			(effects
+				(font
+					(size 1.27 1.27)
+				)
+				(justify left)
+				(hide yes)
+			)
+		)
+		(property "Datasheet" "~"
+			(at 185.42 59.055 0)
+			(effects
+				(font
+					(size 1.27 1.27)
+				)
+				(hide yes)
+			)
+		)
+		(property "Description" "Resettable fuse, polymeric positive temperature coefficient, small symbol"
+			(at 185.42 59.055 0)
+			(effects
+				(font
+					(size 1.27 1.27)
+				)
+				(hide yes)
+			)
+		)
+		(property "Мин. кол-во" "1"
+			(at 185.42 59.055 0)
+			(effects
+				(font
+					(size 1.27 1.27)
+				)
+				(hide yes)
+			)
+		)
+		(property "Ссылка" "https://www.promelec.ru/product/465739/"
+			(at 185.42 59.055 0)
+			(effects
+				(font
+					(size 1.27 1.27)
+				)
+				(hide yes)
+			)
+		)
+		(property "Цена" "28"
+			(at 185.42 59.055 0)
+			(effects
+				(font
+					(size 1.27 1.27)
+				)
+				(hide yes)
+			)
+		)
+		(property "Человекопонятное название" "Самовосстанавливающийся предохранитель"
+			(at 185.42 59.055 0)
+			(effects
+				(font
+					(size 1.27 1.27)
+				)
+				(hide yes)
+			)
+		)
+		(pin "1"
+		)
+		(pin "2"
+		)
+		(instances
+			(project "impeller18"
+				(path "/4ccab03b-4b1c-4c61-9fa8-19853ef32b4d/36ec6b10-e9ff-4e61-94d3-a2b8a8777c75"
+					(reference "F2")
+					(unit 1)
+				)
