File: Hardware/ciam/impeller18/fan.kicad_sch (KiCad schematic)
At the start: 21 parts, among them J23 430450415, U75 HCPL-0600, U76 LDL1117S50R, U77 SMU02M-12

Commit message: added footprints
Parts:
- C111, C112, C113, C114, C115, C116: footprint (none) -> Capacitor_SMD:C_0603_1608Metric
- J23: footprint (none) -> Connector_Molex:Molex_Micro-Fit_3.0_43045-0415_2x02_P3.00mm_Vertical
- R279, R280, R281, R282, R283: footprint (none) -> Resistor_SMD:R_0603_1608Metric
- TP33, TP34, TP35, TP36: footprint (none) -> TestPoint:TestPoint_THTPad_D1.5mm_Drill0.7mm
- U75: footprint (none) -> Package_SO:SO-8_3.9x4.9mm_P1.27mm
- U76: footprint (none) -> Package_TO_SOT_SMD:SOT-223-3_TabPin2
Changed lines of the file:
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@@
 			)
 		)
-		(property "Footprint" ""
+		(property "Footprint" "TestPoint:TestPoint_THTPad_D1.5mm_Drill0.7mm"
 			(at 60.325 107.315 0)
 			(effects
@@
 			)
 		)
-		(property "Footprint" ""
+		(property "Footprint" "Capacitor_SMD:C_0603_1608Metric"
 			(at 134.9502 94.615 0)
 			(effects
@@
 			)
 		)
-		(property "Footprint" ""
+		(property "Footprint" "Resistor_SMD:R_0603_1608Metric"
 			(at 96.52 52.07 0)
 			(effects
@@
 			)
 		)
-		(property "Footprint" ""
+		(property "Footprint" "TestPoint:TestPoint_THTPad_D1.5mm_Drill0.7mm"
 			(at 60.325 102.87 0)
 			(effects
@@
 			)
 		)
-		(property "Footprint" ""
+		(property "Footprint" "Capacitor_SMD:C_0603_1608Metric"
 			(at 77.47 90.17 0)
 			(effects
@@
 			)
 		)
-		(property "Footprint" ""
+		(property "Footprint" "TestPoint:TestPoint_THTPad_D1.5mm_Drill0.7mm"
 			(at 123.19 100.965 0)
 			(effects
@@
 			)
 		)
-		(property "Footprint" ""
+		(property "Footprint" "Resistor_SMD:R_0603_1608Metric"
 			(at 133.35 45.72 0)
 			(effects
@@
 			)
 		)
-		(property "Footprint" ""
+		(property "Footprint" "TestPoint:TestPoint_THTPad_D1.5mm_Drill0.7mm"
 			(at 123.19 105.41 0)
 			(effects
@@
 			)
 		)
-		(property "Footprint" ""
+		(property "Footprint" "Resistor_SMD:R_0603_1608Metric"
 			(at 175.895 83.82 0)
 			(effects
@@
 			)
 		)
-		(property "Footprint" ""
+		(property "Footprint" "Capacitor_SMD:C_0603_1608Metric"
 			(at 52.07 90.17 0)
 			(effects
@@
 			)
 		)
-		(property "Footprint" ""
+		(property "Footprint" "Capacitor_SMD:C_0603_1608Metric"
 			(at 108.2802 94.615 0)
 			(effects
@@
 			)
 		)
-		(property "Footprint" ""
+		(property "Footprint" "Package_SO:SO-8_3.9x4.9mm_P1.27mm"
 			(at 108.585 64.77 0)
 			(effects
@@
 			)
 		)
-		(property "Footprint" ""
+		(property "Footprint" "Package_TO_SOT_SMD:SOT-223-3_TabPin2"
 			(at 123.19 80.645 0)
 			(effects
@@
 			)
 		)
-		(property "Footprint" ""
+		(property "Footprint" "Resistor_SMD:R_0603_1608Metric"
 			(at 125.095 45.72 0)
 			(effects
@@
 			)
 		)
-		(property "Footprint" ""
+		(property "Footprint" "Capacitor_SMD:C_0603_1608Metric"
 			(at 146.3802 94.615 0)
 			(effects
@@
 			)
 		)
-		(property "Footprint" ""
+		(property "Footprint" "Connector_Molex:Molex_Micro-Fit_3.0_43045-0415_2x02_P3.00mm_Vertical"
 			(at 148.59 52.07 0)
 			(effects
@@
 			)
 		)
-		(property "Footprint" ""
+		(property "Footprint" "Resistor_SMD:R_0603_1608Metric"
 			(at 199.39 83.82 0)
 			(effects
@@
 			)
 		)
-		(property "Footprint" ""
+		(property "Footprint" "Capacitor_SMD:C_0603_1608Metric"
 			(at 96.8502 94.615 0)
 			(effects

Commit message: Minor changes
Other:
- moved on the sheet: TP33, TP34, TP35, TP36
Changed lines of the file:
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@@
 	(wire
 		(pts
-			(xy 60.325 107.95) (xy 64.77 107.95)
+			(xy 226.695 81.28) (xy 226.695 76.835)
 		)
 		(stroke
@@
 	(wire
 		(pts
-			(xy 123.19 110.49) (xy 127.635 110.49)
+			(xy 226.695 95.885) (xy 226.695 100.33)
 		)
 		(stroke
@@
 	(wire
 		(pts
-			(xy 60.325 112.395) (xy 64.77 112.395)
+			(xy 243.205 95.885) (xy 243.205 100.33)
 		)
 		(stroke
@@
 	(wire
 		(pts
-			(xy 123.19 106.045) (xy 127.635 106.045)
+			(xy 243.205 81.28) (xy 243.205 76.835)
 		)
 		(stroke
@@
 	(symbol
 		(lib_id "Connector:TestPoint")
-		(at 60.325 112.395 90)
+		(at 243.205 95.885 0)
 		(unit 1)
 		(exclude_from_sim no)
@@
 		(dnp no)
 		(property "Reference" "TP34"
-			(at 52.705 113.03 90)
+			(at 244.475 92.075 0)
 			(effects
 				(font
@@
 		)
 		(property "Value" "TestPoint"
-			(at 55.245 111.125 90)
+			(at 244.475 93.98 0)
 			(effects
 				(font
@@
 		)
 		(property "Footprint" "TestPoint:TestPoint_THTPad_D1.5mm_Drill0.7mm"
-			(at 60.325 107.315 0)
+			(at 248.285 95.885 0)
 			(effects
 				(font
@@
 		)
 		(property "Datasheet" "~"
-			(at 60.325 107.315 0)
+			(at 248.285 95.885 0)
 			(effects
 				(font
@@
 		)
 		(property "Description" "test point"
-			(at 60.325 112.395 0)
+			(at 243.205 95.885 0)
 			(effects
 				(font
@@
 	(symbol
 		(lib_id "power:+12V")
-		(at 64.77 107.95 270)
+		(at 226.695 76.835 0)
 		(unit 1)
 		(exclude_from_sim no)
@@
 		(dnp no)
 		(property "Reference" "#PWR0287"
-			(at 60.96 107.95 0)
+			(at 226.695 80.645 0)
 			(effects
 				(font
@@
 		)
 		(property "Value" "12V0_FAN"
-			(at 73.025 107.95 90)
+			(at 226.695 73.025 0)
 			(effects
 				(font
@@
 		)
 		(property "Footprint" ""
-			(at 64.77 107.95 0)
+			(at 226.695 76.835 0)
 			(effects
 				(font
@@
 		)
 		(property "Datasheet" ""
-			(at 64.77 107.95 0)
+			(at 226.695 76.835 0)
 			(effects
 				(font
@@
 		)
 		(property "Description" "Power symbol creates a global label with name \"+12V\""
-			(at 64.77 107.95 0)
+			(at 226.695 76.835 0)
 			(effects
 				(font
@@
 	(symbol
 		(lib_id "Connector:TestPoint")
-		(at 60.325 107.95 90)
+		(at 226.695 81.28 180)
 		(unit 1)
 		(exclude_from_sim no)
@@
 		(dnp no)
 		(property "Reference" "TP33"
-			(at 52.705 108.585 90)
+			(at 233.045 83.82 0)
 			(effects
 				(font
@@
 		)
 		(property "Value" "TestPoint"
-			(at 55.245 106.68 90)
+			(at 236.855 85.725 0)
 			(effects
 				(font
@@
 		)
 		(property "Footprint" "TestPoint:TestPoint_THTPad_D1.5mm_Drill0.7mm"
-			(at 60.325 102.87 0)
+			(at 221.615 81.28 0)
 			(effects
 				(font
@@
 		)
 		(property "Datasheet" "~"
-			(at 60.325 102.87 0)
+			(at 221.615 81.28 0)
 			(effects
 				(font
@@
 		)
 		(property "Description" "test point"
-			(at 60.325 107.95 0)
+			(at 226.695 81.28 0)
 			(effects
 				(font
@@
 	(symbol
 		(lib_id "Connector:TestPoint")
-		(at 123.19 106.045 90)
+		(at 243.205 81.28 180)
 		(unit 1)
 		(exclude_from_sim no)
@@
 		(dnp no)
 		(property "Reference" "TP35"
-			(at 115.57 106.68 90)
+			(at 249.555 83.82 0)
 			(effects
 				(font
@@
 		)
 		(property "Value" "TestPoint"
-			(at 118.11 104.775 90)
+			(at 253.365 85.725 0)
 			(effects
 				(font
@@
 		)
 		(property "Footprint" "TestPoint:TestPoint_THTPad_D1.5mm_Drill0.7mm"
-			(at 123.19 100.965 0)
+			(at 238.125 81.28 0)
 			(effects
 				(font
@@
 		)
 		(property "Datasheet" "~"
-			(at 123.19 100.965 0)
+			(at 238.125 81.28 0)
 			(effects
 				(font
@@
 		)
 		(property "Description" "test point"
-			(at 123.19 106.045 0)
+			(at 243.205 81.28 0)
 			(effects
 				(font
@@
 	(symbol
 		(lib_id "power:GND")
-		(at 64.77 112.395 90)
+		(at 243.205 100.33 0)
 		(unit 1)
 		(exclude_from_sim no)
@@
 		(dnp no)
 		(property "Reference" "#PWR0288"
-			(at 71.12 112.395 0)
+			(at 243.205 106.68 0)
 			(effects
 				(font
@@
 		)
 		(property "Value" "GND_FAN"
-			(at 72.39 112.395 90)
+			(at 243.205 104.14 0)
 			(effects
 				(font
@@
 		)
 		(property "Footprint" ""
-			(at 64.77 112.395 0)
+			(at 243.205 100.33 0)
 			(effects
 				(font
@@
 		)
 		(property "Datasheet" ""
-			(at 64.77 112.395 0)
+			(at 243.205 100.33 0)
 			(effects
 				(font
@@
 		)
 		(property "Description" "Power symbol creates a global label with name \"GND\" , ground"
-			(at 64.77 112.395 0)
+			(at 243.205 100.33 0)
 			(effects
 				(font
@@
 	(symbol
 		(lib_id "Connector:TestPoint")
-		(at 123.19 110.49 90)
+		(at 226.695 95.885 0)
 		(unit 1)
 		(exclude_from_sim no)
@@
 		(dnp no)
 		(property "Reference" "TP36"
-			(at 115.57 111.125 90)
+			(at 227.965 92.075 0)
 			(effects
 				(font
@@
 		)
 		(property "Value" "TestPoint"
-			(at 118.11 109.22 90)
+			(at 227.965 93.98 0)
 			(effects
 				(font
@@
 		)
 		(property "Footprint" "TestPoint:TestPoint_THTPad_D1.5mm_Drill0.7mm"
-			(at 123.19 105.41 0)
+			(at 231.775 95.885 0)
 			(effects
 				(font
@@
 		)
 		(property "Datasheet" "~"
-			(at 123.19 105.41 0)
+			(at 231.775 95.885 0)
 			(effects
 				(font
@@
 		)
 		(property "Description" "test point"
-			(at 123.19 110.49 0)
+			(at 226.695 95.885 0)
 			(effects
 				(font
@@
 	(symbol
 		(lib_id "power:+12V")
-		(at 127.635 106.045 270)
+		(at 243.205 76.835 0)
 		(unit 1)
 		(exclude_from_sim no)
@@
 		(dnp no)
 		(property "Reference" "#PWR0289"
-			(at 123.825 106.045 0)
+			(at 243.205 80.645 0)
 			(effects
 				(font
@@
 		)
 		(property "Value" "5V0_FAN"
-			(at 135.255 106.045 90)
+			(at 243.205 73.025 0)
 			(effects
 				(font
@@
 		)
 		(property "Footprint" ""
-			(at 127.635 106.045 0)
+			(at 243.205 76.835 0)
 			(effects
 				(font
@@
 		)
 		(property "Datasheet" ""
-			(at 127.635 106.045 0)
+			(at 243.205 76.835 0)
 			(effects
 				(font
@@
 		)
 		(property "Description" "Power symbol creates a global label with name \"+12V\""
-			(at 127.635 106.045 0)
+			(at 243.205 76.835 0)
 			(effects
 				(font
@@
 	(symbol
 		(lib_id "power:GND")
-		(at 127.635 110.49 90)
+		(at 226.695 100.33 0)
 		(unit 1)
 		(exclude_from_sim no)
@@
 		(dnp no)
 		(property "Reference" "#PWR0290"
-			(at 133.985 110.49 0)
+			(at 226.695 106.68 0)
 			(effects
 				(font
@@
 		)
 		(property "Value" "GND_FAN"
-			(at 135.255 110.49 90)
+			(at 226.695 104.14 0)
 			(effects
 				(font
@@
 		)
 		(property "Footprint" ""
-			(at 127.635 110.49 0)
+			(at 226.695 100.33 0)
 			(effects
 				(font
@@
 		)
 		(property "Datasheet" ""
-			(at 127.635 110.49 0)
+			(at 226.695 100.33 0)
 			(effects
 				(font
@@
 		)
 		(property "Description" "Power symbol creates a global label with name \"GND\" , ground"
-			(at 127.635 110.49 0)
+			(at 226.695 100.33 0)
 			(effects
 				(font

Commit message: Updated packeges
Parts:
- added H10, H11, H9: M4, MountingHole:MountingHole_4.3mm_M4_Pad_Via, symbol Mechanical:MountingHole
- J23: footprint Connector_Molex:Molex_Micro-Fit_3.0_43045-0415_2x02_P3.00mm_Vertical -> user_lib:430450415
Changed lines of the file:
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@@
+	)
+	(symbol
+		(lib_id "Mechanical:MountingHole")
+		(at 203.2 38.1 0)
+		(unit 1)
+		(exclude_from_sim yes)
+		(in_bom no)
+		(on_board yes)
+		(dnp no)
+		(fields_autoplaced yes)
+		(property "Reference" "H9"
+			(at 205.74 36.8299 0)
+			(effects
+				(font
+					(size 1.27 1.27)
+				)
+				(justify left)
+			)
+		)
+		(property "Value" "M4"
+			(at 205.74 39.3699 0)
+			(effects
+				(font
+					(size 1.27 1.27)
+				)
+				(justify left)
+			)
+		)
+		(property "Footprint" "MountingHole:MountingHole_4.3mm_M4_Pad_Via"
+			(at 203.2 38.1 0)
+			(effects
+				(font
+					(size 1.27 1.27)
+				)
+				(hide yes)
+			)
+		)
+		(property "Datasheet" "~"
+			(at 203.2 38.1 0)
+			(effects
+				(font
+					(size 1.27 1.27)
+				)
+				(hide yes)
+			)
+		)
+		(property "Description" "Mounting Hole without connection"
+			(at 203.2 38.1 0)
+			(effects
+				(font
+					(size 1.27 1.27)
+				)
+				(hide yes)
+			)
+		)
+		(instances
+			(project "impeller18"
+				(path "/4ccab03b-4b1c-4c61-9fa8-19853ef32b4d/c3c0fd22-6514-4a88-b2de-2515415ad3c7"
+					(reference "H9")
+					(unit 1)
+				)
+			)
+		)
 	)
 	(symbol
@@
 	)
 	(symbol
+		(lib_id "Mechanical:MountingHole")
+		(at 203.2 43.815 0)
+		(unit 1)
+		(exclude_from_sim yes)
+		(in_bom no)
+		(on_board yes)
+		(dnp no)
+		(fields_autoplaced yes)
+		(property "Reference" "H10"
+			(at 205.74 42.5449 0)
+			(effects
+				(font
+					(size 1.27 1.27)
+				)
+				(justify left)
+			)
+		)
+		(property "Value" "M4"
+			(at 205.74 45.0849 0)
+			(effects
+				(font
+					(size 1.27 1.27)
+				)
+				(justify left)
+			)
+		)
+		(property "Footprint" "MountingHole:MountingHole_4.3mm_M4_Pad_Via"
+			(at 203.2 43.815 0)
+			(effects
+				(font
+					(size 1.27 1.27)
+				)
+				(hide yes)
+			)
+		)
+		(property "Datasheet" "~"
+			(at 203.2 43.815 0)
+			(effects
+				(font
+					(size 1.27 1.27)
+				)
+				(hide yes)
+			)
+		)
+		(property "Description" "Mounting Hole without connection"
+			(at 203.2 43.815 0)
+			(effects
+				(font
+					(size 1.27 1.27)
+				)
+				(hide yes)
+			)
+		)
+		(instances
+			(project "impeller18"
+				(path "/4ccab03b-4b1c-4c61-9fa8-19853ef32b4d/c3c0fd22-6514-4a88-b2de-2515415ad3c7"
+					(reference "H10")
+					(unit 1)
+				)
+			)
+		)
+	)
+	(symbol
 		(lib_id "Connector_Generic:Conn_02x02_Odd_Even")
 		(at 148.59 52.07 0)
@@
 			)
 		)
-		(property "Footprint" "Connector_Molex:Molex_Micro-Fit_3.0_43045-0415_2x02_P3.00mm_Vertical"
+		(property "Footprint" "user_lib:430450415"
 			(at 148.59 52.07 0)
 			(effects
@@
 					(unit 1)
 				)
+			)
+		)
+	)
+	(symbol
+		(lib_id "Mechanical:MountingHole")
+		(at 203.2 48.895 0)
+		(unit 1)
+		(exclude_from_sim yes)
+		(in_bom no)
+		(on_board yes)
+		(dnp no)
+		(fields_autoplaced yes)
+		(property "Reference" "H11"
+			(at 205.74 47.6249 0)
+			(effects
+				(font
+					(size 1.27 1.27)
+				)
+				(justify left)
+			)
+		)
+		(property "Value" "M4"
+			(at 205.74 50.1649 0)
+			(effects
+				(font
+					(size 1.27 1.27)
+				)
+				(justify left)
+			)
+		)
+		(property "Footprint" "MountingHole:MountingHole_4.3mm_M4_Pad_Via"
+			(at 203.2 48.895 0)
+			(effects
+				(font
+					(size 1.27 1.27)
+				)
+				(hide yes)
+			)
+		)
+		(property "Datasheet" "~"
+			(at 203.2 48.895 0)
+			(effects
+				(font
+					(size 1.27 1.27)
+				)
+				(hide yes)
+			)
+		)
+		(property "Description" "Mounting Hole without connection"
+			(at 203.2 48.895 0)
+			(effects
+				(font
+					(size 1.27 1.27)
+				)
+				(hide yes)
+			)
+		)
+		(instances
+			(project "impeller18"
+				(path "/4ccab03b-4b1c-4c61-9fa8-19853ef32b4d/c3c0fd22-6514-4a88-b2de-2515415ad3c7"
+					(reference "H11")
+					(unit 1)
+				)
