File: Hardware/ciam/impeller18/fan.kicad_sch (KiCad schematic)
At the start: 24 parts, among them J23 430450415, U75 HCPL-0600, U76 LDL1117S50R, U77 SMU02M-12

Commit message: Updated packeges
Parts:
- added H12: M4, MountingHole:MountingHole_4.3mm_M4_Pad_Via, symbol Mechanical:MountingHole
- U77: footprint (none) -> user_lib:SMU02M-12
Other:
- moved on the sheet: H11
Changed lines of the file:
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@@
 			)
 		)
-		(property "Footprint" ""
+		(property "Footprint" "user_lib:SMU02M-12"
 			(at 64.77 96.647 0)
 			(effects
@@
 				(path "/4ccab03b-4b1c-4c61-9fa8-19853ef32b4d/c3c0fd22-6514-4a88-b2de-2515415ad3c7"
 					(reference "U77")
+					(unit 1)
+				)
+			)
+		)
+	)
+	(symbol
+		(lib_id "Mechanical:MountingHole")
+		(at 203.2 55.245 0)
+		(unit 1)
+		(exclude_from_sim yes)
+		(in_bom no)
+		(on_board yes)
+		(dnp no)
+		(fields_autoplaced yes)
+		(property "Reference" "H12"
+			(at 205.74 53.9749 0)
+			(effects
+				(font
+					(size 1.27 1.27)
+				)
+				(justify left)
+			)
+		)
+		(property "Value" "M4"
+			(at 205.74 56.5149 0)
+			(effects
+				(font
+					(size 1.27 1.27)
+				)
+				(justify left)
+			)
+		)
+		(property "Footprint" "MountingHole:MountingHole_4.3mm_M4_Pad_Via"
+			(at 203.2 55.245 0)
+			(effects
+				(font
+					(size 1.27 1.27)
+				)
+				(hide yes)
+			)
+		)
+		(property "Datasheet" "~"
+			(at 203.2 55.245 0)
+			(effects
+				(font
+					(size 1.27 1.27)
+				)
+				(hide yes)
+			)
+		)
+		(property "Description" "Mounting Hole without connection"
+			(at 203.2 55.245 0)
+			(effects
+				(font
+					(size 1.27 1.27)
+				)
+				(hide yes)
+			)
+		)
+		(instances
+			(project "impeller18"
+				(path "/4ccab03b-4b1c-4c61-9fa8-19853ef32b4d/c3c0fd22-6514-4a88-b2de-2515415ad3c7"
+					(reference "H12")
 					(unit 1)
 				)
@@
 	(symbol
 		(lib_id "Mechanical:MountingHole")
-		(at 203.2 48.895 0)
+		(at 203.2 49.53 0)
 		(unit 1)
 		(exclude_from_sim yes)
@@
 		(fields_autoplaced yes)
 		(property "Reference" "H11"
-			(at 205.74 47.6249 0)
+			(at 205.74 48.2599 0)
 			(effects
 				(font
@@
 		)
 		(property "Value" "M4"
-			(at 205.74 50.1649 0)
+			(at 205.74 50.7999 0)
 			(effects
 				(font
@@
 		)
 		(property "Footprint" "MountingHole:MountingHole_4.3mm_M4_Pad_Via"
-			(at 203.2 48.895 0)
+			(at 203.2 49.53 0)
 			(effects
 				(font
@@
 		)
 		(property "Datasheet" "~"
-			(at 203.2 48.895 0)
+			(at 203.2 49.53 0)
 			(effects
 				(font
@@
 		)
 		(property "Description" "Mounting Hole without connection"
-			(at 203.2 48.895 0)
-			(effects
-				(font
+			(at 203.2 49.53 0)
+			(effects
+				(font

Commit message: Updated 3D models
Parts:
- renumbered C111 to C122, C112 to C123, C113 to C124, C114 to C125, C115 to C126, C116 to C127, D25 to D24, D26 to D25, J23 to J31, R279 to R334, R280 to R335, R281 to R336, R282 to R337, R283 to R338, TP33 to TP42, TP35 to TP43, TP36 to TP44, TP34 to TP45, U75 to U73, U76 to U74, U77 to U75

Commit message: updated bom
Parts:
- added C125, C128: 4u7, Capacitor_SMD:C_1210_3225Metric, symbol Device:C_Small
- renumbered C122 to C126, C123 to C127, C124 to C129, C125 to C130, C126 to C131, C127 to C132
Connections:
- net 12V0: now also C125.1
- net 12V0_FAN: now also C128.1
- net GND_12V: now also C125.2
- net GND_FAN: now also C128.2
Other:
- moved on the sheet: C126, C127, U75

Commit message: Update PCB concept
Connections:
- net GND_FAN: now also U73.5 (GND)
- net GND_12V renamed GND
- net GND: no longer U73.5 (GND)
Changed lines of the file:
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@@
-	)
-	(symbol
-		(lib_id "power:GND")
-		(at 29.21 95.25 0)
-		(unit 1)
-		(exclude_from_sim no)
-		(in_bom yes)
-		(on_board yes)
-		(dnp no)
-		(property "Reference" "#PWR0296"
-			(at 29.21 101.6 0)
-			(effects
-				(font
-					(size 1.27 1.27)
-				)
-				(hide yes)
-			)
-		)
-		(property "Value" "GND_12V"
-			(at 29.21 99.06 0)
-			(effects
-				(font
-					(size 1.27 1.27)
-				)
-			)
-		)
-		(property "Footprint" ""
-			(at 29.21 95.25 0)
-			(effects
-				(font
-					(size 1.27 1.27)
-				)
-				(hide yes)
-			)
-		)
-		(property "Datasheet" ""
-			(at 29.21 95.25 0)
-			(effects
-				(font
-					(size 1.27 1.27)
-				)
-				(hide yes)
-			)
-		)
-		(property "Description" "Power symbol creates a global label with name \"GND\" , ground"
-			(at 29.21 95.25 0)
-			(effects
-				(font
-					(size 1.27 1.27)
-				)
-				(hide yes)
-			)
-		)
-		(pin "1"
-		)
-		(instances
-			(project "impeller18"
-				(path "/4ccab03b-4b1c-4c61-9fa8-19853ef32b4d/c3c0fd22-6514-4a88-b2de-2515415ad3c7"
-					(reference "#PWR0296")
-					(unit 1)
-				)
-			)
-		)
 	)
 	(symbol
@@
 	)
 	(symbol
+		(lib_id "power:GND")
+		(at 119.38 60.325 0)
+		(unit 1)
+		(exclude_from_sim no)
+		(in_bom yes)
+		(on_board yes)
+		(dnp no)
+		(property "Reference" "#PWR0315"
+			(at 119.38 66.675 0)
+			(effects
+				(font
+					(size 1.27 1.27)
+				)
+				(hide yes)
+			)
+		)
+		(property "Value" "GND_FAN"
+			(at 119.38 64.135 0)
+			(effects
+				(font
+					(size 1.27 1.27)
+				)
+			)
+		)
+		(property "Footprint" ""
+			(at 119.38 60.325 0)
+			(effects
+				(font
+					(size 1.27 1.27)
+				)
+				(hide yes)
+			)
+		)
+		(property "Datasheet" ""
+			(at 119.38 60.325 0)
+			(effects
+				(font
+					(size 1.27 1.27)
+				)
+				(hide yes)
+			)
+		)
+		(property "Description" "Power symbol creates a global label with name \"GND\" , ground"
+			(at 119.38 60.325 0)
+			(effects
+				(font
+					(size 1.27 1.27)
+				)
+				(hide yes)
+			)
+		)
+		(pin "1"
+		)
+		(instances
+			(project "impeller18"
+				(path "/4ccab03b-4b1c-4c61-9fa8-19853ef32b4d/c3c0fd22-6514-4a88-b2de-2515415ad3c7"
+					(reference "#PWR0315")
+					(unit 1)
+				)
+			)
+		)
+	)
+	(symbol
 		(lib_id "power:+12V")
 		(at 243.205 76.835 0)
@@
 	)
 	(symbol
-		(lib_id "power:GND")
-		(at 119.38 60.325 0)
-		(unit 1)
-		(exclude_from_sim no)
-		(in_bom yes)
-		(on_board yes)
-		(dnp no)
-		(property "Reference" "#PWR0287"
-			(at 119.38 66.675 0)
-			(effects
-				(font
-					(size 1.27 1.27)
-				)
-				(hide yes)
-			)
-		)
-		(property "Value" "GND_12V"
-			(at 119.38 64.135 0)
-			(effects
-				(font
-					(size 1.27 1.27)
-				)
-			)
-		)
-		(property "Footprint" ""
-			(at 119.38 60.325 0)
-			(effects
-				(font
-					(size 1.27 1.27)
-				)
-				(hide yes)
-			)
-		)
-		(property "Datasheet" ""
-			(at 119.38 60.325 0)
-			(effects
-				(font
-					(size 1.27 1.27)
-				)
-				(hide yes)
-			)
-		)
-		(property "Description" "Power symbol creates a global label with name \"GND\" , ground"
-			(at 119.38 60.325 0)
-			(effects
-				(font
-					(size 1.27 1.27)
-				)
-				(hide yes)
-			)
-		)
-		(pin "1"
-		)
-		(instances
-			(project "impeller18"
-				(path "/4ccab03b-4b1c-4c61-9fa8-19853ef32b4d/c3c0fd22-6514-4a88-b2de-2515415ad3c7"
-					(reference "#PWR0287")
-					(unit 1)
-				)
-			)
-		)
-	)
-	(symbol
 		(lib_id "power:+12V")
 		(at 199.39 78.74 0)
@@
 					(unit 1)
 				)
+			)
+		)
+	)
+	(symbol
+		(lib_id "power:GND")
+		(at 29.21 95.25 0)
+		(unit 1)
+		(exclude_from_sim no)
+		(in_bom yes)
+		(on_board yes)
+		(dnp no)
+		(fields_autoplaced yes)
+		(property "Reference" "#PWR0287"
+			(at 29.21 101.6 0)
+			(effects
+				(font
+					(size 1.27 1.27)
+				)
+				(hide yes)
+			)
+		)
+		(property "Value" "GND"
+			(at 29.21 100.33 0)
+			(effects
+				(font
+					(size 1.27 1.27)
+				)
+			)
+		)
+		(property "Footprint" ""
+			(at 29.21 95.25 0)
+			(effects
+				(font
+					(size 1.27 1.27)
+				)
+				(hide yes)
+			)
+		)
+		(property "Datasheet" ""
+			(at 29.21 95.25 0)
+			(effects
+				(font
+					(size 1.27 1.27)
+				)
+				(hide yes)
+			)
+		)
+		(property "Description" "Power symbol creates a global label with name \"GND\" , ground"
+			(at 29.21 95.25 0)
+			(effects
+				(font
+					(size 1.27 1.27)
+				)
+				(hide yes)
+			)
+		)
+		(pin "1"
+		)
+		(instances
+			(project "impeller18"
+				(path "/4ccab03b-4b1c-4c61-9fa8-19853ef32b4d/c3c0fd22-6514-4a88-b2de-2515415ad3c7"
+					(reference "#PWR0287")
+					(unit 1)
+				)

Commit message: Daily PCB update
Parts:
- renumbered R334 to R338, R335 to R339, R336 to R340, R337 to R341, R338 to R342, TP42 to TP43, TP43 to TP44, TP44 to TP45, TP45 to TP46
Changed lines of the file:
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@@
 		(on_board yes)
 		(dnp no)
-		(property "Reference" "#PWR0297"
+		(property "Reference" "#PWR0309"
 			(at 73.66 101.6 0)
 			(effects
@@
 			(project "impeller18"
 				(path "/4ccab03b-4b1c-4c61-9fa8-19853ef32b4d/c3c0fd22-6514-4a88-b2de-2515415ad3c7"
-					(reference "#PWR0297")
+					(reference "#PWR0309")
 					(unit 1)
 				)
@@
 		(on_board yes)
 		(dnp no)
-		(property "Reference" "#PWR0283"
+		(property "Reference" "#PWR0295"
 			(at 119.38 43.18 0)
 			(effects
@@
 			(project "impeller18"
 				(path "/4ccab03b-4b1c-4c61-9fa8-19853ef32b4d/c3c0fd22-6514-4a88-b2de-2515415ad3c7"
-					(reference "#PWR0283")
+					(reference "#PWR0295")
 					(unit 1)
 				)
@@
 		(on_board yes)
 		(dnp no)
-		(property "Reference" "TP45"
+		(property "Reference" "TP46"
 			(at 244.475 92.075 0)
 			(effects
@@
 			(project "impeller18"
 				(path "/4ccab03b-4b1c-4c61-9fa8-19853ef32b4d/c3c0fd22-6514-4a88-b2de-2515415ad3c7"
-					(reference "TP45")
+					(reference "TP46")
 					(unit 1)
 				)
@@
 		(on_board yes)
 		(dnp no)
-		(property "Reference" "#PWR0288"
+		(property "Reference" "#PWR0300"
 			(at 226.695 80.645 0)
 			(effects
@@
 			(project "impeller18"
 				(path "/4ccab03b-4b1c-4c61-9fa8-19853ef32b4d/c3c0fd22-6514-4a88-b2de-2515415ad3c7"
-					(reference "#PWR0288")
+					(reference "#PWR0300")
 					(unit 1)
 				)
@@
 		(on_board yes)
 		(dnp no)
-		(property "Reference" "R336"
+		(property "Reference" "R340"
 			(at 96.52 50.165 90)
 			(effects
@@
 			(project "impeller18"
 				(path "/4ccab03b-4b1c-4c61-9fa8-19853ef32b4d/c3c0fd22-6514-4a88-b2de-2515415ad3c7"
-					(reference "R336")
+					(reference "R340")
 					(unit 1)
 				)
@@
 		(on_board yes)
 		(dnp no)
-		(property "Reference" "TP42"
+		(property "Reference" "TP43"
 			(at 233.045 83.82 0)
 			(effects
@@
 			(project "impeller18"
 				(path "/4ccab03b-4b1c-4c61-9fa8-19853ef32b4d/c3c0fd22-6514-4a88-b2de-2515415ad3c7"
-					(reference "TP42")
+					(reference "TP43")
 					(unit 1)
 				)
@@
 		(on_board yes)
 		(dnp no)
-		(property "Reference" "#PWR0300"
+		(property "Reference" "#PWR0312"
 			(at 199.39 105.41 0)
 			(effects
@@
 			(project "impeller18"
 				(path "/4ccab03b-4b1c-4c61-9fa8-19853ef32b4d/c3c0fd22-6514-4a88-b2de-2515415ad3c7"
-					(reference "#PWR0300")
+					(reference "#PWR0312")
 					(unit 1)
 				)
@@
 		(on_board yes)
 		(dnp no)
-		(property "Reference" "#PWR0299"
+		(property "Reference" "#PWR0311"
 			(at 175.895 105.41 0)
 			(effects
@@
 			(project "impeller18"
 				(path "/4ccab03b-4b1c-4c61-9fa8-19853ef32b4d/c3c0fd22-6514-4a88-b2de-2515415ad3c7"
-					(reference "#PWR0299")
+					(reference "#PWR0311")
 					(unit 1)
 				)
@@
 		(on_board yes)
 		(dnp no)
-		(property "Reference" "#PWR0293"
+		(property "Reference" "#PWR0305"
 			(at 145.415 86.36 0)
 			(effects
@@
 			(project "impeller18"
 				(path "/4ccab03b-4b1c-4c61-9fa8-19853ef32b4d/c3c0fd22-6514-4a88-b2de-2515415ad3c7"
-					(reference "#PWR0293")
+					(reference "#PWR0305")
 					(unit 1)
 				)
@@
 		(on_board yes)
 		(dnp no)
-		(property "Reference" "#PWR0286"
+		(property "Reference" "#PWR0298"
 			(at 162.56 63.5 0)
 			(effects
@@
 			(project "impeller18"
 				(path "/4ccab03b-4b1c-4c61-9fa8-19853ef32b4d/c3c0fd22-6514-4a88-b2de-2515415ad3c7"
-					(reference "#PWR0286")
+					(reference "#PWR0298")
 					(unit 1)
 				)
@@
 		(on_board yes)
 		(dnp no)
-		(property "Reference" "TP43"
+		(property "Reference" "TP44"
 			(at 249.555 83.82 0)
 			(effects
@@
 			(project "impeller18"
 				(path "/4ccab03b-4b1c-4c61-9fa8-19853ef32b4d/c3c0fd22-6514-4a88-b2de-2515415ad3c7"
-					(reference "TP43")
+					(reference "TP44")
 					(unit 1)
 				)
@@
 		(on_board yes)
 		(dnp no)
-		(property "Reference" "#PWR0302"
+		(property "Reference" "#PWR0314"
 			(at 243.205 106.68 0)
 			(effects
@@
 			(project "impeller18"
 				(path "/4ccab03b-4b1c-4c61-9fa8-19853ef32b4d/c3c0fd22-6514-4a88-b2de-2515415ad3c7"
-					(reference "#PWR0302")
+					(reference "#PWR0314")
 					(unit 1)
 				)
@@
 		(on_board yes)
 		(dnp no)
-		(property "Reference" "R335"
+		(property "Reference" "R339"
 			(at 139.7 44.45 0)
 			(effects
@@
 			(project "impeller18"
 				(path "/4ccab03b-4b1c-4c61-9fa8-19853ef32b4d/c3c0fd22-6514-4a88-b2de-2515415ad3c7"
-					(reference "R335")
+					(reference "R339")
 					(unit 1)
 				)
@@
 		(dnp no)
 		(fields_autoplaced yes)
-		(property "Reference" "#PWR0284"
+		(property "Reference" "#PWR0296"
 			(at 90.17 50.8 0)
 			(effects
@@
 			(project "impeller18"
 				(path "/4ccab03b-4b1c-4c61-9fa8-19853ef32b4d/c3c0fd22-6514-4a88-b2de-2515415ad3c7"
-					(reference "#PWR0284")
+					(reference "#PWR0296")
 					(unit 1)
 				)
@@
 		(on_board yes)
 		(dnp no)
-		(property "Reference" "TP44"
+		(property "Reference" "TP45"
 			(at 227.965 92.075 0)
 			(effects
@@
 			(project "impeller18"
 				(path "/4ccab03b-4b1c-4c61-9fa8-19853ef32b4d/c3c0fd22-6514-4a88-b2de-2515415ad3c7"
-					(reference "TP44")
+					(reference "TP45")
 					(unit 1)
 				)
@@
 		(on_board yes)
 		(dnp no)
-		(property "Reference" "R337"
+		(property "Reference" "R341"
 			(at 179.705 82.55 0)
 			(effects
@@
 			(project "impeller18"
 				(path "/4ccab03b-4b1c-4c61-9fa8-19853ef32b4d/c3c0fd22-6514-4a88-b2de-2515415ad3c7"
-					(reference "R337")
+					(reference "R341")
 					(unit 1)
 				)
@@
 		(on_board yes)
 		(dnp no)
-		(property "Reference" "#PWR0298"
+		(property "Reference" "#PWR0310"
 			(at 95.885 105.41 0)
 			(effects
@@
 			(project "impeller18"
 				(path "/4ccab03b-4b1c-4c61-9fa8-19853ef32b4d/c3c0fd22-6514-4a88-b2de-2515415ad3c7"
-					(reference "#PWR0298")
+					(reference "#PWR0310")
 					(unit 1)
 				)
@@
 		(on_board yes)
 		(dnp no)
-		(property "Reference" "#PWR0292"
+		(property "Reference" "#PWR0304"
 			(at 95.885 86.36 0)
 			(effects
@@
 			(project "impeller18"
 				(path "/4ccab03b-4b1c-4c61-9fa8-19853ef32b4d/c3c0fd22-6514-4a88-b2de-2515415ad3c7"
-					(reference "#PWR0292")
+					(reference "#PWR0304")
 					(unit 1)
 				)
@@
 		(on_board yes)
 		(dnp no)
-		(property "Reference" "#PWR0315"
+		(property "Reference" "#PWR0299"
 			(at 119.38 66.675 0)
 			(effects
@@
 			(project "impeller18"
 				(path "/4ccab03b-4b1c-4c61-9fa8-19853ef32b4d/c3c0fd22-6514-4a88-b2de-2515415ad3c7"
-					(reference "#PWR0315")
+					(reference "#PWR0299")
 					(unit 1)
 				)
@@
 		(on_board yes)
 		(dnp no)
-		(property "Reference" "#PWR0289"
+		(property "Reference" "#PWR0301"
 			(at 243.205 80.645 0)
 			(effects
@@
 			(project "impeller18"
 				(path "/4ccab03b-4b1c-4c61-9fa8-19853ef32b4d/c3c0fd22-6514-4a88-b2de-2515415ad3c7"
-					(reference "#PWR0289")
+					(reference "#PWR0301")
 					(unit 1)
 				)
@@
 		(on_board yes)
 		(dnp no)
-		(property "Reference" "#PWR0290"
+		(property "Reference" "#PWR0302"
 			(at 175.895 82.55 0)
 			(effects
@@
 			(project "impeller18"
 				(path "/4ccab03b-4b1c-4c61-9fa8-19853ef32b4d/c3c0fd22-6514-4a88-b2de-2515415ad3c7"
-					(reference "#PWR0290")
+					(reference "#PWR0302")
 					(unit 1)
 				)
@@
 		(on_board yes)
 		(dnp no)
-		(property "Reference" "#PWR0291"
+		(property "Reference" "#PWR0303"
 			(at 199.39 82.55 0)
 			(effects
@@
 			(project "impeller18"
 				(path "/4ccab03b-4b1c-4c61-9fa8-19853ef32b4d/c3c0fd22-6514-4a88-b2de-2515415ad3c7"
-					(reference "#PWR0291")
+					(reference "#PWR0303")
 					(unit 1)
 				)
@@
 		(on_board yes)
 		(dnp no)
-		(property "Reference" "#PWR0294"
+		(property "Reference" "#PWR0306"
 			(at 73.66 87.63 0)
 			(effects
@@
 			(project "impeller18"
 				(path "/4ccab03b-4b1c-4c61-9fa8-19853ef32b4d/c3c0fd22-6514-4a88-b2de-2515415ad3c7"
-					(reference "#PWR0294")
+					(reference "#PWR0306")
 					(unit 1)
 				)
@@
 		(dnp no)
 		(fields_autoplaced yes)
-		(property "Reference" "#PWR0287"
+		(property "Reference" "#PWR0308"
 			(at 29.21 101.6 0)
 			(effects
@@
 			(project "impeller18"
 				(path "/4ccab03b-4b1c-4c61-9fa8-19853ef32b4d/c3c0fd22-6514-4a88-b2de-2515415ad3c7"
-					(reference "#PWR0287")
+					(reference "#PWR0308")
 					(unit 1)
 				)
@@
 		(on_board yes)
 		(dnp no)
-		(property "Reference" "#PWR0285"
+		(property "Reference" "#PWR0297"
 			(at 162.56 52.07 0)
 			(effects
@@
 			(project "impeller18"
 				(path "/4ccab03b-4b1c-4c61-9fa8-19853ef32b4d/c3c0fd22-6514-4a88-b2de-2515415ad3c7"
-					(reference "#PWR0285")
+					(reference "#PWR0297")
 					(unit 1)
 				)
@@
 		(on_board yes)
 		(dnp no)
-		(property "Reference" "R334"
+		(property "Reference" "R338"
 			(at 131.445 44.45 0)
 			(effects
@@
 			(project "impeller18"
 				(path "/4ccab03b-4b1c-4c61-9fa8-19853ef32b4d/c3c0fd22-6514-4a88-b2de-2515415ad3c7"
-					(reference "R334")
+					(reference "R338")
 					(unit 1)
 				)
@@
 		(dnp no)
 		(fields_autoplaced yes)
-		(property "Reference" "#PWR0295"
+		(property "Reference" "#PWR0307"
 			(at 29.21 88.265 0)
 			(effects
@@
 			(project "impeller18"
 				(path "/4ccab03b-4b1c-4c61-9fa8-19853ef32b4d/c3c0fd22-6514-4a88-b2de-2515415ad3c7"
-					(reference "#PWR0295")
+					(reference "#PWR0307")
 					(unit 1)
 				)
@@
 		(on_board yes)
 		(dnp no)
-		(property "Reference" "R338"
+		(property "Reference" "R342"
 			(at 203.2 82.55 0)
 			(effects
@@
 			(project "impeller18"
 				(path "/4ccab03b-4b1c-4c61-9fa8-19853ef32b4d/c3c0fd22-6514-4a88-b2de-2515415ad3c7"
-					(reference "R338")
+					(reference "R342")
 					(unit 1)
 				)
@@
 		(on_board yes)
 		(dnp no)
-		(property "Reference" "#PWR0301"
+		(property "Reference" "#PWR0313"
 			(at 226.695 106.68 0)
 			(effects
@@
 			(project "impeller18"
 				(path "/4ccab03b-4b1c-4c61-9fa8-19853ef32b4d/c3c0fd22-6514-4a88-b2de-2515415ad3c7"
-					(reference "#PWR0301")
+					(reference "#PWR0313")
 					(unit 1)
 				)

Commit message: Update PCB concept
Parts:
- C125, C128: footprint Capacitor_SMD:C_1210_3225Metric -> Capacitor_SMD:C_0603_1608Metric; Мин. кол-во 17 -> 200; Ссылка https://www.promelec.ru/product/384583/ -> https://www.promelec.ru/product/315964/; Цена 29 -> 4; Человекопонятное название Керамический ЧИП-конденсатор 1210 X7S 4.7мкФ -> Керамический ЧИП-конденсатор 0603 X5R 4.7мкФ
- H10, H11, H12, H9: footprint MountingHole:MountingHole_4.3mm_M4_Pad_Via -> user_lib:MountingHole_M4_PCHSS4-22
- TP37: renamed from TP43; footprint TestPoint:TestPoint_THTPad_D1.5mm_Drill0.7mm -> TestPoint:TestPoint_THTPad_D2.0mm_Drill1.0mm
- TP38: renamed from TP44; footprint TestPoint:TestPoint_THTPad_D1.5mm_Drill0.7mm -> TestPoint:TestPoint_THTPad_D2.0mm_Drill1.0mm
- TP39: renamed from TP45; footprint TestPoint:TestPoint_THTPad_D1.5mm_Drill0.7mm -> TestPoint:TestPoint_THTPad_D2.0mm_Drill1.0mm
- TP40: renamed from TP46; footprint TestPoint:TestPoint_THTPad_D1.5mm_Drill0.7mm -> TestPoint:TestPoint_THTPad_D2.0mm_Drill1.0mm
- renumbered J31 to J34, R338 to R335, R339 to R336, R340 to R337, R341 to R338, R342 to R339
Connections:
- net 12V0: now also C125.2; no longer C125.1
- net 3V3: now also U73.2 (A); no longer R337.1
- net FAN_PWM_3V3: now also R337.1; no longer U73.3 (C)
- net GND: now also C125.1; no longer C125.2
- net at R337.2: now also U73.3 (C); no longer U73.2 (A)
Other:
- moved on the sheet: R337

Commit message: Zone borders
Parts:
- removed C127: 100n, Capacitor_SMD:C_0603_1608Metric, symbol Device:C_Small
- removed TP40: TestPoint, TestPoint:TestPoint_THTPad_D2.0mm_Drill1.0mm, symbol Connector:TestPoint
- D24, D25: footprint LED_SMD:LED_0603_1608Metric -> user_lib:LED_0603_1608Metric
- J34: symbol Connector_Generic:Conn_02x02_Odd_Even -> Connector_Generic:Conn_02x02_Counter_Clockwise
Connections:
- net 12V0_FAN: now also D24.2 (A), J34.3 (Pin_3); no longer J34.2 (Pin_2), R338.2
- net 5V0_FAN: now also D25.2 (A); no longer R339.2
- net FAN_PWM_5V0: now also J34.2 (Pin_2); no longer J34.1 (Pin_1)
- net GND_FAN: now also R338.1, R339.1; no longer D24.1 (K), D25.1 (K)
- new net: D24.1 (K), R338.2
- new net: D25.1 (K), R339.2
Other:
- moved on the sheet: D24, D25, R338, R339

Commit message: Sch ready
Parts:
- added TP6: TestPoint, TestPoint:TestPoint_THTPad_D2.0mm_Drill1.0mm, symbol Connector:TestPoint
Connections:
- net FAN_PWM_3V3: now also TP6.1
Changed lines of the file:
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@@
 	(paper "A3")
+	(junction
+		(at 90.805 57.15)
+		(diameter 0)
+		(color 0 0 0 0)
+	)
 	(junction
 		(at 38.735 92.71)
@@
 	(wire
 		(pts
+			(xy 90.805 57.15) (xy 93.98 57.15)
+		)
+		(stroke
+			(width 0)
+			(type default)
+		)
+	)
+	(wire
+		(pts
 			(xy 29.21 84.455) (xy 29.21 86.36)
 		)
@@
 	(wire
 		(pts
+			(xy 90.805 54.61) (xy 90.805 57.15)
+		)
+		(stroke
+			(width 0)
+			(type default)
+		)
+	)
+	(wire
+		(pts
 			(xy 116.205 49.53) (xy 125.095 49.53)
 		)
@@
 	(wire
 		(pts
-			(xy 89.535 57.15) (xy 93.98 57.15)
+			(xy 88.265 57.15) (xy 90.805 57.15)
 		)
 		(stroke
@@
 	(global_label "FAN_PWM_3V3"
 		(shape input)
-		(at 89.535 57.15 180)
+		(at 88.265 57.15 180)
 		(fields_autoplaced yes)
 		(effects
@@
 		)
 		(property "Intersheetrefs" "${INTERSHEET_REFS}"
-			(at 73.4265 57.15 0)
+			(at 72.1565 57.15 0)
 			(effects
 				(font
@@
 					(unit 1)
 				)
+			)
+		)
+	)
+	(symbol
+		(lib_id "Connector:TestPoint")
+		(at 90.805 54.61 0)
+		(unit 1)
+		(exclude_from_sim no)
+		(in_bom yes)
+		(on_board yes)
+		(dnp no)
+		(property "Reference" "TP6"
+			(at 84.455 52.07 0)
+			(effects
+				(font
+					(size 1.27 1.27)
+				)
+				(justify left)
+			)
+		)
+		(property "Value" "TestPoint"
+			(at 80.645 50.165 0)
+			(effects
+				(font
+					(size 1.27 1.27)
+				)
+				(justify left)
+			)
+		)
+		(property "Footprint" "TestPoint:TestPoint_THTPad_D2.0mm_Drill1.0mm"
+			(at 95.885 54.61 0)
+			(effects
+				(font
+					(size 1.27 1.27)
+				)
+				(hide yes)
+			)
+		)
+		(property "Datasheet" "~"
+			(at 95.885 54.61 0)
+			(effects
+				(font
+					(size 1.27 1.27)
+				)
+				(hide yes)
+			)
+		)
+		(property "Description" "test point"
+			(at 90.805 54.61 0)
+			(effects
+				(font
+					(size 1.27 1.27)
+				)
+				(hide yes)
+			)
+		)
+		(pin "1"
+		)
+		(instances
+			(project "impeller18"
+				(path "/4ccab03b-4b1c-4c61-9fa8-19853ef32b4d/c3c0fd22-6514-4a88-b2de-2515415ad3c7"
+					(reference "TP6")
+					(unit 1)
+				)
