File: Hardware/ciam/impeller18/impeller18.kicad_pcb (KiCad board)
At the start: 2 copper layers, 77 parts, among them J10 430450600, J11 430450600, J12 430450600, J13 430451800, J14 430451800, J15 430451600, J16 430450600, J17 430451600, J18 TF-01, J19 USB_B_Micro, J6 430451800, J7 430451800, J8 430451800, J9 430451000, Q1 BSS138, Q34 BSS138, Q35 BSS138, Q36 BSS138, SW1 SW_RESET, U1 STM32F427ZGTx, U71 W25Q128FVSIG, U72 USBLC6-2SC6, U9 LD1084V, Y1 X322516MLB4SI, Y2 KSE-7K32768KDY2400A3

Commit message: added footprints
Parts:
- removed J7: 430451800, Connector_Molex:Molex_Micro-Fit_3.0_43045-1800_2x09_P3.00mm_Horizontal
- added C10: 100n, Capacitor_SMD:C_0603_1608Metric, F.Cu at (153.3, 119.3)
- added C100: 1u, Capacitor_SMD:C_0603_1608Metric, F.Cu at (147.3, 29.3)
- added C101: 100n, Capacitor_SMD:C_0603_1608Metric, F.Cu at (147.3, 31.8)
- added C102: 4u7, Capacitor_SMD:C_0603_1608Metric, F.Cu at (147.3, 34.3)
- added C103: 100n, Capacitor_SMD:C_0603_1608Metric, F.Cu at (151.4, 19.3)
- added C104: 10n, Capacitor_SMD:C_0603_1608Metric, F.Cu at (151.4, 21.8)
- added C105: 100n, Capacitor_SMD:C_0603_1608Metric, F.Cu at (151.4, 24.3)
- added C106: 1u, Capacitor_SMD:C_0603_1608Metric, F.Cu at (151.4, 26.8)
- added C107: 100n, Capacitor_SMD:C_0603_1608Metric, F.Cu at (151.4, 29.3)
- added C11: 100n, Capacitor_SMD:C_0603_1608Metric, F.Cu at (153.3, 121.8)
- added C111: 100n, Capacitor_SMD:C_0603_1608Metric, F.Cu at (54.0, 149.2)
- added C112: 100n, Capacitor_SMD:C_0603_1608Metric, F.Cu at (54.0, 151.7)
- added C113: 1u, Capacitor_SMD:C_0603_1608Metric, F.Cu at (54.0, 154.2)
- added C114: 100n, Capacitor_SMD:C_0603_1608Metric, F.Cu at (54.0, 156.7)
- added C115: 4u7, Capacitor_SMD:C_0603_1608Metric, F.Cu at (54.0, 159.3)
- added C116: 100n, Capacitor_SMD:C_0603_1608Metric, F.Cu at (54.0, 161.8)
- added C117: 1u, Capacitor_SMD:C_0603_1608Metric, F.Cu at (108.7, 24.3)
- added C118: 100n, Capacitor_SMD:C_0603_1608Metric, F.Cu at (108.7, 26.8)
- added C119: 10u, Capacitor_SMD:C_0603_1608Metric, F.Cu at (108.7, 29.3)
- added C12: 100n, Capacitor_SMD:C_0603_1608Metric, F.Cu at (153.3, 124.3)
- added C120: 100n, Capacitor_SMD:C_0603_1608Metric, F.Cu at (108.7, 31.8)
- added C13: 100n, Capacitor_SMD:C_0603_1608Metric, F.Cu at (153.3, 126.8)
- added C14: 100n, Capacitor_SMD:C_0603_1608Metric, F.Cu at (153.3, 129.4)
- added C15: 100n, Capacitor_SMD:C_0603_1608Metric, F.Cu at (157.3, 114.3)
- added C16: 100n, Capacitor_SMD:C_0603_1608Metric, F.Cu at (157.3, 116.8)
- added C17: 1u, Capacitor_SMD:C_0603_1608Metric, F.Cu at (157.3, 119.3)
- added C18: 100n, Capacitor_SMD:C_0603_1608Metric, F.Cu at (157.3, 121.8)
- added C19: 1u, Capacitor_SMD:C_0603_1608Metric, F.Cu at (157.3, 124.3)
- added C20: 100n, Capacitor_SMD:C_0603_1608Metric, F.Cu at (157.3, 126.8)
- added C26: 10u, Capacitor_THT:CP_Radial_D10.0mm_P5.00mm, F.Cu at (132.0, 43.9)
- added C27: 47u, Capacitor_THT:CP_Radial_D12.5mm_P5.00mm, F.Cu at (93.2, 25.1)
- added C28: 470u, Capacitor_THT:CP_Radial_D12.5mm_P5.00mm, F.Cu at (93.2, 39.1)
- added C29: 1u, Capacitor_SMD:C_0603_1608Metric, F.Cu at (104.7, 19.3)
- added C3: 4u7, Capacitor_SMD:C_0603_1608Metric, F.Cu at (149.3, 119.3)
- added C30: 100n, Capacitor_SMD:C_0603_1608Metric, F.Cu at (104.7, 21.8)
- added C31: 4u7, Capacitor_SMD:C_0603_1608Metric, F.Cu at (104.7, 24.3)
- added C32: 100n, Capacitor_SMD:C_0603_1608Metric, F.Cu at (104.7, 26.8)
- added C33: 330p, Capacitor_SMD:C_1206_3216Metric, F.Cu at (105.5, 64.2)
- added C34: 330p, Capacitor_SMD:C_1206_3216Metric, F.Cu at (105.5, 67.6)
- added C35: 330p, Capacitor_SMD:C_1206_3216Metric, F.Cu at (105.5, 70.9)
- added C36: 330p, Capacitor_SMD:C_1206_3216Metric, F.Cu at (105.5, 74.3)
- added C37: 22u, Capacitor_THT:CP_Radial_D6.3mm_P2.50mm, F.Cu at (119.1, 69.9)
- added C38: 4u7, Capacitor_SMD:C_1210_3225Metric, F.Cu at (127.5, 73.2)
- added C39: 470u, Capacitor_THT:CP_Radial_D12.5mm_P5.00mm, F.Cu at (93.2, 53.2)
- added C4: 100n, Capacitor_SMD:C_0603_1608Metric, F.Cu at (149.3, 121.8)
- added C40: 100u, Capacitor_THT:CP_Radial_D8.0mm_P3.50mm, F.Cu at (136.3, 64.7)
- added C41: 100n, Capacitor_SMD:C_0603_1608Metric, F.Cu at (104.7, 29.3)
- added C42: 100n, Capacitor_SMD:C_0603_1608Metric, F.Cu at (104.7, 31.8)
- added C43: 10u, Capacitor_SMD:C_0603_1608Metric, F.Cu at (104.7, 34.3)
- added C44: 10u, Capacitor_SMD:C_0603_1608Metric, F.Cu at (104.7, 36.9)
- added C45: 100n, Capacitor_SMD:C_0603_1608Metric, F.Cu at (108.7, 19.3)
- added C46: 100n, Capacitor_SMD:C_0603_1608Metric, F.Cu at (108.7, 21.8)
- added C47: 1u, Capacitor_SMD:C_0603_1608Metric, F.Cu at (82.5, 91.0)
- added C48: 1u, Capacitor_SMD:C_0603_1608Metric, F.Cu at (82.5, 93.5)
- added C49: 100n, Capacitor_SMD:C_0603_1608Metric, F.Cu at (82.5, 96.0)
- added C5: 100n, Capacitor_SMD:C_0603_1608Metric, F.Cu at (149.3, 124.3)
- added C50: 100n, Capacitor_SMD:C_0603_1608Metric, F.Cu at (82.5, 98.5)
- added C51: 1u, Capacitor_SMD:C_0603_1608Metric, F.Cu at (82.5, 101.0)
- added C52: 1u, Capacitor_SMD:C_0603_1608Metric, F.Cu at (82.5, 103.6)
- added C53: 100n, Capacitor_SMD:C_0603_1608Metric, F.Cu at (82.5, 106.1)
- added C54: 22p, Capacitor_SMD:C_0603_1608Metric, F.Cu at (82.5, 108.6)
- added C55: 22p, Capacitor_SMD:C_0603_1608Metric, F.Cu at (82.5, 111.1)
- added C56: 100n, Capacitor_SMD:C_0603_1608Metric, F.Cu at (86.5, 91.0)
- added C57: 10u, Capacitor_SMD:C_0603_1608Metric, F.Cu at (86.5, 93.5)
- added C58: 10u, Capacitor_SMD:C_0603_1608Metric, F.Cu at (86.5, 96.0)
- added C59: 100n, Capacitor_SMD:C_0603_1608Metric, F.Cu at (86.5, 98.5)
- added C6: 100n, Capacitor_SMD:C_0603_1608Metric, F.Cu at (149.3, 126.8)
- added C60: 1u, Capacitor_SMD:C_0603_1608Metric, F.Cu at (86.5, 101.0)
- added C61: 1u, Capacitor_SMD:C_0603_1608Metric, F.Cu at (86.5, 103.6)
- added C62: 100n, Capacitor_SMD:C_0603_1608Metric, F.Cu at (86.5, 106.1)
- added C63: 100n, Capacitor_SMD:C_0603_1608Metric, F.Cu at (86.5, 108.6)
- added C64: 1u, Capacitor_SMD:C_0603_1608Metric, F.Cu at (86.5, 111.1)
- added C65: 1u, Capacitor_SMD:C_0603_1608Metric, F.Cu at (90.5, 91.0)
- added C66: 100n, Capacitor_SMD:C_0603_1608Metric, F.Cu at (90.5, 93.5)
- added C67: 22p, Capacitor_SMD:C_0603_1608Metric, F.Cu at (90.5, 96.0)
- added C68: 22p, Capacitor_SMD:C_0603_1608Metric, F.Cu at (90.5, 98.5)
- added C69: 100n, Capacitor_SMD:C_0603_1608Metric, F.Cu at (90.5, 101.0)
- added C7: 100n, Capacitor_SMD:C_0603_1608Metric, F.Cu at (149.3, 129.4)
- added C70: 10u, Capacitor_SMD:C_0603_1608Metric, F.Cu at (90.5, 103.6)
- added C71: 10u, Capacitor_SMD:C_0603_1608Metric, F.Cu at (90.5, 106.1)
- added C72: 100n, Capacitor_SMD:C_0603_1608Metric, F.Cu at (90.5, 108.6)
- added C73: 10u, Capacitor_SMD:C_0603_1608Metric, F.Cu at (110.9, 146.6)
- added C74: 1u, Capacitor_SMD:C_0603_1608Metric, F.Cu at (110.9, 149.1)
- added C75: 100n, Capacitor_SMD:C_0603_1608Metric, F.Cu at (110.9, 151.6)
- added C76: 100n, Capacitor_SMD:C_0603_1608Metric, F.Cu at (49.7, 31.1)
- added C77: 10u, Capacitor_SMD:C_0603_1608Metric, F.Cu at (49.7, 33.6)
- added C78: 10u, Capacitor_SMD:C_0603_1608Metric, F.Cu at (49.7, 36.2)
- added C79: 100n, Capacitor_SMD:C_0603_1608Metric, F.Cu at (49.7, 38.7)
- added C8: 100n, Capacitor_SMD:C_0603_1608Metric, F.Cu at (153.3, 114.3)
- added C80: 100n, Capacitor_SMD:C_0603_1608Metric, F.Cu at (49.7, 41.2)
- added C81: 10u, Capacitor_SMD:C_0603_1608Metric, F.Cu at (49.7, 43.7)
- added C82: 10u, Capacitor_SMD:C_0603_1608Metric, F.Cu at (49.7, 46.2)
- added C83: 100n, Capacitor_SMD:C_0603_1608Metric, F.Cu at (49.7, 48.7)
- added C84: 100n, Capacitor_SMD:C_0603_1608Metric, F.Cu at (31.7, 91.0)
- added C85: 10u, Capacitor_SMD:C_0603_1608Metric, F.Cu at (31.7, 93.5)
- added C86: 10u, Capacitor_SMD:C_0603_1608Metric, F.Cu at (31.7, 96.0)
- added C87: 100n, Capacitor_SMD:C_0603_1608Metric, F.Cu at (31.7, 98.5)
- added C88: 470u, Capacitor_THT:CP_Radial_D12.5mm_P5.00mm, F.Cu at (159.1, 175.9)
- added C89: 100u, Capacitor_THT:CP_Radial_D8.0mm_P3.50mm, F.Cu at (159.4, 144.2)
- added C9: 100n, Capacitor_SMD:C_0603_1608Metric, F.Cu at (153.3, 116.8)
- added C90: 100n, Capacitor_SMD:C_0603_1608Metric, F.Cu at (69.5, 161.3)
- added C91: 10u, Capacitor_SMD:C_0603_1608Metric, F.Cu at (69.5, 163.8)
- added C92: 10u, Capacitor_SMD:C_0603_1608Metric, F.Cu at (69.5, 166.3)
- added C93: 100n, Capacitor_SMD:C_0603_1608Metric, F.Cu at (69.5, 168.8)
- added C94: 100n, Capacitor_SMD:C_0603_1608Metric, F.Cu at (69.5, 171.3)
- added C95: 100n, Capacitor_SMD:C_0603_1608Metric, F.Cu at (69.5, 173.8)
- added C96: 100n, Capacitor_SMD:C_0603_1608Metric, F.Cu at (147.3, 19.3)
- added C97: 10u, Capacitor_SMD:C_0603_1608Metric, F.Cu at (147.3, 21.8)
- added C98: 10u, Capacitor_SMD:C_0603_1608Metric, F.Cu at (147.3, 24.3)
- added C99: 100n, Capacitor_SMD:C_0603_1608Metric, F.Cu at (147.3, 26.8)
- added D1: FYLS-0603BUGC, LED_SMD:LED_0603_1608Metric, F.Cu at (113.4, 62.5)
- added D10: PESD1CAN, Package_TO_SOT_SMD:SOT-23, F.Cu at (75.2, 139.9)
- added D11: FYLS-0603BUGC, LED_SMD:LED_0603_1608Metric, F.Cu at (118.6, 116.2)
- added D14: FYLS-0603BUGC, LED_SMD:LED_0603_1608Metric, F.Cu at (67.9, 81.6)
- added D15: FYLS-0603BUGC, LED_SMD:LED_0603_1608Metric, F.Cu at (67.9, 84.2)
- added D16: FYLS-0603BUGC, LED_SMD:LED_0603_1608Metric, F.Cu at (27.4, 142.3)
- added D17: FYLS-0603BUGC, LED_SMD:LED_0603_1608Metric, F.Cu at (161.8, 150.2)
- added D18: FYLS-0603BUGC, LED_SMD:LED_0603_1608Metric, F.Cu at (104.7, 155.8)
- added D19: FYLS-0603BUGC, LED_SMD:LED_0603_1608Metric, F.Cu at (175.9, 30.5)
- added D2: FYLS-0603BUGC, LED_SMD:LED_0603_1608Metric, F.Cu at (113.4, 65.1)
- added D20: FYLS-0603BUGC, LED_SMD:LED_0603_1608Metric, F.Cu at (175.9, 33.1)
- added D25: FYLS-0603BUGC, LED_SMD:LED_0603_1608Metric, F.Cu at (41.8, 169.8)
- added D26: FYLS-0603BUGC, LED_SMD:LED_0603_1608Metric, F.Cu at (41.8, 172.4)
- added D3: FYLS-0603BUGC, LED_SMD:LED_0603_1608Metric, F.Cu at (113.4, 67.7)
- added D4: ss24, Diode_SMD:D_SMB, F.Cu at (128.9, 62.7)
- added D5: ss24, Diode_SMD:D_SMB, F.Cu at (128.9, 68.3)
- added D6: FYLS-0603BUGC, LED_SMD:LED_0603_1608Metric, F.Cu at (113.4, 70.3)
- added D7: FYLS-0603BUGC, LED_SMD:LED_0603_1608Metric, F.Cu at (113.4, 72.9)
- added D8: PESD1CAN, Package_TO_SOT_SMD:SOT-23, F.Cu at (75.2, 135.2)
- added D9: FYLS-0603BUGC, LED_SMD:LED_0603_1608Metric, F.Cu at (118.6, 113.6)
- added F1: MF-LSMF300/24X-2, Fuse:Fuse_2920_7451Metric, F.Cu at (138.2, 73.0)
- added J1: PLS-6, Connector_PinHeader_2.54mm:PinHeader_1x06_P2.54mm_Vertical, F.Cu at (165.7, 115.4)
- added J2: BH1,27-10-G, Connector_PinHeader_1.27mm:PinHeader_2x05_P1.27mm_Vertical, F.Cu at (161.5, 102.1)
- added J20: 430451600, Connector_Molex:Molex_Micro-Fit_3.0_43045-1600_2x08_P3.00mm_Horizontal, F.Cu at (149.9, 67.9)
- added J22: USB_B_Micro, user_lib:U-F-M5DD-W-2-SUS, F.Cu at (31.3, 168.4)
- added J23: 430450415, Connector_Molex:Molex_Micro-Fit_3.0_43045-0415_2x02_P3.00mm_Vertical, F.Cu at (45.9, 155.0)
- added J24: PLS-5, Connector_PinHeader_2.54mm:PinHeader_1x05_P2.54mm_Vertical, F.Cu at (104.5, 127.9)
- added J25: PLS-5, Connector_PinHeader_2.54mm:PinHeader_1x05_P2.54mm_Vertical, F.Cu at (109.2, 127.9)
- added J26: PLS-3, Connector_PinHeader_2.54mm:PinHeader_1x03_P2.54mm_Vertical, F.Cu at (166.0, 92.1)
- added J3: PLS-3, Connector_PinHeader_2.54mm:PinHeader_1x03_P2.54mm_Vertical, F.Cu at (161.4, 92.1)
- added J4: 430450400, Connector_Molex:Molex_Micro-Fit_3.0_43045-0400_2x02_P3.00mm_Horizontal, F.Cu at (120.9, 48.1)
- added J5: 430450400, Connector_Molex:Molex_Micro-Fit_3.0_43045-0400_2x02_P3.00mm_Horizontal, F.Cu at (101.1, 99.7)
- added JP1: SolderJumper2, Jumper:SolderJumper-2_P1.3mm_Open_RoundedPad1.0x1.5mm, F.Cu at (154.7, 132.4)
- added L1: B82721-K2222-U30, user_lib:B82721-K2222-U30, F.Cu at (132.4, 25.3)
- added L4: 27n, Capacitor_SMD:C_0603_1608Metric, F.Cu at (151.4, 31.8)
- added Q10: BSS138, Package_TO_SOT_SMD:SOT-23, F.Cu at (50.1, 85.5)
- added Q11: BSS138, Package_TO_SOT_SMD:SOT-23, F.Cu at (55.0, 62.4)
- added Q12: BSS138, Package_TO_SOT_SMD:SOT-23, F.Cu at (55.0, 67.0)
- added Q13: BSS138, Package_TO_SOT_SMD:SOT-23, F.Cu at (55.0, 71.7)
- added Q14: BSS138, Package_TO_SOT_SMD:SOT-23, F.Cu at (55.0, 76.3)
- added Q15: BSS138, Package_TO_SOT_SMD:SOT-23, F.Cu at (55.0, 80.9)
- added Q16: BSS138, Package_TO_SOT_SMD:SOT-23, F.Cu at (55.0, 85.5)
- added Q17: BSS138, Package_TO_SOT_SMD:SOT-23, F.Cu at (59.9, 62.4)
- added Q18: BSS138, Package_TO_SOT_SMD:SOT-23, F.Cu at (59.9, 67.0)
- added Q19: BSS138, Package_TO_SOT_SMD:SOT-23, F.Cu at (59.9, 71.7)
- added Q2: AO3401A, Package_TO_SOT_SMD:SOT-23, F.Cu at (113.8, 45.1)
- added Q20: BSS138, Package_TO_SOT_SMD:SOT-23, F.Cu at (59.9, 76.3)
- added Q21: BSS138, Package_TO_SOT_SMD:SOT-23, F.Cu at (59.9, 80.9)
- added Q22: BSS138, Package_TO_SOT_SMD:SOT-23, F.Cu at (59.9, 85.5)
- added Q23: BSS138, Package_TO_SOT_SMD:SOT-23, F.Cu at (32.1, 117.3)
- added Q24: BSS138, Package_TO_SOT_SMD:SOT-23, F.Cu at (32.1, 121.9)
- added Q25: BSS138, Package_TO_SOT_SMD:SOT-23, F.Cu at (32.1, 126.5)
- added Q26: BSS138, Package_TO_SOT_SMD:SOT-23, F.Cu at (32.1, 131.1)
- added Q27: BSS138, Package_TO_SOT_SMD:SOT-23, F.Cu at (32.1, 135.8)
- added Q28: BSS138, Package_TO_SOT_SMD:SOT-23, F.Cu at (37.0, 117.3)
- added Q29: BSS138, Package_TO_SOT_SMD:SOT-23, F.Cu at (37.0, 121.9)
- added Q3: BSS138, Package_TO_SOT_SMD:SOT-23, F.Cu at (113.8, 49.8)
- added Q30: BSS138, Package_TO_SOT_SMD:SOT-23, F.Cu at (37.0, 126.5)
- added Q31: BSS138, Package_TO_SOT_SMD:SOT-23, F.Cu at (37.0, 131.1)
- added Q32: BSS138, Package_TO_SOT_SMD:SOT-23, F.Cu at (37.0, 135.8)
- added Q33: BSS138, Package_TO_SOT_SMD:SOT-23, F.Cu at (41.9, 117.3)
- added Q37: BSS138, Package_TO_SOT_SMD:SOT-23, F.Cu at (171.4, 27.0)
- added Q38: BSS138, Package_TO_SOT_SMD:SOT-23, F.Cu at (171.4, 31.6)
- added Q39: BSS138, Package_TO_SOT_SMD:SOT-23, F.Cu at (113.8, 59.0)
- added Q4: BSS138, Package_TO_SOT_SMD:SOT-23, F.Cu at (113.8, 54.4)
- added Q5: BSS138, Package_TO_SOT_SMD:SOT-23, F.Cu at (50.1, 62.4)
- added Q6: BSS138, Package_TO_SOT_SMD:SOT-23, F.Cu at (50.1, 67.0)
- added Q7: BSS138, Package_TO_SOT_SMD:SOT-23, F.Cu at (50.1, 71.7)
- added Q8: BSS138, Package_TO_SOT_SMD:SOT-23, F.Cu at (50.1, 76.3)
- added Q9: BSS138, Package_TO_SOT_SMD:SOT-23, F.Cu at (50.1, 80.9)
- added R100: 360k, Resistor_SMD:R_0603_1608Metric, F.Cu at (69.7, 48.7)
- added R101: 360, Resistor_SMD:R_0603_1608Metric, F.Cu at (69.7, 51.2)
- added R102: 10k, Resistor_SMD:R_0603_1608Metric, F.Cu at (69.7, 53.7)
- added R103: 360, Resistor_SMD:R_0603_1608Metric, F.Cu at (69.7, 56.2)
- added R104: 10k, Resistor_SMD:R_0603_1608Metric, F.Cu at (69.7, 58.7)
- added R105: 1M, Resistor_SMD:R_0603_1608Metric, F.Cu at (73.7, 31.1)
- added R106: 1M, Resistor_SMD:R_0603_1608Metric, F.Cu at (73.7, 33.6)
- added R107: 360k, Resistor_SMD:R_0603_1608Metric, F.Cu at (73.7, 36.2)
- added R108: 360k, Resistor_SMD:R_0603_1608Metric, F.Cu at (73.7, 38.7)
- added R109: 360, Resistor_SMD:R_0603_1608Metric, F.Cu at (73.7, 41.2)
- added R110: 10k, Resistor_SMD:R_0603_1608Metric, F.Cu at (73.7, 43.7)
- added R111: 360, Resistor_SMD:R_0603_1608Metric, F.Cu at (73.7, 46.2)
- added R112: 10k, Resistor_SMD:R_0603_1608Metric, F.Cu at (73.7, 48.7)
- added R113: 360, Resistor_SMD:R_0603_1608Metric, F.Cu at (73.7, 51.2)
- added R114: 360, Resistor_SMD:R_0603_1608Metric, F.Cu at (73.7, 53.7)
- added R115: 1M, Resistor_SMD:R_0603_1608Metric, F.Cu at (31.7, 101.0)
- added R116: 360k, Resistor_SMD:R_0603_1608Metric, F.Cu at (31.7, 103.6)
- added R117: 360, Resistor_SMD:R_0603_1608Metric, F.Cu at (31.7, 106.1)
- added R118: 10k, Resistor_SMD:R_0603_1608Metric, F.Cu at (31.7, 108.6)
- added R119: 1M, Resistor_SMD:R_0603_1608Metric, F.Cu at (31.7, 111.1)
- added R12: 100, Resistor_SMD:R_0603_1608Metric, F.Cu at (116.7, 19.3)
- added R120: 360k, Resistor_SMD:R_0603_1608Metric, F.Cu at (31.7, 113.6)
- added R121: 360, Resistor_SMD:R_0603_1608Metric, F.Cu at (35.7, 91.0)
- added R122: 10k, Resistor_SMD:R_0603_1608Metric, F.Cu at (35.7, 93.5)
- added R123: 1M, Resistor_SMD:R_0603_1608Metric, F.Cu at (35.7, 96.0)
- added R124: 360k, Resistor_SMD:R_0603_1608Metric, F.Cu at (35.7, 98.5)
- added R125: 360, Resistor_SMD:R_0603_1608Metric, F.Cu at (35.7, 101.0)
- added R126: 10k, Resistor_SMD:R_0603_1608Metric, F.Cu at (35.7, 103.6)
- added R127: 1M, Resistor_SMD:R_0603_1608Metric, F.Cu at (35.7, 106.1)
- added R128: 360k, Resistor_SMD:R_0603_1608Metric, F.Cu at (35.7, 108.6)
- added R129: 360, Resistor_SMD:R_0603_1608Metric, F.Cu at (35.7, 111.1)
- added R13: 130, Resistor_SMD:R_2512_6332Metric, F.Cu at (107.0, 40.6)
- added R130: 10k, Resistor_SMD:R_0603_1608Metric, F.Cu at (35.7, 113.6)
- added R131: 1M, Resistor_SMD:R_0603_1608Metric, F.Cu at (39.7, 91.0)
- added R132: 360k, Resistor_SMD:R_0603_1608Metric, F.Cu at (39.7, 93.5)
- added R133: 360, Resistor_SMD:R_0603_1608Metric, F.Cu at (39.7, 96.0)
- added R134: 360, Resistor_SMD:R_0603_1608Metric, F.Cu at (39.7, 98.5)
- added R135: 10k, Resistor_SMD:R_0603_1608Metric, F.Cu at (39.7, 101.0)
- added R136: 1M, Resistor_SMD:R_0603_1608Metric, F.Cu at (39.7, 103.6)
- added R137: 360k, Resistor_SMD:R_0603_1608Metric, F.Cu at (39.7, 106.1)
- added R138: 360, Resistor_SMD:R_0603_1608Metric, F.Cu at (39.7, 108.6)
- added R139: 10k, Resistor_SMD:R_0603_1608Metric, F.Cu at (39.7, 111.1)
- added R14: 130, Resistor_SMD:R_2512_6332Metric, F.Cu at (107.0, 45.4)
- added R140: 1M, Resistor_SMD:R_0603_1608Metric, F.Cu at (39.7, 113.6)
- added R141: 360k, Resistor_SMD:R_0603_1608Metric, F.Cu at (43.7, 91.0)
- added R142: 360, Resistor_SMD:R_0603_1608Metric, F.Cu at (43.7, 93.5)
- added R143: 10k, Resistor_SMD:R_0603_1608Metric, F.Cu at (43.7, 96.0)
- added R144: 1M, Resistor_SMD:R_0603_1608Metric, F.Cu at (43.7, 98.5)
- added R145: 360k, Resistor_SMD:R_0603_1608Metric, F.Cu at (43.7, 101.0)
- added R146: 360, Resistor_SMD:R_0603_1608Metric, F.Cu at (43.7, 103.6)
- added R147: 10k, Resistor_SMD:R_0603_1608Metric, F.Cu at (43.7, 106.1)
- added R148: 1M, Resistor_SMD:R_0603_1608Metric, F.Cu at (43.7, 108.6)
- added R149: 360k, Resistor_SMD:R_0603_1608Metric, F.Cu at (43.7, 111.1)
- added R15: 0m62, Resistor_SMD:R_2512_6332Metric, F.Cu at (107.0, 50.3)
- added R150: 360, Resistor_SMD:R_0603_1608Metric, F.Cu at (43.7, 113.6)
- added R151: 10k, Resistor_SMD:R_0603_1608Metric, F.Cu at (47.7, 91.0)
- added R152: 1M, Resistor_SMD:R_0603_1608Metric, F.Cu at (47.7, 93.5)
- added R153: 360k, Resistor_SMD:R_0603_1608Metric, F.Cu at (47.7, 96.0)
- added R154: 360, Resistor_SMD:R_0603_1608Metric, F.Cu at (47.7, 98.5)
- added R155: 10k, Resistor_SMD:R_0603_1608Metric, F.Cu at (47.7, 101.0)
- added R156: 1M, Resistor_SMD:R_0603_1608Metric, F.Cu at (47.7, 103.6)
- added R157: 360k, Resistor_SMD:R_0603_1608Metric, F.Cu at (47.7, 106.1)
- added R158: 360, Resistor_SMD:R_0603_1608Metric, F.Cu at (47.7, 108.6)
- added R159: 10k, Resistor_SMD:R_0603_1608Metric, F.Cu at (47.7, 111.1)
- added R16: 10k, Resistor_SMD:R_0603_1608Metric, F.Cu at (116.7, 21.8)
- added R160: 1M, Resistor_SMD:R_0603_1608Metric, F.Cu at (47.7, 113.6)
- added R161: 360k, Resistor_SMD:R_0603_1608Metric, F.Cu at (51.7, 91.0)
- added R162: 360, Resistor_SMD:R_0603_1608Metric, F.Cu at (51.7, 93.5)
- added R163: 10k, Resistor_SMD:R_0603_1608Metric, F.Cu at (51.7, 96.0)
- added R164: 1M, Resistor_SMD:R_0603_1608Metric, F.Cu at (51.7, 98.5)
- added R165: 360k, Resistor_SMD:R_0603_1608Metric, F.Cu at (51.7, 101.0)
- added R166: 360, Resistor_SMD:R_0603_1608Metric, F.Cu at (51.7, 103.6)
- added R167: 10k, Resistor_SMD:R_0603_1608Metric, F.Cu at (51.7, 106.1)
- added R168: 220, Resistor_SMD:R_0603_1608Metric, F.Cu at (125.0, 170.1)
- added R169: 220, Resistor_SMD:R_0603_1608Metric, F.Cu at (125.0, 172.6)
- added R17: 1k, Resistor_SMD:R_0603_1608Metric, F.Cu at (116.7, 24.3)
- added R170: 220, Resistor_SMD:R_0603_1608Metric, F.Cu at (125.0, 175.1)
- added R171: 220, Resistor_SMD:R_0603_1608Metric, F.Cu at (125.0, 177.6)
- added R172: 220, Resistor_SMD:R_0603_1608Metric, F.Cu at (125.0, 180.1)
- added R173: 220, Resistor_SMD:R_0603_1608Metric, F.Cu at (125.0, 182.6)
- added R174: 220, Resistor_SMD:R_0603_1608Metric, F.Cu at (129.0, 170.1)
- added R175: 220, Resistor_SMD:R_0603_1608Metric, F.Cu at (129.0, 172.6)
- added R176: 220, Resistor_SMD:R_0603_1608Metric, F.Cu at (129.0, 175.1)
- added R177: 220, Resistor_SMD:R_0603_1608Metric, F.Cu at (129.0, 177.6)
- added R178: 220, Resistor_SMD:R_0603_1608Metric, F.Cu at (129.0, 180.1)
- added R179: 220, Resistor_SMD:R_0603_1608Metric, F.Cu at (129.0, 182.6)
- added R18: 10k, Resistor_SMD:R_0603_1608Metric, F.Cu at (116.7, 26.8)
- added R180: 220, Resistor_SMD:R_0603_1608Metric, F.Cu at (133.0, 170.1)
- added R181: 220, Resistor_SMD:R_0603_1608Metric, F.Cu at (133.0, 172.6)
- added R182: 220, Resistor_SMD:R_0603_1608Metric, F.Cu at (133.0, 175.1)
- added R183: 220, Resistor_SMD:R_0603_1608Metric, F.Cu at (133.0, 177.6)
- added R184: 220, Resistor_SMD:R_0603_1608Metric, F.Cu at (133.0, 180.1)
- added R185: 220, Resistor_SMD:R_0603_1608Metric, F.Cu at (133.0, 182.6)
- added R186: 220, Resistor_SMD:R_0603_1608Metric, F.Cu at (137.0, 170.1)
- added R187: 220, Resistor_SMD:R_0603_1608Metric, F.Cu at (137.0, 172.6)
- added R188: 220, Resistor_SMD:R_0603_1608Metric, F.Cu at (137.0, 175.1)
- added R189: 470, Resistor_SMD:R_0603_1608Metric, F.Cu at (137.0, 177.6)
- added R19: 100, Resistor_SMD:R_0603_1608Metric, F.Cu at (116.7, 29.3)
- added R190: 360, Resistor_SMD:R_0603_1608Metric, F.Cu at (69.5, 176.3)
- added R191: 1M, Resistor_SMD:R_0603_1608Metric, F.Cu at (69.5, 178.8)
- added R192: 200k, Resistor_SMD:R_0603_1608Metric, F.Cu at (73.6, 161.3)
- added R193: 1M, Resistor_SMD:R_0603_1608Metric, F.Cu at (73.6, 163.8)
- added R194: 10k, Resistor_SMD:R_0603_1608Metric, F.Cu at (73.6, 166.3)
- added R195: 200k, Resistor_SMD:R_0603_1608Metric, F.Cu at (73.6, 168.8)
- added R196: 10k, Resistor_SMD:R_0603_1608Metric, F.Cu at (73.6, 171.3)
- added R197: 180, Resistor_SMD:R_0603_1608Metric, F.Cu at (73.6, 173.8)
- added R198: 10k, Resistor_SMD:R_0603_1608Metric, F.Cu at (73.6, 176.3)
- added R199: 1M, Resistor_SMD:R_0603_1608Metric, F.Cu at (73.6, 178.8)
- added R2: PWR_REG, Resistor_SMD:R_0603_1608Metric, F.Cu at (108.7, 34.3)
- added R20: 130, Resistor_SMD:R_2512_6332Metric, F.Cu at (107.0, 55.2)
- added R200: 200k, Resistor_SMD:R_0603_1608Metric, F.Cu at (77.6, 161.3)
- added R201: 180, Resistor_SMD:R_0603_1608Metric, F.Cu at (77.6, 163.8)
- added R202: 10k, Resistor_SMD:R_0603_1608Metric, F.Cu at (77.6, 166.3)
- added R203: 10k, Resistor_SMD:R_0603_1608Metric, F.Cu at (77.6, 168.8)
- added R204: 1M, Resistor_SMD:R_0603_1608Metric, F.Cu at (77.6, 171.3)
- added R207: 180, Resistor_SMD:R_0603_1608Metric, F.Cu at (77.6, 178.8)
- added R208: 10k, Resistor_SMD:R_0603_1608Metric, F.Cu at (81.6, 161.3)
- added R209: 1M, Resistor_SMD:R_0603_1608Metric, F.Cu at (81.6, 163.8)
- added R21: 130, Resistor_SMD:R_2512_6332Metric, F.Cu at (107.0, 60.1)
- added R210: 200k, Resistor_SMD:R_0603_1608Metric, F.Cu at (81.6, 166.3)
- added R211: 1M, Resistor_SMD:R_0603_1608Metric, F.Cu at (81.6, 168.8)
- added R212: 10k, Resistor_SMD:R_0603_1608Metric, F.Cu at (81.6, 171.3)
- added R213: 10k, Resistor_SMD:R_0603_1608Metric, F.Cu at (81.6, 173.8)
- added R214: 10k, Resistor_SMD:R_0603_1608Metric, F.Cu at (81.6, 176.3)
- added R215: 200k, Resistor_SMD:R_0603_1608Metric, F.Cu at (81.6, 178.8)
- added R216: 470, Resistor_SMD:R_0603_1608Metric, F.Cu at (85.6, 161.3)
- added R217: 1M, Resistor_SMD:R_0603_1608Metric, F.Cu at (85.6, 163.8)
- added R218: 200k, Resistor_SMD:R_0603_1608Metric, F.Cu at (85.6, 166.3)
- added R219: 1M, Resistor_SMD:R_0603_1608Metric, F.Cu at (85.6, 168.8)
- added R22: 10k, Resistor_SMD:R_0603_1608Metric, F.Cu at (116.7, 31.8)
- added R220: 200k, Resistor_SMD:R_0603_1608Metric, F.Cu at (85.6, 171.3)
- added R221: 360, Resistor_SMD:R_0603_1608Metric, F.Cu at (151.4, 34.3)
- added R222: 360, Resistor_SMD:R_0603_1608Metric, F.Cu at (155.4, 19.3)
- added R223: 10k, Resistor_SMD:R_0603_1608Metric, F.Cu at (155.4, 21.8)
- added R224: 10k, Resistor_SMD:R_0603_1608Metric, F.Cu at (155.4, 24.3)
- added R225: 180, Resistor_SMD:R_0603_1608Metric, F.Cu at (155.4, 26.8)
- added R226: 10k, Resistor_SMD:R_0603_1608Metric, F.Cu at (155.4, 29.3)
- added R227: 1k, Resistor_SMD:R_0603_1608Metric, F.Cu at (155.4, 31.8)
- added R228: 2k, Resistor_SMD:R_0603_1608Metric, F.Cu at (155.4, 34.3)
- added R23: 120, Resistor_SMD:R_0603_1608Metric, F.Cu at (116.7, 34.3)
- added R231: 10k, Resistor_SMD:R_0603_1608Metric, F.Cu at (159.4, 24.3)
- added R234: 180, Resistor_SMD:R_0603_1608Metric, F.Cu at (159.4, 31.8)
- added R235: 10k, Resistor_SMD:R_0603_1608Metric, F.Cu at (159.4, 34.3)
- added R236: 2k, Resistor_SMD:R_0603_1608Metric, F.Cu at (163.4, 19.3)
- added R237: 10k, Resistor_SMD:R_0603_1608Metric, F.Cu at (163.4, 21.8)
- added R238: 10k, Resistor_SMD:R_0603_1608Metric, F.Cu at (163.4, 24.3)
- added R239: 180, Resistor_SMD:R_0603_1608Metric, F.Cu at (163.4, 26.8)
- added R24: 470, Resistor_SMD:R_0603_1608Metric, F.Cu at (116.7, 36.9)
- added R240: 10k, Resistor_SMD:R_0603_1608Metric, F.Cu at (163.4, 29.3)
- added R241: 10k, Resistor_SMD:R_0603_1608Metric, F.Cu at (163.4, 31.8)
- added R242: 180, Resistor_SMD:R_0603_1608Metric, F.Cu at (163.4, 34.3)
- added R243: 390, Resistor_SMD:R_0603_1608Metric, F.Cu at (166.6, 73.9)
- added R244: 10k, Resistor_SMD:R_0603_1608Metric, F.Cu at (166.6, 76.5)
- added R245: 390, Resistor_SMD:R_0603_1608Metric, F.Cu at (166.6, 79.0)
- added R246: 10k, Resistor_SMD:R_0603_1608Metric, F.Cu at (166.6, 81.5)
- added R247: 390, Resistor_SMD:R_0603_1608Metric, F.Cu at (166.6, 84.0)
- added R248: 10k, Resistor_SMD:R_0603_1608Metric, F.Cu at (166.6, 86.5)
- added R249: 390, Resistor_SMD:R_0603_1608Metric, F.Cu at (170.7, 73.9)
- added R25: 390, Resistor_SMD:R_0603_1608Metric, F.Cu at (120.7, 19.3)
- added R250: 10k, Resistor_SMD:R_0603_1608Metric, F.Cu at (170.7, 76.5)
- added R26: 470, Resistor_SMD:R_0603_1608Metric, F.Cu at (120.7, 21.8)
- added R27: 120, Resistor_SMD:R_0603_1608Metric, F.Cu at (90.5, 111.1)
- added R271: 220, Resistor_SMD:R_0603_1608Metric, F.Cu at (20.5, 166.8)
- added R272: 220, Resistor_SMD:R_0603_1608Metric, F.Cu at (24.5, 149.2)
- added R273: 220, Resistor_SMD:R_0603_1608Metric, F.Cu at (24.5, 151.7)
- added R274: 220, Resistor_SMD:R_0603_1608Metric, F.Cu at (24.5, 154.2)
- added R275: 220, Resistor_SMD:R_0603_1608Metric, F.Cu at (24.5, 156.7)
- added R276: 220, Resistor_SMD:R_0603_1608Metric, F.Cu at (24.5, 159.3)
- added R277: 10k, Resistor_SMD:R_0603_1608Metric, F.Cu at (24.5, 161.8)
- added R278: 10k, Resistor_SMD:R_0603_1608Metric, F.Cu at (24.5, 164.3)
- added R279: 10k, Resistor_SMD:R_0603_1608Metric, F.Cu at (58.0, 149.2)
- added R28: 0, Resistor_SMD:R_0603_1608Metric, F.Cu at (94.5, 91.0)
- added R280: 10k, Resistor_SMD:R_0603_1608Metric, F.Cu at (58.0, 151.7)
- added R281: 220, Resistor_SMD:R_0603_1608Metric, F.Cu at (58.0, 154.2)
- added R282: 470, Resistor_SMD:R_0603_1608Metric, F.Cu at (58.0, 156.7)
- added R283: 360, Resistor_SMD:R_0603_1608Metric, F.Cu at (58.0, 159.3)
- added R284: 1M, Resistor_SMD:R_0603_1608Metric, F.Cu at (120.7, 24.3)
- added R285: 1M, Resistor_SMD:R_0603_1608Metric, F.Cu at (120.7, 26.8)
- added R286: 1M, Resistor_SMD:R_0603_1608Metric, F.Cu at (120.7, 29.3)
- added R287: 1M, Resistor_SMD:R_0603_1608Metric, F.Cu at (120.7, 31.8)
- added R29: 10k, Resistor_SMD:R_0603_1608Metric, F.Cu at (94.5, 93.5)
- added R3: PWR_REG, Resistor_SMD:R_0603_1608Metric, F.Cu at (108.7, 36.9)
- added R30: 360, Resistor_SMD:R_0603_1608Metric, F.Cu at (94.5, 96.0)
- added R31: 120, Resistor_SMD:R_0603_1608Metric, F.Cu at (94.5, 98.5)
- added R32: 0, Resistor_SMD:R_0603_1608Metric, F.Cu at (94.5, 101.0)
- added R33: 10k, Resistor_SMD:R_0603_1608Metric, F.Cu at (94.5, 103.6)
- added R34: 360, Resistor_SMD:R_0603_1608Metric, F.Cu at (94.5, 106.1)
- added R4: 360, Resistor_SMD:R_0603_1608Metric, F.Cu at (112.7, 19.3)
- added R41: 1M, Resistor_SMD:R_0603_1608Metric, F.Cu at (49.7, 51.2)
- added R42: 1M, Resistor_SMD:R_0603_1608Metric, F.Cu at (49.7, 53.7)
- added R43: 360k, Resistor_SMD:R_0603_1608Metric, F.Cu at (49.7, 56.2)
- added R44: 360k, Resistor_SMD:R_0603_1608Metric, F.Cu at (49.7, 58.7)
- added R45: 360, Resistor_SMD:R_0603_1608Metric, F.Cu at (53.7, 31.1)
- added R46: 10k, Resistor_SMD:R_0603_1608Metric, F.Cu at (53.7, 33.6)
- added R47: 360, Resistor_SMD:R_0603_1608Metric, F.Cu at (53.7, 36.2)
- added R48: 10k, Resistor_SMD:R_0603_1608Metric, F.Cu at (53.7, 38.7)
- added R49: 1M, Resistor_SMD:R_0603_1608Metric, F.Cu at (53.7, 41.2)
- added R5: 220, Resistor_SMD:R_0603_1608Metric, F.Cu at (112.7, 21.8)
- added R50: 1M, Resistor_SMD:R_0603_1608Metric, F.Cu at (53.7, 43.7)
- added R51: 360k, Resistor_SMD:R_0603_1608Metric, F.Cu at (53.7, 46.2)
- added R52: 360k, Resistor_SMD:R_0603_1608Metric, F.Cu at (53.7, 48.7)
- added R53: 360, Resistor_SMD:R_0603_1608Metric, F.Cu at (53.7, 51.2)
- added R54: 10k, Resistor_SMD:R_0603_1608Metric, F.Cu at (53.7, 53.7)
- added R55: 360, Resistor_SMD:R_0603_1608Metric, F.Cu at (53.7, 56.2)
- added R56: 10k, Resistor_SMD:R_0603_1608Metric, F.Cu at (53.7, 58.7)
- added R57: 1M, Resistor_SMD:R_0603_1608Metric, F.Cu at (57.7, 31.1)
- added R58: 1M, Resistor_SMD:R_0603_1608Metric, F.Cu at (57.7, 33.6)
- added R59: 360k, Resistor_SMD:R_0603_1608Metric, F.Cu at (57.7, 36.2)
- added R6: 470, Resistor_SMD:R_0603_1608Metric, F.Cu at (112.7, 24.3)
- added R60: 360k, Resistor_SMD:R_0603_1608Metric, F.Cu at (57.7, 38.7)
- added R61: 360, Resistor_SMD:R_0603_1608Metric, F.Cu at (57.7, 41.2)
- added R62: 10k, Resistor_SMD:R_0603_1608Metric, F.Cu at (57.7, 43.7)
- added R63: 360, Resistor_SMD:R_0603_1608Metric, F.Cu at (57.7, 46.2)
- added R64: 10k, Resistor_SMD:R_0603_1608Metric, F.Cu at (57.7, 48.7)
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Connections:
- C110 pad 1: Net-(J19-VBUS) -> Net-(J22-VBUS)
- J10 pad 1: /Switches_2/SWITCH_3.6_EXT -> /Switches_1/SWITCH_2.1_EXT
- J10 pad 3: /Switches_2/SWITCH_3.7_EXT -> /Switches_1/SWITCH_2.2_EXT
- J10 pad 5: /Switches_2/SWITCH_3.8_EXT -> /Switches_1/SWITCH_2.3_EXT
- J11 pad 1: /Switches_2/SWITCH_4.1_EXT -> /Switches_2/SWITCH_3.1_EXT
- J11 pad 3: /Switches_2/SWITCH_4.2_EXT -> /Switches_2/SWITCH_3.2_EXT
- J11 pad 5: /Switches_2/SWITCH_4.3_EXT -> /Switches_2/SWITCH_3.3_EXT
- J12 pad 1: /LED_indicators/LED19_EXT_12V -> /Switches_2/SWITCH_3.6_EXT
- J12 pad 2: 12V0_LED -> VIN
- J12 pad 3: /LED_indicators/LED20_EXT_12V -> /Switches_2/SWITCH_3.7_EXT
- J12 pad 4: 12V0_LED -> VIN
- J12 pad 5: /LED_indicators/LED21_EXT_12V -> /Switches_2/SWITCH_3.8_EXT
- J12 pad 6: 12V0_LED -> VIN
- J13 pad 1: /LED_indicators/LED1_EXT_12V -> /Switches_2/SWITCH_3.9_EXT
- J13 pad 2: 12V0_LED -> VIN
- J13 pad 3: /LED_indicators/LED2_EXT_12V -> /Switches_2/SWITCH_3.10_EXT
- J13 pad 4: 12V0_LED -> VIN
- J14 pad 1: /LED_indicators/LED10_EXT_12V -> /Switches_2/SWITCH_4.1_EXT
- J14 pad 2: 12V0_LED -> VIN
- J14 pad 3: /LED_indicators/LED11_EXT_12V -> /Switches_2/SWITCH_4.2_EXT
- J14 pad 4: 12V0_LED -> VIN
- J14 pad 5: /LED_indicators/LED12_EXT_12V -> /Switches_2/SWITCH_4.3_EXT
- J14 pad 6: 12V0_LED -> VIN
- J15 pad 1: /ADC8/ADC_30V_IN_1 -> /LED_indicators/LED19_EXT_12V
- J15 pad 2: GND_ADC -> 12V0_LED
- J15 pad 3: /ADC8/ADC_30V_IN_3 -> /LED_indicators/LED20_EXT_12V
- J15 pad 4: GND_ADC -> 12V0_LED
- J15 pad 5: /ADC8/ADC_30V_IN_2 -> /LED_indicators/LED21_EXT_12V
- J15 pad 6: GND_ADC -> 12V0_LED
- J16 pad 1: 5V0_ADC_RUD -> /LED_indicators/LED1_EXT_12V
- J16 pad 2: 5V0_ADC_RUD -> 12V0_LED
- J16 pad 3: /ADC_RUD/ADC_RUD_5V_1 -> /LED_indicators/LED2_EXT_12V
- J16 pad 4: /ADC_RUD/ADC_RUD_5V_2 -> 12V0_LED
- J16 pad 5: GND_ADC_RUD -> /LED_indicators/LED3_EXT_12V
- J16 pad 6: GND_ADC_RUD -> 12V0_LED
- J17 pad 1: /Digital inputs 5V/INPUT_1_POS -> /LED_indicators/LED10_EXT_12V
- J17 pad 10: /Digital inputs 5V/INPUT_5_NEG -> 12V0_LED
- J17 pad 11: /Digital inputs 5V/INPUT_6_POS -> /LED_indicators/LED15_EXT_12V
- J17 pad 12: /Digital inputs 5V/INPUT_6_NEG -> 12V0_LED
- J17 pad 13: /Digital inputs 5V/INPUT_7_POS -> /LED_indicators/LED16_EXT_12V
- J17 pad 14: /Digital inputs 5V/INPUT_7_NEG -> 12V0_LED
- J17 pad 15: /Digital inputs 5V/INPUT_8_POS -> /LED_indicators/LED17_EXT_12V
- J17 pad 16: /Digital inputs 5V/INPUT_8_NEG -> 12V0_LED
- J17 pad 2: /Digital inputs 5V/INPUT_1_NEG -> 12V0_LED
- J17 pad 3: /Digital inputs 5V/INPUT_2_POS -> /LED_indicators/LED11_EXT_12V
- J17 pad 4: /Digital inputs 5V/INPUT_2_NEG -> 12V0_LED
- J17 pad 5: /Digital inputs 5V/INPUT_3_POS -> /LED_indicators/LED12_EXT_12V
- J17 pad 6: /Digital inputs 5V/INPUT_3_NEG -> 12V0_LED
- J17 pad 7: /Digital inputs 5V/INPUT_4_POS -> /LED_indicators/LED13_EXT_12V
- J17 pad 8: /Digital inputs 5V/INPUT_4_NEG -> 12V0_LED
- J17 pad 9: /Digital inputs 5V/INPUT_5_POS -> /LED_indicators/LED14_EXT_12V
- J18 pad 1: SDIO_DAT2 -> /ADC8/ADC_30V_IN_1
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
Commit message: bugfixes
Parts:
- added F2: MF-LSMF300/24X-2, Fuse:Fuse_2920_7451Metric, F.Cu at (174.6, 123.5)
- added J27: PLS-6, Connector_PinHeader_2.54mm:PinHeader_1x06_P2.54mm_Vertical, F.Cu at (136.7, 171.4)
- added J28: 430450800, Connector_Molex:Molex_Micro-Fit_3.0_43045-0800_2x04_P3.00mm_Horizontal, F.Cu at (174.1, 113.2)
- added J29: PLS-8, Connector_PinHeader_2.54mm:PinHeader_1x08_P2.54mm_Vertical, F.Cu at (59.0, 91.1)
- added R288: 220, Resistor_SMD:R_0603_1608Metric, F.Cu at (148.4, 145.4)
- added R289: 10k, Resistor_SMD:R_0603_1608Metric, F.Cu at (73.3, 120.8)
- added R290: 10k, Resistor_SMD:R_0603_1608Metric, F.Cu at (73.3, 123.3)
- added R291: 10k, Resistor_SMD:R_0603_1608Metric, F.Cu at (73.3, 125.8)
- added SW6: B3F1060, Button_Switch_THT:SW_PUSH_6mm_H5mm, F.Cu at (22.3, 99.3)
- added SW7: B3F1060, Button_Switch_THT:SW_PUSH_6mm_H5mm, F.Cu at (22.3, 107.9)
- added SW8: B3F1060, Button_Switch_THT:SW_PUSH_6mm_H5mm, F.Cu at (22.3, 116.4)
- added SW9: B3F1060, Button_Switch_THT:SW_PUSH_6mm_H5mm, F.Cu at (22.3, 125.0)
- added TP39: TestPoint, TestPoint:TestPoint_THTPad_D1.5mm_Drill0.7mm, F.Cu at (126.1, 46.0)
- added TP40: TestPoint, TestPoint:TestPoint_THTPad_D1.5mm_Drill0.7mm, F.Cu at (129.6, 38.9)
- added TP41: TestPoint, TestPoint:TestPoint_THTPad_D1.5mm_Drill0.7mm, F.Cu at (129.6, 42.4)
- added TP42: TestPoint, TestPoint:TestPoint_THTPad_D1.5mm_Drill0.7mm, F.Cu at (129.6, 46.0)
- added TP43: TestPoint, TestPoint:TestPoint_THTPad_D1.5mm_Drill0.7mm, F.Cu at (133.2, 38.9)
- added TP44: TestPoint, TestPoint:TestPoint_THTPad_D1.5mm_Drill0.7mm, F.Cu at (133.2, 42.4)
- added TP45: TestPoint, TestPoint:TestPoint_THTPad_D1.5mm_Drill0.7mm, F.Cu at (133.2, 46.0)
- added TP46: TestPoint, TestPoint:TestPoint_THTPad_D1.5mm_Drill0.7mm, F.Cu at (67.8, 97.6)
- added TP47: TestPoint, TestPoint:TestPoint_THTPad_D1.5mm_Drill0.7mm, F.Cu at (67.8, 101.2)
- D4, D5: value ss24 -> ss54; footprint Diode_SMD:D_SMB -> Diode_SMD:D_SMC
- R221: value 360 -> 10k
- moved R264 153.5 mm to (172.9, 130.4)
- moved R265 153.5 mm to (172.9, 132.9)
- moved R266 153.5 mm to (172.9, 135.4)
- moved R267 153.5 mm to (172.9, 137.9)
- moved R268 153.5 mm to (172.9, 140.4)
- moved R269 153.5 mm to (172.9, 142.9)
- moved R270 153.5 mm to (172.9, 145.4)
- moved R271 153.5 mm to (172.9, 148.0)
- moved R272 153.5 mm to (176.9, 130.4)
- moved R273 153.5 mm to (176.9, 132.9)
- moved R274 153.5 mm to (176.9, 135.4)
- moved R275 153.5 mm to (176.9, 137.9)
- moved R276 153.5 mm to (176.9, 140.4)
- moved R277 153.5 mm to (176.9, 142.9)
- moved R278 153.5 mm to (176.9, 145.4)
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Connections:
- net SPI0_RPi_MOSI renamed SPI1_RPi_MOSI
- C73 pad 2: 5V0 -> Net-(C73-Pad2)
- C74 pad 2: 5V0 -> Net-(C73-Pad2)
- C75 pad 2: 5V0 -> Net-(C73-Pad2)
- J3 pad 1: UART1_STM32_RX -> UART1_STM32_TX
- J3 pad 2: UART1_STM32_TX -> UART1_STM32_RX
- R221 pad 1: Net-(D19-A) -> /BUTTON_1
- R221 pad 2: ADC_RUD_INT -> 3V3
- TP10 pad 1: 5V0 -> 7V4
- TP11 pad 1: 3V3 -> 5V0

Commit message: Updated packeges
Parts:
- removed BT1: KLS5-CR2032-01, user_lib:KLS5-CR2032-01
- removed C100: 1u, Capacitor_SMD:C_0603_1608Metric
- removed C101, C103: 100n, Capacitor_SMD:C_0603_1608Metric
- removed C102: 4u7, Capacitor_SMD:C_0603_1608Metric
- removed C26: 10u, Capacitor_THT:CP_Radial_D10.0mm_P5.00mm
- removed C33, C34, C35, C36: 330p, Capacitor_SMD:C_1206_3216Metric
- removed D19: FYLS-0603BUGC, LED_SMD:LED_0603_1608Metric
- removed J13, J4, J5, J6: 430450400, Connector_Molex:Molex_Micro-Fit_3.0_43045-0400_2x02_P3.00mm_Horizontal
- removed R227, R232: 1k, Resistor_SMD:R_0603_1608Metric
- removed R228, R236: 2k, Resistor_SMD:R_0603_1608Metric
- removed R288: 220, Resistor_SMD:R_0603_1608Metric
- removed TP31, TP32: TestPoint, TestPoint:TestPoint_THTPad_D1.5mm_Drill0.7mm
- removed U64: LDL1117S33R, Package_TO_SOT_SMD:SOT-223-3_TabPin2
- added C121: 10u, Capacitor_THT:CP_Radial_D10.0mm_P5.00mm, F.Cu at (70.1, 81.7)
- added H1: M4, MountingHole:MountingHole_4.3mm_M4_Pad_Via, F.Cu at (35.1, 153.6)
- added H10: M4, MountingHole:MountingHole_4.3mm_M4_Pad_Via, F.Cu at (133.2, 181.9)
- added H11: M4, MountingHole:MountingHole_4.3mm_M4_Pad_Via, F.Cu at (133.2, 192.0)
- added H2: M4, MountingHole:MountingHole_4.3mm_M4_Pad_Via, F.Cu at (35.1, 163.7)
- added H3: M4, MountingHole:MountingHole_4.3mm_M4_Pad_Via, F.Cu at (35.1, 173.9)
- added H4: M4, MountingHole:MountingHole_4.3mm_M4_Pad_Via, F.Cu at (35.1, 184.0)
- added H5: M2.5, MountingHole:MountingHole_2.7mm_M2.5_Pad_Via, F.Cu at (352.6, 37.8)
- added H6: M2.5, MountingHole:MountingHole_2.7mm_M2.5_Pad_Via, F.Cu at (310.0, 36.9)
- added H7: M2.5, MountingHole:MountingHole_2.7mm_M2.5_Pad_Via, F.Cu at (315.5, 99.7)
- added H8: M2.5, MountingHole:MountingHole_2.7mm_M2.5_Pad_Via, F.Cu at (352.5, 97.5)
- added H9: M4, MountingHole:MountingHole_4.3mm_M4_Pad_Via, F.Cu at (133.2, 171.7)
- added J30: PLS-2, Connector_PinHeader_2.54mm:PinHeader_1x02_P2.54mm_Vertical, F.Cu at (21.8, 85.1)
- added J31: PLS-2, Connector_PinHeader_2.54mm:PinHeader_1x02_P2.54mm_Vertical, F.Cu at (26.5, 85.1)
- added J7: Raspberry Pi 4, Connector_PinHeader_2.54mm:PinHeader_2x20_P2.54mm_Vertical, B.Cu at (352.0, 92.0)
- added K1: 1-1415899-9, user_lib:1-1415899-9, F.Cu at (90.7, 16.8)
- added K2: 1-1415899-9, user_lib:1-1415899-9, F.Cu at (90.7, 30.8)
- added K3: 1-1415899-9, user_lib:1-1415899-9, F.Cu at (90.7, 44.7)
- added U10: HY2213-BB3A, Package_TO_SOT_SMD:SOT-23-6, F.Cu at (55.6, 87.3)
- added U4: VDRI15W12, user_lib:VDRI25, F.Cu at (36.3, 24.6)
- added U6: HY2213-BB3A, Package_TO_SOT_SMD:SOT-23-6, F.Cu at (55.6, 82.6)
- added U7: VDRI25W05, user_lib:VDRI25, F.Cu at (36.3, 46.6)
- F1, F2: footprint Fuse:Fuse_2920_7451Metric -> user_lib:Fuse_2920_7451Metric
- J10, J16, J17, J8, J9: footprint Connector_Molex:Molex_Micro-Fit_3.0_43045-1800_2x09_P3.00mm_Horizontal -> user_lib:430451800
- J11: footprint Connector_Molex:Molex_Micro-Fit_3.0_43045-1000_2x05_P3.00mm_Horizontal -> user_lib:430451000
- J12, J14, J15, J19: footprint Connector_Molex:Molex_Micro-Fit_3.0_43045-0600_2x03_P3.00mm_Horizontal -> user_lib:430450600
- J18, J20: footprint Connector_Molex:Molex_Micro-Fit_3.0_43045-1600_2x08_P3.00mm_Horizontal -> user_lib:430451600
- J23: footprint Connector_Molex:Molex_Micro-Fit_3.0_43045-0415_2x02_P3.00mm_Vertical -> user_lib:430450415
- J28: footprint Connector_Molex:Molex_Micro-Fit_3.0_43045-0800_2x04_P3.00mm_Horizontal -> user_lib:430450800
- R239, R242: value 180 -> 360
- U11, U12, U15, U16: footprint Package_SO:SOP-8_6.62x9.15mm_P2.54mm -> user_lib:ISO1050DUB
- U23, U24, U30, U31, U32, U33, U34: footprint Package_SO:SOIC-4_4.55x2.6mm_P1.27mm -> user_lib:TLP291
- U73: footprint Package_SO:SOIC-8_5.23x5.23mm_P1.27mm -> user_lib:SOIC-8_5.23x5.23mm_P1.27mm
- U9: footprint Package_TO_SOT_THT:TO-220-3_Vertical -> user_lib:TO-220-3_Vertical_radiator
- moved R245 149.7 mm to (183.0, 187.6)
- moved R251 149.7 mm to (187.0, 187.6)
- moved R257 149.7 mm to (191.0, 187.6)
- moved J20 149.7 mm to (166.3, 176.6)
- moved R243 149.7 mm to (183.0, 182.6)
- moved R244 149.7 mm to (183.0, 185.1)
- moved R246 149.7 mm to (183.0, 190.1)
- moved R247 149.7 mm to (183.0, 192.6)
- moved R249 149.7 mm to (187.0, 182.6)
- moved R250 149.7 mm to (187.0, 185.1)
- moved R252 149.7 mm to (187.0, 190.1)
- moved R253 149.7 mm to (187.0, 192.6)
- moved R255 149.7 mm to (191.0, 182.6)
- moved R256 149.7 mm to (191.0, 185.1)
- moved R258 149.7 mm to (191.0, 190.1)
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Connections:
- C96 pad 1: 5V0_ADC_RUD -> ADC_RUD_INT
- C97 pad 1: 5V0_ADC_RUD -> ADC_RUD_INT
- J19 pad 1: 5V0_ADC_RUD -> ADC_RUD_INT
- J19 pad 2: 5V0_ADC_RUD -> ADC_RUD_INT
- R222 pad 2: 5V0_ADC_RUD -> ADC_RUD_INT
- R223 pad 1: 5V0_ADC_RUD -> ADC_RUD_INT
- R224 pad 2: 5V0_ADC_RUD -> ADC_RUD_INT
- R231 pad 1: 5V0_ADC_RUD -> ADC_RUD_INT
- R233 pad 2: 5V0_ADC_RUD -> ADC_RUD_INT
- R239 pad 1: ADC_RUD_INT -> Net-(U70-A1)
- R239 pad 2: Net-(U70-A1) -> ADC_RUD_INT
- R242 pad 1: ADC_RUD_INT -> Net-(U70-A2)
- R242 pad 2: Net-(U70-A2) -> ADC_RUD_INT
- TP29 pad 1: 5V0_ADC_RUD -> ADC_RUD_INT
- U65 pad 8: 5V0_ADC_RUD -> ADC_RUD_INT
- U66 pad 8: 5V0_ADC_RUD -> ADC_RUD_INT
- U67 pad 8: 5V0_ADC_RUD -> ADC_RUD_INT
- U68 pad 10: /ADC_RUD/ADC_RUD_3V3_2 -> /ADC_RUD/ADC_RUD_5V_2
- U68 pad 11: /ADC_RUD/ADC_RUD_3V3_1 -> /ADC_RUD/ADC_RUD_5V_1
- U69 pad 1: /ADC_RUD/ADC_RUD_3V3_1 -> /ADC_RUD/ADC_RUD_5V_1
- U69 pad 3: /ADC_RUD/ADC_RUD_3V3_2 -> /ADC_RUD/ADC_RUD_5V_2
