File: Hardware/ciam/impeller18/impeller18.kicad_pcb (KiCad board)
At the start: 2 copper layers, 617 parts, among them J1 PLS-6, J10 430451800, J11 430451000, J12 430450600, J14 430450600, J15 430450600, J16 430451800, J17 430451800, J18 430451600, J19 430450600, J2 BH1,27-10-G, J20 430451600, J22 USB_B_Micro, J23 430450415, J24 PLS-5, J25 PLS-5, J26 PLS-3, J27 PLS-6, J28 430450800, J29 PLS-8, J3 PLS-3, J30 PLS-2, J31 PLS-2, J7 Raspberry Pi 4, J8 430451800, J9 430451800, K1 1-1415899-9, K2 1-1415899-9, K3 1-1415899-9, Q1 BSS138, Q10 BSS138, Q11 BSS138, Q12 BSS138, Q13 BSS138, Q14 BSS138, Q15 BSS138, Q16 BSS138, Q17 BSS138, Q18 BSS138, Q19 BSS138, Q2 AO3401A, Q20 BSS138, Q21 BSS138, Q22 BSS138, Q23 BSS138, Q24 BSS138, Q25 BSS138, Q26 BSS138, Q27 BSS138, Q28 BSS138, Q29 BSS138, Q3 BSS138, Q30 BSS138, Q31 BSS138, Q32 BSS138, Q33 BSS138, Q34 BSS138, Q35 BSS138, Q36 BSS138, Q37 BSS138, Q38 BSS138, Q39 BSS138, Q4 BSS138, Q5 BSS138, Q6 BSS138, Q7 BSS138, Q8 BSS138, Q9 BSS138, SW1 B3F1060, SW2 MSS-12D16, SW3 MSS-12D16, SW4 MSS-12D16, SW5 MSS-12D16, SW6 B3F1060, SW7 B3F1060, SW8 B3F1060, SW9 B3F1060, U1 STM32F427ZGTx, U10 HY2213-BB3A, U11 ISO1050DUB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

Commit message: Updated packeges
Parts:
- removed C121: 10u, Capacitor_THT:CP_Radial_D10.0mm_P5.00mm
- removed C27: 47u, Capacitor_THT:CP_Radial_D12.5mm_P5.00mm
- removed C28, C39: 470u, Capacitor_THT:CP_Radial_D12.5mm_P5.00mm
- removed C37: 22u, Capacitor_THT:CP_Radial_D6.3mm_P2.50mm
- removed C38: 4u7, Capacitor_SMD:C_1210_3225Metric
- removed C40: 100u, Capacitor_THT:CP_Radial_D8.0mm_P3.50mm
- removed L1: B82721-K2222-U30, user_lib:B82721-K2222-U30
- added BT2: Battery_Cell, user_lib:bat_18350, F.Cu at (44.2, 26.7)
- added BT3: Battery_Cell, user_lib:bat_18350, F.Cu at (44.2, 49.7)
- added C100: 10u, Capacitor_THT:CP_Radial_D10.0mm_P5.00mm, F.Cu at (83.1, 90.1)
- added C101: 4u7, Capacitor_SMD:C_1210_3225Metric, F.Cu at (94.2, 83.5)
- added C102: 10u, Capacitor_SMD:C_1210_3225Metric, F.Cu at (94.2, 87.7)
- added C103: 47u, Capacitor_THT:CP_Radial_D12.5mm_P5.00mm, F.Cu at (50.6, 82.3)
- added C122: 47u, Capacitor_THT:CP_Radial_D12.5mm_P5.00mm, F.Cu at (50.6, 96.4)
- added C123: 4u7, Capacitor_SMD:C_1210_3225Metric, F.Cu at (94.2, 92.0)
- added C124: 4u7, Capacitor_SMD:C_1210_3225Metric, F.Cu at (99.9, 83.5)
- added C125: 10u, Capacitor_SMD:C_1210_3225Metric, F.Cu at (99.9, 87.7)
- added C126: 10u, Capacitor_SMD:C_1210_3225Metric, F.Cu at (99.9, 92.0)
- added C127: 10u, Capacitor_SMD:C_1210_3225Metric, F.Cu at (105.5, 83.5)
- added C128: 10u, Capacitor_SMD:C_1210_3225Metric, F.Cu at (105.5, 87.7)
- added C129: 10u, Capacitor_SMD:C_1210_3225Metric, F.Cu at (105.5, 92.0)
- added C130: 4u7, Capacitor_SMD:C_1210_3225Metric, F.Cu at (111.2, 83.5)
- added C131: 4u7, Capacitor_SMD:C_1210_3225Metric, F.Cu at (111.2, 87.7)
- added C132: 4u7, Capacitor_SMD:C_1210_3225Metric, F.Cu at (111.2, 92.0)
- added C133: 4700p, Capacitor_SMD:C_1206_3216Metric, F.Cu at (109.2, 36.7)
- added C134: 4700p, Capacitor_SMD:C_1206_3216Metric, F.Cu at (109.2, 40.1)
- added C26: 4700p, Capacitor_SMD:C_1206_3216Metric, F.Cu at (109.2, 30.0)
- added C33: 4700p, Capacitor_SMD:C_1206_3216Metric, F.Cu at (109.2, 33.4)
- added C34: 47u, Capacitor_THT:CP_Radial_D12.5mm_P5.00mm, F.Cu at (50.6, 68.3)
- added C35: 68u, Capacitor_THT:CP_Radial_D10.0mm_P5.00mm, F.Cu at (83.1, 67.0)
- added C36: 10u, Capacitor_THT:CP_Radial_D10.0mm_P5.00mm, F.Cu at (83.1, 78.6)
- added H12: M4, MountingHole:MountingHole_4.3mm_M4_Pad_Via, F.Cu at (193.5, 50.7)
- added J21: TF-01, sd:TF01A-NEW, F.Cu at (195.8, 74.6)
- added L2: B82790C0513N201, user_lib:B82790C0513N201, F.Cu at (179.6, 145.6)
- added L3: B82790C0513N201, user_lib:B82790C0513N201, F.Cu at (179.6, 153.1)
- added L5: B82721-K2222-U30, user_lib:B82721-K2222-U30, F.Cu at (69.8, 68.5)
- added L6: B82721-K2222-U30, user_lib:B82721-K2222-U30, F.Cu at (69.8, 82.9)
- added R227: PWR_REG, Resistor_SMD:R_0603_1608Metric, F.Cu at (105.4, 77.6)
- added R228: PWR_REG, Resistor_SMD:R_0603_1608Metric, F.Cu at (105.4, 80.1)
- added R232: PWR_REG, Resistor_SMD:R_0603_1608Metric, F.Cu at (109.4, 62.5)
- added R236: PWR_REG, Resistor_SMD:R_0603_1608Metric, F.Cu at (109.4, 65.0)
- added R288: 10k, Resistor_SMD:R_0603_1608Metric, F.Cu at (176.1, 48.4)
- added R292: 10k, Resistor_SMD:R_0603_1608Metric, F.Cu at (176.1, 50.9)
- added R293: 10k, Resistor_SMD:R_0603_1608Metric, F.Cu at (176.1, 53.4)
- added R294: 10k, Resistor_SMD:R_0603_1608Metric, F.Cu at (176.1, 55.9)
- added R295: 10k, Resistor_SMD:R_0603_1608Metric, F.Cu at (176.1, 58.4)
- added R296: 10k, Resistor_SMD:R_0603_1608Metric, F.Cu at (180.1, 28.3)
- added R297: 10k, Resistor_SMD:R_0603_1608Metric, F.Cu at (180.1, 30.8)
- added R298: 10k, Resistor_SMD:R_0603_1608Metric, F.Cu at (180.1, 33.3)
- added R299: 10k, Resistor_SMD:R_0603_1608Metric, F.Cu at (180.1, 35.8)
- added R300: 10k, Resistor_SMD:R_0603_1608Metric, F.Cu at (180.1, 38.3)
- added R301: 10k, Resistor_SMD:R_0603_1608Metric, F.Cu at (180.1, 40.8)
- added R302: 10k, Resistor_SMD:R_0603_1608Metric, F.Cu at (180.1, 43.3)
- added R303: 10k, Resistor_SMD:R_0603_1608Metric, F.Cu at (180.1, 45.8)
- added R304: 10k, Resistor_SMD:R_0603_1608Metric, F.Cu at (180.1, 48.4)
- added R305: 10k, Resistor_SMD:R_0603_1608Metric, F.Cu at (115.0, 135.4)
- added R306: 10k, Resistor_SMD:R_0603_1608Metric, F.Cu at (115.0, 138.0)
- added R307: 10k, Resistor_SMD:R_0603_1608Metric, F.Cu at (115.0, 140.5)
- added R308: 10k, Resistor_SMD:R_0603_1608Metric, F.Cu at (119.0, 117.9)
- added R309: 10k, Resistor_SMD:R_0603_1608Metric, F.Cu at (119.0, 120.4)
- added R310: 10k, Resistor_SMD:R_0603_1608Metric, F.Cu at (119.0, 122.9)
- added R311: 10k, Resistor_SMD:R_0603_1608Metric, F.Cu at (119.0, 125.4)
- added R312: 10k, Resistor_SMD:R_0603_1608Metric, F.Cu at (119.0, 127.9)
- added R313: 10k, Resistor_SMD:R_0603_1608Metric, F.Cu at (119.0, 130.4)
- added R314: 10k, Resistor_SMD:R_0603_1608Metric, F.Cu at (119.0, 132.9)
- added R315: 10k, Resistor_SMD:R_0603_1608Metric, F.Cu at (119.0, 135.4)
- added R316: 10k, Resistor_SMD:R_0603_1608Metric, F.Cu at (119.0, 138.0)
- added R317: 10k, Resistor_SMD:R_0603_1608Metric, F.Cu at (119.0, 140.5)
- added U35: G3VM61VY2, user_lib:G3VM-61VY2TR, F.Cu at (19.9, 119.1)
- added U36: G3VM61VY2, user_lib:G3VM-61VY2TR, F.Cu at (19.9, 124.2)
- added U37: G3VM61VY2, user_lib:G3VM-61VY2TR, F.Cu at (19.9, 129.2)
- added U38: G3VM61VY2, user_lib:G3VM-61VY2TR, F.Cu at (19.9, 134.3)
- added U39: G3VM61VY2, user_lib:G3VM-61VY2TR, F.Cu at (19.9, 139.3)
- added U40: G3VM61VY2, user_lib:G3VM-61VY2TR, F.Cu at (19.9, 144.4)
- added U41: G3VM61VY2, user_lib:G3VM-61VY2TR, F.Cu at (19.9, 149.4)
- added U42: G3VM61VY2, user_lib:G3VM-61VY2TR, F.Cu at (19.9, 154.5)
- added U43: G3VM61VY2, user_lib:G3VM-61VY2TR, F.Cu at (28.7, 119.1)
- added U44: G3VM61VY2, user_lib:G3VM-61VY2TR, F.Cu at (28.7, 124.2)
- added U45: G3VM61VY2, user_lib:G3VM-61VY2TR, F.Cu at (28.7, 129.2)
- added U46: G3VM61VY2, user_lib:G3VM-61VY2TR, F.Cu at (28.7, 134.3)
- added U47: G3VM61VY2, user_lib:G3VM-61VY2TR, F.Cu at (28.7, 139.3)
- added U48: G3VM61VY2, user_lib:G3VM-61VY2TR, F.Cu at (28.7, 144.4)
- added U49: G3VM61VY2, user_lib:G3VM-61VY2TR, F.Cu at (28.7, 149.4)
- added U50: G3VM61VY2, user_lib:G3VM-61VY2TR, F.Cu at (28.7, 154.5)
- added U51: G3VM61VY2, user_lib:G3VM-61VY2TR, F.Cu at (37.5, 119.1)
- added U52: G3VM61VY2, user_lib:G3VM-61VY2TR, F.Cu at (37.5, 124.2)
- added U53: G3VM61VY2, user_lib:G3VM-61VY2TR, F.Cu at (37.5, 129.2)
- added U54: G3VM61VY2, user_lib:G3VM-61VY2TR, F.Cu at (37.5, 134.3)
- added U55: G3VM61VY2, user_lib:G3VM-61VY2TR, F.Cu at (37.5, 139.3)
- added U56: SCWN06A-12, user_lib:SCWN06A-12, F.Cu at (58.8, 127.8)
- added U77: SMU02M-12, user_lib:SMU02M-12, F.Cu at (205.1, 48.7)
- R2, R3, R7, R8: value PWR_REG -> 10k
- moved C111 163.0 mm to (200.6, 16.4)
- moved C112 163.0 mm to (200.6, 18.9)
- moved C113 163.0 mm to (200.6, 21.4)
- moved C114 163.0 mm to (200.6, 24.0)
- moved C115 163.0 mm to (200.6, 26.5)
- moved C116 163.0 mm to (200.6, 29.0)
- moved H10 163.0 mm to (193.5, 30.4)
- moved H11 163.0 mm to (193.5, 40.5)
- moved H9 163.0 mm to (193.5, 20.2)
- moved J23 163.0 mm to (204.7, 37.2)
- moved R279 163.0 mm to (204.6, 16.4)
- moved R280 163.0 mm to (204.6, 18.9)
- moved R281 163.0 mm to (204.6, 21.4)
- moved R282 163.0 mm to (204.6, 24.0)
- moved R283 163.0 mm to (204.6, 26.5)
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Connections:
- Q10 pad 2: Net-(Q10-S) -> GND_IN
- Q10 pad 3: 5V0_SWITCHES_2 -> Net-(Q10-D)
- Q11 pad 2: Net-(Q11-S) -> GND_IN
- Q11 pad 3: 5V0_SWITCHES_1 -> Net-(Q11-D)
- Q12 pad 2: Net-(Q12-S) -> GND_IN
- Q12 pad 3: 5V0_SWITCHES_2 -> Net-(Q12-D)
- Q13 pad 2: Net-(Q13-S) -> GND_IN
- Q13 pad 3: 5V0_SWITCHES_1 -> Net-(Q13-D)
- Q14 pad 2: Net-(Q14-S) -> GND_IN
- Q14 pad 3: 5V0_SWITCHES_2 -> Net-(Q14-D)
- Q15 pad 2: Net-(Q15-S) -> GND_IN
- Q15 pad 3: 5V0_SWITCHES_1 -> Net-(Q15-D)
- Q16 pad 2: Net-(Q16-S) -> GND_IN
- Q16 pad 3: 5V0_SWITCHES_2 -> Net-(Q16-D)
- Q17 pad 2: Net-(Q17-S) -> GND_IN
- Q17 pad 3: 5V0_SWITCHES_1 -> Net-(Q17-D)
- Q18 pad 2: Net-(Q18-S) -> GND_IN
- Q18 pad 3: 5V0_SWITCHES_2 -> Net-(Q18-D)
- Q19 pad 2: Net-(Q19-S) -> GND_IN
- Q19 pad 3: 5V0_SWITCHES_1 -> Net-(Q19-D)
- Q20 pad 2: Net-(Q20-S) -> GND_IN
- Q20 pad 3: 5V0_SWITCHES_2 -> Net-(Q20-D)
- Q21 pad 2: Net-(Q21-S) -> GND_IN
- Q21 pad 3: 5V0_SWITCHES_1 -> Net-(Q21-D)
- Q22 pad 2: Net-(Q22-S) -> GND_IN
- Q22 pad 3: 5V0_SWITCHES_2 -> Net-(Q22-D)
- Q23 pad 2: Net-(Q23-S) -> GND_IN
- Q23 pad 3: 5V0_SWITCHES_3 -> Net-(Q23-D)
- Q24 pad 2: Net-(Q24-S) -> GND_IN
- Q24 pad 3: 5V0_SWITCHES_3 -> Net-(Q24-D)
- Q25 pad 2: Net-(Q25-S) -> GND_IN
- Q25 pad 3: 5V0_SWITCHES_3 -> Net-(Q25-D)
- Q26 pad 2: Net-(Q26-S) -> GND_IN
- Q26 pad 3: 5V0_SWITCHES_3 -> Net-(Q26-D)
- Q27 pad 2: Net-(Q27-S) -> GND_IN
- Q27 pad 3: 5V0_SWITCHES_3 -> Net-(Q27-D)
- Q28 pad 2: Net-(Q28-S) -> GND_IN
- Q28 pad 3: 5V0_SWITCHES_3 -> Net-(Q28-D)
- Q29 pad 2: Net-(Q29-S) -> GND_IN
- Q29 pad 3: 5V0_SWITCHES_3 -> Net-(Q29-D)
- Q30 pad 2: Net-(Q30-S) -> GND_IN
- Q30 pad 3: 5V0_SWITCHES_3 -> Net-(Q30-D)
- Q31 pad 2: Net-(Q31-S) -> GND_IN
- Q31 pad 3: 5V0_SWITCHES_3 -> Net-(Q31-D)
- Q32 pad 2: Net-(Q32-S) -> GND_IN
- Q32 pad 3: 5V0_SWITCHES_3 -> Net-(Q32-D)
- Q33 pad 2: Net-(Q33-S) -> GND_IN
- Q33 pad 3: 5V0_SWITCHES_3 -> Net-(Q33-D)
- Q34 pad 2: Net-(Q34-S) -> GND_IN
- Q34 pad 3: 5V0_SWITCHES_3 -> Net-(Q34-D)
- Q35 pad 2: Net-(Q35-S) -> GND_IN
- Q35 pad 3: 5V0_SWITCHES_3 -> Net-(Q35-D)
- Q5 pad 2: Net-(Q5-S) -> GND_IN
- Q5 pad 3: 5V0_SWITCHES_1 -> Net-(Q5-D)
- Q6 pad 2: Net-(Q6-S) -> GND_IN
- Q6 pad 3: 5V0_SWITCHES_2 -> Net-(Q6-D)
- Q7 pad 2: Net-(Q7-S) -> GND_IN
- Q7 pad 3: 5V0_SWITCHES_1 -> Net-(Q7-D)
- Q8 pad 2: Net-(Q8-S) -> GND_IN
- Q8 pad 3: 5V0_SWITCHES_2 -> Net-(Q8-D)
- Q9 pad 2: Net-(Q9-S) -> GND_IN
- Q9 pad 3: 5V0_SWITCHES_1 -> Net-(Q9-D)
- R101 pad 1: Net-(Q19-S) -> Net-(Q19-D)
- R103 pad 1: Net-(Q20-S) -> Net-(Q20-D)
- R109 pad 1: Net-(Q21-S) -> Net-(Q21-D)
- R111 pad 1: Net-(Q22-S) -> Net-(Q22-D)
- R117 pad 1: Net-(Q23-S) -> Net-(Q23-D)
- R121 pad 1: Net-(Q24-S) -> Net-(Q24-D)
- R125 pad 1: Net-(Q25-S) -> Net-(Q25-D)
- R129 pad 1: Net-(Q26-S) -> Net-(Q26-D)
- R134 pad 1: Net-(Q27-S) -> Net-(Q27-D)
- R138 pad 1: Net-(Q28-S) -> Net-(Q28-D)
- R142 pad 1: Net-(Q29-S) -> Net-(Q29-D)
- R146 pad 1: Net-(Q30-S) -> Net-(Q30-D)
- R150 pad 1: Net-(Q31-S) -> Net-(Q31-D)
- R154 pad 1: Net-(Q32-S) -> Net-(Q32-D)
- R158 pad 1: Net-(Q33-S) -> Net-(Q33-D)
- R162 pad 1: Net-(Q34-S) -> Net-(Q34-D)
- R166 pad 1: Net-(Q35-S) -> Net-(Q35-D)
- R2 pad 1: 5V0 -> 5V0_SWITCHES_1
- R2 pad 2: Net-(R2-Pad2) -> Net-(Q7-D)
- R3 pad 1: Net-(R2-Pad2) -> 5V0_SWITCHES_1
- R3 pad 2: GND -> Net-(Q5-D)
- R45 pad 1: Net-(Q5-S) -> Net-(Q5-D)
- R47 pad 1: Net-(Q6-S) -> Net-(Q6-D)
- R53 pad 1: Net-(Q7-S) -> Net-(Q7-D)
- R55 pad 1: Net-(Q8-S) -> Net-(Q8-D)
- R61 pad 1: Net-(Q9-S) -> Net-(Q9-D)
- R63 pad 1: Net-(Q10-S) -> Net-(Q10-D)
- R69 pad 1: Net-(Q11-S) -> Net-(Q11-D)
- R7 pad 1: 12V0 -> 5V0_SWITCHES_1
- R7 pad 2: Net-(R7-Pad2) -> Net-(Q9-D)
- R71 pad 1: Net-(Q12-S) -> Net-(Q12-D)
- R77 pad 1: Net-(Q13-S) -> Net-(Q13-D)
- R79 pad 1: Net-(Q14-S) -> Net-(Q14-D)
- R8 pad 1: Net-(R7-Pad2) -> 5V0_SWITCHES_1
- R8 pad 2: GND_12V -> Net-(Q11-D)
- R85 pad 1: Net-(Q15-S) -> Net-(Q15-D)
- R87 pad 1: Net-(Q16-S) -> Net-(Q16-D)
- R93 pad 1: Net-(Q17-S) -> Net-(Q17-D)
- R95 pad 1: Net-(Q18-S) -> Net-(Q18-D)
- U19 pad 1: Net-(R45-Pad2) -> 5V0_SWITCHES_1
- U19 pad 2: GND_IN -> Net-(R45-Pad2)
- U19 pad 3: Net-(R53-Pad2) -> 5V0_SWITCHES_1
- U19 pad 4: GND_IN -> Net-(R53-Pad2)
- U19 pad 5: Net-(R61-Pad2) -> 5V0_SWITCHES_1
- U19 pad 6: GND_IN -> Net-(R61-Pad2)
- U19 pad 7: Net-(R69-Pad2) -> 5V0_SWITCHES_1
- U19 pad 8: GND_IN -> Net-(R69-Pad2)
- U20 pad 1: Net-(R47-Pad2) -> 5V0_SWITCHES_2
- U20 pad 2: GND_IN -> Net-(R47-Pad2)
- U20 pad 3: Net-(R55-Pad2) -> 5V0_SWITCHES_2
- U20 pad 4: GND_IN -> Net-(R55-Pad2)
- U20 pad 5: Net-(R63-Pad2) -> 5V0_SWITCHES_2
- U20 pad 6: GND_IN -> Net-(R63-Pad2)
- U20 pad 7: Net-(R71-Pad2) -> 5V0_SWITCHES_2
- U20 pad 8: GND_IN -> Net-(R71-Pad2)
- U21 pad 1: Net-(R77-Pad2) -> 5V0_SWITCHES_1
- U21 pad 2: GND_IN -> Net-(R77-Pad2)
- U21 pad 3: Net-(R85-Pad2) -> 5V0_SWITCHES_1
- U21 pad 4: GND_IN -> Net-(R85-Pad2)
- U21 pad 5: Net-(R93-Pad2) -> 5V0_SWITCHES_1
- U21 pad 6: GND_IN -> Net-(R93-Pad2)
- U21 pad 7: Net-(R101-Pad2) -> 5V0_SWITCHES_1
- U21 pad 8: GND_IN -> Net-(R101-Pad2)
- U22 pad 1: Net-(R79-Pad2) -> 5V0_SWITCHES_2
- U22 pad 2: GND_IN -> Net-(R79-Pad2)
- U22 pad 3: Net-(R87-Pad2) -> 5V0_SWITCHES_2
- U22 pad 4: GND_IN -> Net-(R87-Pad2)
- U22 pad 5: Net-(R95-Pad2) -> 5V0_SWITCHES_2
- U22 pad 6: GND_IN -> Net-(R95-Pad2)
- U22 pad 7: Net-(R103-Pad2) -> 5V0_SWITCHES_2
- U22 pad 8: GND_IN -> Net-(R103-Pad2)
- U23 pad 1: Net-(R109-Pad2) -> 5V0_SWITCHES_1
- U23 pad 2: GND_IN -> Net-(R109-Pad2)
- U24 pad 1: Net-(R111-Pad2) -> 5V0_SWITCHES_2
- U24 pad 2: GND_IN -> Net-(R111-Pad2)
- U27 pad 1: Net-(R117-Pad2) -> 5V0_SWITCHES_3
- U27 pad 2: GND_IN -> Net-(R117-Pad2)
- U27 pad 3: Net-(R121-Pad2) -> 5V0_SWITCHES_3
- U27 pad 4: GND_IN -> Net-(R121-Pad2)
- U27 pad 5: Net-(R125-Pad2) -> 5V0_SWITCHES_3
- U27 pad 6: GND_IN -> Net-(R125-Pad2)
- U27 pad 7: Net-(R129-Pad2) -> 5V0_SWITCHES_3
- U27 pad 8: GND_IN -> Net-(R129-Pad2)
- U28 pad 1: Net-(R134-Pad2) -> 5V0_SWITCHES_3
- U28 pad 2: GND_IN -> Net-(R134-Pad2)
- U28 pad 3: Net-(R138-Pad2) -> 5V0_SWITCHES_3
- U28 pad 4: GND_IN -> Net-(R138-Pad2)
- U28 pad 5: Net-(R142-Pad2) -> 5V0_SWITCHES_3
- U28 pad 6: GND_IN -> Net-(R142-Pad2)
- U28 pad 7: Net-(R146-Pad2) -> 5V0_SWITCHES_3
- U28 pad 8: GND_IN -> Net-(R146-Pad2)
- U30 pad 1: Net-(R150-Pad2) -> 5V0_SWITCHES_3
- U30 pad 2: GND_IN -> Net-(R150-Pad2)
- U31 pad 1: Net-(R154-Pad2) -> 5V0_SWITCHES_3
- U31 pad 2: GND_IN -> Net-(R154-Pad2)
- U32 pad 1: Net-(R158-Pad2) -> 5V0_SWITCHES_3
- U32 pad 2: GND_IN -> Net-(R158-Pad2)
- U33 pad 1: Net-(R162-Pad2) -> 5V0_SWITCHES_3
- U33 pad 2: GND_IN -> Net-(R162-Pad2)
- U34 pad 1: Net-(R166-Pad2) -> 5V0_SWITCHES_3
- U34 pad 2: GND_IN -> Net-(R166-Pad2)
- U4 pad 11: unconnected-(U4-REG-Pad11) -> Net-(U4-REG)
- U4 pad 14: unconnected-(U4-+VOUT-Pad14) -> 12V0
- U4 pad 16: unconnected-(U4--VOUT-Pad16) -> GND_12V
- U4 pad 2: unconnected-(U4--VIN-Pad2) -> Net-(C101-Pad2)
- U4 pad 22: unconnected-(U4-+VIN-Pad22) -> Net-(C101-Pad1)
- U4 pad 23: unconnected-(U4-+VIN-Pad23) -> Net-(C101-Pad1)
- U4 pad 3: unconnected-(U4--VIN-Pad3) -> Net-(C101-Pad2)
- U7 pad 11: unconnected-(U7-REG-Pad11) -> Net-(U7-REG)
- U7 pad 14: unconnected-(U7-+VOUT-Pad14) -> 5V0
- U7 pad 16: unconnected-(U7--VOUT-Pad16) -> GND
- U7 pad 2: unconnected-(U7--VIN-Pad2) -> Net-(C102-Pad2)
- U7 pad 22: unconnected-(U7-+VIN-Pad22) -> Net-(C102-Pad1)
- U7 pad 23: unconnected-(U7-+VIN-Pad23) -> Net-(C102-Pad1)
- U7 pad 3: unconnected-(U7--VIN-Pad3) -> Net-(C102-Pad2)
Other:
- board text added: "программаторный разъём"
