File: Hardware/ciam/impeller18/stm32_peripherals.kicad_sch (KiCad schematic)
At the start: 8 parts, among them J1 Micro_SD_Card_Con

Commit message: updated impeller18 schematics
Parts:
- added C105, C106: 100n, Capacitor_SMD:C_0603_1608Metric, symbol Device:C_Small
- added D10, D11, D8, D9: FYLS-3528RGBC, user_lib:LED_RGB_promelec, symbol Device:LED_RGBA
- added J14: USB_B_Micro, user_lib:U-F-M5DD-W-2-SUS, symbol Connector:USB_B_Micro
- added R205, R206, R207, R208, R209, R210, R211, R212, R213, R214, R215, R216: 220, Resistor_SMD:R_0603_1608Metric, symbol Device:R
- added R217, R218: 10k, Resistor_SMD:R_0603_1608Metric, symbol Device:R_Small
- added U53: W25Q128FVSIG, Package_SO:SOIC-8_5.23x5.23mm_P1.27mm, symbol Memory_Flash:W25Q32JVSS
- added U54: USBLC6-2SC6, Package_TO_SOT_SMD:SOT-23-6, symbol Power_Protection:USBLC6-2SC6
- J1: value Micro_SD_Card_Con -> TF-01
- R2, R3, R4, R5, R6, R7: value 100k -> 10k
Connections:
- net GND: now also C26.2, C105.1, C106.2, J14.5 (GND), J14.6 (Shield), R218.2, U53.4 (GND), U54.2 (GND); no longer C26.1
- net VDD_3V3 renamed 3V3
- net 3V3: now also C26.1, C105.2, D10.2 (A), D11.2 (A), D8.2 (A), D9.2 (A), U53.7 (IO3), U53.8 (VCC); no longer C26.2
- new net: D8.3 (BK), R207.1
- new net: D9.1 (RK), R208.1
- new net: D9.4 (GK), R209.1
- new net: D8.4 (GK), R206.1
- new net: D10.3 (BK), R213.1
- new net: D11.4 (GK), R215.1
- new net: D11.1 (RK), R214.1
- new net: C106.1, J14.1 (VBUS), R217.1, U54.5 (VBUS)
- new net: D9.3 (BK), R210.1
- new net: D8.1 (RK), R205.1
- new net: D10.1 (RK), R211.1
- new net: D10.4 (GK), R212.1
- new net: D11.3 (BK), R216.1
- new net LED1_RGB_BLUE: R207.2
- new net LED1_RGB_GREEN: R206.2
- new net LED1_RGB_RED: R205.2
- new net LED2_RGB_BLUE: R210.2
- new net LED2_RGB_GREEN: R209.2
- new net LED2_RGB_RED: R208.2
- new net LED3_RGB_BLUE: R213.2
- new net LED3_RGB_GREEN: R212.2
- new net LED3_RGB_RED: R211.2
- new net LED4_RGB_BLUE: R216.2
- new net LED4_RGB_GREEN: R215.2
- new net LED4_RGB_RED: R214.2
- new net SPI1_STM32_CLK: U53.6 (CLK)
- new net SPI1_STM32_FLASH_CS: U53.1 (~{CS})
- new net SPI1_STM32_MISO: U53.2 (DO(IO1))
- new net SPI1_STM32_MOSI: U53.5 (DI(IO0))
- new net USB_D+: U54.1 (I/O1)
- new net USB_D-: U54.3 (I/O2)
- new net USB_VBUS: R217.2, R218.1
- new net usb_conn_d+: J14.3 (D+), U54.6 (I/O1)
- new net usb_conn_d-: J14.2 (D-), U54.4 (I/O2)
- no-connect marks 0 -> 2
Other:
- note added: "Flash memory"
- note added: "LED RGB"
- note added: "Micro SD card"
- note added: "USB"
- note removed: "Micro SD"
- moved on the sheet: R2

Commit message: updated schematics
Parts:
- renumbered C26 to C100, C105 to C101, C106 to C102, D8 to D14, D10 to D15, D9 to D16, D11 to D17, J1 to J17, J14 to J18, R205 to R226, R211 to R227, R2 to R228, R3 to R229, R4 to R230, R5 to R231, R6 to R232, R7 to R233, R206 to R234, R212 to R235, R207 to R236, R213 to R237, R208 to R238, R214 to R239, R209 to R240, R215 to R241, R210 to R242, R216 to R243, R217 to R244, R218 to R245, U53 to U64, U54 to U65

Commit message: updated schematics
Parts:
- renumbered C100 to C108, C101 to C109, C102 to C110, D14 to D21, D15 to D22, D16 to D23, D17 to D24, J17 to J18, J18 to J19, R226 to R251, R227 to R252, R228 to R253, R229 to R254, R230 to R255, R231 to R256, R232 to R257, R233 to R258, R234 to R259, R235 to R260, R236 to R261, R237 to R262, R238 to R263, R239 to R264, R240 to R265, R241 to R266, R242 to R267, R243 to R268, R244 to R269, R245 to R270, U64 to U71, U65 to U72

Commit message: updated schematics
Parts:
- C108, C109, C110: footprint Capacitor_SMD:C_0603_1608Metric -> (none); Мин. кол-во (none) -> 300; Ссылка (none) -> https://www.promelec.ru/product/323633/; Цена (none) -> 2; Человекопонятное название (none) -> Керамический ЧИП-конденсатор 0603 X7R 0.1мкФ
- D21, D22, D23, D24: footprint user_lib:LED_RGB_promelec -> (none); Мин. кол-во (none) -> 2; Ссылка (none) -> https://www.promelec.ru/product/337147/; Цена (none) -> 8; Человекопонятное название (none) -> Светодиод smd 3,5х2,8мм/красный/625нм/200мкд - зеленый/520н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
- J21: renamed from J18; footprint sd:TF01A -> (none)
- J22: renamed from J19; footprint user_lib:U-F-M5DD-W-2-SUS -> (none)
- R259: renamed from R251; footprint Resistor_SMD:R_0603_1608Metric -> (none); Мин. кол-во (none) -> 100; Ссылка (none) -> https://www.promelec.ru/product/46446/; Цена (none) -> 1; Человекопонятное название (none) -> Толстопленочный ЧИП-резистор 0603 220Ом
- R260: renamed from R252; footprint Resistor_SMD:R_0603_1608Metric -> (none); Мин. кол-во (none) -> 100; Ссылка (none) -> https://www.promelec.ru/product/46446/; Цена (none) -> 1; Человекопонятное название (none) -> Толстопленочный ЧИП-резистор 0603 220Ом
- R261: renamed from R253; footprint Resistor_SMD:R_0603_1608Metric -> (none); Мин. кол-во (none) -> 1000; Ссылка (none) -> https://www.promelec.ru/product/344748/; Цена (none) -> 1; Человекопонятное название (none) -> Толстопленочный ЧИП-резистор 0603 10кОм
- R262: renamed from R254; footprint Resistor_SMD:R_0603_1608Metric -> (none); Мин. кол-во (none) -> 1000; Ссылка (none) -> https://www.promelec.ru/product/344748/; Цена (none) -> 1; Человекопонятное название (none) -> Толстопленочный ЧИП-резистор 0603 10кОм
- R263: renamed from R255; footprint Resistor_SMD:R_0603_1608Metric -> (none); Мин. кол-во (none) -> 1000; Ссылка (none) -> https://www.promelec.ru/product/344748/; Цена (none) -> 1; Человекопонятное название (none) -> Толстопленочный ЧИП-резистор 0603 10кОм
- R264: renamed from R256; footprint Resistor_SMD:R_0603_1608Metric -> (none); Мин. кол-во (none) -> 1000; Ссылка (none) -> https://www.promelec.ru/product/344748/; Цена (none) -> 1; Человекопонятное название (none) -> Толстопленочный ЧИП-резистор 0603 10кОм
- R265: renamed from R257; footprint Resistor_SMD:R_0603_1608Metric -> (none); Мин. кол-во (none) -> 1000; Ссылка (none) -> https://www.promelec.ru/product/344748/; Цена (none) -> 1; Человекопонятное название (none) -> Толстопленочный ЧИП-резистор 0603 10кОм
- R266: renamed from R258; footprint Resistor_SMD:R_0603_1608Metric -> (none); Мин. кол-во (none) -> 1000; Ссылка (none) -> https://www.promelec.ru/product/344748/; Цена (none) -> 1; Человекопонятное название (none) -> Толстопленочный ЧИП-резистор 0603 10кОм
- R267: renamed from R259; footprint Resistor_SMD:R_0603_1608Metric -> (none); Мин. кол-во (none) -> 100; Ссылка (none) -> https://www.promelec.ru/product/46446/; Цена (none) -> 1; Человекопонятное название (none) -> Толстопленочный ЧИП-резистор 0603 220Ом
- R268: renamed from R260; footprint Resistor_SMD:R_0603_1608Metric -> (none); Мин. кол-во (none) -> 100; Ссылка (none) -> https://www.promelec.ru/product/46446/; Цена (none) -> 1; Человекопонятное название (none) -> Толстопленочный ЧИП-резистор 0603 220Ом
- R269: renamed from R261; footprint Resistor_SMD:R_0603_1608Metric -> (none); Мин. кол-во (none) -> 100; Ссылка (none) -> https://www.promelec.ru/product/46446/; Цена (none) -> 1; Человекопонятное название (none) -> Толстопленочный ЧИП-резистор 0603 220Ом
- R270: renamed from R262; footprint Resistor_SMD:R_0603_1608Metric -> (none); Мин. кол-во (none) -> 100; Ссылка (none) -> https://www.promelec.ru/product/46446/; Цена (none) -> 1; Человекопонятное название (none) -> Толстопленочный ЧИП-резистор 0603 220Ом
- R271: renamed from R263; footprint Resistor_SMD:R_0603_1608Metric -> (none); Мин. кол-во (none) -> 100; Ссылка (none) -> https://www.promelec.ru/product/46446/; Цена (none) -> 1; Человекопонятное название (none) -> Толстопленочный ЧИП-резистор 0603 220Ом
- R272: renamed from R264; footprint Resistor_SMD:R_0603_1608Metric -> (none); Мин. кол-во (none) -> 100; Ссылка (none) -> https://www.promelec.ru/product/46446/; Цена (none) -> 1; Человекопонятное название (none) -> Толстопленочный ЧИП-резистор 0603 220Ом
- R273: renamed from R265; footprint Resistor_SMD:R_0603_1608Metric -> (none); Мин. кол-во (none) -> 100; Ссылка (none) -> https://www.promelec.ru/product/46446/; Цена (none) -> 1; Человекопонятное название (none) -> Толстопленочный ЧИП-резистор 0603 220Ом
- R274: renamed from R266; footprint Resistor_SMD:R_0603_1608Metric -> (none); Мин. кол-во (none) -> 100; Ссылка (none) -> https://www.promelec.ru/product/46446/; Цена (none) -> 1; Человекопонятное название (none) -> Толстопленочный ЧИП-резистор 0603 220Ом
- R275: renamed from R267; footprint Resistor_SMD:R_0603_1608Metric -> (none); Мин. кол-во (none) -> 100; Ссылка (none) -> https://www.promelec.ru/product/46446/; Цена (none) -> 1; Человекопонятное название (none) -> Толстопленочный ЧИП-резистор 0603 220Ом
- R276: renamed from R268; footprint Resistor_SMD:R_0603_1608Metric -> (none); Мин. кол-во (none) -> 100; Ссылка (none) -> https://www.promelec.ru/product/46446/; Цена (none) -> 1; Человекопонятное название (none) -> Толстопленочный ЧИП-резистор 0603 220Ом
- R277: renamed from R269; footprint Resistor_SMD:R_0603_1608Metric -> (none); Мин. кол-во (none) -> 1000; Ссылка (none) -> https://www.promelec.ru/product/344748/; Цена (none) -> 1; Человекопонятное название (none) -> Толстопленочный ЧИП-резистор 0603 10кОм
- R278: renamed from R270; footprint Resistor_SMD:R_0603_1608Metric -> (none); Мин. кол-во (none) -> 1000; Ссылка (none) -> https://www.promelec.ru/product/344748/; Цена (none) -> 1; Человекопонятное название (none) -> Толстопленочный ЧИП-резистор 0603 10кОм
- U73: renamed from U71; footprint Package_SO:SOIC-8_5.23x5.23mm_P1.27mm -> (none); Мин. кол-во (none) -> 2; Ссылка (none) -> https://www.promelec.ru/product/342088/; Цена (none) -> 127; Человекопонятное название (none) -> Флэш-память
- U74: renamed from U72; footprint Package_TO_SOT_SMD:SOT-23-6 -> (none); Мин. кол-во (none) -> 1; Ссылка (none) -> https://www.promelec.ru/product/128262/; Цена (none) -> 13; Человекопонятное название (none) -> Защита интерфейса USB от электростатических разрядов

Commit message: added footprints
Parts:
- C108, C109, C110: footprint (none) -> Capacitor_SMD:C_0603_1608Metric
- D21, D22, D23, D24: footprint (none) -> user_lib:LED_RGB_promelec
- J22: footprint (none) -> user_lib:U-F-M5DD-W-2-SUS
- R259, R260, R261, R262, R263, R264, R265, R266, R267, R268, R269, R270, R271, R272, R273, R274, R275, R276, R277, R278: footprint (none) -> Resistor_SMD:R_0603_1608Metric
- U73: footprint (none) -> Package_SO:SOIC-8_5.23x5.23mm_P1.27mm
- U74: footprint (none) -> Package_TO_SOT_SMD:SOT-23-6
Changed lines of the file:
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@@
 			)
 		)
-		(property "Footprint" ""
+		(property "Footprint" "Resistor_SMD:R_0603_1608Metric"
 			(at 249.555 40.513 90)
 			(effects
@@
 			)
 		)
-		(property "Footprint" ""
+		(property "Footprint" "Resistor_SMD:R_0603_1608Metric"
 			(at 249.555 57.658 90)
 			(effects
@@
 			)
 		)
-		(property "Footprint" ""
+		(property "Footprint" "Resistor_SMD:R_0603_1608Metric"
 			(at 249.555 62.738 90)
 			(effects
@@
 			)
 		)
-		(property "Footprint" ""
+		(property "Footprint" "Resistor_SMD:R_0603_1608Metric"
 			(at 57.785 32.385 0)
 			(effects
@@
 			)
 		)
-		(property "Footprint" ""
+		(property "Footprint" "Resistor_SMD:R_0603_1608Metric"
 			(at 249.555 35.433 90)
 			(effects
@@
 			)
 		)
-		(property "Footprint" ""
+		(property "Footprint" "Resistor_SMD:R_0603_1608Metric"
 			(at 308.61 40.513 90)
 			(effects
@@
 			)
 		)
-		(property "Footprint" ""
+		(property "Footprint" "Resistor_SMD:R_0603_1608Metric"
 			(at 308.61 62.738 90)
 			(effects
@@
 			)
 		)
-		(property "Footprint" ""
+		(property "Footprint" "Package_SO:SOIC-8_5.23x5.23mm_P1.27mm"
 			(at 189.23 49.53 0)
 			(effects
@@
 			)
 		)
-		(property "Footprint" ""
+		(property "Footprint" "Resistor_SMD:R_0603_1608Metric"
 			(at 308.61 57.658 90)
 			(effects
@@
 			)
 		)
-		(property "Footprint" ""
+		(property "Footprint" "Resistor_SMD:R_0603_1608Metric"
 			(at 73.025 32.385 0)
 			(effects
@@
 			)
 		)
-		(property "Footprint" ""
+		(property "Footprint" "Capacitor_SMD:C_0603_1608Metric"
 			(at 30.48 114.935 0)
 			(effects
@@
 			)
 		)
-		(property "Footprint" ""
+		(property "Footprint" "Resistor_SMD:R_0603_1608Metric"
 			(at 120.015 119.38 0)
 			(effects
@@
 			)
 		)
-		(property "Footprint" ""
+		(property "Footprint" "Resistor_SMD:R_0603_1608Metric"
 			(at 50.165 32.385 0)
 			(effects
@@
 			)
 		)
-		(property "Footprint" ""
+		(property "Footprint" "Capacitor_SMD:C_0603_1608Metric"
 			(at 202.565 49.53 0)
 			(effects
@@
 			)
 		)
-		(property "Footprint" ""
+		(property "Footprint" "Package_TO_SOT_SMD:SOT-23-6"
 			(at 85.725 128.27 0)
 			(effects
@@
 			)
 		)
-		(property "Footprint" ""
+		(property "Footprint" "Resistor_SMD:R_0603_1608Metric"
 			(at 65.405 32.385 0)
 			(effects
@@
 			)
 		)
-		(property "Footprint" ""
+		(property "Footprint" "Resistor_SMD:R_0603_1608Metric"
 			(at 249.555 67.818 90)
 			(effects
@@
 			)
 		)
-		(property "Footprint" ""
+		(property "Footprint" "user_lib:U-F-M5DD-W-2-SUS"
 			(at 43.815 115.57 0)
 			(effects
@@
 			)
 		)
-		(property "Footprint" ""
+		(property "Footprint" "Resistor_SMD:R_0603_1608Metric"
 			(at 249.555 30.353 90)
 			(effects
@@
 			)
 		)
-		(property "Footprint" ""
+		(property "Footprint" "Resistor_SMD:R_0603_1608Metric"
 			(at 80.645 32.385 0)
 			(effects
@@
 			)
 		)
-		(property "Footprint" ""
+		(property "Footprint" "user_lib:LED_RGB_promelec"
 			(at 297.18 34.925 0)
 			(effects
@@
 			)
 		)
-		(property "Footprint" ""
+		(property "Footprint" "user_lib:LED_RGB_promelec"
 			(at 238.125 34.925 0)
 			(effects
@@
 			)
 		)
-		(property "Footprint" ""
+		(property "Footprint" "user_lib:LED_RGB_promelec"
 			(at 297.18 62.23 0)
 			(effects
@@
 			)
 		)
-		(property "Footprint" ""
+		(property "Footprint" "Resistor_SMD:R_0603_1608Metric"
 			(at 308.61 35.433 90)
 			(effects
@@
 			)
 		)
-		(property "Footprint" ""
+		(property "Footprint" "Resistor_SMD:R_0603_1608Metric"
 			(at 308.61 30.353 90)
 			(effects
@@
 			)
 		)
-		(property "Footprint" ""
+		(property "Footprint" "Resistor_SMD:R_0603_1608Metric"
 			(at 308.61 67.818 90)
 			(effects
@@
 			)
 		)
-		(property "Footprint" ""
+		(property "Footprint" "Resistor_SMD:R_0603_1608Metric"
 			(at 42.545 32.385 0)
 			(effects
@@
 			)
 		)
-		(property "Footprint" ""
+		(property "Footprint" "user_lib:LED_RGB_promelec"
 			(at 238.125 62.23 0)
 			(effects
@@
 			)
 		)
-		(property "Footprint" ""
+		(property "Footprint" "Capacitor_SMD:C_0603_1608Metric"
 			(at 97.79 28.575 0)
 			(effects
@@
 			)
 		)
-		(property "Footprint" ""
+		(property "Footprint" "Resistor_SMD:R_0603_1608Metric"
 			(at 120.015 109.22 0)
 			(effects

Commit message: Minor changes
Other:
- note added: "ПРОВЕРИТЬ СВЕТОДИОДЫ"
Changed lines of the file:
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@@
+		)
+	)
+	(text "ПРОВЕРИТЬ СВЕТОДИОДЫ"
+		(exclude_from_sim no)
+		(at 278.765 90.805 0)
+		(effects
+			(font
+				(size 1.27 1.27)
+			)
 		)
 	)

Commit message: Updated packeges
Parts:
- U73: footprint Package_SO:SOIC-8_5.23x5.23mm_P1.27mm -> user_lib:SOIC-8_5.23x5.23mm_P1.27mm
Other:
- note removed: "ПРОВЕРИТЬ СВЕТОДИОДЫ"
Changed lines of the file:
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@@
-		)
-	)
-	(text "ПРОВЕРИТЬ СВЕТОДИОДЫ"
-		(exclude_from_sim no)
-		(at 278.765 90.805 0)
-		(effects
-			(font
-				(size 1.27 1.27)
-			)
 		)
 	)
@@
 			)
 		)
-		(property "Footprint" "Package_SO:SOIC-8_5.23x5.23mm_P1.27mm"
+		(property "Footprint" "user_lib:SOIC-8_5.23x5.23mm_P1.27mm"
 			(at 189.23 49.53 0)
 			(effects

Commit message: Updated packeges
Parts:
- J21: footprint (none) -> sd:TF01A-NEW
Changed lines of the file:
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@@
 			)
 		)
-		(property "Footprint" ""
+		(property "Footprint" "sd:TF01A-NEW"
 			(at 170.18 33.655 0)
 			(effects
