File: Hardware/ciam/impeller18/switches_2.kicad_sch (KiCad schematic)
At the start: 85 parts, among them J11 430451000, J12 430450600, J13 430450400, J14 430450600, Q23 BSS138, Q24 BSS138, Q25 BSS138, Q26 BSS138, Q27 BSS138, Q28 BSS138, Q29 BSS138, Q30 BSS138, Q31 BSS138, Q32 BSS138, Q33 BSS138, Q34 BSS138, Q35 BSS138, U27 TLP291-4, U28 TLP291-4, U29 B0505MT-1WR4, U30 TLP291, U31 TLP291, U32 TLP291, U33 TLP291, U34 TLP291

Commit message: bugfixes
Parts:
- added J28: 430450800, Connector_Molex:Molex_Micro-Fit_3.0_43045-0800_2x04_P3.00mm_Horizontal, symbol Connector_Generic:Conn_02x04_Odd_Even
Connections:
- net SWITCH_3.1_EXT: now also J28.1 (Pin_1)
- net SWITCH_3.2_EXT: now also J28.3 (Pin_3)
- net SWITCH_3.3_EXT: now also J28.5 (Pin_5)
- net SWITCH_3.4_EXT: now also J28.7 (Pin_7)
- net SWITCH_3.5_EXT: now also J28.2 (Pin_2)
- net SWITCH_3.6_EXT: now also J28.4 (Pin_4)
- net SWITCH_3.7_EXT: now also J28.6 (Pin_6)
- net SWITCH_3.8_EXT: now also J28.8 (Pin_8)
Other:
- note added: "что планируется кроме большой красной кнопки и что мы посылаем в РУ1?"

Commit message: Updated packeges
Parts:
- J11: footprint Connector_Molex:Molex_Micro-Fit_3.0_43045-1000_2x05_P3.00mm_Horizontal -> user_lib:430451000
- J12, J14: footprint Connector_Molex:Molex_Micro-Fit_3.0_43045-0600_2x03_P3.00mm_Horizontal -> user_lib:430450600
- J13: footprint Connector_Molex:Molex_Micro-Fit_3.0_43045-0400_2x02_P3.00mm_Horizontal -> user_lib:430454000
- J28: footprint Connector_Molex:Molex_Micro-Fit_3.0_43045-0800_2x04_P3.00mm_Horizontal -> user_lib:430450800
- U30, U31, U32, U33, U34: footprint Package_SO:SOIC-4_4.55x2.6mm_P1.27mm -> user_lib:TLP291
Other:
- note added: "0.5 м"
- note added: "0.9 м"
- note added: "1.8"
- note added: "14 м"
- note added: "4 м"
- note added: "8 м"
Changed lines of the file:
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@@
 		)
 	)
+	(text "0.5 м\n"
+		(exclude_from_sim no)
+		(at 305.435 132.08 0)
+		(effects
+			(font
+				(size 1.27 1.27)
+			)
+		)
+	)
 	(text "большая красная кнопка"
 		(exclude_from_sim no)
@@
 		)
 	)
+	(text "1.8\n"
+		(exclude_from_sim no)
+		(at 272.415 179.705 0)
+		(effects
+			(font
+				(size 1.27 1.27)
+			)
+		)
+	)
 	(text "800/24\nАэрПит\nПитСис"
 		(exclude_from_sim no)
@@
 		)
 	)
+	(text "8 м"
+		(exclude_from_sim no)
+		(at 231.775 148.59 0)
+		(effects
+			(font
+				(size 1.27 1.27)
+			)
+		)
+	)
 	(text "что планируется кроме большой красной кнопки и что мы посылаем в РУ1?"
 		(exclude_from_sim no)
@@
 		)
 	)
+	(text "4 м"
+		(exclude_from_sim no)
+		(at 379.095 147.955 0)
+		(effects
+			(font
+				(size 1.27 1.27)
+			)
+		)
+	)
+	(text "0.5 м\n"
+		(exclude_from_sim no)
+		(at 237.49 156.21 0)
+		(effects
+			(font
+				(size 1.27 1.27)
+			)
+		)
+	)
 	(text "АКБ1\nАКБ2\nАКБ3\nАКБ4\nОбщ-"
 		(exclude_from_sim no)
@@
 		)
 	)
+	(text "0.9 м"
+		(exclude_from_sim no)
+		(at 237.49 171.45 0)
+		(effects
+			(font
+				(size 1.27 1.27)
+			)
+		)
+	)
+	(text "0.5 м\n"
+		(exclude_from_sim no)
+		(at 307.975 156.21 0)
+		(effects
+			(font
+				(size 1.27 1.27)
+			)
+		)
+	)
+	(text "0.5 м\n"
+		(exclude_from_sim no)
+		(at 234.95 132.08 0)
+		(effects
+			(font
+				(size 1.27 1.27)
+			)
+		)
+	)
+	(text " 14 м"
+		(exclude_from_sim no)
+		(at 353.06 169.545 0)
+		(effects
+			(font
+				(size 12.7 12.7)
+				(thickness 2.54)
+				(bold yes)
+			)
+		)
+	)
+	(text "0.9 м"
+		(exclude_from_sim no)
+		(at 323.215 172.085 0)
+		(effects
+			(font
+				(size 1.27 1.27)
+			)
+		)
+	)
 	(label "SWITCH_3.8_EXT"
 		(at 240.665 161.925 0)
@@
 			)
 		)
-		(property "Footprint" "Connector_Molex:Molex_Micro-Fit_3.0_43045-1000_2x05_P3.00mm_Horizontal"
+		(property "Footprint" "user_lib:430451000"
 			(at 271.145 137.16 0)
 			(effects
@@
 			)
 		)
-		(property "Footprint" "Package_SO:SOIC-4_4.55x2.6mm_P1.27mm"
+		(property "Footprint" "user_lib:TLP291"
 			(at 128.905 265.43 0)
 			(effects
@@
 			)
 		)
-		(property "Footprint" "Connector_Molex:Molex_Micro-Fit_3.0_43045-0800_2x04_P3.00mm_Horizontal"
+		(property "Footprint" "user_lib:430450800"
 			(at 343.535 147.955 0)
 			(effects
@@
 			)
 		)
-		(property "Footprint" "Connector_Molex:Molex_Micro-Fit_3.0_43045-0600_2x03_P3.00mm_Horizontal"
+		(property "Footprint" "user_lib:430450600"
 			(at 269.875 196.215 0)
 			(effects
@@
 			)
 		)
-		(property "Footprint" "Package_SO:SOIC-4_4.55x2.6mm_P1.27mm"
+		(property "Footprint" "user_lib:TLP291"
 			(at 128.905 252.095 0)
 			(effects
@@
 			)
 		)
-		(property "Footprint" "Package_SO:SOIC-4_4.55x2.6mm_P1.27mm"
+		(property "Footprint" "user_lib:TLP291"
 			(at 128.905 238.76 0)
 			(effects
@@
 			)
 		)
-		(property "Footprint" "Package_SO:SOIC-4_4.55x2.6mm_P1.27mm"
+		(property "Footprint" "user_lib:TLP291"
 			(at 122.555 183.515 0)
 			(effects
@@
 			)
 		)
-		(property "Footprint" "Connector_Molex:Molex_Micro-Fit_3.0_43045-0600_2x03_P3.00mm_Horizontal"
+		(property "Footprint" "user_lib:430450600"
 			(at 270.51 159.385 0)
 			(effects
@@
 			)
 		)
-		(property "Footprint" "Connector_Molex:Molex_Micro-Fit_3.0_43045-0400_2x02_P3.00mm_Horizontal"
+		(property "Footprint" "user_lib:430454000"
 			(at 271.145 172.72 0)
 			(effects
@@
 			)
 		)
-		(property "Footprint" "Package_SO:SOIC-4_4.55x2.6mm_P1.27mm"
+		(property "Footprint" "user_lib:TLP291"
 			(at 122.555 196.85 0)
 			(effects

Commit message: fixed switches
Parts:
- added R305, R306, R307, R308, R309, R310, R311, R312, R313, R314, R315, R316, R317: 10k, Resistor_SMD:R_0603_1608Metric, symbol Device:R_Small
Connections:
- net 5V0_SWITCHES_3: now also U27.1, U27.3, U27.5, U27.7, U28.1, U28.3, U28.5, U28.7, U30.1, U31.1, U32.1, U33.1, U34.1, R305.1, R306.1, R307.1, R308.1, R309.1, R310.1, R311.1, R312.1, R313.1, R314.1, R315.1, R316.1, R317.1; no longer Q23.3 (D), Q24.3 (D), Q25.3 (D), Q26.3 (D), Q27.3 (D), Q28.3 (D), Q29.3 (D), Q30.3 (D), Q31.3 (D), Q32.3 (D), Q33.3 (D), Q34.3 (D), Q35.3 (D)
- net GND_IN: now also Q23.2 (S), Q24.2 (S), Q25.2 (S), Q26.2 (S), Q27.2 (S), Q28.2 (S), Q29.2 (S), Q30.2 (S), Q31.2 (S), Q32.2 (S), Q33.2 (S), Q34.2 (S), Q35.2 (S); no longer U27.2, U27.4, U27.6, U27.8, U28.2, U28.4, U28.6, U28.8, U30.2, U31.2, U32.2, U33.2, U34.2
- net at R158.1: now also Q33.3 (D), R315.2; no longer Q33.2 (S)
- net at R158.2: now also U32.2; no longer U32.1
- net at R146.1: now also Q30.3 (D), R312.2; no longer Q30.2 (S)
- net at R146.2: now also U28.8; no longer U28.7
- net at R117.2: now also U27.2; no longer U27.1
- net at R150.1: now also Q31.3 (D), R313.2; no longer Q31.2 (S)
- net at R150.2: now also U30.2; no longer U30.1
- net at R125.1: now also Q25.3 (D), R307.2; no longer Q25.2 (S)
- net at R142.1: now also Q29.3 (D), R311.2; no longer Q29.2 (S)
- net at R166.2: now also U34.2; no longer U34.1
- net at R154.1: now also Q32.3 (D), R314.2; no longer Q32.2 (S)
- net at R154.2: now also U31.2; no longer U31.1
- net at R121.2: now also U27.4; no longer U27.3
- net at R142.2: now also U28.6; no longer U28.5
- net at R134.1: now also Q27.3 (D), R309.2; no longer Q27.2 (S)
- net at R166.1: now also Q35.3 (D), R317.2; no longer Q35.2 (S)
- net at R162.2: now also U33.2; no longer U33.1
- net at R129.1: now also Q26.3 (D), R308.2; no longer Q26.2 (S)
- net at R138.1: now also Q28.3 (D), R310.2; no longer Q28.2 (S)
- net at R138.2: now also U28.4; no longer U28.3
- net at R121.1: now also Q24.3 (D), R306.2; no longer Q24.2 (S)
- net at R117.1: now also Q23.3 (D), R305.2; no longer Q23.2 (S)
- net at R129.2: now also U27.8; no longer U27.7
- net at R125.2: now also U27.6; no longer U27.5
- net at R162.1: now also Q34.3 (D), R316.2; no longer Q34.2 (S)
- net at R134.2: now also U28.2; no longer U28.1
Other:
- moved on the sheet: Q23, Q24, Q25, Q26, Q27, Q28, Q29, Q30, Q31, Q32, Q33, Q34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

Commit message: Updated 3D models
Parts:
- U26: renamed from U27; Мин. кол-во 1 -> 7; Ссылка https://www.chipdip.ru/product/tlp291-4-gb-tp-e-t -> https://www.promelec.ru/product/247137/; Цена 340 -> 76
- U27: renamed from U28; Мин. кол-во 1 -> 7; Ссылка https://www.chipdip.ru/product/tlp291-4-gb-tp-e-t -> https://www.promelec.ru/product/247137/; Цена 340 -> 76
- U29: renamed from U30; Мин. кол-во 1 -> 31; Ссылка https://www.chipdip.ru/product/tlp291-gb-tp-se-t -> https://www.promelec.ru/product/247129/; Цена 62 -> 17
- U30: renamed from U31; Мин. кол-во 1 -> 31; Ссылка https://www.chipdip.ru/product/tlp291-gb-tp-se-t -> https://www.promelec.ru/product/247129/; Цена 62 -> 17
- U31: renamed from U32; Мин. кол-во 1 -> 31; Ссылка https://www.chipdip.ru/product/tlp291-gb-tp-se-t -> https://www.promelec.ru/product/247129/; Цена 62 -> 17
- U32: renamed from U33; Мин. кол-во 1 -> 31; Ссылка https://www.chipdip.ru/product/tlp291-gb-tp-se-t -> https://www.promelec.ru/product/247129/; Цена 62 -> 17
- U33: renamed from U34; Мин. кол-во 1 -> 31; Ссылка https://www.chipdip.ru/product/tlp291-gb-tp-se-t -> https://www.promelec.ru/product/247129/; Цена 62 -> 17
- renumbered C85 to C100, C86 to C101, C87 to C102, C84 to C99, J11 to J18, J28 to J19, J12 to J20, J13 to J21, J14 to J22, Q23 to Q24, Q24 to Q25, Q25 to Q26, Q26 to Q27, Q27 to Q28, Q28 to Q29, Q29 to Q30, Q30 to Q31, Q31 to Q32, Q32 to Q33, Q33 to Q34, Q34 to Q35, Q35 to Q36, R115 to R141, R116 to R142, R305 to R143, R117 to R144, R119 to R145, R120 to R146, R118 to R147, R306 to R148, R121 to R149, R123 to R150, R124 to R151, R122 to R152, R307 to R153, R125 to R154, R127 to R155, R128 to R156, R126 to R157, R308 to R158, R129 to R159, R131 to R160, R132 to R161, R130 to R162, R309 to R163, R133 to R164, R134 to R165, R136 to R166, R137 to R167, R135 to R168, R310 to R169, R138 to R170, R140 to R171, R141 to R172, R139 to R173, R311 to R174, R142 to R175, R144 to R176, R145 to R177, R143 to R178, R312 to R179, R146 to R180, R147 to R181, R148 to R182, R149 to R183, R313 to R184, R150 to R185, R152 to R186, R153 to R187, R151 to R188, R314 to R189, R154 to R190, R155 to R191, R156 to R192, R157 to R193, R315 to R194, R158 to R195, R160 to R196, R161 to R197, R159 to R198, R316 to R199, R162 to R200, R164 to R201, R165 to R202, R163 to R203, R317 to R204, R166 to R205, R167 to R206, TP21 to TP34, TP22 to TP35, U29 to U28

Commit message: updated bom
Parts:
- renumbered C99 to C101, C100 to C102, C101 to C103, C102 to C104
Changed lines of the file:
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@@
 		(on_board yes)
 		(dnp no)
-		(property "Reference" "C99"
+		(property "Reference" "C101"
 			(at 243.205 100.33 0)
 			(effects
@@
 			(project "impeller18"
 				(path "/4ccab03b-4b1c-4c61-9fa8-19853ef32b4d/f8c6dd6a-e404-4019-a2ea-749009c88df2"
-					(reference "C99")
+					(reference "C101")
 					(unit 1)
 				)
@@
 		(on_board yes)
 		(dnp no)
-		(property "Reference" "C101"
+		(property "Reference" "C103"
 			(at 289.56 100.33 0)
 			(effects
@@
 			(project "impeller18"
 				(path "/4ccab03b-4b1c-4c61-9fa8-19853ef32b4d/f8c6dd6a-e404-4019-a2ea-749009c88df2"
-					(reference "C101")
+					(reference "C103")
 					(unit 1)
 				)
@@
 		(on_board yes)
 		(dnp no)
-		(property "Reference" "C100"
+		(property "Reference" "C102"
 			(at 252.73 100.33 0)
 			(effects
@@
 			(project "impeller18"
 				(path "/4ccab03b-4b1c-4c61-9fa8-19853ef32b4d/f8c6dd6a-e404-4019-a2ea-749009c88df2"
-					(reference "C100")
+					(reference "C102")
 					(unit 1)
 				)
@@
 		(on_board yes)
 		(dnp no)
-		(property "Reference" "C102"
+		(property "Reference" "C104"
 			(at 299.085 100.33 0)
 			(effects
@@
 			(project "impeller18"
 				(path "/4ccab03b-4b1c-4c61-9fa8-19853ef32b4d/f8c6dd6a-e404-4019-a2ea-749009c88df2"
-					(reference "C102")
+					(reference "C104")
 					(unit 1)
 				)

Commit message: PCB concept
Parts:
- J21: footprint user_lib:430454000 -> user_lib:430450400
Other:
- note added: "зачем 24 вольт?"
Changed lines of the file:
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@@
 		)
 	)
+	(polyline
+		(pts
+			(xy 300.99 179.705) (xy 300.99 217.17)
+		)
+		(stroke
+			(width 0)
+			(type default)
+		)
+	)
 	(wire
 		(pts
@@
 		)
 	)
+	(arc
+		(start 299.085 181.61)
+		(mid 299.9698 180.5898)
+		(end 300.99 179.705)
+		(stroke
+			(width 0)
+			(type default)
+		)
+		(fill
+			(type none)
+		)
+	)
+	(arc
+		(start 300.99 179.705)
+		(mid 302.0102 180.5898)
+		(end 302.895 181.61)
+		(stroke
+			(width 0)
+			(type default)
+		)
+		(fill
+			(type none)
+		)
+	)
 	(text "0.5 м\n"
 		(exclude_from_sim no)
@@
 		)
 	)
+	(text "зачем 24 вольт?"
+		(exclude_from_sim no)
+		(at 325.755 226.695 0)
+		(effects
+			(font
+				(size 12 12)
+				(thickness 2.4)
+				(bold yes)
+			)
+		)
+	)
 	(text " 14 м"
 		(exclude_from_sim no)
@@
 			)
 		)
-		(property "Footprint" "user_lib:430454000"
+		(property "Footprint" "user_lib:430450400"
 			(at 271.145 172.72 0)
 			(effects

Commit message: Update PCB concept
Connections:
- net SWITCH_3.1_EXT: now also J18.6 (Pin_6); no longer J18.1 (Pin_1), J19.1 (Pin_1)
- net SWITCH_3.2_EXT: now also J18.7 (Pin_7); no longer J18.3 (Pin_3), J19.3 (Pin_3)
- net SWITCH_3.3_EXT: now also J18.8 (Pin_8); no longer J18.5 (Pin_5), J19.5 (Pin_5)
- net SWITCH_3.4_EXT: now also J18.9 (Pin_9); no longer J18.7 (Pin_7), J19.7 (Pin_7)
- net SWITCH_3.5_EXT: now also J18.10 (Pin_10); no longer J18.9 (Pin_9), J19.2 (Pin_2)
- net SWITCH_3.6_EXT: now also J20.4 (Pin_4); no longer J19.4 (Pin_4), J20.1 (Pin_1)
- net SWITCH_3.7_EXT: now also J20.5 (Pin_5); no longer J19.6 (Pin_6), J20.3 (Pin_3)
- net SWITCH_3.8_EXT: now also J20.6 (Pin_6); no longer J19.8 (Pin_8), J20.5 (Pin_5)
- net SWITCH_3.9_EXT: now also J21.4 (Pin_4); no longer J21.1 (Pin_1)
- net SWITCH_4.1_EXT: now also J22.4 (Pin_4); no longer J22.1 (Pin_1)
- net SWITCH_4.2_EXT: now also J22.5 (Pin_5); no longer J22.3 (Pin_3)
- net SWITCH_4.3_EXT: now also J22.6 (Pin_6); no longer J22.5 (Pin_5)
- net VIN: now also J18.1 (Pin_1), J18.3 (Pin_3), J18.5 (Pin_5), J20.1 (Pin_1), J20.3 (Pin_3), J21.1 (Pin_1), J22.1 (Pin_1), J22.3 (Pin_3); no longer J18.10 (Pin_10), J18.6 (Pin_6), J18.8 (Pin_8), J20.4 (Pin_4), J20.6 (Pin_6), J21.4 (Pin_4), J22.4 (Pin_4), J22.6 (Pin_6)
