File: Hardware/ciam/impeller18/can.kicad_sch (KiCad schematic)
At the start: 66 parts, among them J24 PLS-5, J25 PLS-5, J5 430450400, J6 430450400, SW4 MSS-12D16, SW5 MSS-12D16, U11 ISO1050DUB, U12 ISO1050DUB, U13 MCP2515-I/SO, U14 B0505MT-1WR4, U15 ISO1050DUB, U16 ISO1050DUB, U17 MCP2515-I/SO, U18 B0505MT-1WR4, Y3 X322516MLB4SI, Y4 X322516MLB4SI

Commit message: Minor changes
Connections:
- net SPI0_RPi_MOSI renamed SPI1_RPi_MOSI
Other:
- moved on the sheet: D11, D9, R30, R34, TP15, TP16, TP19, TP20

Commit message: Updated packeges
Parts:
- J5, J6: footprint Connector_Molex:Molex_Micro-Fit_3.0_43045-0400_2x02_P3.00mm_Horizontal -> user_lib:430454000
- U11, U12, U15, U16: footprint Package_SO:SOP-8_6.62x9.15mm_P2.54mm -> user_lib:ISO1050DUB
Other:
- note added: "1.5 м"
Changed lines of the file:
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@@
 		)
 	)
+	(text "1.5 м"
+		(exclude_from_sim no)
+		(at 53.975 72.39 0)
+		(effects
+			(font
+				(size 12.7 12.7)
+				(bold yes)
+			)
+		)
+	)
+	(text "1.5 м"
+		(exclude_from_sim no)
+		(at 53.975 167.64 0)
+		(effects
+			(font
+				(size 12.7 12.7)
+				(bold yes)
+			)
+		)
+	)
 	(text "https://files.waveshare.com/upload/1/15/2-CH-CAN-HAT-Schematic.pdf\nшилд"
 		(exclude_from_sim no)
@@
 			)
 		)
-		(property "Footprint" "Package_SO:SOP-8_6.62x9.15mm_P2.54mm"
+		(property "Footprint" "user_lib:ISO1050DUB"
 			(at 176.53 50.165 0)
 			(effects
@@
 			)
 		)
-		(property "Footprint" "Package_SO:SOP-8_6.62x9.15mm_P2.54mm"
+		(property "Footprint" "user_lib:ISO1050DUB"
 			(at 176.53 150.495 0)
 			(effects
@@
 			)
 		)
-		(property "Footprint" "Package_SO:SOP-8_6.62x9.15mm_P2.54mm"
+		(property "Footprint" "user_lib:ISO1050DUB"
 			(at 176.53 78.74 0)
 			(effects
@@
 			)
 		)
-		(property "Footprint" "Connector_Molex:Molex_Micro-Fit_3.0_43045-0400_2x02_P3.00mm_Horizontal"
+		(property "Footprint" "user_lib:430454000"
 			(at 50.165 45.72 0)
 			(effects
@@
 			)
 		)
-		(property "Footprint" "Package_SO:SOP-8_6.62x9.15mm_P2.54mm"
+		(property "Footprint" "user_lib:ISO1050DUB"
 			(at 176.53 179.07 0)
 			(effects
@@
 			)
 		)
-		(property "Footprint" "Connector_Molex:Molex_Micro-Fit_3.0_43045-0400_2x02_P3.00mm_Horizontal"
+		(property "Footprint" "user_lib:430454000"
 			(at 50.165 146.05 0)
 			(effects

Commit message: Updated packeges
Parts:
- L2, L3: footprint (none) -> user_lib:B82790C0513N201
Changed lines of the file:
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@@
 			)
 		)
-		(property "Footprint" ""
+		(property "Footprint" "user_lib:B82790C0513N201"
 			(at 97.79 48.26 0)
 			(effects
@@
 			)
 		)
-		(property "Footprint" ""
+		(property "Footprint" "user_lib:B82790C0513N201"
 			(at 97.79 148.59 0)
 			(effects

Commit message: Updated 3D models
Parts:
- renumbered C47 to C62, C48 to C63, C49 to C64, C50 to C65, C51 to C66, C52 to C67, C53 to C68, C54 to C69, C55 to C70, C56 to C71, C57 to C72, C58 to C73, C59 to C74, C60 to C75, C61 to C76, C62 to C77, C63 to C78, C64 to C79, C65 to C80, C66 to C81, C67 to C82, C68 to C83, C69 to C84, C70 to C85, C71 to C86, C72 to C87, J24 to J10, J6 to J11, J25 to J12, J5 to J9, L2 to L3, L3 to L4, R27 to R35, R28 to R36, R29 to R37, R30 to R38, R31 to R39, R32 to R40, R33 to R41, R34 to R42, SW4 to SW8, SW5 to SW9, TP3 to TP20, TP4 to TP21, TP37 to TP22, TP15 to TP23, TP16 to TP24, TP5 to TP25, TP6 to TP26, TP38 to TP27, TP19 to TP28, TP20 to TP29, U11 to U10, U12 to U11, U13 to U12, U14 to U13, U15 to U14, U16 to U15, U17 to U16, U18 to U17

Commit message: updated bom
Parts:
- renumbered C62 to C64, C63 to C65, C64 to C66, C65 to C67, C66 to C68, C67 to C69, C68 to C70, C69 to C71, C70 to C72, C71 to C73, C72 to C74, C73 to C75, C74 to C76, C75 to C77, C76 to C78, C77 to C79, C78 to C80, C79 to C81, C80 to C82, C81 to C83, C82 to C84, C83 to C85, C84 to C86, C85 to C87, C86 to C88, C87 to C89
Changed lines of the file:
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@@
 		(on_board yes)
 		(dnp no)
-		(property "Reference" "C62"
+		(property "Reference" "C64"
 			(at 150.495 41.275 0)
 			(effects
@@
 			(project "impeller18"
 				(path "/4ccab03b-4b1c-4c61-9fa8-19853ef32b4d/ab594f26-bead-49a9-873a-c6155ff4b923"
-					(reference "C62")
+					(reference "C64")
 					(unit 1)
 				)
@@
 		(on_board yes)
 		(dnp no)
-		(property "Reference" "C72"
+		(property "Reference" "C74"
 			(at 159.385 99.06 0)
 			(effects
@@
 			(project "impeller18"
 				(path "/4ccab03b-4b1c-4c61-9fa8-19853ef32b4d/ab594f26-bead-49a9-873a-c6155ff4b923"
-					(reference "C72")
+					(reference "C74")
 					(unit 1)
 				)
@@
 		(on_board yes)
 		(dnp no)
-		(property "Reference" "C78"
+		(property "Reference" "C80"
 			(at 293.37 145.415 90)
 			(effects
@@
 			(project "impeller18"
 				(path "/4ccab03b-4b1c-4c61-9fa8-19853ef32b4d/ab594f26-bead-49a9-873a-c6155ff4b923"
-					(reference "C78")
+					(reference "C80")
 					(unit 1)
 				)
@@
 		(on_board yes)
 		(dnp no)
-		(property "Reference" "C85"
+		(property "Reference" "C87"
 			(at 159.385 199.39 0)
 			(effects
@@
 			(project "impeller18"
 				(path "/4ccab03b-4b1c-4c61-9fa8-19853ef32b4d/ab594f26-bead-49a9-873a-c6155ff4b923"
-					(reference "C85")
+					(reference "C87")
 					(unit 1)
 				)
@@
 		(on_board yes)
 		(dnp no)
-		(property "Reference" "C67"
+		(property "Reference" "C69"
 			(at 210.185 69.85 0)
 			(effects
@@
 			(project "impeller18"
 				(path "/4ccab03b-4b1c-4c61-9fa8-19853ef32b4d/ab594f26-bead-49a9-873a-c6155ff4b923"
-					(reference "C67")
+					(reference "C69")
 					(unit 1)
 				)
@@
 		(on_board yes)
 		(dnp no)
-		(property "Reference" "C65"
+		(property "Reference" "C67"
 			(at 293.37 45.085 90)
 			(effects
@@
 			(project "impeller18"
 				(path "/4ccab03b-4b1c-4c61-9fa8-19853ef32b4d/ab594f26-bead-49a9-873a-c6155ff4b923"
-					(reference "C65")
+					(reference "C67")
 					(unit 1)
 				)
@@
 		(on_board yes)
 		(dnp no)
-		(property "Reference" "C75"
+		(property "Reference" "C77"
 			(at 150.495 141.605 0)
 			(effects
@@
 			(project "impeller18"
 				(path "/4ccab03b-4b1c-4c61-9fa8-19853ef32b4d/ab594f26-bead-49a9-873a-c6155ff4b923"
-					(reference "C75")
+					(reference "C77")
 					(unit 1)
 				)
@@
 		(on_board yes)
 		(dnp no)
-		(property "Reference" "C87"
+		(property "Reference" "C89"
 			(at 205.74 199.39 0)
 			(effects
@@
 			(project "impeller18"
 				(path "/4ccab03b-4b1c-4c61-9fa8-19853ef32b4d/ab594f26-bead-49a9-873a-c6155ff4b923"
-					(reference "C87")
+					(reference "C89")
 					(unit 1)
 				)
@@
 		(on_board yes)
 		(dnp no)
-		(property "Reference" "C63"
+		(property "Reference" "C65"
 			(at 210.185 41.275 0)
 			(effects
@@
 			(project "impeller18"
 				(path "/4ccab03b-4b1c-4c61-9fa8-19853ef32b4d/ab594f26-bead-49a9-873a-c6155ff4b923"
-					(reference "C63")
+					(reference "C65")
 					(unit 1)
 				)
@@
 		(on_board yes)
 		(dnp no)
-		(property "Reference" "C84"
+		(property "Reference" "C86"
 			(at 149.86 199.39 0)
 			(effects
@@
 			(project "impeller18"
 				(path "/4ccab03b-4b1c-4c61-9fa8-19853ef32b4d/ab594f26-bead-49a9-873a-c6155ff4b923"
-					(reference "C84")
+					(reference "C86")
 					(unit 1)
 				)
@@
 		(on_board yes)
 		(dnp no)
-		(property "Reference" "C73"
+		(property "Reference" "C75"
 			(at 196.215 99.06 0)
 			(effects
@@
 			(project "impeller18"
 				(path "/4ccab03b-4b1c-4c61-9fa8-19853ef32b4d/ab594f26-bead-49a9-873a-c6155ff4b923"
-					(reference "C73")
+					(reference "C75")
 					(unit 1)
 				)
@@
 		(on_board yes)
 		(dnp no)
-		(property "Reference" "C69"
+		(property "Reference" "C71"
 			(at 245.745 72.39 90)
 			(effects
@@
 			(project "impeller18"
 				(path "/4ccab03b-4b1c-4c61-9fa8-19853ef32b4d/ab594f26-bead-49a9-873a-c6155ff4b923"
-					(reference "C69")
+					(reference "C71")
 					(unit 1)
 				)
@@
 		(on_board yes)
 		(dnp no)
-		(property "Reference" "C83"
+		(property "Reference" "C85"
 			(at 245.745 180.34 90)
 			(effects
@@
 			(project "impeller18"
 				(path "/4ccab03b-4b1c-4c61-9fa8-19853ef32b4d/ab594f26-bead-49a9-873a-c6155ff4b923"
-					(reference "C83")
+					(reference "C85")
 					(unit 1)
 				)
@@
 		(on_board yes)
 		(dnp no)
-		(property "Reference" "C80"
+		(property "Reference" "C82"
 			(at 210.185 170.18 0)
 			(effects
@@
 			(project "impeller18"
 				(path "/4ccab03b-4b1c-4c61-9fa8-19853ef32b4d/ab594f26-bead-49a9-873a-c6155ff4b923"
-					(reference "C80")
+					(reference "C82")
 					(unit 1)
 				)
@@
 		(on_board yes)
 		(dnp no)
-		(property "Reference" "C68"
+		(property "Reference" "C70"
 			(at 219.075 69.85 0)
 			(effects
@@
 			(project "impeller18"
 				(path "/4ccab03b-4b1c-4c61-9fa8-19853ef32b4d/ab594f26-bead-49a9-873a-c6155ff4b923"
-					(reference "C68")
+					(reference "C70")
 					(unit 1)
 				)
@@
 		(on_board yes)
 		(dnp no)
-		(property "Reference" "C82"
+		(property "Reference" "C84"
 			(at 245.745 172.72 90)
 			(effects
@@
 			(project "impeller18"
 				(path "/4ccab03b-4b1c-4c61-9fa8-19853ef32b4d/ab594f26-bead-49a9-873a-c6155ff4b923"
-					(reference "C82")
+					(reference "C84")
 					(unit 1)
 				)
@@
 		(on_board yes)
 		(dnp no)
-		(property "Reference" "C79"
+		(property "Reference" "C81"
 			(at 150.495 170.18 0)
 			(effects
@@
 			(project "impeller18"
 				(path "/4ccab03b-4b1c-4c61-9fa8-19853ef32b4d/ab594f26-bead-49a9-873a-c6155ff4b923"
-					(reference "C79")
+					(reference "C81")
 					(unit 1)
 				)
@@
 		(on_board yes)
 		(dnp no)
-		(property "Reference" "C71"
+		(property "Reference" "C73"
 			(at 149.86 99.06 0)
 			(effects
@@
 			(project "impeller18"
 				(path "/4ccab03b-4b1c-4c61-9fa8-19853ef32b4d/ab594f26-bead-49a9-873a-c6155ff4b923"
-					(reference "C71")
+					(reference "C73")
 					(unit 1)
 				)
@@
 		(on_board yes)
 		(dnp no)
-		(property "Reference" "C70"
+		(property "Reference" "C72"
 			(at 245.745 80.01 90)
 			(effects
@@
 			(project "impeller18"
 				(path "/4ccab03b-4b1c-4c61-9fa8-19853ef32b4d/ab594f26-bead-49a9-873a-c6155ff4b923"
-					(reference "C70")
+					(reference "C72")
 					(unit 1)
 				)
@@
 		(on_board yes)
 		(dnp no)
-		(property "Reference" "C77"
+		(property "Reference" "C79"
 			(at 219.075 141.605 0)
 			(effects
@@
 			(project "impeller18"
 				(path "/4ccab03b-4b1c-4c61-9fa8-19853ef32b4d/ab594f26-bead-49a9-873a-c6155ff4b923"
-					(reference "C77")
+					(reference "C79")
 					(unit 1)
 				)
@@
 		(on_board yes)
 		(dnp no)
-		(property "Reference" "C74"
+		(property "Reference" "C76"
 			(at 205.74 99.06 0)
 			(effects
@@
 			(project "impeller18"
 				(path "/4ccab03b-4b1c-4c61-9fa8-19853ef32b4d/ab594f26-bead-49a9-873a-c6155ff4b923"
-					(reference "C74")
+					(reference "C76")
 					(unit 1)
 				)
@@
 		(on_board yes)
 		(dnp no)
-		(property "Reference" "C81"
+		(property "Reference" "C83"
 			(at 219.075 170.18 0)
 			(effects
@@
 			(project "impeller18"
 				(path "/4ccab03b-4b1c-4c61-9fa8-19853ef32b4d/ab594f26-bead-49a9-873a-c6155ff4b923"
-					(reference "C81")
+					(reference "C83")
 					(unit 1)
 				)
@@
 		(on_board yes)
 		(dnp no)
-		(property "Reference" "C64"
+		(property "Reference" "C66"
 			(at 219.075 41.275 0)
 			(effects
@@
 			(project "impeller18"
 				(path "/4ccab03b-4b1c-4c61-9fa8-19853ef32b4d/ab594f26-bead-49a9-873a-c6155ff4b923"
-					(reference "C64")
+					(reference "C66")
 					(unit 1)
 				)
@@
 		(on_board yes)
 		(dnp no)
-		(property "Reference" "C66"
+		(property "Reference" "C68"
 			(at 150.495 69.85 0)
 			(effects
@@
 			(project "impeller18"
 				(path "/4ccab03b-4b1c-4c61-9fa8-19853ef32b4d/ab594f26-bead-49a9-873a-c6155ff4b923"
-					(reference "C66")
+					(reference "C68")
 					(unit 1)
 				)
@@
 		(on_board yes)
 		(dnp no)
-		(property "Reference" "C86"
+		(property "Reference" "C88"
 			(at 196.215 199.39 0)
 			(effects
@@
 			(project "impeller18"
 				(path "/4ccab03b-4b1c-4c61-9fa8-19853ef32b4d/ab594f26-bead-49a9-873a-c6155ff4b923"
-					(reference "C86")
+					(reference "C88")
 					(unit 1)
 				)
@@
 		(on_board yes)
 		(dnp no)
-		(property "Reference" "C76"
+		(property "Reference" "C78"
 			(at 210.185 141.605 0)
 			(effects
@@
 			(project "impeller18"
 				(path "/4ccab03b-4b1c-4c61-9fa8-19853ef32b4d/ab594f26-bead-49a9-873a-c6155ff4b923"
-					(reference "C76")
+					(reference "C78")
 					(unit 1)
 				)

Commit message: PCB concept
Parts:
- added TP46: TestPoint, TestPoint:TestPoint_THTPad_D1.5mm_Drill0.7mm, symbol Connector:TestPoint
- J11, J9: footprint user_lib:430454000 -> user_lib:430450400
Connections:
- net GND: now also TP46.1
Changed lines of the file:
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@@
 	(wire
 		(pts
+			(xy 267.97 204.47) (xy 267.97 198.755)
+		)
+		(stroke
+			(width 0)
+			(type default)
+		)
+	)
+	(wire
+		(pts
 			(xy 121.92 87.63) (xy 121.92 90.17)
 		)
@@
 			)
 		)
-		(property "Footprint" "user_lib:430454000"
+		(property "Footprint" "user_lib:430450400"
 			(at 50.165 45.72 0)
 			(effects
@@
 	)
 	(symbol
+		(lib_id "Connector:TestPoint")
+		(at 267.97 198.755 0)
+		(unit 1)
+		(exclude_from_sim no)
+		(in_bom yes)
+		(on_board yes)
+		(dnp no)
+		(property "Reference" "TP46"
+			(at 266.065 191.77 0)
+			(effects
+				(font
+					(size 1.27 1.27)
+				)
+				(justify left)
+			)
+		)
+		(property "Value" "TestPoint"
+			(at 263.525 193.675 0)
+			(effects
+				(font
+					(size 1.27 1.27)
+				)
+				(justify left)
+			)
+		)
+		(property "Footprint" "TestPoint:TestPoint_THTPad_D1.5mm_Drill0.7mm"
+			(at 273.05 198.755 0)
+			(effects
+				(font
+					(size 1.27 1.27)
+				)
+				(hide yes)
+			)
+		)
+		(property "Datasheet" "~"
+			(at 273.05 198.755 0)
+			(effects
+				(font
+					(size 1.27 1.27)
+				)
+				(hide yes)
+			)
+		)
+		(property "Description" "test point"
+			(at 267.97 198.755 0)
+			(effects
+				(font
+					(size 1.27 1.27)
+				)
+				(hide yes)
+			)
+		)
+		(pin "1"
+		)
+		(instances
+			(project "impeller18"
+				(path "/4ccab03b-4b1c-4c61-9fa8-19853ef32b4d/ab594f26-bead-49a9-873a-c6155ff4b923"
+					(reference "TP46")
+					(unit 1)
+				)
+			)
+		)
+	)
+	(symbol
 		(lib_id "power:+5V")
 		(at 203.835 94.615 0)
@@
 	)
 	(symbol
+		(lib_id "power:GND")
+		(at 267.97 204.47 0)
+		(unit 1)
+		(exclude_from_sim no)
+		(in_bom yes)
+		(on_board yes)
+		(dnp no)
+		(property "Reference" "#PWR0303"
+			(at 267.97 210.82 0)
+			(effects
+				(font
+					(size 1.27 1.27)
+				)
+				(hide yes)
+			)
+		)
+		(property "Value" "GND"
+			(at 267.97 208.28 0)
+			(effects
+				(font
+					(size 1.27 1.27)
+				)
+			)
+		)
+		(property "Footprint" ""
+			(at 267.97 204.47 0)
+			(effects
+				(font
+					(size 1.27 1.27)
+				)
+				(hide yes)
+			)
+		)
+		(property "Datasheet" ""
+			(at 267.97 204.47 0)
+			(effects
+				(font
+					(size 1.27 1.27)
+				)
+				(hide yes)
+			)
+		)
+		(property "Description" ""
+			(at 267.97 204.47 0)
+			(effects
+				(font
+					(size 1.27 1.27)
+				)
+				(hide yes)
+			)
+		)
+		(pin "1"
+		)
+		(instances
+			(project "impeller18"
+				(path "/4ccab03b-4b1c-4c61-9fa8-19853ef32b4d/ab594f26-bead-49a9-873a-c6155ff4b923"
+					(reference "#PWR0303")
+					(unit 1)
+				)
+			)
+		)
+	)
+	(symbol
 		(lib_id "Device:R_Small")
 		(at 121.92 194.31 180)
@@
 			)
 		)
-		(property "Footprint" "user_lib:430454000"
+		(property "Footprint" "user_lib:430450400"
 			(at 50.165 146.05 0)
 			(effects

Commit message: Update PCB concept
Connections:
- net CAN0-: now also J9.3 (Pin_3); no longer J9.2 (Pin_2)
- net CAN1-: now also J11.3 (Pin_3); no longer J11.2 (Pin_2)
- net GND_CAN0: now also J9.2 (Pin_2); no longer J9.3 (Pin_3)
- net GND_CAN1: now also J11.2 (Pin_2); no longer J11.3 (Pin_3)
Changed lines of the file:
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@@
 	)
 	(symbol
+		(lib_name "Conn_02x02_Odd_Even_1")
 		(lib_id "Connector_Generic:Conn_02x02_Odd_Even")
 		(at 50.165 45.72 0)

Commit message: Daily PCB update
Parts:
- renumbered R35 to R39, R36 to R40, R37 to R41, R38 to R42, R39 to R43, R40 to R44, R41 to R45, R42 to R46, TP46 to TP29, TP29 to TP30
