File: Hardware/ciam/impeller18/digital_inputs.kicad_sch (KiCad schematic)
At the start: 19 parts, among them J8 430451600, U39 TLP291-4, U40 TLP291-4

Commit message: updated schematics
Parts:
- renumbered J8 to J13, R171 to R189, R172 to R190, R173 to R191, R174 to R192, R175 to R193, R176 to R194, R177 to R195, R178 to R196, R179 to R197, R180 to R198, R181 to R199, R182 to R200, R183 to R201, R184 to R202, R185 to R203, R186 to R204, U39 to U51, U40 to U52
Changed lines of the file:
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@@
 		(on_board yes)
 		(dnp no)
-		(property "Reference" "R176"
+		(property "Reference" "R194"
 			(at 111.76 78.105 90)
 			(effects
@@
 			(project "impeller18"
 				(path "/4ccab03b-4b1c-4c61-9fa8-19853ef32b4d/f0192a6c-39ea-409b-b3a4-616780c2a8a3"
-					(reference "R176")
+					(reference "R194")
 					(unit 1)
 				)
@@
 		(on_board yes)
 		(dnp no)
-		(property "Reference" "U39"
+		(property "Reference" "U51"
 			(at 87.63 88.9 0)
 			(effects
@@
 			(project "impeller18"
 				(path "/4ccab03b-4b1c-4c61-9fa8-19853ef32b4d/f0192a6c-39ea-409b-b3a4-616780c2a8a3"
-					(reference "U39")
+					(reference "U51")
 					(unit 4)
 				)
@@
 		(on_board yes)
 		(dnp no)
-		(property "Reference" "R179"
+		(property "Reference" "R197"
 			(at 74.295 104.775 90)
 			(effects
@@
 			(project "impeller18"
 				(path "/4ccab03b-4b1c-4c61-9fa8-19853ef32b4d/f0192a6c-39ea-409b-b3a4-616780c2a8a3"
-					(reference "R179")
+					(reference "R197")
 					(unit 1)
 				)
@@
 		(dnp no)
 		(fields_autoplaced yes)
-		(property "Reference" "J8"
+		(property "Reference" "J13"
 			(at 97.155 172.72 0)
 			(effects
@@
 			(project "impeller18"
 				(path "/4ccab03b-4b1c-4c61-9fa8-19853ef32b4d/f0192a6c-39ea-409b-b3a4-616780c2a8a3"
-					(reference "J8")
+					(reference "J13")
 					(unit 1)
 				)
@@
 		(on_board yes)
 		(dnp no)
-		(property "Reference" "R185"
+		(property "Reference" "R203"
 			(at 74.295 144.78 90)
 			(effects
@@
 			(project "impeller18"
 				(path "/4ccab03b-4b1c-4c61-9fa8-19853ef32b4d/f0192a6c-39ea-409b-b3a4-616780c2a8a3"
-					(reference "R185")
+					(reference "R203")
 					(unit 1)
 				)
@@
 		(on_board yes)
 		(dnp no)
-		(property "Reference" "R174"
+		(property "Reference" "R192"
 			(at 111.76 64.77 90)
 			(effects
@@
 			(project "impeller18"
 				(path "/4ccab03b-4b1c-4c61-9fa8-19853ef32b4d/f0192a6c-39ea-409b-b3a4-616780c2a8a3"
-					(reference "R174")
+					(reference "R192")
 					(unit 1)
 				)
@@
 		(on_board yes)
 		(dnp no)
-		(property "Reference" "U39"
+		(property "Reference" "U51"
 			(at 87.63 48.895 0)
 			(effects
@@
 			(project "impeller18"
 				(path "/4ccab03b-4b1c-4c61-9fa8-19853ef32b4d/f0192a6c-39ea-409b-b3a4-616780c2a8a3"
-					(reference "U39")
+					(reference "U51")
 					(unit 1)
 				)
@@
 		(on_board yes)
 		(dnp no)
-		(property "Reference" "U40"
+		(property "Reference" "U52"
 			(at 87.63 115.57 0)
 			(effects
@@
 			(project "impeller18"
 				(path "/4ccab03b-4b1c-4c61-9fa8-19853ef32b4d/f0192a6c-39ea-409b-b3a4-616780c2a8a3"
-					(reference "U40")
+					(reference "U52")
 					(unit 2)
 				)
@@
 		(on_board yes)
 		(dnp no)
-		(property "Reference" "U39"
+		(property "Reference" "U51"
 			(at 87.63 75.565 0)
 			(effects
@@
 			(project "impeller18"
 				(path "/4ccab03b-4b1c-4c61-9fa8-19853ef32b4d/f0192a6c-39ea-409b-b3a4-616780c2a8a3"
-					(reference "U39")
+					(reference "U51")
 					(unit 3)
 				)
@@
 		(on_board yes)
 		(dnp no)
-		(property "Reference" "R186"
+		(property "Reference" "R204"
 			(at 111.76 144.78 90)
 			(effects
@@
 			(project "impeller18"
 				(path "/4ccab03b-4b1c-4c61-9fa8-19853ef32b4d/f0192a6c-39ea-409b-b3a4-616780c2a8a3"
-					(reference "R186")
+					(reference "R204")
 					(unit 1)
 				)
@@
 		(on_board yes)
 		(dnp no)
-		(property "Reference" "R180"
+		(property "Reference" "R198"
 			(at 111.76 104.775 90)
 			(effects
@@
 			(project "impeller18"
 				(path "/4ccab03b-4b1c-4c61-9fa8-19853ef32b4d/f0192a6c-39ea-409b-b3a4-616780c2a8a3"
-					(reference "R180")
+					(reference "R198")
 					(unit 1)
 				)
@@
 		(on_board yes)
 		(dnp no)
-		(property "Reference" "R175"
+		(property "Reference" "R193"
 			(at 74.295 78.105 90)
 			(effects
@@
 			(project "impeller18"
 				(path "/4ccab03b-4b1c-4c61-9fa8-19853ef32b4d/f0192a6c-39ea-409b-b3a4-616780c2a8a3"
-					(reference "R175")
+					(reference "R193")
 					(unit 1)
 				)
@@
 		(on_board yes)
 		(dnp no)
-		(property "Reference" "U40"
+		(property "Reference" "U52"
 			(at 87.63 142.24 0)
 			(effects
@@
 			(project "impeller18"
 				(path "/4ccab03b-4b1c-4c61-9fa8-19853ef32b4d/f0192a6c-39ea-409b-b3a4-616780c2a8a3"
-					(reference "U40")
+					(reference "U52")
 					(unit 4)
 				)
@@
 		(on_board yes)
 		(dnp no)
-		(property "Reference" "R177"
+		(property "Reference" "R195"
 			(at 74.295 91.44 90)
 			(effects
@@
 			(project "impeller18"
 				(path "/4ccab03b-4b1c-4c61-9fa8-19853ef32b4d/f0192a6c-39ea-409b-b3a4-616780c2a8a3"
-					(reference "R177")
+					(reference "R195")
 					(unit 1)
 				)
@@
 		(on_board yes)
 		(dnp no)
-		(property "Reference" "U40"
+		(property "Reference" "U52"
 			(at 87.63 102.235 0)
 			(effects
@@
 			(project "impeller18"
 				(path "/4ccab03b-4b1c-4c61-9fa8-19853ef32b4d/f0192a6c-39ea-409b-b3a4-616780c2a8a3"
-					(reference "U40")
+					(reference "U52")
 					(unit 1)
 				)
@@
 		(on_board yes)
 		(dnp no)
-		(property "Reference" "R184"
+		(property "Reference" "R202"
 			(at 111.76 131.445 90)
 			(effects
@@
 			(project "impeller18"
 				(path "/4ccab03b-4b1c-4c61-9fa8-19853ef32b4d/f0192a6c-39ea-409b-b3a4-616780c2a8a3"
-					(reference "R184")
+					(reference "R202")
 					(unit 1)
 				)
@@
 		(on_board yes)
 		(dnp no)
-		(property "Reference" "R172"
+		(property "Reference" "R190"
 			(at 111.76 51.435 90)
 			(effects
@@
 			(project "impeller18"
 				(path "/4ccab03b-4b1c-4c61-9fa8-19853ef32b4d/f0192a6c-39ea-409b-b3a4-616780c2a8a3"
-					(reference "R172")
+					(reference "R190")
 					(unit 1)
 				)
@@
 		(on_board yes)
 		(dnp no)
-		(property "Reference" "R171"
+		(property "Reference" "R189"
 			(at 74.295 51.435 90)
 			(effects
@@
 			(project "impeller18"
 				(path "/4ccab03b-4b1c-4c61-9fa8-19853ef32b4d/f0192a6c-39ea-409b-b3a4-616780c2a8a3"
-					(reference "R171")
+					(reference "R189")
 					(unit 1)
 				)
@@
 		(on_board yes)
 		(dnp no)
-		(property "Reference" "U40"
+		(property "Reference" "U52"
 			(at 87.63 128.905 0)
 			(effects
@@
 			(project "impeller18"
 				(path "/4ccab03b-4b1c-4c61-9fa8-19853ef32b4d/f0192a6c-39ea-409b-b3a4-616780c2a8a3"
-					(reference "U40")
+					(reference "U52")
 					(unit 3)
 				)
@@
 		(on_board yes)
 		(dnp no)
-		(property "Reference" "U39"
+		(property "Reference" "U51"
 			(at 87.63 62.23 0)
 			(effects
@@
 			(project "impeller18"
 				(path "/4ccab03b-4b1c-4c61-9fa8-19853ef32b4d/f0192a6c-39ea-409b-b3a4-616780c2a8a3"
-					(reference "U39")
+					(reference "U51")
 					(unit 2)
 				)
@@
 		(on_board yes)
 		(dnp no)
-		(property "Reference" "R173"
+		(property "Reference" "R191"
 			(at 74.295 64.77 90)
 			(effects
@@
 			(project "impeller18"
 				(path "/4ccab03b-4b1c-4c61-9fa8-19853ef32b4d/f0192a6c-39ea-409b-b3a4-616780c2a8a3"
-					(reference "R173")
+					(reference "R191")
 					(unit 1)
 				)
@@
 		(on_board yes)
 		(dnp no)
-		(property "Reference" "R183"
+		(property "Reference" "R201"
 			(at 74.295 131.445 90)
 			(effects
@@
 			(project "impeller18"
 				(path "/4ccab03b-4b1c-4c61-9fa8-19853ef32b4d/f0192a6c-39ea-409b-b3a4-616780c2a8a3"
-					(reference "R183")
+					(reference "R201")
 					(unit 1)
 				)
@@
 		(on_board yes)
 		(dnp no)
-		(property "Reference" "R181"
+		(property "Reference" "R199"
 			(at 74.295 118.11 90)
 			(effects
@@
 			(project "impeller18"
 				(path "/4ccab03b-4b1c-4c61-9fa8-19853ef32b4d/f0192a6c-39ea-409b-b3a4-616780c2a8a3"
-					(reference "R181")
+					(reference "R199")
 					(unit 1)
 				)
@@
 		(on_board yes)
 		(dnp no)
-		(property "Reference" "R182"
+		(property "Reference" "R200"
 			(at 111.76 118.11 90)
 			(effects
@@
 			(project "impeller18"
 				(path "/4ccab03b-4b1c-4c61-9fa8-19853ef32b4d/f0192a6c-39ea-409b-b3a4-616780c2a8a3"
-					(reference "R182")
+					(reference "R200")
 					(unit 1)
 				)
@@
 		(on_board yes)
 		(dnp no)
-		(property "Reference" "#PWR0124"
+		(property "Reference" "#PWR0176"
 			(at 99.695 161.29 0)
 			(effects
@@
 			(project "impeller18"
 				(path "/4ccab03b-4b1c-4c61-9fa8-19853ef32b4d/f0192a6c-39ea-409b-b3a4-616780c2a8a3"
-					(reference "#PWR0124")
+					(reference "#PWR0176")
 					(unit 1)
 				)
@@
 		(on_board yes)
 		(dnp no)
-		(property "Reference" "R178"
+		(property "Reference" "R196"
 			(at 111.76 91.44 90)
 			(effects
@@
 			(project "impeller18"
 				(path "/4ccab03b-4b1c-4c61-9fa8-19853ef32b4d/f0192a6c-39ea-409b-b3a4-616780c2a8a3"
-					(reference "R178")
+					(reference "R196")
 					(unit 1)
 				)
@@
 		(dnp no)
 		(fields_autoplaced yes)
-		(property "Reference" "#PWR0123"
+		(property "Reference" "#PWR0175"
 			(at 135.255 54.61 0)
 			(effects
@@
 			(project "impeller18"
 				(path "/4ccab03b-4b1c-4c61-9fa8-19853ef32b4d/f0192a6c-39ea-409b-b3a4-616780c2a8a3"
-					(reference "#PWR0123")
-					(unit 1)
-				)
+					(reference "#PWR0175")
+					(unit 1)
+				)

Commit message: updated schematics
Parts:
- renumbered J13 to J16, R189 to R210, R190 to R211, R191 to R212, R192 to R213, R193 to R214, R194 to R215, R195 to R216, R196 to R217, R197 to R218, R198 to R219, R199 to R220, R200 to R221, R201 to R222, R202 to R223, R203 to R224, R204 to R225, U51 to U62, U52 to U63
Changed lines of the file:
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@@
 		(on_board yes)
 		(dnp no)
-		(property "Reference" "R194"
+		(property "Reference" "R215"
 			(at 111.76 78.105 90)
 			(effects
@@
 			(project "impeller18"
 				(path "/4ccab03b-4b1c-4c61-9fa8-19853ef32b4d/f0192a6c-39ea-409b-b3a4-616780c2a8a3"
-					(reference "R194")
+					(reference "R215")
 					(unit 1)
 				)
@@
 		(on_board yes)
 		(dnp no)
-		(property "Reference" "U51"
+		(property "Reference" "U62"
 			(at 87.63 88.9 0)
 			(effects
@@
 			(project "impeller18"
 				(path "/4ccab03b-4b1c-4c61-9fa8-19853ef32b4d/f0192a6c-39ea-409b-b3a4-616780c2a8a3"
-					(reference "U51")
+					(reference "U62")
 					(unit 4)
 				)
@@
 		(on_board yes)
 		(dnp no)
-		(property "Reference" "R197"
+		(property "Reference" "R218"
 			(at 74.295 104.775 90)
 			(effects
@@
 			(project "impeller18"
 				(path "/4ccab03b-4b1c-4c61-9fa8-19853ef32b4d/f0192a6c-39ea-409b-b3a4-616780c2a8a3"
-					(reference "R197")
+					(reference "R218")
 					(unit 1)
 				)
@@
 		(dnp no)
 		(fields_autoplaced yes)
-		(property "Reference" "J13"
+		(property "Reference" "J16"
 			(at 97.155 172.72 0)
 			(effects
@@
 			(project "impeller18"
 				(path "/4ccab03b-4b1c-4c61-9fa8-19853ef32b4d/f0192a6c-39ea-409b-b3a4-616780c2a8a3"
-					(reference "J13")
+					(reference "J16")
 					(unit 1)
 				)
@@
 		(on_board yes)
 		(dnp no)
-		(property "Reference" "R203"
+		(property "Reference" "R224"
 			(at 74.295 144.78 90)
 			(effects
@@
 			(project "impeller18"
 				(path "/4ccab03b-4b1c-4c61-9fa8-19853ef32b4d/f0192a6c-39ea-409b-b3a4-616780c2a8a3"
-					(reference "R203")
+					(reference "R224")
 					(unit 1)
 				)
@@
 		(on_board yes)
 		(dnp no)
-		(property "Reference" "R192"
+		(property "Reference" "R213"
 			(at 111.76 64.77 90)
 			(effects
@@
 			(project "impeller18"
 				(path "/4ccab03b-4b1c-4c61-9fa8-19853ef32b4d/f0192a6c-39ea-409b-b3a4-616780c2a8a3"
-					(reference "R192")
+					(reference "R213")
 					(unit 1)
 				)
@@
 		(on_board yes)
 		(dnp no)
-		(property "Reference" "U51"
+		(property "Reference" "U62"
 			(at 87.63 48.895 0)
 			(effects
@@
 			(project "impeller18"
 				(path "/4ccab03b-4b1c-4c61-9fa8-19853ef32b4d/f0192a6c-39ea-409b-b3a4-616780c2a8a3"
-					(reference "U51")
+					(reference "U62")
 					(unit 1)
 				)
@@
 		(on_board yes)
 		(dnp no)
-		(property "Reference" "U52"
+		(property "Reference" "U63"
 			(at 87.63 115.57 0)
 			(effects
@@
 			(project "impeller18"
 				(path "/4ccab03b-4b1c-4c61-9fa8-19853ef32b4d/f0192a6c-39ea-409b-b3a4-616780c2a8a3"
-					(reference "U52")
+					(reference "U63")
 					(unit 2)
 				)
@@
 		(on_board yes)
 		(dnp no)
-		(property "Reference" "U51"
+		(property "Reference" "U62"
 			(at 87.63 75.565 0)
 			(effects
@@
 			(project "impeller18"
 				(path "/4ccab03b-4b1c-4c61-9fa8-19853ef32b4d/f0192a6c-39ea-409b-b3a4-616780c2a8a3"
-					(reference "U51")
+					(reference "U62")
 					(unit 3)
 				)
@@
 		(on_board yes)
 		(dnp no)
-		(property "Reference" "R204"
+		(property "Reference" "R225"
 			(at 111.76 144.78 90)
 			(effects
@@
 			(project "impeller18"
 				(path "/4ccab03b-4b1c-4c61-9fa8-19853ef32b4d/f0192a6c-39ea-409b-b3a4-616780c2a8a3"
-					(reference "R204")
+					(reference "R225")
 					(unit 1)
 				)
@@
 		(on_board yes)
 		(dnp no)
-		(property "Reference" "R198"
+		(property "Reference" "R219"
 			(at 111.76 104.775 90)
 			(effects
@@
 			(project "impeller18"
 				(path "/4ccab03b-4b1c-4c61-9fa8-19853ef32b4d/f0192a6c-39ea-409b-b3a4-616780c2a8a3"
-					(reference "R198")
+					(reference "R219")
 					(unit 1)
 				)
@@
 		(on_board yes)
 		(dnp no)
-		(property "Reference" "R193"
+		(property "Reference" "R214"
 			(at 74.295 78.105 90)
 			(effects
@@
 			(project "impeller18"
 				(path "/4ccab03b-4b1c-4c61-9fa8-19853ef32b4d/f0192a6c-39ea-409b-b3a4-616780c2a8a3"
-					(reference "R193")
+					(reference "R214")
 					(unit 1)
 				)
@@
 		(on_board yes)
 		(dnp no)
-		(property "Reference" "U52"
+		(property "Reference" "U63"
 			(at 87.63 142.24 0)
 			(effects
@@
 			(project "impeller18"
 				(path "/4ccab03b-4b1c-4c61-9fa8-19853ef32b4d/f0192a6c-39ea-409b-b3a4-616780c2a8a3"
-					(reference "U52")
+					(reference "U63")
 					(unit 4)
 				)
@@
 		(on_board yes)
 		(dnp no)
-		(property "Reference" "R195"
+		(property "Reference" "R216"
 			(at 74.295 91.44 90)
 			(effects
@@
 			(project "impeller18"
 				(path "/4ccab03b-4b1c-4c61-9fa8-19853ef32b4d/f0192a6c-39ea-409b-b3a4-616780c2a8a3"
-					(reference "R195")
+					(reference "R216")
 					(unit 1)
 				)
@@
 		(on_board yes)
 		(dnp no)
-		(property "Reference" "U52"
+		(property "Reference" "U63"
 			(at 87.63 102.235 0)
 			(effects
@@
 			(project "impeller18"
 				(path "/4ccab03b-4b1c-4c61-9fa8-19853ef32b4d/f0192a6c-39ea-409b-b3a4-616780c2a8a3"
-					(reference "U52")
+					(reference "U63")
 					(unit 1)
 				)
@@
 		(on_board yes)
 		(dnp no)
-		(property "Reference" "R202"
+		(property "Reference" "R223"
 			(at 111.76 131.445 90)
 			(effects
@@
 			(project "impeller18"
 				(path "/4ccab03b-4b1c-4c61-9fa8-19853ef32b4d/f0192a6c-39ea-409b-b3a4-616780c2a8a3"
-					(reference "R202")
+					(reference "R223")
 					(unit 1)
 				)
@@
 		(on_board yes)
 		(dnp no)
-		(property "Reference" "R190"
+		(property "Reference" "R211"
 			(at 111.76 51.435 90)
 			(effects
@@
 			(project "impeller18"
 				(path "/4ccab03b-4b1c-4c61-9fa8-19853ef32b4d/f0192a6c-39ea-409b-b3a4-616780c2a8a3"
-					(reference "R190")
+					(reference "R211")
 					(unit 1)
 				)
@@
 		(on_board yes)
 		(dnp no)
-		(property "Reference" "R189"
+		(property "Reference" "R210"
 			(at 74.295 51.435 90)
 			(effects
@@
 			(project "impeller18"
 				(path "/4ccab03b-4b1c-4c61-9fa8-19853ef32b4d/f0192a6c-39ea-409b-b3a4-616780c2a8a3"
-					(reference "R189")
+					(reference "R210")
 					(unit 1)
 				)
@@
 		(on_board yes)
 		(dnp no)
-		(property "Reference" "U52"
+		(property "Reference" "U63"
 			(at 87.63 128.905 0)
 			(effects
@@
 			(project "impeller18"
 				(path "/4ccab03b-4b1c-4c61-9fa8-19853ef32b4d/f0192a6c-39ea-409b-b3a4-616780c2a8a3"
-					(reference "U52")
+					(reference "U63")
 					(unit 3)
 				)
@@
 		(on_board yes)
 		(dnp no)
-		(property "Reference" "U51"
+		(property "Reference" "U62"
 			(at 87.63 62.23 0)
 			(effects
@@
 			(project "impeller18"
 				(path "/4ccab03b-4b1c-4c61-9fa8-19853ef32b4d/f0192a6c-39ea-409b-b3a4-616780c2a8a3"
-					(reference "U51")
+					(reference "U62")
 					(unit 2)
 				)
@@
 		(on_board yes)
 		(dnp no)
-		(property "Reference" "R191"
+		(property "Reference" "R212"
 			(at 74.295 64.77 90)
 			(effects
@@
 			(project "impeller18"
 				(path "/4ccab03b-4b1c-4c61-9fa8-19853ef32b4d/f0192a6c-39ea-409b-b3a4-616780c2a8a3"
-					(reference "R191")
+					(reference "R212")
 					(unit 1)
 				)
@@
 		(on_board yes)
 		(dnp no)
-		(property "Reference" "R201"
+		(property "Reference" "R222"
 			(at 74.295 131.445 90)
 			(effects
@@
 			(project "impeller18"
 				(path "/4ccab03b-4b1c-4c61-9fa8-19853ef32b4d/f0192a6c-39ea-409b-b3a4-616780c2a8a3"
-					(reference "R201")
+					(reference "R222")
 					(unit 1)
 				)
@@
 		(on_board yes)
 		(dnp no)
-		(property "Reference" "R199"
+		(property "Reference" "R220"
 			(at 74.295 118.11 90)
 			(effects
@@
 			(project "impeller18"
 				(path "/4ccab03b-4b1c-4c61-9fa8-19853ef32b4d/f0192a6c-39ea-409b-b3a4-616780c2a8a3"
-					(reference "R199")
+					(reference "R220")
 					(unit 1)
 				)
@@
 		(on_board yes)
 		(dnp no)
-		(property "Reference" "R200"
+		(property "Reference" "R221"
 			(at 111.76 118.11 90)
 			(effects
@@
 			(project "impeller18"
 				(path "/4ccab03b-4b1c-4c61-9fa8-19853ef32b4d/f0192a6c-39ea-409b-b3a4-616780c2a8a3"
-					(reference "R200")
+					(reference "R221")
 					(unit 1)
 				)
@@
 		(on_board yes)
 		(dnp no)
-		(property "Reference" "#PWR0176"
+		(property "Reference" "#PWR0201"
 			(at 99.695 161.29 0)
 			(effects
@@
 			(project "impeller18"
 				(path "/4ccab03b-4b1c-4c61-9fa8-19853ef32b4d/f0192a6c-39ea-409b-b3a4-616780c2a8a3"
-					(reference "#PWR0176")
+					(reference "#PWR0201")
 					(unit 1)
 				)
@@
 		(on_board yes)
 		(dnp no)
-		(property "Reference" "R196"
+		(property "Reference" "R217"
 			(at 111.76 91.44 90)
 			(effects
@@
 			(project "impeller18"
 				(path "/4ccab03b-4b1c-4c61-9fa8-19853ef32b4d/f0192a6c-39ea-409b-b3a4-616780c2a8a3"
-					(reference "R196")
+					(reference "R217")
 					(unit 1)
 				)
@@
 		(dnp no)
 		(fields_autoplaced yes)
-		(property "Reference" "#PWR0175"
+		(property "Reference" "#PWR0200"
 			(at 135.255 54.61 0)
 			(effects
@@
 			(project "impeller18"
 				(path "/4ccab03b-4b1c-4c61-9fa8-19853ef32b4d/f0192a6c-39ea-409b-b3a4-616780c2a8a3"
-					(reference "#PWR0175")
-					(unit 1)
-				)
+					(reference "#PWR0200")
+					(unit 1)
+				)
