File: Hardware/ciam/impeller18/digital_inputs.kicad_sch (KiCad schematic)
At the start: 19 parts, among them J16 430451600, U62 TLP291-4, U63 TLP291-4

Commit message: updated schematics
Parts:
- J17: renamed from J16; footprint (none) -> Connector_Molex:Molex_Micro-Fit_3.0_43045-1600_2x08_P3.00mm_Horizontal
- renumbered R210 to R235, R211 to R236, R212 to R237, R213 to R238, R214 to R239, R215 to R240, R216 to R241, R217 to R242, R218 to R243, R219 to R244, R220 to R245, R221 to R246, R222 to R247, R223 to R248, R224 to R249, R225 to R250, U62 to U69, U63 to U70
Changed lines of the file:
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@@
 		(on_board yes)
 		(dnp no)
-		(property "Reference" "R215"
+		(property "Reference" "R240"
 			(at 111.76 78.105 90)
 			(effects
@@
 			(project "impeller18"
 				(path "/4ccab03b-4b1c-4c61-9fa8-19853ef32b4d/f0192a6c-39ea-409b-b3a4-616780c2a8a3"
-					(reference "R215")
+					(reference "R240")
 					(unit 1)
 				)
@@
 		(on_board yes)
 		(dnp no)
-		(property "Reference" "U62"
+		(property "Reference" "U69"
 			(at 87.63 88.9 0)
 			(effects
@@
 			(project "impeller18"
 				(path "/4ccab03b-4b1c-4c61-9fa8-19853ef32b4d/f0192a6c-39ea-409b-b3a4-616780c2a8a3"
-					(reference "U62")
+					(reference "U69")
 					(unit 4)
 				)
@@
 		(on_board yes)
 		(dnp no)
-		(property "Reference" "R218"
+		(property "Reference" "R243"
 			(at 74.295 104.775 90)
 			(effects
@@
 			(project "impeller18"
 				(path "/4ccab03b-4b1c-4c61-9fa8-19853ef32b4d/f0192a6c-39ea-409b-b3a4-616780c2a8a3"
-					(reference "R218")
+					(reference "R243")
 					(unit 1)
 				)
@@
 		(dnp no)
 		(fields_autoplaced yes)
-		(property "Reference" "J16"
+		(property "Reference" "J17"
 			(at 97.155 172.72 0)
 			(effects
@@
 			)
 		)
-		(property "Footprint" ""
+		(property "Footprint" "Connector_Molex:Molex_Micro-Fit_3.0_43045-1600_2x08_P3.00mm_Horizontal"
 			(at 95.885 186.055 0)
 			(effects
@@
 			(project "impeller18"
 				(path "/4ccab03b-4b1c-4c61-9fa8-19853ef32b4d/f0192a6c-39ea-409b-b3a4-616780c2a8a3"
-					(reference "J16")
+					(reference "J17")
 					(unit 1)
 				)
@@
 		(on_board yes)
 		(dnp no)
-		(property "Reference" "R224"
+		(property "Reference" "R249"
 			(at 74.295 144.78 90)
 			(effects
@@
 			(project "impeller18"
 				(path "/4ccab03b-4b1c-4c61-9fa8-19853ef32b4d/f0192a6c-39ea-409b-b3a4-616780c2a8a3"
-					(reference "R224")
+					(reference "R249")
 					(unit 1)
 				)
@@
 		(on_board yes)
 		(dnp no)
-		(property "Reference" "R213"
+		(property "Reference" "R238"
 			(at 111.76 64.77 90)
 			(effects
@@
 			(project "impeller18"
 				(path "/4ccab03b-4b1c-4c61-9fa8-19853ef32b4d/f0192a6c-39ea-409b-b3a4-616780c2a8a3"
-					(reference "R213")
+					(reference "R238")
 					(unit 1)
 				)
@@
 		(on_board yes)
 		(dnp no)
-		(property "Reference" "U62"
+		(property "Reference" "U69"
 			(at 87.63 48.895 0)
 			(effects
@@
 			(project "impeller18"
 				(path "/4ccab03b-4b1c-4c61-9fa8-19853ef32b4d/f0192a6c-39ea-409b-b3a4-616780c2a8a3"
-					(reference "U62")
+					(reference "U69")
 					(unit 1)
 				)
@@
 		(on_board yes)
 		(dnp no)
-		(property "Reference" "U63"
+		(property "Reference" "U70"
 			(at 87.63 115.57 0)
 			(effects
@@
 			(project "impeller18"
 				(path "/4ccab03b-4b1c-4c61-9fa8-19853ef32b4d/f0192a6c-39ea-409b-b3a4-616780c2a8a3"
-					(reference "U63")
+					(reference "U70")
 					(unit 2)
 				)
@@
 		(on_board yes)
 		(dnp no)
-		(property "Reference" "U62"
+		(property "Reference" "U69"
 			(at 87.63 75.565 0)
 			(effects
@@
 			(project "impeller18"
 				(path "/4ccab03b-4b1c-4c61-9fa8-19853ef32b4d/f0192a6c-39ea-409b-b3a4-616780c2a8a3"
-					(reference "U62")
+					(reference "U69")
 					(unit 3)
 				)
@@
 		(on_board yes)
 		(dnp no)
-		(property "Reference" "R225"
+		(property "Reference" "R250"
 			(at 111.76 144.78 90)
 			(effects
@@
 			(project "impeller18"
 				(path "/4ccab03b-4b1c-4c61-9fa8-19853ef32b4d/f0192a6c-39ea-409b-b3a4-616780c2a8a3"
-					(reference "R225")
+					(reference "R250")
 					(unit 1)
 				)
@@
 		(on_board yes)
 		(dnp no)
-		(property "Reference" "R219"
+		(property "Reference" "R244"
 			(at 111.76 104.775 90)
 			(effects
@@
 			(project "impeller18"
 				(path "/4ccab03b-4b1c-4c61-9fa8-19853ef32b4d/f0192a6c-39ea-409b-b3a4-616780c2a8a3"
-					(reference "R219")
+					(reference "R244")
 					(unit 1)
 				)
@@
 		(on_board yes)
 		(dnp no)
-		(property "Reference" "R214"
+		(property "Reference" "R239"
 			(at 74.295 78.105 90)
 			(effects
@@
 			(project "impeller18"
 				(path "/4ccab03b-4b1c-4c61-9fa8-19853ef32b4d/f0192a6c-39ea-409b-b3a4-616780c2a8a3"
-					(reference "R214")
+					(reference "R239")
 					(unit 1)
 				)
@@
 		(on_board yes)
 		(dnp no)
-		(property "Reference" "U63"
+		(property "Reference" "U70"
 			(at 87.63 142.24 0)
 			(effects
@@
 			(project "impeller18"
 				(path "/4ccab03b-4b1c-4c61-9fa8-19853ef32b4d/f0192a6c-39ea-409b-b3a4-616780c2a8a3"
-					(reference "U63")
+					(reference "U70")
 					(unit 4)
 				)
@@
 		(on_board yes)
 		(dnp no)
-		(property "Reference" "R216"
+		(property "Reference" "R241"
 			(at 74.295 91.44 90)
 			(effects
@@
 			(project "impeller18"
 				(path "/4ccab03b-4b1c-4c61-9fa8-19853ef32b4d/f0192a6c-39ea-409b-b3a4-616780c2a8a3"
-					(reference "R216")
+					(reference "R241")
 					(unit 1)
 				)
@@
 		(on_board yes)
 		(dnp no)
-		(property "Reference" "U63"
+		(property "Reference" "U70"
 			(at 87.63 102.235 0)
 			(effects
@@
 			(project "impeller18"
 				(path "/4ccab03b-4b1c-4c61-9fa8-19853ef32b4d/f0192a6c-39ea-409b-b3a4-616780c2a8a3"
-					(reference "U63")
+					(reference "U70")
 					(unit 1)
 				)
@@
 		(on_board yes)
 		(dnp no)
-		(property "Reference" "R223"
+		(property "Reference" "R248"
 			(at 111.76 131.445 90)
 			(effects
@@
 			(project "impeller18"
 				(path "/4ccab03b-4b1c-4c61-9fa8-19853ef32b4d/f0192a6c-39ea-409b-b3a4-616780c2a8a3"
-					(reference "R223")
+					(reference "R248")
 					(unit 1)
 				)
@@
 		(on_board yes)
 		(dnp no)
-		(property "Reference" "R211"
+		(property "Reference" "R236"
 			(at 111.76 51.435 90)
 			(effects
@@
 			(project "impeller18"
 				(path "/4ccab03b-4b1c-4c61-9fa8-19853ef32b4d/f0192a6c-39ea-409b-b3a4-616780c2a8a3"
-					(reference "R211")
+					(reference "R236")
 					(unit 1)
 				)
@@
 		(on_board yes)
 		(dnp no)
-		(property "Reference" "R210"
+		(property "Reference" "R235"
 			(at 74.295 51.435 90)
 			(effects
@@
 			(project "impeller18"
 				(path "/4ccab03b-4b1c-4c61-9fa8-19853ef32b4d/f0192a6c-39ea-409b-b3a4-616780c2a8a3"
-					(reference "R210")
+					(reference "R235")
 					(unit 1)
 				)
@@
 		(on_board yes)
 		(dnp no)
-		(property "Reference" "U63"
+		(property "Reference" "U70"
 			(at 87.63 128.905 0)
 			(effects
@@
 			(project "impeller18"
 				(path "/4ccab03b-4b1c-4c61-9fa8-19853ef32b4d/f0192a6c-39ea-409b-b3a4-616780c2a8a3"
-					(reference "U63")
+					(reference "U70")
 					(unit 3)
 				)
@@
 		(on_board yes)
 		(dnp no)
-		(property "Reference" "U62"
+		(property "Reference" "U69"
 			(at 87.63 62.23 0)
 			(effects
@@
 			(project "impeller18"
 				(path "/4ccab03b-4b1c-4c61-9fa8-19853ef32b4d/f0192a6c-39ea-409b-b3a4-616780c2a8a3"
-					(reference "U62")
+					(reference "U69")
 					(unit 2)
 				)
@@
 		(on_board yes)
 		(dnp no)
-		(property "Reference" "R212"
+		(property "Reference" "R237"
 			(at 74.295 64.77 90)
 			(effects
@@
 			(project "impeller18"
 				(path "/4ccab03b-4b1c-4c61-9fa8-19853ef32b4d/f0192a6c-39ea-409b-b3a4-616780c2a8a3"
-					(reference "R212")
+					(reference "R237")
 					(unit 1)
 				)
@@
 		(on_board yes)
 		(dnp no)
-		(property "Reference" "R222"
+		(property "Reference" "R247"
 			(at 74.295 131.445 90)
 			(effects
@@
 			(project "impeller18"
 				(path "/4ccab03b-4b1c-4c61-9fa8-19853ef32b4d/f0192a6c-39ea-409b-b3a4-616780c2a8a3"
-					(reference "R222")
+					(reference "R247")
 					(unit 1)
 				)
@@
 		(on_board yes)
 		(dnp no)
-		(property "Reference" "R220"
+		(property "Reference" "R245"
 			(at 74.295 118.11 90)
 			(effects
@@
 			(project "impeller18"
 				(path "/4ccab03b-4b1c-4c61-9fa8-19853ef32b4d/f0192a6c-39ea-409b-b3a4-616780c2a8a3"
-					(reference "R220")
+					(reference "R245")
 					(unit 1)
 				)
@@
 		(on_board yes)
 		(dnp no)
-		(property "Reference" "R221"
+		(property "Reference" "R246"
 			(at 111.76 118.11 90)
 			(effects
@@
 			(project "impeller18"
 				(path "/4ccab03b-4b1c-4c61-9fa8-19853ef32b4d/f0192a6c-39ea-409b-b3a4-616780c2a8a3"
-					(reference "R221")
+					(reference "R246")
 					(unit 1)
 				)
@@
 		(on_board yes)
 		(dnp no)
-		(property "Reference" "#PWR0201"
+		(property "Reference" "#PWR0223"
 			(at 99.695 161.29 0)
 			(effects
@@
 			(project "impeller18"
 				(path "/4ccab03b-4b1c-4c61-9fa8-19853ef32b4d/f0192a6c-39ea-409b-b3a4-616780c2a8a3"
-					(reference "#PWR0201")
+					(reference "#PWR0223")
 					(unit 1)
 				)
@@
 		(on_board yes)
 		(dnp no)
-		(property "Reference" "R217"
+		(property "Reference" "R242"
 			(at 111.76 91.44 90)
 			(effects
@@
 			(project "impeller18"
 				(path "/4ccab03b-4b1c-4c61-9fa8-19853ef32b4d/f0192a6c-39ea-409b-b3a4-616780c2a8a3"
-					(reference "R217")
+					(reference "R242")
 					(unit 1)
 				)
@@
 		(dnp no)
 		(fields_autoplaced yes)
-		(property "Reference" "#PWR0200"
+		(property "Reference" "#PWR0222"
 			(at 135.255 54.61 0)
 			(effects
@@
 			(project "impeller18"
 				(path "/4ccab03b-4b1c-4c61-9fa8-19853ef32b4d/f0192a6c-39ea-409b-b3a4-616780c2a8a3"
-					(reference "#PWR0200")
-					(unit 1)
-				)
+					(reference "#PWR0222")
+					(unit 1)
+				)

Commit message: updated schematics
Parts:
- J20: renamed from J17; footprint Connector_Molex:Molex_Micro-Fit_3.0_43045-1600_2x08_P3.00mm_Horizontal -> (none); Мин. кол-во (none) -> 3; Ссылка (none) -> https://www.promelec.ru/product/362588/; Цена (none) -> 197; Человекопонятное название (none) -> Прямоугольный разъем, Серия Micro-Fit 3.0 43045, 16 контакт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
- R243: renamed from R235; Мин. кол-во (none) -> 100; Ссылка (none) -> https://www.promelec.ru/product/15311/; Цена (none) -> 1; Человекопонятное название (none) -> Толстопленочный ЧИП-резистор 0603 390Ом
- R244: renamed from R236; Мин. кол-во (none) -> 1000; Ссылка (none) -> https://www.promelec.ru/product/344748/; Цена (none) -> 1; Человекопонятное название (none) -> Толстопленочный ЧИП-резистор 0603 10кОм
- R245: renamed from R237; Мин. кол-во (none) -> 100; Ссылка (none) -> https://www.promelec.ru/product/15311/; Цена (none) -> 1; Человекопонятное название (none) -> Толстопленочный ЧИП-резистор 0603 390Ом
- R246: renamed from R238; Мин. кол-во (none) -> 1000; Ссылка (none) -> https://www.promelec.ru/product/344748/; Цена (none) -> 1; Человекопонятное название (none) -> Толстопленочный ЧИП-резистор 0603 10кОм
- R247: renamed from R239; Мин. кол-во (none) -> 100; Ссылка (none) -> https://www.promelec.ru/product/15311/; Цена (none) -> 1; Человекопонятное название (none) -> Толстопленочный ЧИП-резистор 0603 390Ом
- R248: renamed from R240; Мин. кол-во (none) -> 1000; Ссылка (none) -> https://www.promelec.ru/product/344748/; Цена (none) -> 1; Человекопонятное название (none) -> Толстопленочный ЧИП-резистор 0603 10кОм
- R249: renamed from R241; Мин. кол-во (none) -> 100; Ссылка (none) -> https://www.promelec.ru/product/15311/; Цена (none) -> 1; Человекопонятное название (none) -> Толстопленочный ЧИП-резистор 0603 390Ом
- R250: renamed from R242; Мин. кол-во (none) -> 1000; Ссылка (none) -> https://www.promelec.ru/product/344748/; Цена (none) -> 1; Человекопонятное название (none) -> Толстопленочный ЧИП-резистор 0603 10кОм
- R251: renamed from R243; Мин. кол-во (none) -> 100; Ссылка (none) -> https://www.promelec.ru/product/15311/; Цена (none) -> 1; Человекопонятное название (none) -> Толстопленочный ЧИП-резистор 0603 390Ом
- R252: renamed from R244; Мин. кол-во (none) -> 1000; Ссылка (none) -> https://www.promelec.ru/product/344748/; Цена (none) -> 1; Человекопонятное название (none) -> Толстопленочный ЧИП-резистор 0603 10кОм
- R253: renamed from R245; Мин. кол-во (none) -> 100; Ссылка (none) -> https://www.promelec.ru/product/15311/; Цена (none) -> 1; Человекопонятное название (none) -> Толстопленочный ЧИП-резистор 0603 390Ом
- R254: renamed from R246; Мин. кол-во (none) -> 1000; Ссылка (none) -> https://www.promelec.ru/product/344748/; Цена (none) -> 1; Человекопонятное название (none) -> Толстопленочный ЧИП-резистор 0603 10кОм
- R255: renamed from R247; Мин. кол-во (none) -> 100; Ссылка (none) -> https://www.promelec.ru/product/15311/; Цена (none) -> 1; Человекопонятное название (none) -> Толстопленочный ЧИП-резистор 0603 390Ом
- R256: renamed from R248; Мин. кол-во (none) -> 1000; Ссылка (none) -> https://www.promelec.ru/product/344748/; Цена (none) -> 1; Человекопонятное название (none) -> Толстопленочный ЧИП-резистор 0603 10кОм
- R257: renamed from R249; Мин. кол-во (none) -> 100; Ссылка (none) -> https://www.promelec.ru/product/15311/; Цена (none) -> 1; Человекопонятное название (none) -> Толстопленочный ЧИП-резистор 0603 390Ом
- R258: renamed from R250; Мин. кол-во (none) -> 1000; Ссылка (none) -> https://www.promelec.ru/product/344748/; Цена (none) -> 1; Человекопонятное название (none) -> Толстопленочный ЧИП-резистор 0603 10кОм
- U71: renamed from U69; Мин. кол-во (none) -> 1; Ссылка (none) -> https://www.chipdip.ru/product/tlp291-4-gb-tp-e-t; Цена (none) -> 340; Человекопонятное название (none) -> Оптопара с транзисторным выходом 4-х канальная
- U72: renamed from U70; Мин. кол-во (none) -> 1; Ссылка (none) -> https://www.chipdip.ru/product/tlp291-4-gb-tp-e-t; Цена (none) -> 340; Человекопонятное название (none) -> Оптопара с транзисторным выходом 4-х канальная

Commit message: added footprints
Parts:
- J20: footprint (none) -> Connector_Molex:Molex_Micro-Fit_3.0_43045-1600_2x08_P3.00mm_Horizontal
- R243, R244, R245, R246, R247, R248, R249, R250, R251, R252, R253, R254, R255, R256, R257, R258: footprint (none) -> Resistor_SMD:R_0603_1608Metric
- U71, U72: footprint (none) -> Package_SO:SOIC-16_4.55x10.3mm_P1.27mm
Changed lines of the file:
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@@
 			)
 		)
-		(property "Footprint" ""
+		(property "Footprint" "Resistor_SMD:R_0603_1608Metric"
 			(at 111.76 80.01 0)
 			(effects
@@
 			)
 		)
-		(property "Footprint" ""
+		(property "Footprint" "Package_SO:SOIC-16_4.55x10.3mm_P1.27mm"
 			(at 82.55 100.965 0)
 			(effects
@@
 			)
 		)
-		(property "Footprint" ""
+		(property "Footprint" "Resistor_SMD:R_0603_1608Metric"
 			(at 74.295 106.68 0)
 			(effects
@@
 			)
 		)
-		(property "Footprint" ""
+		(property "Footprint" "Connector_Molex:Molex_Micro-Fit_3.0_43045-1600_2x08_P3.00mm_Horizontal"
 			(at 95.885 186.055 0)
 			(effects
@@
 			)
 		)
-		(property "Footprint" ""
+		(property "Footprint" "Resistor_SMD:R_0603_1608Metric"
 			(at 74.295 146.685 0)
 			(effects
@@
 			)
 		)
-		(property "Footprint" ""
+		(property "Footprint" "Resistor_SMD:R_0603_1608Metric"
 			(at 111.76 66.675 0)
 			(effects
@@
 			)
 		)
-		(property "Footprint" ""
+		(property "Footprint" "Package_SO:SOIC-16_4.55x10.3mm_P1.27mm"
 			(at 82.55 60.96 0)
 			(effects
@@
 			)
 		)
-		(property "Footprint" ""
+		(property "Footprint" "Package_SO:SOIC-16_4.55x10.3mm_P1.27mm"
 			(at 82.55 127.635 0)
 			(effects
@@
 			)
 		)
-		(property "Footprint" ""
+		(property "Footprint" "Package_SO:SOIC-16_4.55x10.3mm_P1.27mm"
 			(at 82.55 87.63 0)
 			(effects
@@
 			)
 		)
-		(property "Footprint" ""
+		(property "Footprint" "Resistor_SMD:R_0603_1608Metric"
 			(at 111.76 146.685 0)
 			(effects
@@
 			)
 		)
-		(property "Footprint" ""
+		(property "Footprint" "Resistor_SMD:R_0603_1608Metric"
 			(at 111.76 106.68 0)
 			(effects
@@
 			)
 		)
-		(property "Footprint" ""
+		(property "Footprint" "Resistor_SMD:R_0603_1608Metric"
 			(at 74.295 80.01 0)
 			(effects
@@
 			)
 		)
-		(property "Footprint" ""
+		(property "Footprint" "Package_SO:SOIC-16_4.55x10.3mm_P1.27mm"
 			(at 82.55 154.305 0)
 			(effects
@@
 			)
 		)
-		(property "Footprint" ""
+		(property "Footprint" "Resistor_SMD:R_0603_1608Metric"
 			(at 74.295 93.345 0)
 			(effects
@@
 			)
 		)
-		(property "Footprint" ""
+		(property "Footprint" "Package_SO:SOIC-16_4.55x10.3mm_P1.27mm"
 			(at 82.55 114.3 0)
 			(effects
@@
 			)
 		)
-		(property "Footprint" ""
+		(property "Footprint" "Resistor_SMD:R_0603_1608Metric"
 			(at 111.76 133.35 0)
 			(effects
@@
 			)
 		)
-		(property "Footprint" ""
+		(property "Footprint" "Resistor_SMD:R_0603_1608Metric"
 			(at 111.76 53.34 0)
 			(effects
@@
 			)
 		)
-		(property "Footprint" ""
+		(property "Footprint" "Resistor_SMD:R_0603_1608Metric"
 			(at 74.295 53.34 0)
 			(effects
@@
 			)
 		)
-		(property "Footprint" ""
+		(property "Footprint" "Package_SO:SOIC-16_4.55x10.3mm_P1.27mm"
 			(at 82.55 140.97 0)
 			(effects
@@
 			)
 		)
-		(property "Footprint" ""
+		(property "Footprint" "Package_SO:SOIC-16_4.55x10.3mm_P1.27mm"
 			(at 82.55 74.295 0)
 			(effects
@@
 			)
 		)
-		(property "Footprint" ""
+		(property "Footprint" "Resistor_SMD:R_0603_1608Metric"
 			(at 74.295 66.675 0)
 			(effects
@@
 			)
 		)
-		(property "Footprint" ""
+		(property "Footprint" "Resistor_SMD:R_0603_1608Metric"
 			(at 74.295 133.35 0)
 			(effects
@@
 			)
 		)
-		(property "Footprint" ""
+		(property "Footprint" "Resistor_SMD:R_0603_1608Metric"
 			(at 74.295 120.015 0)
 			(effects
@@
 			)
 		)
-		(property "Footprint" ""
+		(property "Footprint" "Resistor_SMD:R_0603_1608Metric"
 			(at 111.76 120.015 0)
 			(effects
@@
 			)
 		)
-		(property "Footprint" ""
+		(property "Footprint" "Resistor_SMD:R_0603_1608Metric"
 			(at 111.76 93.345 0)
 			(effects

Commit message: Updated packeges
Parts:
- J20: footprint Connector_Molex:Molex_Micro-Fit_3.0_43045-1600_2x08_P3.00mm_Horizontal -> user_lib:430451600
Changed lines of the file:
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@@
 			)
 		)
-		(property "Footprint" "Connector_Molex:Molex_Micro-Fit_3.0_43045-1600_2x08_P3.00mm_Horizontal"
+		(property "Footprint" "user_lib:430451600"
 			(at 95.885 186.055 0)
 			(effects

Commit message: Updated 3D models
Parts:
- U69: renamed from U71; Мин. кол-во 1 -> 7; Ссылка https://www.chipdip.ru/product/tlp291-4-gb-tp-e-t -> https://www.promelec.ru/product/247137/; Цена 340 -> 76
- U70: renamed from U72; Мин. кол-во 1 -> 7; Ссылка https://www.chipdip.ru/product/tlp291-4-gb-tp-e-t -> https://www.promelec.ru/product/247137/; Цена 340 -> 76
- renumbered J20 to J28, R243 to R298, R244 to R299, R245 to R300, R246 to R301, R247 to R302, R248 to R303, R249 to R304, R250 to R305, R251 to R306, R252 to R307, R253 to R308, R254 to R309, R255 to R310, R256 to R311, R257 to R312, R258 to R313
