File: Hardware/ciam/impeller18/digital_inputs.kicad_sch (KiCad schematic)
At the start: 19 parts, among them J28 430451600, U69 TLP291-4, U70 TLP291-4

Commit message: Daily PCB update
Parts:
- renumbered R298 to R302, R299 to R303, R300 to R304, R301 to R305, R302 to R306, R303 to R307, R304 to R308, R305 to R309, R306 to R310, R307 to R311, R308 to R312, R309 to R313, R310 to R314, R311 to R315, R312 to R316, R313 to R317
Changed lines of the file:
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@@
 		(on_board yes)
 		(dnp no)
-		(property "Reference" "R303"
+		(property "Reference" "R307"
 			(at 111.76 78.105 90)
 			(effects
@@
 			(project "impeller18"
 				(path "/4ccab03b-4b1c-4c61-9fa8-19853ef32b4d/f0192a6c-39ea-409b-b3a4-616780c2a8a3"
-					(reference "R303")
+					(reference "R307")
 					(unit 1)
 				)
@@
 		(on_board yes)
 		(dnp no)
-		(property "Reference" "R306"
+		(property "Reference" "R310"
 			(at 74.295 104.775 90)
 			(effects
@@
 			(project "impeller18"
 				(path "/4ccab03b-4b1c-4c61-9fa8-19853ef32b4d/f0192a6c-39ea-409b-b3a4-616780c2a8a3"
-					(reference "R306")
+					(reference "R310")
 					(unit 1)
 				)
@@
 		(on_board yes)
 		(dnp no)
-		(property "Reference" "R312"
+		(property "Reference" "R316"
 			(at 74.295 144.78 90)
 			(effects
@@
 			(project "impeller18"
 				(path "/4ccab03b-4b1c-4c61-9fa8-19853ef32b4d/f0192a6c-39ea-409b-b3a4-616780c2a8a3"
-					(reference "R312")
+					(reference "R316")
 					(unit 1)
 				)
@@
 		(on_board yes)
 		(dnp no)
-		(property "Reference" "R301"
+		(property "Reference" "R305"
 			(at 111.76 64.77 90)
 			(effects
@@
 			(project "impeller18"
 				(path "/4ccab03b-4b1c-4c61-9fa8-19853ef32b4d/f0192a6c-39ea-409b-b3a4-616780c2a8a3"
-					(reference "R301")
+					(reference "R305")
 					(unit 1)
 				)
@@
 		(on_board yes)
 		(dnp no)
-		(property "Reference" "R313"
+		(property "Reference" "R317"
 			(at 111.76 144.78 90)
 			(effects
@@
 			(project "impeller18"
 				(path "/4ccab03b-4b1c-4c61-9fa8-19853ef32b4d/f0192a6c-39ea-409b-b3a4-616780c2a8a3"
-					(reference "R313")
+					(reference "R317")
 					(unit 1)
 				)
@@
 		(on_board yes)
 		(dnp no)
-		(property "Reference" "R307"
+		(property "Reference" "R311"
 			(at 111.76 104.775 90)
 			(effects
@@
 			(project "impeller18"
 				(path "/4ccab03b-4b1c-4c61-9fa8-19853ef32b4d/f0192a6c-39ea-409b-b3a4-616780c2a8a3"
-					(reference "R307")
+					(reference "R311")
 					(unit 1)
 				)
@@
 		(on_board yes)
 		(dnp no)
-		(property "Reference" "R302"
+		(property "Reference" "R306"
 			(at 74.295 78.105 90)
 			(effects
@@
 			(project "impeller18"
 				(path "/4ccab03b-4b1c-4c61-9fa8-19853ef32b4d/f0192a6c-39ea-409b-b3a4-616780c2a8a3"
-					(reference "R302")
+					(reference "R306")
 					(unit 1)
 				)
@@
 		(on_board yes)
 		(dnp no)
-		(property "Reference" "R304"
+		(property "Reference" "R308"
 			(at 74.295 91.44 90)
 			(effects
@@
 			(project "impeller18"
 				(path "/4ccab03b-4b1c-4c61-9fa8-19853ef32b4d/f0192a6c-39ea-409b-b3a4-616780c2a8a3"
-					(reference "R304")
+					(reference "R308")
 					(unit 1)
 				)
@@
 		(on_board yes)
 		(dnp no)
-		(property "Reference" "R311"
+		(property "Reference" "R315"
 			(at 111.76 131.445 90)
 			(effects
@@
 			(project "impeller18"
 				(path "/4ccab03b-4b1c-4c61-9fa8-19853ef32b4d/f0192a6c-39ea-409b-b3a4-616780c2a8a3"
-					(reference "R311")
+					(reference "R315")
 					(unit 1)
 				)
@@
 		(on_board yes)
 		(dnp no)
-		(property "Reference" "R299"
+		(property "Reference" "R303"
 			(at 111.76 51.435 90)
 			(effects
@@
 			(project "impeller18"
 				(path "/4ccab03b-4b1c-4c61-9fa8-19853ef32b4d/f0192a6c-39ea-409b-b3a4-616780c2a8a3"
-					(reference "R299")
+					(reference "R303")
 					(unit 1)
 				)
@@
 		(on_board yes)
 		(dnp no)
-		(property "Reference" "R298"
+		(property "Reference" "R302"
 			(at 74.295 51.435 90)
 			(effects
@@
 			(project "impeller18"
 				(path "/4ccab03b-4b1c-4c61-9fa8-19853ef32b4d/f0192a6c-39ea-409b-b3a4-616780c2a8a3"
-					(reference "R298")
+					(reference "R302")
 					(unit 1)
 				)
@@
 		(on_board yes)
 		(dnp no)
-		(property "Reference" "R300"
+		(property "Reference" "R304"
 			(at 74.295 64.77 90)
 			(effects
@@
 			(project "impeller18"
 				(path "/4ccab03b-4b1c-4c61-9fa8-19853ef32b4d/f0192a6c-39ea-409b-b3a4-616780c2a8a3"
-					(reference "R300")
+					(reference "R304")
 					(unit 1)
 				)
@@
 		(on_board yes)
 		(dnp no)
-		(property "Reference" "R310"
+		(property "Reference" "R314"
 			(at 74.295 131.445 90)
 			(effects
@@
 			(project "impeller18"
 				(path "/4ccab03b-4b1c-4c61-9fa8-19853ef32b4d/f0192a6c-39ea-409b-b3a4-616780c2a8a3"
-					(reference "R310")
+					(reference "R314")
 					(unit 1)
 				)
@@
 		(on_board yes)
 		(dnp no)
-		(property "Reference" "R308"
+		(property "Reference" "R312"
 			(at 74.295 118.11 90)
 			(effects
@@
 			(project "impeller18"
 				(path "/4ccab03b-4b1c-4c61-9fa8-19853ef32b4d/f0192a6c-39ea-409b-b3a4-616780c2a8a3"
-					(reference "R308")
+					(reference "R312")
 					(unit 1)
 				)
@@
 		(on_board yes)
 		(dnp no)
-		(property "Reference" "R309"
+		(property "Reference" "R313"
 			(at 111.76 118.11 90)
 			(effects
@@
 			(project "impeller18"
 				(path "/4ccab03b-4b1c-4c61-9fa8-19853ef32b4d/f0192a6c-39ea-409b-b3a4-616780c2a8a3"
-					(reference "R309")
+					(reference "R313")
 					(unit 1)
 				)
@@
 		(on_board yes)
 		(dnp no)
-		(property "Reference" "#PWR0273"
+		(property "Reference" "#PWR0285"
 			(at 99.695 161.29 0)
 			(effects
@@
 			(project "impeller18"
 				(path "/4ccab03b-4b1c-4c61-9fa8-19853ef32b4d/f0192a6c-39ea-409b-b3a4-616780c2a8a3"
-					(reference "#PWR0273")
+					(reference "#PWR0285")
 					(unit 1)
 				)
@@
 		(on_board yes)
 		(dnp no)
-		(property "Reference" "R305"
+		(property "Reference" "R309"
 			(at 111.76 91.44 90)
 			(effects
@@
 			(project "impeller18"
 				(path "/4ccab03b-4b1c-4c61-9fa8-19853ef32b4d/f0192a6c-39ea-409b-b3a4-616780c2a8a3"
-					(reference "R305")
+					(reference "R309")
 					(unit 1)
 				)
@@
 		(dnp no)
 		(fields_autoplaced yes)
-		(property "Reference" "#PWR0272"
+		(property "Reference" "#PWR0284"
 			(at 135.255 54.61 0)
 			(effects
@@
 			(project "impeller18"
 				(path "/4ccab03b-4b1c-4c61-9fa8-19853ef32b4d/f0192a6c-39ea-409b-b3a4-616780c2a8a3"
-					(reference "#PWR0272")
+					(reference "#PWR0284")
 					(unit 1)
 				)
