File: Hardware/ciam/impeller18/digital_inputs.kicad_sch (KiCad schematic)
At the start: 19 parts, among them J28 430451600, U69 TLP291-4, U70 TLP291-4

Commit message: Update PCB concept
Parts:
- renumbered J28 to J31, R302 to R299, R303 to R300, R304 to R301, R305 to R302, R306 to R303, R307 to R304, R308 to R305, R309 to R306, R310 to R307, R311 to R308, R312 to R309, R313 to R310, R314 to R311, R315 to R312, R316 to R313, R317 to R314
Connections:
- net DIGITAL_IN_1: now also U69.10; no longer U69.16
- net DIGITAL_IN_2: now also U69.12; no longer U69.14
- net DIGITAL_IN_3: now also U69.14; no longer U69.12
- net DIGITAL_IN_4: now also U69.16; no longer U69.10
- net DIGITAL_IN_5: now also U70.10; no longer U70.16
- net DIGITAL_IN_6: now also U70.12; no longer U70.14
- net DIGITAL_IN_7: now also U70.14; no longer U70.12
- net DIGITAL_IN_8: now also U70.16; no longer U70.10
- net INPUT_1_NEG: now also J31.9 (Pin_9), U69.8; no longer J31.2 (Pin_2), U69.2
- net INPUT_2_NEG: now also J31.10 (Pin_10), U69.6; no longer J31.4 (Pin_4), U69.4
- net INPUT_2_POS: now also J31.2 (Pin_2); no longer J31.3 (Pin_3)
- net INPUT_3_NEG: now also J31.11 (Pin_11), U69.4; no longer J31.6 (Pin_6), U69.6
- net INPUT_3_POS: now also J31.3 (Pin_3); no longer J31.5 (Pin_5)
- net INPUT_4_NEG: now also J31.12 (Pin_12), U69.2; no longer J31.8 (Pin_8), U69.8
- net INPUT_4_POS: now also J31.4 (Pin_4); no longer J31.7 (Pin_7)
- net INPUT_5_NEG: now also J31.13 (Pin_13), U70.8; no longer J31.10 (Pin_10), U70.2
- net INPUT_5_POS: now also J31.5 (Pin_5); no longer J31.9 (Pin_9)
- net INPUT_6_NEG: now also J31.14 (Pin_14), U70.6; no longer J31.12 (Pin_12), U70.4
- net INPUT_6_POS: now also J31.6 (Pin_6); no longer J31.11 (Pin_11)
- net INPUT_7_NEG: now also J31.15 (Pin_15), U70.4; no longer J31.14 (Pin_14), U70.6
- net INPUT_7_POS: now also J31.7 (Pin_7); no longer J31.13 (Pin_13)
- net INPUT_8_NEG: now also U70.2; no longer U70.8
- net INPUT_8_POS: now also J31.8 (Pin_8); no longer J31.15 (Pin_15)
- net at U69.7: now also R299.2; no longer R305.2
- net at R307.2: now also U70.7; no longer U70.1
- net at R313.2: now also U70.1; no longer U70.7
- net at U69.1: now also R305.2; no longer R299.2
- net at U70.3: now also R311.2; no longer R309.2
- net at U69.5: now also R301.2; no longer R303.2
- net at U70.5: now also R309.2; no longer R311.2
- net at U69.3: now also R303.2; no longer R301.2
Other:
- moved on the sheet: U69A, U69B, U69C, U69D, U70A, U70B, U70C, U70D

Commit message: Silkscreen bugfix
Parts:
- renumbered J31 to J34, R299 to R313, R300 to R314, R301 to R315, R302 to R316, R303 to R317, R304 to R318, R305 to R319, R306 to R320, R307 to R321, R308 to R322, R309 to R323, R310 to R324, R311 to R325, R312 to R326, R313 to R327, R314 to R328
Changed lines of the file:
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@@
 		(on_board yes)
 		(dnp no)
-		(property "Reference" "R304"
+		(property "Reference" "R318"
 			(at 111.76 78.105 90)
 			(effects
@@
 			(project "impeller18"
 				(path "/4ccab03b-4b1c-4c61-9fa8-19853ef32b4d/f0192a6c-39ea-409b-b3a4-616780c2a8a3"
-					(reference "R304")
+					(reference "R318")
 					(unit 1)
 				)
@@
 		(on_board yes)
 		(dnp no)
-		(property "Reference" "R307"
+		(property "Reference" "R321"
 			(at 74.295 104.775 90)
 			(effects
@@
 			(project "impeller18"
 				(path "/4ccab03b-4b1c-4c61-9fa8-19853ef32b4d/f0192a6c-39ea-409b-b3a4-616780c2a8a3"
-					(reference "R307")
+					(reference "R321")
 					(unit 1)
 				)
@@
 		(on_board yes)
 		(dnp no)
-		(property "Reference" "J31"
+		(property "Reference" "J34"
 			(at 97.155 172.72 0)
 			(effects
@@
 			(project "impeller18"
 				(path "/4ccab03b-4b1c-4c61-9fa8-19853ef32b4d/f0192a6c-39ea-409b-b3a4-616780c2a8a3"
-					(reference "J31")
+					(reference "J34")
 					(unit 1)
 				)
@@
 		(on_board yes)
 		(dnp no)
-		(property "Reference" "R313"
+		(property "Reference" "R327"
 			(at 74.295 144.78 90)
 			(effects
@@
 			(project "impeller18"
 				(path "/4ccab03b-4b1c-4c61-9fa8-19853ef32b4d/f0192a6c-39ea-409b-b3a4-616780c2a8a3"
-					(reference "R313")
+					(reference "R327")
 					(unit 1)
 				)
@@
 		(on_board yes)
 		(dnp no)
-		(property "Reference" "R302"
+		(property "Reference" "R316"
 			(at 111.76 64.77 90)
 			(effects
@@
 			(project "impeller18"
 				(path "/4ccab03b-4b1c-4c61-9fa8-19853ef32b4d/f0192a6c-39ea-409b-b3a4-616780c2a8a3"
-					(reference "R302")
+					(reference "R316")
 					(unit 1)
 				)
@@
 		(on_board yes)
 		(dnp no)
-		(property "Reference" "R314"
+		(property "Reference" "R328"
 			(at 111.76 144.78 90)
 			(effects
@@
 			(project "impeller18"
 				(path "/4ccab03b-4b1c-4c61-9fa8-19853ef32b4d/f0192a6c-39ea-409b-b3a4-616780c2a8a3"
-					(reference "R314")
+					(reference "R328")
 					(unit 1)
 				)
@@
 		(on_board yes)
 		(dnp no)
-		(property "Reference" "R308"
+		(property "Reference" "R322"
 			(at 111.76 104.775 90)
 			(effects
@@
 			(project "impeller18"
 				(path "/4ccab03b-4b1c-4c61-9fa8-19853ef32b4d/f0192a6c-39ea-409b-b3a4-616780c2a8a3"
-					(reference "R308")
+					(reference "R322")
 					(unit 1)
 				)
@@
 		(on_board yes)
 		(dnp no)
-		(property "Reference" "R303"
+		(property "Reference" "R317"
 			(at 74.295 78.105 90)
 			(effects
@@
 			(project "impeller18"
 				(path "/4ccab03b-4b1c-4c61-9fa8-19853ef32b4d/f0192a6c-39ea-409b-b3a4-616780c2a8a3"
-					(reference "R303")
+					(reference "R317")
 					(unit 1)
 				)
@@
 		(on_board yes)
 		(dnp no)
-		(property "Reference" "R305"
+		(property "Reference" "R319"
 			(at 74.295 91.44 90)
 			(effects
@@
 			(project "impeller18"
 				(path "/4ccab03b-4b1c-4c61-9fa8-19853ef32b4d/f0192a6c-39ea-409b-b3a4-616780c2a8a3"
-					(reference "R305")
+					(reference "R319")
 					(unit 1)
 				)
@@
 		(on_board yes)
 		(dnp no)
-		(property "Reference" "R312"
+		(property "Reference" "R326"
 			(at 111.76 131.445 90)
 			(effects
@@
 			(project "impeller18"
 				(path "/4ccab03b-4b1c-4c61-9fa8-19853ef32b4d/f0192a6c-39ea-409b-b3a4-616780c2a8a3"
-					(reference "R312")
+					(reference "R326")
 					(unit 1)
 				)
@@
 		(on_board yes)
 		(dnp no)
-		(property "Reference" "R300"
+		(property "Reference" "R314"
 			(at 111.76 51.435 90)
 			(effects
@@
 			(project "impeller18"
 				(path "/4ccab03b-4b1c-4c61-9fa8-19853ef32b4d/f0192a6c-39ea-409b-b3a4-616780c2a8a3"
-					(reference "R300")
+					(reference "R314")
 					(unit 1)
 				)
@@
 		(on_board yes)
 		(dnp no)
-		(property "Reference" "R299"
+		(property "Reference" "R313"
 			(at 74.295 51.435 90)
 			(effects
@@
 			(project "impeller18"
 				(path "/4ccab03b-4b1c-4c61-9fa8-19853ef32b4d/f0192a6c-39ea-409b-b3a4-616780c2a8a3"
-					(reference "R299")
+					(reference "R313")
 					(unit 1)
 				)
@@
 		(on_board yes)
 		(dnp no)
-		(property "Reference" "R301"
+		(property "Reference" "R315"
 			(at 74.295 64.77 90)
 			(effects
@@
 			(project "impeller18"
 				(path "/4ccab03b-4b1c-4c61-9fa8-19853ef32b4d/f0192a6c-39ea-409b-b3a4-616780c2a8a3"
-					(reference "R301")
+					(reference "R315")
 					(unit 1)
 				)
@@
 		(on_board yes)
 		(dnp no)
-		(property "Reference" "R311"
+		(property "Reference" "R325"
 			(at 74.295 131.445 90)
 			(effects
@@
 			(project "impeller18"
 				(path "/4ccab03b-4b1c-4c61-9fa8-19853ef32b4d/f0192a6c-39ea-409b-b3a4-616780c2a8a3"
-					(reference "R311")
+					(reference "R325")
 					(unit 1)
 				)
@@
 		(on_board yes)
 		(dnp no)
-		(property "Reference" "R309"
+		(property "Reference" "R323"
 			(at 74.295 118.11 90)
 			(effects
@@
 			(project "impeller18"
 				(path "/4ccab03b-4b1c-4c61-9fa8-19853ef32b4d/f0192a6c-39ea-409b-b3a4-616780c2a8a3"
-					(reference "R309")
+					(reference "R323")
 					(unit 1)
 				)
@@
 		(on_board yes)
 		(dnp no)
-		(property "Reference" "R310"
+		(property "Reference" "R324"
 			(at 111.76 118.11 90)
 			(effects
@@
 			(project "impeller18"
 				(path "/4ccab03b-4b1c-4c61-9fa8-19853ef32b4d/f0192a6c-39ea-409b-b3a4-616780c2a8a3"
-					(reference "R310")
+					(reference "R324")
 					(unit 1)
 				)
@@
 		(on_board yes)
 		(dnp no)
-		(property "Reference" "#PWR0279"
+		(property "Reference" "#PWR0280"
 			(at 99.695 161.29 0)
 			(effects
@@
 			(project "impeller18"
 				(path "/4ccab03b-4b1c-4c61-9fa8-19853ef32b4d/f0192a6c-39ea-409b-b3a4-616780c2a8a3"
-					(reference "#PWR0279")
+					(reference "#PWR0280")
 					(unit 1)
 				)
@@
 		(on_board yes)
 		(dnp no)
-		(property "Reference" "R306"
+		(property "Reference" "R320"
 			(at 111.76 91.44 90)
 			(effects
@@
 			(project "impeller18"
 				(path "/4ccab03b-4b1c-4c61-9fa8-19853ef32b4d/f0192a6c-39ea-409b-b3a4-616780c2a8a3"
-					(reference "R306")
+					(reference "R320")
 					(unit 1)
 				)
@@
 		(dnp no)
 		(fields_autoplaced yes)
-		(property "Reference" "#PWR0278"
+		(property "Reference" "#PWR0279"
 			(at 135.255 54.61 0)
 			(effects
@@
 			(project "impeller18"
 				(path "/4ccab03b-4b1c-4c61-9fa8-19853ef32b4d/f0192a6c-39ea-409b-b3a4-616780c2a8a3"
-					(reference "#PWR0278")
+					(reference "#PWR0279")
 					(unit 1)
 				)
