File: Hardware/ciam/impeller18/power.kicad_sch (KiCad schematic)
At the start: 117 parts, among them J6 430450400, J7 PLS-2, J8 PLS-2, K1 1393219-3, K2 1393219-3, K3 1393219-3, Q1 BSS138, Q2 BSS138, Q3 AO3401A, Q4 BSS138, Q5 BSS138, U2 LDL1117S33R, U3 VDRI25W05, U4 VDRI15W12, U5 HY2213-BB3A, U6 bq2057WSN, U7 HY2213-BB3A, U8 LD1084V, U9 MCP3001-I/SN

Commit message: Daily PCB update
Parts:
- renumbered R339 to R30, R30 to R31, R340 to R32, R31 to R33, R341 to R34, R32 to R35, R33 to R36, R342 to R37, R34 to R38
Connections:
- net GND_IN: now also L1.1, L2.1; no longer L1.2, L2.2
- net VIN: now also L1.2, L2.2; no longer L1.1, L2.1
- net at C34.2, C35.2, C36.2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: now also L1.4; no longer L1.3
- net at C34.1, C35.1, C36.1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: now also L1.3; no longer L1.4
- net at C45.2, C46.2, C47.2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: now also L2.4; no longer L2.3
- net at C45.1, C46.1, C47.1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: now also L2.3; no longer L2.4
Changed lines of the file:
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@@
 		(on_board yes)
 		(dnp no)
-		(property "Reference" "R340"
+		(property "Reference" "R32"
 			(at 84.455 231.775 0)
 			(effects
@@
 			(project "impeller18"
 				(path "/4ccab03b-4b1c-4c61-9fa8-19853ef32b4d/1159e494-0aef-4f6c-ae01-1217066bb411"
-					(reference "R340")
+					(reference "R32")
 					(unit 1)
 				)
@@
 		(on_board yes)
 		(dnp no)
-		(property "Reference" "#PWR089"
+		(property "Reference" "#PWR091"
 			(at 208.915 264.16 0)
 			(effects
@@
 			(project "impeller18"
 				(path "/4ccab03b-4b1c-4c61-9fa8-19853ef32b4d/1159e494-0aef-4f6c-ae01-1217066bb411"
-					(reference "#PWR089")
+					(reference "#PWR091")
 					(unit 1)
 				)
@@
 		(on_board yes)
 		(dnp no)
-		(property "Reference" "R342"
+		(property "Reference" "R37"
 			(at 84.455 247.65 0)
 			(effects
@@
 			(project "impeller18"
 				(path "/4ccab03b-4b1c-4c61-9fa8-19853ef32b4d/1159e494-0aef-4f6c-ae01-1217066bb411"
-					(reference "R342")
+					(reference "R37")
 					(unit 1)
 				)
@@
 		(lib_id "Device:L_Coupled")
 		(at 69.215 90.17 0)
+		(mirror x)
 		(unit 1)
 		(exclude_from_sim no)
@@
 		(dnp no)
 		(property "Reference" "L2"
-			(at 69.215 83.82 0)
+			(at 69.215 79.375 0)
 			(effects
 				(font
@@
 		)
 		(property "Value" "B82721-K2222-U30"
-			(at 69.215 81.28 0)
+			(at 69.215 81.915 0)
 			(effects
 				(font
@@
 		(on_board yes)
 		(dnp no)
-		(property "Reference" "R31"
+		(property "Reference" "R33"
 			(at 205.105 229.87 0)
 			(effects
@@
 			(project "impeller18"
 				(path "/4ccab03b-4b1c-4c61-9fa8-19853ef32b4d/1159e494-0aef-4f6c-ae01-1217066bb411"
-					(reference "R31")
+					(reference "R33")
 					(unit 1)
 				)
@@
 		(dnp no)
 		(fields_autoplaced yes)
-		(property "Reference" "#PWR0314"
+		(property "Reference" "#PWR090"
 			(at 85.725 257.175 0)
 			(effects
@@
 			(project "impeller18"
 				(path "/4ccab03b-4b1c-4c61-9fa8-19853ef32b4d/1159e494-0aef-4f6c-ae01-1217066bb411"
-					(reference "#PWR0314")
+					(reference "#PWR090")
 					(unit 1)
 				)
@@
 		(dnp no)
 		(fields_autoplaced yes)
-		(property "Reference" "#PWR084"
+		(property "Reference" "#PWR085"
 			(at 208.915 229.87 0)
 			(effects
@@
 			(project "impeller18"
 				(path "/4ccab03b-4b1c-4c61-9fa8-19853ef32b4d/1159e494-0aef-4f6c-ae01-1217066bb411"
-					(reference "#PWR084")
+					(reference "#PWR085")
 					(unit 1)
 				)
@@
 		(on_board yes)
 		(dnp no)
-		(property "Reference" "R339"
+		(property "Reference" "R30"
 			(at 84.455 225.425 0)
 			(effects
@@
 			(project "impeller18"
 				(path "/4ccab03b-4b1c-4c61-9fa8-19853ef32b4d/1159e494-0aef-4f6c-ae01-1217066bb411"
-					(reference "R339")
+					(reference "R30")
 					(unit 1)
 				)
@@
 		(dnp no)
 		(fields_autoplaced yes)
-		(property "Reference" "#PWR085"
+		(property "Reference" "#PWR086"
 			(at 236.22 233.68 0)
 			(effects
@@
 			(project "impeller18"
 				(path "/4ccab03b-4b1c-4c61-9fa8-19853ef32b4d/1159e494-0aef-4f6c-ae01-1217066bb411"
-					(reference "#PWR085")
+					(reference "#PWR086")
 					(unit 1)
 				)
@@
 		(lib_id "Device:L_Coupled")
 		(at 69.215 54.61 0)
+		(mirror x)
 		(unit 1)
 		(exclude_from_sim no)
@@
 		(dnp no)
 		(property "Reference" "L1"
-			(at 69.215 48.26 0)
+			(at 69.215 43.815 0)
 			(effects
 				(font
@@
 		)
 		(property "Value" "B82721-K2222-U30"
-			(at 69.215 45.72 0)
+			(at 69.215 46.355 0)
 			(effects
 				(font
@@
 		(on_board yes)
 		(dnp no)
-		(property "Reference" "#PWR088"
+		(property "Reference" "#PWR089"
 			(at 262.255 245.11 0)
 			(effects
@@
 			(project "impeller18"
 				(path "/4ccab03b-4b1c-4c61-9fa8-19853ef32b4d/1159e494-0aef-4f6c-ae01-1217066bb411"
-					(reference "#PWR088")
+					(reference "#PWR089")
 					(unit 1)
 				)
@@
 		(on_board yes)
 		(dnp no)
-		(property "Reference" "R32"
+		(property "Reference" "R35"
 			(at 205.105 236.855 0)
 			(effects
@@
 			(project "impeller18"
 				(path "/4ccab03b-4b1c-4c61-9fa8-19853ef32b4d/1159e494-0aef-4f6c-ae01-1217066bb411"
-					(reference "R32")
+					(reference "R35")
 					(unit 1)
 				)
@@
 		(on_board yes)
 		(dnp no)
-		(property "Reference" "#PWR087"
+		(property "Reference" "#PWR088"
 			(at 224.155 243.205 0)
 			(effects
@@
 			(project "impeller18"
 				(path "/4ccab03b-4b1c-4c61-9fa8-19853ef32b4d/1159e494-0aef-4f6c-ae01-1217066bb411"
-					(reference "#PWR087")
+					(reference "#PWR088")
 					(unit 1)
 				)
@@
 		(on_board yes)
 		(dnp no)
-		(property "Reference" "R30"
+		(property "Reference" "R31"
 			(at 347.98 229.87 0)
 			(effects
@@
 			(project "impeller18"
 				(path "/4ccab03b-4b1c-4c61-9fa8-19853ef32b4d/1159e494-0aef-4f6c-ae01-1217066bb411"
-					(reference "R30")
+					(reference "R31")
 					(unit 1)
 				)
@@
 		(dnp no)
 		(fields_autoplaced yes)
-		(property "Reference" "#PWR086"
+		(property "Reference" "#PWR087"
 			(at 381 241.935 0)
 			(effects
@@
 			(project "impeller18"
 				(path "/4ccab03b-4b1c-4c61-9fa8-19853ef32b4d/1159e494-0aef-4f6c-ae01-1217066bb411"
-					(reference "#PWR086")
+					(reference "#PWR087")
 					(unit 1)
 				)
@@
 		(dnp no)
 		(fields_autoplaced yes)
-		(property "Reference" "#PWR083"
+		(property "Reference" "#PWR084"
 			(at 238.76 227.965 0)
 			(effects
@@
 			(project "impeller18"
 				(path "/4ccab03b-4b1c-4c61-9fa8-19853ef32b4d/1159e494-0aef-4f6c-ae01-1217066bb411"
-					(reference "#PWR083")
+					(reference "#PWR084")
 					(unit 1)
 				)
@@
 		(on_board yes)
 		(dnp no)
-		(property "Reference" "R341"
+		(property "Reference" "R34"
 			(at 84.455 238.125 0)
 			(effects
@@
 			(project "impeller18"
 				(path "/4ccab03b-4b1c-4c61-9fa8-19853ef32b4d/1159e494-0aef-4f6c-ae01-1217066bb411"
-					(reference "R341")
+					(reference "R34")
 					(unit 1)
 				)
@@
 		(on_board yes)
 		(dnp no)
-		(property "Reference" "R33"
+		(property "Reference" "R36"
 			(at 205.105 244.475 0)
 			(effects
@@
 			(project "impeller18"
 				(path "/4ccab03b-4b1c-4c61-9fa8-19853ef32b4d/1159e494-0aef-4f6c-ae01-1217066bb411"
-					(reference "R33")
+					(reference "R36")
 					(unit 1)
 				)
@@
 		(dnp no)
 		(fields_autoplaced yes)
-		(property "Reference" "#PWR0296"
+		(property "Reference" "#PWR083"
 			(at 85.725 222.885 0)
 			(effects
@@
 			(project "impeller18"
 				(path "/4ccab03b-4b1c-4c61-9fa8-19853ef32b4d/1159e494-0aef-4f6c-ae01-1217066bb411"
-					(reference "#PWR0296")
+					(reference "#PWR083")
 					(unit 1)
 				)
@@
 		(on_board yes)
 		(dnp no)
-		(property "Reference" "R34"
+		(property "Reference" "R38"
 			(at 205.105 251.46 0)
 			(effects
@@
 			(project "impeller18"
 				(path "/4ccab03b-4b1c-4c61-9fa8-19853ef32b4d/1159e494-0aef-4f6c-ae01-1217066bb411"
-					(reference "R34")
+					(reference "R38")
 					(unit 1)
 				)
@@
 		(on_board yes)
 		(dnp no)
-		(property "Reference" "#PWR090"
+		(property "Reference" "#PWR092"
 			(at 237.49 267.335 0)
 			(effects
@@
 			(project "impeller18"
 				(path "/4ccab03b-4b1c-4c61-9fa8-19853ef32b4d/1159e494-0aef-4f6c-ae01-1217066bb411"
-					(reference "#PWR090")
+					(reference "#PWR092")
 					(unit 1)
 				)

Commit message: Update PCB concept
Parts:
- removed TP19: TestPoint, TestPoint:TestPoint_THTPad_D1.5mm_Drill0.7mm, symbol Connector:TestPoint
- added D26, D27: FYLS-0603BUGC, LED_SMD:LED_0603_1608Metric, symbol Device:LED
- added J8: PLS-2, Connector_PinHeader_2.54mm:PinHeader_1x02_P2.54mm_Vertical, symbol Connector_Generic:Conn_01x02
- added R340, R341: 220, Resistor_SMD:R_0603_1608Metric, symbol Device:R_Small
- added R346: 0, Resistor_SMD:R_0603_1608Metric, symbol Device:R_Small
- added R348, R351, R352: DNP, Resistor_SMD:R_0603_1608Metric, symbol Device:R_Small
- added TP41: TestPoint, TestPoint:TestPoint_THTPad_D2.0mm_Drill1.0mm, symbol Connector:TestPoint
- C56, C59: footprint Capacitor_SMD:C_1210_3225Metric -> Capacitor_SMD:C_0603_1608Metric; Мин. кол-во 17 -> 200; Ссылка https://www.promelec.ru/product/384583/ -> https://www.promelec.ru/product/315964/; Цена 29 -> 4; Человекопонятное название Керамический ЧИП-конденсатор 1210 X7S 4.7мкФ -> Керамический ЧИП-конденсатор 0603 X5R 4.7мкФ
- TP10: renamed from TP11; footprint TestPoint:TestPoint_THTPad_D1.5mm_Drill0.7mm -> TestPoint:TestPoint_THTPad_D2.0mm_Drill1.0mm
- TP11: renamed from TP12; footprint TestPoint:TestPoint_THTPad_D1.5mm_Drill0.7mm -> TestPoint:TestPoint_THTPad_D2.0mm_Drill1.0mm
- TP12: renamed from TP13; footprint TestPoint:TestPoint_THTPad_D1.5mm_Drill0.7mm -> TestPoint:TestPoint_THTPad_D2.0mm_Drill1.0mm
- TP13: renamed from TP14; footprint TestPoint:TestPoint_THTPad_D1.5mm_Drill0.7mm -> TestPoint:TestPoint_THTPad_D2.0mm_Drill1.0mm
- TP14: renamed from TP15; footprint TestPoint:TestPoint_THTPad_D1.5mm_Drill0.7mm -> TestPoint:TestPoint_THTPad_D2.0mm_Drill1.0mm
- TP15: renamed from TP16; footprint TestPoint:TestPoint_THTPad_D1.5mm_Drill0.7mm -> TestPoint:TestPoint_THTPad_D2.0mm_Drill1.0mm
- TP16: renamed from TP17; footprint TestPoint:TestPoint_THTPad_D1.5mm_Drill0.7mm -> TestPoint:TestPoint_THTPad_D2.0mm_Drill1.0mm
- TP17: renamed from TP18; footprint TestPoint:TestPoint_THTPad_D1.5mm_Drill0.7mm -> TestPoint:TestPoint_THTPad_D2.0mm_Drill1.0mm
- TP4: renamed from TP5; footprint TestPoint:TestPoint_THTPad_D1.5mm_Drill0.7mm -> TestPoint:TestPoint_THTPad_D2.0mm_Drill1.0mm
- TP5: renamed from TP6; footprint TestPoint:TestPoint_THTPad_D1.5mm_Drill0.7mm -> TestPoint:TestPoint_THTPad_D2.0mm_Drill1.0mm
- TP6: renamed from TP7; footprint TestPoint:TestPoint_THTPad_D1.5mm_Drill0.7mm -> TestPoint:TestPoint_THTPad_D2.0mm_Drill1.0mm
- TP7: renamed from TP8; footprint TestPoint:TestPoint_THTPad_D1.5mm_Drill0.7mm -> TestPoint:TestPoint_THTPad_D2.0mm_Drill1.0mm
- TP8: renamed from TP9; footprint TestPoint:TestPoint_THTPad_D1.5mm_Drill0.7mm -> TestPoint:TestPoint_THTPad_D2.0mm_Drill1.0mm
- TP9: renamed from TP10; footprint TestPoint:TestPoint_THTPad_D1.5mm_Drill0.7mm -> TestPoint:TestPoint_THTPad_D2.0mm_Drill1.0mm
- renumbered C55 to C54, C54 to C55, J8 to J9
Connections:
- net 12V0_SENS: now also TP41.1
- net 5V0: now also K1.A2, K2.A2, K3.A2; no longer K1.A1, K2.A1, K3.A1
- net 7V4: now also C56.1, K1.14, K2.11, J8.1 (Pin_1); no longer C56.2, K1.11, K2.14
- net BAT_CHRG_TOGGLE: now also R340.1
- net BAT_CHRG_TOGGLE_: now also K1.A1, K3.A1; no longer K1.A2, K3.A2
- net BAT_RELAY_TOGGLE: now also R341.1
- net BAT_RELAY_TOGGLE_: now also K2.A1; no longer K2.A2
- net GND: now also C56.2, D26.1 (K), D27.1 (K), R346.2, R351.2; no longer C56.1, R31.1
- net PACK_CHARGE+: now also K1.11; no longer K1.14
- net at BT2.2 (-), BT3.1 (+), J9.2 (Pin_2)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: now also K3.14; no longer K3.11
- net at C52.2, J9.1 (Pin_1), Q4.2 (S)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: now also K3.11; no longer K3.14
- net at F1.1: now also K2.14, J8.2 (Pin_2); no longer K2.11
- net at R29.2, U8.1 (ADJ): now also R31.1, R348.1; no longer R31.2
- new net: D27.2 (A), R341.2
- new net: R348.2, R351.1, R352.1
- new net: R31.2, R346.1, R352.2
- new net: D26.2 (A), R340.2
Other:
- note added: "+gnd"
- note removed: "2 м"
- note removed: "можно поменять стороны реле"
- note removed: "размыкать питание 5v0 при выключении/отключать всю малину от питания"
- moved on the sheet: BT2, BT3, C52, C54, C55, D1, D2, D3, F1, J6, J7, J9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

Commit message: Zone borders
Parts:
- removed TP11, TP6: TestPoint, TestPoint:TestPoint_THTPad_D2.0mm_Drill1.0mm, symbol Connector:TestPoint
- D1, D2, D26, D27, D3, D5, D6: footprint LED_SMD:LED_0603_1608Metric -> user_lib:LED_0603_1608Metric
Other:
- moved on the sheet: D26, D27, Q1, Q2, R12, R13, R15, R16, R340, R341, TP12, TP13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
