File: Hardware/ciam/impeller18/adc_rud.kicad_sch (KiCad schematic)
At the start: 51 parts, among them J19 430450600, Q37 BSS138, Q38 BSS138, U64 LDL1117S33R, U65 B0505MT-1WR4, U66 HCPL-0600, U67 HCPL-0630, U68 ADS1120-PW, U69 IP4220, U70 HCPL-0630

Commit message: changed ads1120 supply voltaged to 5v0
Parts:
- removed C100: 1u, Capacitor_SMD:C_0603_1608Metric, symbol Device:C
- removed C101, C103: 100n, Capacitor_SMD:C_0603_1608Metric, symbol Device:C
- removed C102: 4u7, Capacitor_SMD:C_0603_1608Metric, symbol Device:C
- removed D19: FYLS-0603BUGC, LED_SMD:LED_0603_1608Metric, symbol Device:LED
- removed R227, R232: 1k, Resistor_SMD:R_0603_1608Metric, symbol Device:R_Small
- removed R228, R236: 2k, Resistor_SMD:R_0603_1608Metric, symbol Device:R_Small
- removed R288: 220, Resistor_SMD:R_0603_1608Metric, symbol Device:R_Small
- removed TP31, TP32: TestPoint, TestPoint:TestPoint_THTPad_D1.5mm_Drill0.7mm, symbol Connector:TestPoint
- removed U64: LDL1117S33R, Package_TO_SOT_SMD:SOT-223-3_TabPin2, symbol Regulator_Linear:LD1117S33TR_SOT223
- R239, R242: value 180 -> 360; Ссылка https://www.promelec.ru/product/108141/ -> https://www.promelec.ru/product/46471/; Человекопонятное название Толстопленочный ЧИП-резистор 0603 180Ом -> Толстопленочный ЧИП-резистор 0603 360Ом
Connections:
- net ADC_RUD_3V3_1 is gone; now on net ADC_RUD_5V_1: U68.11 (AIN0/REFP1), U69.1 (IO1)
- net ADC_RUD_3V3_2 is gone; now on net ADC_RUD_5V_2: U68.10 (AIN1), U69.3 (IO2)
- net 5V0_ADC_RUD: now also C107.1, L4.2, Q38.2 (S), R239.2, R241.2, R242.2, U68.13 (DVDD), U68.14 (~{DRDY}), U68.15 (DOUT/~{DRDY}), U69.5 (VDD), U70.2 (C1), U70.3 (C2)
- net at U70.1 (A1): now also R239.1; no longer R239.2
- net at U70.4 (A2): now also R242.1; no longer R242.2
- removed net 3V3_ADC_RUD: C107.1, L4.2, Q38.2 (S), R239.1, R241.2, R242.1, U68.13 (DVDD), U68.14 (~{DRDY}), U68.15 (DOUT/~{DRDY}), U69.5 (VDD), U70.2 (C1), U70.3 (C2)
Other:
- moved on the sheet: J19, U69

Commit message: Updated packeges
Parts:
- J19: footprint Connector_Molex:Molex_Micro-Fit_3.0_43045-0600_2x03_P3.00mm_Horizontal -> user_lib:430450600
Changed lines of the file:
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@@
 			)
 		)
-		(property "Footprint" "Connector_Molex:Molex_Micro-Fit_3.0_43045-0600_2x03_P3.00mm_Horizontal"
+		(property "Footprint" "user_lib:430450600"
 			(at 65.405 145.415 0)
 			(effects

Commit message: Updated 3D models
Parts:
- renumbered C96 to C111, C97 to C112, C98 to C113, C99 to C114, C104 to C115, C105 to C116, C106 to C117, C107 to C118, D20 to D19, J19 to J27, L4 to L5, Q37 to Q59, Q38 to Q60, R222 to R281, R223 to R282, R224 to R283, R225 to R284, R226 to R285, R229 to R286, R230 to R287, R231 to R288, R233 to R289, R234 to R290, R235 to R291, R237 to R292, R238 to R293, R239 to R294, R240 to R295, R241 to R296, R242 to R297, TP29 to TP40, TP30 to TP41, U65 to U63, U66 to U64, U67 to U65, U69 to U66, U68 to U67, U70 to U68
Other:
- moved on the sheet: R295, R296

Commit message: updated bom
Parts:
- renumbered C111 to C114, C112 to C115, C113 to C116, C114 to C117, C115 to C118, C116 to C119, C117 to C120, C118 to C121
Changed lines of the file:
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@@
 		(on_board yes)
 		(dnp no)
-		(property "Reference" "C116"
+		(property "Reference" "C119"
 			(at 227.965 126.365 0)
 			(effects
@@
 			(project "impeller18"
 				(path "/4ccab03b-4b1c-4c61-9fa8-19853ef32b4d/55d85deb-4ae6-4900-939b-1dd08916ec93"
-					(reference "C116")
+					(reference "C119")
 					(unit 1)
 				)
@@
 		(on_board yes)
 		(dnp no)
-		(property "Reference" "#PWR0266"
+		(property "Reference" "#PWR0265"
 			(at 312.42 160.02 0)
 			(effects
@@
 			(project "impeller18"
 				(path "/4ccab03b-4b1c-4c61-9fa8-19853ef32b4d/55d85deb-4ae6-4900-939b-1dd08916ec93"
-					(reference "#PWR0266")
+					(reference "#PWR0265")
 					(unit 1)
 				)
@@
 		(on_board yes)
 		(dnp no)
-		(property "Reference" "#PWR0264"
+		(property "Reference" "#PWR0266"
 			(at 57.785 160.655 0)
 			(effects
@@
 			(project "impeller18"
 				(path "/4ccab03b-4b1c-4c61-9fa8-19853ef32b4d/55d85deb-4ae6-4900-939b-1dd08916ec93"
-					(reference "#PWR0264")
+					(reference "#PWR0266")
 					(unit 1)
 				)
@@
 		(on_board yes)
 		(dnp no)
-		(property "Reference" "C115"
+		(property "Reference" "C118"
 			(at 220.98 126.365 0)
 			(effects
@@
 			(project "impeller18"
 				(path "/4ccab03b-4b1c-4c61-9fa8-19853ef32b4d/55d85deb-4ae6-4900-939b-1dd08916ec93"
-					(reference "C115")
+					(reference "C118")
 					(unit 1)
 				)
@@
 		(on_board yes)
 		(dnp no)
-		(property "Reference" "C118"
+		(property "Reference" "C121"
 			(at 199.39 126.365 90)
 			(effects
@@
 			(project "impeller18"
 				(path "/4ccab03b-4b1c-4c61-9fa8-19853ef32b4d/55d85deb-4ae6-4900-939b-1dd08916ec93"
-					(reference "C118")
+					(reference "C121")
 					(unit 1)
 				)
@@
 		(on_board yes)
 		(dnp no)
-		(property "Reference" "C112"
+		(property "Reference" "C115"
 			(at 111.76 43.815 0)
 			(effects
@@
 			(project "impeller18"
 				(path "/4ccab03b-4b1c-4c61-9fa8-19853ef32b4d/55d85deb-4ae6-4900-939b-1dd08916ec93"
-					(reference "C112")
+					(reference "C115")
 					(unit 1)
 				)
@@
 		(on_board yes)
 		(dnp no)
-		(property "Reference" "C117"
+		(property "Reference" "C120"
 			(at 236.22 126.365 0)
 			(effects
@@
 			(project "impeller18"
 				(path "/4ccab03b-4b1c-4c61-9fa8-19853ef32b4d/55d85deb-4ae6-4900-939b-1dd08916ec93"
-					(reference "C117")
+					(reference "C120")
 					(unit 1)
 				)
@@
 		(on_board yes)
 		(dnp no)
-		(property "Reference" "C113"
+		(property "Reference" "C116"
 			(at 148.59 43.815 0)
 			(effects
@@
 			(project "impeller18"
 				(path "/4ccab03b-4b1c-4c61-9fa8-19853ef32b4d/55d85deb-4ae6-4900-939b-1dd08916ec93"
-					(reference "C113")
+					(reference "C116")
 					(unit 1)
 				)
@@
 		(on_board yes)
 		(dnp no)
-		(property "Reference" "C111"
+		(property "Reference" "C114"
 			(at 102.235 43.815 0)
 			(effects
@@
 			(project "impeller18"
 				(path "/4ccab03b-4b1c-4c61-9fa8-19853ef32b4d/55d85deb-4ae6-4900-939b-1dd08916ec93"
-					(reference "C111")
+					(reference "C114")
 					(unit 1)
 				)
@@
 		(on_board yes)
 		(dnp no)
-		(property "Reference" "C114"
+		(property "Reference" "C117"
 			(at 158.115 43.815 0)
 			(effects
@@
 			(project "impeller18"
 				(path "/4ccab03b-4b1c-4c61-9fa8-19853ef32b4d/55d85deb-4ae6-4900-939b-1dd08916ec93"
-					(reference "C114")
+					(reference "C117")
 					(unit 1)
 				)
@@
 		(on_board yes)
 		(dnp no)
-		(property "Reference" "#PWR0265"
+		(property "Reference" "#PWR0264"
 			(at 130.81 160.02 0)
 			(effects
@@
 			(project "impeller18"
 				(path "/4ccab03b-4b1c-4c61-9fa8-19853ef32b4d/55d85deb-4ae6-4900-939b-1dd08916ec93"
-					(reference "#PWR0265")
+					(reference "#PWR0264")
 					(unit 1)
 				)

Commit message: Daily PCB update
Parts:
- renumbered R281 to R285, R282 to R286, R283 to R287, R284 to R288, R285 to R289, R286 to R290, R287 to R291, R288 to R292, R289 to R293, R290 to R294, R291 to R295, R292 to R296, R293 to R297, R294 to R298, R295 to R299, R296 to R300, R297 to R301, TP40 to TP41, TP41 to TP42

Commit message: Update PCB concept
Parts:
- removed R289, R291, R292, R293, R295: 10k, Resistor_SMD:R_0603_1608Metric, symbol Device:R_Small
- added R284, R285, R286, R288: 1k, Resistor_SMD:R_0603_1608Metric, symbol Device:R_Small
- J30: renamed from J27; symbol Connector_Generic:Conn_02x03_Odd_Even -> Connector_Generic:Conn_02x03_Counter_Clockwise
- R287: value 10k -> 1k; Мин. кол-во 1000 -> 100; Ссылка https://www.promelec.ru/product/344748/ -> https://www.promelec.ru/product/22771/; Человекопонятное название Толстопленочный ЧИП-резистор 0603 10кОм -> Толстопленочный ЧИП-резистор 0603 1кОм
- TP35: renamed from TP41; footprint TestPoint:TestPoint_THTPad_D1.5mm_Drill0.7mm -> TestPoint:TestPoint_THTPad_D2.0mm_Drill1.0mm
- TP36: renamed from TP42; footprint TestPoint:TestPoint_THTPad_D1.5mm_Drill0.7mm -> TestPoint:TestPoint_THTPad_D2.0mm_Drill1.0mm
- renumbered C121 to C118, C118 to C119, C119 to C120, C120 to C121, R285 to R283, R286 to R289, R288 to R290, R290 to R291, R294 to R292, R296 to R293, R297 to R294, R298 to R295, R299 to R296, R300 to R297, R301 to R298, U67 to U65, U65 to U66, U66 to U67
Connections:
- net 3V3: now also U64.2 (A), U66.1 (A1), U66.4 (A2); no longer R290.2, R291.2, R292.2
- net 5V0_ADC_RUD: now also D19.2 (A), J30.5 (Pin_5), R289.2, U68.1 (A1), U68.4 (A2), R284.2, R285.2, R286.2, R288.2; no longer J30.1 (Pin_1), Q60.2 (S), R283.2, R289.1, R295.2, R297.2, R298.2, U65.14 (~{DRDY}), U65.15 (DOUT/~{DRDY}), U68.2 (C1), U68.3 (C2)
- net ADC_RUD_5V_1: now also J30.1 (Pin_1), U67.4 (IO3); no longer J30.3 (Pin_3), U67.1 (IO1)
- net GND: no longer C118.2, C119.1, C120.1, C121.1
- net GND_ADC_RUD: now also C118.2, C119.1, C120.1, C121.1, J30.3 (Pin_3), R283.1; no longer D19.1 (K), J30.5 (Pin_5)
- net SPI1_STM32_ADC8_CS: now also R292.1; no longer U66.3 (C2)
- net SPI1_STM32_CLK: now also R290.1; no longer U64.3 (C)
- net SPI1_STM32_MOSI: now also R291.2; no longer U66.2 (C1)
- net SPI_ADC_RUD_CLK: now also U66.6 (VO2), R284.1; no longer R287.1, U64.6 (VO)
- net SPI_ADC_RUD_CS: now also R287.1, U66.7 (VO1); no longer U66.6 (VO2)
- net SPI_ADC_RUD_MOSI: now also U64.6 (VO), R286.1; no longer U66.7 (VO1)
- net at R295.1: now also U68.2 (C1); no longer U68.1 (A1)
- net at R291.1: now also U66.2 (C1); no longer U66.1 (A1)
- net SPI_ADC_RUD_MISO: now reaches R298.1
- net SPI_ADC_RUD_MISO: now also U65.15 (DOUT/~{DRDY}), R285.1; no longer U68.4 (A2)
- net at U64.7 (EN): now also R289.1; no longer R289.2
- new net: D19.1 (K), R283.2
- new net: R292.2, U66.3 (C2)
- new net: R298.2, U68.3 (C2)
- new net: R290.2, U64.3 (C)
- new net ADC_RUD_INT: Q60.2 (S), R288.1, R295.2, R297.2, U65.14 (~{DRDY})
Other:
- note added: "перeкинуть резистор????"
- moved on the sheet: C118, C119, C120, C121, D19, J30, L5, R283, R289, R290, R291, R292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

Commit message: Zone borders
Parts:
- D19: footprint LED_SMD:LED_0603_1608Metric -> user_lib:LED_0603_1608Metric
Changed lines of the file:
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@@
 			)
 		)
-		(property "Footprint" "LED_SMD:LED_0603_1608Metric"
+		(property "Footprint" "user_lib:LED_0603_1608Metric"
 			(at 266.065 45.72 0)
 			(effects

Commit message: Sch ready
Connections:
- net ADC_RUD_INT: no longer R288.1, R295.2, U65.14 (~{DRDY})
- net SPI1_STM32_ADC8_CS renamed SPI1_STM32_ADC_RUD_CS
- new net ADC_RUD_INT_: R288.1, R295.2, U65.14 (~{DRDY})
Other:
- note removed: "вопросы к работе этой части"
- note removed: "перeкинуть резистор????"
Changed lines of the file:
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@@
 	(wire
 		(pts
-			(xy 368.3 194.31) (xy 373.126 194.31)
+			(xy 368.3 194.31) (xy 373.38 194.31)
 		)
 		(stroke
@@
 		)
 	)
-	(text "перeкинуть резистор????"
-		(exclude_from_sim no)
-		(at 277.495 187.96 90)
-		(effects
-			(font
-				(size 1.27 1.27)
-			)
-		)
-	)
 	(text "VDDA"
 		(exclude_from_sim no)
@@
 		)
 	)
-	(text "вопросы к работе этой части"
-		(exclude_from_sim no)
-		(at 320.04 93.345 0)
-		(effects
-			(font
-				(size 1.27 1.27)
-			)
-		)
-	)
 	(label "SPI_ADC_RUD_MISO"
 		(at 284.48 191.77 0)
@@
 		)
 	)
-	(label "ADC_RUD_INT"
-		(at 284.48 186.69 0)
-		(fields_autoplaced yes)
-		(effects
-			(font
-				(size 1.27 1.27)
-			)
-			(justify left bottom)
+	(label "ADC_RUD_INT_"
+		(at 208.915 191.135 180)
+		(fields_autoplaced yes)
+		(effects
+			(font
+				(size 1.27 1.27)
+			)
+			(justify right bottom)
 		)
 	)
@@
 		)
 	)
+	(label "ADC_RUD_INT_"
+		(at 284.48 186.69 0)
+		(fields_autoplaced yes)
+		(effects
+			(font
+				(size 1.27 1.27)
+			)
+			(justify left bottom)
+		)
+	)
 	(label "ADC_RUD_5V_2"
 		(at 167.005 105.41 180)
@@
 		)
 	)
-	(label "ADC_RUD_INT"
-		(at 208.915 191.135 180)
-		(fields_autoplaced yes)
-		(effects
-			(font
-				(size 1.27 1.27)
-			)
-			(justify right bottom)
-		)
-	)
 	(label "SPI_ADC_RUD_CLK"
 		(at 292.1 140.97 0)
@@
 		)
 	)
-	(global_label "ADC_RUD_INT"
+	(global_label "SPI1_STM32_ADC_RUD_CS"
 		(shape input)
-		(at 373.126 194.31 0)
+		(at 349.885 138.43 0)
 		(fields_autoplaced yes)
 		(effects
@@
 		)
 		(property "Intersheetrefs" "${INTERSHEET_REFS}"
-			(at 388.4484 194.31 0)
+			(at 377.0605 138.43 0)
 			(effects
 				(font
@@
 		)
 	)
-	(global_label "SPI1_STM32_ADC8_CS"
+	(global_label "ADC_RUD_INT"
 		(shape input)
-		(at 349.885 138.43 0)
+		(at 373.38 194.31 0)
 		(fields_autoplaced yes)
 		(effects
@@
 		)
 		(property "Intersheetrefs" "${INTERSHEET_REFS}"
-			(at 373.4319 138.43 0)
+			(at 388.7024 194.31 0)
 			(effects
 				(font
